File: 09_ham_radio.kicad_sch (KiCad schematic)
At the start: 42 parts, among them J240 2m/VHF internal/PCB antenna f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, J241 2m/VHF rear external SMA/u.FL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, J250 70cm/UHF internal/PCB antenna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, J251 70cm/UHF rear external SMA/u.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, J70 DRA818V 2m FM module socket, J71 DRA818U 70cm FM module socket, J72 DNP radio audio/codec harness, U240 2m/VHF RF SPDT antenna switch, U250 70cm/UHF RF SPDT antenna swit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, U70 TPS54302 SYS_5V -> RADIO_4V0

Commit message: Publish the current Ducktop2 design
Parts:
- removed C241: 2m/VHF LPF C2 39pF C0G, Capacitor_SMD:C_0603_1608Metric, symbol Device:C
- removed C242: 2m/VHF LPF C3 12pF C0G, Capacitor_SMD:C_0603_1608Metric, symbol Device:C
- removed C251: 70cm/UHF LPF C2 12pF C0G, Capacitor_SMD:C_0603_1608Metric, symbol Device:C
- removed C252: 70cm/UHF LPF C3 3.9pF C0G, Capacitor_SMD:C_0603_1608Metric, symbol Device:C
- removed J70: DRA818V 2m FM module socket, Connector_PinHeader_1.27mm:PinHeader_1x18_P1.27mm_Vertical, symbol Connector_Generic:Conn_01x18
- removed J71: DRA818U 70cm FM module socket, Connector_PinHeader_1.27mm:PinHeader_1x18_P1.27mm_Vertical, symbol Connector_Generic:Conn_01x18
- removed L240: 2m/VHF LPF L1 75nH RF inductor, Inductor_SMD:L_0603_1608Metric, symbol Device:L
- removed L241: 2m/VHF LPF L2 75nH RF inductor, Inductor_SMD:L_0603_1608Metric, symbol Device:L
- removed L250: 70cm/UHF LPF L1 24nH RF inductor, Inductor_SMD:L_0603_1608Metric, symbol Device:L
- removed L251: 70cm/UHF LPF L2 24nH RF inductor, Inductor_SMD:L_0603_1608Metric, symbol Device:L
- removed U240: 2m/VHF RF SPDT antenna switch, Package_LGA:Infineon_PG-TSNP-6-10_0.7x1.1mm_0.7x1.1mm_P0.4mm, symbol RF_Switch:BGS12WN6E6327
- removed U250: 70cm/UHF RF SPDT antenna switch, Package_LGA:Infineon_PG-TSNP-6-10_0.7x1.1mm_0.7x1.1mm_P0.4mm, symbol RF_Switch:BGS12WN6E6327
- added C223: 100n 50V X7R radio HF, Capacitor_SMD:C_0603_1608Metric, symbol Device:C
- added C224: 56p C0G TPS54302 feed-forward, Capacitor_SMD:C_0402_1005Metric, symbol Device:C
- added C243, C253: 10n PE42820 VDD bypass per eval board, Capacitor_SMD:C_0603_1608Metric, symbol Device:C
- added C244, C254: 100p PE42820 V1 RF bypass per eval board, Capacitor_SMD:C_0603_1608Metric, symbol Device:C
- added C245, C255: DNP 0.2p PE42820 RFC match candidate, Capacitor_SMD:C_0603_1608Metric, symbol Device:C
- added C246: 100n VHF fail-safe buffer local, Capacitor_SMD:C_0603_1608Metric, symbol Device:C
- added C256: 100n UHF fail-safe buffer local, Capacitor_SMD:C_0603_1608Metric, symbol Device:C
- added C260, C261: 100n PTT interlock local, Capacitor_SMD:C_0603_1608Metric, symbol Device:C
- added FL240: Mini-Circuits LFCN-160+ 2m/VHF LPF, Filter:Filter_Mini-Circuits_FV1206, symbol RF_Filter:LFCN-160
- added FL250: Mini-Circuits ULP-470+ 70cm/UHF LPF, ducktop2:MiniCircuits_QA2224_PL484, symbol MiniCircuits_ULP:MiniCircuits_ULP
- added J70: DRA818V 2m FM module, ducktop2:DRA818_Castellated, symbol DRA818:DRA818
- added J71: DRA818U 70cm FM module, ducktop2:DRA818_Castellated, symbol DRA818:DRA818
- added R225: 100k VHF default sleep, Resistor_SMD:R_0603_1608Metric, symbol Device:R
- added R226: 100k UHF default sleep, Resistor_SMD:R_0603_1608Metric, symbol Device:R
- added R227: 47k 1% VHF antenna select default internal; PE428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, Resistor_SMD:R_0603_1608Metric, symbol Device:R
- added R228: 47k 1% UHF antenna select default internal; PE428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, Resistor_SMD:R_0603_1608Metric, symbol Device:R
- added R242: 10k 1% VHF PE42820 control divider top, Resistor_SMD:R_0603_1608Metric, symbol Device:R
- added R243: 1k VHF module TXD isolation, Resistor_SMD:R_0603_1608Metric, symbol Device:R
- added R244: 100k VHF EC TX default low, Resistor_SMD:R_0603_1608Metric, symbol Device:R
- added R260: 10k 1% UHF PE42820 control divider top, Resistor_SMD:R_0603_1608Metric, symbol Device:R
- added R261: 1k UHF module TXD isolation, Resistor_SMD:R_0603_1608Metric, symbol Device:R
- added R262: 100k UHF EC TX default low, Resistor_SMD:R_0603_1608Metric, symbol Device:R
- added U240: PE42820B-X 2m/VHF 43dBm-CW RF switch, ducktop2:PE42820_QFN-32-1EP_5x5mm_P0.5mm, symbol PE42820:PE42820
- added U241: SN74LVC1G373DCKR VHF transmit-safe RF-select latch, Package_TO_SOT_SMD:SOT-363_SC-70-6, symbol 74xGxx:74LVC1G373
- added U242: SN74LVC3G34DCUR VHF fail-safe control buffer, Package_SO:VSSOP-8_2.3x2mm_P0.5mm, symbol 74xGxx:74LVC3G34
- added U250: PE42820B-X 70cm/UHF 43dBm-CW RF switch, ducktop2:PE42820_QFN-32-1EP_5x5mm_P0.5mm, symbol PE42820:PE42820
- added U251: SN74LVC1G373DCKR UHF transmit-safe RF-select latch, Package_TO_SOT_SMD:SOT-363_SC-70-6, symbol 74xGxx:74LVC1G373
- added U252: SN74LVC3G34DCUR UHF fail-safe control buffer, Package_SO:VSSOP-8_2.3x2mm_P0.5mm, symbol 74xGxx:74LVC3G34
- added unit 3 of U261
- added unit 2 of U261
- C220: value 10u radio VIN -> 10u 25V X7R radio VIN; MPN (none) -> GRM31CR71E106KA12L; Manufacturer (none) -> Murata
- C222: value 47u radio rail bulk -> 22u 16V X7R radio output; MPN (none) -> GRM31CZ71C226ME15L; Manufacturer (none) -> Murata
- C225: renamed from C223; value 100n radio rail -> 22u 16V X7R radio output; footprint Capacitor_SMD:C_0603_1608Metric -> Capacitor_SMD:C_1206_3216Metric; MPN (none) -> GRM31CZ71C226ME15L; Manufacturer (none) -> Murata
- C240: value 2m/VHF LPF C1 12pF C0G -> 100n VHF RF-select latch local
- C250: value 70cm/UHF LPF C1 3.9pF C0G -> 100n UHF RF-select latch local
- J240, J250: MPN (none) -> U.FL-R-SMT-1(01); Manufacturer (none) -> Hirose
- J241, J251: MPN (none) -> 73251-1153; Manufacturer (none) -> Molex
- L70: value 2.2uH >=2A -> 3.3uH 20% 6.0A Isat20; footprint Inductor_SMD:L_1210_3225Metric -> ducktop2:Coilcraft_XGL5030; MPN (none) -> XGL5030-332MEC; Manufacturer (none) -> Coilcraft
- R221: value 576k 1% 4.0V FB hi -> 100k 1% 4.0V FB hi
- R222: value 100k 1% 4.0V FB lo -> 17.4k 1% 4.0V FB lo
- R229: value 0R VHF H/L default low power -> 0R VHF H/L LOW POWER - FIT; AssemblyState (none) -> MUST_FIT_FOR_PROTOTYPE; VariantRule (none) -> FIT=LOW_0.5W;LFCN160_POWER_MARGIN_DOES_NOT_WAIVE_RF_SPECTRU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
- R230: value DNP 0R VHF H/L high power -> 100k VHF RF-select EC reset default internal; now fitted; now in the parts list
- R231: value 0R UHF H/L default low power -> 0R UHF H/L LOW POWER - FIT; AssemblyState (none) -> MUST_FIT_FOR_PROTOTYPE; VariantRule (none) -> FIT=LOW_0.5W;OMIT=FLOAT_HIGH_1W_ONLY_AFTER_RF_RELEASE
- R232: value DNP 0R UHF H/L high power -> 100k UHF RF-select EC reset default internal; now fitted; now in the parts list
- U260: renamed from R227; value 100k VHF antenna select default internal -> SN74LVC2G04DCKR PTT request inverter; footprint Resistor_SMD:R_0603_1608Metric -> Package_TO_SOT_SMD:SOT-363_SC-70-6; symbol Device:R -> 74xGxx:74LVC2G04; MPN (none) -> SN74LVC2G04DCKR; Manufacturer (none) -> Texas Instruments; SafetyContract (none) -> BOTH_PTT_REQUESTS_ASSERTED_FORCES_BOTH_MODULE_PTT_OUTPUTS_I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
- U260: renamed from R225; value 100k VHF PD default pulled up -> SN74LVC2G04DCKR PTT request inverter; footprint Resistor_SMD:R_0603_1608Metric -> Package_TO_SOT_SMD:SOT-363_SC-70-6; symbol Device:R -> 74xGxx:74LVC2G04; MPN (none) -> SN74LVC2G04DCKR; Manufacturer (none) -> Texas Instruments; SafetyContract (none) -> BOTH_PTT_REQUESTS_ASSERTED_FORCES_BOTH_MODULE_PTT_OUTPUTS_I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
- U260: renamed from R226; value 100k UHF PD default pulled up -> SN74LVC2G04DCKR PTT request inverter; footprint Resistor_SMD:R_0603_1608Metric -> Package_TO_SOT_SMD:SOT-363_SC-70-6; symbol Device:R -> 74xGxx:74LVC2G04; MPN (none) -> SN74LVC2G04DCKR; Manufacturer (none) -> Texas Instruments; SafetyContract (none) -> BOTH_PTT_REQUESTS_ASSERTED_FORCES_BOTH_MODULE_PTT_OUTPUTS_I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
- U261: renamed from R228; value 100k UHF antenna select default internal -> SN74LVC2G32DCUR dual-radio PTT interlock; footprint Resistor_SMD:R_0603_1608Metric -> Package_SO:VSSOP-8_2.3x2mm_P0.5mm; symbol Device:R -> 74xGxx:74LVC2G32; MPN (none) -> SN74LVC2G32DCUR; Manufacturer (none) -> Texas Instruments; SafetyContract (none) -> BOTH_PTT_REQUESTS_ASSERTED_FORCES_BOTH_MODULE_PTT_OUTPUTS_I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
- U70: MPN (none) -> TPS54302DDCR; Manufacturer (none) -> Texas Instruments
Connections:
- net RADIO_UHF_RF_SEL is gone; now on net RADIO_VHF_PTT_N: U261.1
- net GND: now also R230.2, R232.2, C223.2, C243.2, C244.2, C245.2, C246.2, C253.2, C254.2, C255.2, C256.2, C260.2, C261.2, FL240.2 (GND), FL240.4 (GND), FL250.2 (GND), FL250.4 (GND), FL250.5 (GND), FL250.6 (GND), J70.10 (GND), J70.9 (GND), J71.10 (GND), J71.9 (GND), R225.2, R226.2, R227.2, R228.2, R244.2, R262.2, U240.1 (GND), U240.10 (GND), U240.11 (GND), U240.14 (GND), U240.15 (GND), U240.16 (VSS_EXT), U240.17 (GND), U240.18 (GND), U240.19 (GND), U240.20 (GND), U240.21 (GND), U240.22 (GND), U240.24 (GND), U240.25 (GND), U240.26 (GND), U240.27 (GND), U240.29 (GND), U240.3 (GND), U240.30 (GND), U240.31 (GND), U240.32 (GND), U240.33 (EP_GND), U240.4 (GND), U240.5 (GND), U240.6 (GND), U240.7 (GND), U240.8 (GND), U240.9 (GND), U241.2 (GND), U241.6 (~{OE}), U242.4 (GND), U250.1 (GND), U250.10 (GND), U250.11 (GND), U250.14 (GND), U250.15 (GND), U250.16 (VSS_EXT), U250.17 (GND), U250.18 (GND), U250.19 (GND), U250.20 (GND), U250.21 (GND), U250.22 (GND), U250.24 (GND), U250.25 (GND), U250.26 (GND), U250.27 (GND), U250.29 (GND), U250.3 (GND), U250.30 (GND), U250.31 (GND), U250.32 (GND), U250.33 (EP_GND), U250.4 (GND), U250.5 (GND), U250.6 (GND), U250.7 (GND), U250.8 (GND), U250.9 (GND), U251.2 (GND), U251.6 (~{OE}), U252.4 (GND), U261.4 (GND); no longer U261.2
- net MCU_3V3: now also U260.5 (VCC), C260.1, C261.1, U261.8 (VCC); no longer R230.2, R232.2, U260.1, U260.1
- net RADIO_4V0: now also C240.1, C250.1, C223.1, C224.1, C243.1, C246.1, C253.1, C256.1, J70.8 (VBAT), J71.8 (VBAT), U240.12 (VDD), U241.5 (VCC), U242.8 (VCC), U250.12 (VDD), U251.5 (VCC), U252.8 (VCC)
- net RADIO_BUCK_FB: now also C224.2
- net RADIO_UHF_MIC_IN: now also J71.18 (MIC_IN)
- net RADIO_UHF_PD_N: now also R226.1, U252.3; no longer U260.2
- net RADIO_UHF_PTT_N: now also U260.3, U261.5
- net RADIO_UHF_SQL: now also J71.1 (SQ)
- net RADIO_UHF_UART_RX: now also R261.2
- net RADIO_UHF_UART_TX: now also R262.1, U252.1
- net RADIO_VHF_MIC_IN: now also J70.18 (MIC_IN)
- net RADIO_VHF_PD_N: now also R225.1, U242.3; no longer U260.2
- net RADIO_VHF_PTT_N: now also U260.1
- net RADIO_VHF_SQL: now also J70.1 (SQ)
- net RADIO_VHF_UART_RX: now also R243.2
- net RADIO_VHF_UART_TX: now also R244.1, U242.1
- net UHF_AF_OUT: now also J71.3 (AF_OUT)
- net UHF_ANT_EXTERNAL: now also U250.2 (RF1)
- net UHF_ANT_ONBOARD: now also U250.23 (RF2)
- net UHF_HL: now also J71.7 (H/L); no longer R232.1
- net UHF_RF_FILTERED: now also C255.1, FL250.3 (RF2), U250.28 (RFC)
- net UHF_RF_RAW: now also FL250.1 (RF1), J71.12 (ANT); no longer C250.1
- net VHF_AF_OUT: now also J70.3 (AF_OUT)
- net VHF_ANT_EXTERNAL: now also U240.2 (RF1)
- net VHF_ANT_ONBOARD: now also U240.23 (RF2)
- net VHF_HL: now also J70.7 (H/L); no longer R230.1
- net VHF_RF_FILTERED: now also C245.1, FL240.3 (OUT), U240.28 (RFC)
- net VHF_RF_RAW: now also FL240.1 (IN), J70.12 (ANT); no longer C240.1
- removed net RADIO_VHF_RF_SEL: U260.1
- new net RADIO_UHF_PD_LOCAL_N: J71.6 (PD), U252.5
- new net RADIO_UHF_PTT_LOCAL_N: J71.5 (PTT_N), U252.2
- new net RADIO_UHF_PTT_REQ: U260.4, U261.2
- new net RADIO_UHF_PTT_SAFE_N: U251.1 (LE), U252.6, U261.3
- new net RADIO_UHF_RF_SEL_3V3: R232.1, U251.3 (D)
- new net RADIO_UHF_RF_SEL_4V0: C254.1, R228.1, R260.2, U250.13 (V1)
- new net RADIO_UHF_RF_SEL_4V0_RAW: R260.1, U251.4 (Q)
- new net RADIO_UHF_UART_RXD: J71.16 (RXD), U252.7
- new net RADIO_UHF_UART_TXD: J71.17 (TXD), R261.1
- new net RADIO_VHF_PD_LOCAL_N: J70.6 (PD), U242.5
- new net RADIO_VHF_PTT_LOCAL_N: J70.5 (PTT_N), U242.2
- new net RADIO_VHF_PTT_REQ: U260.6, U261.6
- new net RADIO_VHF_PTT_SAFE_N: U241.1 (LE), U242.6, U261.7
- new net RADIO_VHF_RF_SEL_3V3: R230.1, U241.3 (D)
- new net RADIO_VHF_RF_SEL_4V0: C244.1, R227.1, R242.2, U240.13 (V1)
- new net RADIO_VHF_RF_SEL_4V0_RAW: R242.1, U241.4 (Q)
- new net RADIO_VHF_UART_RXD: J70.16 (RXD), U242.7
- new net RADIO_VHF_UART_TXD: J70.17 (TXD), R243.1
- no-connect marks 10 -> 12
Other:
- note added: "== DRA818V/U castellated radio modules =="
- note added: "Dorji pinout: pins 9/10 GND; pins 2/4/11/13/14/15 NC; pin12 ANT 50 ohm; pin16 RXD; pin17 TXD."
- note added: "FL240 LFCN-160+ (8W at 25C) and FL250 ULP-470+ (2W) are fitted LPFs; calculate both 50-ohm launches from the final stackup."
- note added: "H/L is never driven high: fitted 0R selects low power; omitted 0R floats for high power only after RF release."
- note added: "PE42820 is rated 43dBm CW through 2GHz when powered; RADIO_4V0 powers switch and module together."
- note added: "R225/R226 set safe EC defaults; radio-powered Ioff buffers prevent injection into unpowered DRA818 inputs."
- note added: "R229/R231 select 0.5W prototype power. Filter ratings do not prove emissions compliance; verify both outputs on a spectrum analyzer."
- note added: "U260/U261 force both radios out of TX for simultaneous requests; U241/U251 freeze antenna selection for the full transmit interval."
- note added: "VHF uses the DRA818V 2m module; UHF uses the DRA818U 70cm module."
- note added: "Validate antenna match/VSWR, enclosure detuning, duty cycle, harmonics, and GNSS/Wi-Fi isolation before RF release."
- note removed: "== DRA818/SA818-compatible module sockets =="
- note removed: "BGS12 control low selects RF1/pin3 internal feed; high selects RF2/pin1 rear external feed."
- note removed: "DRA818V/U pinout is locked to Dorji V1.23: pin16 RXD<-EC_TX, pin17 TXD->EC_RX, pin12 RF 50 ohm."
- note removed: "Default RF switch state selects the internal/PCB antenna feed; rear external SMA/u.FL is the high-performance option."
- note removed: "LPF values are 5th-order Butterworth starting points; simulate/bench-check harmonics for Part 97 before fab."
- note removed: "RF switch truth table, RF layout, and filter parasitics remain RF-review items; DRA818 module pinout is set."
- note removed: "Use board-edge keepouts around rear external SMA paths; internal antennas need separation from GPS and Wi-Fi antennas."
- note removed: "VHF uses DRA818V/SA818-compatible 2m module; UHF uses DRA818U/SA818-compatible 70cm module."
- moved on the sheet: C225
