File: 13_radio_audio_codec.kicad_sch (KiCad schematic)
At the start: 23 parts, among them J330 DNP radio audio codec probe, U330 PCM2902 USB audio codec, Y330 12MHz PCM2902

Commit message: Publish the current Ducktop2 design
Parts:
- removed C336: 4.7u codec 3V3 bulk, Capacitor_SMD:C_0805_2012Metric, symbol Device:C
- removed C342: 1u TX audio AC couple, Capacitor_SMD:C_0805_2012Metric, symbol Device:C
- removed R332: 100k line-in L bleed, Resistor_SMD:R_0603_1608Metric, symbol Device:R
- removed R333: 100k line-in R bleed, Resistor_SMD:R_0603_1608Metric, symbol Device:R
- removed Y330: 12MHz PCM2902, Crystal:Crystal_SMD_3225-4Pin_3.2x2.5mm, symbol Device:Crystal_GND24
- added C330: 1u PCM2902C VBUS, Capacitor_SMD:C_0805_2012Metric, symbol Device:C
- added C338: 18p C0G 5% PCM2902 crystal load, Capacitor_SMD:C_0603_1608Metric, symbol Device:C
- added D390, D391, D392, D393: BAT54WS PTT/suspend mute OR, Diode_SMD:D_SOD-323, symbol Device:D_Schottky
- added J330: DNP radio audio codec probe, Connector_PinHeader_2.54mm:PinHeader_1x08_P2.54mm_Vertical, symbol Connector_Generic:Conn_01x08
- added Q330: 2N7002KT1G VHF PTT/suspend fail-mute shunt, Package_TO_SOT_SMD:SOT-23, symbol Q_NMOS_SOT23_GSD:Q_NMOS_SOT23_GSD
- added Q331: 2N7002KT1G UHF PTT/suspend fail-mute shunt, Package_TO_SOT_SMD:SOT-23, symbol Q_NMOS_SOT23_GSD:Q_NMOS_SOT23_GSD
- added Q332: BSS84LT1G codec-loss force-mute, Package_TO_SOT_SMD:SOT-23, symbol Transistor_FET:Q_PMOS_GSD
- added R336: 1k 1% VHF mic attenuator shunt, Resistor_SMD:R_0603_1608Metric, symbol Device:R
- added R338: 1.5k USB D+ pull-up per TI Figure 39, Resistor_SMD:R_0603_1608Metric, symbol Device:R
- added R340: 1M crystal feedback, Resistor_SMD:R_0603_1608Metric, symbol Device:R
- added R341: 1k 1% UHF mic attenuator shunt, Resistor_SMD:R_0603_1608Metric, symbol Device:R
- added R342: 100k SSPND fail-low pull-down, Resistor_SMD:R_0603_1608Metric, symbol Device:R
- added R343: 100k force-mute pull-down, Resistor_SMD:R_0603_1608Metric, symbol Device:R
- added R344: 100k VHF mute-gate pull-down, Resistor_SMD:R_0603_1608Metric, symbol Device:R
- added R345: 100k UHF mute-gate pull-down, Resistor_SMD:R_0603_1608Metric, symbol Device:R
- C331: value 100n codec VBUS -> 10u VCCCI; footprint Capacitor_SMD:C_0603_1608Metric -> Capacitor_SMD:C_1206_3216Metric
- C332: value 100n codec 3V3 -> 1u VCCP1I (<2u); footprint Capacitor_SMD:C_0603_1608Metric -> Capacitor_SMD:C_0805_2012Metric
- C333: value 100n codec 3V3 -> 1u VCCP2I (<2u); footprint Capacitor_SMD:C_0603_1608Metric -> Capacitor_SMD:C_0805_2012Metric
- C334: value 100n codec 3V3 -> 1u VCCXI (<2u); footprint Capacitor_SMD:C_0603_1608Metric -> Capacitor_SMD:C_0805_2012Metric
- C335: value 100n codec 3V3 -> 1u VDDI (<2u); footprint Capacitor_SMD:C_0603_1608Metric -> Capacitor_SMD:C_0805_2012Metric
- C337: value 1u VCOM -> 10u VCOM; footprint Capacitor_SMD:C_0805_2012Metric -> Capacitor_SMD:C_1206_3216Metric
- C339: value 18p -> 18p C0G 5% PCM2902 crystal load
- C342: renamed from R334; value 10k VHF mic feed -> 1u VHF TX audio AC couple; footprint Resistor_SMD:R_0603_1608Metric -> Capacitor_SMD:C_0805_2012Metric; symbol Device:R -> Device:C
- C343: renamed from R335; value 10k UHF mic feed -> 1u UHF TX audio AC couple; footprint Resistor_SMD:R_0603_1608Metric -> Capacitor_SMD:C_0805_2012Metric; symbol Device:R -> Device:C
- R334: renamed from R336; value 100k TX audio bleed -> 82k 1% VHF mic attenuator series; ReleaseGate (none) -> CALIBRATE_DEVIATION_AND_LOCK_DRA818_MIC_INPUT_IMPEDANCE
- R335: renamed from J330; value DNP radio audio codec probe -> 82k 1% UHF mic attenuator series; footprint Connector_PinHeader_2.54mm:PinHeader_1x08_P2.54mm_Vertical -> Resistor_SMD:R_0603_1608Metric; symbol Connector_Generic:Conn_01x08 -> Device:R; ReleaseGate (none) -> CALIBRATE_DEVIATION_AND_LOCK_DRA818_MIC_INPUT_IMPEDANCE; now fitted; now in the parts list
- R337: renamed from C330; value 10u codec VBUS -> 2.2R PCM2902C VBUS filter; footprint Capacitor_SMD:C_1206_3216Metric -> Resistor_SMD:R_0603_1608Metric; symbol Device:C -> Device:R
- U330: value PCM2902 USB audio codec -> PCM2902CDBR USB audio codec; MPN (none) -> PCM2902CDBR; Manufacturer (none) -> Texas Instruments; ReferenceCircuit (none) -> PCM2902C Figure 39 bus-powered configuration
- Y330: renamed from C338; value 18p -> ABM8G-106-12.000MHZ-T 12MHz 10pF CL; footprint Capacitor_SMD:C_0603_1608Metric -> Crystal:Crystal_SMD_3225-4Pin_3.2x2.5mm; symbol Device:C -> Device:Crystal_GND24; LoadCalculation (none) -> 18pF each leg gives about 10pF with approximately 1pF pin/P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; MPN (none) -> ABM8G-106-12.000MHZ-T; Manufacturer (none) -> Abracon
Connections:
- net CODEC_USB_DP: now also R338.2
- net CODEC_XTI: now also C338.1, R340.1
- net CODEC_XTO: now also Y330.3, R340.2
- net GND: now also Y330.4 (G), C330.2, C338.2, J330.1 (Pin_1), J330.8 (Pin_8), Q330.2 (S), Q331.2 (S), R336.2, R341.2, R342.2, R343.2, R344.2, R345.2; no longer R334.2, R335.1 (Pin_1), R335.8 (Pin_8), R337.2, U330.5 (HID0), U330.6 (HID1), U330.7 (HID2), U330.8 (SEL0), U330.9 (SEL1)
- net RADIO_UHF_AUDIO_OUT: now also J330.3 (Pin_3); no longer R335.3 (Pin_3)
- net RADIO_UHF_MIC_IN: now also R335.2, J330.7 (Pin_7), Q331.3 (D), R341.1; no longer C343.2, R335.6 (Pin_6)
- net RADIO_VHF_AUDIO_OUT: now also J330.2 (Pin_2); no longer R335.2 (Pin_2)
- net RADIO_VHF_MIC_IN: now also R334.2, J330.6 (Pin_6), Q330.3 (D), R336.1; no longer C342.2, R335.5 (Pin_5)
- net CODEC_TX_UHF: now reaches U330.15 (VOUTR)
- net CODEC_TX_UHF: now also C343.1
- net CODEC_SSPND: now reaches U330.28 (~{SSPND})
- net CODEC_SSPND: now also Q332.1 (G), R342.1
- net AUDIO_USB_DM renamed RADIO_CODEC_USB_DM
- net AUDIO_USB_DP renamed RADIO_CODEC_USB_DP
- removed net CODEC_3V3: C332.1, C333.1, C334.1, C335.1, U330.10 (VCCCI), U330.17 (VCCP1I), U330.19 (VCCP2I), U330.23 (VCCXI), U330.27 (VDDI)
- net CODEC_TX_L renamed CODEC_TX_VHF
- net CODEC_TX_VHF: now also C342.1
- removed net RADIO_TX_AUDIO: C342.1, C343.1, R334.1, R335.4 (Pin_4)
- removed net SYS_5V: C331.1, R335.7 (Pin_7), R337.1, U330.3 (VBUS)
- new net CODEC_FORCE_MUTE: D391.2 (A), D393.2 (A), Q332.3 (D), R343.1
- new net CODEC_VBUS: C330.1, R337.2, U330.3 (VBUS)
- new net CODEC_VCCCI: C331.1, U330.10 (VCCCI)
- new net CODEC_VCCP1I: C332.1, U330.17 (VCCP1I)
- new net CODEC_VCCP2I: C333.1, U330.19 (VCCP2I)
- new net CODEC_VCCXI: C334.1, U330.23 (VCCXI)
- new net CODEC_VDDI: C335.1, R338.1, U330.27 (VDDI), U330.8 (SEL0), U330.9 (SEL1)
- new net MCU_3V3: Q332.2 (S)
- new net RADIO_CODEC_USB_VBUS: R337.1
- new net RADIO_UHF_PTT_N: D392.2 (A)
- new net RADIO_VHF_PTT_N: D390.2 (A)
- new net UHF_MUTE_GATE: D392.1 (K), D393.1 (K), Q331.1 (G), R345.1
- new net UHF_TX_AUDIO: C343.2, J330.5 (Pin_5), R335.1
- new net VHF_MUTE_GATE: D390.1 (K), D391.1 (K), Q330.1 (G), R344.1
- new net VHF_TX_AUDIO: C342.2, J330.4 (Pin_4), R334.1
- no-connect marks 4 -> 5
Other:
- note added: "== U330 PCM2902CDBR USB audio codec; TI Figure 39 core network =="
- note added: "Independent 82k/1k dividers produce about 8.4mVrms open-circuit; Q330/Q331 mute on PTT_N high, USB suspend, or codec power loss."
- note added: "No codec-side bleed: PCM2902 biases VINL/VINR internally to VCOM through 30k."
- note added: "PCM2902CDBR is downstream port 1 of the internal system-audio hub on Mu USB2_P5."
- note added: "RELEASE GATE: measure MIC impedance and deviation per band; preserve Ham R223/R224 pull-ups and hard-interlock both PTT_N signals."
- note added: "TI Figure 39 core is implemented: SEL0/SEL1 direct-high, 1.5k D+ pull-up, filtered VBUS, and separate rail capacitors."
- note added: "VHF/UHF use independent stereo ADC/DAC channels; each TX path is attenuated and fail-muted by its PTT_N signal."
- note removed: "== U330 PCM2902 USB audio codec =="
- note removed: "Final DRA818 audio gain/attenuation values require bench measurements; current values are safe first-pass starts."
- note removed: "Host software handles APRS/audio decoding through USB audio; EC GPIO still owns PTT, PD, SQL, and antenna select."
- note removed: "Only assert one PTT at a time; both radio mic inputs receive the same isolated DAC audio through large resistors."
- note removed: "PCM2902 appears to the host as a USB audio device on Mu USB2_P5."
- note removed: "VHF/UHF receive feed stereo inputs; left DAC output feeds both radio mic inputs through isolation resistors."
- moved on the sheet: R334
