File: 06_tcp0_external_hdmi.kicad_sch (KiCad schematic)
At the start: 61 parts, among them J30 External HDMI-A from TCP0, Q50 BSS138 HDMI bias gate, U50 TPD13S523PWR HDMI control ESD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, U51 PCA9306DCTR HDMI DDC level tr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, U53 SN74LVC1G17DBVR HDMI HPD buff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, U54 TPS22975NDSGR host-active SYS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, U55 TPS22975NDSGR host-active SYS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

Commit message: Regenerate child schematics to sync with current generators
The committed .kicad_sch carried stale embedded Manufacturer/MPN properties from the old per-component BOM approach (MPNs now live in verification/BOM_MPN_ASSIGNMENTS.md). Regenerating from the current generators strips those stale properties and clears the pre-existing Generated-source identity release-check failure. No connectivity change; ERC still 0 errors / 27 intentional warnings; schematic closure 1569/0.
Parts:
- C164, C165: MPN GRM155R71C472KA01D -> (none); Manufacturer Murata -> (none)
- R164, R166, R168, R169: MPN RC0402FR-07100KL -> (none); Manufacturer Yageo -> (none)
- R165: MPN RC0402FR-072K2L -> (none); Manufacturer Yageo -> (none)
Changed lines of the file:
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@@
   (property "Footprint" "Resistor_SMD:R_0402_1005Metric" (at 529.59 177.8 0) (effects (font (size 1.27 1.27)) (hide yes)))
   (property "Datasheet" "" (at 529.59 177.8 0) (effects (font (size 1.27 1.27)) (hide yes)))
-  (property "Manufacturer" "Yageo" (at 529.59 177.8 0) (effects (font (size 1.27 1.27)) (hide yes)))
-  (property "MPN" "RC0402FR-072K2L" (at 529.59 177.8 0) (effects (font (size 1.27 1.27)) (hide yes)))
   (pin "1")
   (pin "2")
@@
   (property "Footprint" "Resistor_SMD:R_0402_1005Metric" (at 529.59 190.5 0) (effects (font (size 1.27 1.27)) (hide yes)))
   (property "Datasheet" "" (at 529.59 190.5 0) (effects (font (size 1.27 1.27)) (hide yes)))
-  (property "Manufacturer" "Yageo" (at 529.59 190.5 0) (effects (font (size 1.27 1.27)) (hide yes)))
-  (property "MPN" "RC0402FR-07100KL" (at 529.59 190.5 0) (effects (font (size 1.27 1.27)) (hide yes)))
   (pin "1")
   (pin "2")
@@
   (property "Footprint" "Capacitor_SMD:C_0402_1005Metric" (at 454.66 38.1 0) (effects (font (size 1.27 1.27)) (hide yes)))
   (property "Datasheet" "" (at 454.66 38.1 0) (effects (font (size 1.27 1.27)) (hide yes)))
-  (property "Manufacturer" "Murata" (at 454.66 38.1 0) (effects (font (size 1.27 1.27)) (hide yes)))
-  (property "MPN" "GRM155R71C472KA01D" (at 454.66 38.1 0) (effects (font (size 1.27 1.27)) (hide yes)))
   (pin "1")
   (pin "2")
@@
   (property "Footprint" "Capacitor_SMD:C_0402_1005Metric" (at 454.66 101.6 0) (effects (font (size 1.27 1.27)) (hide yes)))
   (property "Datasheet" "" (at 454.66 101.6 0) (effects (font (size 1.27 1.27)) (hide yes)))
-  (property "Manufacturer" "Murata" (at 454.66 101.6 0) (effects (font (size 1.27 1.27)) (hide yes)))
-  (property "MPN" "GRM155R71C472KA01D" (at 454.66 101.6 0) (effects (font (size 1.27 1.27)) (hide yes)))
   (pin "1")
   (pin "2")
@@
   (property "Footprint" "Resistor_SMD:R_0402_1005Metric" (at 454.66 50.8 0) (effects (font (size 1.27 1.27)) (hide yes)))
   (property "Datasheet" "" (at 454.66 50.8 0) (effects (font (size 1.27 1.27)) (hide yes)))
-  (property "Manufacturer" "Yageo" (at 454.66 50.8 0) (effects (font (size 1.27 1.27)) (hide yes)))
-  (property "MPN" "RC0402FR-07100KL" (at 454.66 50.8 0) (effects (font (size 1.27 1.27)) (hide yes)))
   (pin "1")
   (pin "2")
@@
   (property "Footprint" "Resistor_SMD:R_0402_1005Metric" (at 454.66 114.3 0) (effects (font (size 1.27 1.27)) (hide yes)))
   (property "Datasheet" "" (at 454.66 114.3 0) (effects (font (size 1.27 1.27)) (hide yes)))
-  (property "Manufacturer" "Yageo" (at 454.66 114.3 0) (effects (font (size 1.27 1.27)) (hide yes)))
-  (property "MPN" "RC0402FR-07100KL" (at 454.66 114.3 0) (effects (font (size 1.27 1.27)) (hide yes)))
   (pin "1")
   (pin "2")
@@
   (property "Footprint" "Resistor_SMD:R_0402_1005Metric" (at 650.24 132.08 0) (effects (font (size 1.27 1.27)) (hide yes)))
   (property "Datasheet" "" (at 650.24 132.08 0) (effects (font (size 1.27 1.27)) (hide yes)))
-  (property "Manufacturer" "Yageo" (at 650.24 132.08 0) (effects (font (size 1.27 1.27)) (hide yes)))
-  (property "MPN" "RC0402FR-07100KL" (at 650.24 132.08 0) (effects (font (size 1.27 1.27)) (hide yes)))
-  (pin "1")
-  (pin "2")
+  (pin "1")
+  (pin "2")
