File: 08_internal_services.kicad_sch (KiCad schematic)
At the start: 48 parts, among them J50 DNP EC USB probe, J51 DNP alternate touchscreen USB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, J52 4-wire 5V PWM blower/fan: GND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, J53 Lid/hall switch, J54 Skin/hinge NTC, J55 DNP low-speed display/backlig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, J56 Mu heatsink/spreader NTC, J57 DNP trackpad FFC fallback: US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, J58 Internal USB-C receptacle for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, Q200 Fan PWM open-drain sink, U60 USBLC6-2P6 EC USB ESD, U61 USBLC6-2P6 touch USB ESD, U62 USBLC6-2P6 trackpad USB ESD

Commit message: Publish the current Ducktop2 design
Parts:
- removed C200: 10u touch VBUS local, Capacitor_SMD:C_1206_3216Metric, symbol Device:C
- removed C201: 100n touch local, Capacitor_SMD:C_0603_1608Metric, symbol Device:C
- removed C203: 10u display service bulk, Capacitor_SMD:C_1206_3216Metric, symbol Device:C
- removed C204: 100n display service, Capacitor_SMD:C_0603_1608Metric, symbol Device:C
- removed F201: 500mA trackpad 5V polyfuse, Fuse:Fuse_1206_3216Metric, symbol Device:Fuse
- removed J51: DNP alternate touchscreen USB/control, Connector_PinHeader_2.54mm:PinHeader_1x06_P2.54mm_Vertical, symbol Connector_Generic:Conn_01x06
- removed J52: 4-wire 5V PWM blower/fan: GND, fused 5V, tach, PWM, Connector_JST:JST_XH_B4B-XH-A_1x04_P2.50mm_Vertical, symbol Connector_Generic:Conn_01x04
- removed J55: DNP low-speed display/backlight service FFC, Connector_FFC-FPC:Hirose_FH12-20S-0.5SH_1x20-1MP_P0.50mm_Horizontal, symbol Connector_Generic:Conn_01x20
- removed J57: DNP trackpad FFC fallback: USB HID plus optional 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, Connector_FFC-FPC:Hirose_FH12-10S-0.5SH_1x10-1MP_P0.50mm_Horizontal, symbol Connector_Generic:Conn_01x10
- removed R202: 22R touch DP series, Resistor_SMD:R_0603_1608Metric, symbol Device:R
- removed R204: 100k touch reset pull-up, Resistor_SMD:R_0603_1608Metric, symbol Device:R
- removed R205: 100k touch INT pull-up, Resistor_SMD:R_0603_1608Metric, symbol Device:R
- removed R211: 100k panel power default off, Resistor_SMD:R_0603_1608Metric, symbol Device:R
- removed R212: 100k backlight EN default off, Resistor_SMD:R_0603_1608Metric, symbol Device:R
- removed R213: 100R backlight PWM series, Resistor_SMD:R_0603_1608Metric, symbol Device:R
- removed R214: 100k panel reset pull-up, Resistor_SMD:R_0603_1608Metric, symbol Device:R
- removed R216: DNP 10k fan PWM pull-up, Resistor_SMD:R_0603_1608Metric, symbol Device:R
- removed R253: 100k trackpad reset pull-up, Resistor_SMD:R_0603_1608Metric, symbol Device:R
- removed R255: 56k USB-C Rp default current CC2, Resistor_SMD:R_0603_1608Metric, symbol Device:R
- removed U62: USBLC6-2P6 trackpad USB ESD, Package_TO_SOT_SMD:SOT-666, symbol Power_Protection:USBLC6-2P6
- added C209: 3.9n fan FG filter, Capacitor_SMD:C_0402_1005Metric, symbol Device:C
- added C282: 100n TPS25810 AUX, Capacitor_SMD:C_0603_1608Metric, symbol Device:C
- added C283: 10u trackpad VBUS, Capacitor_SMD:C_1206_3216Metric, symbol Device:C
- added C284: 150u 10V TPS25810 input reservoir, Capacitor_Tantalum_SMD:CP_EIA-7343-31_Kemet-D, symbol Device:C_Polarized
- added Q60: 2N7002 physical host-VBUS USB connect gate, Package_TO_SOT_SMD:SOT-23, symbol Q_NMOS_SOT23_GSD:Q_NMOS_SOT23_GSD
- added R207: 100R fan PWM gate series, Resistor_SMD:R_0603_1608Metric, symbol Device:R
- added R256: 10k trackpad fault pull-up, Resistor_SMD:R_0603_1608Metric, symbol Device:R
- added U60: USBLC6-2P6 EC USB ESD, Package_TO_SOT_SMD:SOT-666, symbol Power_Protection:USBLC6-2P6
- added U62: TPD4E05U06 trackpad USB2/CC ESD, Package_SON:USON-10_2.5x1.0mm_P0.5mm, symbol Power_Protection:TPD4EUSB30
- added U63: TPS25810 attach-controlled trackpad Type-C source, Package_DFN_QFN:Texas_RVC0020A_WQFN-20-1EP_3x4mm_P0.5mm_EP1.6x2.6mm, symbol Interface_USB:TPS25810RVC
- added U64: TPS2553DDBVR trackpad 0.61A branch switch, Package_TO_SOT_SMD:SOT-23-6, symbol TPS2553D:TPS2553D
- C205: value 10u fan local bulk -> 10u 25V X7R fan local bulk; MPN (none) -> GRM31CR71E106KA12L; Manufacturer (none) -> Murata
- C206: value 100n fan local -> 100n 25V X7R fan local; MPN (none) -> GRM188R71E104KA01D; Manufacturer (none) -> Murata
- C208: renamed from U61; value USBLC6-2P6 touch USB ESD -> 100n EC USB switch local; footprint Package_TO_SOT_SMD:SOT-666 -> Capacitor_SMD:C_0603_1608Metric; symbol Power_Protection:USBLC6-2P6 -> Device:C
- C280: value 10u trackpad 5V local -> 100n TPS2553 input bypass; footprint Capacitor_SMD:C_1206_3216Metric -> Capacitor_SMD:C_0603_1608Metric
- C281: value 100n trackpad 3V3 sideband -> 100n TPS25810 input
- F200: value 750mA fan polyfuse -> 750mA 16V fan polyfuse; MPN (none) -> 1206L075/16WR; Manufacturer (none) -> Littelfuse
- J52: renamed from R207; value 100R fan PWM gate series -> Delta BFB04512HHA-CZ0T: GND, fused 12V, FG, PWM; footprint Resistor_SMD:R_0603_1608Metric -> Connector_JST:JST_GH_SM04B-GHS-TB_1x04-1MP_P1.25mm_Horizontal; symbol Device:R -> Connector_Generic:Conn_01x04; Contacts (none) -> SSHL-002T-P0.2; EndpointDatasheet (none) -> https://www.delta-fan.com/Download/Spec/BFB04512HHA-CZ0T.pdf; EndpointElectricalContract (none) -> 12V_NOMINAL_5.0_TO_13.5V;0.26A_MAX;25KHZ_OPEN_DRAIN_PWM;FLO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; EndpointMPN (none) -> BFB04512HHA-CZ0T; EndpointManufacturer (none) -> Delta Electronics; EndpointWireMap (none) -> 1=BLACK/GND;2=RED/+12V;3=WHITE/FG;4=YELLOW/PWM; MPN (none) -> SM04B-GHS-TB; Manufacturer (none) -> JST; MatingHousing (none) -> GHR-04V-S
- J53, J54, J56: footprint Connector_PinHeader_2.54mm:PinHeader_1x02_P2.54mm_Vertical -> Connector_JST:JST_GH_SM02B-GHS-TB_1x02-1MP_P1.25mm_Horizontal; Contacts (none) -> SSHL-002T-P0.2; MPN (none) -> SM02B-GHS-TB; Manufacturer (none) -> JST; MatingHousing (none) -> GHR-02V-S
- J58: MPN (none) -> 105450-0101; Manufacturer (none) -> Molex
- Q200: value Fan PWM open-drain sink -> 2N7002KT1G fan PWM open-drain sink; MPN (none) -> 2N7002KT1G; Manufacturer (none) -> onsemi
- R202: renamed from R203; value 22R touch DM series -> 10k EC USB default-disconnect pull-up
- R206: value 10k fan tach pull-up -> 8.2k fan FG pull-up; MPN (none) -> RC0603FR-078K2L; Manufacturer (none) -> Yageo
- R208: value 100k fan PWM default off -> 100k gate pull-down; fan defaults full speed; MPN (none) -> RC0603FR-07100KL; Manufacturer (none) -> Yageo
- R252: value 10k trackpad INT pull-up -> 43.2k 1% TPS2553 trackpad ILIM 0.61A nominal; MPN (none) -> RC0603FR-0743K2L; Manufacturer (none) -> Yageo
- R254: value 56k USB-C Rp default current CC1 -> 100k 1% <=100ppm TPS25810 REF
- U61: renamed from U60; value USBLC6-2P6 EC USB ESD -> TS3USB30EDGSR EC USB host-state isolation; footprint Package_TO_SOT_SMD:SOT-666 -> Package_SO:TSSOP-10_3x3mm_P0.5mm; symbol Power_Protection:USBLC6-2P6 -> Interface_USB:TS3USB30EDGSR; MPN (none) -> TS3USB30EDGSR; Manufacturer (none) -> Texas Instruments
Connections:
- net TOUCH_USB_DM is gone; now on net MCU_3V3: R202.1
- net TPAD_INT_N is gone; now on net GND: R252.2
- net EC_HOST_USB_DM: now also U61.8 (D1-), U60.3 (I/O2), U60.4 (I/O2); no longer R201.1, U61.3 (I/O2), U61.4 (I/O2)
- net EC_HOST_USB_DP: now also U61.2 (D1+), U60.1 (I/O1), U60.6 (I/O1); no longer R200.1, U61.1 (I/O1), U61.6 (I/O1)
- net FAN_PWM: now also R207.1; no longer J52.1
- net FAN_PWM_CONN: now also J52.4 (Pin_4)
- net FAN_PWM_GATE: now also R207.2; no longer J52.2
- net FAN_TACH: now also J52.3 (Pin_3), C209.1
- net GND: now also J52.1 (Pin_1), U61.1 (S), U61.5 (GND), C209.2, C282.2, C283.2, C284.2, Q60.2 (S), U60.2 (GND), U62.3 (GND), U62.8 (GND), U63.12 (GND), U63.21 (GND), U63.7 (CHG), U63.8 (CHG_HI), U64.2 (GND); no longer J58.A5 (CC1), J58.B5 (CC2), R254.2, U61.2 (GND)
- net SYS_3V3: now also C282.1, U63.5 (AUX)
- net SYS_5V: now also C280.1, U64.1 (IN); no longer C208.5 (VBUS), F200.1
- net TPAD_CONN_DM: now also U62.2 (D1-)
- net TPAD_CONN_DP: now also U62.1 (D1+)
- net FAN_5V renamed FAN_12V
- net FAN_12V: now also J52.2 (Pin_2)
- removed net LCD_BL_EN: C280.1, C281.1, J50.4 (Pin_4), J58.A4 (VBUS), J58.A9 (VBUS), J58.B4 (VBUS), J58.B9 (VBUS), R206.1, R209.1, R210.1, R215.1, R252.1, R254.1, U61.5 (VBUS)
- removed net TOUCH_CONN_DM: C208.3 (I/O2), C208.4 (I/O2), R202.2
- net TOUCH_CONN_DP renamed MCU_3V3
- net MCU_3V3: now also J50.4 (Pin_4), R206.1, R209.1, R210.1, R215.1, U61.10 (VCC), R256.1, U60.5 (VBUS); no longer C208.6 (I/O1)
- new net EC_USB_ISO_DM: R201.1, U61.6 (D-)
- new net EC_USB_ISO_DP: R200.1, U61.4 (D+)
- new net EC_USB_OE_N: Q60.3 (D), R202.2, U61.9 (~{OE})
- new net INTERNAL_USB_VBUS_VALID: Q60.1 (G)
- new net MU_12V: F200.1
- new net MU_HOST_ACTIVE: U63.6 (EN), U64.3 (EN)
- new net TPAD_5V: C283.1, J58.A4 (VBUS), J58.A9 (VBUS), J58.B4 (VBUS), J58.B9 (VBUS), U63.14 (OUT), U63.15 (OUT)
- new net TPAD_5V_PRE: C281.1, C284.1, U63.2 (IN1), U63.3 (IN1), U63.4 (IN2), U64.6 (OUT)
- new net TPAD_CC1: J58.A5 (CC1), U62.4 (D2+), U63.11 (CC1)
- new net TPAD_CC2: J58.B5 (CC2), U62.5 (D2-), U63.13 (CC2)
- new net TPAD_ILIM: R252.1, U64.5 (ILIM)
- new net TPAD_REF: R254.1, U63.10 (REF)
- new net TPAD_REF_RTN: R254.2, U63.9 (REF_RTN)
- new net TRACKPAD_FAULT_N: R256.2, U63.1 (~{FAULT}), U64.4 (~{FAULT})
- no-connect marks 18 -> 21
Other:
- note added: "== Internal laptop services: EC USB, trackpad, fan, lid, thermal =="
- note added: "Cooling default is copper spreader/heatpipe/vapor chamber plus the released Delta blower; no Peltier/TEC in the base design. Solid-state AirJet-style modules are a future mechanical option only."
- note added: "Delta contract: 0.26A maximum, 35% minimum start duty, FG is open collector at 2 pulses/revolution, and 0% PWM stops the fan. Gate pull-down makes an unpowered/reset EC command full fan speed, not fan-off."
- note added: "EC enumerates over Mu USB2_P3 only after the carrier-generated physical INTERNAL_USB_VBUS is above the supervisor threshold. U61 defaults disconnected so an always-powered EC cannot back-drive an off host PHY."
- note added: "J52 is released for Delta BFB04512HHA-CZ0T: fused MU_12V, 8.2k/3.9n FG interface, and 25kHz open-drain PWM. Floating PWM commands full speed; firmware never drives the fan PWM node high."
- note added: "J58 is the only trackpad connector. TPS2553 isolates the 150uF input reservoir; TPS25810 applies connector VBUS only after attach."
- note added: "The Intehill controller remains a bench fixture/fallback and is not populated on the motherboard."
- note added: "The blower shares MU_12V: it is available whenever the Mu is powered. Thermal policy commands full fan and host throttle/shutdown before any final MU_12V cut; after a cut the passive coldplate/heatpipe/fin stack absorbs residual heat while heat generation is removed."
- note added: "The internal display uses the Mu onboard eDP connector and needs no motherboard USB path."
- note added: "The verified B160QAN03.K panel is non-touch; USB2_P4 is paired with native USB-C port 2."
- note added: "Trackpad uses Mu USB2_P8 as a direct internal USB HID device. TRACKPAD_FAULT_N is pulled up to the EC; S3 removes trackpad VBUS, so wake-from-trackpad is not supported."
- note removed: "== DNP low-speed display/backlight service harness =="
- note removed: "== Internal laptop services: EC USB, touch, trackpad, fan, lid, display service =="
- note removed: "== Internal touchscreen USB2 link on Mu USB2_P4 =="
- note removed: "Cooling default is copper spreader/heatpipe/vapor chamber plus quiet blower; no Peltier/TEC in the base design."
- note removed: "Display-specific retained-controller and raw-panel paths live on sheets 10 and 11."
- note removed: "EC enumerates to the x86 host as a plain USB device over Mu USB2_P3; firmware exposes keyboard/power/telemetry."
- note removed: "Fan PWM/tach are EC-owned. J52 uses fused 5V, 3.3V tach pull-up, and an open-drain PWM sink."
- note removed: "J51 and J55 are DNP alternate/service harnesses; sheets 10/11 own the real display video paths."
- note removed: "J58 is the normal trackpad connector for a USB-C cable trackpad. J57 is DNP fallback only if the trackpad is gutted to FFC/wires."
- note removed: "Solid-state AirJet-style modules are a future mechanical option, not the assumed electrical baseline."
- note removed: "Touchscreen USB is separate on Mu USB2_P4; sheet 11 owns the retained Intehill USB-C touch/power path."
- note removed: "Trackpad uses Mu USB2_P8 as a direct internal USB HID pointing device; EC only owns reset/interrupt/sideband."
- moved on the sheet: R202

Commit message: Wire the trackpad directly over USB2 and record audit holds
Parts:
- removed C281: 100n TPS25810 input, Capacitor_SMD:C_0603_1608Metric, symbol Device:C
- removed C282: 100n TPS25810 AUX, Capacitor_SMD:C_0603_1608Metric, symbol Device:C
- removed C284: 150u 10V TPS25810 input reservoir, Capacitor_Tantalum_SMD:CP_EIA-7343-31_Kemet-D, symbol Device:C_Polarized
- removed J58: Internal USB-C receptacle for cable-attached USB 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, Connector_USB:USB_C_Receptacle_Molex_105450-0101, symbol USB_C_Receptacle_Passive:USB_C_Receptacle_Passive
- removed R254: 100k 1% <=100ppm TPS25810 REF, Resistor_SMD:R_0603_1608Metric, symbol Device:R
- removed U64: TPS2553DDBVR trackpad 0.61A branch switch, Package_TO_SOT_SMD:SOT-23-6, symbol TPS2553D:TPS2553D
- added J58: Field-soldered trackpad USB2 cable: GND/D-/D+/VBUS, ducktop2:USB2_Trackpad_Cable_SolderPads_1x04_P2.54mm, symbol Connector_Generic:Conn_01x04
- C283: value 10u trackpad VBUS -> 10u trackpad cable VBUS
- U62: value TPD4E05U06 trackpad USB2/CC ESD -> TPD4E05U06 wired trackpad USB2 ESD
- U64: renamed from U63; value TPS25810 attach-controlled trackpad Type-C source -> TPS2553DDBVR trackpad 0.61A branch switch; footprint Package_DFN_QFN:Texas_RVC0020A_WQFN-20-1EP_3x4mm_P0.5mm_EP1.6x2.6mm -> Package_TO_SOT_SMD:SOT-23-6; symbol Interface_USB:TPS25810RVC -> TPS2553D:TPS2553D; MPN TPS25810RVCR -> TPS2553DDBVR
Connections:
- net SYS_3V3 is gone; now on net TPAD_ILIM: U64.5 (ILIM)
- net GND: now also U64.2 (GND), J58.1 (Pin_1); no longer U64.12 (GND), U64.21 (GND), U64.7 (CHG), U64.8 (CHG_HI)
- net MU_HOST_ACTIVE: now also U64.3 (EN); no longer U64.6 (EN)
- net SYS_5V: now also U64.1 (IN)
- net TPAD_5V: now also U64.6 (OUT), J58.4 (Pin_4); no longer U64.14 (OUT), U64.15 (OUT)
- net TPAD_CONN_DM: now also J58.2 (Pin_2)
- net TPAD_CONN_DP: now also J58.3 (Pin_3)
- net TRACKPAD_FAULT_N: now also U64.4 (~{FAULT}); no longer U64.1 (~{FAULT})
- removed net TPAD_5V_PRE: U64.2 (IN1), U64.3 (IN1), U64.4 (IN2)
- net TPAD_CC1: no longer names the net of U62.4 (D2+)
- net TPAD_CC1: no longer U64.11 (CC1)
- net TPAD_CC2: no longer names the net of U62.5 (D2-)
- net TPAD_CC2: no longer U64.13 (CC2)
- removed net TPAD_REF: U64.10 (REF)
- removed net TPAD_REF_RTN: U64.9 (REF_RTN)
- no-connect marks 21 -> 8
Other:
- note added: "J58 is four field-soldered pads for a cut USB 2.0 Standard-A-to-USB-C cable: 1=GND, 2=D-, 3=D+, 4=VBUS. The USB-C plug's compliant 56k Rp handles trackpad-side CC; U64 provides current limiting and host-off isolation."
- note removed: "J58 is the only trackpad connector. TPS2553 isolates the 150uF input reservoir; TPS25810 applies connector VBUS only after attach."

Commit message: Fix trackpad USB and duplicate footprints
Parts:
- C280: MPN (none) -> GRM188R71E104KA01D; Manufacturer (none) -> Murata
- C283: MPN (none) -> GRM31CR71E106KA12L; Manufacturer (none) -> Murata
Changed lines of the file:
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@@
   (property "Footprint" "Capacitor_SMD:C_0603_1608Metric" (at 330.2 271.78 0) (effects (font (size 1.27 1.27)) (hide yes)))
   (property "Datasheet" "" (at 330.2 271.78 0) (effects (font (size 1.27 1.27)) (hide yes)))
+  (property "Manufacturer" "Murata" (at 330.2 271.78 0) (effects (font (size 1.27 1.27)) (hide yes)))
+  (property "MPN" "GRM188R71E104KA01D" (at 330.2 271.78 0) (effects (font (size 1.27 1.27)) (hide yes)))
   (pin "1")
   (pin "2")
@@
   (property "Footprint" "Capacitor_SMD:C_1206_3216Metric" (at 330.2 309.88 0) (effects (font (size 1.27 1.27)) (hide yes)))
   (property "Datasheet" "" (at 330.2 309.88 0) (effects (font (size 1.27 1.27)) (hide yes)))
+  (property "Manufacturer" "Murata" (at 330.2 309.88 0) (effects (font (size 1.27 1.27)) (hide yes)))
+  (property "MPN" "GRM31CR71E106KA12L" (at 330.2 309.88 0) (effects (font (size 1.27 1.27)) (hide yes)))
   (pin "1")
   (pin "2")

Commit message: Assign 327 BOM MPNs across 11 schematic sheets (370→43 gaps)
Closes 370 BOM procurement gaps by assigning Yageo resistor and Murata
capacitor MPNs to all passive components in the project's 11 schematic
sheets. 43 intentional holds remain for design-review items (crystal
loads, audio AC-coupling, VCAP, C0G timing, maker MCU 4.7u 0402s).

Key changes:
- 205 resistors assigned (Yageo RC0603/RT0603 series)
- 124 capacitors assigned (Murata GRM series, matching footprint body size)
- Fixed C183: 4.7u MPN→1u (GRM21BR71A105KA01L)
- Fixed C795/C840: upgraded to 50V rating (GRM21BR71H105KA12L)
- Generated fresh inventory: 1173 components, 43 remaining gaps
Parts:
- C202, C207, C208: MPN (none) -> GRM188R71H104KA93D; Manufacturer (none) -> Murata
- R200, R201, R250, R251: MPN (none) -> RC0603FR-0722RL; Manufacturer (none) -> Yageo
- R202, R209, R210, R215, R256: MPN (none) -> RC0603FR-0710KL; Manufacturer (none) -> Yageo
Changed lines of the file:
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@@
   (property "Footprint" "Resistor_SMD:R_0603_1608Metric" (at 20.32 76.2 0) (effects (font (size 1.27 1.27)) (hide yes)))
   (property "Datasheet" "" (at 20.32 76.2 0) (effects (font (size 1.27 1.27)) (hide yes)))
+  (property "Manufacturer" "Yageo" (at 20.32 76.2 0) (effects (font (size 1.27 1.27)) (hide yes)))
+  (property "MPN" "RC0603FR-0722RL" (at 20.32 76.2 0) (effects (font (size 1.27 1.27)) (hide yes)))
   (pin "1")
   (pin "2")
@@
   (property "Footprint" "Resistor_SMD:R_0603_1608Metric" (at 20.32 88.9 0) (effects (font (size 1.27 1.27)) (hide yes)))
   (property "Datasheet" "" (at 20.32 88.9 0) (effects (font (size 1.27 1.27)) (hide yes)))
+  (property "Manufacturer" "Yageo" (at 20.32 88.9 0) (effects (font (size 1.27 1.27)) (hide yes)))
+  (property "MPN" "RC0603FR-0722RL" (at 20.32 88.9 0) (effects (font (size 1.27 1.27)) (hide yes)))
   (pin "1")
   (pin "2")
@@
   (property "Footprint" "Resistor_SMD:R_0603_1608Metric" (at 195.58 63.5 0) (effects (font (size 1.27 1.27)) (hide yes)))
   (property "Datasheet" "" (at 195.58 63.5 0) (effects (font (size 1.27 1.27)) (hide yes)))
+  (property "Manufacturer" "Yageo" (at 195.58 63.5 0) (effects (font (size 1.27 1.27)) (hide yes)))
+  (property "MPN" "RC0603FR-0710KL" (at 195.58 63.5 0) (effects (font (size 1.27 1.27)) (hide yes)))
   (pin "1")
   (pin "2")
@@
   (property "Footprint" "Capacitor_SMD:C_0603_1608Metric" (at 284.48 63.5 0) (effects (font (size 1.27 1.27)) (hide yes)))
   (property "Datasheet" "" (at 284.48 63.5 0) (effects (font (size 1.27 1.27)) (hide yes)))
+  (property "Manufacturer" "Murata" (at 284.48 63.5 0) (effects (font (size 1.27 1.27)) (hide yes)))
+  (property "MPN" "GRM188R71H104KA93D" (at 284.48 63.5 0) (effects (font (size 1.27 1.27)) (hide yes)))
   (pin "1")
   (pin "2")
@@
   (property "Footprint" "Resistor_SMD:R_0603_1608Metric" (at 20.32 259.08 0) (effects (font (size 1.27 1.27)) (hide yes)))
   (property "Datasheet" "" (at 20.32 259.08 0) (effects (font (size 1.27 1.27)) (hide yes)))
+  (property "Manufacturer" "Yageo" (at 20.32 259.08 0) (effects (font (size 1.27 1.27)) (hide yes)))
+  (property "MPN" "RC0603FR-0722RL" (at 20.32 259.08 0) (effects (font (size 1.27 1.27)) (hide yes)))
   (pin "1")
   (pin "2")
@@
   (property "Footprint" "Resistor_SMD:R_0603_1608Metric" (at 20.32 271.78 0) (effects (font (size 1.27 1.27)) (hide yes)))
   (property "Datasheet" "" (at 20.32 271.78 0) (effects (font (size 1.27 1.27)) (hide yes)))
+  (property "Manufacturer" "Yageo" (at 20.32 271.78 0) (effects (font (size 1.27 1.27)) (hide yes)))
+  (property "MPN" "RC0603FR-0722RL" (at 20.32 271.78 0) (effects (font (size 1.27 1.27)) (hide yes)))
   (pin "1")
   (pin "2")
@@
   (property "Footprint" "Resistor_SMD:R_0603_1608Metric" (at 379.73 322.58 0) (effects (font (size 1.27 1.27)) (hide yes)))
   (property "Datasheet" "" (at 379.73 322.58 0) (effects (font (size 1.27 1.27)) (hide yes)))
+  (property "Manufacturer" "Yageo" (at 379.73 322.58 0) (effects (font (size 1.27 1.27)) (hide yes)))
+  (property "MPN" "RC0603FR-0710KL" (at 379.73 322.58 0) (effects (font (size 1.27 1.27)) (hide yes)))
   (pin "1")
   (pin "2")
@@
   (property "Footprint" "Resistor_SMD:R_0603_1608Metric" (at 330.2 130.81 0) (effects (font (size 1.27 1.27)) (hide yes)))
   (property "Datasheet" "" (at 330.2 130.81 0) (effects (font (size 1.27 1.27)) (hide yes)))
+  (property "Manufacturer" "Yageo" (at 330.2 130.81 0) (effects (font (size 1.27 1.27)) (hide yes)))
+  (property "MPN" "RC0603FR-0710KL" (at 330.2 130.81 0) (effects (font (size 1.27 1.27)) (hide yes)))
   (pin "1")
   (pin "2")
@@
   (property "Footprint" "Resistor_SMD:R_0603_1608Metric" (at 330.2 160.02 0) (effects (font (size 1.27 1.27)) (hide yes)))
   (property "Datasheet" "" (at 330.2 160.02 0) (effects (font (size 1.27 1.27)) (hide yes)))
+  (property "Manufacturer" "Yageo" (at 330.2 160.02 0) (effects (font (size 1.27 1.27)) (hide yes)))
+  (property "MPN" "RC0603FR-0710KL" (at 330.2 160.02 0) (effects (font (size 1.27 1.27)) (hide yes)))
   (pin "1")
   (pin "2")
@@
   (property "Footprint" "Capacitor_SMD:C_0603_1608Metric" (at 330.2 172.72 0) (effects (font (size 1.27 1.27)) (hide yes)))
   (property "Datasheet" "" (at 330.2 172.72 0) (effects (font (size 1.27 1.27)) (hide yes)))
+  (property "Manufacturer" "Murata" (at 330.2 172.72 0) (effects (font (size 1.27 1.27)) (hide yes)))
+  (property "MPN" "GRM188R71H104KA93D" (at 330.2 172.72 0) (effects (font (size 1.27 1.27)) (hide yes)))
   (pin "1")
   (pin "2")
@@
   (property "Footprint" "Resistor_SMD:R_0603_1608Metric" (at 490.22 160.02 0) (effects (font (size 1.27 1.27)) (hide yes)))
   (property "Datasheet" "" (at 490.22 160.02 0) (effects (font (size 1.27 1.27)) (hide yes)))
+  (property "Manufacturer" "Yageo" (at 490.22 160.02 0) (effects (font (size 1.27 1.27)) (hide yes)))
+  (property "MPN" "RC0603FR-0710KL" (at 490.22 160.02 0) (effects (font (size 1.27 1.27)) (hide yes)))
   (pin "1")
   (pin "2")
@@
   (property "Footprint" "Capacitor_SMD:C_0603_1608Metric" (at 490.22 172.72 0) (effects (font (size 1.27 1.27)) (hide yes)))
   (property "Datasheet" "" (at 490.22 172.72 0) (effects (font (size 1.27 1.27)) (hide yes)))
-  (pin "1")
-  (pin "2")
+  (property "Manufacturer" "Murata" (at 490.22 172.72 0) (effects (font (size 1.27 1.27)) (hide yes)))
+  (property "MPN" "GRM188R71H104KA93D" (at 490.22 172.72 0) (effects (font (size 1.27 1.27)) (hide yes)))
+  (pin "1")
+  (pin "2")

Commit message: P1.5: Add EC DFU programming path: BOOT0 button (SW2) + rear-edge USB-C prog port (J70/U70/U71/D70) in 08_internal_services
Parts:
- added C220: 1u prog VBUS LDO input, Capacitor_SMD:C_0603_1608Metric, symbol Device:C
- added C221: 100n prog 3V3 LDO output, Capacitor_SMD:C_0603_1608Metric, symbol Device:C
- added D70: BAT54WS prog VBUS OR-ing, Diode_SMD:D_SOD-323, symbol Device:D_Schottky
- added J70: USB-C EC prog, Connector_USB:USB_C_Receptacle_Molex_105450-0101, symbol Connector:USB_C_Receptacle
- added R220: 5.1k prog CC1 pulldown, Resistor_SMD:R_0603_1608Metric, symbol Device:R
- added R221: 5.1k prog CC2 pulldown, Resistor_SMD:R_0603_1608Metric, symbol Device:R
- added R222: 22R prog DP series, Resistor_SMD:R_0603_1608Metric, symbol Device:R
- added R223: 22R prog DM series, Resistor_SMD:R_0603_1608Metric, symbol Device:R
- added U70: USBLC6-2P6 prog port USB ESD, Package_TO_SOT_SMD:SOT-666, symbol Power_Protection:USBLC6-2P6
- added U71: AP2112K-3.3 prog VBUS LDO 600mA, Package_TO_SOT_SMD:SOT-23-5, symbol ducktop2:AP2112K-3.3
Connections:
- net MCU_USB_DM: now also U70.3 (I/O2)
- new net EC_PROG_3V3: C221.1
- new net EC_PROG_CONN_DM: R223.2
- new net EC_PROG_CONN_DP: R222.2
- new net EC_PROG_DM: R223.1
- new net EC_PROG_DP: R222.1
- new net EC_PROG_VBUS: C220.1
Other:
- note added: "== EC programming USB-C port (rear PCB edge, STM32 DFU bootloader) =="
- note added: "== Programming USB-C port section (DFU bootloader access) =="
- note added: "Hold BOOT0 (SW2) and tap Reset (SW1) on power-up to enter DFU. USB VBUS powers U71 LDO -> D70 -> MCU_3V3 rail when system is off."
- note added: "U70/R222/R223 tap MCU_USB_DP/DM. Unpowered U61 is high-Z, so no bus conflict during DFU."

Commit message: Fix ERC + annotation issues in EC DFU programming section (08)
- Move 7 stranded GND labels onto their correct pin connection points
- Reposition #PWR2ac409aa onto U71 GND pin (was double-moved off-point)
- Rename power symbols to digit-terminated refs (#PWR2302-2308); letter-
  terminated refs (e.g. #PWRf564ab8b) made SCH_REFERENCE::Split flag them
  as unannotated, triggering the netlist 'annotation errors' warning
- Align property Reference with instances reference for all 7 power symbols
- Add power:PWR_FLAG (#FLG071) on EC_PROG_VBUS to drive U71 VIN

ERC for /Internal Services/ section now reports zero violations (64 total
remaining are all pre-existing project-wide baseline). Netlist exports
cleanly with full section connectivity verified.
Connections:
- net EC_PROG_3V3: now also D70.1 (K), U71.5 (VOUT)
- net EC_PROG_CC1: now also J70.A5 (CC1), R220.1
- net EC_PROG_CC2: now also J70.B5 (CC2), R221.1
- net EC_PROG_CONN_DM: now also J70.A7 (D-), J70.B7 (D-)
- net EC_PROG_CONN_DP: now also J70.A6 (D+), J70.B6 (D+)
- net EC_PROG_DM: now also U70.3 (I/O2)
- net EC_PROG_DP: now also U70.1 (I/O1)
- net EC_PROG_VBUS: now also J70.A4 (VBUS), J70.A9 (VBUS), J70.B4 (VBUS), J70.B9 (VBUS), U70.5 (VBUS), U71.1 (VIN), U71.3 (EN)
- net GND: now also C220.2, C221.2, J70.A1 (GND), J70.A12 (GND), J70.B1 (GND), J70.B12 (GND), J70.SH (SHIELD), R220.2, R221.2, U70.2 (GND), U71.2 (GND)
- net MCU_3V3: now also D70.2 (A)
- net MCU_USB_DM: now also U70.4 (I/O2); no longer U70.3 (I/O2)
- net MCU_USB_DP: now also U70.6 (I/O1)
- no-connect marks 8 -> 18

Commit message: Regenerate child schematics to sync with current generators
The committed .kicad_sch carried stale embedded Manufacturer/MPN properties from the old per-component BOM approach (MPNs now live in verification/BOM_MPN_ASSIGNMENTS.md). Regenerating from the current generators strips those stale properties and clears the pre-existing Generated-source identity release-check failure. No connectivity change; ERC still 0 errors / 27 intentional warnings; schematic closure 1569/0.
Parts:
- removed C220: 1u prog VBUS LDO input, Capacitor_SMD:C_0603_1608Metric, symbol Device:C
- removed C221: 100n prog 3V3 LDO output, Capacitor_SMD:C_0603_1608Metric, symbol Device:C
- removed D70: BAT54WS prog VBUS OR-ing, Diode_SMD:D_SOD-323, symbol Device:D_Schottky
- removed J70: USB-C EC prog, Connector_USB:USB_C_Receptacle_Molex_105450-0101, symbol Connector:USB_C_Receptacle
- removed R220: 5.1k prog CC1 pulldown, Resistor_SMD:R_0603_1608Metric, symbol Device:R
- removed R221: 5.1k prog CC2 pulldown, Resistor_SMD:R_0603_1608Metric, symbol Device:R
- removed R222: 22R prog DP series, Resistor_SMD:R_0603_1608Metric, symbol Device:R
- removed R223: 22R prog DM series, Resistor_SMD:R_0603_1608Metric, symbol Device:R
- removed U70: USBLC6-2P6 prog port USB ESD, Package_TO_SOT_SMD:SOT-666, symbol Power_Protection:USBLC6-2P6
- removed U71: AP2112K-3.3 prog VBUS LDO 600mA, Package_TO_SOT_SMD:SOT-23-5, symbol ducktop2:AP2112K-3.3
- C202, C207, C208: MPN GRM188R71H104KA93D -> (none); Manufacturer Murata -> (none)
- R200, R201, R250, R251: MPN RC0603FR-0722RL -> (none); Manufacturer Yageo -> (none)
- R202, R209, R210, R215, R256: MPN RC0603FR-0710KL -> (none); Manufacturer Yageo -> (none)
Connections:
- no-connect marks 18 -> 8
Other:
- note removed: "== EC programming USB-C port (rear PCB edge, STM32 DFU bootloader) =="
- note removed: "== Programming USB-C port section (DFU bootloader access) =="
- note removed: "Hold BOOT0 (SW2) and tap Reset (SW1) on power-up to enter DFU. USB VBUS powers U71 LDO -> D70 -> MCU_3V3 rail when system is off."
- note removed: "U70/R222/R223 tap MCU_USB_DP/DM. Unpowered U61 is high-Z, so no bus conflict during DFU."
