File: 12_keyboard_daughterboard.kicad_sch (KiCad schematic)
At the start: 134 parts, among them J320 Keyboard FFC: MX ULP 5x14 mat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, J321 DNP keyboard bring-up/debug, SW320 Esc 1u, SW321 1 1u, SW322 2 1u, SW323 3 1u, SW324 4 1u, SW325 5 1u, SW326 6 1u, SW327 7 1u, SW328 8 1u, SW329 9 1u, SW330 0 1u, SW331 Minus 1u, SW332 Equal 1u, SW333 Backspace 1.75u, SW334 Tab 1.25u, SW335 Q 1u, SW336 W 1u, SW337 E 1u, SW338 R 1u, SW339 T 1u, SW340 Y 1u, SW341 U 1u, SW342 I 1u, SW343 O 1u, SW344 P 1u, SW345 [ 1u, SW346 ] 1u, SW347 Backslash 1u, SW348 Caps 1.5u, SW349 A 1u, SW350 S 1u, SW351 D 1u, SW352 F 1u, SW353 G 1u, SW354 H 1u, SW355 J 1u, SW356 K 1u, SW357 L 1u, SW358 Semicolon 1u, SW359 Quote 1u, SW360 Enter 1.75u, SW361 Shift L 1.75u, SW362 Z 1u, SW363 X 1u, SW364 C 1u, SW365 V 1u, SW366 B 1u, SW367 N 1u, SW368 M 1u, SW369 Comma 1u, SW370 Period 1u, SW371 Slash 1u, SW372 Up 1u, SW373 Shift R 1.25u, SW374 Ctrl 1u, SW375 Fn 1u, SW376 Super 1u, SW377 Alt L 1u, SW378 Space L 2.25u, SW379 Space R 2.25u, SW380 Alt R 1u, SW381 Menu 1u, SW382 Left 1u, SW383 Down 1u, SW384 Right 1u

Commit message: Publish the current Ducktop2 design
Parts:
- C320, C321, J321: ReleasedRevA (none) -> Not fitted; footprint omitted from manufactured PCB
- J320: symbol Connector_Generic:Conn_01x30 -> Conn_01x30_FFC_MP:Conn_01x30_FFC_MP; ReleasedRevA (none) -> Populated; MP hold-down pads are mechanical and netless
Other:
- note added: "J320 mirrors mainboard J310. Its MP hold-down pads are intentionally netless on manufactured Rev A; C320/C321/J321 are DNP and excluded from that PCB."
- note added: "Manufactured Rev A envelope is 273.5 x 80.0 mm; this schematic records its released population and connector contract."
- note removed: "J320 keeps the current 30-pin motherboard connector. KB_ROW5..7 and KB_COL14..15 are unused on this 65-key layout and may become spare EC GPIO."
- note removed: "Target physical envelope is about 300 x 80 mm using roughly 18.0-18.5 mm horizontal pitch and 16 mm row pitch."
Changed lines of the file:
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@@
 (text "== Ducktop2 MX ULP keyboard daughterboard ==" (at 20.32 12.7 0) (effects (font (size 1.27 1.27))))
 (text "65-key compact laptop-style layout, Cherry MX Ultra Low Profile tactile switches, one diode per key." (at 20.32 20.32 0) (effects (font (size 1.27 1.27))))
-(text "Target physical envelope is about 300 x 80 mm using roughly 18.0-18.5 mm horizontal pitch and 16 mm row pitch." (at 20.32 27.94 0) (effects (font (size 1.27 1.27))))
+(text "Manufactured Rev A envelope is 273.5 x 80.0 mm; this schematic records its released population and connector contract." (at 20.32 27.94 0) (effects (font (size 1.27 1.27))))
 (text "This sheet is the keyboard PCB itself: switches, matrix diodes, EC FFC, and bring-up notes." (at 20.32 35.56 0) (effects (font (size 1.27 1.27))))
 (text "== 5x14 switch matrix, diode direction locked for EC firmware ==" (at 20.32 55.88 0) (effects (font (size 1.27 1.27))))
@@
 (text "== J320 keyboard FFC / board-to-board connector ==" (at 20.32 250.19 0) (effects (font (size 1.27 1.27))))
 (symbol
-  (lib_id "Connector_Generic:Conn_01x30")
+  (lib_id "Conn_01x30_FFC_MP:Conn_01x30_FFC_MP")
   (at 165.1 340.36 0)
   (unit 1)
@@
   (property "Footprint" "Connector_FFC-FPC:Hirose_FH12-30S-0.5SH_1x30-1MP_P0.50mm_Horizontal" (at 165.1 340.36 0) (effects (font (size 1.27 1.27)) (hide yes)))
   (property "Datasheet" "" (at 165.1 340.36 0) (effects (font (size 1.27 1.27)) (hide yes)))
+  (property "ReleasedRevA" "Populated; MP hold-down pads are mechanical and netless" (at 165.1 340.36 0) (effects (font (size 1.27 1.27)) (hide yes)))
   (pin "1")
   (pin "2")
@@
   (pin "29")
   (pin "30")
+  (pin "MP")
   (instances
     (project "ducktop2"
@@
   (exclude_from_sim no)
   (in_bom no)
-  (on_board yes)
+  (on_board no)
   (dnp yes)
   (property "Reference" "C320" (at 350.52 274.32 0) (effects (font (size 1.27 1.27))))
@@
   (property "Footprint" "Capacitor_SMD:C_0603_1608Metric" (at 350.52 276.86 0) (effects (font (size 1.27 1.27)) (hide yes)))
   (property "Datasheet" "" (at 350.52 276.86 0) (effects (font (size 1.27 1.27)) (hide yes)))
+  (property "ReleasedRevA" "Not fitted; footprint omitted from manufactured PCB" (at 350.52 276.86 0) (effects (font (size 1.27 1.27)) (hide yes)))
   (pin "1")
   (pin "2")
@@
   (exclude_from_sim no)
   (in_bom no)
-  (on_board yes)
+  (on_board no)
   (dnp yes)
   (property "Reference" "C321" (at 350.52 289.56 0) (effects (font (size 1.27 1.27))))
@@
   (property "Footprint" "Capacitor_SMD:C_1206_3216Metric" (at 350.52 292.1 0) (effects (font (size 1.27 1.27)) (hide yes)))
   (property "Datasheet" "" (at 350.52 292.1 0) (effects (font (size 1.27 1.27)) (hide yes)))
+  (property "ReleasedRevA" "Not fitted; footprint omitted from manufactured PCB" (at 350.52 292.1 0) (effects (font (size 1.27 1.27)) (hide yes)))
   (pin "1")
   (pin "2")
@@
   (exclude_from_sim no)
   (in_bom no)
-  (on_board yes)
+  (on_board no)
   (dnp yes)
   (property "Reference" "J321" (at 350.52 337.82 0) (effects (font (size 1.27 1.27))))
@@
   (property "Footprint" "Connector_PinHeader_2.54mm:PinHeader_1x04_P2.54mm_Vertical" (at 350.52 340.36 0) (effects (font (size 1.27 1.27)) (hide yes)))
   (property "Datasheet" "" (at 350.52 340.36 0) (effects (font (size 1.27 1.27)) (hide yes)))
+  (property "ReleasedRevA" "Not fitted; footprint omitted from manufactured PCB" (at 350.52 340.36 0) (effects (font (size 1.27 1.27)) (hide yes)))
   (pin "1")
   (pin "2")
@@
 (text "Use MX6C-T3NB Cherry MX ULP tactile switches. The project footprint has unnumbered mechanical solder tabs; only switch pins 1/2 enter the matrix." (at 20.32 429.26 0) (effects (font (size 1.27 1.27))))
 (text "D320-D384 are 1N4148W/SOD-323 class signal diodes. Diode pin 2 is anode on KB_ROWn; pin 1 is cathode at the per-key switch node." (at 20.32 436.88 0) (effects (font (size 1.27 1.27))))
-(text "J320 keeps the current 30-pin motherboard connector. KB_ROW5..7 and KB_COL14..15 are unused on this 65-key layout and may become spare EC GPIO." (at 20.32 444.5 0) (effects (font (size 1.27 1.27))))
+(text "J320 mirrors mainboard J310. Its MP hold-down pads are intentionally netless on manufactured Rev A; C320/C321/J321 are DNP and excluded from that PCB." (at 20.32 444.5 0) (effects (font (size 1.27 1.27))))
 (text "MX ULP hotswap is not planned: use stencil + reflow/hot plate for production and validate rework on a small coupon first." (at 20.32 452.12 0) (effects (font (size 1.27 1.27))))
 (text "Use split space in rev A. Treat Backspace, Enter, left Shift, and both Space keys as mechanical stabilizer/keycap-risk items before full board release." (at 20.32 459.74 0) (effects (font (size 1.27 1.27))))
@@
 (sheet_instances
   (path "/e5f63080-4501-5e30-a9d3-cbf1e4a2a151"
-    (page "13")
+    (page "K1")
   )
 )

Commit message: Apply BOM to radio + keyboard daughterboards, add Cherry MX switch 3D models
radio_daughterboard/:
- 74 MPNs assigned (33 resistors, 41 caps) across 4 schematic sheets
- 129 BOM gaps reduced to 7 (mounting holes H1-H4, DNP connectors J44/J72/J330)

12_keyboard_daughterboard/:
- 134 MPNs assigned: 65× 1N4148W-7-F diodes, 65× Cherry MX4A-L1NA switches,
  2× caps, 2× connectors
- BOM gaps eliminated: 134 → 0

3D models:
- Added Cherry_MX_ULP_SMD.step to ducktop2.3dshapes/ (65 Cherry MX switch
  footprints on keyboard daughterboard now have 3D models)
- Created gen/add_pcb_3d_models.py script for future 3D model assignments
- 57 footprints remain without models (MountingHole, TestPoint, Tag-Connect,
  and custom ducktop2 components — need manufacturer STEP files)

gen/:
- apply_bom_radio_daughterboard.py: radio daughterboard BOM catalog
- apply_bom_keyboard_daughterboard.py: keyboard daughterboard BOM catalog
- add_pcb_3d_models.py: automated 3D model path inserter
Parts:
- C320: MPN (none) -> GRM188R71H104KA93D; Manufacturer (none) -> Murata
- C321: MPN (none) -> GRM31CR71E106KA12L; Manufacturer (none) -> Murata
- D320, D321, D322, D323, D324, D325, D326, D327, D328, D329, D330, D331, D332, D333, D334, D335, D336, D337, D338, D339, D340, D341, D342, D343, D344, D345, D346, D347, D348, D349, D350, D351, D352, D353, D354, D355, D356, D357, D358, D359, D360, D361, D362, D363, D364, D365, D366, D367, D368, D369, D370, D371, D372, D373, D374, D375, D376, D377, D378, D379, D380, D381, D382, D383, D384: MPN (none) -> 1N4148W-7-F; Manufacturer (none) -> Diodes Incorporated
- J320: MPN (none) -> FH12-30S-0.5SH(55); Manufacturer (none) -> Hirose
- J321: MPN (none) -> TMM-104-01-T-S; Manufacturer (none) -> Samtec
- SW320, SW321, SW322, SW323, SW324, SW325, SW326, SW327, SW328, SW329, SW330, SW331, SW332, SW333, SW334, SW335, SW336, SW337, SW338, SW339, SW340, SW341, SW342, SW343, SW344, SW345, SW346, SW347, SW348, SW349, SW350, SW351, SW352, SW353, SW354, SW355, SW356, SW357, SW358, SW359, SW360, SW361, SW362, SW363, SW364, SW365, SW366, SW367, SW368, SW369, SW370, SW371, SW372, SW373, SW374, SW375, SW376, SW377, SW378, SW379, SW380, SW381, SW382, SW383, SW384: MPN (none) -> MX4A-L1NA; Manufacturer (none) -> Cherry

Commit message: Regenerate child schematics to sync with current generators
The committed .kicad_sch carried stale embedded Manufacturer/MPN properties from the old per-component BOM approach (MPNs now live in verification/BOM_MPN_ASSIGNMENTS.md). Regenerating from the current generators strips those stale properties and clears the pre-existing Generated-source identity release-check failure. No connectivity change; ERC still 0 errors / 27 intentional warnings; schematic closure 1569/0.
Parts:
- C320: MPN GRM188R71H104KA93D -> (none); Manufacturer Murata -> (none)
- C321: MPN GRM31CR71E106KA12L -> (none); Manufacturer Murata -> (none)
- D320, D321, D322, D323, D324, D325, D326, D327, D328, D329, D330, D331, D332, D333, D334, D335, D336, D337, D338, D339, D340, D341, D342, D343, D344, D345, D346, D347, D348, D349, D350, D351, D352, D353, D354, D355, D356, D357, D358, D359, D360, D361, D362, D363, D364, D365, D366, D367, D368, D369, D370, D371, D372, D373, D374, D375, D376, D377, D378, D379, D380, D381, D382, D383, D384: MPN 1N4148W-7-F -> (none); Manufacturer Diodes Incorporated -> (none)
- J320: MPN FH12-30S-0.5SH(55) -> (none); Manufacturer Hirose -> (none)
- J321: MPN TMM-104-01-T-S -> (none); Manufacturer Samtec -> (none)
- SW320, SW321, SW322, SW323, SW324, SW325, SW326, SW327, SW328, SW329, SW330, SW331, SW332, SW333, SW334, SW335, SW336, SW337, SW338, SW339, SW340, SW341, SW342, SW343, SW344, SW345, SW346, SW347, SW348, SW349, SW350, SW351, SW352, SW353, SW354, SW355, SW356, SW357, SW358, SW359, SW360, SW361, SW362, SW363, SW364, SW365, SW366, SW367, SW368, SW369, SW370, SW371, SW372, SW373, SW374, SW375, SW376, SW377, SW378, SW379, SW380, SW381, SW382, SW383, SW384: MPN MX4A-L1NA -> (none); Manufacturer Cherry -> (none)
