File: ducktop2.kicad_pcb (KiCad board)
At the start: 6 copper layers, 358 x 185 mm, 1170 parts, among them J10 Amphenol MDT420M01001 M-key N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, J11 USB-C dual-role data/PD port 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, J12 USB-C source-only data port J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, J16 Case power/reset button harne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, J190 AUX/SOLAR protected screw ter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, J2 3S pack power + cell-tap harn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, J21 USB-C dual-role data/PD port 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, J22 USB-C source-only data port J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, J23 USB-C source-only data port J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, J2300 DF40C 60-pin optional radio d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, J30 External HDMI-A from TCP0, J310 Mainboard keyboard FFC to MX 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, J4 TC2030 Cortex SWD: VTref/SWDI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, J40 Amphenol MDT420E01001 E-key W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, J41 SSD1306 OLED A 4-pin GND/VDD/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, J420 Left 8-ohm BTL speaker; pin 1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, J421 Right 8-ohm BTL speaker; pin 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, J45 SSD1306 OLED B 4-pin GND/VDD/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, J500 JXD1-1022NL recessed 1GbE RJ45, J52 Delta BFB04512HHA-CZ0T: GND, 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, J53 Lid/hall switch, J54 Skin/hinge NTC, J56 Mu heatsink/spreader NTC, J58 Field-soldered trackpad USB2 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, J9 RTC backup coin-cell header, J901 JST PUD 2x20 protected maker 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, J902 TC2030 Cortex SWD: VTref/SWDI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, Q11 CSD18540Q5B reverse-pack FET A, Q12 CSD18540Q5B reverse-pack FET B, Q13 CSD19537Q3 100V AUX reverse F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, Q14 BSS138 fast reverse-gate pull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, Q15 SiSS4409DN 40V reverse-blocki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, Q16 SiSS4409DN 40V reverse-blocki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, Q17 SiSS4409DN 40V reverse-blocki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, Q18 SiSS4409DN 40V reverse-blocki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, Q200 2N7002KT1G fan PWM open-drain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, Q2001 2N7002K DFP USB2 enable inver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, Q2002 2N7002K DFP USB2 enable inver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, Q21 SiSS4409DN 40V reverse-blocki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, Q22 SiSS4409DN 40V reverse-blocki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, Q23 SiSS4409DN 40V reverse-blocki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, Q2300 2N7002K radio-PG USB enable, Q24 SiSS4409DN 40V reverse-blocki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, Q25 CSD17575Q3 BQ25798 ship FET, Q50 BSS138 HDMI bias gate, Q60 2N7002 physical host-VBUS USB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, Q700 BSS138 active-high charger en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, Q701 BSS138 pack protector latch r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, Q702 BSS138 QON open-drain pulse, Q703 CSD18540Q5B BQ77915 discharge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, Q704 CSD18540Q5B BQ77915 charge FET, Q750 BSS138 fail-off EN/UVLO clamp, Q751 BSS138 active-high enable rel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, Q901 2N7002 physical host-VBUS USB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, Q903 2N7002 maker header isolation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, SW1 Reset, SW2 Mu Power, SW3 Mu Reset, SW900 Maker reset/RUN, SW901 Maker BOOTSEL, U10 BQ34Z100-G1 protected-pack ga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, U11 LTC4368IMS-1 bidirectional pa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, U12 TPS26630RGER 3A AUX eFuse / s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, U14 LTC4418IUF#PBF dual-input PD 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, U15 LTC4418IUF#PBF dual-input sel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, U170 SN74LVC3G34DCUR E-key control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, U1700 USB7206C-I/KDX six-port USB 3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, U1701 TPS62823DLC 3A USB7206C 1.146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, U1702 TLV803EA29 USB hub reset supe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, U1703 TPS56637RPAR VSYS to USB_PORT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, U1704 SN74LVC1G08 hub 3V3/core-PG r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, U1740 TPS2553DDBVR 1.3A USB branch, U1741 TPS25810RVCR Type-C DFP contr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, U1742 HD3SS6126RUAR USB3 orientatio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, U1743 TPD1S514-1YZR 5.9V VBUS OVP, U1745 TPD4E05U06 USB2/CC ESD, U1760 TPS2553DDBVR 1.3A USB branch, U1761 TPS25810RVCR Type-C DFP contr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, U1762 HD3SS6126RUAR USB3 orientatio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, U1763 TPD1S514-1YZR 5.9V VBUS OVP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

Commit message: Add impedance-driven net classes and base design rules to mainboard
Other:
- net class DIFF_100 added: clearance 0.2, trace_width 0.215, via_dia 0.6, via_drill 0.3
- net class DIFF_85 added: clearance 0.2, trace_width 0.29, via_dia 0.6, via_drill 0.3
- net class DIFF_90 added: clearance 0.2, trace_width 0.26, via_dia 0.6, via_drill 0.3
- net class Default added: clearance 0.2, trace_width 0.25, via_dia 0.6, via_drill 0.3
- net class USB2_45 added: clearance 0.2, trace_width 0.262, via_dia 0.6, via_drill 0.3
Changed lines of the file:
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@@
 		)
 	)
+(net_class "Default" "Default net class"
+	(clearance 0.2)
+	(trace_width 0.25)
+	(via_dia 0.6)
+	(via_drill 0.3)
+	(diff_pair_width 0.25)
+	(diff_pair_gap 0.25)
+)
+(net_class "DIFF_85" "PCIe Gen3 85 ohm differential (NVMe x4, Wi-Fi x1, REFCLK)"
+	(clearance 0.2)
+	(trace_width 0.29)
+	(via_dia 0.6)
+	(via_drill 0.3)
+	(diff_pair_width 0.29)
+	(diff_pair_gap 0.8)
+	(add_net "/Mu Carrier/PCIE_M_L0_RX_N")
+	(add_net "/Mu Carrier/PCIE_M_L0_RX_P")
+	(add_net "/Mu Carrier/PCIE_M_L0_TX_N")
+	(add_net "/Mu Carrier/PCIE_M_L0_TX_P")
+	(add_net "/Mu Carrier/PCIE_M_L0_TX_RAW_N")
+	(add_net "/Mu Carrier/PCIE_M_L0_TX_RAW_P")
+	(add_net "/Mu Carrier/PCIE_M_L1_RX_N")
+	(add_net "/Mu Carrier/PCIE_M_L1_RX_P")
+	(add_net "/Mu Carrier/PCIE_M_L1_TX_N")
+	(add_net "/Mu Carrier/PCIE_M_L1_TX_P")
+	(add_net "/Mu Carrier/PCIE_M_L1_TX_RAW_N")
+	(add_net "/Mu Carrier/PCIE_M_L1_TX_RAW_P")
+	(add_net "/Mu Carrier/PCIE_M_L2_RX_N")
+	(add_net "/Mu Carrier/PCIE_M_L2_RX_P")
+	(add_net "/Mu Carrier/PCIE_M_L2_TX_N")
+	(add_net "/Mu Carrier/PCIE_M_L2_TX_P")
+	(add_net "/Mu Carrier/PCIE_M_L2_TX_RAW_N")
+	(add_net "/Mu Carrier/PCIE_M_L2_TX_RAW_P")
+	(add_net "/Mu Carrier/PCIE_M_L3_RX_N")
+	(add_net "/Mu Carrier/PCIE_M_L3_RX_P")
+	(add_net "/Mu Carrier/PCIE_M_L3_TX_N")
+	(add_net "/Mu Carrier/PCIE_M_L3_TX_P")
+	(add_net "/Mu Carrier/PCIE_M_L3_TX_RAW_N")
+	(add_net "/Mu Carrier/PCIE_M_L3_TX_RAW_P")
+	(add_net "/Mu Carrier/PCIE_M_REFCLK_N")
+	(add_net "/Mu Carrier/PCIE_M_REFCLK_P")
+	(add_net "/Mu Carrier/PCIE_M_REFCLK_SRC_N")
+	(add_net "/Mu Carrier/PCIE_M_REFCLK_SRC_P")
+	(add_net "/Mu Carrier/WIFI_PCIE_TX_RAW_N")
+	(add_net "/Mu Carrier/WIFI_PCIE_TX_RAW_P")
+	(add_net "/WIFI_PCIE_RX_N")
+	(add_net "/WIFI_PCIE_RX_P")
+	(add_net "/WIFI_PCIE_TX_N")
+	(add_net "/WIFI_PCIE_TX_P")
+	(add_net "/WIFI_REFCLK_N")
+	(add_net "/WIFI_REFCLK_P")
+	(add_net "/Wi-Fi{slash}Bluetooth & OLEDs/WIFI_REFCLK_E_N")
+	(add_net "/Wi-Fi{slash}Bluetooth & OLEDs/WIFI_REFCLK_E_P")
+)
+(net_class "DIFF_90" "USB 3.x / USB-C 90 ohm differential"
+	(clearance 0.2)
+	(trace_width 0.26)
+	(via_dia 0.6)
+	(via_drill 0.3)
+	(diff_pair_width 0.26)
+	(diff_pair_gap 0.612)
+	(add_net "/HUB_DS1_SSRX_N")
+	(add_net "/HUB_DS1_SSRX_P")
+	(add_net "/HUB_DS1_SSTX_N")
+	(add_net "/HUB_DS1_SSTX_P")
+	(add_net "/Mu Carrier/USBC1_SSTX_RAW_N")
+	(add_net "/Mu Carrier/USBC1_SSTX_RAW_P")
+	(add_net "/Mu Carrier/USBC2_SSTX_RAW_N")
+	(add_net "/Mu Carrier/USBC2_SSTX_RAW_P")
+	(add_net "/Native USB-C I{slash}O/HUB_DS1_TX_RAW_N")
+	(add_net "/Native USB-C I{slash}O/HUB_DS1_TX_RAW_P")
+	(add_net "/Native USB-C I{slash}O/HUB_DS2_SSRX_N")
+	(add_net "/Native USB-C I{slash}O/HUB_DS2_SSRX_P")
+	(add_net "/Native USB-C I{slash}O/HUB_DS2_SSTX_N")
+	(add_net "/Native USB-C I{slash}O/HUB_DS2_SSTX_P")
+	(add_net "/Native USB-C I{slash}O/HUB_DS2_TX_RAW_N")
+	(add_net "/Native USB-C I{slash}O/HUB_DS2_TX_RAW_P")
+	(add_net "/Native USB-C I{slash}O/HUB_DS3_SSRX_N")
+	(add_net "/Native USB-C I{slash}O/HUB_DS3_SSRX_P")
+	(add_net "/Native USB-C I{slash}O/HUB_DS3_SSTX_N")
+	(add_net "/Native USB-C I{slash}O/HUB_DS3_SSTX_P")
+	(add_net "/Native USB-C I{slash}O/HUB_DS3_TX_RAW_N")
+	(add_net "/Native USB-C I{slash}O/HUB_DS3_TX_RAW_P")
+	(add_net "/Native USB-C I{slash}O/HUB_DS4_SSRX_N")
+	(add_net "/Native USB-C I{slash}O/HUB_DS4_SSRX_P")
+	(add_net "/Native USB-C I{slash}O/HUB_DS4_SSTX_N")
+	(add_net "/Native USB-C I{slash}O/HUB_DS4_SSTX_P")
+	(add_net "/Native USB-C I{slash}O/HUB_DS4_TX_RAW_N")
+	(add_net "/Native USB-C I{slash}O/HUB_DS4_TX_RAW_P")
+	(add_net "/Native USB-C I{slash}O/HUB_UP_TX_RAW_N")
+	(add_net "/Native USB-C I{slash}O/HUB_UP_TX_RAW_P")
+	(add_net "/Native USB-C I{slash}O/J12_RX1_N")
+	(add_net "/Native USB-C I{slash}O/J12_RX1_P")
+	(add_net "/Native USB-C I{slash}O/J12_RX2_N")
+	(add_net "/Native USB-C I{slash}O/J12_RX2_P")
+	(add_net "/Native USB-C I{slash}O/J12_TX1_N")
+	(add_net "/Native USB-C I{slash}O/J12_TX1_P")
+	(add_net "/Native USB-C I{slash}O/J12_TX2_N")
+	(add_net "/Native USB-C I{slash}O/J12_TX2_P")
+	(add_net "/Power Inputs/PD1_SSRX_RAW_N")
+	(add_net "/Power Inputs/PD1_SSRX_RAW_P")
+	(add_net "/Power Inputs/PD2_SSRX_RAW_N")
+	(add_net "/Power Inputs/PD2_SSRX_RAW_P")
+	(add_net "/USBC1_SSRX_N")
+	(add_net "/USBC1_SSRX_P")
+	(add_net "/USBC1_SSTX_N")
+	(add_net "/USBC1_SSTX_P")
+	(add_net "/USBC2_SSRX_N")
+	(add_net "/USBC2_SSRX_P")
+	(add_net "/USBC2_SSTX_N")
+	(add_net "/USBC2_SSTX_P")
+)
+(net_class "DIFF_100" "HDMI + Ethernet MDI 100 ohm differential"
+	(clearance 0.2)
+	(trace_width 0.215)
+	(via_dia 0.6)
+	(via_drill 0.3)
+	(diff_pair_width 0.215)
+	(diff_pair_gap 0.679)
+	(add_net "/GBE_HOST_RX_N")
+	(add_net "/GBE_HOST_RX_P")
+	(add_net "/GBE_HOST_TX_N")
+	(add_net "/GBE_HOST_TX_P")
+	(add_net "/GBE_REFCLK_N")
+	(add_net "/GBE_REFCLK_P")
+	(add_net "/Gigabit Ethernet/ETH_MDI0_N")
+	(add_net "/Gigabit Ethernet/ETH_MDI0_P")
+	(add_net "/Gigabit Ethernet/ETH_MDI1_N")
+	(add_net "/Gigabit Ethernet/ETH_MDI1_P")
+	(add_net "/Gigabit Ethernet/ETH_MDI2_N")
+	(add_net "/Gigabit Ethernet/ETH_MDI2_P")
+	(add_net "/Gigabit Ethernet/ETH_MDI3_N")
+	(add_net "/Gigabit Ethernet/ETH_MDI3_P")
+	(add_net "/Gigabit Ethernet/GBE_HSI_N")
+	(add_net "/Gigabit Ethernet/GBE_HSI_P")
+	(add_net "/Gigabit Ethernet/GBE_HSO_N")
+	(add_net "/Gigabit Ethernet/GBE_HSO_P")
+	(add_net "/TCP0 External HDMI/EXT_HDMI_CK_N")
+	(add_net "/TCP0 External HDMI/EXT_HDMI_CK_P")
+	(add_net "/TCP0 External HDMI/EXT_HDMI_D0_N")
+	(add_net "/TCP0 External HDMI/EXT_HDMI_D0_P")
+	(add_net "/TCP0 External HDMI/EXT_HDMI_D1_N")
+	(add_net "/TCP0 External HDMI/EXT_HDMI_D1_P")
+	(add_net "/TCP0 External HDMI/EXT_HDMI_D2_N")
+	(add_net "/TCP0 External HDMI/EXT_HDMI_D2_P")
+)
+(net_class "USB2_45" "USB 2.0 D+/D- 45 ohm single-ended"
+	(clearance 0.2)
+	(trace_width 0.262)
+	(via_dia 0.6)
+	(via_drill 0.3)
+	(diff_pair_width 0.262)
+	(diff_pair_gap 0.25)
+	(add_net "/AUDIO_USB_DM")
+	(add_net "/AUDIO_USB_DP")
+	(add_net "/EC_HOST_USB_DM")
+	(add_net "/EC_HOST_USB_DP")
+	(add_net "/HUB_DS1_DM")
+	(add_net "/HUB_DS1_DP")
+	(add_net "/Internal Services/EC_USB_ISO_DM")
+	(add_net "/Internal Services/EC_USB_ISO_DP")
+	(add_net "/Internal Services/TPAD_CONN_DM")
+	(add_net "/Internal Services/TPAD_CONN_DP")
+	(add_net "/MAKER_USB_DM")
+	(add_net "/MAKER_USB_DP")
+	(add_net "/MCU_USB_DM")
+	(add_net "/MCU_USB_DP")
+	(add_net "/Maker MCU/MAKER_USB_ISO_DM")
+	(add_net "/Maker MCU/MAKER_USB_ISO_DP")
+	(add_net "/Native USB-C I{slash}O/HUB_DIS5_DM")
+	(add_net "/Native USB-C I{slash}O/HUB_DIS5_DP")
+	(add_net "/Native USB-C I{slash}O/HUB_DIS6_DM")
+	(add_net "/Native USB-C I{slash}O/HUB_DIS6_DP")
+	(add_net "/Native USB-C I{slash}O/HUB_DS2_DM")
+	(add_net "/Native USB-C I{slash}O/HUB_DS2_DP")
+	(add_net "/Native USB-C I{slash}O/HUB_DS3_DM")
+	(add_net "/Native USB-C I{slash}O/HUB_DS3_DP")
+	(add_net "/Native USB-C I{slash}O/HUB_DS4_DM")
+	(add_net "/Native USB-C I{slash}O/HUB_DS4_DP")
+	(add_net "/System Audio/CODEC_USB_DM")
+	(add_net "/System Audio/CODEC_USB_DP")
+	(add_net "/System Audio/SYSTEM_DAC_USB_DM")
+	(add_net "/System Audio/SYSTEM_DAC_USB_DP")
+	(add_net "/TRACKPAD_USB_DM")
+	(add_net "/TRACKPAD_USB_DP")
+	(add_net "/USBC1_DM")
+	(add_net "/USBC1_DP")
+	(add_net "/USBC2_DM")
+	(add_net "/USBC2_DP")
+	(add_net "/WIFI_USB_DP")
+)
 	(footprint "Package_DFN_QFN:Diodes_UDFN-10_1x2.5mm_P0.5mm"
 		(layer "F.Cu")
