File: ducktop2.kicad_pcb (KiCad board)
At the start: 6 copper layers, 358 x 185 mm, 1181 parts, among them J10 Amphenol MDT420M01001 M-key N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, J11 USB-C dual-role data/PD port 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, J12 USB-C source-only data port J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, J16 Case power/reset button harne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, J190 AUX/SOLAR protected screw ter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, J2 3S pack power + cell-tap harn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, J21 USB-C dual-role data/PD port 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, J22 USB-C source-only data port J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, J23 USB-C source-only data port J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, J2300 DF40C 60-pin optional radio d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, J30 External HDMI-A from TCP0, J310 Mainboard keyboard FFC to MX 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, J4 TC2030 Cortex SWD: VTref/SWDI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, J40 Amphenol MDT420E01001 E-key W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, J41 SSD1306 OLED A 4-pin GND/VDD/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, J420 Left 8-ohm BTL speaker; pin 1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, J421 Right 8-ohm BTL speaker; pin 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, J422 CUI SJ1-3535NG rear 3.5mm ste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, J45 SSD1306 OLED B 4-pin GND/VDD/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, J500 JXD1-1022NL recessed 1GbE RJ45, J52 Delta BFB04512HHA-CZ0T: GND, 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, J53 Lid/hall switch, J54 Skin/hinge NTC, J56 Mu heatsink/spreader NTC, J58 Field-soldered trackpad USB2 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, J9 RTC backup coin-cell header, J901 JST PUD 2x20 protected maker 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, J902 TC2030 Cortex SWD: VTref/SWDI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, Q11 CSD18540Q5B reverse-pack FET A, Q12 CSD18540Q5B reverse-pack FET B, Q13 CSD19537Q3 100V AUX reverse F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, Q14 BSS138 fast reverse-gate pull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, Q15 SiSS4409DN 40V reverse-blocki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, Q16 SiSS4409DN 40V reverse-blocki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, Q17 SiSS4409DN 40V reverse-blocki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, Q18 SiSS4409DN 40V reverse-blocki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, Q200 2N7002KT1G fan PWM open-drain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, Q2001 2N7002K DFP USB2 enable inver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, Q2002 2N7002K DFP USB2 enable inver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, Q21 SiSS4409DN 40V reverse-blocki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, Q22 SiSS4409DN 40V reverse-blocki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, Q23 SiSS4409DN 40V reverse-blocki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, Q2300 2N7002K radio-PG USB enable, Q24 SiSS4409DN 40V reverse-blocki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, Q25 CSD17575Q3 BQ25798 ship FET, Q50 BSS138 HDMI bias gate, Q60 2N7002 physical host-VBUS USB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, Q700 BSS138 active-high charger en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, Q701 BSS138 pack protector latch r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, Q702 BSS138 QON open-drain pulse, Q703 CSD18540Q5B BQ77915 discharge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, Q704 CSD18540Q5B BQ77915 charge FET, Q750 BSS138 fail-off EN/UVLO clamp, Q751 BSS138 active-high enable rel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, Q901 2N7002 physical host-VBUS USB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, Q903 2N7002 maker header isolation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, SW1 Reset, SW2 Mu Power, SW3 Mu Reset, SW900 Maker reset/RUN, SW901 Maker BOOTSEL, U10 BQ34Z100-G1 protected-pack ga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, U11 LTC4368IMS-1 bidirectional pa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, U12 TPS26630RGER 3A AUX eFuse / s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, U14 LTC4418IUF#PBF dual-input PD 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, U15 LTC4418IUF#PBF dual-input sel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, U170 SN74LVC3G34DCUR E-key control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, U1700 USB7206C-I/KDX six-port USB 3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, U1701 TPS62823DLC 3A USB7206C 1.146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, U1702 TLV803EA29 USB hub reset supe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, U1703 TPS56637RPAR VSYS to USB_PORT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, U1704 SN74LVC1G08 hub 3V3/core-PG r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, U1740 TPS2553DDBVR 1.3A USB branch, U1741 TPS25810RVCR Type-C DFP contr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, U1742 HD3SS6126RUAR USB3 orientatio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, U1743 TPD1S514-1YZR 5.9V VBUS OVP, U1745 TPD4E05U06 USB2/CC ESD, U1760 TPS2553DDBVR 1.3A USB branch, U1761 TPS25810RVCR Type-C DFP contr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, U1762 HD3SS6126RUAR USB3 orientatio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

Commit message: Placement fixer pass 3: 59 more passive moves (shorts 97->54)
Parts:
- moved C2081 21.6 mm to (349.7, 20.1)
- moved H4 20.3 mm to (213.5, 177.4)
- moved C796 18.0 mm to (241.2, 166.8)
- moved C701 17.8 mm to (69.0, 123.2)
- moved D710 17.8 mm to (207.5, 174.8)
- moved C441 16.3 mm to (98.5, 171.8)
- moved Y500 12.7 mm to (324.4, 115.2)
- moved C703 7.62 mm to (72.1, 128.5)
- moved C768 7.62 mm to (279.1, 58.5)
- moved R708 7.18 mm to (307.5, 115.5)
- moved C423 7.18 mm to (90.6, 187.1)
- moved C705 7.18 mm to (58.8, 116.8)
- moved R1750 7.18 mm to (54.0, 68.5)
- moved C722 5.08 mm to (89.6, 187.1)
- moved C758 5.08 mm to (147.7, 74.0)
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