File: 02_ec_mcu.kicad_sch (KiCad schematic)
At the start: 35 parts, among them J4 SWD (VDD/SWDIO/SWCLK/GND), J5 KB rows (PE0-7), J6 KB columns (PD0-15), J7 EC_GPIO0-15 expansion, SW1 Reset, U4 STM32F407VGTx, U5 TPS54202DDC, Y1 8MHz HSE, Y2 32.768kHz LSE

Commit message: Checkpoint ducktop2 generated schematic baseline
Parts:
- removed Y1: 8MHz HSE, Crystal:Crystal_SMD_3225-4Pin_3.2x2.5mm, symbol Device:Crystal
- added J13: Laptop service GPIO map, Connector_PinHeader_2.54mm:PinHeader_1x16_P2.54mm_Vertical, symbol Connector_Generic:Conn_01x16
- added J14: Ham radio EC GPIO map, Connector_PinHeader_2.54mm:PinHeader_1x16_P2.54mm_Vertical, symbol Connector_Generic:Conn_01x16
- added J15: Exposed EC-owned GPIO header, Connector_PinHeader_2.54mm:PinHeader_1x16_P2.54mm_Vertical, symbol Connector_Generic:Conn_01x16
- added J16: Case power/reset button harness, Connector_JST:JST_XH_B4B-XH-A_1x04_P2.50mm_Vertical, symbol Connector_Generic:Conn_01x04
- added Y1: 8MHz HSE, Crystal:Crystal_SMD_3225-4Pin_3.2x2.5mm, symbol Device:Crystal_GND24
- C39: value 22u (TBD - verify output ripple) -> 22u MCU_3V3 output
- J5: value KB rows (PE0-7) -> DNP KB row probe; R5-R7 spare in MX ULP rev A; now not fitted; now left out of the parts list
- J6: value KB columns (PD0-15) -> DNP KB column probe; C14-C15 spare in MX ULP rev A; now not fitted; now left out of the parts list
- J7: value EC_GPIO0-15 expansion -> EC power controls + spare GPIO expansion
- L3: value 3.3uH (typ, verify per fsw) -> 3.3uH >=3A
- R35: value 31.6k (FB divider hi) -> 45.3k 1% (3.3V FB hi)
- R36: value 10k (FB divider lo) -> 10k 1% (3.3V FB lo)
Connections:
- net GND: now also J13.16 (Pin_16), J14.16 (Pin_16), J15.12 (Pin_12), J15.16 (Pin_16), J15.2 (Pin_2), J16.1 (Pin_1), Y1.2 (G), Y1.4 (G)
- net HSE_IN: now also Y1.1
- net HSE_OUT: now also Y1.3
- net I2C_SCL: now also J15.3 (Pin_3)
- net I2C_SDA: now also J15.4 (Pin_4)
- net MCU_3V3: now also J13.14 (Pin_14), J14.15 (Pin_15), J15.1 (Pin_1), J15.11 (Pin_11), J16.4 (Pin_4)
- net MCU_USB_DM: now also J13.13 (Pin_13)
- net MCU_USB_DP: now also J13.12 (Pin_12)
- net VSYS: now also J13.15 (Pin_15)
- net USER_GPIO0_SPI_SCK: now reaches U4.15 (PC0)
- net USER_GPIO0_SPI_SCK: now also J15.5 (Pin_5)
- net USER_GPIO1_SPI_MISO: now reaches U4.16 (PC1)
- net USER_GPIO1_SPI_MISO: now also J15.6 (Pin_6)
- net USER_GPIO2_SPI_MOSI: now reaches U4.17 (PC2)
- net USER_GPIO2_SPI_MOSI: now also J15.7 (Pin_7)
- net USER_GPIO3_SPI_CS_N: now reaches U4.18 (PC3)
- net USER_GPIO3_SPI_CS_N: now also J15.8 (Pin_8)
- net FAN_PWM: now reaches U4.33 (PC4)
- net FAN_PWM: now also J13.1 (Pin_1)
- net FAN_TACH: now reaches U4.34 (PC5)
- net FAN_TACH: now also J13.2 (Pin_2)
- net LCD_BL_PWM: now reaches U4.39 (PE8)
- net LCD_BL_PWM: now also J13.3 (Pin_3)
- net LCD_BL_EN: now reaches U4.40 (PE9)
- net LCD_BL_EN: now also J13.4 (Pin_4)
- net LID_CLOSED_N: now reaches U4.41 (PE10)
- net LID_CLOSED_N: now also J13.5 (Pin_5)
- net TPAD_RESET_N: now reaches U4.42 (PE11)
- net TPAD_RESET_N: now also J7.4 (Pin_4)
- net TOUCH_RESET_N: now reaches U4.43 (PE12)
- net TOUCH_RESET_N: now also J13.8 (Pin_8)
- net PANEL_PWR_EN: now reaches U4.44 (PE13)
- net PANEL_PWR_EN: now also J13.10 (Pin_10)
- net PANEL_RESET_N: now reaches U4.45 (PE14)
- net PANEL_RESET_N: now also J13.11 (Pin_11)
- net TOUCH_INT_N: now reaches U4.46 (PE15)
- net TOUCH_INT_N: now also J13.9 (Pin_9)
- net RADIO_VHF_UART_TX: now reaches U4.47 (PB10)
- net RADIO_VHF_UART_TX: now also J14.1 (Pin_1)
- net RADIO_VHF_UART_RX: now reaches U4.48 (PB11)
- net RADIO_VHF_UART_RX: now also J14.2 (Pin_2)
- net RADIO_UHF_UART_TX: now reaches U4.54 (PB15)
- net RADIO_UHF_UART_TX: now also J14.3 (Pin_3)
- net RADIO_UHF_UART_RX: now reaches U4.63 (PC6)
- net RADIO_UHF_UART_RX: now also J14.4 (Pin_4)
- net RADIO_VHF_PTT_N: now reaches U4.64 (PC7)
- net RADIO_VHF_PTT_N: now also J14.5 (Pin_5)
- net RADIO_UHF_PTT_N: now reaches U4.65 (PC8)
- net RADIO_UHF_PTT_N: now also J14.6 (Pin_6)
- net RADIO_VHF_PD_N: now reaches U4.66 (PC9)
- net RADIO_VHF_PD_N: now also J14.7 (Pin_7)
- net USER_GPIO4: now reaches U4.7 (PC13)
- net USER_GPIO4: now also J15.9 (Pin_9)
- net RADIO_UHF_PD_N: now reaches U4.78 (PC10)
- net RADIO_UHF_PD_N: now also J14.8 (Pin_8)
- net RADIO_VHF_SQL: now reaches U4.79 (PC11)
- net RADIO_VHF_SQL: now also J14.9 (Pin_9)
- net RADIO_UHF_SQL: now reaches U4.80 (PC12)
- net RADIO_UHF_SQL: now also J14.10 (Pin_10)
- net RADIO_VHF_RF_SEL: now reaches U4.89 (PB3)
- net RADIO_VHF_RF_SEL: now also J14.11 (Pin_11)
- net RADIO_UHF_RF_SEL: now reaches U4.90 (PB4)
- net RADIO_UHF_RF_SEL: now also J14.12 (Pin_12)
- net RADIO_AUDIO_SEL: now reaches U4.91 (PB5)
- net RADIO_AUDIO_SEL: now also J14.13 (Pin_13)
- net EC_GPIO0 renamed MU_PWRBTN_N
- net MU_PWRBTN_N: now also J16.2 (Pin_2)
- net EC_GPIO1 renamed MU_RSTBTN_N
- net MU_RSTBTN_N: now also J16.3 (Pin_3)
- net EC_GPIO10 renamed EC_SPARE_GPIO5
- net EC_SPARE_GPIO5: now also J7.6 (Pin_6); no longer J7.11 (Pin_11)
- net EC_GPIO11 renamed GNSS_EXTINT
- net GNSS_EXTINT: now also J7.15 (Pin_15); no longer J7.12 (Pin_12)
- net EC_GPIO12 renamed GNSS_RESET_N
- net GNSS_RESET_N: now also U4.52 (PB13); no longer U4.96 (PB9)
- net EC_GPIO13 renamed GNSS_PPS
- net GNSS_PPS: now also U4.53 (PB14); no longer U4.51 (PB12)
- removed net EC_GPIO14: J7.15 (Pin_15), U4.52 (PB13)
- net EC_GPIO15 renamed RADIO_GPIO0
- net RADIO_GPIO0: now also U4.96 (PB9), J14.14 (Pin_14), J15.10 (Pin_10); no longer U4.53 (PB14)
- net EC_GPIO2 renamed AUX_DC_ADC
- net EC_GPIO3 renamed THERM_SKIN_ADC
- net THERM_SKIN_ADC: now also J13.6 (Pin_6); no longer J7.4 (Pin_4)
- net EC_GPIO4 renamed TPAD_INT_N
- net TPAD_INT_N: now also U4.36 (PB1); no longer U4.67 (PA8)
- net EC_GPIO5 renamed WIFI_W_DISABLE2_N
- net WIFI_W_DISABLE2_N: now also J7.9 (Pin_9); no longer J7.6 (Pin_6)
- net EC_GPIO6 renamed GNSS_UART_RX
- net GNSS_UART_RX: now also J7.10 (Pin_10); no longer J7.7 (Pin_7)
- net EC_GPIO7 renamed GNSS_UART_TX
- net GNSS_UART_TX: now also J7.11 (Pin_11); no longer J7.8 (Pin_8)
- net EC_GPIO8 renamed THERM_MU_ADC
- net THERM_MU_ADC: now also J7.7 (Pin_7), J13.7 (Pin_7); no longer J7.9 (Pin_9)
- removed net EC_GPIO9: J7.10 (Pin_10), U4.36 (PB1)
- new net OLED_RESET_N: J7.12 (Pin_12), U4.51 (PB12)
- new net WIFI_W_DISABLE1_N: J7.8 (Pin_8), U4.67 (PA8)
- no-connect marks 28 -> 3
Other:
- note added: "== EC GPIO expansion / laptop power controls =="
- note added: "== Keyboard Matrix GPIO bank (MX ULP rev A uses 5 rows x 14 cols) =="
- note added: "AUX_DC_ADC monitors the screw-terminal wide-DC input so firmware can classify and current-limit that source."
- note added: "Anti-ghosting diodes for the keyboard matrix live on the separate MX ULP keyboard PCB."
- note added: "EC can assert Mu PWRBTN_N/RSTBTN_N as open-drain GPIOs; J16 also allows physical case buttons."
- note added: "J15 is the user-facing EC GPIO header: EC I2C, five GPIO/SPI-capable signals, power, and grounds."
- note added: "PA7/PB0 are assigned to skin and Mu-heatsink thermistors; fan PWM/tach remain EC-owned."
- note added: "Second spare GPIO bank is assigned to E-key radio disables, GNSS UART/control/PPS, OLED reset, trackpad reset/INT, and one spare radio GPIO."
- note added: "U5 uses TPS54202/TPS54302-style 0.596V feedback; R35/R36 set MCU_3V3 to about 3.30V."
- note removed: "== EC_GPIO expansion header (16 spare GPIO) =="
- note removed: "== Keyboard Matrix (8 rows x 16 cols, diodes on membrane PCB) =="
- note removed: "Anti-ghosting diodes for the keyboard matrix live on the keyboard membrane PCB, not this board."

Commit message: Publish the current Ducktop2 design
Parts:
- removed C34: 12p, Capacitor_SMD:C_0603_1608Metric, symbol Device:C
- removed J14: Ham radio EC GPIO map, Connector_PinHeader_2.54mm:PinHeader_1x16_P2.54mm_Vertical, symbol Connector_Generic:Conn_01x16
- removed J15: Exposed EC-owned GPIO header, Connector_PinHeader_2.54mm:PinHeader_1x16_P2.54mm_Vertical, symbol Connector_Generic:Conn_01x16
- removed J16: Case power/reset button harness, Connector_JST:JST_XH_B4B-XH-A_1x04_P2.50mm_Vertical, symbol Connector_Generic:Conn_01x04
- removed J7: EC power controls + spare GPIO expansion, Connector_PinHeader_2.54mm:PinHeader_1x16_P2.54mm_Vertical, symbol Connector_Generic:Conn_01x16
- removed R32: 10k, Resistor_SMD:R_0603_1608Metric, symbol Device:R
- added C291: 22u 16V X7R MCU_3V3 output, Capacitor_SMD:C_1206_3216Metric, symbol Device:C
- added C292: 56p C0G TPS54202 feed-forward, Capacitor_SMD:C_0402_1005Metric, symbol Device:C
- added C30: 2.2u (VCAP_2, mandatory), Capacitor_SMD:C_0805_2012Metric, symbol Device:C
- added C780: 100n source-manager local, Capacitor_SMD:C_0603_1608Metric, symbol Device:C
- added C781: 100n service-mux reset gate local, Capacitor_SMD:C_0603_1608Metric, symbol Device:C
- added R172: 100k service mux reset-request pull-up, Resistor_SMD:R_0603_1608Metric, symbol Device:R
- added R33: 10k, Resistor_SMD:R_0603_1608Metric, symbol Device:R
- added R37: 0R HSE drive/tuning position, Resistor_SMD:R_0603_1608Metric, symbol Device:R
- added R780: 10k source-manager INT pull-up, Resistor_SMD:R_0603_1608Metric, symbol Device:R
- added R781: 10k aggregate AON fault pull-up, Resistor_SMD:R_0603_1608Metric, symbol Device:R
- added R782, R783, R784: 100k unused source-manager I/O pulldown, Resistor_SMD:R_0603_1608Metric, symbol Device:R
- added U46: SN74LVC1G08DBVR EC-reset-qualified service mux re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, Package_TO_SOT_SMD:SOT-23-5, symbol 74xGxx:74LVC1G08
- C29: renamed from C30; value 2.2u (VCAP_2, mandatory) -> 2.2u (VCAP_1, mandatory)
- C290: renamed from C29; value 2.2u (VCAP_1, mandatory) -> 10n (VDDA high-frequency); footprint Capacitor_SMD:C_0805_2012Metric -> Capacitor_SMD:C_0603_1608Metric
- C31: renamed from SW1; value Reset -> 100n; footprint Button_Switch_SMD:SW_SPST_B3S-1000 -> Capacitor_SMD:C_0603_1608Metric; symbol Switch:SW_Push -> Device:C
- C32, C33: value 18p -> 10p C0G 0.25pF HSE load; MPN (none) -> C0603C100C5GACTU; Manufacturer (none) -> KEMET
- C34: renamed from J4; value SWD (VDD/SWDIO/SWCLK/GND) -> 6.8p C0G 0.25pF LSE load; footprint Connector_PinHeader_2.54mm:PinHeader_1x04_P2.54mm_Vertical -> Capacitor_SMD:C_0603_1608Metric; symbol Connector_Generic:Conn_01x04 -> Device:C; MPN (none) -> C0603C689C5GACTU; Manufacturer (none) -> KEMET
- C35: value 12p -> 6.8p C0G 0.25pF LSE load; MPN (none) -> C0603C689C5GACTU; Manufacturer (none) -> KEMET
- C36: value 10u (VIN bulk) -> 10u 50V X7R VIN; MPN (none) -> CGA5L1X7R1H106K160AC; Manufacturer (none) -> TDK
- C37: value 100n (VIN bypass) -> 100n 50V X7R VIN HF; MPN (none) -> GRM188R71H104KA93D; Manufacturer (none) -> Murata
- C39: value 22u MCU_3V3 output -> 22u 16V X7R MCU_3V3 output; MPN (none) -> GRM31CZ71C226ME15L; Manufacturer (none) -> Murata
- J16: renamed from J6; value DNP KB column probe; C14-C15 spare in MX ULP rev A -> Case power/reset button harness: GND/CASE_PWR/RESET; footprint Connector_PinHeader_2.54mm:PinHeader_1x16_P2.54mm_Vertical -> Connector_JST:JST_SH_SM03B-SRSS-TB_1x03-1MP_P1.00mm_Horizontal; symbol Connector_Generic:Conn_01x16 -> Connector_Generic:Conn_01x03; MPN (none) -> SM03B-SRSS-TB; Manufacturer (none) -> JST; now fitted; now in the parts list
- J4: renamed from J5; value DNP KB row probe; R5-R7 spare in MX ULP rev A -> TC2030 Cortex SWD: VTref/SWDIO/NRST/SWCLK/GND/NC; footprint Connector_PinHeader_2.54mm:PinHeader_1x08_P2.54mm_Vertical -> Connector:Tag-Connect_TC2030-IDC-NL_2x03_P1.27mm_Vertical; symbol Connector_Generic:Conn_01x08 -> Connector_Generic:Conn_01x06; FixtureCable (none) -> TC2030-CTX-NL external programming cable; not fitted; ProcurementClass (none) -> PCB copper test feature; now fitted
- L3: value 3.3uH >=3A -> 10uH 20% 3.3A Isat20; footprint Inductor_SMD:L_1210_3225Metric -> ducktop2:Coilcraft_XGL5030; MPN (none) -> XGL5030-103MEC; Manufacturer (none) -> Coilcraft
- R32: renamed from C31; value 100n -> 10k; footprint Capacitor_SMD:C_0603_1608Metric -> Resistor_SMD:R_0603_1608Metric; symbol Device:C -> Device:R
- R34: value 100k (EN pull-up, always-on) -> 0R VTref sense link
- R35: value 45.3k 1% (3.3V FB hi) -> 100k 1% (3.3V FB hi)
- R36: value 10k 1% (3.3V FB lo) -> 22.1k 1% (3.3V FB lo)
- SW1: renamed from R33; value 10k -> Reset; footprint Resistor_SMD:R_0603_1608Metric -> Button_Switch_SMD:SW_SPST_B3S-1000; symbol Device:R -> Switch:SW_Push; MPN (none) -> B3S-1000; Manufacturer (none) -> Omron
- U4: MPN (none) -> STM32F407VGT6; Manufacturer (none) -> STMicroelectronics
- U44: renamed from J13; value Laptop service GPIO map -> TCA9539PWR resettable source manager @0x20; footprint Connector_PinHeader_2.54mm:PinHeader_1x16_P2.54mm_Vertical -> Package_SO:TSSOP-24_4.4x7.8mm_P0.65mm; symbol Connector_Generic:Conn_01x16 -> Interface_Expansion:PCA9539xD; MPN (none) -> TCA9539PWR; Manufacturer (none) -> Texas Instruments; ResetContract (none) -> Pin 3 follows EC NRST; all P-ports reset to inputs and exte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
- U5: MPN (none) -> TPS54202DDCR; Manufacturer (none) -> Texas Instruments
- Y1: value 8MHz HSE -> J32SMX-K-F-G-I-8M0 8MHz CL8pF; MPN (none) -> J32SMX-K-F-G-I-8M0; Manufacturer (none) -> Jauch Quartz
- Y2: value 32.768kHz LSE -> X1A000141000612 32.768kHz CL6pF; MPN (none) -> X1A000141000612; Manufacturer (none) -> Epson
Connections:
- net WIFI_W_DISABLE2_N is gone; now on net GNSS_UART_TX: U4.68 (PA9)
- net BOOT0_NET: now also R33.1; no longer SW1.1
- net BUCK_FB: now also C292.2
- net FAN_PWM: now also U4.40 (PE9); no longer U4.33 (PC4), U44.1 (Pin_1)
- net FAN_TACH: no longer U44.2 (Pin_2)
- net GND: now also C34.2, J16.1 (Pin_1), J4.5 (Pin_5), U44.12 (V_{SS}), U44.2 (A1), U44.21 (A0), C291.2, C30.2, C780.2, C781.2, R33.2, R782.2, R783.2, R784.2, U46.3 (GND); no longer C34.4 (Pin_4), R32.2, U44.16 (Pin_16)
- net GNSS_UART_TX: no longer U4.77 (PA15)
- net HSE_OUT: now also R37.2; no longer C33.1, Y1.3
- net I2C_SCL: now also U44.22 (SCL)
- net I2C_SDA: now also U44.23 (SDA)
- net KB_COL0: no longer J16.1 (Pin_1)
- net KB_COL1: no longer J16.2 (Pin_2)
- net KB_COL10: no longer J16.11 (Pin_11)
- net KB_COL11: no longer J16.12 (Pin_12)
- net KB_COL12: no longer J16.13 (Pin_13)
- net KB_COL13: no longer J16.14 (Pin_14)
- net KB_COL14: no longer J16.15 (Pin_15)
- net KB_COL2: no longer J16.3 (Pin_3)
- net KB_COL3: no longer J16.4 (Pin_4)
- net KB_COL4: no longer J16.5 (Pin_5)
- net KB_COL5: no longer J16.6 (Pin_6)
- net KB_COL6: no longer J16.7 (Pin_7)
- net KB_COL7: no longer J16.8 (Pin_8)
- net KB_COL8: no longer J16.9 (Pin_9)
- net KB_COL9: no longer J16.10 (Pin_10)
- net KB_ROW0: no longer J4.1 (Pin_1)
- net KB_ROW1: no longer J4.2 (Pin_2)
- net KB_ROW2: no longer J4.3 (Pin_3)
- net KB_ROW3: no longer J4.4 (Pin_4)
- net KB_ROW4: no longer J4.5 (Pin_5)
- net KB_ROW5: no longer J4.6 (Pin_6)
- net KB_ROW6: no longer J4.7 (Pin_7)
- net KB_ROW7: no longer J4.8 (Pin_8)
- net LID_CLOSED_N: no longer U44.5 (Pin_5)
- net LSE_IN: now also C34.1
- net MCU_3V3: now also C290.1, R32.1, R34.1, U44.24 (V_{DD}), C291.1, C292.1, C780.1, C781.1, R172.1, R780.1, R781.1, U46.5 (VCC); no longer C34.1 (Pin_1), U44.14 (Pin_14)
- net MCU_USB_DM: no longer U44.13 (Pin_13)
- net MCU_USB_DP: no longer U44.12 (Pin_12)
- net MU_RSTBTN_N: now also J16.3 (Pin_3)
- net NRST_NET: now also J4.3 (Pin_3), R32.2, SW1.1, U44.3 (~{RESET}), U46.1; no longer R32.1
- net RADIO_UHF_UART_RX: now also U4.64 (PC7); no longer U4.63 (PC6)
- net RADIO_UHF_UART_TX: now also U4.63 (PC6); no longer U4.54 (PB15)
- net RADIO_VHF_PTT_N: now also U4.54 (PB15); no longer U4.64 (PC7)
- net SWCLK_NET: now also J4.4 (Pin_4); no longer C34.3 (Pin_3)
- net SWDIO_NET: now also J4.2 (Pin_2); no longer C34.2 (Pin_2)
- net THERM_MU_ADC: no longer U44.7 (Pin_7)
- net THERM_SKIN_ADC: no longer U44.6 (Pin_6)
- net VCAP1_NODE: now also C29.1; no longer C290.1
- net VCAP2_NODE: now also C30.1; no longer C29.1
- net BUCK_EN: no longer names the net of U5.5 (EN)
- net BUCK_EN: no longer R34.2
- net CHG_CE_N renamed CHG_ENABLE
- net EC_SPARE_GPIO5 renamed PD2_VALID_N
- net KB_COL15 renamed KB_RGB_DATA_3V3
- net KB_RGB_DATA_3V3: no longer J16.16 (Pin_16)
- net LCD_BL_EN renamed PD1_PATH_EN
- net PD1_PATH_EN: no longer U4.40 (PE9)
- net LCD_BL_PWM renamed PD3_VALID_N
- net PD3_VALID_N: no longer U44.3 (Pin_3)
- net OLED_RESET_N renamed SERVICE_MUX_RESET_REQ_N
- net SERVICE_MUX_RESET_REQ_N: now also R172.2, U46.2
- net PANEL_PWR_EN renamed MU_12V_ENABLE
- net MU_12V_ENABLE: no longer U44.10 (Pin_10)
- net PANEL_RESET_N renamed AUX_FAULT_N
- net AUX_FAULT_N: no longer U4.45 (PE14)
- net PMIC_QON renamed PMIC_QON_ASSERT
- net RADIO_UHF_RF_SEL: no longer names the net of U4.90 (PB4)
- net RADIO_VHF_RF_SEL renamed INTERNAL_USB_VBUS_FAULT_N
- net TOUCH_INT_N renamed MU_12V_PG
- net MU_12V_PG: no longer U44.9 (Pin_9)
- net TOUCH_RESET_N renamed AUDIO_AMP_EC_EN
- net AUDIO_AMP_EC_EN: no longer U44.8 (Pin_8)
- net TPAD_INT_N renamed TRACKPAD_FAULT_N
- net TPAD_RESET_N renamed AUDIO_MIC_EN
- net USER_GPIO0_SPI_SCK renamed KB_RGB_PWR_EN
- net USER_GPIO1_SPI_MISO renamed KB_RGB_FAULT_N
- net USER_GPIO2_SPI_MOSI renamed RADIO_VHF_RF_SEL_3V3
- net USER_GPIO3_SPI_CS_N renamed RADIO_UHF_RF_SEL_3V3
- net USER_GPIO4 renamed SOURCE_MGR_INT_N
- net SOURCE_MGR_INT_N: now also U44.1 (~{INT}), R780.2
- net VSYS renamed EC_AON_IN
- net EC_AON_IN: no longer R34.1, U44.15 (Pin_15)
- net WIFI_W_DISABLE1_N renamed WIFI_W_DISABLE1_N_EC
- new net AON_FAULT_N: R781.2, U44.17 (IO1_4)
- new net AUX_PGOOD: U44.14 (IO1_1)
- new net CASE_PWRBTN_N: J16.2 (Pin_2)
- new net EC_SWD_VTREF: J4.1 (Pin_1), R34.2
- new net HSE_XTAL_OUT: C33.1, R37.1, Y1.3
- new net MAIN_AUX_VALID_N: U44.16 (IO1_3)
- new net MAIN_USB_VALID_N: U44.15 (IO1_2)
- new net MU_S0_HIGH: U4.45 (PE14)
- new net PACK_FAULT_N: U44.10 (IO0_6)
- new net PACK_RETRY_PULSE: U44.13 (IO1_0)
- new net PD1_EFUSE_FAULT_N: U44.7 (IO0_3)
- new net PD1_VALID_N: U4.33 (PC4)
- new net PD2_EFUSE_FAULT_N: U44.8 (IO0_4)
- new net PD2_PATH_EN: U44.5 (IO0_1)
- new net PD3_EFUSE_FAULT_N: U44.9 (IO0_5)
- new net PD3_PATH_EN: U44.6 (IO0_2)
- new net SERVICE_MUX_RESET_N: U46.4
- new net SOURCE_MGR_SPARE1: R782.1, U44.18 (IO1_5)
- new net SOURCE_MGR_SPARE2: R783.1, U44.19 (IO1_6)
- new net SOURCE_MGR_SPARE3: R784.1, U44.20 (IO1_7)
- new net WIFI_W_DISABLE2_N_EC: U4.77 (PA15)
Other:
- note added: "-- Standard TC2030 Cortex SWD target pads --"
- note added: "== Final case controls (no exposed EC/service-map headers) =="
- note added: "== U44 resettable always-on source manager I/O expander =="
- note added: "== U5 TPS54202DDC EC_AON_IN -> MCU_3V3 Buck (3.3V, 2A) =="
- note added: "EC can assert Mu PWRBTN_N/RSTBTN_N; J16 case power is diode-isolated to Mu PWRBTN and charger QON."
- note added: "Hardware UARTs: VHF USART3 on PB10/PB11, UHF USART6 on PC6/PC7, GNSS USART1 on PA9/PA10."
- note added: "MCU_USB_DP/DM (PA12/PA11, OTG_FS device mode) are unrelated to the power-only USB-C PD sink ports."
- note added: "PA7/PB0 are thermal ADCs; fan PWM uses timer-capable PE9/TIM1_CH1 and tach remains EC-owned."
- note added: "PE13 drives active-high MU_12V_ENABLE; PE14 reads MU_S0_HIGH; PE15 reads MU_12V_PG; PB1 reads TRACKPAD_FAULT_N."
- note added: "The EC has no user GPIO header; all tinkering I/O is isolated to the integrated RP2350 maker domain."
- note added: "U5 EN is intentionally floated: TI specifies an internal pull-up that enables the converter when EN is open."
- note added: "U5 follows the TPS54202 3.3V table and runs from EC_AON_IN so source validation firmware can execute before arbitration."
- note removed: "-- SWD debug header --"
- note removed: "== EC GPIO expansion / laptop power controls =="
- note removed: "== Keyboard Matrix GPIO bank (MX ULP rev A uses 5 rows x 14 cols) =="
- note removed: "== U5 TPS54202DDC VSYS -> MCU_3V3 Buck (3.3V, 2A) =="
- note removed: "EC can assert Mu PWRBTN_N/RSTBTN_N as open-drain GPIOs; J16 also allows physical case buttons."
- note removed: "J15 is the user-facing EC GPIO header: EC I2C, five GPIO/SPI-capable signals, power, and grounds."
- note removed: "MCU_USB_DP/DM (PA12/PA11, OTG_FS device mode) intentionally distinct from Power sheet's USB_DP1/DM1 (PD sink port)."
- note removed: "PA7/PB0 are assigned to skin and Mu-heatsink thermistors; fan PWM/tach remain EC-owned."
- note removed: "Second spare GPIO bank is assigned to E-key radio disables, GNSS UART/control/PPS, OLED reset, trackpad reset/INT, and one spare radio GPIO."
- note removed: "U5 uses TPS54202/TPS54302-style 0.596V feedback; R35/R36 set MCU_3V3 to about 3.30V."

Commit message: Finish USB-C policy and split out radio board
Parts:
- removed U46: SN74LVC1G08DBVR EC-reset-qualified service mux re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, Package_TO_SOT_SMD:SOT-23-5, symbol 74xGxx:74LVC1G08
- C780: renamed from R784; value 100k unused source-manager I/O pulldown -> 100n source-manager local; footprint Resistor_SMD:R_0603_1608Metric -> Capacitor_SMD:C_0603_1608Metric; symbol Device:R -> Device:C
- R172: renamed from C780; value 100n source-manager local -> 100k service mux reset-request pull-up; footprint Capacitor_SMD:C_0603_1608Metric -> Resistor_SMD:R_0603_1608Metric; symbol Device:C -> Device:R; MPN (none) -> RC0603FR-07100KL; Manufacturer (none) -> Yageo
- U44: value TCA9539PWR resettable source manager @0x20 -> TCA9539PWR resettable source manager @0x74; I2CAddress7Bit (none) -> 0x74
- U46: renamed from R172; value 100k service mux reset-request pull-up -> SN74LVC1G08DBVR EC-reset-qualified service mux reset; footprint Resistor_SMD:R_0603_1608Metric -> Package_TO_SOT_SMD:SOT-23-5; symbol Device:R -> 74xGxx:74LVC1G08; MPN RC0603FR-07100KL -> SN74LVC1G08DBVR; Manufacturer Yageo -> Texas Instruments; ResetContract (none) -> U45 RESET_N = EC NRST AND firmware reset request
Connections:
- net PD3_EFUSE_FAULT_N is gone; now on net SOURCE_MGR_SPARE2: U44.9 (IO0_5)
- net PD3_PATH_EN is gone; now on net SOURCE_MGR_SPARE1: U44.6 (IO0_2)
- net GND: now also U46.3 (GND); no longer R172.2
- net MCU_3V3: now also C780.1, U46.5 (VCC); no longer U46.1
- net NRST_NET: now also U46.1
- net SERVICE_MUX_RESET_N: now also U46.4
- net SERVICE_MUX_RESET_REQ_N: now also R172.2
- net SOURCE_MGR_SPARE1: no longer U44.18 (IO1_5)
- net SOURCE_MGR_SPARE2: no longer U44.19 (IO1_6)
- net PD2_TCPC_IRQ_N: now reaches U4.90 (PB4)
- net PD3_VALID_N renamed PD1_TCPC_IRQ_N
- net RADIO_AUDIO_SEL renamed RADIO_DB_PWR_EN
- net RADIO_GPIO0 renamed PD_PROTECT_FAULT_N
- net SOURCE_MGR_SPARE3 renamed RADIO_DB_PRESENT_N
- net RADIO_DB_PRESENT_N: no longer C780.1
- new net RADIO_DB_FAULT_N: U44.19 (IO1_6)
- new net RADIO_DB_PG: U44.18 (IO1_5)
- no-connect marks 3 -> 2
Changed lines of the file:
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@@
   (effects (font (size 1.27 1.27)) (justify left bottom))
 )
-(hierarchical_label "PD3_VALID_N"
+(hierarchical_label "PD1_TCPC_IRQ_N"
   (shape bidirectional)
   (at 224.79 379.73 0)
@@
   (effects (font (size 1.27 1.27)) (justify left bottom))
 )
-(no_connect (at 275.59 389.89))
-(hierarchical_label "RADIO_AUDIO_SEL"
+(hierarchical_label "PD2_TCPC_IRQ_N"
+  (shape bidirectional)
+  (at 275.59 389.89 0)
+  (effects (font (size 1.27 1.27)) (justify left bottom))
+)
+(hierarchical_label "RADIO_DB_PWR_EN"
   (shape bidirectional)
   (at 275.59 392.43 0)
@@
   (effects (font (size 1.27 1.27)) (justify left bottom))
 )
-(hierarchical_label "RADIO_GPIO0"
+(hierarchical_label "PD_PROTECT_FAULT_N"
   (shape bidirectional)
   (at 275.59 402.59 0)
@@
   (dnp no)
   (property "Reference" "U44" (at 699.77 327.66 0) (effects (font (size 1.27 1.27))))
-  (property "Value" "TCA9539PWR resettable source manager @0x20" (at 699.77 332.74 0) (effects (font (size 1.27 1.27))))
+  (property "Value" "TCA9539PWR resettable source manager @0x74" (at 699.77 332.74 0) (effects (font (size 1.27 1.27))))
   (property "Footprint" "Package_SO:TSSOP-24_4.4x7.8mm_P0.65mm" (at 699.77 330.2 0) (effects (font (size 1.27 1.27)) (hide yes)))
   (property "Datasheet" "" (at 699.77 330.2 0) (effects (font (size 1.27 1.27)) (hide yes)))
@@
   (property "MPN" "TCA9539PWR" (at 699.77 330.2 0) (effects (font (size 1.27 1.27)) (hide yes)))
   (property "Datasheet" "https://www.ti.com/lit/ds/symlink/tca9539.pdf" (at 699.77 330.2 0) (effects (font (size 1.27 1.27)) (hide yes)))
+  (property "I2CAddress7Bit" "0x74" (at 699.77 330.2 0) (effects (font (size 1.27 1.27)) (hide yes)))
   (property "ResetContract" "Pin 3 follows EC NRST; all P-ports reset to inputs and external SHDN pulldowns force every PD path off" (at 699.77 330.2 0) (effects (font (size 1.27 1.27)) (hide yes)))
   (pin "1")
@@
   (effects (font (size 1.27 1.27)) (justify left bottom))
 )
-(hierarchical_label "PD3_PATH_EN"
-  (shape bidirectional)
+(label "SOURCE_MGR_SPARE1"
   (at 712.47 314.96 0)
   (effects (font (size 1.27 1.27)) (justify left bottom))
@@
   (effects (font (size 1.27 1.27)) (justify left bottom))
 )
-(hierarchical_label "PD3_EFUSE_FAULT_N"
-  (shape bidirectional)
+(label "SOURCE_MGR_SPARE2"
   (at 712.47 322.58 0)
   (effects (font (size 1.27 1.27)) (justify left bottom))
@@
   (effects (font (size 1.27 1.27)) (justify left bottom))
 )
-(label "SOURCE_MGR_SPARE1"
+(hierarchical_label "RADIO_DB_PG"
+  (shape bidirectional)
   (at 712.47 345.44 0)
   (effects (font (size 1.27 1.27)) (justify left bottom))
 )
-(label "SOURCE_MGR_SPARE2"
+(hierarchical_label "RADIO_DB_FAULT_N"
+  (shape bidirectional)
   (at 712.47 347.98 0)
   (effects (font (size 1.27 1.27)) (justify left bottom))
 )
-(label "SOURCE_MGR_SPARE3"
+(hierarchical_label "RADIO_DB_PRESENT_N"
+  (shape bidirectional)
   (at 712.47 350.52 0)
   (effects (font (size 1.27 1.27)) (justify left bottom))
@@
   (effects (font (size 1.27 1.27)) (justify left bottom))
 )
-(symbol
-  (lib_id "Device:R")
-  (at 650.24 312.42 0)
-  (unit 1)
-  (exclude_from_sim no)
-  (in_bom yes)
-  (on_board yes)
-  (dnp no)
-  (property "Reference" "R784" (at 650.24 309.88 0) (effects (font (size 1.27 1.27))))
-  (property "Value" "100k unused source-manager I/O pulldown" (at 650.24 314.96 0) (effects (font (size 1.27 1.27))))
-  (property "Footprint" "Resistor_SMD:R_0603_1608Metric" (at 650.24 312.42 0) (effects (font (size 1.27 1.27)) (hide yes)))
-  (property "Datasheet" "" (at 650.24 312.42 0) (effects (font (size 1.27 1.27)) (hide yes)))
-  (pin "1")
-  (pin "2")
-  (instances
-    (project "ducktop2"
-      (path "/ed7eaa34-1bd3-577a-ab85-6415c5cdb1f8"
-        (reference "R784")
-        (unit 1)
-      )
-    )
-  )
-)
-(label "SOURCE_MGR_SPARE3"
-  (at 650.24 308.61 0)
-  (effects (font (size 1.27 1.27)) (justify left bottom))
-)
-(label "GND"
-  (at 650.24 316.23 0)
-  (effects (font (size 1.27 1.27)) (justify left bottom))
-)
