File: 03_mu_carrier.kicad_sch (KiCad schematic)
At the start: 140 parts, among them J10 Amphenol MDT420M01001 M-key N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, J8 DNP Mu SIO UART debug (IO vol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, J9 RTC backup coin-cell header, Q750 BSS138 fail-off EN/UVLO clamp, Q751 BSS138 active-high enable rel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, SW2 Mu Power, SW3 Mu Reset, U6 TPS56637RPAR VSYS -> SYS_5V (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, U7 TPS56637RPAR VSYS -> SYS_3V3 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, U750 TPS552892RYQR 12V buck-boost, U769 SN74LVC1G08DBVR qualified hos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, U770 TPS2553DDBVR internal host VB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, U771 TPS3897ADRYR internal VBUS su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, U772 TPS22975NDSGR switched PCIe e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

Commit message: Stamp generation-time BOM catalog; close 378 procurement gaps
Parts:
- C42, C770, C773, C791, C793: MPN (none) -> GRM188R71H104KA93D; Manufacturer (none) -> Murata
- C43, C47: MPN (none) -> C1608X7R1C104K080AA; Manufacturer (none) -> TDK
- C767, C774, C775: MPN (none) -> GRM188R71H103KA01; Manufacturer (none) -> Murata
- C771: MPN (none) -> GRM188R71H472KA01; Manufacturer (none) -> Murata
- C772: MPN (none) -> GRM1885C1H101JA01; Manufacturer (none) -> Murata
- R42, R770: MPN (none) -> RC0603FR-07169KL; Manufacturer (none) -> Yageo
- R43: MPN (none) -> RC0603FR-0745K3L; Manufacturer (none) -> Yageo
- R44, R768: MPN (none) -> RC0603FR-0710KL; Manufacturer (none) -> Yageo
- R45, R771: MPN (none) -> RC0603FR-0736K1L; Manufacturer (none) -> Yageo
- R46, R761, R762, R763, R766, R767, R769, R772: MPN (none) -> RC0603FR-07100KL; Manufacturer (none) -> Yageo
- R47, R48, R49, R757, R758: MPN (none) -> RC0603FR-070RL; Manufacturer (none) -> Yageo
- R750, R751: MPN (none) -> RC0603FR-0710RL; Manufacturer (none) -> Yageo
- R752: MPN (none) -> RC0603FR-0749R9L; Manufacturer (none) -> Yageo
- R753: MPN (none) -> RT0603BRD07102KL; Manufacturer (none) -> Yageo
- R754: MPN (none) -> RT0603BRD0711K3L; Manufacturer (none) -> Yageo
- R755: MPN (none) -> RC0603FR-0715KL; Manufacturer (none) -> Yageo
- R756: MPN (none) -> RC0603FR-0749K9L; Manufacturer (none) -> Yageo
- R759: MPN (none) -> RC0603FR-07150KL; Manufacturer (none) -> Yageo
- R760: MPN (none) -> RC0603FR-0723K7L; Manufacturer (none) -> Yageo

Commit message: Complete EC DFU port (J73) + DB power rework; verify schematic and board
- Add rear USB-C EC firmware programming port J73 (UFP/DFU) on Internal
  Services sheet: USBLC6-2P6 ESD (U63), 5.1k CC Rd resistors (R205/R211),
  22R series on D+/D- (R203/R204), mux-select hookup so BOOT0 high forces
  the USB mux to the DFU port
- Rename port ref J70->J73 after ham-radio collision; sync all net names
  (J73_CC1/J73_CC2)
- DB power rework: S5 gating + 3V3_STBY split, dual DCDC paths, GND
  returns on the standby rails; regenerate all sheets and re-verify
- sync_main_pcb_from_netlist: anchor placement for the 9 new footprints,
  scoped ECO support
- Board: rebuild main PCB with J73 footprint block (lib-sourced, net
  injection from netlist name attribute), sync pad nets for the 5 stale
  refs, remove duplicate R205/R211 copies
- Verified: check_schematic self-check OK (0 errors), radio DB contracts
  OK, ERC 0 errors, board DRC 0 electrical violations, board-vs-schematic
  net parity 0 conflicts, no duplicate refs
Parts:
- R42, R770: value 169k 1% TPS56637 EN high -> 100k 1% TPS56637 EN high (host-active gate)
- R45, R771: value 36.1k 1% TPS56637 EN low -> 100k 1% TPS56637 EN low
Connections:
- net MU_HOST_ACTIVE: now also R42.1, R770.1
- net VSYS: no longer R42.1, R770.1
Changed lines of the file:
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@@
   (dnp no)
   (property "Reference" "R42" (at 299.72 121.92 0) (effects (font (size 1.27 1.27))))
-  (property "Value" "169k 1% TPS56637 EN high" (at 299.72 127 0) (effects (font (size 1.27 1.27))))
+  (property "Value" "100k 1% TPS56637 EN high (host-active gate)" (at 299.72 127 0) (effects (font (size 1.27 1.27))))
   (property "Footprint" "Resistor_SMD:R_0603_1608Metric" (at 299.72 124.46 0) (effects (font (size 1.27 1.27)) (hide yes)))
   (property "Datasheet" "" (at 299.72 124.46 0) (effects (font (size 1.27 1.27)) (hide yes)))
@@
   )
 )
-(hierarchical_label "VSYS"
+(hierarchical_label "MU_HOST_ACTIVE"
   (shape bidirectional)
   (at 299.72 120.65 0)
@@
   (dnp no)
   (property "Reference" "R45" (at 299.72 132.08 0) (effects (font (size 1.27 1.27))))
-  (property "Value" "36.1k 1% TPS56637 EN low" (at 299.72 137.16 0) (effects (font (size 1.27 1.27))))
+  (property "Value" "100k 1% TPS56637 EN low" (at 299.72 137.16 0) (effects (font (size 1.27 1.27))))
   (property "Footprint" "Resistor_SMD:R_0603_1608Metric" (at 299.72 134.62 0) (effects (font (size 1.27 1.27)) (hide yes)))
   (property "Datasheet" "" (at 299.72 134.62 0) (effects (font (size 1.27 1.27)) (hide yes)))
@@
   (dnp no)
   (property "Reference" "R770" (at 355.6 52.07 0) (effects (font (size 1.27 1.27))))
-  (property "Value" "169k 1% TPS56637 EN high" (at 355.6 57.15 0) (effects (font (size 1.27 1.27))))
+  (property "Value" "100k 1% TPS56637 EN high (host-active gate)" (at 355.6 57.15 0) (effects (font (size 1.27 1.27))))
   (property "Footprint" "Resistor_SMD:R_0603_1608Metric" (at 355.6 54.61 0) (effects (font (size 1.27 1.27)) (hide yes)))
   (property "Datasheet" "" (at 355.6 54.61 0) (effects (font (size 1.27 1.27)) (hide yes)))
@@
   )
 )
-(hierarchical_label "VSYS"
+(hierarchical_label "MU_HOST_ACTIVE"
   (shape bidirectional)
   (at 355.6 50.8 0)
@@
   (dnp no)
   (property "Reference" "R771" (at 355.6 62.23 0) (effects (font (size 1.27 1.27))))
-  (property "Value" "36.1k 1% TPS56637 EN low" (at 355.6 67.31 0) (effects (font (size 1.27 1.27))))
+  (property "Value" "100k 1% TPS56637 EN low" (at 355.6 67.31 0) (effects (font (size 1.27 1.27))))
   (property "Footprint" "Resistor_SMD:R_0603_1608Metric" (at 355.6 64.77 0) (effects (font (size 1.27 1.27)) (hide yes)))
   (property "Datasheet" "" (at 355.6 64.77 0) (effects (font (size 1.27 1.27)) (hide yes)))

Commit message: Close remaining electronics-review items: FAN1_TAC, SLS_S3, SIO UART, F5/F6
- P2-2: fan FG (FAN_TACH, 8.2k MCU_3V3 pull-up) now feeds Mu FAN1_TAC
  (A1 pin 4; SIO GP52 tach input per LattePanda-Mu pin tables) so the
  module's thermal policy sees real fan speed
- P3-2: Mu SLS_S3 (A1 pin 7; SoC GPD5, high in S0/S3 per Mu pin tables)
  observed on the TCA9539 spare input; R783 100k default-low pulldown so an
  absent Mu reads off
- P3-1: Mu SIO console (3.3V Super I/O UART, SIO JP3/GP41) exposed on
  on-board probe pads TP16/TP17 with 100k MCU_3V3 idle pull-ups (R779/R784)
  on the rear service edge; EC has no spare UART-capable pin (documented)
- F5: move H15 (240,70) -> (252,70) per retention doc (was under the Mu
  courtyard); move SW4/R212 on-board at (185/196,180) (were off-board at
  y=195/200); npth_inside_courtyard cleared
- F6: apply DIFF_85/90/100 + USB2_45 net classes with the impedance-doc
  geometries and project-default 0.15mm clearance (idempotent apply);
  include DFU_CONN/EC_DFU USB2 pairs in USB2_45
- F7: verified already released (commits 91c4f3b/caf6ffb documented the
  ethernet notch + mounting pattern as contracts)
- Root-sheet builder: auto-expand sheet blocks to fit their pin count
- Pin-review contracts updated for the new A1/U44 wiring
- Verified: check_schematic self-check OK, ERC 0 errors, radio DB contracts
  OK, board DRC 0 electrical violations (shorts/mask-bridges/npth all 0),
  board-vs-schematic net parity 0 conflicts
Parts:
- removed C590, C591: 220n 10V X7R Wi-Fi TX AC, Capacitor_SMD:C_0402_1005Metric, symbol Device:C
- removed C597: 220n 10V X7R NVMe TX AC, Capacitor_SMD:C_0402_1005Metric, symbol Device:C
- removed C836: 10u 6.3V NVMe socket local bulk, Capacitor_SMD:C_1206_3216Metric, symbol Device:C
- removed R763: 100k CC pull-up, Resistor_SMD:R_0603_1608Metric, symbol Device:R
- removed R768: 10k LattePanda PSON required pull-up, Resistor_SMD:R_0603_1608Metric, symbol Device:R
- removed R777: 78.7k 1% VBUS sense top divider, Resistor_SMD:R_0603_1608Metric, symbol Device:R
- removed TP6: SYS_3V3 test, TestPoint:TestPoint_Pad_D1.0mm, symbol Connector:TestPoint
- removed U769: SN74LVC1G08DBVR qualified host-active AND, Package_TO_SOT_SMD:SOT-23-5, symbol 74xGxx:74LVC1G08
- added C592: 220n 10V X7R NVMe TX AC, Capacitor_SMD:C_0402_1005Metric, symbol Device:C
- added C793: 100n qualified host-active gate local, Capacitor_SMD:C_0603_1608Metric, symbol Device:C
- added H13: M2.5 isolated mainboard mounting hole, MountingHole:MountingHole_2.7mm_M2.5, symbol Mechanical:MountingHole
- added J9: RTC backup coin-cell header, Connector_JST:JST_GH_SM02B-GHS-TB_1x02-1MP_P1.25mm_Horizontal, symbol Connector_Generic:Conn_01x02
- added R47: 0R / PERST isolation, Resistor_SMD:R_0603_1608Metric, symbol Device:R
- added R48: 0R / REFCLK+ isolation, Resistor_SMD:R_0603_1608Metric, symbol Device:R
- added R49: 0R / REFCLK- isolation, Resistor_SMD:R_0603_1608Metric, symbol Device:R
- added R769: 100k MU_HOST_ACTIVE fail-low, Resistor_SMD:R_0603_1608Metric, symbol Device:R
- added R779: 100k MU_SIO_UART_TX idle pull-up, Resistor_SMD:R_0603_1608Metric, symbol Device:R
- added R784: 100k MU_SIO_UART_RX idle pull-up, Resistor_SMD:R_0603_1608Metric, symbol Device:R
- added TP15: Internal USB VBUS fault test, TestPoint:TestPoint_Pad_D1.0mm, symbol Connector:TestPoint
- added TP17: Mu SIO UART RX probe pad, TestPoint:TestPoint_Pad_D1.0mm, symbol Connector:TestPoint
- added TP5: SYS_5V test, TestPoint:TestPoint_Pad_D1.0mm, symbol Connector:TestPoint
- C590: renamed from R48; value 0R / REFCLK+ isolation -> 220n 10V X7R Wi-Fi TX AC; footprint Resistor_SMD:R_0603_1608Metric -> Capacitor_SMD:C_0402_1005Metric; symbol Device:R -> Device:C; MPN RC0603FR-070RL -> GRM155R71A224KE01D; Manufacturer Yageo -> Murata
- C591: renamed from R49; value 0R / REFCLK- isolation -> 220n 10V X7R Wi-Fi TX AC; footprint Resistor_SMD:R_0603_1608Metric -> Capacitor_SMD:C_0402_1005Metric; symbol Device:R -> Device:C; MPN RC0603FR-070RL -> GRM155R71A224KE01D; Manufacturer Yageo -> Murata
- C597: renamed from R47; value 0R / PERST isolation -> 220n 10V X7R NVMe TX AC; footprint Resistor_SMD:R_0603_1608Metric -> Capacitor_SMD:C_0402_1005Metric; symbol Device:R -> Device:C; MPN RC0603FR-070RL -> GRM155R71A224KE01D; Manufacturer Yageo -> Murata
- C836: renamed from H13; value M2.5 isolated mainboard mounting hole -> 10u 6.3V NVMe socket local bulk; footprint MountingHole:MountingHole_2.7mm_M2.5 -> Capacitor_SMD:C_1206_3216Metric; symbol Mechanical:MountingHole -> Device:C; Hardware_Spec 2.7mm isolated NPTH for M2.5 chassis screw; no electrical c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 -> (none); MPN (none) -> GRM21BR60J106ME19L; Manufacturer (none) -> Murata; now in the parts list
- J8: value DNP Mu SIO UART debug (IO voltage unverified) -> DNP Mu SIO UART debug header (3.3V, SIO console; probe via TP16/TP17)
- R763: renamed from TP5; value SYS_5V test -> 100k CC pull-up; footprint TestPoint:TestPoint_Pad_D1.0mm -> Resistor_SMD:R_0603_1608Metric; symbol Connector:TestPoint -> Device:R; MPN (none) -> RC0603FR-07100KL; Manufacturer (none) -> Yageo; ProcurementClass PCB copper test feature -> (none); now in the parts list
- R768: renamed from C793; value 100n qualified host-active gate local -> 10k LattePanda PSON required pull-up; footprint Capacitor_SMD:C_0603_1608Metric -> Resistor_SMD:R_0603_1608Metric; symbol Device:C -> Device:R; MPN GRM188R71H104KA93D -> RC0603FR-0710KL; Manufacturer Murata -> Yageo; ReferenceCircuit (none) -> LattePanda Mu Power Control and Status design guide
- R777: renamed from TP15; value Internal USB VBUS fault test -> 78.7k 1% VBUS sense top divider; footprint TestPoint:TestPoint_Pad_D1.0mm -> Resistor_SMD:R_0603_1608Metric; symbol Connector:TestPoint -> Device:R; MPN (none) -> RC0603FR-0778K7L; Manufacturer (none) -> Yageo; ProcurementClass PCB copper test feature -> (none); now in the parts list
- TP16: renamed from J9; value RTC backup coin-cell header -> Mu SIO UART TX probe pad; footprint Connector_JST:JST_GH_SM02B-GHS-TB_1x02-1MP_P1.25mm_Horizontal -> TestPoint:TestPoint_Pad_D1.0mm; symbol Connector_Generic:Conn_01x02 -> Connector:TestPoint; Contacts SSHL-002T-P0.2 -> (none); MPN SM02B-GHS-TB -> (none); Manufacturer JST -> (none); MatingHousing GHR-02V-S -> (none); ProcurementClass (none) -> PCB copper test feature; now left out of the parts list
- TP6: renamed from C592; value 220n 10V X7R NVMe TX AC -> SYS_3V3 test; footprint Capacitor_SMD:C_0402_1005Metric -> TestPoint:TestPoint_Pad_D1.0mm; symbol Device:C -> Connector:TestPoint; MPN GRM155R71A224KE01D -> (none); Manufacturer Murata -> (none); ProcurementClass (none) -> PCB copper test feature; now left out of the parts list
- U769: renamed from R769; value 100k MU_HOST_ACTIVE fail-low -> SN74LVC1G08DBVR qualified host-active AND; footprint Resistor_SMD:R_0603_1608Metric -> Package_TO_SOT_SMD:SOT-23-5; symbol Device:R -> 74xGxx:74LVC1G08; LogicContract (none) -> MU_HOST_ACTIVE=MU_S0_HIGH_AND_MU_12V_PG; MPN RC0603FR-07100KL -> SN74LVC1G08DBVR; Manufacturer Yageo -> Texas Instruments
Connections:
- net GND: now also C836.2, U769.3 (GND), C793.2, J9.2 (Pin_2), R769.2; no longer R768.2, TP16.2 (Pin_2), U769.2
- net INTERNAL_USB_VBUS: now also R777.1
- net INTERNAL_USB_VBUS_FAULT_N: now also TP15.1; no longer R777.1
- net INTERNAL_USB_VBUS_SENSE: now also R777.2
- net MCU_3V3: now also U769.5 (VCC), C793.1, R779.1, R784.1
- net MU12_CC_N: now also R763.2
- net MU12_VCC: now also R763.1
- net MU_12V_PG: now also U769.2
- net MU_HOST_ACTIVE: now also U769.4, R769.1; no longer U769.1
- net MU_S0_HIGH: now also R768.2, U769.1
- net MU_SIO_UART_RX: now also R784.2, TP17.1
- net MU_SIO_UART_TX: now also TP16.1, R779.2
- net PCIE_3V3: now also C836.1
- net PCIE_M_L1_TX_P: now also C592.2; no longer TP6.2
- net PCIE_M_L1_TX_RAW_P: now also C592.1; no longer TP6.1
- net PCIE_M_L3_TX_N: now also C597.2
- net PCIE_M_L3_TX_RAW_N: now also C597.1
- net PCIE_M_PERST_N: now also R47.2; no longer C597.2
- net PCIE_M_REFCLK_N: now also R49.2; no longer C591.2
- net PCIE_M_REFCLK_P: now also R48.2; no longer C590.2
- net PCIE_M_REFCLK_SRC_N: now also R49.1; no longer C591.1
- net PCIE_M_REFCLK_SRC_P: now also R48.1; no longer C590.1
- net PLTRST_SRC_N: now also R47.1; no longer C597.1
- net RTC_BAT: now also J9.1 (Pin_1); no longer TP16.1 (Pin_1)
- net SYS_3V3: now also TP6.1
- net SYS_5V: now also TP5.1; no longer R763.1
- net WIFI_PCIE_TX_N: now also C591.2
- net WIFI_PCIE_TX_P: now also C590.2
- net WIFI_PCIE_TX_RAW_N: now also C591.1
- net WIFI_PCIE_TX_RAW_P: now also C590.1
- net FAN_TACH: now reaches A1.4 (FAN1_TAC)
- net SLS_S3: now reaches A1.7 (SLS_S3)
- no-connect marks 137 -> 135
Changed lines of the file:
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@@
   (effects (font (size 1.27 1.27)) (justify left bottom))
 )
-(no_connect (at 200.66 55.88))
+(hierarchical_label "FAN_TACH"
+  (shape bidirectional)
+  (at 200.66 55.88 0)
+  (effects (font (size 1.27 1.27)) (justify left bottom))
+)
 (label "PCIE_M_L0_RX_P"
   (at 119.38 116.84 0)
@@
   (effects (font (size 1.27 1.27)) (justify left bottom))
 )
-(no_connect (at 119.38 58.42))
+(hierarchical_label "SLS_S3"
+  (shape bidirectional)
+  (at 119.38 58.42 0)
+  (effects (font (size 1.27 1.27)) (justify left bottom))
+)
 (hierarchical_label "USBC2_DP"
   (shape bidirectional)
@@
   (dnp yes)
   (property "Reference" "J8" (at 30.48 97.79 0) (effects (font (size 1.27 1.27))))
-  (property "Value" "DNP Mu SIO UART debug (IO voltage unverified)" (at 30.48 102.87 0) (effects (font (size 1.27 1.27))))
+  (property "Value" "DNP Mu SIO UART debug header (3.3V, SIO console; probe via TP16/TP17)" (at 30.48 102.87 0) (effects (font (size 1.27 1.27))))
   (property "Footprint" "Connector_PinHeader_2.54mm:PinHeader_1x04_P2.54mm_Vertical" (at 30.48 100.33 0) (effects (font (size 1.27 1.27)) (hide yes)))
   (property "Datasheet" "" (at 30.48 100.33 0) (effects (font (size 1.27 1.27)) (hide yes)))
@@
   (effects (font (size 1.27 1.27)) (justify left bottom))
 )
+(symbol
+  (lib_id "Connector:TestPoint")
+  (at 39.37 100.33 0)
+  (unit 1)
+  (exclude_from_sim no)
+  (in_bom no)
+  (on_board yes)
+  (dnp no)
+  (property "Reference" "TP16" (at 39.37 97.79 0) (effects (font (size 1.27 1.27))))
+  (property "Value" "Mu SIO UART TX probe pad" (at 39.37 102.87 0) (effects (font (size 1.27 1.27))))
+  (property "Footprint" "TestPoint:TestPoint_Pad_D1.0mm" (at 39.37 100.33 0) (effects (font (size 1.27 1.27)) (hide yes)))
+  (property "Datasheet" "" (at 39.37 100.33 0) (effects (font (size 1.27 1.27)) (hide yes)))
+  (property "ProcurementClass" "PCB copper test feature" (at 39.37 100.33 0) (effects (font (size 1.27 1.27)) (hide yes)))
+  (pin "1")
+  (instances
+    (project "ducktop2"
+      (path "/7f3572a2-a529-5ef0-93eb-27f85c0119a9"
+        (reference "TP16")
+        (unit 1)
+      )
+    )
+  )
+)
+(label "MU_SIO_UART_TX"
+  (at 39.37 100.33 0)
+  (effects (font (size 1.27 1.27)) (justify left bottom))
+)
+(symbol
+  (lib_id "Connector:TestPoint")
+  (at 49.53 100.33 0)
+  (unit 1)
+  (exclude_from_sim no)
+  (in_bom no)
+  (on_board yes)
+  (dnp no)
+  (property "Reference" "TP17" (at 49.53 97.79 0) (effects (font (size 1.27 1.27))))
+  (property "Value" "Mu SIO UART RX probe pad" (at 49.53 102.87 0) (effects (font (size 1.27 1.27))))
+  (property "Footprint" "TestPoint:TestPoint_Pad_D1.0mm" (at 49.53 100.33 0) (effects (font (size 1.27 1.27)) (hide yes)))
+  (property "Datasheet" "" (at 49.53 100.33 0) (effects (font (size 1.27 1.27)) (hide yes)))
+  (property "ProcurementClass" "PCB copper test feature" (at 49.53 100.33 0) (effects (font (size 1.27 1.27)) (hide yes)))
+  (pin "1")
+  (instances
+    (project "ducktop2"
+      (path "/7f3572a2-a529-5ef0-93eb-27f85c0119a9"
+        (reference "TP17")
+        (unit 1)
+      )
+    )
+  )
+)
+(label "MU_SIO_UART_RX"
+  (at 49.53 100.33 0)
+  (effects (font (size 1.27 1.27)) (justify left bottom))
+)
+(symbol
+  (lib_id "Device:R")
+  (at 39.37 110.49 0)
+  (unit 1)
+  (exclude_from_sim no)
+  (in_bom yes)
+  (on_board yes)
+  (dnp no)
+  (property "Reference" "R779" (at 39.37 107.95 0) (effects (font (size 1.27 1.27))))
+  (property "Value" "100k MU_SIO_UART_TX idle pull-up" (at 39.37 113.03 0) (effects (font (size 1.27 1.27))))
+  (property "Footprint" "Resistor_SMD:R_0603_1608Metric" (at 39.37 110.49 0) (effects (font (size 1.27 1.27)) (hide yes)))
+  (property "Datasheet" "" (at 39.37 110.49 0) (effects (font (size 1.27 1.27)) (hide yes)))
+  (pin "1")
+  (pin "2")
+  (instances
+    (project "ducktop2"
+      (path "/7f3572a2-a529-5ef0-93eb-27f85c0119a9"
+        (reference "R779")
+        (unit 1)
+      )
+    )
+  )
+)
+(hierarchical_label "MCU_3V3"
+  (shape bidirectional)
+  (at 39.37 106.68 0)
+  (effects (font (size 1.27 1.27)) (justify left bottom))
+)
+(label "MU_SIO_UART_TX"
+  (at 39.37 114.3 0)
+  (effects (font (size 1.27 1.27)) (justify left bottom))
+)
+(symbol
+  (lib_id "Device:R")
+  (at 49.53 110.49 0)
+  (unit 1)
+  (exclude_from_sim no)
+  (in_bom yes)
+  (on_board yes)
+  (dnp no)
+  (property "Reference" "R784" (at 49.53 107.95 0) (effects (font (size 1.27 1.27))))
+  (property "Value" "100k MU_SIO_UART_RX idle pull-up" (at 49.53 113.03 0) (effects (font (size 1.27 1.27))))
+  (property "Footprint" "Resistor_SMD:R_0603_1608Metric" (at 49.53 110.49 0) (effects (font (size 1.27 1.27)) (hide yes)))
+  (property "Datasheet" "" (at 49.53 110.49 0) (effects (font (size 1.27 1.27)) (hide yes)))
+  (pin "1")
+  (pin "2")
+  (instances
+    (project "ducktop2"
+      (path "/7f3572a2-a529-5ef0-93eb-27f85c0119a9"
+        (reference "R784")
+        (unit 1)
+      )
+    )
+  )
+)
+(hierarchical_label "MCU_3V3"
+  (shape bidirectional)
+  (at 49.53 106.68 0)
+  (effects (font (size 1.27 1.27)) (justify left bottom))
+)
+(label "MU_SIO_UART_RX"
+  (at 49.53 114.3 0)
+  (effects (font (size 1.27 1.27)) (justify left bottom))
+)
