File: 03_mu_carrier.kicad_sch (KiCad schematic)
At the start: 144 parts, among them J10 Amphenol MDT420M01001 M-key N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, J8 DNP Mu SIO UART debug header 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, J9 RTC backup coin-cell header, Q750 BSS138 fail-off EN/UVLO clamp, Q751 BSS138 active-high enable rel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, SW2 Mu Power, SW3 Mu Reset, U6 TPS56637RPAR VSYS -> SYS_5V (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, U7 TPS56637RPAR VSYS -> SYS_3V3 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, U750 TPS552892RYQR 12V buck-boost, U769 SN74LVC1G08DBVR qualified hos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, U770 TPS2553DDBVR internal host VB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, U771 TPS3897ADRYR internal VBUS su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, U772 TPS22975NDSGR switched PCIe e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

Commit message: NVMe power headroom + pack-backed RTC (coin cell removed)
- Add dedicated PCIe endpoint buck U773 (TPS56637, VSYS -> PCIE_3V3_IN),
  host-gated like U6/U7: moves ~3A endpoint load (NVMe 1.5-2.5A peak,
  Wi-Fi, GbE) off SYS_3V3; SYS_3V3 peak drops ~6A -> ~3A, endpoint rail
  now has ~50% headroom at the 6A buck.  U772 switch input re-railed to
  PCIE_3V3_IN.
- RTC: replace the coin-cell header J9 with a 1N5819HW diode-OR from the
  always-on MCU_3V3 + 1u hold cap (C783) on the freed J9 footprint spot;
  clock persists while the pack or AC is connected, resets on pack removal
  (the tradeoff requested).  Saves the coin cell, holder and header.
- Layer-count gates updated 6 -> 8; sync add/remove gates updated
- Verified: ERC 0, gate pass, net parity 0 conflicts, board DRC 0
  electrical / 0 clearance, courtyards 167 (below baseline); residual 6
  silk-text items on the dense buck cluster are cosmetic (baseline class)
Parts:
- removed C40, C46: 10u 50V X7R TPS56637 VIN, Capacitor_SMD:C_1206_3216Metric, symbol Device:C
- removed C793: 100n qualified host-active gate local, Capacitor_SMD:C_0603_1608Metric, symbol Device:C
- removed L750: 4.7uH 10.1A Isat / 6.9A Irms, Inductor_SMD:L_Coilcraft_XAL7030-472, symbol Device:L
- removed R761: 100k fail-off gate divider low, Resistor_SMD:R_0603_1608Metric, symbol Device:R
- removed R773: 43.2k 1% internal host VBUS 0.61A ILIM, Resistor_SMD:R_0603_1608Metric, symbol Device:R
- removed R775: 10k internal host VBUS valid pull-up, Resistor_SMD:R_0603_1608Metric, symbol Device:R
- removed R776: 100k PCIe endpoint rail fail-low, Resistor_SMD:R_0603_1608Metric, symbol Device:R
- added C587: 100n 10V X7R Mu USB3 TX AC, Capacitor_SMD:C_0402_1005Metric, symbol Device:C
- added C776, C777: 10u 50V X7R TPS56637 VIN, Capacitor_SMD:C_1206_3216Metric, symbol Device:C
- added C778: 100n 50V X7R TPS56637 VIN HF, Capacitor_SMD:C_0603_1608Metric, symbol Device:C
- added C782: 47u 6.3V PCIE_3V3_IN rail bulk, Capacitor_SMD:C_1206_3216Metric, symbol Device:C
- added C783: 1u RTC_BAT hold, Capacitor_SMD:C_0805_2012Metric, symbol Device:C
- added C833: 4.7n PCIe endpoint controlled slew, Capacitor_SMD:C_0402_1005Metric, symbol Device:C
- added C834: 47u 6.3V PCIe endpoint rail bulk, Capacitor_SMD:C_1206_3216Metric, symbol Device:C
- added L1702: XAL7070-222MEC 2.2uH 19.6A Isat30%, Inductor_SMD:L_Coilcraft_XAL7070-XXX, symbol Device:L
- added Q750: BSS138 fail-off EN/UVLO clamp, Package_TO_SOT_SMD:SOT-23, symbol Q_NMOS_SOT23_GSD:Q_NMOS_SOT23_GSD
- added R785: 45.3k 1% TPS56637 FB high, Resistor_SMD:R_0603_1608Metric, symbol Device:R
- added R786: 10k 1% TPS56637 FB low, Resistor_SMD:R_0603_1608Metric, symbol Device:R
- added R787: 100k 1% TPS56637 EN high (host-active gate), Resistor_SMD:R_0603_1608Metric, symbol Device:R
- added R788: 100k 1% TPS56637 EN low, Resistor_SMD:R_0603_1608Metric, symbol Device:R
- added R789: 100k PCIE_3V3_PG pull-up, Resistor_SMD:R_0603_1608Metric, symbol Device:R
- added TP13: Internal USB VBUS test, TestPoint:TestPoint_Pad_D1.0mm, symbol Connector:TestPoint
- added TP5: SYS_5V test, TestPoint:TestPoint_Pad_D1.0mm, symbol Connector:TestPoint
- added U7: TPS56637RPAR VSYS -> SYS_3V3 (3.32V, 6A class), ducktop2:Texas_RPA0010A_VQFN-HR-10_3x3mm, symbol TPS56637:TPS56637
- added U769: SN74LVC1G08DBVR qualified host-active AND, Package_TO_SOT_SMD:SOT-23-5, symbol 74xGxx:74LVC1G08
- added U770: TPS2553DDBVR internal host VBUS 0.61A, Package_TO_SOT_SMD:SOT-23-6, symbol TPS2553D:TPS2553D
- added U771: TPS3897ADRYR internal VBUS supervisor (always-pow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, Package_SON:Texas_USON-6_1x1.45mm_P0.5mm_SMD, symbol TPS3897ADRYR:TPS3897ADRYR
- C41: renamed from C42; value 100n 50V X7R TPS56637 VIN HF -> 10u 50V X7R TPS56637 VIN; footprint Capacitor_SMD:C_0603_1608Metric -> Capacitor_SMD:C_1206_3216Metric; MPN GRM188R71H104KA93D -> CGA5L1X7R1H106K160AC; Manufacturer Murata -> TDK
- C42: renamed from C43; value 100n 16V X7R TPS56637 BOOT -> 100n 50V X7R TPS56637 VIN HF; MPN C1608X7R1C104K080AA -> GRM188R71H104KA93D; Manufacturer TDK -> Murata
- C43: renamed from L4; value XAL7070-332MEC 3.3uH 19.4A Isat30% -> 100n 16V X7R TPS56637 BOOT; footprint Inductor_SMD:L_Coilcraft_XAL7070-XXX -> Capacitor_SMD:C_0603_1608Metric; symbol Device:L -> Device:C; MPN XAL7070-332MEC -> C1608X7R1C104K080AA; Manufacturer Coilcraft -> TDK
- C45: renamed from U7; value TPS56637RPAR VSYS -> SYS_3V3 (3.32V, 6A class) -> 22u 16V X7R TPS56637 OUT; footprint ducktop2:Texas_RPA0010A_VQFN-HR-10_3x3mm -> Capacitor_SMD:C_1206_3216Metric; symbol TPS56637:TPS56637 -> Device:C; MPN TPS56637RPAR -> GRM31CZ71C226ME15L; Manufacturer Texas Instruments -> Murata
- C47: renamed from L5; value XAL7070-222MEC 2.2uH 19.6A Isat30% -> 100n 16V X7R TPS56637 BOOT; footprint Inductor_SMD:L_Coilcraft_XAL7070-XXX -> Capacitor_SMD:C_0603_1608Metric; symbol Device:L -> Device:C; MPN XAL7070-222MEC -> C1608X7R1C104K080AA; Manufacturer Coilcraft -> TDK
- C750: renamed from C751; value 10u 50V X7R input -> 68u 50V hybrid input bulk; footprint Capacitor_SMD:C_1206_3216Metric -> Capacitor_SMD:CP_Elec_8x10; symbol Device:C -> Device:C_Polarized; MPN CGA5L1X7R1H106K160AC -> EEHZA1H680P; Manufacturer TDK -> Panasonic
- C752: renamed from C753; value 1u 50V X5R input -> 10u 50V X7R input; footprint Capacitor_SMD:C_0603_1608Metric -> Capacitor_SMD:C_1206_3216Metric; MPN GRT188R61H105ME13D -> CGA5L1X7R1H106K160AC; Manufacturer Murata -> TDK
- C753: renamed from C754; value 100n 50V X7R input HF -> 1u 50V X5R input; footprint Capacitor_SMD:C_0402_1005Metric -> Capacitor_SMD:C_0603_1608Metric; MPN GRM155R71H104ME14D -> GRT188R61H105ME13D
- C755: renamed from C756; value 100n 50V X7R output HF -> 100n 50V X7R input HF
- C757: renamed from C758; value 1u 50V X5R output -> 100n 50V X7R output HF; footprint Capacitor_SMD:C_0603_1608Metric -> Capacitor_SMD:C_0402_1005Metric; MPN GRT188R61H105ME13D -> GRM155R71H104ME14D
- C758: renamed from C759; value 10u 50V X7R output -> 1u 50V X5R output; footprint Capacitor_SMD:C_1206_3216Metric -> Capacitor_SMD:C_0603_1608Metric; MPN CGA5L1X7R1H106K160AC -> GRT188R61H105ME13D; Manufacturer TDK -> Murata
- C761: renamed from C762; value 100u 35V hybrid output bulk -> 10u 50V X7R output; footprint Capacitor_SMD:CP_Elec_6.3x5.8 -> Capacitor_SMD:C_1206_3216Metric; symbol Device:C_Polarized -> Device:C; MPN EEHZK1V101XP -> CGA5L1X7R1H106K160AC; Manufacturer Panasonic -> TDK
- C762: renamed from C763; value 1u 50V post-sense load-side bypass -> 100u 35V hybrid output bulk; footprint Capacitor_SMD:C_0603_1608Metric -> Capacitor_SMD:CP_Elec_6.3x5.8; symbol Device:C -> Device:C_Polarized; MPN GRT188R61H105ME13D -> EEHZK1V101XP; Manufacturer Murata -> Panasonic
- C763: renamed from C764; value 22u 16V X7R VCC mandatory; effective >4.7u -> 1u 50V post-sense load-side bypass; footprint Capacitor_SMD:C_1206_3216Metric -> Capacitor_SMD:C_0603_1608Metric; MPN GRM31CZ71C226ME15L -> GRT188R61H105ME13D
- C764: renamed from C765; value 100n 50V X8L bootstrap -> 22u 16V X7R VCC mandatory; effective >4.7u; footprint Capacitor_SMD:C_0603_1608Metric -> Capacitor_SMD:C_1206_3216Metric; MPN GCM188L81H104KA57D -> GRM31CZ71C226ME15L
- C766: renamed from R764; value DNP 2.2R 0.25W switch-node snubber -> 100n 50V X8L bootstrap; footprint Resistor_SMD:R_1206_3216Metric -> Capacitor_SMD:C_0603_1608Metric; symbol Device:R -> Device:C; MPN ERJ-8RQF2R2V -> GCM188L81H104KA57D; Manufacturer Panasonic -> Murata; now fitted; now in the parts list
- C767: renamed from R757; value 0R MODE forced-PWM -> 10n DITH/SYNC spreading; footprint Resistor_SMD:R_0603_1608Metric -> Capacitor_SMD:C_0603_1608Metric; symbol Device:R -> Device:C; MPN RC0603FR-070RL -> GRM188R71H103KA01; Manufacturer Yageo -> Murata
- C768: renamed from R765; value DNP 2.2R 0.25W switch-node snubber -> DNP 2.2n 250V X7R switch-node snubber; footprint Resistor_SMD:R_1206_3216Metric -> Capacitor_SMD:C_0805_2012Metric; symbol Device:R -> Device:C; MPN ERJ-8RQF2R2V -> GRM21AR72E222KW01D; Manufacturer Panasonic -> Murata
- C769: renamed from R750; value 10R ISP Kelvin filter -> DNP 2.2n 250V X7R switch-node snubber; footprint Resistor_SMD:R_0603_1608Metric -> Capacitor_SMD:C_0805_2012Metric; symbol Device:R -> Device:C; MPN RC0603FR-0710RL -> GRM21AR72E222KW01D; Manufacturer Yageo -> Murata; now not fitted; now left out of the parts list
- C770: renamed from R752; value 49.9R FB isolation -> 100n differential current-sense filter; footprint Resistor_SMD:R_0603_1608Metric -> Capacitor_SMD:C_0603_1608Metric; symbol Device:R -> Device:C; MPN RC0603FR-0749R9L -> GRM188R71H104KA93D; Manufacturer Yageo -> Murata
- C771: renamed from C772; value 100p C0G COMP HF -> 4.7n COMP; MPN GRM1885C1H101JA01 -> GRM188R71H472KA01
- C772: renamed from R756; value 49.9k 1% FSW = 400kHz -> 100p C0G COMP HF; footprint Resistor_SMD:R_0603_1608Metric -> Capacitor_SMD:C_0603_1608Metric; symbol Device:R -> Device:C; MPN RC0603FR-0749K9L -> GRM1885C1H101JA01; Manufacturer Yageo -> Murata
- C773: renamed from Q750; value BSS138 fail-off EN/UVLO clamp -> 100n UVLO noise filter; footprint Package_TO_SOT_SMD:SOT-23 -> Capacitor_SMD:C_0603_1608Metric; symbol Q_NMOS_SOT23_GSD:Q_NMOS_SOT23_GSD -> Device:C; MPN BSS138LT1G -> GRM188R71H104KA93D; Manufacturer onsemi -> Murata
- C779: renamed from TP5; value SYS_5V test -> 100n 16V X7R TPS56637 BOOT; footprint TestPoint:TestPoint_Pad_D1.0mm -> Capacitor_SMD:C_0603_1608Metric; symbol Connector:TestPoint -> Device:C; ProcurementClass PCB copper test feature -> (none); now in the parts list
- C790: renamed from C791; value 100n 50V X7R TPS56637 VIN HF -> 10u 50V X7R TPS56637 VIN; footprint Capacitor_SMD:C_0603_1608Metric -> Capacitor_SMD:C_1206_3216Metric; MPN GRM188R71H104KA93D -> CGA5L1X7R1H106K160AC; Manufacturer Murata -> TDK
- C791: renamed from C47; value 100n 16V X7R TPS56637 BOOT -> 100n 50V X7R TPS56637 VIN HF; MPN C1608X7R1C104K080AA -> GRM188R71H104KA93D; Manufacturer TDK -> Murata
- C792: renamed from C66; value 100n 10V X7R Mu USB3 TX AC -> 22u 16V X7R TPS56637 OUT; footprint Capacitor_SMD:C_0402_1005Metric -> Capacitor_SMD:C_1206_3216Metric; MPN GRM155R71A104KA01D -> GRM31CZ71C226ME15L
- C793: renamed from R769; value 100k MU_HOST_ACTIVE fail-low -> 100n qualified host-active gate local; footprint Resistor_SMD:R_0603_1608Metric -> Capacitor_SMD:C_0603_1608Metric; symbol Device:R -> Device:C; MPN RC0603FR-07100KL -> GRM188R71H104KA93D; Manufacturer Yageo -> Murata
- C794: renamed from C830; value 10u internal host VBUS output -> 1u internal host VBUS switch input; footprint Capacitor_SMD:C_1206_3216Metric -> Capacitor_SMD:C_0805_2012Metric; MPN GRM21BR61A106KE19L -> GRM188R71A105KA61D
- C830: renamed from U771; value TPS3897ADRYR internal VBUS supervisor (always-powered) -> 10u internal host VBUS output; footprint Package_SON:Texas_USON-6_1x1.45mm_P0.5mm_SMD -> Capacitor_SMD:C_1206_3216Metric; symbol TPS3897ADRYR:TPS3897ADRYR -> Device:C; Function Assert VBUS valid only after SENSE (divided INTERNAL_USB_VB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 -> (none); MPN TPS3897ADRYR -> GRM21BR61A106KE19L; Manufacturer Texas Instruments -> Murata
- C831: renamed from R777; value 78.7k 1% VBUS sense top divider -> 100n TPS3897 VCC bypass; footprint Resistor_SMD:R_0603_1608Metric -> Capacitor_SMD:C_0603_1608Metric; symbol Device:R -> Device:C; MPN RC0603FR-0778K7L -> GRM188R71A104KA01D; Manufacturer Yageo -> Murata
- C832: renamed from C833; value 4.7n PCIe endpoint controlled slew -> 1u PCIe endpoint switch input; footprint Capacitor_SMD:C_0402_1005Metric -> Capacitor_SMD:C_0805_2012Metric; MPN GRM155R71H472KA01D -> GRM188R60J105KA01D
- D1824: renamed from J9; value RTC backup coin-cell header -> 1N5819HW RTC_BAT diode-OR from MCU_3V3; footprint Connector_JST:JST_GH_SM02B-GHS-TB_1x02-1MP_P1.25mm_Horizontal -> Diode_SMD:Nexperia_CFP3_SOD-123W; symbol Connector_Generic:Conn_01x02 -> Device:D_Schottky; Contacts SSHL-002T-P0.2 -> (none); MPN SM02B-GHS-TB -> 1N5819HW; Manufacturer JST -> STMicroelectronics; MatingHousing GHR-02V-S -> (none)
- L4: renamed from R40; value 76.8k 0.1% TPS56637 FB high -> XAL7070-332MEC 3.3uH 19.4A Isat30%; footprint Resistor_SMD:R_0603_1608Metric -> Inductor_SMD:L_Coilcraft_XAL7070-XXX; symbol Device:R -> Device:L; MPN RT0603BRD0776K8L -> XAL7070-332MEC; Manufacturer Yageo -> Coilcraft
- L5: renamed from R43; value 45.3k 1% TPS56637 FB high -> XAL7070-222MEC 2.2uH 19.6A Isat30%; footprint Resistor_SMD:R_0603_1608Metric -> Inductor_SMD:L_Coilcraft_XAL7070-XXX; symbol Device:R -> Device:L; MPN RC0603FR-0745K3L -> XAL7070-222MEC; Manufacturer Yageo -> Coilcraft
- L750: renamed from RS750; value 15mOhm 1% 1W; 3.33A output current limit -> 4.7uH 10.1A Isat / 6.9A Irms; footprint Resistor_SMD:R_1206_3216Metric -> Inductor_SMD:L_Coilcraft_XAL7030-472; symbol Device:R -> Device:L; MPN ERJ8BWFR015V -> XAL7030-472MEC; Manufacturer Panasonic -> Coilcraft
- R40: renamed from R41; value 10k 0.1% TPS56637 FB low -> 76.8k 0.1% TPS56637 FB high; MPN RT0603BRD0710KL -> RT0603BRD0776K8L
- R41: renamed from R42; value 100k 1% TPS56637 EN high (host-active gate) -> 10k 0.1% TPS56637 FB low; MPN RC0603FR-07169KL -> RT0603BRD0710KL
- R42: renamed from R45; value 100k 1% TPS56637 EN low -> 100k 1% TPS56637 EN high (host-active gate); MPN RC0603FR-0736K1L -> RC0603FR-07169KL
- R43: renamed from R44; value 10k 1% TPS56637 FB low -> 45.3k 1% TPS56637 FB high; MPN RC0603FR-0710KL -> RC0603FR-0745K3L
- R44: renamed from R770; value 100k 1% TPS56637 EN high (host-active gate) -> 10k 1% TPS56637 FB low; MPN RC0603FR-07169KL -> RC0603FR-0710KL
- R45: renamed from R46; value 100k SYS_5V PG pull-up -> 100k 1% TPS56637 EN low; MPN RC0603FR-07100KL -> RC0603FR-0736K1L
- R46: renamed from C44; value 22u 16V X7R TPS56637 OUT -> 100k SYS_5V PG pull-up; footprint Capacitor_SMD:C_1206_3216Metric -> Resistor_SMD:R_0603_1608Metric; symbol Device:C -> Device:R; MPN GRM31CZ71C226ME15L -> RC0603FR-07100KL; Manufacturer Murata -> Yageo
- R750: renamed from R751; value 10R ISN Kelvin filter -> 10R ISP Kelvin filter
- R751: renamed from C770; value 100n differential current-sense filter -> 10R ISN Kelvin filter; footprint Capacitor_SMD:C_0603_1608Metric -> Resistor_SMD:R_0603_1608Metric; symbol Device:C -> Device:R; MPN GRM188R71H104KA93D -> RC0603FR-0710RL; Manufacturer Murata -> Yageo
- R752: renamed from R753; value 102k 0.1% 12V FB high -> 49.9R FB isolation; MPN RT0603BRD07102KL -> RC0603FR-0749R9L
- R753: renamed from R754; value 11.3k 0.1% 12V FB low -> 102k 0.1% 12V FB high; MPN RT0603BRD0711K3L -> RT0603BRD07102KL
- R754: renamed from R755; value 15k COMP series -> 11.3k 0.1% 12V FB low; MPN RC0603FR-0715KL -> RT0603BRD0711K3L
- R755: renamed from C771; value 4.7n COMP -> 15k COMP series; footprint Capacitor_SMD:C_0603_1608Metric -> Resistor_SMD:R_0603_1608Metric; symbol Device:C -> Device:R; MPN GRM188R71H472KA01 -> RC0603FR-0715KL; Manufacturer Murata -> Yageo
- R756: renamed from C767; value 10n DITH/SYNC spreading -> 49.9k 1% FSW = 400kHz; footprint Capacitor_SMD:C_0603_1608Metric -> Resistor_SMD:R_0603_1608Metric; symbol Device:C -> Device:R; MPN GRM188R71H103KA01 -> RC0603FR-0749K9L; Manufacturer Murata -> Yageo
- R757: renamed from R758; value 0R EXTVCC selects internal LDO -> 0R MODE forced-PWM
- R758: renamed from R759; value 150k 1% UVLO high; 9.0V rising -> 0R EXTVCC selects internal LDO; MPN RC0603FR-07150KL -> RC0603FR-070RL
- R759: renamed from R760; value 23.7k 1% UVLO low -> 150k 1% UVLO high; 9.0V rising; MPN RC0603FR-0723K7L -> RC0603FR-07150KL
- R760: renamed from C773; value 100n UVLO noise filter -> 23.7k 1% UVLO low; footprint Capacitor_SMD:C_0603_1608Metric -> Resistor_SMD:R_0603_1608Metric; symbol Device:C -> Device:R; MPN GRM188R71H104KA93D -> RC0603FR-0723K7L; Manufacturer Murata -> Yageo
- R761: renamed from R766; value 100k fail-off gate divider high -> 100k fail-off gate divider low
- R764: renamed from C768; value DNP 2.2n 250V X7R switch-node snubber -> DNP 2.2R 0.25W switch-node snubber; footprint Capacitor_SMD:C_0805_2012Metric -> Resistor_SMD:R_1206_3216Metric; symbol Device:C -> Device:R; MPN GRM21AR72E222KW01D -> ERJ-8RQF2R2V; Manufacturer Murata -> Panasonic
- R765: renamed from C769; value DNP 2.2n 250V X7R switch-node snubber -> DNP 2.2R 0.25W switch-node snubber; footprint Capacitor_SMD:C_0805_2012Metric -> Resistor_SMD:R_1206_3216Metric; symbol Device:C -> Device:R; MPN GRM21AR72E222KW01D -> ERJ-8RQF2R2V; Manufacturer Murata -> Panasonic
- R766: renamed from R767; value 100k MU_12V_ENABLE reset pulldown -> 100k fail-off gate divider high
- R767: renamed from R768; value 10k LattePanda PSON required pull-up -> 100k MU_12V_ENABLE reset pulldown; MPN RC0603FR-0710KL -> RC0603FR-07100KL; ReferenceCircuit LattePanda Mu Power Control and Status design guide -> (none)
- R768: renamed from U769; value SN74LVC1G08DBVR qualified host-active AND -> 10k LattePanda PSON required pull-up; footprint Package_TO_SOT_SMD:SOT-23-5 -> Resistor_SMD:R_0603_1608Metric; symbol 74xGxx:74LVC1G08 -> Device:R; LogicContract MU_HOST_ACTIVE=MU_S0_HIGH_AND_MU_12V_PG -> (none); MPN SN74LVC1G08DBVR -> RC0603FR-0710KL; Manufacturer Texas Instruments -> Yageo; ReferenceCircuit (none) -> LattePanda Mu Power Control and Status design guide
- R769: renamed from U770; value TPS2553DDBVR internal host VBUS 0.61A -> 100k MU_HOST_ACTIVE fail-low; footprint Package_TO_SOT_SMD:SOT-23-6 -> Resistor_SMD:R_0603_1608Metric; symbol TPS2553D:TPS2553D -> Device:R; Function Carrier-generated physical VBUS for permanently attached Mu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 -> (none); MPN TPS2553DDBVR -> RC0603FR-07100KL; Manufacturer Texas Instruments -> Yageo
- R770: renamed from R771; value 100k 1% TPS56637 EN low -> 100k 1% TPS56637 EN high (host-active gate); MPN RC0603FR-0736K1L -> RC0603FR-07169KL
- R771: renamed from R772; value 100k SYS_3V3 PG pull-up -> 100k 1% TPS56637 EN low; MPN RC0603FR-07100KL -> RC0603FR-0736K1L
- R772: renamed from C48; value 22u 16V X7R TPS56637 OUT -> 100k SYS_3V3 PG pull-up; footprint Capacitor_SMD:C_1206_3216Metric -> Resistor_SMD:R_0603_1608Metric; symbol Device:C -> Device:R; MPN GRM31CZ71C226ME15L -> RC0603FR-07100KL; Manufacturer Murata -> Yageo
- R773: renamed from R774; value 10k internal host VBUS fault pull-up -> 43.2k 1% internal host VBUS 0.61A ILIM; MPN RC0603FR-0710KL -> RC0603FR-0743K2L
- R774: renamed from C794; value 1u internal host VBUS switch input -> 10k internal host VBUS fault pull-up; footprint Capacitor_SMD:C_0805_2012Metric -> Resistor_SMD:R_0603_1608Metric; symbol Device:C -> Device:R; MPN GRM188R71A105KA61D -> RC0603FR-0710KL; Manufacturer Murata -> Yageo
- R775: renamed from C831; value 100n TPS3897 VCC bypass -> 10k internal host VBUS valid pull-up; footprint Capacitor_SMD:C_0603_1608Metric -> Resistor_SMD:R_0603_1608Metric; symbol Device:C -> Device:R; MPN GRM188R71A104KA01D -> RC0603FR-0710KL; Manufacturer Murata -> Yageo
- R776: renamed from C832; value 1u PCIe endpoint switch input -> 100k PCIe endpoint rail fail-low; footprint Capacitor_SMD:C_0805_2012Metric -> Resistor_SMD:R_0603_1608Metric; symbol Device:C -> Device:R; MPN GRM188R60J105KA01D -> RC0603FR-07100KL; Manufacturer Murata -> Yageo
- R777: renamed from R778; value 10.0k 1% VBUS sense bottom divider -> 78.7k 1% VBUS sense top divider; MPN RC0603FR-0710KL -> RC0603FR-0778K7L
- R778: renamed from TP13; value Internal USB VBUS test -> 10.0k 1% VBUS sense bottom divider; footprint TestPoint:TestPoint_Pad_D1.0mm -> Resistor_SMD:R_0603_1608Metric; symbol Connector:TestPoint -> Device:R; MPN (none) -> RC0603FR-0710KL; Manufacturer (none) -> Yageo; ProcurementClass PCB copper test feature -> (none); now in the parts list
- RS750: renamed from C750; value 68u 50V hybrid input bulk -> 15mOhm 1% 1W; 3.33A output current limit; footprint Capacitor_SMD:CP_Elec_8x10 -> Resistor_SMD:R_1206_3216Metric; symbol Device:C_Polarized -> Device:R; MPN EEHZA1H680P -> ERJ8BWFR015V
- U773: renamed from C834; value 47u 6.3V PCIe endpoint rail bulk -> TPS56637RPAR VSYS -> PCIE_3V3_IN (3.32V, 6A class, dedicated endpoint rail); footprint Capacitor_SMD:C_1206_3216Metric -> ducktop2:Texas_RPA0010A_VQFN-HR-10_3x3mm; symbol Device:C -> TPS56637:TPS56637; MPN GRM32ER60J476ME20L -> TPS56637RPAR; Manufacturer Murata -> Texas Instruments
- renumbered C41 to C40, C45 to C44, C790 to C46, C792 to C48, C587 to C586, C67 to C66, C586 to C67, C752 to C751, C755 to C754, C757 to C756, C760 to C759, C761 to C760, C766 to C765
Connections:
- net BUCK33_BOOT: now also C47.1, U7.7 (BOOT); no longer C45.7 (BOOT), C791.1
- net BUCK33_EN: now also R770.2, R771.1, U7.1 (EN); no longer C45.1 (EN), R44.2, R770.1
- net BUCK33_FB: now also R43.2, R44.1, U7.2 (FB); no longer C45.2 (FB), L5.2, R43.1
- net BUCK33_SW: now also C47.2, L5.1, U7.6 (SW); no longer C45.6 (SW), C47.1, C791.2
- net BUCK5_BOOT: now also C43.1; no longer C42.1
- net BUCK5_EN: now also R42.2, R45.1; no longer R41.2, R42.1
- net BUCK5_FB: now also R40.2, R41.1; no longer L4.2, R40.1
- net BUCK5_SW: now also C43.2, L4.1; no longer C42.2, C43.1
- net GND: now also C42.2, C45.2, C764.2, C767.2, C768.2, C769.2, C791.2, C792.2, C831.2, R41.2, R44.2, R45.2, R754.2, R761.2, R767.2, R771.2, R773.2, R778.2, U773.10 (MODE), U773.3 (AGND), U773.9 (PGND), C776.2, C777.2, C778.2, C782.2, C783.2, C833.2, C834.2, Q750.2 (S), R786.2, R788.2, U7.10 (MODE), U7.3 (AGND), U7.9 (PGND), U769.3 (GND), U770.2 (GND), U771.2 (GND); no longer C45.10 (MODE), C45.3 (AGND), C45.9 (PGND), D1824.2 (Pin_2), R40.2, R42.2, R43.2, R46.2, R753.2, R755.2, R759.2, R764.2, R765.2, R766.2, R768.3 (GND), R770.2, R772.2, R774.2, R775.2, R777.2, RS750.2, U773.2
- net INTERNAL_USB_VBUS: now also C830.1, R777.1, TP13.1, U770.6 (OUT); no longer C794.1, C831.1, R769.6 (OUT), R778.1
- net INTERNAL_USB_VBUS_FAULT_N: now also R774.2, U770.4 (~{FAULT}); no longer R769.4 (~{FAULT}), R773.2
- net INTERNAL_USB_VBUS_ILIM: now also R773.1, U770.5 (ILIM); no longer R769.5 (ILIM)
- net INTERNAL_USB_VBUS_SENSE: now also R777.2, R778.1, U771.3 (SENSE); no longer C830.3 (SENSE), C831.2, R777.1
- net INTERNAL_USB_VBUS_VALID: now also R775.2, U771.4 (SENSE_OUT); no longer C830.4 (SENSE_OUT)
- net MCU_3V3: now also C793.1, C831.1, D1824.1 (K), R46.1, R768.1, R772.1, R774.1, R789.1, U769.5 (VCC), U771.1 (ENABLE), U771.6 (VCC); no longer C830.1 (ENABLE), C830.6 (VCC), R45.1, R767.1, R768.5 (VCC), R771.1, R773.1
- net MU12_BOOT1: now also C765.1; no longer C764.1
- net MU12_BOOT2: now also C766.1; no longer C765.1
- net MU12_COMP: now also C772.1, R755.1; no longer C771.1, R754.1
- net MU12_COMP_RC: now also C771.1, R755.2; no longer R754.2, R755.1
- net MU12_DITH: now also C767.1; no longer R756.1
- net MU12_EN_UVLO: now also C773.1, R759.2, Q750.3 (D); no longer C773.3 (D), R758.2, R759.1
- net MU12_EXTVCC: now also R758.2; no longer R757.2
- net MU12_FB: now also R753.2, R754.1; no longer R752.2, R753.1
- net MU12_FB_TOP: now also R752.2, R753.1; no longer C770.2, R752.1
- net MU12_FORCE_OFF: now also R761.1, R766.2, Q750.1 (G); no longer C773.1 (G), R761.2
- net MU12_FSW: now also R756.1; no longer C772.1
- net MU12_ISN: now also C770.2; no longer R750.2
- net MU12_ISP: now also C770.1, R750.2; no longer C769.2, R751.1
- net MU12_MODE: now also R757.2; no longer C767.2
- net MU12_PRE_SENSE: now also C762.1, R750.1, RS750.1; no longer C755.1, C769.1, L750.1
- net MU12_SNUB1: now also C768.1, R764.2; no longer C766.2, R764.1
- net MU12_SNUB2: now also C769.1, R765.2; no longer C768.2, R765.1
- net MU12_SW1: now also C765.2, L750.1, R764.1; no longer C764.2, C766.1
- net MU12_SW2: now also C766.2, L750.2, R765.1; no longer C765.2, C768.1
- net MU12_VCC: now also C764.1, R758.1; no longer C763.1, C767.1
- net MU_12V: now also C763.1, R751.1, R752.1, RS750.2; no longer C762.1, C770.1, L750.2, R750.1
- net MU_12V_ENABLE: now also R767.1; no longer R766.1
- net MU_12V_PG: now also U769.2; no longer R768.2
- net MU_HOST_ACTIVE: now also R42.1, R769.1, R770.1, R776.1, R787.1, U769.4, U770.3 (EN); no longer C793.1, R41.1, R44.1, R768.4, R769.3 (EN)
- net MU_S0_HIGH: now also R768.2, U769.1; no longer R767.2, R768.1
- net PCIE_3V3: now also C834.1; no longer U773.1
- net PCIE_3V3_CT: now also C833.1; no longer C832.1
- net RTC_BAT: now also D1824.2 (A), C783.1; no longer D1824.1 (Pin_1)
- net SYS_3V3: now also C792.1, L5.2, R43.1; no longer C47.2, L5.1, R772.1, R776.1, U772.1 (VIN), U772.2 (VIN), U772.4 (VBIAS)
- net SYS_3V3_PG: now also R772.2, U7.4 (PG); no longer C45.4 (PG), R771.2
- net SYS_5V: now also C45.1, C794.1, L4.2, R40.1, TP5.1, U770.1 (IN); no longer C43.2, C779.1, L4.1, R46.1, R769.1 (IN), R774.1
- net SYS_5V_PG: now also R46.2; no longer R45.2
- net USBC1_SSTX_N: now also C67.2; no longer C66.2
- net USBC1_SSTX_P: now also C66.2; no longer C792.2
- net USBC1_SSTX_RAW_N: now also C67.1; no longer C66.1
- net USBC1_SSTX_RAW_P: now also C66.1; no longer C792.1
- net USBC2_SSTX_N: now also C587.2; no longer C586.2
- net USBC2_SSTX_P: now also C586.2; no longer C67.2
- net USBC2_SSTX_RAW_N: now also C587.1; no longer C586.1
- net USBC2_SSTX_RAW_P: now also C586.1; no longer C67.1
- net VSYS: now also C42.1, C755.1, C791.1, R759.1, R766.1, U773.8 (VIN), C776.1, C777.1, C778.1, U7.8 (VIN); no longer C45.8 (VIN), R758.1, R761.1, RS750.1
- new net BUCKPE_BOOT: C779.1, U773.7 (BOOT)
- new net BUCKPE_EN: R787.2, R788.1, U773.1 (EN)
- new net BUCKPE_FB: R785.2, R786.1, U773.2 (FB)
- new net BUCKPE_SW: C779.2, L1702.1, U773.6 (SW)
- new net PCIE_3V3_IN: C782.1, C832.1, L1702.2, R785.1, U772.1 (VIN), U772.2 (VIN), U772.4 (VBIAS)
- new net PCIE_3V3_PG: R789.2, U773.4 (PG)
- no-connect marks 135 -> 136
Other:
- moved on the sheet: C40, C41, C42, C44, C46, C48, C586, C66, C67, C751, C752, C753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
