File: 04_usb_c_io.kicad_sch (KiCad schematic)
At the start: 183 parts, among them J12 USB-C source-only data port J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, J22 USB-C source-only data port J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, J23 USB-C source-only data port J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, U1700 USB7206C-I/KDX six-port USB 3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, U1701 TPS62823DLC 3A USB7206C 1.146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, U1702 TLV803EA29 USB hub reset supe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, U1703 TPS56637RPAR VSYS to USB_PORT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, U1704 SN74LVC1G08 hub 3V3/core-PG r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, U1740 TPS2553DDBVR 1.3A USB branch, U1741 TPS25810RVCR Type-C DFP contr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, U1742 HD3SS6126RUAR USB3 orientatio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, U1743 TPD1S514-1YZR 5.9V VBUS OVP, U1745 TPD4E05U06 USB2/CC ESD, U1760 TPS2553DDBVR 1.3A USB branch, U1761 TPS25810RVCR Type-C DFP contr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, U1762 HD3SS6126RUAR USB3 orientatio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, U1763 TPD1S514-1YZR 5.9V VBUS OVP, U1765 TPD4E05U06 USB2/CC ESD, U1780 TPS2553DDBVR 1.3A USB branch, U1781 TPS25810RVCR Type-C DFP contr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, U1782 HD3SS6126RUAR USB3 orientatio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, U1783 TPD1S514-1YZR 5.9V VBUS OVP, U1785 TPD4E05U06 USB2/CC ESD, Y1700 25.000MHz 3.3V USB hub oscill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

Commit message: USB-A spare-port headers: hub DIS5 (USB3) + DIS6 (USB2)
Wire the hub's previously-strapped spare DIS5/DIS6 ports to two internal
USB-A receptacles on the left edge:
- J24 USB 3.0 Type-A (XKB U231-091N-4BLRA00-S): hub DIS5 D+/D- via
  USBLC6-2P6 (U1801), SuperSpeed lanes (pins 83/84/86/87) via TPD4E05U06
  (U1802), SSTX through 100n C0G series AC caps (C1852/C1853)
- J25 USB 2.0 Type-A (GCT USB1046): hub DIS6 D+/D- via USBLC6-2P6 (U1804)
- VBUS per port from USB_PORT_5V via TPS2553 (U1800/U1803) with 20k ILIM,
  gated by INTERNAL_USB_VBUS_VALID; 10u+100n bulk/HF cap each
Remove the four 0R disable straps (R1730-R1733); new USB3_A 9-pin symbol
+ sym-lib-table registration. ERC: 0 errors.
Parts:
- removed C1717: 100n hub reset-gate bypass, Capacitor_SMD:C_0603_1608Metric, symbol Device:C
- removed C1817: 100n USB7206C VDD33 local, Capacitor_SMD:C_0603_1608Metric, symbol Device:C
- removed C1836: 1n USB7206C VDD33 HF, Capacitor_SMD:C_0402_1005Metric, symbol Device:C
- removed R1730, R1731, R1732, R1733: 0R unused-port disable strap to 3V3, Resistor_SMD:R_0603_1608Metric, symbol Device:R
- removed Y1700: 25.000MHz 3.3V USB hub oscillator, Oscillator:Oscillator_SMD_Abracon_ASDMB-4Pin_2.5x2.0mm, symbol Oscillator:ASDMB-xxxMHz
- added C1726: 100n USB 3.2 TX AC coupling, Capacitor_SMD:C_0402_1005Metric, symbol Device:C
- added C1816: 100n USB7206C VDD33 local, Capacitor_SMD:C_0603_1608Metric, symbol Device:C
- added C1835: 1n USB7206C VDD33 HF, Capacitor_SMD:C_0402_1005Metric, symbol Device:C
- added C1850: 10u 10V USB3-A VBUS bulk, Capacitor_SMD:C_1206_3216Metric, symbol Device:C
- added C1851: 100n USB3-A VBUS HF, Capacitor_SMD:C_0603_1608Metric, symbol Device:C
- added C1852: 100n C0G USB3-A SSTX+ series AC, Capacitor_SMD:C_0402_1005Metric, symbol Device:C
- added C1853: 100n C0G USB3-A SSTX- series AC, Capacitor_SMD:C_0402_1005Metric, symbol Device:C
- added C1854: 10u 10V USB2-A VBUS bulk, Capacitor_SMD:C_1206_3216Metric, symbol Device:C
- added C1855: 100n USB2-A VBUS HF, Capacitor_SMD:C_0603_1608Metric, symbol Device:C
- added J24: USB 3.0 Type-A internal header (hub DIS5), Connector_USB:USB_A_Receptacle_XKB_U231-091N-4BLRA00-S, symbol USB3_A:USB3_A
- added J25: USB 2.0 Type-A internal header (hub DIS6), Connector_USB:USB_A_Receptacle_GCT_USB1046, symbol Connector:USB_A
- added R1780, R1850, R1851: 20.0k 1% TPS2553 1.3A ILIM, Resistor_SMD:R_0603_1608Metric, symbol Device:R
- added U1781: TPS25810RVCR Type-C DFP controller, Package_DFN_QFN:Texas_RVC0020A_WQFN-20-1EP_3x4mm_P0.5mm_EP1.6x2.6mm, symbol Interface_USB:TPS25810RVC
- added U1800: TPS2553DDBVR USB3-A VBUS branch 1.3A, Package_TO_SOT_SMD:SOT-23-6, symbol TPS2553D:TPS2553D
- added U1801: USBLC6-2P6 USB3-A D+/D- ESD, Package_TO_SOT_SMD:SOT-666, symbol Power_Protection:USBLC6-2P6
- added U1802: TPD4E05U06 USB3-A SuperSpeed ESD, Package_SON:USON-10_2.5x1.0mm_P0.5mm, symbol Power_Protection:TPD4EUSB30
- added U1804: USBLC6-2P6 USB2-A D+/D- ESD, Package_TO_SOT_SMD:SOT-666, symbol Power_Protection:USBLC6-2P6
- C1717: renamed from C1835; value 1n USB7206C VDD33 HF -> 100n hub reset-gate bypass; footprint Capacitor_SMD:C_0402_1005Metric -> Capacitor_SMD:C_0603_1608Metric; MPN GRM155R71H102KA01D -> GRM188R71H104KA93D
- C1817: renamed from U1781; value TPS25810RVCR Type-C DFP controller -> 100n USB7206C VDD33 local; footprint Package_DFN_QFN:Texas_RVC0020A_WQFN-20-1EP_3x4mm_P0.5mm_EP1.6x2.6mm -> Capacitor_SMD:C_0603_1608Metric; symbol Interface_USB:TPS25810RVC -> Device:C; MPN TPS25810RVCR -> GRM188R71H104KA93D; Manufacturer Texas Instruments -> Murata
- C1836: renamed from R1780; value 20.0k 1% TPS2553 1.3A ILIM -> 1n USB7206C VDD33 HF; footprint Resistor_SMD:R_0603_1608Metric -> Capacitor_SMD:C_0402_1005Metric; symbol Device:R -> Device:C; MPN RC0603FR-0720KL -> GRM155R71H102KA01D; Manufacturer Yageo -> Murata
- U1803: renamed from C1726; value 100n USB 3.2 TX AC coupling -> TPS2553DDBVR USB2-A VBUS branch 1.3A; footprint Capacitor_SMD:C_0402_1005Metric -> Package_TO_SOT_SMD:SOT-23-6; symbol Device:C -> TPS2553D:TPS2553D; MPN GRM155R71C104KA88D -> TPS2553DDBVR; Manufacturer Murata -> Texas Instruments
- Y1700: renamed from C1816; value 100n USB7206C VDD33 local -> 25.000MHz 3.3V USB hub oscillator; footprint Capacitor_SMD:C_0603_1608Metric -> Oscillator:Oscillator_SMD_Abracon_ASDMB-4Pin_2.5x2.0mm; symbol Device:C -> Oscillator:ASDMB-xxxMHz; MPN GRM188R71H104KA93D -> ASDMB-25.000MHZ-LC-T; Manufacturer Murata -> Abracon
Connections:
- net GND: now also C1817.2, U1803.2 (GND), C1816.2, C1835.2, C1850.2, C1851.2, C1854.2, C1855.2, J24.4 (GND), J24.7 (GND_DRAIN), J25.4 (GND), J25.SH (Shield), R1780.2, R1850.2, R1851.2, U1781.12 (GND), U1781.21 (GND), U1781.7 (CHG), U1781.8 (CHG_HI), U1800.2 (GND), U1801.2 (GND), U1801.5 (VBUS), U1802.3 (GND), U1802.8 (GND), U1804.2 (GND), U1804.5 (VBUS); no longer C1817.12 (GND), C1817.21 (GND), C1817.7 (CHG), C1817.8 (CHG_HI)
- net HUB_CLK: now also Y1700.3 (Out)
- net HUB_DIS5_DM: now also J24.2 (D-), U1801.3 (I/O2), U1801.4 (I/O2)
- net HUB_DIS5_DP: now also J24.3 (D+), U1801.1 (I/O1), U1801.6 (I/O1)
- net HUB_DIS6_DM: now also J25.2 (D-), U1804.3 (I/O2), U1804.4 (I/O2)
- net HUB_DIS6_DP: now also J25.3 (D+), U1804.1 (I/O1), U1804.6 (I/O1)
- net HUB_DS4_SSTX_P: now also C1726.2; no longer U1803.2
- net HUB_DS4_TX_RAW_P: now also C1726.1; no longer U1803.1
- net HUB_PRT_CTL2: now also U1781.1 (~{FAULT}), U1781.6 (EN); no longer C1817.1 (~{FAULT}), C1817.6 (EN)
- net INTERNAL_USB_VBUS_VALID: now also U1803.3 (EN), U1800.3 (EN)
- net J22_5V_PRE: now also U1781.2 (IN1), U1781.3 (IN1), U1781.4 (IN2); no longer C1817.2 (IN1), C1817.3 (IN1), C1817.4 (IN2)
- net J22_CC1: now also U1781.11 (CC1); no longer C1817.11 (CC1)
- net J22_CC2: now also U1781.13 (CC2); no longer C1817.13 (CC2)
- net J22_ILIM: now also R1780.1; no longer C1836.1
- net J22_POL_N: now also U1781.18 (~{POL}); no longer C1817.18 (~{POL})
- net J22_REF: now also U1781.10 (REF); no longer C1817.10 (REF)
- net J22_REF_RTN: now also U1781.9 (REF_RTN); no longer C1817.9 (REF_RTN)
- net J22_VBUS_SYS: now also U1781.14 (OUT), U1781.15 (OUT); no longer C1817.14 (OUT), C1817.15 (OUT)
- net SYS_3V3: now also C1817.1, C1836.1, Y1700.4 (VDD), C1816.1, C1835.1, U1781.5 (AUX); no longer C1817.5 (AUX)
- net USB_PORT_5V: now also U1803.1 (IN), U1800.1 (IN)
- new net HUB_DIS5_RX_N: J24.5 (StdA_SSRX-), U1802.5 (D2-)
- new net HUB_DIS5_RX_P: J24.6 (StdA_SSRX+), U1802.4 (D2+)
- new net HUB_DIS5_TX_N: C1853.1, U1802.2 (D1-)
- new net HUB_DIS5_TX_P: C1852.1, U1802.1 (D1+)
- new net J24_5V_PRE: C1850.1, C1851.1, J24.1 (VBUS), U1800.6 (OUT)
- new net J24_ILIM: R1850.1, U1800.5 (ILIM)
- new net J24_SSTX_N: C1853.2, J24.8 (StdA_SSTX-)
- new net J24_SSTX_P: C1852.2, J24.9 (StdA_SSTX+)
- new net J25_5V_PRE: C1854.1, C1855.1, J25.1 (VBUS), U1803.6 (OUT)
- new net J25_ILIM: R1851.1, U1803.5 (ILIM)
- no-connect marks 120 -> 126
Other:
- note added: "== Internal USB-A spare ports: hub DIS5 (USB3) + DIS6 (USB2) =="
- moved on the sheet: C1717
