File: 16_gigabit_ethernet.kicad_sch (KiCad schematic)
At the start: 29 parts, among them J500 JXD1-1022NL recessed 1GbE RJ45, U500 RTL8111H-CG-RH PCIe Gigabit E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, U501 D3V3XA4B10LP-7 four-channel 0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, U502 D3V3XA4B10LP-7 four-channel 0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, Y500 ECS-250-8-33-AGN-TR 25MHz 8pF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

Commit message: Stamp generation-time BOM catalog; close 378 procurement gaps
Parts:
- C504, C505, C506, C507, C508, C509, C510, C511, C513: MPN (none) -> GRM155R71C104KA88D; Manufacturer (none) -> Murata
- C512: MPN (none) -> GRM31CR71E106KA12L; Manufacturer (none) -> Murata
- C515, C516: MPN (none) -> GRM1555C1H120JA01; Manufacturer (none) -> Murata
- R500: MPN (none) -> RC0402FR-071ML; Manufacturer (none) -> Yageo
- R502, R503: MPN (none) -> RC0402FR-0710KL; Manufacturer (none) -> Yageo
- R504, R505: MPN (none) -> RC0402FR-07470RL; Manufacturer (none) -> Yageo
Changed lines of the file:
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@@
   (property "Footprint" "Capacitor_SMD:C_0402_1005Metric" (at 20.32 137.16 0) (effects (font (size 1.27 1.27)) (hide yes)))
   (property "Datasheet" "" (at 20.32 137.16 0) (effects (font (size 1.27 1.27)) (hide yes)))
+  (property "Manufacturer" "Murata" (at 20.32 137.16 0) (effects (font (size 1.27 1.27)) (hide yes)))
+  (property "MPN" "GRM155R71C104KA88D" (at 20.32 137.16 0) (effects (font (size 1.27 1.27)) (hide yes)))
   (pin "1")
   (pin "2")
@@
   (property "Footprint" "Capacitor_SMD:C_0402_1005Metric" (at 20.32 149.86 0) (effects (font (size 1.27 1.27)) (hide yes)))
   (property "Datasheet" "" (at 20.32 149.86 0) (effects (font (size 1.27 1.27)) (hide yes)))
+  (property "Manufacturer" "Murata" (at 20.32 149.86 0) (effects (font (size 1.27 1.27)) (hide yes)))
+  (property "MPN" "GRM155R71C104KA88D" (at 20.32 149.86 0) (effects (font (size 1.27 1.27)) (hide yes)))
   (pin "1")
   (pin "2")
@@
   (property "Footprint" "Capacitor_SMD:C_0402_1005Metric" (at 20.32 162.56 0) (effects (font (size 1.27 1.27)) (hide yes)))
   (property "Datasheet" "" (at 20.32 162.56 0) (effects (font (size 1.27 1.27)) (hide yes)))
+  (property "Manufacturer" "Murata" (at 20.32 162.56 0) (effects (font (size 1.27 1.27)) (hide yes)))
+  (property "MPN" "GRM155R71C104KA88D" (at 20.32 162.56 0) (effects (font (size 1.27 1.27)) (hide yes)))
   (pin "1")
   (pin "2")
@@
   (property "Footprint" "Capacitor_SMD:C_0402_1005Metric" (at 129.54 137.16 0) (effects (font (size 1.27 1.27)) (hide yes)))
   (property "Datasheet" "" (at 129.54 137.16 0) (effects (font (size 1.27 1.27)) (hide yes)))
+  (property "Manufacturer" "Murata" (at 129.54 137.16 0) (effects (font (size 1.27 1.27)) (hide yes)))
+  (property "MPN" "GRM155R71C104KA88D" (at 129.54 137.16 0) (effects (font (size 1.27 1.27)) (hide yes)))
   (pin "1")
   (pin "2")
@@
   (property "Footprint" "Capacitor_SMD:C_0402_1005Metric" (at 129.54 149.86 0) (effects (font (size 1.27 1.27)) (hide yes)))
   (property "Datasheet" "" (at 129.54 149.86 0) (effects (font (size 1.27 1.27)) (hide yes)))
+  (property "Manufacturer" "Murata" (at 129.54 149.86 0) (effects (font (size 1.27 1.27)) (hide yes)))
+  (property "MPN" "GRM155R71C104KA88D" (at 129.54 149.86 0) (effects (font (size 1.27 1.27)) (hide yes)))
   (pin "1")
   (pin "2")
@@
   (property "Footprint" "Capacitor_SMD:C_0402_1005Metric" (at 129.54 162.56 0) (effects (font (size 1.27 1.27)) (hide yes)))
   (property "Datasheet" "" (at 129.54 162.56 0) (effects (font (size 1.27 1.27)) (hide yes)))
+  (property "Manufacturer" "Murata" (at 129.54 162.56 0) (effects (font (size 1.27 1.27)) (hide yes)))
+  (property "MPN" "GRM155R71C104KA88D" (at 129.54 162.56 0) (effects (font (size 1.27 1.27)) (hide yes)))
   (pin "1")
   (pin "2")
@@
   (property "Footprint" "Capacitor_SMD:C_0402_1005Metric" (at 129.54 175.26 0) (effects (font (size 1.27 1.27)) (hide yes)))
   (property "Datasheet" "" (at 129.54 175.26 0) (effects (font (size 1.27 1.27)) (hide yes)))
+  (property "Manufacturer" "Murata" (at 129.54 175.26 0) (effects (font (size 1.27 1.27)) (hide yes)))
+  (property "MPN" "GRM155R71C104KA88D" (at 129.54 175.26 0) (effects (font (size 1.27 1.27)) (hide yes)))
   (pin "1")
   (pin "2")
@@
   (property "Footprint" "Capacitor_SMD:C_0402_1005Metric" (at 129.54 187.96 0) (effects (font (size 1.27 1.27)) (hide yes)))
   (property "Datasheet" "" (at 129.54 187.96 0) (effects (font (size 1.27 1.27)) (hide yes)))
+  (property "Manufacturer" "Murata" (at 129.54 187.96 0) (effects (font (size 1.27 1.27)) (hide yes)))
+  (property "MPN" "GRM155R71C104KA88D" (at 129.54 187.96 0) (effects (font (size 1.27 1.27)) (hide yes)))
   (pin "1")
   (pin "2")
@@
   (property "Footprint" "Capacitor_SMD:C_1206_3216Metric" (at 129.54 200.66 0) (effects (font (size 1.27 1.27)) (hide yes)))
   (property "Datasheet" "" (at 129.54 200.66 0) (effects (font (size 1.27 1.27)) (hide yes)))
+  (property "Manufacturer" "Murata" (at 129.54 200.66 0) (effects (font (size 1.27 1.27)) (hide yes)))
+  (property "MPN" "GRM31CR71E106KA12L" (at 129.54 200.66 0) (effects (font (size 1.27 1.27)) (hide yes)))
   (pin "1")
   (pin "2")
@@
   (property "Footprint" "Resistor_SMD:R_0402_1005Metric" (at 20.32 200.66 0) (effects (font (size 1.27 1.27)) (hide yes)))
   (property "Datasheet" "" (at 20.32 200.66 0) (effects (font (size 1.27 1.27)) (hide yes)))
+  (property "Manufacturer" "Yageo" (at 20.32 200.66 0) (effects (font (size 1.27 1.27)) (hide yes)))
+  (property "MPN" "RC0402FR-0710KL" (at 20.32 200.66 0) (effects (font (size 1.27 1.27)) (hide yes)))
   (pin "1")
   (pin "2")
@@
   (property "Footprint" "Resistor_SMD:R_0402_1005Metric" (at 20.32 213.36 0) (effects (font (size 1.27 1.27)) (hide yes)))
   (property "Datasheet" "" (at 20.32 213.36 0) (effects (font (size 1.27 1.27)) (hide yes)))
+  (property "Manufacturer" "Yageo" (at 20.32 213.36 0) (effects (font (size 1.27 1.27)) (hide yes)))
+  (property "MPN" "RC0402FR-0710KL" (at 20.32 213.36 0) (effects (font (size 1.27 1.27)) (hide yes)))
   (pin "1")
   (pin "2")
@@
   (property "Footprint" "Resistor_SMD:R_0402_1005Metric" (at 149.86 271.78 0) (effects (font (size 1.27 1.27)) (hide yes)))
   (property "Datasheet" "" (at 149.86 271.78 0) (effects (font (size 1.27 1.27)) (hide yes)))
+  (property "Manufacturer" "Yageo" (at 149.86 271.78 0) (effects (font (size 1.27 1.27)) (hide yes)))
+  (property "MPN" "RC0402FR-071ML" (at 149.86 271.78 0) (effects (font (size 1.27 1.27)) (hide yes)))
   (pin "1")
   (pin "2")
@@
   (property "Footprint" "Capacitor_SMD:C_0402_1005Metric" (at 20.32 266.7 0) (effects (font (size 1.27 1.27)) (hide yes)))
   (property "Datasheet" "" (at 20.32 266.7 0) (effects (font (size 1.27 1.27)) (hide yes)))
+  (property "Manufacturer" "Murata" (at 20.32 266.7 0) (effects (font (size 1.27 1.27)) (hide yes)))
+  (property "MPN" "GRM1555C1H120JA01" (at 20.32 266.7 0) (effects (font (size 1.27 1.27)) (hide yes)))
   (pin "1")
   (pin "2")
@@
   (property "Footprint" "Capacitor_SMD:C_0402_1005Metric" (at 20.32 279.4 0) (effects (font (size 1.27 1.27)) (hide yes)))
   (property "Datasheet" "" (at 20.32 279.4 0) (effects (font (size 1.27 1.27)) (hide yes)))
+  (property "Manufacturer" "Murata" (at 20.32 279.4 0) (effects (font (size 1.27 1.27)) (hide yes)))
+  (property "MPN" "GRM1555C1H120JA01" (at 20.32 279.4 0) (effects (font (size 1.27 1.27)) (hide yes)))
   (pin "1")
   (pin "2")
@@
   (property "Footprint" "Capacitor_SMD:C_0402_1005Metric" (at 519.43 243.84 0) (effects (font (size 1.27 1.27)) (hide yes)))
   (property "Datasheet" "" (at 519.43 243.84 0) (effects (font (size 1.27 1.27)) (hide yes)))
+  (property "Manufacturer" "Murata" (at 519.43 243.84 0) (effects (font (size 1.27 1.27)) (hide yes)))
+  (property "MPN" "GRM155R71C104KA88D" (at 519.43 243.84 0) (effects (font (size 1.27 1.27)) (hide yes)))
   (pin "1")
   (pin "2")
@@
   (property "Footprint" "Resistor_SMD:R_0402_1005Metric" (at 570.23 256.54 0) (effects (font (size 1.27 1.27)) (hide yes)))
   (property "Datasheet" "" (at 570.23 256.54 0) (effects (font (size 1.27 1.27)) (hide yes)))
+  (property "Manufacturer" "Yageo" (at 570.23 256.54 0) (effects (font (size 1.27 1.27)) (hide yes)))
+  (property "MPN" "RC0402FR-07470RL" (at 570.23 256.54 0) (effects (font (size 1.27 1.27)) (hide yes)))
   (pin "1")
   (pin "2")
@@
   (property "Footprint" "Resistor_SMD:R_0402_1005Metric" (at 570.23 269.24 0) (effects (font (size 1.27 1.27)) (hide yes)))
   (property "Datasheet" "" (at 570.23 269.24 0) (effects (font (size 1.27 1.27)) (hide yes)))
-  (pin "1")
-  (pin "2")
+  (property "Manufacturer" "Yageo" (at 570.23 269.24 0) (effects (font (size 1.27 1.27)) (hide yes)))
+  (property "MPN" "RC0402FR-07470RL" (at 570.23 269.24 0) (effects (font (size 1.27 1.27)) (hide yes)))
+  (pin "1")
+  (pin "2")
