File: 05_power_inputs.kicad_sch (KiCad schematic)
At the start: 21 parts, among them J21 USB-C PD input 1, J22 USB-C PD input 2, J23 USB-C PD input 3, U41 CH224K 15V sink 1, U42 CH224K 15V sink 2, U43 CH224K 15V sink 3

Commit message: Publish the current Ducktop2 design
Parts:
- removed U41: CH224K 15V sink 1, Package_SO:SSOP-10-1EP_3.9x4.9mm_P1mm_EP2.1x3.3mm, symbol Interface_USB:CH224K
- removed U42: CH224K 15V sink 2, Package_SO:SSOP-10-1EP_3.9x4.9mm_P1mm_EP2.1x3.3mm, symbol Interface_USB:CH224K
- removed U43: CH224K 15V sink 3, Package_SO:SSOP-10-1EP_3.9x4.9mm_P1mm_EP2.1x3.3mm, symbol Interface_USB:CH224K
- added C730, C731, C732, C733, C734, C735: 100n 50V selector local, Capacitor_SMD:C_0603_1608Metric, symbol Device:C
- added C736: 10u 25V selected-PD output, Capacitor_SMD:C_1206_3216Metric, symbol Device:C
- added C737: 100u 35V hybrid selected-PD hold-up, Capacitor_SMD:CP_Elec_6.3x5.8, symbol Device:C_Polarized
- added C800, C810, C820: 1u 50V PD eFuse input, Capacitor_SMD:C_0805_2012Metric, symbol Device:C
- added C801, C811, C821: 100n 50V PD eFuse input HF, Capacitor_SMD:C_0603_1608Metric, symbol Device:C
- added C802, C812, C822: 10u 50V PD eFuse output, Capacitor_SMD:C_1206_3216Metric, symbol Device:C
- added C803, C813, C823: 22n PD eFuse dVdT, Capacitor_SMD:C_0402_1005Metric, symbol Device:C
- added Q15, Q16, Q17, Q18, Q19, Q20: SiSS4409DN 40V reverse-blocking PMOS, Package_SO:Vishay_PowerPAK_1212-8_Single, symbol Q_PMOS_1G_234S_5D:Q_PMOS_1G_234S_5D
- added R123, R133, R143: 100R CH224A SCL series damping, Resistor_SMD:R_0603_1608Metric, symbol Device:R
- added R124, R134, R144: 100R CH224A SDA series damping, Resistor_SMD:R_0603_1608Metric, symbol Device:R
- added R720, R723, R726: 1.00M 0.1% 15V UV top, Resistor_SMD:R_0603_1608Metric, symbol Device:R
- added R721, R724, R727: 19.6k 0.1% 15V window middle, Resistor_SMD:R_0603_1608Metric, symbol Device:R
- added R722, R725, R728: 63.4k 0.1% 15V OV bottom, Resistor_SMD:R_0603_1608Metric, symbol Device:R
- added R736, R737, R738: 10k VALID open-drain pull-up, Resistor_SMD:R_0603_1608Metric, symbol Device:R
- added R800, R810, R820: 887k 0.1% PD eFuse UV/OV top, Resistor_SMD:R_0603_1608Metric, symbol Device:R
- added R801, R811, R821: 27.4k 0.1% PD eFuse UV/OV middle, Resistor_SMD:R_0603_1608Metric, symbol Device:R
- added R802, R812, R822: 68.1k 0.1% PD eFuse UV/OV bottom, Resistor_SMD:R_0603_1608Metric, symbol Device:R
- added R803, R813, R823: 6.04k 1% PD eFuse 2.98A ILIM, Resistor_SMD:R_0603_1608Metric, symbol Device:R
- added R804, R814, R824: 47k PD eFuse SHDN default-off pulldown, Resistor_SMD:R_0603_1608Metric, symbol Device:R
- added R805, R815, R825: 10k PD path-enable series, Resistor_SMD:R_0603_1608Metric, symbol Device:R
- added R806, R816, R826: 10k PD eFuse FLT pull-up, Resistor_SMD:R_0603_1608Metric, symbol Device:R
- added U123: TPD4E05U06 CC ESD port 1, Package_SON:USON-10_2.5x1.0mm_P0.5mm, symbol Power_Protection:TPD4E05U06DQA
- added U133: TPD4E05U06 CC ESD port 2, Package_SON:USON-10_2.5x1.0mm_P0.5mm, symbol Power_Protection:TPD4E05U06DQA
- added U14: LTC4417IGN#PBF three-input PD selector, Package_SO:SSOP-24_3.9x8.7mm_P0.635mm, symbol Power_Management:LTC4417CGN
- added U143: TPD4E05U06 CC ESD port 3, Package_SON:USON-10_2.5x1.0mm_P0.5mm, symbol Power_Protection:TPD4E05U06DQA
- added U41: CH224A 15V sink 1, Package_SO:SSOP-10-1EP_3.9x4.9mm_P1mm_EP2.1x3.3mm, symbol CH224A:CH224A
- added U42: CH224A 15V sink 2, Package_SO:SSOP-10-1EP_3.9x4.9mm_P1mm_EP2.1x3.3mm, symbol CH224A:CH224A
- added U43: CH224A 15V sink 3, Package_SO:SSOP-10-1EP_3.9x4.9mm_P1mm_EP2.1x3.3mm, symbol CH224A:CH224A
- added U720: TPS26630RGER PD1 default-off 3A eFuse, Package_DFN_QFN:Texas_RGE0024H_VQFN-24-1EP_4x4mm_P0.5mm_EP2.7x2.7mm_ThermalVias, symbol Power_Management:TPS26630RGE
- added U721: TPS26630RGER PD2 default-off 3A eFuse, Package_DFN_QFN:Texas_RGE0024H_VQFN-24-1EP_4x4mm_P0.5mm_EP2.7x2.7mm_ThermalVias, symbol Power_Management:TPS26630RGE
- added U722: TPS26630RGER PD3 default-off 3A eFuse, Package_DFN_QFN:Texas_RGE0024H_VQFN-24-1EP_4x4mm_P0.5mm_EP2.7x2.7mm_ThermalVias, symbol Power_Management:TPS26630RGE
- C120, C130, C140: value 1u CH224 VDD -> 1u 50V X7R CH224A VHV; MPN (none) -> GRM21BR71H105KA12L; Manufacturer (none) -> Murata
- C121, C131, C141: value 10u port VBUS -> 1u 50V X7R port VBUS; footprint Capacitor_SMD:C_1206_3216Metric -> Capacitor_SMD:C_0805_2012Metric; MPN (none) -> GRM21BR71H105KA12L; Manufacturer (none) -> Murata
- J21, J22, J23: MPN (none) -> 105450-0101; Manufacturer (none) -> Molex
- R120, R130, R140: value 5.1k CH224 VDD feed -> 0R CH224A VHV link; MPN (none) -> RC0603JR-070RL; Manufacturer (none) -> Yageo
- R121, R131, R141: value 5.1k VBUS sense -> 0R CH224A VBUS sense link; MPN (none) -> RC0603JR-070RL; Manufacturer (none) -> Yageo
- R122, R132, R142: MPN (none) -> RC0603FR-0756KL; Manufacturer (none) -> Yageo
Connections:
- net GND: now also C730.2, C731.2, C732.2, C733.2, C734.2, C735.2, C736.2, C737.2, C800.2, C801.2, C802.2, C803.2, C810.2, C811.2, C812.2, C813.2, C820.2, C821.2, C822.2, C823.2, R722.2, R725.2, R728.2, R802.2, R803.2, R804.2, R812.2, R813.2, R814.2, R822.2, R823.2, R824.2, U123.3 (GND), U123.8 (GND), U133.3 (GND), U133.8 (GND), U14.13 (GND), U14.3 (HYS), U143.3 (GND), U143.8 (GND), U41.11 (GND), U42.11 (GND), U43.11 (GND), U720.15 (PGTH), U720.25 (GND), U720.8 (GND), U721.15 (PGTH), U721.25 (GND), U721.8 (GND), U722.15 (PGTH), U722.25 (GND), U722.8 (GND)
- net PD1_CC1: now also U123.1 (D1+), U41.7 (CC1)
- net PD1_CC2: now also U123.2 (D1-), U41.6 (CC2)
- net PD1_CFG1: now also U41.9 (CFG1)
- net PD1_CH224_VBUS_SENSE: now also U41.8 (VBUS)
- net PD2_CC1: now also U133.1 (D1+), U42.7 (CC1)
- net PD2_CC2: now also U133.2 (D1-), U42.6 (CC2)
- net PD2_CFG1: now also U42.9 (CFG1)
- net PD2_CH224_VBUS_SENSE: now also U42.8 (VBUS)
- net PD3_CC1: now also U143.1 (D1+), U43.7 (CC1)
- net PD3_CC2: now also U143.2 (D1-), U43.6 (CC2)
- net PD3_CFG1: now also U43.9 (CFG1)
- net PD3_CH224_VBUS_SENSE: now also U43.8 (VBUS)
- net PD1_CH224_VDD renamed PD1_CH224_VHV
- net PD1_CH224_VHV: now also U41.1 (VHV)
- net PD2_CH224_VDD renamed PD2_CH224_VHV
- net PD2_CH224_VHV: now also U42.1 (VHV)
- net PD3_CH224_VDD renamed PD3_CH224_VHV
- net PD3_CH224_VHV: now also U43.1 (VHV)
- net USB_DM1: no longer names the net of J21.A7 (D-)
- net USB_DM1: no longer J21.B7 (D-)
- net USB_DP1: no longer names the net of J21.A6 (D+)
- net USB_DP1: no longer J21.B6 (D+)
- net VBUS_PD1 renamed PD1_VBUS_RAW
- net PD1_VBUS_RAW: now also C800.1, C801.1, R800.1, U720.1 (IN), U720.2 (IN), U720.5 (IN_SYS)
- net VBUS_PD2 renamed PD2_VBUS_RAW
- net PD2_VBUS_RAW: now also C810.1, C811.1, R810.1, U721.1 (IN), U721.2 (IN), U721.5 (IN_SYS)
- net VBUS_PD3 renamed PD3_VBUS_RAW
- net PD3_VBUS_RAW: now also C820.1, C821.1, R820.1, U722.1 (IN), U722.2 (IN), U722.5 (IN_SYS)
- new net MCU_3V3: R736.1, R737.1, R738.1, R806.1, R816.1, R826.1
- new net PD1_CH224_SCL: R123.2, U41.2 (CFG2/SCL)
- new net PD1_CH224_SDA: R124.2, U41.3 (CFG3/SDA)
- new net PD1_EFUSE_DVDT: C803.1, U720.9 (dVdT)
- new net PD1_EFUSE_FAULT_N: R806.2, U720.14 (~{FLT})
- new net PD1_EFUSE_ILIM: R803.1, U720.10 (ILIM)
- new net PD1_EFUSE_OV: R801.2, R802.1, U720.7 (OVP)
- new net PD1_EFUSE_SHDN_N: R804.1, R805.2, U720.12 (~{SHDN})
- new net PD1_EFUSE_UV: R800.2, R801.1, U720.6 (UVLO)
- new net PD1_FET_COMMON: C733.1, Q15.2 (S), Q15.3 (S), Q15.4 (S), Q16.2 (S), Q16.3 (S), Q16.4 (S), U14.21 (VS1)
- new net PD1_GATE: Q15.1 (G), Q16.1 (G), U14.20 (G1)
- new net PD1_I2C_SCL: R123.1
- new net PD1_I2C_SDA: R124.1
- new net PD1_OV: R721.2, R722.1, U14.5 (OV1)
- new net PD1_PATH_EN: R805.1
- new net PD1_UV: R720.2, R721.1, U14.4 (UV1)
- new net PD1_VALID_N: R736.2, U14.10 (~{VALID1})
- new net PD1_VBUS_GATED: C730.1, C802.1, Q15.5 (D(5-8)), R720.1, U14.24 (V1), U720.17 (OUT), U720.18 (OUT)
- new net PD2_CH224_SCL: R133.2, U42.2 (CFG2/SCL)
- new net PD2_CH224_SDA: R134.2, U42.3 (CFG3/SDA)
- new net PD2_EFUSE_DVDT: C813.1, U721.9 (dVdT)
- new net PD2_EFUSE_FAULT_N: R816.2, U721.14 (~{FLT})
- new net PD2_EFUSE_ILIM: R813.1, U721.10 (ILIM)
- new net PD2_EFUSE_OV: R811.2, R812.1, U721.7 (OVP)
- new net PD2_EFUSE_SHDN_N: R814.1, R815.2, U721.12 (~{SHDN})
- new net PD2_EFUSE_UV: R810.2, R811.1, U721.6 (UVLO)
- new net PD2_FET_COMMON: C734.1, Q17.2 (S), Q17.3 (S), Q17.4 (S), Q18.2 (S), Q18.3 (S), Q18.4 (S), U14.19 (VS2)
- new net PD2_GATE: Q17.1 (G), Q18.1 (G), U14.18 (G2)
- new net PD2_I2C_SCL: R133.1
- new net PD2_I2C_SDA: R134.1
- new net PD2_OV: R724.2, R725.1, U14.7 (OV2)
- new net PD2_PATH_EN: R815.1
- new net PD2_UV: R723.2, R724.1, U14.6 (UV2)
- new net PD2_VALID_N: R737.2, U14.11 (~{VALID2})
- new net PD2_VBUS_GATED: C731.1, C812.1, Q17.5 (D(5-8)), R723.1, U14.23 (V2), U721.17 (OUT), U721.18 (OUT)
- new net PD3_CH224_SCL: R143.2, U43.2 (CFG2/SCL)
- new net PD3_CH224_SDA: R144.2, U43.3 (CFG3/SDA)
- new net PD3_EFUSE_DVDT: C823.1, U722.9 (dVdT)
- new net PD3_EFUSE_FAULT_N: R826.2, U722.14 (~{FLT})
- new net PD3_EFUSE_ILIM: R823.1, U722.10 (ILIM)
- new net PD3_EFUSE_OV: R821.2, R822.1, U722.7 (OVP)
- new net PD3_EFUSE_SHDN_N: R824.1, R825.2, U722.12 (~{SHDN})
- new net PD3_EFUSE_UV: R820.2, R821.1, U722.6 (UVLO)
- new net PD3_FET_COMMON: C735.1, Q19.2 (S), Q19.3 (S), Q19.4 (S), Q20.2 (S), Q20.3 (S), Q20.4 (S), U14.17 (VS3)
- new net PD3_GATE: Q19.1 (G), Q20.1 (G), U14.16 (G3)
- new net PD3_I2C_SCL: R143.1
- new net PD3_I2C_SDA: R144.1
- new net PD3_OV: R727.2, R728.1, U14.9 (OV3)
- new net PD3_PATH_EN: R825.1
- new net PD3_UV: R726.2, R727.1, U14.8 (UV3)
- new net PD3_VALID_N: R738.2, U14.12 (~{VALID3})
- new net PD3_VBUS_GATED: C732.1, C822.1, Q19.5 (D(5-8)), R726.1, U14.22 (V3), U722.17 (OUT), U722.18 (OUT)
- new net USB_PD_SELECTED: C736.1, C737.1, Q16.5 (D(5-8)), Q18.5 (D(5-8)), Q20.5 (D(5-8)), U14.15 (VOUT)
- no-connect marks 47 -> 105
Other:
- note added: "== J21 USB-C PD sink input 1: CH224A requests 15V and reports PDO current =="
- note added: "== J22 USB-C PD sink input 2: CH224A requests 15V and reports PDO current =="
- note added: "== J23 USB-C PD sink input 3: CH224A requests 15V and reports PDO current =="
- note added: "== U14 LTC4417IGN: qualified, prioritized selection of the three negotiated 15V inputs =="
- note added: "== USB-C power inputs: three CH224A PD sink controllers =="
- note added: "All three ports are power-only. USB D+/D- stay open because the selected source can change after arbitration."
- note added: "C737 provides low-ESR hold-up through LTC4417 break-before-make adapter switching."
- note added: "CH224A reports negotiated PDO current; LTC4417 validates, prioritizes, and reverse-isolates the three adapters."
- note added: "EN/SHDN use LTC4417 internal pull-ups; HYS is grounded; VALID1/2/3 have external 10k pull-ups to always-on MCU_3V3."
- note added: "J21: power-only PD input; CH224A D+/D- are NC; 100R-damped muxed I2C reports PDO current."
- note added: "J22: power-only PD input; CH224A D+/D- are NC; 100R-damped muxed I2C reports PDO current."
- note added: "J23: power-only PD input; CH224A D+/D- are NC; 100R-damped muxed I2C reports PDO current."
- note added: "Only a source offering the 15V PDO crosses the 6.06-6.36V AON UVLO and boots the EC; a 5V-only source leaves the laptop off."
- note added: "Priority is J21, then J22, then J23; every input must validate inside approximately 13.1V to 17.1V."
- note added: "Q15-Q20 are common-source back-to-back pairs, so inactive adapters are reverse-isolated instead of diode-ORed."
- note added: "Raw 5V attachment powers CH224A directly; CFG1=56k autonomously requests 15V without EC firmware."
- note added: "U720-U722 enforce 3A current limits and default off; EC validates CH224A PDO current before enabling exactly one path."
- note removed: "== J21 USB-C PD sink input 1: CH224K requests 15V =="
- note removed: "== J22 USB-C PD sink input 2: CH224K requests 15V =="
- note removed: "== J23 USB-C PD sink input 3: CH224K requests 15V =="
- note removed: "== USB-C power inputs: three CH224K PD sink triggers =="
- note removed: "CH224K performs USB-C PD negotiation; BQ25798 on sheet 1 is the buck-boost charger / NVDC power path."
- note removed: "Each CH224K uses resistor mode: CFG1=56k to GND requests 15V; CFG2/CFG3 are NC."
- note removed: "J21: D+/D- route to BQ25798 USB_DP1/USB_DM1 for fallback detection."
- note removed: "J22: power-only PD input; connector D+/D- are intentionally NC."
- note removed: "J23: power-only PD input; connector D+/D- are intentionally NC."
- note removed: "Only J21 carries USB2 D+/D- to BQ25798; J22/J23 are power-only charge inputs."

Commit message: Finish USB-C policy and split out radio board
Parts:
- removed C120, C130, C140: 1u 50V X7R CH224A VHV, Capacitor_SMD:C_0805_2012Metric, symbol Device:C
- removed C121, C131, C141: 1u 50V X7R port VBUS, Capacitor_SMD:C_0805_2012Metric, symbol Device:C
- removed C730, C731, C732, C733: 100n 50V selector local, Capacitor_SMD:C_0603_1608Metric, symbol Device:C
- removed C800, C810, C820: 1u 50V PD eFuse input, Capacitor_SMD:C_0805_2012Metric, symbol Device:C
- removed C801, C811, C821: 100n 50V PD eFuse input HF, Capacitor_SMD:C_0603_1608Metric, symbol Device:C
- removed C802, C812, C822: 10u 50V PD eFuse output, Capacitor_SMD:C_1206_3216Metric, symbol Device:C
- removed C803, C813, C823: 22n PD eFuse dVdT, Capacitor_SMD:C_0402_1005Metric, symbol Device:C
- removed J22: USB-C PD input 2, Connector_USB:USB_C_Receptacle_Molex_105450-0101, symbol Connector:USB_C_Receptacle
- removed J23: USB-C PD input 3, Connector_USB:USB_C_Receptacle_Molex_105450-0101, symbol Connector:USB_C_Receptacle
- removed Q19, Q20: SiSS4409DN 40V reverse-blocking PMOS, Package_SO:Vishay_PowerPAK_1212-8_Single, symbol Q_PMOS_1G_234S_5D:Q_PMOS_1G_234S_5D
- removed R120, R130, R140: 0R CH224A VHV link, Resistor_SMD:R_0603_1608Metric, symbol Device:R
- removed R121, R131, R141: 0R CH224A VBUS sense link, Resistor_SMD:R_0603_1608Metric, symbol Device:R
- removed R122, R132, R142: 56k CFG1 to GND (15V), Resistor_SMD:R_0603_1608Metric, symbol Device:R
- removed R123, R133, R143: 100R CH224A SCL series damping, Resistor_SMD:R_0603_1608Metric, symbol Device:R
- removed R124, R134, R144: 100R CH224A SDA series damping, Resistor_SMD:R_0603_1608Metric, symbol Device:R
- removed R720, R723, R726: 1.00M 0.1% 15V UV top, Resistor_SMD:R_0603_1608Metric, symbol Device:R
- removed R721, R724, R727: 19.6k 0.1% 15V window middle, Resistor_SMD:R_0603_1608Metric, symbol Device:R
- removed R722, R725, R728: 63.4k 0.1% 15V OV bottom, Resistor_SMD:R_0603_1608Metric, symbol Device:R
- removed R736, R737, R738: 10k VALID open-drain pull-up, Resistor_SMD:R_0603_1608Metric, symbol Device:R
- removed R800, R810, R820: 887k 0.1% PD eFuse UV/OV top, Resistor_SMD:R_0603_1608Metric, symbol Device:R
- removed R801, R811, R821: 27.4k 0.1% PD eFuse UV/OV middle, Resistor_SMD:R_0603_1608Metric, symbol Device:R
- removed R802, R812, R822: 68.1k 0.1% PD eFuse UV/OV bottom, Resistor_SMD:R_0603_1608Metric, symbol Device:R
- removed R803, R813, R823: 6.04k 1% PD eFuse 2.98A ILIM, Resistor_SMD:R_0603_1608Metric, symbol Device:R
- removed R804, R814, R824: 47k PD eFuse SHDN default-off pulldown, Resistor_SMD:R_0603_1608Metric, symbol Device:R
- removed R805, R815, R825: 10k PD path-enable series, Resistor_SMD:R_0603_1608Metric, symbol Device:R
- removed R806, R816, R826: 10k PD eFuse FLT pull-up, Resistor_SMD:R_0603_1608Metric, symbol Device:R
- removed U123: TPD4E05U06 CC ESD port 1, Package_SON:USON-10_2.5x1.0mm_P0.5mm, symbol Power_Protection:TPD4E05U06DQA
- removed U133: TPD4E05U06 CC ESD port 2, Package_SON:USON-10_2.5x1.0mm_P0.5mm, symbol Power_Protection:TPD4E05U06DQA
- removed U14: LTC4417IGN#PBF three-input PD selector, Package_SO:SSOP-24_3.9x8.7mm_P0.635mm, symbol Power_Management:LTC4417CGN
- removed U143: TPD4E05U06 CC ESD port 3, Package_SON:USON-10_2.5x1.0mm_P0.5mm, symbol Power_Protection:TPD4E05U06DQA
- removed U41: CH224A 15V sink 1, Package_SO:SSOP-10-1EP_3.9x4.9mm_P1mm_EP2.1x3.3mm, symbol CH224A:CH224A
- removed U42: CH224A 15V sink 2, Package_SO:SSOP-10-1EP_3.9x4.9mm_P1mm_EP2.1x3.3mm, symbol CH224A:CH224A
- removed U43: CH224A 15V sink 3, Package_SO:SSOP-10-1EP_3.9x4.9mm_P1mm_EP2.1x3.3mm, symbol CH224A:CH224A
- removed U722: TPS26630RGER PD3 default-off 3A eFuse, Package_DFN_QFN:Texas_RGE0024H_VQFN-24-1EP_4x4mm_P0.5mm_EP2.7x2.7mm_ThermalVias, symbol Power_Management:TPS26630RGE
- added C2000, C2040: 100n 100V TPD4S201 VBIAS, Capacitor_SMD:C_0805_2012Metric, symbol Device:C
- added C2001, C2041: 820n 10V TPD4S201 VPWR, Capacitor_SMD:C_0805_2012Metric, symbol Device:C
- added C2002: 100n EEPROM local, Capacitor_SMD:C_0603_1608Metric, symbol Device:C
- added C2003, C2043: 100n mux-control buffer local, Capacitor_SMD:C_0603_1608Metric, symbol Device:C
- added C2004, C2044: 10u TUSB1142 local, Capacitor_SMD:C_1206_3216Metric, symbol Device:C
- added C2005, C2006, C2007, C2008, C2045, C2046, C2047, C2048: 100n TUSB1142 VCC local, Capacitor_SMD:C_0603_1608Metric, symbol Device:C
- added C2009, C2010, C2011, C2012, C2013, C2014, C2049, C2050, C2051, C2052, C2053, C2054: 220n USB3 TX AC coupling, Capacitor_SMD:C_0402_1005Metric, symbol Device:C
- added C2015, C2055: 4.7u 25V raw VBUS; pre-attach total below 10uF, Capacitor_SMD:C_1206_3216Metric, symbol Device:C
- added C2016, C2017, C2018, C2019, C2056, C2057, C2058, C2059: 10n 50V connector VBUS HF, Capacitor_SMD:C_0402_1005Metric, symbol Device:C
- added C2020, C2060: 6.8u 25V X7R TPS25751A LDO3V3; verify >=5u effect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, Capacitor_SMD:C_1206_3216Metric, symbol Device:C
- added C2021, C2061: 10u 16V X7R TPS25751A LDO1V5; verify 4.5-12u effe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, Capacitor_SMD:C_1206_3216Metric, symbol Device:C
- added C2022, C2062: 10u TPS25751A VIN3V3, Capacitor_SMD:C_1206_3216Metric, symbol Device:C
- added C2023, C2063: 270p C0G CC1 total-capacitance component, Capacitor_SMD:C_0402_1005Metric, symbol Device:C
- added C2024, C2064: 270p C0G CC2 total-capacitance component, Capacitor_SMD:C_0402_1005Metric, symbol Device:C
- added C2025, C2026, C2065, C2066: 100u 10V PP5V source bulk, Capacitor_Tantalum_SMD:CP_EIA-7343-31_Kemet-D, symbol Device:C_Polarized
- added C2027, C2067: 10u PP5V local ceramic, Capacitor_SMD:C_1206_3216Metric, symbol Device:C
- added C2028, C2068: 68u 25V PPHV sink bulk, Capacitor_Tantalum_SMD:CP_EIA-7343-31_Kemet-D, symbol Device:C_Polarized
- added C2029, C2069: 100n 50V PPHV local, Capacitor_SMD:C_0603_1608Metric, symbol Device:C
- added C2030, C2070: 100n USB2 switch local, Capacitor_SMD:C_0603_1608Metric, symbol Device:C
- added C2080, C2090: 100n 50V eFuse input local, Capacitor_SMD:C_0603_1608Metric, symbol Device:C
- added C2081, C2091: 10u 25V eFuse output, Capacitor_SMD:C_1206_3216Metric, symbol Device:C
- added C2082, C2092: 22n eFuse dVdT, Capacitor_SMD:C_0402_1005Metric, symbol Device:C
- added C2140: 100n selector INTVCC, Capacitor_SMD:C_0603_1608Metric, symbol Device:C
- added C2141: 15n selector TMR approx 240ms, Capacitor_SMD:C_0402_1005Metric, symbol Device:C
- added C2142, C2143, C2144, C2145: 100n 50V selector local, Capacitor_SMD:C_0603_1608Metric, symbol Device:C
- added C2146: 100u 35V selected-PD hold-up, Capacitor_SMD:CP_Elec_6.3x5.8, symbol Device:C_Polarized
- added D2080, D2090: B340A eFuse output negative-transient clamp, Diode_SMD:D_SMA, symbol Device:D_Schottky
- added D2100, D2101, D2102, D2103, D2104, D2105, D2106, D2107, D2120, D2121, D2122, D2123, D2124, D2125, D2126, D2127: TPD1E0B04DPLR 0.13pF USB3 ESD, Diode_SMD:D_0201_0603Metric, symbol TPD1E0B04:TPD1E0B04
- added J11: USB-C dual-role data/PD port J11, Connector_USB:USB_C_Receptacle_Molex_105450-0101, symbol Connector:USB_C_Receptacle
- added Q2001, Q2002: 2N7002K DFP USB2 enable inverter, Package_TO_SOT_SMD:SOT-23, symbol Q_NMOS_SOT23_GSD:Q_NMOS_SOT23_GSD
- added R2000, R2040: 10k shared CC/USB2 protector FLT pull-up, Resistor_SMD:R_0603_1608Metric, symbol Device:R
- added R2001: 2.2k EEPROM SDA pull-up, Resistor_SMD:R_0603_1608Metric, symbol Device:R
- added R2002: 2.2k EEPROM SCL pull-up, Resistor_SMD:R_0603_1608Metric, symbol Device:R
- added R2003, R2043: 4.7k TCPC SDA pull-up, Resistor_SMD:R_0603_1608Metric, symbol Device:R
- added R2004, R2044: 4.7k TCPC SCL pull-up, Resistor_SMD:R_0603_1608Metric, symbol Device:R
- added R2005, R2045: 10k TCPC IRQ pull-up, Resistor_SMD:R_0603_1608Metric, symbol Device:R
- added R2006, R2046: 10k mux FLIP pull-up, Resistor_SMD:R_0603_1608Metric, symbol Device:R
- added R2007, R2047: 10k mux EN pull-up, Resistor_SMD:R_0603_1608Metric, symbol Device:R
- added R2008, R2048: 1k TUSB1142 MODE=0 strap, Resistor_SMD:R_0603_1608Metric, symbol Device:R
- added R2009, R2049: 1k TUSB1142 VIO=3V3 strap, Resistor_SMD:R_0603_1608Metric, symbol Device:R
- added R2010, R2050: 1k TUSB1142 EQCFG=0 strap, Resistor_SMD:R_0603_1608Metric, symbol Device:R
- added R2011, R2051: 1k TUSB1142 SSEQ1=0 strap, Resistor_SMD:R_0603_1608Metric, symbol Device:R
- added R2012, R2052: 10k TUSB1142 SLP_S0# pull-up, Resistor_SMD:R_0603_1608Metric, symbol Device:R
- added R2013, R2053: 100k mux FLIP input default-low, Resistor_SMD:R_0603_1608Metric, symbol Device:R
- added R2014, R2054: 100k data-attach input default-low, Resistor_SMD:R_0603_1608Metric, symbol Device:R
- added R2015: 10k I2Cc IRQ inactive pull-up, Resistor_SMD:R_0603_1608Metric, symbol Device:R
- added R2016, R2056: 100k USB2 switch default-disable pull-up, Resistor_SMD:R_0603_1608Metric, symbol Device:R
- added R2017, R2057: 0R protector FLT wired-OR link, Resistor_SMD:R_0603_1608Metric, symbol Device:R
- added R2018, R2058: 100k DFP-role input default-low, Resistor_SMD:R_0603_1608Metric, symbol Device:R
- added R2080, R2090: 887k 0.1% 15V eFuse UV/OV top, Resistor_SMD:R_0603_1608Metric, symbol Device:R
- added R2081, R2091: 27.4k 0.1% 15V eFuse UV/OV middle, Resistor_SMD:R_0603_1608Metric, symbol Device:R
- added R2082, R2092: 68.1k 0.1% 15V eFuse UV/OV bottom, Resistor_SMD:R_0603_1608Metric, symbol Device:R
- added R2083, R2093: 6.04k 1% eFuse 2.98A ILIM, Resistor_SMD:R_0603_1608Metric, symbol Device:R
- added R2084, R2094: 47k eFuse default-off pulldown, Resistor_SMD:R_0603_1608Metric, symbol Device:R
- added R2085, R2095: 10k path-enable series, Resistor_SMD:R_0603_1608Metric, symbol Device:R
- added R2086, R2096: 10k eFuse FLT pull-up, Resistor_SMD:R_0603_1608Metric, symbol Device:R
- added R2140, R2143: 1.00M 0.1% 15V UV top, Resistor_SMD:R_0603_1608Metric, symbol Device:R
- added R2141, R2144: 19.6k 0.1% 15V window middle, Resistor_SMD:R_0603_1608Metric, symbol Device:R
- added R2142, R2145: 63.4k 0.1% 15V OV bottom, Resistor_SMD:R_0603_1608Metric, symbol Device:R
- added R2146: 10k PD1 VALID pull-up, Resistor_SMD:R_0603_1608Metric, symbol Device:R
- added R2147: 10k PD2 VALID pull-up, Resistor_SMD:R_0603_1608Metric, symbol Device:R
- added U14: LTC4418IUF#PBF dual-input PD selector, ducktop2:ADI_UF20_QFN20_4x4_P0.5_EP2.45, symbol LTC4418IUF:LTC4418IUF
- added U2000, U2010: TUSB1142 USB 3.2 Gen 2 orientation redriver, Package_DFN_QFN:Texas_RNQ0040A_WQFN-40-1EP_6x4mm_P0.4mm_EP4.7x2.7mm_ThermalVias, symbol TUSB1142:TUSB1142
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Connections:
- net GND: now also U720.11 (MODE), U721.11 (MODE), C2000.2, C2001.2, C2002.2, C2003.2, C2004.2, C2005.2, C2006.2, C2007.2, C2008.2, C2015.2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; no longer R2041.2, R2042.2, R2055.2
- net MCU_3V3: now also C2022.1, C2062.1, R2000.1, R2003.1, R2004.1, R2005.1, R2040.1, R2043.1, R2044.1, R2045.1, R2086.1, R2096.1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
- net PD1_EFUSE_DVDT: now also C2082.1
- net PD1_EFUSE_FAULT_N: now also R2086.2
- net PD1_EFUSE_ILIM: now also R2083.1
- net PD1_EFUSE_OV: now also R2081.2, R2082.1
- net PD1_EFUSE_UV: now also R2080.2, R2081.1
- net PD1_I2C_SCL: now also R2004.2, U41.9 (I2Ct_SCL)
- net PD1_I2C_SDA: now also R2003.2, U41.8 (I2Ct_SDA)
- net PD1_PATH_EN: now also R2085.1
- net PD1_VALID_N: now also R2146.2, U14.9 (~{VALID1})
- net PD1_VBUS_GATED: now also C2081.1, C2142.1, D2080.1 (K), R2140.1, U14.17 (V1)
- net PD1_VBUS_RAW: now also C2015.1, C2016.1, C2017.1, C2018.1, C2019.1, U2005.4 (IN), U2005.5 (IN), U2005.6 (IN), U41.23 (VBUS_IN_(23-25)), U41.32 (VBUS_(32-33)); no longer U720.1 (IN), U720.2 (IN), U720.5 (IN_SYS)
- net PD2_EFUSE_DVDT: now also C2092.1
- net PD2_EFUSE_FAULT_N: now also R2096.2
- net PD2_EFUSE_ILIM: now also R2093.1
- net PD2_EFUSE_OV: now also R2091.2, R2092.1
- net PD2_EFUSE_UV: now also R2090.2, R2091.1
- net PD2_I2C_SCL: now also R2044.2, U42.9 (I2Ct_SCL)
- net PD2_I2C_SDA: now also R2043.2, U42.8 (I2Ct_SDA)
- net PD2_PATH_EN: now also R2095.1
- net PD2_VALID_N: now also R2147.2, U14.10 (~{VALID2})
- net PD2_VBUS_GATED: now also C2091.1, C2144.1, D2090.1 (K), R2143.1, U14.16 (V2)
- net PD2_VBUS_RAW: now also C2055.1, C2056.1, C2057.1, C2058.1, C2059.1, J11.A4 (VBUS), J11.A9 (VBUS), J11.B4 (VBUS), J11.B9 (VBUS), U2015.4 (IN), U2015.5 (IN), U2015.6 (IN)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; no longer U721.1 (IN), U721.2 (IN), U721.5 (IN_SYS)
- net USB_PD_SELECTED: now also C2146.1, U14.15 (VOUT); no longer C2042.1, R2055.1
- net PD1_RX2_N: now reaches J21.A10 (RX2-)
- net PD1_RX2_N: now also D2107.1 (IO), U2000.36 (CRX2n)
- net PD1_RX2_P: now reaches J21.A11 (RX2+)
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Other:
- note added: "== J11: USB 3.2 Gen 2 data plus USB-PD charging, side port 2 =="
- note added: "== J21: USB 3.2 Gen 2 data plus USB-PD charging, side port 1 =="
- note added: "== Two rear USB-C data/charging ports: J21 left and J11 right =="
- note added: "== U14: two-input qualified PD selector; J21 has priority over J11 =="
- note added: "Both ports carry USB 3.2 Gen 2 plus USB2 and can sink negotiated 15V or source protected default USB current."
- note added: "Firmware must reject any configuration that advertises more than default USB current and must shed optional ports on rail fault."
- note added: "Five-port source budget: 5 x 0.9A maximum advertised load = 4.5A on the dedicated 6A USB_PORT_5V rail."
- note added: "GPIO4 AND GPIO7 qualifies both host USB2 and SuperSpeed. They remain disconnected through reset, detach, and sink-only operation."
- note added: "J11: EEPROM configures DRP prefer-sink, 15V/3A sink, 5V/0.9A source, default Rp, GPIO6 FLIP, GPIO4 DFP, and GPIO7 data-attached."
- note added: "J21: EEPROM configures DRP prefer-sink, 15V/3A sink, 5V/0.9A source, default Rp, GPIO6 FLIP, GPIO4 DFP, and GPIO7 data-attached."
- note added: "LTC4418 independently validates approximately 13.1V to 17.1V and prevents either attached adapter from backfeeding the other."
- note added: "TPS25751A loads a versioned 32KB EEPROM image while powered from dead-battery VBUS; no EC is needed to obtain the first 15V contract."
- note added: "The EC reads each TPS25751A contract first, programs the BQ25798 input limit, then enables exactly one default-off TPS26630 path."
- note added: "The raw 5V attach rail stays below the Type-C pre-attach capacitance limit; large sink bulk is behind the integrated PD switch."
- note removed: "== J21 USB-C PD sink input 1: CH224A requests 15V and reports PDO current =="
- note removed: "== J22 USB-C PD sink input 2: CH224A requests 15V and reports PDO current =="
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
Commit message: Phase 2.0: convert J11/J12 to USB2-only (board split prep)
J11 and J12 lose their SuperSpeed lanes as part of the 4-board split
(no USB3 host port remains on the right side; hub DS1/DS4 become
USB2-only downstream ports).

- generate_power_inputs_sheet.py: add_dual_role_port gains usb2_only;
  J11 drops the TUSB1142 redriver, SS coupling caps, and SS ESD; SS
  connector pins become NC. PD charging (15V sink / 5V 0.9A source),
  CC, USB2 (via hub DS1 D+/D-), VBUS/PPHV/LDO protection all kept.
- generate_usb_c_io_sheet.py: add_source_port gains usb2_only; J12
  drops the HD3SS6126 mux + SS chain; hub DS1/DS4 SS pins (7/8/10/11,
  36/37/39/40) retired to NC. DS2/DS3/UP unchanged.
- verify_design_contracts.py: J11/J12 SS pins now NC, U1700 DS1/DS4 SS
  pins NC, TUSB1142/strap contracts gated on usb2_only.
- verify_schematic_closure.py: closure audit accepts NC SS pins
  (unconnected-* pseudo-nets) for J12 and the retired hub pins.
- generate_pin_review_table.py: J12 SS pins NC, U1700 retired pins NC,
  U2010 removed from required set.
- Regenerated 04_usb_c_io / 05_power_inputs / root sheets.

16 SS nets removed. Verified: schematic gate PASS (closure 1574/0,
contracts OK, ERC 0, pin review 2602/2602, generated-source identity
PASS).
Parts:
- removed C2021: 10u 16V X7R TPS25751A LDO1V5; verify 4.5-12u effe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, Capacitor_SMD:C_1206_3216Metric, symbol Device:C
- removed C2022: 10u TPS25751A VIN3V3, Capacitor_SMD:C_1206_3216Metric, symbol Device:C
- removed C2044: 10u TUSB1142 local, Capacitor_SMD:C_1206_3216Metric, symbol Device:C
- removed C2045, C2046, C2047, C2048: 100n TUSB1142 VCC local, Capacitor_SMD:C_0603_1608Metric, symbol Device:C
- removed C2049, C2050, C2051, C2052, C2053, C2054: 220n USB3 TX AC coupling, Capacitor_SMD:C_0402_1005Metric, symbol Device:C
- removed D2120, D2121, D2122, D2123, D2124, D2125, D2126, D2127: TPD1E0B04DPLR 0.13pF USB3 ESD, Diode_SMD:D_0201_0603Metric, symbol TPD1E0B04:TPD1E0B04
- removed Q15: SiSS4409DN 40V reverse-blocking PMOS, Package_SO:Vishay_PowerPAK_1212-8_Single, symbol Q_PMOS_1G_234S_5D:Q_PMOS_1G_234S_5D
- removed R2048: 1k TUSB1142 MODE=0 strap, Resistor_SMD:R_0603_1608Metric, symbol Device:R
- removed R2049: 1k TUSB1142 VIO=3V3 strap, Resistor_SMD:R_0603_1608Metric, symbol Device:R
- removed R2050: 1k TUSB1142 EQCFG=0 strap, Resistor_SMD:R_0603_1608Metric, symbol Device:R
- removed R2051: 1k TUSB1142 SSEQ1=0 strap, Resistor_SMD:R_0603_1608Metric, symbol Device:R
- removed R2052: 10k TUSB1142 SLP_S0# pull-up, Resistor_SMD:R_0603_1608Metric, symbol Device:R
- removed R2053: 100k mux FLIP input default-low, Resistor_SMD:R_0603_1608Metric, symbol Device:R
- removed R2054: 100k data-attach input default-low, Resistor_SMD:R_0603_1608Metric, symbol Device:R
- removed R2058: 100k DFP-role input default-low, Resistor_SMD:R_0603_1608Metric, symbol Device:R
- removed U2015: TVS2200 22V USB VBUS surge clamp, Package_SON:WSON-6-1EP_2x2mm_P0.65mm_EP1x1.6mm, symbol Power_Protection:TVS2200DRV
- added C2066: 100u 10V PP5V source bulk, Capacitor_Tantalum_SMD:CP_EIA-7343-31_Kemet-D, symbol Device:C_Polarized
- added D2101, D2102: TPD1E0B04DPLR 0.13pF USB3 ESD, Diode_SMD:D_0201_0603Metric, symbol TPD1E0B04:TPD1E0B04
- C2015: renamed from C2023; value 270p C0G CC1 total-capacitance component -> 4.7u 25V raw VBUS; pre-attach total below 10uF; footprint Capacitor_SMD:C_0402_1005Metric -> Capacitor_SMD:C_1206_3216Metric; MPN GRM1555C1H271JA01D -> GRM31CR71E475KA88L
- C2016: renamed from C2024; value 270p C0G CC2 total-capacitance component -> 10n 50V connector VBUS HF; MPN GRM1555C1H271JA01D -> GRM155R71H103KA88D
- C2017: renamed from C2025; value 100u 10V PP5V source bulk -> 10n 50V connector VBUS HF; footprint Capacitor_Tantalum_SMD:CP_EIA-7343-31_Kemet-D -> Capacitor_SMD:C_0402_1005Metric; symbol Device:C_Polarized -> Device:C; MPN T520D107M010ATE070 -> GRM155R71H103KA88D; Manufacturer KEMET -> Murata
- C2018: renamed from C2026; value 100u 10V PP5V source bulk -> 10n 50V connector VBUS HF; footprint Capacitor_Tantalum_SMD:CP_EIA-7343-31_Kemet-D -> Capacitor_SMD:C_0402_1005Metric; symbol Device:C_Polarized -> Device:C; MPN T520D107M010ATE070 -> GRM155R71H103KA88D; Manufacturer KEMET -> Murata
- C2019: renamed from C2027; value 10u PP5V local ceramic -> 10n 50V connector VBUS HF; footprint Capacitor_SMD:C_1206_3216Metric -> Capacitor_SMD:C_0402_1005Metric; MPN GRM31CR71A106KA01L -> GRM155R71H103KA88D
- C2020: renamed from C2028; value 68u 25V PPHV sink bulk -> 6.8u 25V X7R TPS25751A LDO3V3; verify >=5u effective; footprint Capacitor_Tantalum_SMD:CP_EIA-7343-31_Kemet-D -> Capacitor_SMD:C_1206_3216Metric; symbol Device:C_Polarized -> Device:C; MPN T521V686M025ATE050 -> GRM31CR71E685KA88L; Manufacturer KEMET -> Murata
- C2021: renamed from C2029; value 100n 50V PPHV local -> 10u 16V X7R TPS25751A LDO1V5; verify 4.5-12u effective; footprint Capacitor_SMD:C_0603_1608Metric -> Capacitor_SMD:C_1206_3216Metric; MPN GRM188R71H104KA93D -> GRM31CR71C106KA01L
- C2022: renamed from D2100; value TPD1E0B04DPLR 0.13pF USB3 ESD -> 10u TPS25751A VIN3V3; footprint Diode_SMD:D_0201_0603Metric -> Capacitor_SMD:C_1206_3216Metric; symbol TPD1E0B04:TPD1E0B04 -> Device:C; MPN TPD1E0B04DPLR -> GRM31CR71A106KA01L; Manufacturer Texas Instruments -> Murata
- C2023: renamed from D2101; value TPD1E0B04DPLR 0.13pF USB3 ESD -> 270p C0G CC1 total-capacitance component; footprint Diode_SMD:D_0201_0603Metric -> Capacitor_SMD:C_0402_1005Metric; symbol TPD1E0B04:TPD1E0B04 -> Device:C; MPN TPD1E0B04DPLR -> GRM1555C1H271JA01D; Manufacturer Texas Instruments -> Murata
- C2024: renamed from D2102; value TPD1E0B04DPLR 0.13pF USB3 ESD -> 270p C0G CC2 total-capacitance component; footprint Diode_SMD:D_0201_0603Metric -> Capacitor_SMD:C_0402_1005Metric; symbol TPD1E0B04:TPD1E0B04 -> Device:C; MPN TPD1E0B04DPLR -> GRM1555C1H271JA01D; Manufacturer Texas Instruments -> Murata
- C2025: renamed from D2103; value TPD1E0B04DPLR 0.13pF USB3 ESD -> 100u 10V PP5V source bulk; footprint Diode_SMD:D_0201_0603Metric -> Capacitor_Tantalum_SMD:CP_EIA-7343-31_Kemet-D; symbol TPD1E0B04:TPD1E0B04 -> Device:C_Polarized; MPN TPD1E0B04DPLR -> T520D107M010ATE070; Manufacturer Texas Instruments -> KEMET
- C2026: renamed from D2104; value TPD1E0B04DPLR 0.13pF USB3 ESD -> 100u 10V PP5V source bulk; footprint Diode_SMD:D_0201_0603Metric -> Capacitor_Tantalum_SMD:CP_EIA-7343-31_Kemet-D; symbol TPD1E0B04:TPD1E0B04 -> Device:C_Polarized; MPN TPD1E0B04DPLR -> T520D107M010ATE070; Manufacturer Texas Instruments -> KEMET
- C2027: renamed from D2105; value TPD1E0B04DPLR 0.13pF USB3 ESD -> 10u PP5V local ceramic; footprint Diode_SMD:D_0201_0603Metric -> Capacitor_SMD:C_1206_3216Metric; symbol TPD1E0B04:TPD1E0B04 -> Device:C; MPN TPD1E0B04DPLR -> GRM31CR71A106KA01L; Manufacturer Texas Instruments -> Murata
- C2028: renamed from D2106; value TPD1E0B04DPLR 0.13pF USB3 ESD -> 68u 25V PPHV sink bulk; footprint Diode_SMD:D_0201_0603Metric -> Capacitor_Tantalum_SMD:CP_EIA-7343-31_Kemet-D; symbol TPD1E0B04:TPD1E0B04 -> Device:C_Polarized; MPN TPD1E0B04DPLR -> T521V686M025ATE050; Manufacturer Texas Instruments -> KEMET
- C2029: renamed from D2107; value TPD1E0B04DPLR 0.13pF USB3 ESD -> 100n 50V PPHV local; footprint Diode_SMD:D_0201_0603Metric -> Capacitor_SMD:C_0603_1608Metric; symbol TPD1E0B04:TPD1E0B04 -> Device:C; MPN TPD1E0B04DPLR -> GRM188R71H104KA93D; Manufacturer Texas Instruments -> Murata
- D2100: renamed from U2005; value TVS2200 22V USB VBUS surge clamp -> TPD1E0B04DPLR 0.13pF USB3 ESD; footprint Package_SON:WSON-6-1EP_2x2mm_P0.65mm_EP1x1.6mm -> Diode_SMD:D_0201_0603Metric; symbol Power_Protection:TVS2200DRV -> TPD1E0B04:TPD1E0B04; MPN TVS2200DRVR -> TPD1E0B04DPLR
- D2103: renamed from C2015; value 4.7u 25V raw VBUS; pre-attach total below 10uF -> TPD1E0B04DPLR 0.13pF USB3 ESD; footprint Capacitor_SMD:C_1206_3216Metric -> Diode_SMD:D_0201_0603Metric; symbol Device:C -> TPD1E0B04:TPD1E0B04; MPN GRM31CR71E475KA88L -> TPD1E0B04DPLR; Manufacturer Murata -> Texas Instruments
- D2104: renamed from C2016; value 10n 50V connector VBUS HF -> TPD1E0B04DPLR 0.13pF USB3 ESD; footprint Capacitor_SMD:C_0402_1005Metric -> Diode_SMD:D_0201_0603Metric; symbol Device:C -> TPD1E0B04:TPD1E0B04; MPN GRM155R71H103KA88D -> TPD1E0B04DPLR; Manufacturer Murata -> Texas Instruments
- D2105: renamed from C2017; value 10n 50V connector VBUS HF -> TPD1E0B04DPLR 0.13pF USB3 ESD; footprint Capacitor_SMD:C_0402_1005Metric -> Diode_SMD:D_0201_0603Metric; symbol Device:C -> TPD1E0B04:TPD1E0B04; MPN GRM155R71H103KA88D -> TPD1E0B04DPLR; Manufacturer Murata -> Texas Instruments
- D2106: renamed from C2018; value 10n 50V connector VBUS HF -> TPD1E0B04DPLR 0.13pF USB3 ESD; footprint Capacitor_SMD:C_0402_1005Metric -> Diode_SMD:D_0201_0603Metric; symbol Device:C -> TPD1E0B04:TPD1E0B04; MPN GRM155R71H103KA88D -> TPD1E0B04DPLR; Manufacturer Murata -> Texas Instruments
- D2107: renamed from C2019; value 10n 50V connector VBUS HF -> TPD1E0B04DPLR 0.13pF USB3 ESD; footprint Capacitor_SMD:C_0402_1005Metric -> Diode_SMD:D_0201_0603Metric; symbol Device:C -> TPD1E0B04:TPD1E0B04; MPN GRM155R71H103KA88D -> TPD1E0B04DPLR; Manufacturer Murata -> Texas Instruments
- Q15: renamed from C2066; value 100u 10V PP5V source bulk -> SiSS4409DN 40V reverse-blocking PMOS; footprint Capacitor_Tantalum_SMD:CP_EIA-7343-31_Kemet-D -> Package_SO:Vishay_PowerPAK_1212-8_Single; symbol Device:C_Polarized -> Q_PMOS_1G_234S_5D:Q_PMOS_1G_234S_5D; MPN T520D107M010ATE070 -> SiSS4409DN-T1-GE3; Manufacturer KEMET -> Vishay
- U2005: renamed from C2020; value 6.8u 25V X7R TPS25751A LDO3V3; verify >=5u effective -> TVS2200 22V USB VBUS surge clamp; footprint Capacitor_SMD:C_1206_3216Metric -> Package_SON:WSON-6-1EP_2x2mm_P0.65mm_EP1x1.6mm; symbol Device:C -> Power_Protection:TVS2200DRV; MPN GRM31CR71E685KA88L -> TVS2200DRVR; Manufacturer Murata -> Texas Instruments
- U2015: renamed from U2010; value TUSB1142 USB 3.2 Gen 2 orientation redriver -> TVS2200 22V USB VBUS surge clamp; footprint Package_DFN_QFN:Texas_RNQ0040A_WQFN-40-1EP_6x4mm_P0.4mm_EP4.7x2.7mm_ThermalVias -> Package_SON:WSON-6-1EP_2x2mm_P0.65mm_EP1x1.6mm; symbol TUSB1142:TUSB1142 -> Power_Protection:TVS2200DRV; MPN TUSB1142IRNQR -> TVS2200DRVR; StrapMode GPIO_MODE;FULL_AEQ;4P5DB_HOST_EQ;VIO_3V3 -> (none)
Connections:
- net PD2_MUX_EQCFG is gone; now on net GND: U2015.3 (GND)
- net PD2_MUX_SLEEP_N is gone; now on net PD2_VBUS_RAW: U2015.4 (IN)
- net PD2_MUX_SSEQ1 is gone; now on net GND: U2015.2 (GND)
- net GND: now also U2005.1 (GND), U2005.3 (GND), U2005.7 (GND), U2015.1 (GND), U2015.7 (GND), C2066.2, D2101.2 (IO), D2102.2 (IO); no longer D2100.1 (GND), D2100.3 (GND), D2100.7 (GND), Q15.2, U2015.22 (AEQENZ/SDA), U2015.27 (TEST1), U2015.41 (GND)
- net MCU_3V3: now also C2022.1
- net PD1_CC1_SYS: now also C2023.1; no longer C2015.1
- net PD1_CC2_SYS: now also C2024.1; no longer C2016.1
- net PD1_LDO1V5: now also C2021.1
- net PD1_LDO3V3: now also C2020.1; no longer U2005.1
- net PD1_PPHV: now also C2028.1, C2029.1; no longer C2020.1, C2021.1
- net PD1_RX1_N: now also D2105.1 (IO); no longer C2027.1 (IO)
- net PD1_RX1_P: now also D2104.1 (IO); no longer C2026.1 (IO)
- net PD1_RX2_N: now also D2107.1 (IO); no longer C2029.1 (IO)
- net PD1_RX2_P: now also D2106.1 (IO); no longer C2028.1 (IO)
- net PD1_SEL_FET_COMMON: now also Q15.2 (S), Q15.3 (S), Q15.4 (S)
- net PD1_SEL_GATE: now also Q15.1 (G)
- net PD1_TX1_N: now also D2101.1 (IO); no longer C2023.1 (IO)
- net PD1_TX1_P: now also D2100.1 (IO); no longer C2022.1 (IO)
- net PD1_TX2_N: now also D2103.1 (IO); no longer C2025.1 (IO)
- net PD1_TX2_P: now also D2102.1 (IO); no longer C2024.1 (IO)
- net PD1_VBUS_GATED: now also Q15.5 (D(5-8))
- net PD1_VBUS_RAW: now also C2015.1, C2016.1, C2017.1, C2018.1, C2019.1, U2005.4 (IN), U2005.5 (IN), U2005.6 (IN); no longer D2100.4 (IN), D2100.5 (IN), D2100.6 (IN), D2103.1, D2104.1, D2105.1, D2106.1, D2107.1
- net PD2_MUX_EN: no longer U2015.26 (EN)
- net PD2_MUX_FLIP: no longer U2015.21 (FLIP/SCL)
- net PD2_VBUS_RAW: now also U2015.5 (IN), U2015.6 (IN)
- net SYS_3V3: no longer U2015.1 (VCC), U2015.20 (VCC), U2015.28 (VCC), U2015.6 (VCC)
- net USB_PORT_5V: now also C2025.1, C2026.1, C2027.1, C2066.1; no longer C2017.1, C2018.1, C2019.1, Q15.1
- removed net HUB_DS1_SSTX_N: U2015.15 (SSTXn)
- removed net HUB_DS1_SSTX_P: U2015.16 (SSTXp)
- removed net PD2_CTX1_RAW_N: U2015.34 (CTX1n)
- removed net PD2_CTX1_RAW_P: U2015.33 (CTX1p)
- removed net PD2_CTX2_RAW_N: U2015.39 (CTX2n)
- removed net PD2_CTX2_RAW_P: U2015.40 (CTX2p)
- removed net PD2_MUX_MODE: U2015.17 (MODE)
- removed net PD2_MUX_VIO: U2015.14 (VIO_SEL)
- net PD2_RX1_N: no longer names the net of J11.B10 (RX1-)
- net PD2_RX1_N: no longer U2015.31 (CRX1n)
- net PD2_RX1_P: no longer names the net of J11.B11 (RX1+)
- net PD2_RX1_P: no longer U2015.30 (CRX1p)
- net PD2_RX2_N: no longer names the net of J11.A10 (RX2-)
- net PD2_RX2_N: no longer U2015.36 (CRX2n)
- net PD2_RX2_P: no longer names the net of J11.A11 (RX2+)
- net PD2_RX2_P: no longer U2015.37 (CRX2p)
- removed net PD2_SSRX_RAW_N: U2015.18 (SSRXn)
- removed net PD2_SSRX_RAW_P: U2015.19 (SSRXp)
- net PD2_TX1_N: no longer names the net of J11.A3 (TX1-)
- net PD2_TX1_P: no longer names the net of J11.A2 (TX1+)
- net PD2_TX2_N: no longer names the net of J11.B3 (TX2-)
- net PD2_TX2_P: no longer names the net of J11.B2 (TX2+)
- no-connect marks 67 -> 60
Other:
- note added: "== J11: USB 2.0 data plus USB-PD charging, side port 2 =="
- note added: "== Two rear USB-C data/charging ports: J21 left (USB3) and J11 right (USB2) =="
- note added: "J21 carries USB 3.2 Gen 2 plus USB2. J11 is USB2-only (split architecture: no USB3 host port remains on the right side); both can sink negotiated 15V or source protected default USB current."
- note removed: "== J11: USB 3.2 Gen 2 data plus USB-PD charging, side port 2 =="
- note removed: "== Two rear USB-C data/charging ports: J21 left and J11 right =="
- note removed: "Both ports carry USB 3.2 Gen 2 plus USB2 and can sink negotiated 15V or source protected default USB current."
- moved on the sheet: C2015, C2016, C2019, C2021, C2025, C2026, C2028
