File: 01_power_battery.kicad_sch (KiCad schematic)
At the start: 79 parts, among them J1 Battery balance taps (JST-XH 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, J2 Battery power leads (heavy ga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, J3 Solar panel input, Q1 Q_DSG (10A NMOS, TBD p/n), Q2 Q_CHG (10A NMOS, TBD p/n), Q3 Q_HI solar buck (TBD p/n), Q4 Q_LO solar buck (TBD p/n), U1 BQ76920PW, U2 BQ25798, U3 BQ24650

Commit message: Checkpoint ducktop2 generated schematic baseline
Parts:
- removed F2: 3A (TBD), Fuse:Fuse_1206_3216Metric, symbol Device:Fuse
- removed J3: Solar panel input, Connector_JST:JST_XH_B2B-XH-A_1x02_P2.50mm_Vertical, symbol Connector_Generic:Conn_01x02
- removed Q1: Q_DSG (10A NMOS, TBD p/n), Package_TO_SOT_SMD:TO-252-2, symbol Device:Q_NMOS
- removed Q2: Q_CHG (10A NMOS, TBD p/n), Package_TO_SOT_SMD:TO-252-2, symbol Device:Q_NMOS
- removed Q3: Q_HI solar buck (TBD p/n), Package_TO_SOT_SMD:TO-252-2, symbol Device:Q_NMOS
- removed Q4: Q_LO solar buck (TBD p/n), Package_TO_SOT_SMD:TO-252-2, symbol Device:Q_NMOS
- added C180: 100n BAT filter, Capacitor_SMD:C_0603_1608Metric, symbol Device:C
- added C181: 100n sense filter, Capacitor_SMD:C_0603_1608Metric, symbol Device:C
- added C182: 100n REGIN/VCC, Capacitor_SMD:C_0603_1608Metric, symbol Device:C
- added C183: 1u REG25, Capacitor_SMD:C_0805_2012Metric, symbol Device:C
- added C184: 1nF SDRV cap, ship FET unused, Capacitor_SMD:C_0402_1005Metric, symbol Device:C
- added C190: 10u AUX input bulk, Capacitor_SMD:C_1206_3216Metric, symbol Device:C
- added C191: 100n AUX input, Capacitor_SMD:C_0603_1608Metric, symbol Device:C
- added C192: 100n AUX ADC filter, Capacitor_SMD:C_0603_1608Metric, symbol Device:C
- added D190: SMBJ24CA-class AUX/SOLAR input TVS, Diode_SMD:D_SOD-123, symbol Device:D_TVS
- added D191: POP default AUX -> BQ25798 reverse block, Diode_SMD:D_SMB, symbol Device:D_Schottky
- added F190: 3A AUX/SOLAR input fuse/polyfuse, Fuse:Fuse_1206_3216Metric, symbol Device:Fuse
- added J190: AUX/SOLAR wide-DC screw terminal 6-24V nominal, TerminalBlock_Phoenix:TerminalBlock_Phoenix_MKDS-1,5-2-5.08_1x02_P5.08mm_Horizontal, symbol Connector_Generic:Conn_01x02
- added NTC4: 10k pack NTC, Resistor_SMD:R_0603_1608Metric, symbol Device:Thermistor_NTC
- added Q1: DNP IPD90N04S4L-04 Q_DSG bare-cell pack, Package_TO_SOT_SMD:TO-252-2, symbol Q_NMOS_TO252_GDS:Q_NMOS_TO252_GDS
- added Q2: DNP IPD90N04S4L-04 Q_CHG bare-cell pack, Package_TO_SOT_SMD:TO-252-2, symbol Q_NMOS_TO252_GDS:Q_NMOS_TO252_GDS
- added Q3: DNP IPD50N04S4L-08 solar high-side FET, Package_TO_SOT_SMD:TO-252-2, symbol Q_NMOS_TO252_GDS:Q_NMOS_TO252_GDS
- added Q4: DNP IPD50N04S4L-08 solar low-side FET, Package_TO_SOT_SMD:TO-252-2, symbol Q_NMOS_TO252_GDS:Q_NMOS_TO252_GDS
- added R180: 215k 0.1% pack divider hi, Resistor_SMD:R_0603_1608Metric, symbol Device:R
- added R181: 16.5k 0.1% pack divider lo, Resistor_SMD:R_0603_1608Metric, symbol Device:R
- added R182: 100R BAT filter, Resistor_SMD:R_0603_1608Metric, symbol Device:R
- added R183: 100R SRP filter, Resistor_SMD:R_0603_1608Metric, symbol Device:R
- added R184: 100R SRN filter, Resistor_SMD:R_0603_1608Metric, symbol Device:R
- added R185: 10k CE pull-up, Resistor_SMD:R_0603_1608Metric, symbol Device:R
- added R186: 10k gauge ALERT pull-up, Resistor_SMD:R_0603_1608Metric, symbol Device:R
- added R187: 10k TS pull-up, Resistor_SMD:R_0603_1608Metric, symbol Device:R
- added R188: 0R P2 not-used tie to VSS, Resistor_SMD:R_0603_1608Metric, symbol Device:R
- added R189: 0R P1 not-used tie to VSS, Resistor_SMD:R_0603_1608Metric, symbol Device:R
- added R190: 100k 1% ILIM bottom, Resistor_SMD:R_0603_1608Metric, symbol Device:R
- added R191: 470k 1% AUX ADC top, Resistor_SMD:R_0603_1608Metric, symbol Device:R
- added R192: 56k 1% AUX ADC bottom, Resistor_SMD:R_0603_1608Metric, symbol Device:R
- added R193: 1k AUX ADC series, Resistor_SMD:R_0603_1608Metric, symbol Device:R
- added U10: BQ34Z100-G1 protected-pack gauge, Package_SO:TSSOP-14_4.4x5mm_P0.65mm, symbol BQ34Z100-G1:BQ34Z100-G1
- C1, C14, C15, C2, C3, C4, C5: value 100n -> DNP 100n; now not fitted; now left out of the parts list
- C13: value 100n -> DNP 1u VREF; footprint Capacitor_SMD:C_0603_1608Metric -> Capacitor_SMD:C_0805_2012Metric; now not fitted; now left out of the parts list
- C16, C17, C6: value 1u -> DNP 1u; now not fitted; now left out of the parts list
- C18: value 10u -> DNP 10u solar MPPT input bulk; now not fitted; now left out of the parts list
- D5, D6, D7: footprint Diode_SMD:D_SOD-123 -> Diode_SMD:D_SMB
- D8: value reverse-polarity block -> DNP solar MPPT feed from AUX/SOLAR input; footprint Diode_SMD:D_SOD-123 -> Diode_SMD:D_SMB; now not fitted; now left out of the parts list
- DZ1: value 3.3V -> DNP 3.3V; now not fitted; now left out of the parts list
- DZ2, DZ3, DZ4: value 5.6V -> DNP 5.6V; now not fitted; now left out of the parts list
- F1: value 10A (TBD) -> 10A replaceable pack fuse; footprint Fuse:Fuse_1206_3216Metric -> Fuse:Fuseholder_Blade_Mini_Keystone_3568
- J1: value Battery balance taps (JST-XH 4pin) -> DNP sense-only balance taps (B+/C2/C1/B-); now not fitted; now left out of the parts list
- J2: footprint Connector_JST:JST_XH_B2B-XH-A_1x02_P2.50mm_Vertical -> Connector_Molex:Molex_Mega-Fit_76829-0002_2x01_P5.70mm_Vertical
- L1: value 2.2uH (typ, verify per fsw) -> 2.2uH >=6A buck-boost; footprint (none) -> Inductor_SMD:L_1210_3225Metric
- L2: value 4.7uH (typ, verify) -> DNP 10uH >=3A solar buck; footprint (none) -> Inductor_SMD:L_1210_3225Metric; now not fitted; now left out of the parts list
- LED2: value MPPT STAT1 -> DNP MPPT STAT1; now not fitted; now left out of the parts list
- LED3: value MPPT STAT2 -> DNP MPPT STAT2; now not fitted; now left out of the parts list
- NTC1, NTC3: value 10k NTC -> DNP 10k NTC; now not fitted; now left out of the parts list
- R1, R21, R22, R26, R27, R3, R5, R6, R7, R8, R9: value 1k -> DNP 1k; now not fitted; now left out of the parts list
- R10, R11, R23: value 10k -> DNP 10k; now not fitted; now left out of the parts list
- R13: value 100k -> 100k QON pull-up to 3V3
- R14: value 100k -> 100k CE pull-up to 3V3
- R15: value 10k -> 10k INT pull-up to 3V3
- R17: value TBD (see ILIM_HIZ table) -> 47k 1% ILIM top (3A clamp)
- R18: value TBD (see PROG table) -> 10.5k 1% PROG: 3S, 1.5MHz
- R19: value 100k (TBD-verify MPPT ratio) -> DNP 140k 1% MPPSET top (18V); now not fitted; now left out of the parts list
- R2, R4: value 100k -> DNP 100k; now not fitted; now left out of the parts list
- R20: value 10k (TBD-verify MPPT ratio) -> DNP 10k 1% MPPSET bottom; now not fitted; now left out of the parts list
- R24: value TBD (see VFB table) -> DNP 499k 0.1% 3S charge VFB hi; now not fitted; now left out of the parts list
- R25: value TBD (see VFB table) -> DNP 100k 0.1% 3S charge VFB lo; now not fitted; now left out of the parts list
- R28, R29: value 4.7 -> DNP 4.7; now not fitted; now left out of the parts list
- R30: value 4.7k -> 4.7k I2C SCL pull-up to 3V3
- R31: value 4.7k -> 4.7k I2C SDA pull-up to 3V3
- RS1: value 2mOhm (TBD - size for 10A cont.) -> 5mOhm 1% Kelvin gauge shunt >=5A; footprint (none) -> Resistor_SMD:R_2512_6332Metric
- RS2: value 10mOhm (TBD - size for solar current) -> DNP 40mOhm 1% solar sense, 1A fast-charge; footprint (none) -> Resistor_SMD:R_2512_6332Metric; now not fitted; now left out of the parts list
- U1: value BQ76920PW -> BQ76920PW (DNP if pack BMS remains); now not fitted; now left out of the parts list
- U3: value BQ24650 -> DNP BQ24650 optional solar MPPT; now not fitted; now left out of the parts list
Connections:
- net BQ_ALERT: now also R186.2
- net CHG_GATE: now also Q2.1 (G)
- net DSG_GATE: now also Q1.1 (G)
- net FET_MID: now also Q1.3 (S), Q2.2 (D)
- net GND: now also C180.2, C182.2, C183.2, C184.2, C190.2, C191.2, C192.2, D190.2 (A2), J190.2 (Pin_2), NTC4.2, Q4.3 (S), R181.2, R184.1, R188.2, R189.2, R190.2, R192.2, U10.8 (VSS); no longer R17.2, U2.8 (VAC2), U2.9 (VAC1)
- net I2C_SCL: now also U10.13 (P4/SCL)
- net I2C_SDA: now also U10.14 (P3/SDA)
- net ILIM_SET: now also R17.2, R190.1; no longer R17.1
- net PACK_POS_FUSED: now also R24.1, R27.1, RS2.2, U2.18 (BATP), U2.22 (BAT), U2.23 (BAT), R180.1; no longer J2.1 (Pin_1)
- net QHI_GATE: now also Q3.1 (G)
- net QLO_GATE: now also Q4.1 (G)
- net REGN: now also R17.1; no longer R13.2, R14.2, R15.2, R30.1, R31.1
- net SOLAR_IN: now also Q3.2 (D)
- net SOLAR_SW: now also Q3.3 (S), Q4.2 (D)
- net VBUS_COMBINED: now also U2.8 (VAC2), U2.9 (VAC1), D191.1 (K)
- net SDRV_DAMP: now reaches U2.24 (SDRV)
- net SDRV_DAMP: now also C184.1
- net PACK_NEG renamed CELL0_BAL
- net CELL0_BAL: now also Q1.2 (D); no longer J2.2 (Pin_2)
- removed net PACK_POS: F1.1, J1.1 (Pin_1), R24.1, R27.1, R9.1, RS2.2, U1.10 (BAT), U1.12 (VC5), U1.13 (VC4), U1.9 (REGSRC), U2.18 (BATP), U2.22 (BAT), U2.23 (BAT)
- net RSENSE_HI renamed PACK_NEG_RAW
- net PACK_NEG_RAW: now also J2.2 (Pin_2), Q2.3 (S), R183.1
- net SOLAR_IN_FUSED renamed AUX_DC_FUSED
- net AUX_DC_FUSED: now also C190.1, C191.1, D190.1 (A1), D191.2 (A), F190.2, R191.1
- new net AUX_DC_ADC: C192.1, R193.2
- new net AUX_DC_DIV: R191.2, R192.1, R193.1
- new net AUX_DC_RAW: F190.1, J190.1 (Pin_1)
- new net CELL3_BAL: J1.1 (Pin_1), R9.1, U1.10 (BAT), U1.12 (VC5), U1.13 (VC4), U1.9 (REGSRC)
- new net FG_BAT_DIV: R180.2, R181.1, R182.1
- new net FG_BAT_SENSE: C180.1, R182.2, U10.4 (BAT)
- new net FG_CE: R185.2, U10.5 (CE)
- new net FG_P1_TIE: R189.1, U10.3 (P1)
- new net FG_P2_TIE: R188.1, U10.1 (P2)
- new net FG_REG25: C183.1, U10.7 (REG25)
- new net FG_SRN: C181.2, R184.2, U10.10 (SRN)
- new net FG_SRP: C181.1, R183.2, U10.9 (SRP)
- new net FG_TS: NTC4.1, R187.2, U10.11 (P6/TS)
- new net MCU_3V3: C182.1, R13.2, R14.2, R15.2, R185.1, R186.1, R187.1, R30.1, R31.1, U10.6 (REGIN)
- new net PACK_POS_RAW: F1.1, J2.1 (Pin_1)
- no-connect marks 2 -> 3
Other:
- note added: "== U1 bq76920 3S Battery AFE / Protection (optional/DNP with protected pack) =="
- note added: "== U10 BQ34Z100-G1 3S fuel gauge for protected external pack =="
- note added: "== U2 bq25798 Buck-Boost Charger / NVDC Power Path (VSYS) =="
- note added: "== U3 bq24650 optional solar MPPT from shared AUX/SOLAR input =="
- note added: "AUX divider maps 24V to about 2.56V and 30V abs-max to about 3.19V at the EC ADC."
- note added: "AUX_DC_ADC lets EC firmware detect random bench/DC inputs and reduce BQ25798 input current if the source droops."
- note added: "Balance taps are sense-only and DNP by default; they never feed PACK_POS_FUSED."
- note added: "Charger I2C/INT/QON/CE pull-ups use MCU_3V3 so STM32 pins never see REGN-level logic."
- note added: "D5-D7/D191: K(pin1)=VBUS_COMBINED, A(pin2)=input raw/fused VBUS"
- note added: "DNP Q1/Q2 candidate: Infineon IPD90N04S4L-04, 40V 3.8mR DPAK, active/preferred, pin 1=G 2=D/tab 3=S."
- note added: "DNP Q3/Q4 candidate: Infineon IPD50N04S4L-08, 40V 7.3mR DPAK, lower Qg for BQ24650 6V gate drive."
- note added: "Default BOM should not populate D8 with D191; choose random-DC charger input or solar MPPT behavior for J190."
- note added: "Default build populates D191 for random DC; solar option feeds U3 from same terminal via D8."
- note added: "Do not populate D8 and D191 together unless dual-charger input policy is intentionally reviewed."
- note added: "If solar option is used, U3 starts at 18V nominal MPP, 12.6V 3S regulation, and 1A solar charge current."
- note added: "J190 is shared: default random-DC mode populates D191 to U2; solar mode populates D8/U3 MPPT option."
- note added: "J190 is the single AUX/SOLAR physical input; USB-C PD negotiation remains only on sheet 5."
- note added: "RS1 remains populated as the BQ34Z100-G1 low-side current shunt; Kelvin route SRP/SRN per TI layout guidance."
- note added: "SDRV has 1nF to GND because the ship FET is unused in this first integrated laptop spin."
- note added: "TS1/TS2/TS3/FG_TS use independent thermistor dividers per-IC (not shared) per design decision."
- note added: "The real pack already has a protection-only BMS; U1/Q1/Q2 are optional/DNP unless a bare-cell pack is used."
- note added: "U10 pinout is verified against TI Table 5-1; divider 215k/16.5k gives about 0.90V at 12.6V full-charge 3S."
- note added: "U2 ILIM_HIZ divider sets about 3A input-current clamp from REGN; PROG selects 3S/1.5MHz POR defaults."
- note added: "U2 VAC1/VAC2 tie to VBUS_COMBINED in no-external-mux mode; ACDRV1/2 go to GND."
- note removed: "== U1 bq76920 3S Battery AFE / Protection =="
- note removed: "== U2 bq25798 USB-PD Buck-Boost Charger (VSYS) =="
- note removed: "== U3 bq24650 Solar MPPT Charger =="
- note removed: "D5-D7: K(pin1)=VBUS_COMBINED, A(pin2)=port raw VBUS"
- note removed: "I2C pull-ups R30 (SCL)/R31 (SDA) sourced from U2 REGN only, to avoid cross-LDO backfeed between REGOUT and REGN."
- note removed: "SDRV (U2 pin24) intentionally left NC - ship-mode FET not yet designed."
- note removed: "TS1/TS2/TS3 use independent thermistor dividers per-IC (not shared) per design decision."
- note removed: "VERIFY: pack must expose 4-wire JST-XH balance tap (B-/C1/C2/B+)"

Commit message: Publish the current Ducktop2 design
Parts:
- removed C1, C14, C15, C2, C3, C4, C5: DNP 100n, Capacitor_SMD:C_0603_1608Metric, symbol Device:C
- removed C12: 10u, Capacitor_SMD:C_1206_3216Metric, symbol Device:C
- removed C13: DNP 1u VREF, Capacitor_SMD:C_0805_2012Metric, symbol Device:C
- removed C16, C6: DNP 1u, Capacitor_SMD:C_0805_2012Metric, symbol Device:C
- removed C184: 1nF SDRV cap, ship FET unused, Capacitor_SMD:C_0402_1005Metric, symbol Device:C
- removed C190: 10u AUX input bulk, Capacitor_SMD:C_1206_3216Metric, symbol Device:C
- removed C191: 100n AUX input, Capacitor_SMD:C_0603_1608Metric, symbol Device:C
- removed D191: POP default AUX -> BQ25798 reverse block, Diode_SMD:D_SMB, symbol Device:D_Schottky
- removed D5, D6, D7: (no value), Diode_SMD:D_SMB, symbol Device:D_Schottky
- removed DZ1: DNP 3.3V, Diode_SMD:D_SOD-123, symbol Device:D_Zener
- removed DZ2, DZ3, DZ4: DNP 5.6V, Diode_SMD:D_SOD-123, symbol Device:D_Zener
- removed F1: 10A replaceable pack fuse, Fuse:Fuseholder_Blade_Mini_Keystone_3568, symbol Device:Fuse
- removed J1: DNP sense-only balance taps (B+/C2/C1/B-), Connector_JST:JST_XH_B4B-XH-A_1x04_P2.50mm_Vertical, symbol Connector_Generic:Conn_01x04
- removed J2: Battery power leads (heavy gauge), Connector_Molex:Molex_Mega-Fit_76829-0002_2x01_P5.70mm_Vertical, symbol Connector_Generic:Conn_01x02
- removed LED2: DNP MPPT STAT1, LED_SMD:LED_0603_1608Metric, symbol Device:LED
- removed LED3: DNP MPPT STAT2, LED_SMD:LED_0603_1608Metric, symbol Device:LED
- removed NTC1, NTC3: DNP 10k NTC, Resistor_SMD:R_0603_1608Metric, symbol Device:Thermistor_NTC
- removed NTC2: 10k NTC, Resistor_SMD:R_0603_1608Metric, symbol Device:Thermistor_NTC
- removed NTC4: 10k pack NTC, Resistor_SMD:R_0603_1608Metric, symbol Device:Thermistor_NTC
- removed Q1: DNP IPD90N04S4L-04 Q_DSG bare-cell pack, Package_TO_SOT_SMD:TO-252-2, symbol Q_NMOS_TO252_GDS:Q_NMOS_TO252_GDS
- removed Q2: DNP IPD90N04S4L-04 Q_CHG bare-cell pack, Package_TO_SOT_SMD:TO-252-2, symbol Q_NMOS_TO252_GDS:Q_NMOS_TO252_GDS
- removed Q3: DNP IPD50N04S4L-08 solar high-side FET, Package_TO_SOT_SMD:TO-252-2, symbol Q_NMOS_TO252_GDS:Q_NMOS_TO252_GDS
- removed Q4: DNP IPD50N04S4L-08 solar low-side FET, Package_TO_SOT_SMD:TO-252-2, symbol Q_NMOS_TO252_GDS:Q_NMOS_TO252_GDS
- removed R1, R21, R22, R26, R27, R3, R5, R6, R7, R8, R9: DNP 1k, Resistor_SMD:R_0603_1608Metric, symbol Device:R
- removed R10, R11, R23: DNP 10k, Resistor_SMD:R_0603_1608Metric, symbol Device:R
- removed R187: 10k TS pull-up, Resistor_SMD:R_0603_1608Metric, symbol Device:R
- removed R188: 0R P2 not-used tie to VSS, Resistor_SMD:R_0603_1608Metric, symbol Device:R
- removed R19: DNP 140k 1% MPPSET top (18V), Resistor_SMD:R_0603_1608Metric, symbol Device:R
- removed R2, R4: DNP 100k, Resistor_SMD:R_0603_1608Metric, symbol Device:R
- removed R20: DNP 10k 1% MPPSET bottom, Resistor_SMD:R_0603_1608Metric, symbol Device:R
- removed R24: DNP 499k 0.1% 3S charge VFB hi, Resistor_SMD:R_0603_1608Metric, symbol Device:R
- removed R25: DNP 100k 0.1% 3S charge VFB lo, Resistor_SMD:R_0603_1608Metric, symbol Device:R
- removed R28, R29: DNP 4.7, Resistor_SMD:R_0603_1608Metric, symbol Device:R
- removed unit 2 of U1
- removed U3: DNP BQ24650 optional solar MPPT, Package_DFN_QFN:Texas_RVA_VQFN-16-1EP_3.5x3.5mm_P0.5mm_EP2.14x2.14mm_ThermalVias, symbol ducktop2:BQ24650
- added C700: 3.3nF >=50V LTC4368 CGATE, Capacitor_SMD:C_0402_1005Metric, symbol Device:C
- added C701, C702: 10u 25V X7R VBUS, Capacitor_SMD:C_1206_3216Metric, symbol Device:C
- added C703, C704, C705: 10u 25V X7R PMID, Capacitor_SMD:C_1206_3216Metric, symbol Device:C
- added C706, C707, C708, C709, C710: 10u 25V X7R SYS, Capacitor_SMD:C_1206_3216Metric, symbol Device:C
- added C711: 100n 50V X7R BAT local, Capacitor_SMD:C_0603_1608Metric, symbol Device:C
- added C720: 1u 50V X7R AUX input, Capacitor_SMD:C_0805_2012Metric, symbol Device:C
- added C721: 100n 50V X7R AUX eFuse local, Capacitor_SMD:C_0603_1608Metric, symbol Device:C
- added C722: 10u 50V X7R AUX output, Capacitor_SMD:C_1206_3216Metric, symbol Device:C
- added C723: 100n AUX eFuse dVdT approx 50ms at 24V, Capacitor_SMD:C_0603_1608Metric, symbol Device:C
- added C724: 4.7nF >=50V pack hot-swap slew, Capacitor_SMD:C_0402_1005Metric, symbol Device:C
- added C725: 10u 25V X7R LTC4368 VOUT, Capacitor_SMD:C_0805_2012Metric, symbol Device:C
- added C740: 100n 10V INTVCC, Capacitor_SMD:C_0603_1608Metric, symbol Device:C
- added C741: 15n 50V TMR approx 240ms, Capacitor_SMD:C_0402_1005Metric, symbol Device:C
- added C742: 100n 50V USB V1 local, Capacitor_SMD:C_0603_1608Metric, symbol Device:C
- added C743: 100n 50V USB VS1 local, Capacitor_SMD:C_0603_1608Metric, symbol Device:C
- added C744: 100n 50V AUX V2 local, Capacitor_SMD:C_0603_1608Metric, symbol Device:C
- added C745: 100n 50V AUX VS2 local, Capacitor_SMD:C_0603_1608Metric, symbol Device:C
- added C746: 100u 35V hybrid selector output hold-up, Capacitor_SMD:CP_Elec_6.3x5.8, symbol Device:C_Polarized
- added C795: 1u 25V AON eFuse input, Capacitor_SMD:C_0805_2012Metric, symbol Device:C
- added C796: 100n 50V AON eFuse input local, Capacitor_SMD:C_0603_1608Metric, symbol Device:C
- added C797: 10u 25V AON eFuse output, Capacitor_SMD:C_1206_3216Metric, symbol Device:C
- added C798: 100n 50V AON eFuse output local, Capacitor_SMD:C_0603_1608Metric, symbol Device:C
- added C799: 3.3n AON eFuse dVdt, Capacitor_SMD:C_0402_1005Metric, symbol Device:C
- added C840: 1u 25V X7R BQ77915 VDD, Capacitor_SMD:C_0805_2012Metric, symbol Device:C
- added C841: 1u 10V X7R BQ77915 AVDD, Capacitor_SMD:C_0805_2012Metric, symbol Device:C
- added C842, C843, C844, C848: 1u 10V X7R BQ77915 internal-balance filter, Capacitor_SMD:C_0805_2012Metric, symbol Device:C
- added C845: 100n BQ77915 SRP-VSS filter, Capacitor_SMD:C_0603_1608Metric, symbol Device:C
- added C846: 100n BQ77915 differential sense filter, Capacitor_SMD:C_0603_1608Metric, symbol Device:C
- added C847: 100n BQ77915 SRN-VSS filter, Capacitor_SMD:C_0603_1608Metric, symbol Device:C
- added D710, D711, D712, D713, D714: B340A 3A 40V EC always-on OR, Diode_SMD:D_SMA, symbol Device:D_Schottky
- added D715: BAT54WS case button to charger QON, Diode_SMD:D_SOD-323, symbol Device:D_Schottky
- added D716: BAT54WS case button to Mu PWRBTN, Diode_SMD:D_SOD-323, symbol Device:D_Schottky
- added J2: 3S pack power + cell-tap harness, Connector_Molex:Molex_Mega-Fit_76829-0006_2x03_P5.70mm_Vertical, symbol Connector_Generic:Conn_02x03_Odd_Even
- added Q11: CSD18540Q5B reverse-pack FET A, ducktop2:CSD18540Q5B_DNK, symbol Q_NMOS_123S_4G_5678D:Q_NMOS_123S_4G_5678D
- added Q12: CSD18540Q5B reverse-pack FET B, ducktop2:CSD18540Q5B_DNK, symbol Q_NMOS_123S_4G_5678D:Q_NMOS_123S_4G_5678D
- added Q13: CSD19537Q3 100V AUX reverse FET, ducktop2:CSD19537Q3_DQG, symbol Q_NMOS_123S_4G_5678D:Q_NMOS_123S_4G_5678D
- added Q14: BSS138 fast reverse-gate pulldown, Package_TO_SOT_SMD:SOT-23, symbol Q_NMOS_SOT23_GSD:Q_NMOS_SOT23_GSD
- added Q21, Q22, Q23, Q24: SiSS4409DN 40V reverse-blocking PMOS, Package_SO:Vishay_PowerPAK_1212-8_Single, symbol Q_PMOS_1G_234S_5D:Q_PMOS_1G_234S_5D
- added Q25: CSD17575Q3 BQ25798 ship FET, ducktop2:CSD19537Q3_DQG, symbol Q_NMOS_123S_4G_5678D:Q_NMOS_123S_4G_5678D
- added Q700: BSS138 active-high charger enable pull-down, Package_TO_SOT_SMD:SOT-23, symbol Q_NMOS_SOT23_GSD:Q_NMOS_SOT23_GSD
- added Q701: BSS138 pack protector latch reset, Package_TO_SOT_SMD:SOT-23, symbol Q_NMOS_SOT23_GSD:Q_NMOS_SOT23_GSD
- added Q702: BSS138 QON open-drain pulse, Package_TO_SOT_SMD:SOT-23, symbol Q_NMOS_SOT23_GSD:Q_NMOS_SOT23_GSD
- added Q703: CSD18540Q5B BQ77915 discharge FET, ducktop2:CSD18540Q5B_DNK, symbol Q_NMOS_123S_4G_5678D:Q_NMOS_123S_4G_5678D
- added Q704: CSD18540Q5B BQ77915 charge FET, ducktop2:CSD18540Q5B_DNK, symbol Q_NMOS_123S_4G_5678D:Q_NMOS_123S_4G_5678D
- added R700: 3.09M 1% BAT UV/OV top, Resistor_SMD:R_0603_1608Metric, symbol Device:R
- added R701: 73.2k 1% BAT UV/OV middle, Resistor_SMD:R_0603_1608Metric, symbol Device:R
- added R702: 121k 1% BAT UV/OV bottom, Resistor_SMD:R_0603_1608Metric, symbol Device:R
- added R703: 22k LTC4368 CGATE series, Resistor_SMD:R_0603_1608Metric, symbol Device:R
- added R704: 100R BATP Kelvin filter, Resistor_SMD:R_0603_1608Metric, symbol Device:R
- added R705: 7.50k 1% fixed-valid TS bottom, Resistor_SMD:R_0603_1608Metric, symbol Device:R
- added R707: 100k pack protector SHDN pull-up, Resistor_SMD:R_0603_1608Metric, symbol Device:R
- added R708: 10k pack FAULT pull-up, Resistor_SMD:R_0603_1608Metric, symbol Device:R
- added R709: 100k pack retry gate pulldown, Resistor_SMD:R_0603_1608Metric, symbol Device:R
- added R710: 6.04k 1% AUX 3A current limit, Resistor_SMD:R_0603_1608Metric, symbol Device:R
- added R711: 300k 0.1% AUX UV/OV top, Resistor_SMD:R_0603_1608Metric, symbol Device:R
- added R712: 63.2k 0.1% AUX UV/OV middle, Resistor_SMD:R_0603_1608Metric, symbol Device:R
- added R713: 20.0k 0.1% AUX UV/OV bottom, Resistor_SMD:R_0603_1608Metric, symbol Device:R
- added R714: 31R AUX reverse-FET pulldown gate, Resistor_SMD:R_0603_1608Metric, symbol Device:R
- added R715: 10k AUX eFuse FLT pull-up, Resistor_SMD:R_0603_1608Metric, symbol Device:R
- added R716: 10k AUX eFuse PGOOD pull-up, Resistor_SMD:R_0603_1608Metric, symbol Device:R
- added R717: 10k main USB VALID pull-up, Resistor_SMD:R_0603_1608Metric, symbol Device:R
- added R718: 10k main AUX VALID pull-up, Resistor_SMD:R_0603_1608Metric, symbol Device:R
- added R719: 100k charger-enable gate pulldown, Resistor_SMD:R_0603_1608Metric, symbol Device:R
- added R730: 1.00M 0.1% USB UV top, Resistor_SMD:R_0603_1608Metric, symbol Device:R
- added R731: 19.6k 0.1% USB window middle, Resistor_SMD:R_0603_1608Metric, symbol Device:R
- added R732: 63.4k 0.1% USB OV bottom, Resistor_SMD:R_0603_1608Metric, symbol Device:R
- added R733: 383k 0.1% AUX UV top, Resistor_SMD:R_0603_1608Metric, symbol Device:R
- added R734: 63.4k 0.1% AUX window middle, Resistor_SMD:R_0603_1608Metric, symbol Device:R
- added R735: 20.0k 0.1% AUX OV bottom, Resistor_SMD:R_0603_1608Metric, symbol Device:R
- added R739: 332k 0.1% AUX PGOOD threshold top, Resistor_SMD:R_0603_1608Metric, symbol Device:R
- added R740: 97.6k 0.1% AUX PGOOD threshold bottom, Resistor_SMD:R_0603_1608Metric, symbol Device:R
- added R795: 301k 0.1% AON UV/OV top, Resistor_SMD:R_0603_1608Metric, symbol Device:R
- added R796: 52.3k 0.1% AON UV/OV middle, Resistor_SMD:R_0603_1608Metric, symbol Device:R
- added R797: 20.0k 0.1% AON UV/OV bottom, Resistor_SMD:R_0603_1608Metric, symbol Device:R
- added R798: 2.21k 0.1% AON ILM 1.51A typ, Resistor_SMD:R_0603_1608Metric, symbol Device:R
- added R840: 1k 1% BQ77915 VDD filter, Resistor_SMD:R_0603_1608Metric, symbol Device:R
- added R841, R842, R843, R844: 75R 1% BQ77915 cell/balance filter, Resistor_SMD:R_0603_1608Metric, symbol Device:R
- added R845: 100R BQ77915 SRP filter, Resistor_SMD:R_0603_1608Metric, symbol Device:R
- added R846: 100R BQ77915 SRN filter, Resistor_SMD:R_0603_1608Metric, symbol Device:R
- added R847: 4.53k 1% DSG gate resistor, Resistor_SMD:R_0603_1608Metric, symbol Device:R
- added R848: 1k 1% CHG gate resistor, Resistor_SMD:R_0603_1608Metric, symbol Device:R
- added R849: 1M 5% DSG gate-source, Resistor_SMD:R_0603_1608Metric, symbol Device:R
- added R850: 3.3M 5% CHG gate-source, Resistor_SMD:R_0603_1608Metric, symbol Device:R
- added R851: 453k 1% load-detect resistor, Resistor_SMD:R_0603_1608Metric, symbol Device:R
- added R852: 10k 5% PRES normal-mode pull-up, Resistor_SMD:R_0603_1608Metric, symbol Device:R
- added R853: 10k 1% unused TS to VSS, Resistor_SMD:R_0603_1608Metric, symbol Device:R
- added R854: 604k 1% OCD delay program, Resistor_SMD:R_0603_1608Metric, symbol Device:R
- added R855: 10k unused external TS pulldown, Resistor_SMD:R_0603_1608Metric, symbol Device:R
- added RS10: 11mOhm 1% 2W LTC4368 bounded pack-current shunt, Resistor_SMD:R_2512_6332Metric, symbol Device:R
- added RS11: 8mOhm 1% 2W BQ77915 current shunt, Resistor_SMD:R_2512_6332Metric, symbol Device:R
- added TP1: GND test, TestPoint:TestPoint_Pad_D1.0mm, symbol Connector:TestPoint
- added TP10: PACK_FAULT_N test, TestPoint:TestPoint_Pad_D1.0mm, symbol Connector:TestPoint
- added TP11: AON_FAULT_N test, TestPoint:TestPoint_Pad_D1.0mm, symbol Connector:TestPoint
- added TP2: PACK_POS_FUSED test, TestPoint:TestPoint_Pad_D1.0mm, symbol Connector:TestPoint
- added TP3: VSYS test, TestPoint:TestPoint_Pad_D1.0mm, symbol Connector:TestPoint
- added TP4: EC_AON_IN test, TestPoint:TestPoint_Pad_D1.0mm, symbol Connector:TestPoint
- added TP7: MCU_3V3 test, TestPoint:TestPoint_Pad_D1.0mm, symbol Connector:TestPoint
- added TP9: CHG_INT_N test, TestPoint:TestPoint_Pad_D1.0mm, symbol Connector:TestPoint
- added U11: LTC4368IMS-1 bidirectional pack protector, Package_SO:MSOP-10_3x3mm_P0.5mm, symbol LTC4368-1:LTC4368-1
- added U12: TPS26630RGER 3A AUX eFuse / surge cutoff, Package_DFN_QFN:Texas_RGE0024H_VQFN-24-1EP_4x4mm_P0.5mm_EP2.7x2.7mm_ThermalVias, symbol Power_Management:TPS26630RGE
- added U15: LTC4418IUF#PBF dual-input selector, ducktop2:ADI_UF20_QFN20_4x4_P0.5_EP2.45, symbol LTC4418IUF:LTC4418IUF
- added U718: TPS259470ARPW aggregate EC AON eFuse, ducktop2:Texas_RPW0010A_VQFN-HR-10_2x2mm, symbol TPS259470A:TPS259470A
- added U719: BQ7791500PWR autonomous 3S primary protector, Package_SO:TSSOP-24_4.4x7.8mm_P0.65mm, symbol BQ77915:BQ77915
- C10: value 10u -> 100n 50V X7R PMID local; footprint Capacitor_SMD:C_1206_3216Metric -> Capacitor_SMD:C_0603_1608Metric
- C11: value 10u -> 100n 50V X7R SYS local; footprint Capacitor_SMD:C_1206_3216Metric -> Capacitor_SMD:C_0603_1608Metric
- C12: renamed from C18; value DNP 10u solar MPPT input bulk -> 100n 50V X7R VBUS local; footprint Capacitor_SMD:C_1206_3216Metric -> Capacitor_SMD:C_0603_1608Metric; MPN (none) -> GRM188R71H104KA93D; Manufacturer (none) -> Murata; now fitted; now in the parts list
- C7: value 100n -> 47n 25V X7R BTST1; footprint Capacitor_SMD:C_0603_1608Metric -> Capacitor_SMD:C_0402_1005Metric; MPN (none) -> GRM155R71E473KA88D; Manufacturer (none) -> Murata
- C712: renamed from L2; value DNP 10uH >=3A solar buck -> 10u 25V X7R BAT; footprint Inductor_SMD:L_1210_3225Metric -> Capacitor_SMD:C_1206_3216Metric; symbol Device:L -> Device:C; MPN (none) -> GRM31CR71E106KA12L; Manufacturer (none) -> Murata; now fitted; now in the parts list
- C713: renamed from RS2; value DNP 40mOhm 1% solar sense, 1A fast-charge -> 10u 25V X7R BAT; footprint Resistor_SMD:R_2512_6332Metric -> Capacitor_SMD:C_1206_3216Metric; symbol Device:R -> Device:C; MPN (none) -> GRM31CR71E106KA12L; Manufacturer (none) -> Murata; now fitted; now in the parts list
- C714: renamed from D8; value DNP solar MPPT feed from AUX/SOLAR input -> 2.2u 25V X7R VBUS hot-plug damper; footprint Diode_SMD:D_SMB -> Capacitor_SMD:C_0805_2012Metric; symbol Device:D_Schottky -> Device:C; MPN (none) -> GRM21BR71E225KA73L; Manufacturer (none) -> Murata; now fitted; now in the parts list
- C8: value 100n -> 47n 25V X7R BTST2; footprint Capacitor_SMD:C_0603_1608Metric -> Capacitor_SMD:C_0402_1005Metric; MPN (none) -> GRM155R71E473KA88D; Manufacturer (none) -> Murata
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Connections:
- net DSG_DRV is gone; now on net PACK_POS_RAW: F1.1
- net FG_P2_TIE is gone; now on net BQ_ALERT: U10.1 (P2)
- net SOLAR_SW is gone; now on net BAT_CHARGER: C712.1
- net AUX_DC_FUSED: now also Q13.5 (D(5-8)), U12.1 (IN), U12.2 (IN); no longer C714.2 (A), R191.1
- net CHG_INT_N: now also TP9.1
- net FG_TS: now also R855.1
- net GND: now also C712.2, C713.2, C714.2, R13.2, C700.2, C701.2, C702.2, C703.2, C704.2, C705.2, C706.2, C707.2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; no longer C180.2, C182.2, C183.2, R181.2, R189.2, R706.2, U10.8 (VSS)
- net I2C_SCL: no longer F1.5 (SCL)
- net I2C_SDA: no longer F1.4 (SDA)
- net MCU_3V3: now also R708.1, R715.1, R716.1, R717.1, R718.1, TP7.1; no longer R13.2, R14.2
- net PACK_NEG_RAW: now also C840.2, C841.2, C842.2, C845.2, C847.2, J2.3 (Pin_3), J2.4 (Pin_4), R841.1, R845.1, R853.2, R854.2, RS11.1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; no longer R183.1, RS1.1
- net PACK_POS_FUSED: now also C725.1, Q25.5 (D(5-8)), R704.1, RS10.2, TP2.1, U11.8 (VOUT); no longer C713.2, R180.1, U2.18 (BATP), U2.22 (BAT), U2.23 (BAT)
- net PACK_POS_RAW: now also J2.1 (Pin_1), J2.2 (Pin_2), R840.1, R844.1, R852.1
- net PMID: now also C703.1, C704.1, C705.1
- net REGN: now also R14.1
- net VBUS_COMBINED: now also C12.1, R706.1, C701.1, C702.1, C746.1, Q22.5 (D(5-8)), Q24.5 (D(5-8)), U15.15 (VOUT)
- net VSYS: now also C706.1, C707.1, C708.1, C709.1, C710.1, TP3.1
- removed net CELL0_BAL: F1.3 (VSS)
- net CHG_CE_N renamed CHG_CE_HW_N
- net CHG_CE_HW_N: now also R14.2, Q700.3 (D); no longer R14.1
- net CHG_DRV renamed BAT_PROT_VIN
- net BAT_PROT_VIN: now also R180.1, Q11.5 (D(5-8)), R700.1, R707.1, U11.1 (VIN)
- net PMIC_QON renamed PMIC_QON_ASSERT
- net PMIC_QON_ASSERT: now also Q702.1 (G); no longer U2.12 (~{QON})
- net SDRV_DAMP renamed SDRV_GATE
- net SDRV_GATE: now also Q25.4 (G)
- removed net SOLAR_IN: C12.1, C714.1 (K), R706.1
- net SOLAR_ISNS_HI_RAW renamed BAT_CHARGER
- net BAT_CHARGER: now also U2.22 (BAT), U2.23 (BAT), C711.1, D710.2 (A), Q25.1 (S), Q25.2 (S), Q25.3 (S); no longer C712.2
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Other:
- note added: "== 3S cell entry, autonomous primary protection, fuse and redundant pack protection =="
- note added: "== U15 LTC4418IUF: USB-C PD priority over protected AUX/solar =="
- note added: "A 5V-only USB-C source leaves the laptop off. AON_FAULT_N inhibits charging and Mu start; the service connector remains the assembly hard disconnect."
- note added: "AON UVLO corners are 6.06-6.36V: default 5V USB-C is negotiation-only; CH224A must autonomously obtain its strapped 15V PDO before EC_AON_IN starts."
- note added: "AUX_DC_ADC measures the post-reverse-FET input so firmware can detect droop and reduce BQ25798 input current."
- note added: "BQ25798 /CE is fail-off: REGN pulls it high; active-high CHG_ENABLE turns Q700 on only after EC source validation."
- note added: "BQ25798 TS is fixed at 58.9% REGN by 5.24k/7.50k; firmware sets TS_IGNORE=1. BQ34Z100 TS has 10k to VSS; set TEMPS=0."
- note added: "BQ25798 firmware must set STOP_WD_CHG=1 and TS_IGNORE=1, service faults, validate PDO current, and assert CHG_ENABLE only after safe limits are programmed."
- note added: "C746 provides low-ESR hold-up through LTC4418 break-before-make source switching."
- note added: "J190 is the one 7-22V nominal AUX/solar input; TPS26630 protects it before BQ25798."
- note added: "J2: pins 1/2 PACK+, pins 3/4 PACK-, pin 5 cell1 tap, pin 6 cell2 tap. Verify harness order before first connection."
- note added: "MANDATORY STARTUP: hold MU_12V_ENABLE low; require selected-source VALID; read CH224A PDO current; program VSYSMIN and IINDPM <= min(PDO-0.25A, 2.75A); require VSYS >=10.0V."
- note added: "No motherboard battery thermistors are fitted. U719 TS uses TI's 10k-to-VSS unused-function connection; VTB is NC."
- note added: "Q25 follows BQ25798EVM-842: SDRV disconnects pack discharge for electronic ship/hard-off while adapter charging can wake the pack."
- note added: "RS11=8mOhm gives 7.5A nominal OCD and 15A nominal SCD; U11/RS10 and F1 remain independent tighter/secondary protection."
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
Commit message: Finish USB-C policy and split out radio board
Parts:
- removed D714: B340A 3A 40V EC always-on OR, Diode_SMD:D_SMA, symbol Device:D_Schottky
Other:
- note added: "AON UVLO corners are 6.06-6.36V: default 5V USB-C is negotiation-only; TPS25751A dead-battery boot must obtain a valid higher-voltage PDO before EC_AON_IN starts."
- note added: "MANDATORY STARTUP: hold MU_12V_ENABLE low; read TPS25751A PD Status 0x35 plus Active PDO/RDO 0x31/0x32; program VSYSMIN and IINDPM <= min(PDO-0.25A, 2.75A); require VSYS >=10.0V."
- note added: "U2 ILIM_HIZ divider is a 3.0A hardware ceiling; EC programs a lower IINDPM from the selected TPS25751A Active PDO Contract (0x31)."
- note removed: "AON UVLO corners are 6.06-6.36V: default 5V USB-C is negotiation-only; CH224A must autonomously obtain its strapped 15V PDO before EC_AON_IN starts."
- note removed: "MANDATORY STARTUP: hold MU_12V_ENABLE low; require selected-source VALID; read CH224A PDO current; program VSYSMIN and IINDPM <= min(PDO-0.25A, 2.75A); require VSYS >=10.0V."
- note removed: "U2 ILIM_HIZ divider is a 3.0A hardware ceiling; EC programs a lower IINDPM from the selected CH224A PDO current."
Changed lines of the file:
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@@
-(symbol
-  (lib_id "power:PWR_FLAG")
-  (at 650.24 74.93 0)
-  (unit 0)
-  (exclude_from_sim no)
-  (in_bom yes)
-  (on_board yes)
-  (dnp no)
-  (property "Reference" "#FLG007" (at 650.24 72.39 0) (effects (font (size 1.27 1.27))))
-  (property "Value" "PWR_FLAG" (at 650.24 77.47 0) (effects (font (size 1.27 1.27))))
-  (property "Footprint" "" (at 650.24 74.93 0) (effects (font (size 1.27 1.27)) (hide yes)))
-  (property "Datasheet" "" (at 650.24 74.93 0) (effects (font (size 1.27 1.27)) (hide yes)))
-  (pin "1")
-  (instances
-    (project "ducktop2"
-      (path "/577b7ab7-60d3-5949-82f8-bb269dce837a"
-        (reference "#FLG007")
-        (unit 0)
-      )
-    )
-  )
-)
-(label "USB_PD_SELECTED"
-  (at 650.24 74.93 0)
-  (effects (font (size 1.27 1.27)) (justify left bottom))
-)
 (symbol
   (lib_id "power:PWR_FLAG")
@@
   (on_board yes)
   (dnp no)
-  (property "Reference" "#FLG008" (at 650.24 87.63 0) (effects (font (size 1.27 1.27))))
+  (property "Reference" "#FLG007" (at 650.24 87.63 0) (effects (font (size 1.27 1.27))))
   (property "Value" "PWR_FLAG" (at 650.24 92.71 0) (effects (font (size 1.27 1.27))))
   (property "Footprint" "" (at 650.24 90.17 0) (effects (font (size 1.27 1.27)) (hide yes)))
@@
     (project "ducktop2"
       (path "/577b7ab7-60d3-5949-82f8-bb269dce837a"
-        (reference "#FLG008")
+        (reference "#FLG007")
         (unit 0)
       )
@@
   (on_board yes)
   (dnp no)
-  (property "Reference" "#FLG009" (at 650.24 41.91 0) (effects (font (size 1.27 1.27))))
+  (property "Reference" "#FLG008" (at 650.24 41.91 0) (effects (font (size 1.27 1.27))))
   (property "Value" "PWR_FLAG" (at 650.24 46.99 0) (effects (font (size 1.27 1.27))))
   (property "Footprint" "" (at 650.24 44.45 0) (effects (font (size 1.27 1.27)) (hide yes)))
@@
     (project "ducktop2"
       (path "/577b7ab7-60d3-5949-82f8-bb269dce837a"
-        (reference "#FLG009")
+        (reference "#FLG008")
         (unit 0)
       )
@@
   (on_board yes)
   (dnp no)
-  (property "Reference" "#FLG010" (at 650.24 57.15 0) (effects (font (size 1.27 1.27))))
+  (property "Reference" "#FLG009" (at 650.24 57.15 0) (effects (font (size 1.27 1.27))))
   (property "Value" "PWR_FLAG" (at 650.24 62.23 0) (effects (font (size 1.27 1.27))))
   (property "Footprint" "" (at 650.24 59.69 0) (effects (font (size 1.27 1.27)) (hide yes)))
@@
     (project "ducktop2"
       (path "/577b7ab7-60d3-5949-82f8-bb269dce837a"
-        (reference "#FLG010")
+        (reference "#FLG009")
         (unit 0)
       )
@@
   (shape bidirectional)
   (at 654.05 345.44 0)
-  (effects (font (size 1.27 1.27)) (justify left bottom))
-)
-(symbol
-  (lib_id "Device:D_Schottky")
-  (at 650.24 355.6 0)
-  (unit 1)
-  (exclude_from_sim no)
-  (in_bom yes)
-  (on_board yes)
-  (dnp no)
-  (property "Reference" "D714" (at 650.24 353.06 0) (effects (font (size 1.27 1.27))))
-  (property "Value" "B340A 3A 40V EC always-on OR" (at 650.24 358.14 0) (effects (font (size 1.27 1.27))))
-  (property "Footprint" "Diode_SMD:D_SMA" (at 650.24 355.6 0) (effects (font (size 1.27 1.27)) (hide yes)))
-  (property "Datasheet" "" (at 650.24 355.6 0) (effects (font (size 1.27 1.27)) (hide yes)))
-  (property "Manufacturer" "Diodes Incorporated" (at 650.24 355.6 0) (effects (font (size 1.27 1.27)) (hide yes)))
-  (property "MPN" "B340A-13-F" (at 650.24 355.6 0) (effects (font (size 1.27 1.27)) (hide yes)))
-  (pin "1")
-  (pin "2")
-  (instances
-    (project "ducktop2"
-      (path "/577b7ab7-60d3-5949-82f8-bb269dce837a"
-        (reference "D714")
-        (unit 1)
-      )
-    )
-  )
-)
-(label "AON_OR_RAW"
-  (at 646.43 355.6 0)
-  (effects (font (size 1.27 1.27)) (justify left bottom))
-)
-(hierarchical_label "PD3_VBUS_RAW"
-  (shape bidirectional)
-  (at 654.05 355.6 0)
   (effects (font (size 1.27 1.27)) (justify left bottom))
 )
@@
   (on_board yes)
   (dnp no)
-  (property "Reference" "#FLG011" (at 650.24 367.03 0) (effects (font (size 1.27 1.27))))
+  (property "Reference" "#FLG010" (at 650.24 367.03 0) (effects (font (size 1.27 1.27))))
   (property "Value" "PWR_FLAG" (at 650.24 372.11 0) (effects (font (size 1.27 1.27))))
   (property "Footprint" "" (at 650.24 369.57 0) (effects (font (size 1.27 1.27)) (hide yes)))
@@
     (project "ducktop2"
       (path "/577b7ab7-60d3-5949-82f8-bb269dce837a"
-        (reference "#FLG011")
+        (reference "#FLG010")
         (unit 0)
       )
@@
 (text "No motherboard battery thermistors are fitted. U719 TS uses TI's 10k-to-VSS unused-function connection; VTB is NC." (at 20.32 243.84 0) (effects (font (size 1.27 1.27))))
 (text "BQ25798 /CE is fail-off: REGN pulls it high; active-high CHG_ENABLE turns Q700 on only after EC source validation." (at 20.32 250.19 0) (effects (font (size 1.27 1.27))))
-(text "U2 ILIM_HIZ divider is a 3.0A hardware ceiling; EC programs a lower IINDPM from the selected CH224A PDO current." (at 20.32 256.54 0) (effects (font (size 1.27 1.27))))
+(text "U2 ILIM_HIZ divider is a 3.0A hardware ceiling; EC programs a lower IINDPM from the selected TPS25751A Active PDO Contract (0x31)." (at 20.32 256.54 0) (effects (font (size 1.27 1.27))))
 (text "J190 is the one 7-22V nominal AUX/solar input; TPS26630 protects it before BQ25798." (at 20.32 264.16 0) (effects (font (size 1.27 1.27))))
 (text "Solar MPPT is implemented by BQ25798 firmware on this same input; there is no second charger path." (at 20.32 271.78 0) (effects (font (size 1.27 1.27))))
@@
 (text "U11 accepts about 8.45-13.57V nominal; 11mOhm RS10 gives 4.55A nominal and <=5.51A worst-case trips." (at 20.32 309.88 0) (effects (font (size 1.27 1.27))))
 (text "BQ25798 TS is fixed at 58.9% REGN by 5.24k/7.50k; firmware sets TS_IGNORE=1. BQ34Z100 TS has 10k to VSS; set TEMPS=0." (at 20.32 317.5 0) (effects (font (size 1.27 1.27))))
-(text "MANDATORY STARTUP: hold MU_12V_ENABLE low; require selected-source VALID; read CH224A PDO current; program VSYSMIN and IINDPM <= min(PDO-0.25A, 2.75A); require VSYS >=10.0V." (at 20.32 325.12 0) (effects (font (size 1.27 1.27))))
+(text "MANDATORY STARTUP: hold MU_12V_ENABLE low; read TPS25751A PD Status 0x35 plus Active PDO/RDO 0x31/0x32; program VSYSMIN and IINDPM <= min(PDO-0.25A, 2.75A); require VSYS >=10.0V." (at 20.32 325.12 0) (effects (font (size 1.27 1.27))))
 (text "Then assert MU_12V_ENABLE and require MU_12V_PG within 20ms. Any PG timeout, source-invalid, charger fault, watchdog fault, or VSYS<10V disables the Mu rail." (at 20.32 332.74 0) (effects (font (size 1.27 1.27))))
 (text "BQ25798 firmware must set STOP_WD_CHG=1 and TS_IGNORE=1, service faults, validate PDO current, and assert CHG_ENABLE only after safe limits are programmed." (at 20.32 340.36 0) (effects (font (size 1.27 1.27))))
 (text "U718 is the aggregate AON safety boundary: 1.51A typical limit, true reverse blocking, 6.20V nominal UVLO, and 22.40V nominal OVLO." (at 20.32 347.98 0) (effects (font (size 1.27 1.27))))
-(text "AON UVLO corners are 6.06-6.36V: default 5V USB-C is negotiation-only; CH224A must autonomously obtain its strapped 15V PDO before EC_AON_IN starts." (at 20.32 355.6 0) (effects (font (size 1.27 1.27))))
+(text "AON UVLO corners are 6.06-6.36V: default 5V USB-C is negotiation-only; TPS25751A dead-battery boot must obtain a valid higher-voltage PDO before EC_AON_IN starts." (at 20.32 355.6 0) (effects (font (size 1.27 1.27))))
 (text "A 5V-only USB-C source leaves the laptop off. AON_FAULT_N inhibits charging and Mu start; the service connector remains the assembly hard disconnect." (at 20.32 363.22 0) (effects (font (size 1.27 1.27))))
 (text "C746 provides low-ESR hold-up through LTC4418 break-before-make source switching." (at 20.32 370.84 0) (effects (font (size 1.27 1.27))))
