File: 01_power_battery.kicad_sch (KiCad schematic)
At the start: 167 parts, among them J190 AUX/SOLAR protected screw ter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, J2 3S pack power + cell-tap harn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, Q11 CSD18540Q5B reverse-pack FET A, Q12 CSD18540Q5B reverse-pack FET B, Q13 CSD19537Q3 100V AUX reverse F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, Q14 BSS138 fast reverse-gate pull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, Q21 SiSS4409DN 40V reverse-blocki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, Q22 SiSS4409DN 40V reverse-blocki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, Q23 SiSS4409DN 40V reverse-blocki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, Q24 SiSS4409DN 40V reverse-blocki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, Q25 CSD17575Q3 BQ25798 ship FET, Q700 BSS138 active-high charger en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, Q701 BSS138 pack protector latch r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, Q702 BSS138 QON open-drain pulse, Q703 CSD18540Q5B BQ77915 discharge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, Q704 CSD18540Q5B BQ77915 charge FET, U10 BQ34Z100-G1 protected-pack ga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, U11 LTC4368IMS-1 bidirectional pa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, U12 TPS26630RGER 3A AUX eFuse / s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, U15 LTC4418IUF#PBF dual-input sel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, U2 BQ25798RQMR, U718 TPS259470ARPW aggregate EC AO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, U719 BQ7791500PWR autonomous 3S pr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

Commit message: Stamp generation-time BOM catalog; close 378 procurement gaps
Parts:
- C10, C11, C180, C181, C182, C192, C721, C723, C796, C798, C845, C846, C847: MPN (none) -> GRM188R71H104KA93D; Manufacturer (none) -> Murata
- C183, C841, C842, C843, C844, C848: MPN (none) -> GRM21BR71A105KA01L; Manufacturer (none) -> Murata
- C700, C799: MPN (none) -> GRM155R71H332KA01; Manufacturer (none) -> Murata
- C720: MPN (none) -> GRM21BR71H105KA01; Manufacturer (none) -> Murata
- C724: MPN (none) -> GRM155R71H472KA01; Manufacturer (none) -> Murata
- C795, C840: MPN (none) -> GRM21BR71H105KA12L; Manufacturer (none) -> Murata
- C797: MPN (none) -> GRM31CR71E106KA12L; Manufacturer (none) -> Murata
- R12, R193, R840, R848: MPN (none) -> RC0603FR-071KL; Manufacturer (none) -> Yageo
- R14, R15, R185, R186, R708, R715, R716, R717, R718, R852, R853, R855: MPN (none) -> RC0603FR-0710KL; Manufacturer (none) -> Yageo
- R16: MPN (none) -> RC0603FR-075K24L; Manufacturer (none) -> Yageo
- R18: MPN (none) -> RC0603FR-0710K5L; Manufacturer (none) -> Yageo
- R180: MPN (none) -> RT0603BRD07220KL; Manufacturer (none) -> Yageo
- R181: MPN (none) -> RT0603BRD0716K5L; Manufacturer (none) -> Yageo
- R182, R183, R184, R704, R845, R846: MPN (none) -> RC0603FR-07100RL; Manufacturer (none) -> Yageo
- R189: MPN (none) -> RC0603FR-070RL; Manufacturer (none) -> Yageo
- R191: MPN (none) -> RC0603FR-07470KL; Manufacturer (none) -> Yageo
- R192: MPN (none) -> RC0603FR-0756KL; Manufacturer (none) -> Yageo
- R30, R31: MPN (none) -> RC0603FR-074K7L; Manufacturer (none) -> Yageo
- R700: MPN (none) -> RC0603FR-073M09L; Manufacturer (none) -> Yageo
- R701: MPN (none) -> RC0603FR-0773K2L; Manufacturer (none) -> Yageo
- R702: MPN (none) -> RC0603FR-07121KL; Manufacturer (none) -> Yageo
- R703: MPN (none) -> RC0603FR-0722KL; Manufacturer (none) -> Yageo
- R705: MPN (none) -> RC0603FR-077K50L; Manufacturer (none) -> Yageo
- R706: MPN (none) -> RC0603FR-072RL; Manufacturer (none) -> Yageo
- R707, R709, R719: MPN (none) -> RC0603FR-07100KL; Manufacturer (none) -> Yageo
- R710: MPN (none) -> RC0603FR-076K04L; Manufacturer (none) -> Yageo
- R711: MPN (none) -> RT0603BRD07300KL; Manufacturer (none) -> Yageo
- R712: MPN (none) -> RT0603BRD0763K2L; Manufacturer (none) -> Yageo
- R713: MPN (none) -> RT0603BRD0720K0L; Manufacturer (none) -> Yageo
- R714: MPN (none) -> RC0603FR-0731RL; Manufacturer (none) -> Yageo
- R798: MPN (none) -> RT0603BRD072K21L; Manufacturer (none) -> Yageo
- R841, R842, R843, R844: MPN (none) -> RC0603FR-0775RL; Manufacturer (none) -> Yageo
- R847: MPN (none) -> RC0603FR-074K53L; Manufacturer (none) -> Yageo
- R849: MPN (none) -> RC0603FR-071ML; Manufacturer (none) -> Yageo
- R850: MPN (none) -> RC0603FR-073M3L; Manufacturer (none) -> Yageo
- R851: MPN (none) -> RC0603FR-07453KL; Manufacturer (none) -> Yageo
- R854: MPN (none) -> RC0603FR-07604KL; Manufacturer (none) -> Yageo

Commit message: Board split Phase 2.4: trim center board, FPC boundary contracts, per-project verification
Center (ducktop2) loses the four sheets that moved to the daughterboards:
04_usb_c_io, 05_power_inputs, 06_tcp0_external_hdmi, 16_gigabit_ethernet,
and the pack-protection section of 01_power_battery (BMS board). J190 AUX
terminal moves to the left board. Center keeps 9 sheets: charger/gauge/
ship-FET (U2/U10/Q25/RS1), EC, Mu, radio, internal, radio-DB, keyboard x2,
maker, audio. 717 components.

FPC-1/2/3 boundary contracts declare the crossing nets at the center root
(30 + 35 + 4 shared nets; HUB_DS1_DP/DM are center pass-throughs).

Verification is now per-project:
- verify_design_contracts.py --project {ducktop2,left_io,right_io,bms}
  (five-port USB-C contracts split by port, HDMI/GbE run on right_io,
  pack contracts run on bms, sheet names parameterized)
- verify_schematic_closure.py --pack audits the BMS pack block
- verify_electrical_calculations.py --project bms for pack calcs
- pin review trimmed to center parts; FPC-boundary nets in ERC allowlist

Fixed while trimming: daughterboard root labels now sit on sheet-block pin
endpoints (left/right FPC nets actually connect); duplicate GND pwrflag in
power sheet; sync.parse_netlist respects the radio-daughterboard override.

Schematic gate PASS: self-check, closure audits (89+151), electrical
calcs (67+15), pin review (1625), identity.
Parts:
- removed C181: 100n sense filter, Capacitor_SMD:C_0603_1608Metric, symbol Device:C
- removed C182: 100n REGIN/VCC, Capacitor_SMD:C_0603_1608Metric, symbol Device:C
- removed C183: 1u REG25, Capacitor_SMD:C_0805_2012Metric, symbol Device:C
- removed C700: 3.3nF >=50V LTC4368 CGATE, Capacitor_SMD:C_0402_1005Metric, symbol Device:C
- removed C701, C702: 10u 25V X7R VBUS, Capacitor_SMD:C_1206_3216Metric, symbol Device:C
- removed C724: 4.7nF >=50V pack hot-swap slew, Capacitor_SMD:C_0402_1005Metric, symbol Device:C
- removed C725: 10u 25V X7R LTC4368 VOUT, Capacitor_SMD:C_0805_2012Metric, symbol Device:C
- removed C844, C848: 1u 10V X7R BQ77915 internal-balance filter, Capacitor_SMD:C_0805_2012Metric, symbol Device:C
- removed C845: 100n BQ77915 SRP-VSS filter, Capacitor_SMD:C_0603_1608Metric, symbol Device:C
- removed C846: 100n BQ77915 differential sense filter, Capacitor_SMD:C_0603_1608Metric, symbol Device:C
- removed C847: 100n BQ77915 SRN-VSS filter, Capacitor_SMD:C_0603_1608Metric, symbol Device:C
- removed D713: B340A 3A 40V EC always-on OR, Diode_SMD:D_SMA, symbol Device:D_Schottky
- removed D715: BAT54WS case button to charger QON, Diode_SMD:D_SOD-323, symbol Device:D_Schottky
- removed D716: BAT54WS case button to Mu PWRBTN, Diode_SMD:D_SOD-323, symbol Device:D_Schottky
- removed F1: 10A MINI pack fuse: Littelfuse 0297010.WXNV, Fuse:Fuseholder_Blade_Mini_Keystone_3568, symbol Device:Fuse
- removed J190: AUX/SOLAR protected screw terminal 6-22V nominal, TerminalBlock_Phoenix:TerminalBlock_Phoenix_MKDS-1,5-2-5.08_1x02_P5.08mm_Horizontal, symbol Connector_Generic:Conn_01x02
- removed J2: 3S pack power + cell-tap harness, Connector_Molex:Molex_Mega-Fit_76829-0006_2x03_P5.70mm_Vertical, symbol Connector_Generic:Conn_02x03_Odd_Even
- removed Q11: CSD18540Q5B reverse-pack FET A, ducktop2:CSD18540Q5B_DNK, symbol Q_NMOS_123S_4G_5678D:Q_NMOS_123S_4G_5678D
- removed Q703: CSD18540Q5B BQ77915 discharge FET, ducktop2:CSD18540Q5B_DNK, symbol Q_NMOS_123S_4G_5678D:Q_NMOS_123S_4G_5678D
- removed Q704: CSD18540Q5B BQ77915 charge FET, ducktop2:CSD18540Q5B_DNK, symbol Q_NMOS_123S_4G_5678D:Q_NMOS_123S_4G_5678D
- removed R14: 10k CE hardware-disable pull-up to REGN, Resistor_SMD:R_0603_1608Metric, symbol Device:R
- removed R183: 100R SRP filter, Resistor_SMD:R_0603_1608Metric, symbol Device:R
- removed R184: 100R SRN filter, Resistor_SMD:R_0603_1608Metric, symbol Device:R
- removed R185: 10k CE pull-up, Resistor_SMD:R_0603_1608Metric, symbol Device:R
- removed R189: 0R P1 not-used tie to VSS, Resistor_SMD:R_0603_1608Metric, symbol Device:R
- removed R31: 4.7k I2C SDA pull-up to 3V3, Resistor_SMD:R_0603_1608Metric, symbol Device:R
- removed R700: 3.09M 1% BAT UV/OV top, Resistor_SMD:R_0603_1608Metric, symbol Device:R
- removed R701: 73.2k 1% BAT UV/OV middle, Resistor_SMD:R_0603_1608Metric, symbol Device:R
- removed R702: 121k 1% BAT UV/OV bottom, Resistor_SMD:R_0603_1608Metric, symbol Device:R
- removed R703: 22k LTC4368 CGATE series, Resistor_SMD:R_0603_1608Metric, symbol Device:R
- removed R704: 100R BATP Kelvin filter, Resistor_SMD:R_0603_1608Metric, symbol Device:R
- removed R709: 100k pack retry gate pulldown, Resistor_SMD:R_0603_1608Metric, symbol Device:R
- removed R845: 100R BQ77915 SRP filter, Resistor_SMD:R_0603_1608Metric, symbol Device:R
- removed R846: 100R BQ77915 SRN filter, Resistor_SMD:R_0603_1608Metric, symbol Device:R
- removed R847: 4.53k 1% DSG gate resistor, Resistor_SMD:R_0603_1608Metric, symbol Device:R
- removed R848: 1k 1% CHG gate resistor, Resistor_SMD:R_0603_1608Metric, symbol Device:R
- removed R849: 1M 5% DSG gate-source, Resistor_SMD:R_0603_1608Metric, symbol Device:R
- removed R850: 3.3M 5% CHG gate-source, Resistor_SMD:R_0603_1608Metric, symbol Device:R
- removed R851: 453k 1% load-detect resistor, Resistor_SMD:R_0603_1608Metric, symbol Device:R
- removed R852: 10k 5% PRES normal-mode pull-up, Resistor_SMD:R_0603_1608Metric, symbol Device:R
- removed R853: 10k 1% unused TS to VSS, Resistor_SMD:R_0603_1608Metric, symbol Device:R
- removed R855: 10k unused external TS pulldown, Resistor_SMD:R_0603_1608Metric, symbol Device:R
- removed RS10: 11mOhm 1% 2W LTC4368 bounded pack-current shunt, Resistor_SMD:R_2512_6332Metric, symbol Device:R
- removed RS11: 8mOhm 1% 2W BQ77915 current shunt, Resistor_SMD:R_2512_6332Metric, symbol Device:R
- removed TP4: EC_AON_IN test, TestPoint:TestPoint_Pad_D1.0mm, symbol Connector:TestPoint
- removed U12: TPS26630RGER 3A AUX eFuse / surge cutoff, Package_DFN_QFN:Texas_RGE0024H_VQFN-24-1EP_4x4mm_P0.5mm_EP2.7x2.7mm_ThermalVias, symbol Power_Management:TPS26630RGE
- removed U15: LTC4418IUF#PBF dual-input selector, ducktop2:ADI_UF20_QFN20_4x4_P0.5_EP2.45, symbol LTC4418IUF:LTC4418IUF
- removed U719: BQ7791500PWR autonomous 3S primary protector, Package_SO:TSSOP-24_4.4x7.8mm_P0.65mm, symbol BQ77915:BQ77915
- added C721: 100n 50V X7R AUX eFuse local, Capacitor_SMD:C_0603_1608Metric, symbol Device:C
- added Q14: BSS138 fast reverse-gate pulldown, Package_TO_SOT_SMD:SOT-23, symbol Q_NMOS_SOT23_GSD:Q_NMOS_SOT23_GSD
- added Q700: BSS138 active-high charger enable pull-down, Package_TO_SOT_SMD:SOT-23, symbol Q_NMOS_SOT23_GSD:Q_NMOS_SOT23_GSD
- added RS1: 5mOhm 1% 2W BQ34Z100 Kelvin shunt, Resistor_SMD:R_2512_6332Metric, symbol Device:R
- C181: renamed from C841; value 1u 10V X7R BQ77915 AVDD -> 100n sense filter; footprint Capacitor_SMD:C_0805_2012Metric -> Capacitor_SMD:C_0603_1608Metric; MPN GRM21BR71A105KA01L -> GRM188R71H104KA93D
- C182: renamed from R843; value 75R 1% BQ77915 cell/balance filter -> 100n REGIN/VCC; footprint Resistor_SMD:R_0603_1608Metric -> Capacitor_SMD:C_0603_1608Metric; symbol Device:R -> Device:C; MPN RC0603FR-0775RL -> GRM188R71H104KA93D; Manufacturer Yageo -> Murata
- C183: renamed from R844; value 75R 1% BQ77915 cell/balance filter -> 1u REG25; footprint Resistor_SMD:R_0603_1608Metric -> Capacitor_SMD:C_0805_2012Metric; symbol Device:R -> Device:C; MPN RC0603FR-0775RL -> GRM21BR71A105KA01L; Manufacturer Yageo -> Murata
- C701: renamed from R708; value 10k pack FAULT pull-up -> 10u 25V X7R VBUS; footprint Resistor_SMD:R_0603_1608Metric -> Capacitor_SMD:C_1206_3216Metric; symbol Device:R -> Device:C; MPN RC0603FR-0710KL -> GRM31CR71E106KA12L; Manufacturer Yageo -> Murata
- C702: renamed from Q701; value BSS138 pack protector latch reset -> 10u 25V X7R VBUS; footprint Package_TO_SOT_SMD:SOT-23 -> Capacitor_SMD:C_1206_3216Metric; symbol Q_NMOS_SOT23_GSD:Q_NMOS_SOT23_GSD -> Device:C; MPN BSS138LT1G -> GRM31CR71E106KA12L; Manufacturer onsemi -> Murata
- D713: renamed from Q14; value BSS138 fast reverse-gate pulldown -> B340A 3A 40V EC always-on OR; footprint Package_TO_SOT_SMD:SOT-23 -> Diode_SMD:D_SMA; symbol Q_NMOS_SOT23_GSD:Q_NMOS_SOT23_GSD -> Device:D_Schottky; MPN BSS138LT1G -> B340A-13-F; Manufacturer onsemi -> Diodes Incorporated
- D715: renamed from R854; value 604k 1% OCD delay program -> BAT54WS case button to charger QON; footprint Resistor_SMD:R_0603_1608Metric -> Diode_SMD:D_SOD-323; symbol Device:R -> Device:D_Schottky; MPN RC0603FR-07604KL -> BAT54WS-7-F; Manufacturer Yageo -> Diodes Incorporated
- D716: renamed from RS1; value 5mOhm 1% 2W BQ34Z100 Kelvin shunt -> BAT54WS case button to Mu PWRBTN; footprint Resistor_SMD:R_2512_6332Metric -> Diode_SMD:D_SOD-323; symbol Device:R -> Device:D_Schottky; MPN WSLP2512R0050FEA -> BAT54WS-7-F; Manufacturer Vishay Dale -> Diodes Incorporated
- R14: renamed from U11; value LTC4368IMS-1 bidirectional pack protector -> 10k CE hardware-disable pull-up to REGN; footprint Package_SO:MSOP-10_3x3mm_P0.5mm -> Resistor_SMD:R_0603_1608Metric; symbol LTC4368-1:LTC4368-1 -> Device:R; MPN LTC4368IMS-1#PBF -> RC0603FR-0710KL; Manufacturer Analog Devices -> Yageo
- R183: renamed from R840; value 1k 1% BQ77915 VDD filter -> 100R SRP filter; MPN RC0603FR-071KL -> RC0603FR-07100RL
- R184: renamed from C840; value 1u 25V X7R BQ77915 VDD -> 100R SRN filter; footprint Capacitor_SMD:C_0805_2012Metric -> Resistor_SMD:R_0603_1608Metric; symbol Device:C -> Device:R; MPN GRM21BR71H105KA12L -> RC0603FR-07100RL; Manufacturer Murata -> Yageo
- R185: renamed from R841; value 75R 1% BQ77915 cell/balance filter -> 10k CE pull-up; MPN RC0603FR-0775RL -> RC0603FR-0710KL
- R186: renamed from R842; value 75R 1% BQ77915 cell/balance filter -> 10k gauge ALERT pull-up; MPN RC0603FR-0775RL -> RC0603FR-0710KL
- R189: renamed from C842; value 1u 10V X7R BQ77915 internal-balance filter -> 0R P1 not-used tie to VSS; footprint Capacitor_SMD:C_0805_2012Metric -> Resistor_SMD:R_0603_1608Metric; symbol Device:C -> Device:R; MPN GRM21BR71A105KA01L -> RC0603FR-070RL; Manufacturer Murata -> Yageo
- R31: renamed from Q12; value CSD18540Q5B reverse-pack FET B -> 4.7k I2C SDA pull-up to 3V3; footprint ducktop2:CSD18540Q5B_DNK -> Resistor_SMD:R_0603_1608Metric; symbol Q_NMOS_123S_4G_5678D:Q_NMOS_123S_4G_5678D -> Device:R; MPN CSD18540Q5B -> RC0603FR-074K7L; Manufacturer Texas Instruments -> Yageo
- R704: renamed from R707; value 100k pack protector SHDN pull-up -> 100R BATP Kelvin filter; MPN RC0603FR-07100KL -> RC0603FR-07100RL
- R855: renamed from C843; value 1u 10V X7R BQ77915 internal-balance filter -> 10k unused external TS pulldown; footprint Capacitor_SMD:C_0805_2012Metric -> Resistor_SMD:R_0603_1608Metric; symbol Device:C -> Device:R; MPN GRM21BR71A105KA01L -> RC0603FR-0710KL; Manufacturer Murata -> Yageo
- TP4: renamed from C721; value 100n 50V X7R AUX eFuse local -> EC_AON_IN test; footprint Capacitor_SMD:C_0603_1608Metric -> TestPoint:TestPoint_Pad_D1.0mm; symbol Device:C -> Connector:TestPoint; MPN GRM188R71H104KA93D -> (none); Manufacturer Murata -> (none); ProcurementClass (none) -> PCB copper test feature; now left out of the parts list
- U12: renamed from R186; value 10k gauge ALERT pull-up -> TPS26630RGER 3A AUX eFuse / surge cutoff; footprint Resistor_SMD:R_0603_1608Metric -> Package_DFN_QFN:Texas_RGE0024H_VQFN-24-1EP_4x4mm_P0.5mm_EP2.7x2.7mm_ThermalVias; symbol Device:R -> Power_Management:TPS26630RGE; MPN RC0603FR-0710KL -> TPS26630RGER; Manufacturer Yageo -> Texas Instruments
- U15: renamed from Q700; value BSS138 active-high charger enable pull-down -> LTC4418IUF#PBF dual-input selector; footprint Package_TO_SOT_SMD:SOT-23 -> ducktop2:ADI_UF20_QFN20_4x4_P0.5_EP2.45; symbol Q_NMOS_SOT23_GSD:Q_NMOS_SOT23_GSD -> LTC4418IUF:LTC4418IUF; MPN BSS138LT1G -> LTC4418IUF#PBF; Manufacturer onsemi -> Analog Devices
Connections:
- net BAT_PROT_UV is gone; now on net CHG_CE_HW_N: R14.2
- net BMS_AVDD is gone; now on net FG_SRP: C181.1
- net BMS_OCDP is gone; now on net CASE_PWRBTN_N: D715.1 (K)
- net BMS_VC2 is gone; now on net FG_VSS: C182.2
- net BMS_VC3_TOP is gone; now on net FG_VSS: C183.2
- net CELL1_TAP is gone; now on net MCU_3V3: R186.1
- net CELL2_TAP is gone; now on net MCU_3V3: C182.1
- net PACK_RETRY_PULSE is gone; now on net VBUS_COMBINED: C702.1
- net AON_OR_RAW: now also D713.1 (K)
- net AUX_DC_FUSED: now also U12.1 (IN), U12.2 (IN)
- net AUX_DC_PROTECTED: now also U12.17 (OUT), U12.18 (OUT), U15.16 (V2)
- net AUX_EFUSE_BGATE: now also U12.3 (B_GATE), Q14.3 (D); no longer D713.3 (D)
- net AUX_EFUSE_DRV: now also U12.4 (DRV)
- net AUX_EFUSE_DVDT: now also U12.9 (dVdT)
- net AUX_EFUSE_ILIM: now also U12.10 (ILIM)
- net AUX_EFUSE_IN_SYS: now also U12.5 (IN_SYS), C721.1, Q14.2 (S); no longer D713.2 (S), TP4.1
- net AUX_EFUSE_OV: now also U12.7 (OVP)
- net AUX_EFUSE_Q2_GATE: now also Q14.1 (G); no longer D713.1 (G)
- net AUX_EFUSE_UV: now also U12.6 (UVLO)
- net AUX_FAULT_N: now also U12.14 (~{FLT})
- net AUX_MAIN_FET_COMMON: now also U15.12 (VS2)
- net AUX_MAIN_GATE: now also U15.11 (G2)
- net AUX_MAIN_OV: now also U15.5 (OV2)
- net AUX_MAIN_UV: now also U15.4 (UV2)
- net AUX_PGOOD: now also U12.16 (PGOOD)
- net AUX_PGTH: now also U12.15 (PGTH)
- net BATP_SENSE: now also R704.2
- net BAT_PROT_VIN: no longer R14.1 (VIN), R704.1
- net BQ_ALERT: now also R186.2; no longer U12.2
- net CASE_PWRBTN_N: now also D716.1 (K)
- net CHG_CE_HW_N: now also Q700.3 (D); no longer U15.3 (D)
- net CHG_ENABLE: now also Q700.1 (G); no longer U15.1 (G)
- net EC_AON_IN: now also TP4.1
- net FG_CE: now also R185.2
- net FG_P1_TIE: now also R189.1
- net FG_REG25: now also C183.1
- net FG_SRN: now also C181.2, R184.2
- net FG_SRP: now also R183.2
- net FG_TS: now also R855.1
- net FG_VSS: now also R183.1, R189.2, R855.2, RS1.1; no longer D716.1
- net GND: now also C701.2, R184.1, U12.11 (MODE), U12.25 (GND), U12.8 (GND), U15.20 (HYS), U15.21 (EP/GND), U15.7 (GND), C721.2, Q700.2 (S), RS1.2; no longer D716.2, R14.4 (RETRY), R14.5 (GND), TP4.2, U15.2 (S)
- net I2C_SDA: now also R31.2
- net MAIN_AUX_VALID_N: now also U15.10 (~{VALID2})
- net MAIN_SEL_INTVCC: now also U15.18 (EN), U15.19 (~{SHDN}), U15.8 (INTVCC)
- net MAIN_SEL_TMR: now also U15.1 (TMR)
- net MAIN_USB_VALID_N: now also U15.9 (~{VALID1})
- net MCU_3V3: now also R185.1, R31.1; no longer C701.1, U12.1
- net MU_PWRBTN_N: now also D716.2 (A)
- net PACK_FAULT_N: no longer C701.2, R14.7 (FAULT)
- net PACK_POS_FUSED: now also R704.1; no longer R14.8 (VOUT)
- net PD2_VBUS_RAW: now also D713.2 (A)
- net PMIC_QON_PIN: now also D715.2 (A)
- net REGN: now also R14.1
- net USB_MAIN_FET_COMMON: now also U15.14 (VS1)
- net USB_MAIN_GATE: now also U15.13 (G1)
- net USB_MAIN_OV: now also U15.3 (OV1)
- net USB_MAIN_UV: now also U15.2 (UV1)
- net USB_PD_SELECTED: now also U15.17 (V1)
- net VBUS_COMBINED: now also C701.1, U15.15 (VOUT)
- removed net BAT_PROT_FET_COMMON: R31.1 (S), R31.2 (S), R31.3 (S)
- removed net BAT_PROT_GATE: R14.10 (GATE), R31.4 (G)
- removed net BAT_PROT_OV: R14.3 (OV)
- removed net BAT_PROT_SENSE: R14.9 (SENSE), R31.5 (D(5-8))
- removed net BAT_PROT_SHDN: C702.3 (D), R14.6 (SHDN), R704.2
- removed net BMS_VC0: R185.2, R189.1, R855.2
- removed net BMS_VC1: R186.2, R855.1
- removed net BMS_VDD: R183.2, R184.1
- removed net PACK_NEG_RAW: C181.2, D715.2, R184.2, R185.1, R189.2
- removed net PACK_POS_RAW: C183.1, R183.1
- no-connect marks 18 -> 15
Other:
- note added: "FPC-3 to BMS: PACK_POS_FUSED / PACK_FAULT_N / PACK_RETRY_PULSE cross here"
- note removed: "== 3S cell entry, autonomous primary protection, fuse and redundant pack protection =="
- moved on the sheet: C181, R183, R185, R186, R704

Commit message: Board split Phase 4a: FPC connectors wired through the four split schematics
Connector symbols and sheets now exist in every project and the boundary
nets are pinned through them (same conductor order on both ends, verified
netlist-by-netlist):
  - gen/fpc_contract.py: authoritative FPC-1/2/3 pin maps + center-side
    renames (single source of truth for schematics, board pad nets, cable
    spec, and gate contracts)
  - gen/Conn_01x100_FFC_MP.kicad_sym (derived from the 30-pin pattern)
  - center: real fpc1_left/fpc2_right/fpc3_bms sheets wired to host pins
  - left_io/right_io: left_fpc/right_fpc connector sheets; bms carries
    FPC106 inline
  - connector refs FPC101..FPC106 (valid designators; FPC1_L-style refs
    broke KiCad annotation)
  - pack-rail naming reconciled: center gauge divider BAT_PROT_VIN ->
    PACK_POS_FUSED (same node as the BMS LTC4368 output); BMS ground
    /GND -> GND (pack negative is the system ground)

Boards: daughterboards re-synced from their connector-bearing schematics;
center connectors placed and their pad nets assigned text-side ((net
"name") convention).  Connector pads verified against every other
footprint (0 overlaps) and DRC shows 0 shorts on all four boards (center
16 pre-existing, down from 17).

Fixed two latent generator bugs exposed by the wiring:
  - resolve_connectors used naive +R rotation, placing Phase 3 connectors
    against mirrored phantom positions
  - pad half-extents were computed as footprint_rot+pad_rot, but KiCad
    saves pads with world orientation (FH12-100S pins are 1.3mm wide);
    both verified empirically against pcbnew, plus a connector-nudge pass
    for parts sandwiched between the connector body and pin columns

Gate: SCHEMATIC RELEASE CHECK: PASS (FPC pin contracts added per project;
closure audits 0 FAIL).  Routing remains manual (Phase 4b).
Connections:
- net BAT_PROT_VIN is gone; now on net PACK_POS_FUSED: R180.1
Changed lines of the file:
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@@
   )
 )
-(label "BAT_PROT_VIN"
+(label "PACK_POS_FUSED"
   (at 650.24 30.48 0)
   (effects (font (size 1.27 1.27)) (justify left bottom))
@@
   )
 )
-(label "BAT_PROT_VIN"
+(hierarchical_label "PACK_POS_FUSED"
+  (shape bidirectional)
   (at 170.18 146.05 0)
   (effects (font (size 1.27 1.27)) (justify left bottom))

Commit message: Phase 5: second-opinion audit remediation + rebuilt, verified board pipeline
Second-opinion AI audit found A-tier defects; remediation applied and the
board pipeline rebuilt on a known-good base with the fixes it needed:

- electrical: LTC4418IUF symbol pinout corrected (both selectors were
  dead as drawn); center charge cascade (U15 <- U15B, PD1 > PD2 > AUX);
  pack negative never crosses FPC-3, 15-pin FG_VSS return; power-budgeted
  FPC pin maps (0.4 A/pin derate); J12/DS4 completed; AUX source fuse
- FH41-68S footprint: 13 datasheet-correct SH pads + SH pin in symbol
- connector geometry settled against the Hirose FH12 2D drawing: FFC
  enters opposite the solder pins (mouth = local +Y); reversed side-B
  maps are correct for the 180-deg-mounted pairs; rotations set so mouths
  face across every seam
- pipeline (generate_split_boards.py): per-pin pad-net resync from the
  netlists (kills shadow nets for good), netlist-exact name
  normalization, netlist-only part injection (cascade, probe headers),
  zone refill after outline swap, read-before-write race fixed, orphan
  parts dropped loudly, non-zero exit on unresolved overlaps
- monolith board relocated to old/monolith_ducktop2.kicad_pcb (placement
  oracle for the center cut only)

verified end state: 4 boards 0 shorts / 0 clearance / 0 drill, 0 boundary
crossings, 6/6 connectors contract-exact with mouths facing, 0 shadow
nets, gates PASS x4, ERC 0 x4. routing next (499 nets/board).
Parts:
- removed Q22, Q23: SiSS4409DN 40V reverse-blocking PMOS, Package_SO:Vishay_PowerPAK_1212-8_Single, symbol Q_PMOS_1G_234S_5D:Q_PMOS_1G_234S_5D
- removed R730: 1.00M 0.1% USB UV top, Resistor_SMD:R_0603_1608Metric, symbol Device:R
- removed R731: 19.6k 0.1% USB window middle, Resistor_SMD:R_0603_1608Metric, symbol Device:R
- added C747: 100n 50V stage2 VS1 local, Capacitor_SMD:C_0603_1608Metric, symbol Device:C
- added C748: 100n 50V stage2 out local, Capacitor_SMD:C_0603_1608Metric, symbol Device:C
- added C749: 100n 10V stage2 INTVCC, Capacitor_SMD:C_0603_1608Metric, symbol Device:C
- added D710, D711, D712, D713: B340A 3A 40V EC always-on OR, Diode_SMD:D_SMA, symbol Device:D_Schottky
- added Q21, Q26, Q27, Q28, Q29: SiSS4409DN 40V reverse-blocking PMOS, Package_SO:Vishay_PowerPAK_1212-8_Single, symbol Q_PMOS_1G_234S_5D:Q_PMOS_1G_234S_5D
- added R718: 10k main AUX VALID pull-up, Resistor_SMD:R_0603_1608Metric, symbol Device:R
- added R743: 63.4k 0.1% PD2 OV bottom, Resistor_SMD:R_0603_1608Metric, symbol Device:R
- added R744: 374k 0.1% stage2 UV top, Resistor_SMD:R_0603_1608Metric, symbol Device:R
- added R745: 54.9k 0.1% stage2 window middle, Resistor_SMD:R_0603_1608Metric, symbol Device:R
- added R746: 20.0k 0.1% stage2 OV bottom, Resistor_SMD:R_0603_1608Metric, symbol Device:R
- added R747: 10k PD2 VALID pull-up, Resistor_SMD:R_0603_1608Metric, symbol Device:R
- added TP3: VSYS test, TestPoint:TestPoint_Pad_D1.0mm, symbol Connector:TestPoint
- added U718: TPS259470ARPW aggregate EC AON eFuse, ducktop2:Texas_RPW0010A_VQFN-HR-10_2x2mm, symbol TPS259470A:TPS259470A
- C715: renamed from TP3; value VSYS test -> 15n 50V stage2 TMR approx 240ms; footprint TestPoint:TestPoint_Pad_D1.0mm -> Capacitor_SMD:C_0402_1005Metric; symbol Connector:TestPoint -> Device:C; MPN (none) -> GRM155R71H153KA12D; Manufacturer (none) -> Murata; ProcurementClass PCB copper test feature -> (none); now in the parts list
- C744: value 100n 50V AUX V2 local -> 100n 50V stage2 V2 local
- Q22: renamed from R732; value 63.4k 0.1% USB OV bottom -> SiSS4409DN 40V reverse-blocking PMOS; footprint Resistor_SMD:R_0603_1608Metric -> Package_SO:Vishay_PowerPAK_1212-8_Single; symbol Device:R -> Q_PMOS_1G_234S_5D:Q_PMOS_1G_234S_5D; MPN RT0603BRD0763K4L -> SiSS4409DN-T1-GE3; Manufacturer Yageo -> Vishay
- Q23: renamed from R718; value 10k main AUX VALID pull-up -> SiSS4409DN 40V reverse-blocking PMOS; footprint Resistor_SMD:R_0603_1608Metric -> Package_SO:Vishay_PowerPAK_1212-8_Single; symbol Device:R -> Q_PMOS_1G_234S_5D:Q_PMOS_1G_234S_5D; MPN RC0603FR-0710KL -> SiSS4409DN-T1-GE3; Manufacturer Yageo -> Vishay
- Q25: footprint ducktop2:CSD19537Q3_DQG -> ducktop2:CSD17575Q3_DQG
- R730: renamed from D710; value B340A 3A 40V EC always-on OR -> 1.00M 0.1% USB UV top; footprint Diode_SMD:D_SMA -> Resistor_SMD:R_0603_1608Metric; symbol Device:D_Schottky -> Device:R; MPN B340A-13-F -> RT0603BRD071ML; Manufacturer Diodes Incorporated -> Yageo
- R731: renamed from D711; value B340A 3A 40V EC always-on OR -> 19.6k 0.1% USB window middle; footprint Diode_SMD:D_SMA -> Resistor_SMD:R_0603_1608Metric; symbol Device:D_Schottky -> Device:R; MPN B340A-13-F -> RT0603BRD0719K6L; Manufacturer Diodes Incorporated -> Yageo
- R732: renamed from D712; value B340A 3A 40V EC always-on OR -> 63.4k 0.1% USB OV bottom; footprint Diode_SMD:D_SMA -> Resistor_SMD:R_0603_1608Metric; symbol Device:D_Schottky -> Device:R; MPN B340A-13-F -> RT0603BRD0763K4L; Manufacturer Diodes Incorporated -> Yageo
- R741: renamed from D713; value B340A 3A 40V EC always-on OR -> 1.00M 0.1% PD2 UV top; footprint Diode_SMD:D_SMA -> Resistor_SMD:R_0603_1608Metric; symbol Device:D_Schottky -> Device:R; MPN B340A-13-F -> RT0603BRD071ML; Manufacturer Diodes Incorporated -> Yageo
- R742: renamed from U718; value TPS259470ARPW aggregate EC AON eFuse -> 19.6k 0.1% PD2 window middle; footprint ducktop2:Texas_RPW0010A_VQFN-HR-10_2x2mm -> Resistor_SMD:R_0603_1608Metric; symbol TPS259470A:TPS259470A -> Device:R; MPN TPS259470ARPW -> RT0603BRD0719K6L; Manufacturer Texas Instruments -> Yageo
- U15: value LTC4418IUF#PBF dual-input selector -> LTC4418IUF#PBF dual-input selector (stage 1)
- U15B: renamed from Q21; value SiSS4409DN 40V reverse-blocking PMOS -> LTC4418IUF#PBF dual-input selector (stage 2); footprint Package_SO:Vishay_PowerPAK_1212-8_Single -> ducktop2:ADI_UF20_QFN20_4x4_P0.5_EP2.45; symbol Q_PMOS_1G_234S_5D:Q_PMOS_1G_234S_5D -> LTC4418IUF:LTC4418IUF; MPN SiSS4409DN-T1-GE3 -> LTC4418IUF#PBF; Manufacturer Vishay -> Analog Devices
Connections:
- net AON_EFUSE_DVDT: now also U718.7 (dVdt); no longer R742.7 (dVdt)
- net AON_EFUSE_ILM: now also U718.9 (ILM); no longer R742.9 (ILM)
- net AON_EFUSE_OV: now also U718.2 (OVLO); no longer R742.2 (OVLO)
- net AON_EFUSE_UV: now also U718.1 (EN/UVLO); no longer R742.1 (EN/UVLO)
- net AON_FAULT_N: now also U718.4 (~{FLT}); no longer R742.4 (~{FLT})
- net AON_OR_RAW: now also D710.1 (K), D711.1 (K), D712.1 (K), D713.1 (K), U718.5 (IN); no longer R730.1 (K), R731.1 (K), R732.1 (K), R741.1 (K), R742.5 (IN)
- net AUX_DC_PROTECTED: now also Q23.5 (D(5-8)), U15B.16 (V2), D711.2 (A); no longer R731.2 (A), U15.16 (V2)
- net BAT_CHARGER: now also D710.2 (A); no longer R730.2 (A)
- net EC_AON_IN: now also U718.6 (OUT); no longer R742.6 (OUT)
- net GND: now also C715.2, R732.2, U15.8 (GND), U15B.20 (HYS), U15B.21 (EP/GND), U15B.8 (GND), C747.2, C748.2, C749.2, R743.2, R746.2, U718.8 (GND); no longer Q22.2, R742.8 (GND), U15.7 (GND)
- net MAIN_AUX_VALID_N: now also U15.7 (~{VALID2}), R718.2; no longer Q23.2, U15.10 (~{VALID2})
- net MAIN_SEL_INTVCC: now also U15.10 (INTVCC); no longer U15.8 (INTVCC)
- net MAIN_USB_VALID_N: now also U15.6 (~{VALID1}); no longer U15.9 (~{VALID1})
- net MCU_3V3: now also R718.1, R747.1; no longer Q23.1
- net PD1_VBUS_RAW: now also D712.2 (A); no longer R732.2 (A)
- net PD2_VBUS_RAW: now also D713.2 (A); no longer R741.2 (A)
- net USB_MAIN_FET_COMMON: now also Q22.2 (S), Q22.3 (S), Q22.4 (S), Q21.2 (S), Q21.3 (S), Q21.4 (S); no longer U15B.2 (S), U15B.3 (S), U15B.4 (S)
- net USB_MAIN_GATE: now also Q22.1 (G), Q21.1 (G); no longer U15B.1 (G)
- net USB_MAIN_OV: now also R731.2, R732.1; no longer Q22.1
- net USB_MAIN_UV: now also R730.2, R731.1
- net USB_PD_SELECTED: now also R730.1, Q21.5 (D(5-8)); no longer U15B.5 (D(5-8))
- net VBUS_COMBINED: now also Q22.5 (D(5-8)), Q29.5 (D(5-8)); no longer Q24.5 (D(5-8))
- net VSYS: now also TP3.1; no longer C715.1
- net AUX_MAIN_FET_COMMON renamed ST2_AUX_FET_COMMON
- net ST2_AUX_FET_COMMON: now also Q23.2 (S), Q23.3 (S), Q23.4 (S), U15B.12 (VS2); no longer U15.12 (VS2)
- net AUX_MAIN_GATE renamed ST2_AUX_GATE
- net ST2_AUX_GATE: now also Q23.1 (G), U15B.11 (G2); no longer U15.11 (G2)
- net AUX_MAIN_OV renamed ST2_AUX_OV
- net ST2_AUX_OV: now also U15B.5 (OV2); no longer U15.5 (OV2)
- net AUX_MAIN_UV renamed ST2_AUX_UV
- net ST2_AUX_UV: now also U15B.4 (UV2); no longer U15.4 (UV2)
- new net PD2_VALID_N: R747.2, U15B.6 (~{VALID1})
- new net PD2_VBUS_GATED: Q26.5 (D(5-8)), R741.1, U15B.17 (V1)
- new net SEL_STAGE2: C748.1, Q24.5 (D(5-8)), Q27.5 (D(5-8)), Q28.5 (D(5-8)), R744.1, U15.16 (V2), U15B.15 (VOUT)
- new net ST2_MAIN_FET_COMMON: C747.1, Q28.2 (S), Q28.3 (S), Q28.4 (S), Q29.2 (S), Q29.3 (S), Q29.4 (S), U15.12 (VS2)
- new net ST2_MAIN_GATE: Q28.1 (G), Q29.1 (G), U15.11 (G2)
- new net ST2_MAIN_OV: R745.2, R746.1, U15.5 (OV2)
- new net ST2_MAIN_UV: R744.2, R745.1, U15.4 (UV2)
- new net ST2_SEL_INTVCC: C749.1, U15B.10 (INTVCC), U15B.18 (EN), U15B.19 (~{SHDN})
- new net ST2_SEL_TMR: C715.1, U15B.1 (TMR)
- new net ST2_USB_FET_COMMON: Q26.2 (S), Q26.3 (S), Q26.4 (S), Q27.2 (S), Q27.3 (S), Q27.4 (S), U15B.14 (VS1)
- new net ST2_USB_GATE: Q26.1 (G), Q27.1 (G), U15B.13 (G1)
- new net ST2_USB_OV: R742.2, R743.1, U15B.3 (OV1)
- new net ST2_USB_UV: R741.2, R742.1, U15B.2 (UV1)
- no-connect marks 15 -> 17
Other:
- note added: "== U15/U15B LTC4418IUF cascade: PD1 > PD2 > AUX into VBUS_COMBINED =="
- note added: "U15/U15B cascade validates USB+PD2 near 15V and AUX across 7-22V, prioritizes PD1 > PD2 > AUX, and prevents inactive-source backfeed."
- note removed: "== U15 LTC4418IUF: USB-C PD priority over protected AUX/solar =="
- note removed: "U15 validates USB near 15V and AUX across 7-22V, gives USB priority, and prevents inactive-source backfeed."
