File: 07_radio_oled_gps.kicad_sch (KiCad schematic)
At the start: 32 parts, among them J40 M.2 E-key Wi-Fi/Bluetooth, J41 SSD1306 OLED A 0x3C (3.3V), J42 GNSS passive antenna U.FL, J43 DNP radio/debug expansion, J44 DNP MAX-M10S debug/program, J45 SSD1306 OLED B 0x3D (3.3V), U40 MAX-M10S GNSS

Commit message: Publish the current Ducktop2 design
Parts:
- removed C176: DNP 100p bias RF bypass, Capacitor_SMD:C_0603_1608Metric, symbol Device:C
- removed C177: DNP 100n bias bypass, Capacitor_SMD:C_0603_1608Metric, symbol Device:C
- removed J41: SSD1306 OLED A 0x3C (3.3V), Connector_PinHeader_2.54mm:PinHeader_1x06_P2.54mm_Vertical, symbol Connector_Generic:Conn_01x06
- removed L40: DNP 56nH active antenna RF choke, Inductor_SMD:L_0603_1608Metric, symbol Device:L
- removed R172: 100k OLED reset pull-up, Resistor_SMD:R_0603_1608Metric, symbol Device:R
- removed R175: 100k GNSS EXTINT pulldown, Resistor_SMD:R_0603_1608Metric, symbol Device:R
- removed R195: DNP 0R active antenna bias enable, Resistor_SMD:R_0603_1608Metric, symbol Device:R
- added C185: 100n OLED mux local, Capacitor_SMD:C_0603_1608Metric, symbol Device:C
- added C186: 1u MAX-M10S V_BCKP local decoupling, Capacitor_SMD:C_0805_2012Metric, symbol Device:C
- added C187: 100n E-key control-isolator local, Capacitor_SMD:C_0603_1608Metric, symbol Device:C
- added F10: 2A E-key 3V3 fuse/polyfuse, Fuse:Fuse_1206_3216Metric, symbol Device:Fuse
- added J41: SSD1306 OLED A 4-pin GND/VDD/SCK/SDA, ducktop2:SSD1306_0.96in_Module_4Pin, symbol Connector_Generic:Conn_01x04
- added J45: SSD1306 OLED B 4-pin GND/VDD/SCK/SDA, ducktop2:SSD1306_0.96in_Module_4Pin, symbol Connector_Generic:Conn_01x04
- added R198: 100k WLAN disable default asserted, Resistor_SMD:R_0603_1608Metric, symbol Device:R
- added R199: 100k Bluetooth disable default asserted, Resistor_SMD:R_0603_1608Metric, symbol Device:R
- added U170: SN74LVC3G34DCUR E-key control isolation, Package_SO:VSSOP-8_2.3x2mm_P0.5mm, symbol 74xGxx:74LVC3G34
- C174: value 1u OLED local -> 1u OLED A local
- C175: value 100n OLED local -> 100n OLED A local
- H4: renamed from F10; value 2A E-key 3V3 fuse/polyfuse -> M.2 E-key 2230 M2 grounded standoff 2.5mm; footprint Fuse:Fuse_1206_3216Metric -> ducktop2:SMT_Standoff_M2_H2.5_C4_Tail2.7x1.5; symbol Device:Fuse -> Mechanical:MountingHole_Pad; Buy_Link (none) -> https://item.taobao.com/item.htm?abbucket=8&id=655855111684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; Hardware_Spec (none) -> M2 internal thread; 4mm body; 2.5mm above PCB; 2.7x1.5mm lo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; MPN (none) -> M2XC4X2.5+C2.7X1.5; Manufacturer (none) -> Unbranded; Reference_Design (none) -> LattePanda Mu Lite Carrier V2 f954bf0275fa0aec4c1e9eb168f09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; Supplier (none) -> Taobao; Supplier_SKU (none) -> 4725777108077
- J40: value M.2 E-key Wi-Fi/Bluetooth -> Amphenol MDT420E01001 E-key Wi-Fi/Bluetooth socket; footprint Connector_PCBEdge:M.2_2230-xx-E -> ducktop2:Amphenol_MDT420E01001_H4.2; MPN (none) -> MDT420E01001; Manufacturer (none) -> Amphenol; QualifiedModuleContract (none) -> M2_2230_KEY_E_PCIE_WIFI_USB_BLUETOOTH_NOT_CNVIO2; QualifiedModuleMPN (none) -> AX210.NGWGIE.NV; QualifiedModuleManufacturer (none) -> Intel
- J42: MPN (none) -> U.FL-R-SMT-1(01); Manufacturer (none) -> Hirose
- R173: value 0R SSD1306 SA0=0x3C default -> 4.7k OLED A SCL pull-up
- R179: value DNP 0R SA0=0x3D option -> 4.7k OLED A SDA pull-up; now fitted; now in the parts list
- R196: value 0R SSD1306 B SA0=0x3D default -> 4.7k OLED B SCL pull-up
- R197: value DNP 0R OLED B SA0=0x3C option -> 4.7k OLED B SDA pull-up; now fitted; now in the parts list
- U40: MPN (none) -> MAX-M10S-00B; Manufacturer (none) -> u-blox
- U45: renamed from J45; value SSD1306 OLED B 0x3D (3.3V) -> TCA9548A service I2C mux @0x70; footprint Connector_PinHeader_2.54mm:PinHeader_1x06_P2.54mm_Vertical -> Package_SO:TSSOP-24_4.4x7.8mm_P0.65mm; symbol Connector_Generic:Conn_01x06 -> Interface_Expansion:TCA9548APWR; MPN (none) -> TCA9548APWR; Manufacturer (none) -> Texas Instruments
Connections:
- net OLED_SA0 is gone; now on net MCU_3V3: R173.1, R179.1
- net GND: now also H4.1, U45.12 (GND), U45.2 (A1), U45.21 (A2), C185.2, C186.2, C187.2, J41.1 (Pin_1), J45.1 (Pin_1), R198.2, R199.2, U170.3, U170.4 (GND); no longer R173.2, R197.2
- net I2C_SCL: now also U45.22 (SCL); no longer J40.60 (I2C_CLK), U45.3 (Pin_3)
- net I2C_SDA: now also U45.23 (SDA); no longer J40.58 (I2C_DATA), U45.4 (Pin_4)
- net MCU_3V3: now also C172.1, C173.1, J44.1 (Pin_1), R174.1, R196.1, R197.1, U40.6 (V_BCKP), U40.7 (VCC_IO), U40.8 (VCC), U45.24 (VCC), C185.1, C186.1, J41.2 (Pin_2), J45.2 (Pin_2); no longer R170.1, R171.1, R179.2, R196.2, U45.2 (Pin_2)
- net WIFI_3V3: now also R170.1, R171.1, C187.1, F10.2, U170.8 (VCC); no longer H4.2
- net WIFI_PCIE_RX_N: now also J40.43 (PERn0); no longer J40.37 (PETn0)
- net WIFI_PCIE_RX_P: now also J40.41 (PERp0); no longer J40.35 (PETp0)
- net WIFI_PCIE_TX_N: now also J40.37 (PETn0); no longer J40.43 (PERn0)
- net WIFI_PCIE_TX_P: now also J40.35 (PETp0); no longer J40.41 (PERp0)
- net WIFI_W_DISABLE1_N: now also U170.7
- net WIFI_W_DISABLE2_N: now also U170.2
- removed net OLED2_SA0: R196.1, R197.1, U45.6 (Pin_6)
- net OLED_RESET_N renamed OLED_A_SCL
- net OLED_A_SCL: now also R173.2, J41.3 (Pin_3)
- removed net SYS_3V3: C172.1, C173.1, H4.1, J44.1 (Pin_1), R174.1, U40.6 (V_BCKP), U40.7 (VCC_IO), U40.8 (VCC)
- new net OLED_A_SDA: J41.4 (Pin_4), R179.2, U45.4 (SD0)
- new net OLED_B_SCL: J45.3 (Pin_3), R196.2, U45.7 (SC1)
- new net OLED_B_SDA: J45.4 (Pin_4), R197.2, U45.6 (SD1)
- new net PCIE_3V3: F10.1
- new net PD1_I2C_SCL: U45.9 (SC2)
- new net PD1_I2C_SDA: U45.8 (SD2)
- new net PD2_I2C_SCL: U45.11 (SC3)
- new net PD2_I2C_SDA: U45.10 (SD3)
- new net PD3_I2C_SCL: U45.14 (SC4)
- new net PD3_I2C_SDA: U45.13 (SD4)
- new net SERVICE_MUX_RESET_N: U45.3 (~{RESET})
- new net WIFI_W_DISABLE1_N_EC: R198.1, U170.1
- new net WIFI_W_DISABLE2_N_EC: R199.1, U170.6
- no-connect marks 43 -> 52
Other:
- note added: "GNSS_EXTINT has no external pulldown; the MAX-M10S internal pull-up defines its reset state. EC firmware must leave the pin high-impedance until configured."
- note added: "Hardware-gated SERVICE_MUX_RESET_N asserts during every EC reset; firmware selects only a powered, VALID CH224A channel."
- note added: "J42 is passive-antenna-only. Active antenna bias requires a complete u-blox short-protected supervisor, not a bias-tee strap."
- note added: "M.2 E-key directions are host TX->PET35/37 and PER41/43->host RX; Mu-side TX has 220n AC coupling."
- note added: "MAX-M10S V_BCKP, VCC, and VCC_IO use always-on MCU_3V3 so I/O cannot back-power an unpowered GNSS domain."
- note added: "OLED headers match common 4-pin SSD1306 modules: GND, VDD/3V3, SCK/SCL, SDA. Use 3.3V modules only."
- note added: "Qualified radio is Intel AX210.NGWGIE.NV M.2 2230 Key-E: Wi-Fi over PCIe and Bluetooth over USB; AX211/CNVio2 is prohibited."
- note added: "TCA9548A channels 0/1 isolate the identical 0x3C OLEDs; channels 2/3/4 isolate the three CH224A sinks."
- note added: "U170 isolates powered-off E-key controls; R198/R199 keep WLAN and Bluetooth disabled until EC firmware explicitly enables them."
- note added: "USB2_P1 carries Bluetooth; default-BIOS HSIO3/REFCLK3/CLKREQ3 carry the E-key PCIe function."
- note removed: "Avoid CNVio/CNVio2-only E-key modules unless LattePanda Mu support is explicitly verified."
- note removed: "M.2 E-key PCIe lane follows the existing Mu-host-to-socket naming convention used by the NVMe M-key slot."
- note removed: "MAX-M10S uses EC UART here. VIO_SEL, SAFEBOOT_N, SDA/SCL, VCC_RF, and LNA_EN are NC."
- note removed: "OLED A defaults to 0x3C; OLED B defaults to 0x3D. Do not run both at the same address."
- note removed: "OLED headers are SSD1306 I2C: GND, 3V3, SCL, SDA, RES, SA0. Use 3.3V OLED modules only."
- note removed: "R195/L40/C176/C177 are DNP active-GNSS-antenna bias options; leave open for passive antennas."
- note removed: "Target radio is an Intel AX210-class M.2 2230 Key-E module: Wi-Fi over PCIe, Bluetooth over USB."
- note removed: "USB2_P1 is reserved for the E-key Bluetooth/USB function; HSIO1 is reserved for the E-key PCIe lane."

Commit message: Finish USB-C policy and split out radio board
Parts:
- removed C172: 10u GNSS local, Capacitor_SMD:C_1206_3216Metric, symbol Device:C
- removed C173: 100n GNSS local, Capacitor_SMD:C_0603_1608Metric, symbol Device:C
- removed C186: 1u MAX-M10S V_BCKP local decoupling, Capacitor_SMD:C_0805_2012Metric, symbol Device:C
- removed J42: GNSS passive antenna U.FL, Connector_Coaxial:U.FL_Hirose_U.FL-R-SMT-1_Vertical, symbol Connector:Conn_Coaxial
- removed J43: DNP radio/debug expansion, Connector_PinHeader_2.54mm:PinHeader_1x08_P2.54mm_Vertical, symbol Connector_Generic:Conn_01x08
- removed J44: DNP MAX-M10S debug/program, Connector_PinHeader_2.54mm:PinHeader_1x06_P2.54mm_Vertical, symbol Connector_Generic:Conn_01x06
- removed R174: 100k GNSS reset pull-up, Resistor_SMD:R_0603_1608Metric, symbol Device:R
- removed U40: MAX-M10S GNSS, RF_GPS:ublox_MAX, symbol RF_GPS:MAX-M10S
Connections:
- net PD3_I2C_SCL: no longer names the net of U45.14 (SC4)
- net PD3_I2C_SDA: no longer names the net of U45.13 (SD4)
- no-connect marks 52 -> 48
Other:
- note added: "== Wi-Fi/Bluetooth and dual OLED peripherals =="
- note added: "Both SSD1306 displays remain on the always-on EC service bus and work without the radio daughterboard."
- note added: "Channels 4-7 remain unused and explicitly no-connected for future service expansion."
- note added: "GNSS, amateur-radio modules, RF switching, and the dedicated radio codec are isolated on the removable daughterboard."
- note added: "Hardware-gated SERVICE_MUX_RESET_N asserts during every EC reset; firmware selects one TPS25751A channel and validates PD Status 0x35 plus PDO/RDO 0x31/0x32."
- note added: "M.2 E-key remains on the mainboard; GNSS and amateur-radio hardware moved to the optional radio daughterboard."
- note added: "TCA9548A channels 0/1 isolate the identical 0x3C OLEDs; channels 2/3 isolate the two TPS25751A service buses."
- note added: "The mainboard OLED and Wi-Fi functions do not depend on radio-daughterboard presence or power."
- note added: "The optional-board interface provides independent safe defaults for every radio/GNSS signal."
- note removed: "== J43 low-speed radio/debug expansion =="
- note removed: "== Radio, OLED, and GNSS peripherals =="
- note removed: "== U40 u-blox MAX-M10S GNSS module =="
- note removed: "GNSS RF layout: place U.FL near board edge, route RF_IN as 50 ohm, and keep it away from Wi-Fi antennas/noisy bucks."
- note removed: "GNSS_EXTINT has no external pulldown; the MAX-M10S internal pull-up defines its reset state. EC firmware must leave the pin high-impedance until configured."
- note removed: "Hardware-gated SERVICE_MUX_RESET_N asserts during every EC reset; firmware selects only a powered, VALID CH224A channel."
- note removed: "J42 is passive-antenna-only. Active antenna bias requires a complete u-blox short-protected supervisor, not a bias-tee strap."
- note removed: "M.2 E-key is the main Wi-Fi/Bluetooth path; OLED and GNSS stay on EC-controlled low-speed interfaces."
- note removed: "MAX-M10S V_BCKP, VCC, and VCC_IO use always-on MCU_3V3 so I/O cannot back-power an unpowered GNSS domain."
- note removed: "RF stays inside modules for this pass; antenna, keepout, and exact module qualification are layout-stage work."
- note removed: "TCA9548A channels 0/1 isolate the identical 0x3C OLEDs; channels 2/3/4 isolate the three CH224A sinks."

Commit message: Assign 327 BOM MPNs across 11 schematic sheets (370→43 gaps)
Closes 370 BOM procurement gaps by assigning Yageo resistor and Murata
capacitor MPNs to all passive components in the project's 11 schematic
sheets. 43 intentional holds remain for design-review items (crystal
loads, audio AC-coupling, VCAP, C0G timing, maker MCU 4.7u 0402s).

Key changes:
- 205 resistors assigned (Yageo RC0603/RT0603 series)
- 124 capacitors assigned (Murata GRM series, matching footprint body size)
- Fixed C183: 4.7u MPN→1u (GRM21BR71A105KA01L)
- Fixed C795/C840: upgraded to 50V rating (GRM21BR71H105KA12L)
- Generated fresh inventory: 1173 components, 43 remaining gaps
Parts:
- C170: MPN (none) -> GRM31CR71E106KA12L; Manufacturer (none) -> Murata
- C171, C175, C179, C185, C187: MPN (none) -> GRM188R71H104KA93D; Manufacturer (none) -> Murata
- C174, C178: MPN (none) -> GRM21BR71A105KA01L; Manufacturer (none) -> Murata
- R170, R171: MPN (none) -> RC0603FR-0710KL; Manufacturer (none) -> Yageo
- R173, R179, R196, R197: MPN (none) -> RC0603FR-074K7L; Manufacturer (none) -> Yageo
- R176, R177, R178: MPN (none) -> RC0603FR-070RL; Manufacturer (none) -> Yageo
- R198, R199: MPN (none) -> RC0603FR-07100KL; Manufacturer (none) -> Yageo
Changed lines of the file:
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@@
   (property "Footprint" "Capacitor_SMD:C_1206_3216Metric" (at 20.32 91.44 0) (effects (font (size 1.27 1.27)) (hide yes)))
   (property "Datasheet" "" (at 20.32 91.44 0) (effects (font (size 1.27 1.27)) (hide yes)))
+  (property "Manufacturer" "Murata" (at 20.32 91.44 0) (effects (font (size 1.27 1.27)) (hide yes)))
+  (property "MPN" "GRM31CR71E106KA12L" (at 20.32 91.44 0) (effects (font (size 1.27 1.27)) (hide yes)))
   (pin "1")
   (pin "2")
@@
   (property "Footprint" "Capacitor_SMD:C_0603_1608Metric" (at 20.32 104.14 0) (effects (font (size 1.27 1.27)) (hide yes)))
   (property "Datasheet" "" (at 20.32 104.14 0) (effects (font (size 1.27 1.27)) (hide yes)))
+  (property "Manufacturer" "Murata" (at 20.32 104.14 0) (effects (font (size 1.27 1.27)) (hide yes)))
+  (property "MPN" "GRM188R71H104KA93D" (at 20.32 104.14 0) (effects (font (size 1.27 1.27)) (hide yes)))
   (pin "1")
   (pin "2")
@@
   (property "Footprint" "Resistor_SMD:R_0603_1608Metric" (at 20.32 139.7 0) (effects (font (size 1.27 1.27)) (hide yes)))
   (property "Datasheet" "" (at 20.32 139.7 0) (effects (font (size 1.27 1.27)) (hide yes)))
+  (property "Manufacturer" "Yageo" (at 20.32 139.7 0) (effects (font (size 1.27 1.27)) (hide yes)))
+  (property "MPN" "RC0603FR-0710KL" (at 20.32 139.7 0) (effects (font (size 1.27 1.27)) (hide yes)))
   (pin "1")
   (pin "2")
@@
   (property "Footprint" "Resistor_SMD:R_0603_1608Metric" (at 20.32 152.4 0) (effects (font (size 1.27 1.27)) (hide yes)))
   (property "Datasheet" "" (at 20.32 152.4 0) (effects (font (size 1.27 1.27)) (hide yes)))
+  (property "Manufacturer" "Yageo" (at 20.32 152.4 0) (effects (font (size 1.27 1.27)) (hide yes)))
+  (property "MPN" "RC0603FR-0710KL" (at 20.32 152.4 0) (effects (font (size 1.27 1.27)) (hide yes)))
   (pin "1")
   (pin "2")
@@
   (property "Footprint" "Capacitor_SMD:C_0603_1608Metric" (at 214.63 139.7 0) (effects (font (size 1.27 1.27)) (hide yes)))
   (property "Datasheet" "" (at 214.63 139.7 0) (effects (font (size 1.27 1.27)) (hide yes)))
+  (property "Manufacturer" "Murata" (at 214.63 139.7 0) (effects (font (size 1.27 1.27)) (hide yes)))
+  (property "MPN" "GRM188R71H104KA93D" (at 214.63 139.7 0) (effects (font (size 1.27 1.27)) (hide yes)))
   (pin "1")
   (pin "2")
@@
   (property "Footprint" "Resistor_SMD:R_0603_1608Metric" (at 95.25 152.4 0) (effects (font (size 1.27 1.27)) (hide yes)))
   (property "Datasheet" "" (at 95.25 152.4 0) (effects (font (size 1.27 1.27)) (hide yes)))
+  (property "Manufacturer" "Yageo" (at 95.25 152.4 0) (effects (font (size 1.27 1.27)) (hide yes)))
+  (property "MPN" "RC0603FR-07100KL" (at 95.25 152.4 0) (effects (font (size 1.27 1.27)) (hide yes)))
   (pin "1")
   (pin "2")
@@
   (property "Footprint" "Resistor_SMD:R_0603_1608Metric" (at 124.46 152.4 0) (effects (font (size 1.27 1.27)) (hide yes)))
   (property "Datasheet" "" (at 124.46 152.4 0) (effects (font (size 1.27 1.27)) (hide yes)))
+  (property "Manufacturer" "Yageo" (at 124.46 152.4 0) (effects (font (size 1.27 1.27)) (hide yes)))
+  (property "MPN" "RC0603FR-07100KL" (at 124.46 152.4 0) (effects (font (size 1.27 1.27)) (hide yes)))
   (pin "1")
   (pin "2")
@@
   (property "Footprint" "Resistor_SMD:R_0603_1608Metric" (at 20.32 170.18 0) (effects (font (size 1.27 1.27)) (hide yes)))
   (property "Datasheet" "" (at 20.32 170.18 0) (effects (font (size 1.27 1.27)) (hide yes)))
+  (property "Manufacturer" "Yageo" (at 20.32 170.18 0) (effects (font (size 1.27 1.27)) (hide yes)))
+  (property "MPN" "RC0603FR-070RL" (at 20.32 170.18 0) (effects (font (size 1.27 1.27)) (hide yes)))
   (pin "1")
   (pin "2")
@@
   (property "Footprint" "Resistor_SMD:R_0603_1608Metric" (at 20.32 182.88 0) (effects (font (size 1.27 1.27)) (hide yes)))
   (property "Datasheet" "" (at 20.32 182.88 0) (effects (font (size 1.27 1.27)) (hide yes)))
+  (property "Manufacturer" "Yageo" (at 20.32 182.88 0) (effects (font (size 1.27 1.27)) (hide yes)))
+  (property "MPN" "RC0603FR-070RL" (at 20.32 182.88 0) (effects (font (size 1.27 1.27)) (hide yes)))
   (pin "1")
   (pin "2")
@@
   (property "Footprint" "Resistor_SMD:R_0603_1608Metric" (at 20.32 195.58 0) (effects (font (size 1.27 1.27)) (hide yes)))
   (property "Datasheet" "" (at 20.32 195.58 0) (effects (font (size 1.27 1.27)) (hide yes)))
+  (property "Manufacturer" "Yageo" (at 20.32 195.58 0) (effects (font (size 1.27 1.27)) (hide yes)))
+  (property "MPN" "RC0603FR-070RL" (at 20.32 195.58 0) (effects (font (size 1.27 1.27)) (hide yes)))
   (pin "1")
   (pin "2")
@@
   (property "Footprint" "Resistor_SMD:R_0603_1608Metric" (at 20.32 299.72 0) (effects (font (size 1.27 1.27)) (hide yes)))
   (property "Datasheet" "" (at 20.32 299.72 0) (effects (font (size 1.27 1.27)) (hide yes)))
+  (property "Manufacturer" "Yageo" (at 20.32 299.72 0) (effects (font (size 1.27 1.27)) (hide yes)))
+  (property "MPN" "RC0603FR-074K7L" (at 20.32 299.72 0) (effects (font (size 1.27 1.27)) (hide yes)))
   (pin "1")
   (pin "2")
@@
   (property "Footprint" "Resistor_SMD:R_0603_1608Metric" (at 20.32 312.42 0) (effects (font (size 1.27 1.27)) (hide yes)))
   (property "Datasheet" "" (at 20.32 312.42 0) (effects (font (size 1.27 1.27)) (hide yes)))
+  (property "Manufacturer" "Yageo" (at 20.32 312.42 0) (effects (font (size 1.27 1.27)) (hide yes)))
+  (property "MPN" "RC0603FR-074K7L" (at 20.32 312.42 0) (effects (font (size 1.27 1.27)) (hide yes)))
   (pin "1")
   (pin "2")
@@
   (property "Footprint" "Capacitor_SMD:C_0805_2012Metric" (at 90.17 325.12 0) (effects (font (size 1.27 1.27)) (hide yes)))
   (property "Datasheet" "" (at 90.17 325.12 0) (effects (font (size 1.27 1.27)) (hide yes)))
+  (property "Manufacturer" "Murata" (at 90.17 325.12 0) (effects (font (size 1.27 1.27)) (hide yes)))
+  (property "MPN" "GRM21BR71A105KA01L" (at 90.17 325.12 0) (effects (font (size 1.27 1.27)) (hide yes)))
   (pin "1")
   (pin "2")
@@
   (property "Footprint" "Capacitor_SMD:C_0603_1608Metric" (at 90.17 337.82 0) (effects (font (size 1.27 1.27)) (hide yes)))
   (property "Datasheet" "" (at 90.17 337.82 0) (effects (font (size 1.27 1.27)) (hide yes)))
+  (property "Manufacturer" "Murata" (at 90.17 337.82 0) (effects (font (size 1.27 1.27)) (hide yes)))
+  (property "MPN" "GRM188R71H104KA93D" (at 90.17 337.82 0) (effects (font (size 1.27 1.27)) (hide yes)))
   (pin "1")
   (pin "2")
@@
   (property "Footprint" "Resistor_SMD:R_0603_1608Metric" (at 204.47 312.42 0) (effects (font (size 1.27 1.27)) (hide yes)))
   (property "Datasheet" "" (at 204.47 312.42 0) (effects (font (size 1.27 1.27)) (hide yes)))
+  (property "Manufacturer" "Yageo" (at 204.47 312.42 0) (effects (font (size 1.27 1.27)) (hide yes)))
+  (property "MPN" "RC0603FR-074K7L" (at 204.47 312.42 0) (effects (font (size 1.27 1.27)) (hide yes)))
   (pin "1")
   (pin "2")
@@
   (property "Footprint" "Resistor_SMD:R_0603_1608Metric" (at 204.47 325.12 0) (effects (font (size 1.27 1.27)) (hide yes)))
   (property "Datasheet" "" (at 204.47 325.12 0) (effects (font (size 1.27 1.27)) (hide yes)))
+  (property "Manufacturer" "Yageo" (at 204.47 325.12 0) (effects (font (size 1.27 1.27)) (hide yes)))
+  (property "MPN" "RC0603FR-074K7L" (at 204.47 325.12 0) (effects (font (size 1.27 1.27)) (hide yes)))
   (pin "1")
   (pin "2")
@@
   (property "Footprint" "Capacitor_SMD:C_0805_2012Metric" (at 204.47 350.52 0) (effects (font (size 1.27 1.27)) (hide yes)))
   (property "Datasheet" "" (at 204.47 350.52 0) (effects (font (size 1.27 1.27)) (hide yes)))
+  (property "Manufacturer" "Murata" (at 204.47 350.52 0) (effects (font (size 1.27 1.27)) (hide yes)))
+  (property "MPN" "GRM21BR71A105KA01L" (at 204.47 350.52 0) (effects (font (size 1.27 1.27)) (hide yes)))
   (pin "1")
   (pin "2")
@@
   (property "Footprint" "Capacitor_SMD:C_0603_1608Metric" (at 204.47 363.22 0) (effects (font (size 1.27 1.27)) (hide yes)))
   (property "Datasheet" "" (at 204.47 363.22 0) (effects (font (size 1.27 1.27)) (hide yes)))
+  (property "Manufacturer" "Murata" (at 204.47 363.22 0) (effects (font (size 1.27 1.27)) (hide yes)))
+  (property "MPN" "GRM188R71H104KA93D" (at 204.47 363.22 0) (effects (font (size 1.27 1.27)) (hide yes)))
   (pin "1")
   (pin "2")
@@
   (property "Footprint" "Capacitor_SMD:C_0603_1608Metric" (at 90.17 350.52 0) (effects (font (size 1.27 1.27)) (hide yes)))
   (property "Datasheet" "" (at 90.17 350.52 0) (effects (font (size 1.27 1.27)) (hide yes)))
-  (pin "1")
-  (pin "2")
+  (property "Manufacturer" "Murata" (at 90.17 350.52 0) (effects (font (size 1.27 1.27)) (hide yes)))
+  (property "MPN" "GRM188R71H104KA93D" (at 90.17 350.52 0) (effects (font (size 1.27 1.27)) (hide yes)))
+  (pin "1")
+  (pin "2")
