File: 12_keyboard_interface.kicad_sch (KiCad schematic)
At the start: 40 parts, among them J310 Mainboard keyboard FFC to MX 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, U310 TPS2553D keyboard RGB 5V swit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, U311 SN74AHCT1G126 keyboard RGB 3V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

Commit message: Assign 327 BOM MPNs across 11 schematic sheets (370→43 gaps)
Closes 370 BOM procurement gaps by assigning Yageo resistor and Murata
capacitor MPNs to all passive components in the project's 11 schematic
sheets. 43 intentional holds remain for design-review items (crystal
loads, audio AC-coupling, VCAP, C0G timing, maker MCU 4.7u 0402s).

Key changes:
- 205 resistors assigned (Yageo RC0603/RT0603 series)
- 124 capacitors assigned (Murata GRM series, matching footprint body size)
- Fixed C183: 4.7u MPN→1u (GRM21BR71A105KA01L)
- Fixed C795/C840: upgraded to 50V rating (GRM21BR71H105KA12L)
- Generated fresh inventory: 1173 components, 43 remaining gaps
Parts:
- C319: MPN (none) -> GRM31CR71E106KA12L; Manufacturer (none) -> Murata
- C322, C323, C324: MPN (none) -> GRM188R71H104KA93D; Manufacturer (none) -> Murata
- R360, R361, R362, R363, R364, R365, R366, R367, R368, R369, R370, R371, R372, R373, R374, R376, R377, R378, R379, R380, R381, R382, R383: MPN (none) -> RC0603FR-071KL; Manufacturer (none) -> Yageo
- R375, R384, R385: MPN (none) -> RC0603FR-07100RL; Manufacturer (none) -> Yageo
- R388: MPN (none) -> RC0603FR-0766K5L; Manufacturer (none) -> Yageo
- R389, R391: MPN (none) -> RC0603FR-07100KL; Manufacturer (none) -> Yageo
- R390: MPN (none) -> RC0603FR-0710KL; Manufacturer (none) -> Yageo
