File: ducktop2.kicad_sch (KiCad schematic)
At the start: 0 parts

Commit message: Phase 2.0: convert J11/J12 to USB2-only (board split prep)
J11 and J12 lose their SuperSpeed lanes as part of the 4-board split
(no USB3 host port remains on the right side; hub DS1/DS4 become
USB2-only downstream ports).

- generate_power_inputs_sheet.py: add_dual_role_port gains usb2_only;
  J11 drops the TUSB1142 redriver, SS coupling caps, and SS ESD; SS
  connector pins become NC. PD charging (15V sink / 5V 0.9A source),
  CC, USB2 (via hub DS1 D+/D-), VBUS/PPHV/LDO protection all kept.
- generate_usb_c_io_sheet.py: add_source_port gains usb2_only; J12
  drops the HD3SS6126 mux + SS chain; hub DS1/DS4 SS pins (7/8/10/11,
  36/37/39/40) retired to NC. DS2/DS3/UP unchanged.
- verify_design_contracts.py: J11/J12 SS pins now NC, U1700 DS1/DS4 SS
  pins NC, TUSB1142/strap contracts gated on usb2_only.
- verify_schematic_closure.py: closure audit accepts NC SS pins
  (unconnected-* pseudo-nets) for J12 and the retired hub pins.
- generate_pin_review_table.py: J12 SS pins NC, U1700 retired pins NC,
  U2010 removed from required set.
- Regenerated 04_usb_c_io / 05_power_inputs / root sheets.

16 SS nets removed. Verified: schematic gate PASS (closure 1574/0,
contracts OK, ERC 0, pin review 2602/2602, generated-source identity
PASS).
Other:
- sheet Native USB-C I/O ports: added none; removed HUB_DS1_SSRX_N, HUB_DS1_SSRX_P, HUB_DS1_SSTX_N, HUB_DS1_SSTX_P
- sheet Power Inputs ports: added none; removed HUB_DS1_SSRX_N, HUB_DS1_SSRX_P, HUB_DS1_SSTX_N, HUB_DS1_SSTX_P
Changed lines of the file:
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@@
     (effects (font (size 1.27 1.27)) (justify left))
   )
-  (pin "HUB_DS1_SSRX_P" bidirectional
+  (pin "USBC2_DP" bidirectional
     (at 120.65 234.95 0)
     (effects (font (size 1.27 1.27)) (justify left))
   )
-  (pin "HUB_DS1_SSRX_N" bidirectional
+  (pin "USBC2_DM" bidirectional
     (at 120.65 240.03 0)
     (effects (font (size 1.27 1.27)) (justify left))
   )
-  (pin "USBC2_DP" bidirectional
+  (pin "USBC2_SSTX_P" bidirectional
     (at 120.65 245.11 0)
     (effects (font (size 1.27 1.27)) (justify left))
   )
-  (pin "USBC2_DM" bidirectional
+  (pin "USBC2_SSTX_N" bidirectional
     (at 120.65 250.19 0)
     (effects (font (size 1.27 1.27)) (justify left))
   )
-  (pin "USBC2_SSTX_P" bidirectional
+  (pin "USBC2_SSRX_P" bidirectional
     (at 120.65 255.27 0)
     (effects (font (size 1.27 1.27)) (justify left))
   )
-  (pin "USBC2_SSTX_N" bidirectional
+  (pin "USBC2_SSRX_N" bidirectional
     (at 120.65 260.35 0)
-    (effects (font (size 1.27 1.27)) (justify left))
-  )
-  (pin "HUB_DS1_SSTX_P" bidirectional
-    (at 120.65 265.43 0)
-    (effects (font (size 1.27 1.27)) (justify left))
-  )
-  (pin "HUB_DS1_SSTX_N" bidirectional
-    (at 120.65 270.51 0)
-    (effects (font (size 1.27 1.27)) (justify left))
-  )
-  (pin "USBC2_SSRX_P" bidirectional
-    (at 120.65 275.59 0)
-    (effects (font (size 1.27 1.27)) (justify left))
-  )
-  (pin "USBC2_SSRX_N" bidirectional
-    (at 120.65 280.67 0)
     (effects (font (size 1.27 1.27)) (justify left))
   )
@@
 (sheet
   (at 549.91 490.22)
-  (size 90.17 167.64)
+  (size 90.17 165.1)
   (stroke (width 0.1524) (type solid))
   (fill (color 0 0 0 0.0))
@@
   )
   (property "Sheetfile" "05_power_inputs.kicad_sch"
-    (at 549.91 659.13 0)
+    (at 549.91 656.59 0)
     (effects (font (size 1.27 1.27)) (justify left top))
   )
@@
     (effects (font (size 1.27 1.27)) (justify left))
   )
-  (pin "HUB_DS1_SSTX_N" bidirectional
+  (pin "PD2_EFUSE_FAULT_N" bidirectional
     (at 640.08 607.06 0)
     (effects (font (size 1.27 1.27)) (justify left))
   )
-  (pin "HUB_DS1_SSTX_P" bidirectional
+  (pin "PD2_PATH_EN" bidirectional
     (at 640.08 612.14 0)
     (effects (font (size 1.27 1.27)) (justify left))
   )
-  (pin "HUB_DS1_SSRX_P" bidirectional
+  (pin "PD1_VALID_N" bidirectional
     (at 640.08 617.22 0)
     (effects (font (size 1.27 1.27)) (justify left))
   )
-  (pin "HUB_DS1_SSRX_N" bidirectional
+  (pin "PD2_VALID_N" bidirectional
     (at 640.08 622.3 0)
     (effects (font (size 1.27 1.27)) (justify left))
   )
-  (pin "PD2_EFUSE_FAULT_N" bidirectional
+  (pin "USB_PD_SELECTED" bidirectional
     (at 640.08 627.38 0)
-    (effects (font (size 1.27 1.27)) (justify left))
-  )
-  (pin "PD2_PATH_EN" bidirectional
-    (at 640.08 632.46 0)
-    (effects (font (size 1.27 1.27)) (justify left))
-  )
-  (pin "PD1_VALID_N" bidirectional
-    (at 640.08 637.54 0)
-    (effects (font (size 1.27 1.27)) (justify left))
-  )
-  (pin "PD2_VALID_N" bidirectional
-    (at 640.08 642.62 0)
-    (effects (font (size 1.27 1.27)) (justify left))
-  )
-  (pin "USB_PD_SELECTED" bidirectional
-    (at 640.08 647.7 0)
     (effects (font (size 1.27 1.27)) (justify left))
   )
@@
 )
 (label "USB_PD_SELECTED"
-  (at 640.08 647.7 0)
+  (at 640.08 627.38 0)
   (effects (font (size 1.27 1.27)) (justify left bottom))
 )
@@
 )
 (label "PD1_VALID_N"
-  (at 640.08 637.54 0)
+  (at 640.08 617.22 0)
   (effects (font (size 1.27 1.27)) (justify left bottom))
 )
@@
 )
 (label "PD2_VALID_N"
-  (at 640.08 642.62 0)
+  (at 640.08 622.3 0)
   (effects (font (size 1.27 1.27)) (justify left bottom))
 )
@@
 )
 (label "PD2_PATH_EN"
-  (at 640.08 632.46 0)
+  (at 640.08 612.14 0)
   (effects (font (size 1.27 1.27)) (justify left bottom))
 )
@@
 )
 (label "PD2_EFUSE_FAULT_N"
-  (at 640.08 627.38 0)
+  (at 640.08 607.06 0)
   (effects (font (size 1.27 1.27)) (justify left bottom))
 )
@@
 )
 (label "USBC2_SSRX_P"
-  (at 120.65 275.59 0)
+  (at 120.65 255.27 0)
   (effects (font (size 1.27 1.27)) (justify left bottom))
 )
@@
 )
 (label "USBC2_SSRX_N"
-  (at 120.65 280.67 0)
+  (at 120.65 260.35 0)
   (effects (font (size 1.27 1.27)) (justify left bottom))
 )
@@
 )
 (label "USBC2_DP"
-  (at 120.65 245.11 0)
+  (at 120.65 234.95 0)
   (effects (font (size 1.27 1.27)) (justify left bottom))
 )
@@
 )
 (label "USBC2_DM"
-  (at 120.65 250.19 0)
+  (at 120.65 240.03 0)
   (effects (font (size 1.27 1.27)) (justify left bottom))
 )
@@
 )
 (label "USBC2_SSTX_P"
-  (at 120.65 255.27 0)
+  (at 120.65 245.11 0)
   (effects (font (size 1.27 1.27)) (justify left bottom))
 )
@@
 )
 (label "USBC2_SSTX_N"
-  (at 120.65 260.35 0)
+  (at 120.65 250.19 0)
   (effects (font (size 1.27 1.27)) (justify left bottom))
 )
@@
   (effects (font (size 1.27 1.27)) (justify left bottom))
 )
-(label "HUB_DS1_SSRX_P"
-  (at 120.65 234.95 0)
-  (effects (font (size 1.27 1.27)) (justify left bottom))
-)
-(label "HUB_DS1_SSRX_P"
-  (at 640.08 617.22 0)
-  (effects (font (size 1.27 1.27)) (justify left bottom))
-)
-(label "HUB_DS1_SSRX_N"
-  (at 120.65 240.03 0)
-  (effects (font (size 1.27 1.27)) (justify left bottom))
-)
-(label "HUB_DS1_SSRX_N"
-  (at 640.08 622.3 0)
-  (effects (font (size 1.27 1.27)) (justify left bottom))
-)
-(label "HUB_DS1_SSTX_P"
-  (at 120.65 265.43 0)
-  (effects (font (size 1.27 1.27)) (justify left bottom))
-)
-(label "HUB_DS1_SSTX_P"
-  (at 640.08 612.14 0)
-  (effects (font (size 1.27 1.27)) (justify left bottom))
-)
-(label "HUB_DS1_SSTX_N"
-  (at 120.65 270.51 0)
-  (effects (font (size 1.27 1.27)) (justify left bottom))
-)
-(label "HUB_DS1_SSTX_N"
-  (at 640.08 607.06 0)
-  (effects (font (size 1.27 1.27)) (justify left bottom))
-)

Commit message: Board split Phase 2.4: trim center board, FPC boundary contracts, per-project verification
Center (ducktop2) loses the four sheets that moved to the daughterboards:
04_usb_c_io, 05_power_inputs, 06_tcp0_external_hdmi, 16_gigabit_ethernet,
and the pack-protection section of 01_power_battery (BMS board). J190 AUX
terminal moves to the left board. Center keeps 9 sheets: charger/gauge/
ship-FET (U2/U10/Q25/RS1), EC, Mu, radio, internal, radio-DB, keyboard x2,
maker, audio. 717 components.

FPC-1/2/3 boundary contracts declare the crossing nets at the center root
(30 + 35 + 4 shared nets; HUB_DS1_DP/DM are center pass-throughs).

Verification is now per-project:
- verify_design_contracts.py --project {ducktop2,left_io,right_io,bms}
  (five-port USB-C contracts split by port, HDMI/GbE run on right_io,
  pack contracts run on bms, sheet names parameterized)
- verify_schematic_closure.py --pack audits the BMS pack block
- verify_electrical_calculations.py --project bms for pack calcs
- pin review trimmed to center parts; FPC-boundary nets in ERC allowlist

Fixed while trimming: daughterboard root labels now sit on sheet-block pin
endpoints (left/right FPC nets actually connect); duplicate GND pwrflag in
power sheet; sync.parse_netlist respects the radio-daughterboard override.

Schematic gate PASS: self-check, closure audits (89+151), electrical
calcs (67+15), pin review (1625), identity.
Other:
- removed sheet Gigabit Ethernet
- removed sheet Native USB-C I/O
- removed sheet Power Inputs
- removed sheet TCP0 External HDMI
- sheet Power & Battery ports: added AUX_DC_RAW, FG_VSS, PACK_POS_FUSED; removed PACK_RETRY_PULSE

Commit message: Board split Phase 4a: FPC connectors wired through the four split schematics
Connector symbols and sheets now exist in every project and the boundary
nets are pinned through them (same conductor order on both ends, verified
netlist-by-netlist):
  - gen/fpc_contract.py: authoritative FPC-1/2/3 pin maps + center-side
    renames (single source of truth for schematics, board pad nets, cable
    spec, and gate contracts)
  - gen/Conn_01x100_FFC_MP.kicad_sym (derived from the 30-pin pattern)
  - center: real fpc1_left/fpc2_right/fpc3_bms sheets wired to host pins
  - left_io/right_io: left_fpc/right_fpc connector sheets; bms carries
    FPC106 inline
  - connector refs FPC101..FPC106 (valid designators; FPC1_L-style refs
    broke KiCad annotation)
  - pack-rail naming reconciled: center gauge divider BAT_PROT_VIN ->
    PACK_POS_FUSED (same node as the BMS LTC4368 output); BMS ground
    /GND -> GND (pack negative is the system ground)

Boards: daughterboards re-synced from their connector-bearing schematics;
center connectors placed and their pad nets assigned text-side ((net
"name") convention).  Connector pads verified against every other
footprint (0 overlaps) and DRC shows 0 shorts on all four boards (center
16 pre-existing, down from 17).

Fixed two latent generator bugs exposed by the wiring:
  - resolve_connectors used naive +R rotation, placing Phase 3 connectors
    against mirrored phantom positions
  - pad half-extents were computed as footprint_rot+pad_rot, but KiCad
    saves pads with world orientation (FH12-100S pins are 1.3mm wide);
    both verified empirically against pcbnew, plus a connector-nudge pass
    for parts sandwiched between the connector body and pin columns

Gate: SCHEMATIC RELEASE CHECK: PASS (FPC pin contracts added per project;
closure audits 0 FAIL).  Routing remains manual (Phase 4b).
Other:
- added sheet FPC-1 (Left) (fpc1_left.kicad_sch)
- added sheet FPC-2 (Right) (fpc2_right.kicad_sch)
- added sheet FPC-3 (BMS) (fpc3_bms.kicad_sch)

Commit message: Phase 5: second-opinion audit remediation + rebuilt, verified board pipeline
Second-opinion AI audit found A-tier defects; remediation applied and the
board pipeline rebuilt on a known-good base with the fixes it needed:

- electrical: LTC4418IUF symbol pinout corrected (both selectors were
  dead as drawn); center charge cascade (U15 <- U15B, PD1 > PD2 > AUX);
  pack negative never crosses FPC-3, 15-pin FG_VSS return; power-budgeted
  FPC pin maps (0.4 A/pin derate); J12/DS4 completed; AUX source fuse
- FH41-68S footprint: 13 datasheet-correct SH pads + SH pin in symbol
- connector geometry settled against the Hirose FH12 2D drawing: FFC
  enters opposite the solder pins (mouth = local +Y); reversed side-B
  maps are correct for the 180-deg-mounted pairs; rotations set so mouths
  face across every seam
- pipeline (generate_split_boards.py): per-pin pad-net resync from the
  netlists (kills shadow nets for good), netlist-exact name
  normalization, netlist-only part injection (cascade, probe headers),
  zone refill after outline swap, read-before-write race fixed, orphan
  parts dropped loudly, non-zero exit on unresolved overlaps
- monolith board relocated to old/monolith_ducktop2.kicad_pcb (placement
  oracle for the center cut only)

verified end state: 4 boards 0 shorts / 0 clearance / 0 drill, 0 boundary
crossings, 6/6 connectors contract-exact with mouths facing, 0 shadow
nets, gates PASS x4, ERC 0 x4. routing next (499 nets/board).
Other:
- sheet FPC-1 (Left) ports: added HUB_DS4_DM, HUB_DS4_DP, HUB_PRT_CTL4; removed PD2_VALID_N
- sheet FPC-2 (Right) ports: added HUB_DS4_DM, HUB_DS4_DP, HUB_PRT_CTL4, PD2_VBUS_GATED; removed none
- sheet Power & Battery ports: added PD2_VALID_N, PD2_VBUS_GATED; removed none

Commit message: get the main boards ready for routing
Other:
- sheet EC & MCU ports: added MCU_USB_DN; removed MCU_USB_DM
- sheet FPC-1 (Left) ports: added HUB_DS1_DN, HUB_DS4_DN, USBC1_DN, USBC2_DN; removed HUB_DS1_DM, HUB_DS4_DM, USBC1_DM, USBC2_DM
- sheet FPC-2 (Right) ports: added HUB_DS1_DN, HUB_DS4_DN; removed HUB_DS1_DM, HUB_DS4_DM
- sheet Internal Services ports: added EC_HOST_USB_DN, MCU_USB_DN, TRACKPAD_USB_DN; removed EC_HOST_USB_DM, MCU_USB_DM, TRACKPAD_USB_DM
- sheet Maker MCU ports: added MAKER_USB_DN; removed MAKER_USB_DM
- sheet Mu Carrier ports: added AUDIO_USB_DN, EC_HOST_USB_DN, MAKER_USB_DN, TRACKPAD_USB_DN, USBC1_DN, USBC2_DN; removed AUDIO_USB_DM, EC_HOST_USB_DM, MAKER_USB_DM, TRACKPAD_USB_DM, USBC1_DM, USBC2_DM
- sheet Optional Radio Daughterboard Interface ports: added RADIO_CODEC_USB_HOST_DN, RADIO_CODEC_USB_HOST_DP; removed RADIO_CODEC_USB_DM_HOST, RADIO_CODEC_USB_DP_HOST
- sheet System Audio ports: added AUDIO_USB_DN, RADIO_CODEC_USB_HOST_DN, RADIO_CODEC_USB_HOST_DP; removed AUDIO_USB_DM, RADIO_CODEC_USB_DM_HOST, RADIO_CODEC_USB_DP_HOST
Changed lines of the file:
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@@
     (effects (font (size 1.27 1.27)) (justify left))
   )
-  (pin "MCU_USB_DM" bidirectional
+  (pin "MCU_USB_DN" bidirectional
     (at 219.71 308.61 0)
     (effects (font (size 1.27 1.27)) (justify left))
@@
     (effects (font (size 1.27 1.27)) (justify left))
   )
-  (pin "AUDIO_USB_DM" bidirectional
+  (pin "AUDIO_USB_DN" bidirectional
     (at 359.41 69.85 0)
     (effects (font (size 1.27 1.27)) (justify left))
@@
     (effects (font (size 1.27 1.27)) (justify left))
   )
-  (pin "USBC2_DM" bidirectional
+  (pin "USBC2_DN" bidirectional
     (at 359.41 227.33 0)
     (effects (font (size 1.27 1.27)) (justify left))
   )
-  (pin "USBC1_DM" bidirectional
+  (pin "USBC1_DN" bidirectional
     (at 359.41 232.41 0)
     (effects (font (size 1.27 1.27)) (justify left))
@@
     (effects (font (size 1.27 1.27)) (justify left))
   )
-  (pin "MAKER_USB_DM" bidirectional
+  (pin "MAKER_USB_DN" bidirectional
     (at 359.41 247.65 0)
     (effects (font (size 1.27 1.27)) (justify left))
   )
-  (pin "EC_HOST_USB_DM" bidirectional
+  (pin "EC_HOST_USB_DN" bidirectional
     (at 359.41 252.73 0)
     (effects (font (size 1.27 1.27)) (justify left))
@@
     (effects (font (size 1.27 1.27)) (justify left))
   )
-  (pin "TRACKPAD_USB_DM" bidirectional
+  (pin "TRACKPAD_USB_DN" bidirectional
     (at 359.41 267.97 0)
     (effects (font (size 1.27 1.27)) (justify left))
@@
     (effects (font (size 1.27 1.27)) (justify left))
   )
-  (pin "MCU_USB_DM" bidirectional
+  (pin "MCU_USB_DN" bidirectional
     (at 405.13 400.05 0)
     (effects (font (size 1.27 1.27)) (justify left))
@@
     (effects (font (size 1.27 1.27)) (justify left))
   )
-  (pin "EC_HOST_USB_DM" bidirectional
+  (pin "EC_HOST_USB_DN" bidirectional
     (at 405.13 415.29 0)
     (effects (font (size 1.27 1.27)) (justify left))
@@
     (effects (font (size 1.27 1.27)) (justify left))
   )
-  (pin "TRACKPAD_USB_DM" bidirectional
+  (pin "TRACKPAD_USB_DN" bidirectional
     (at 405.13 435.61 0)
     (effects (font (size 1.27 1.27)) (justify left))
@@
     (effects (font (size 1.27 1.27)) (justify left))
   )
-  (pin "RADIO_CODEC_USB_DP_HOST" bidirectional
+  (pin "RADIO_CODEC_USB_HOST_DP" bidirectional
     (at 535.94 255.27 0)
     (effects (font (size 1.27 1.27)) (justify left))
   )
-  (pin "RADIO_CODEC_USB_DM_HOST" bidirectional
+  (pin "RADIO_CODEC_USB_HOST_DN" bidirectional
     (at 535.94 260.35 0)
     (effects (font (size 1.27 1.27)) (justify left))
@@
     (effects (font (size 1.27 1.27)) (justify left))
   )
-  (pin "MAKER_USB_DM" bidirectional
+  (pin "MAKER_USB_DN" bidirectional
     (at 674.37 454.66 0)
     (effects (font (size 1.27 1.27)) (justify left))
@@
     (effects (font (size 1.27 1.27)) (justify left))
   )
-  (pin "RADIO_CODEC_USB_DM_HOST" bidirectional
+  (pin "RADIO_CODEC_USB_HOST_DN" bidirectional
     (at 814.07 345.44 0)
     (effects (font (size 1.27 1.27)) (justify left))
   )
-  (pin "RADIO_CODEC_USB_DP_HOST" bidirectional
+  (pin "RADIO_CODEC_USB_HOST_DP" bidirectional
     (at 814.07 350.52 0)
     (effects (font (size 1.27 1.27)) (justify left))
@@
     (effects (font (size 1.27 1.27)) (justify left))
   )
-  (pin "AUDIO_USB_DM" bidirectional
+  (pin "AUDIO_USB_DN" bidirectional
     (at 814.07 360.68 0)
     (effects (font (size 1.27 1.27)) (justify left))
@@
     (effects (font (size 1.27 1.27)) (justify left))
   )
-  (pin "HUB_DS4_DM" bidirectional
+  (pin "HUB_DS4_DN" bidirectional
     (at 480.06 125.73 0)
     (effects (font (size 1.27 1.27)) (justify left))
@@
     (effects (font (size 1.27 1.27)) (justify left))
   )
-  (pin "USBC1_DM" bidirectional
+  (pin "USBC1_DN" bidirectional
     (at 480.06 140.97 0)
     (effects (font (size 1.27 1.27)) (justify left))
@@
     (effects (font (size 1.27 1.27)) (justify left))
   )
-  (pin "USBC2_DM" bidirectional
+  (pin "USBC2_DN" bidirectional
     (at 480.06 151.13 0)
     (effects (font (size 1.27 1.27)) (justify left))
@@
     (effects (font (size 1.27 1.27)) (justify left))
   )
-  (pin "HUB_DS1_DM" bidirectional
+  (pin "HUB_DS1_DN" bidirectional
     (at 480.06 161.29 0)
     (effects (font (size 1.27 1.27)) (justify left))
@@
     (effects (font (size 1.27 1.27)) (justify left))
   )
-  (pin "HUB_DS4_DM" bidirectional
+  (pin "HUB_DS4_DN" bidirectional
     (at 549.91 85.09 0)
     (effects (font (size 1.27 1.27)) (justify left))
@@
     (effects (font (size 1.27 1.27)) (justify left))
   )
-  (pin "HUB_DS1_DM" bidirectional
+  (pin "HUB_DS1_DN" bidirectional
     (at 549.91 151.13 0)
     (effects (font (size 1.27 1.27)) (justify left))
@@
   (effects (font (size 1.27 1.27)) (justify left bottom))
 )
-(label "MCU_USB_DM"
+(label "MCU_USB_DN"
   (at 219.71 308.61 0)
   (effects (font (size 1.27 1.27)) (justify left bottom))
 )
-(label "MCU_USB_DM"
+(label "MCU_USB_DN"
   (at 405.13 400.05 0)
   (effects (font (size 1.27 1.27)) (justify left bottom))
@@
   (effects (font (size 1.27 1.27)) (justify left bottom))
 )
-(label "AUDIO_USB_DM"
+(label "AUDIO_USB_DN"
   (at 359.41 69.85 0)
   (effects (font (size 1.27 1.27)) (justify left bottom))
 )
-(label "AUDIO_USB_DM"
+(label "AUDIO_USB_DN"
   (at 814.07 360.68 0)
   (effects (font (size 1.27 1.27)) (justify left bottom))
@@
   (effects (font (size 1.27 1.27)) (justify left bottom))
 )
-(label "USBC2_DM"
+(label "USBC2_DN"
   (at 359.41 227.33 0)
   (effects (font (size 1.27 1.27)) (justify left bottom))
 )
-(label "USBC2_DM"
+(label "USBC2_DN"
   (at 480.06 151.13 0)
   (effects (font (size 1.27 1.27)) (justify left bottom))
 )
-(label "USBC1_DM"
+(label "USBC1_DN"
   (at 359.41 232.41 0)
   (effects (font (size 1.27 1.27)) (justify left bottom))
 )
-(label "USBC1_DM"
+(label "USBC1_DN"
   (at 480.06 140.97 0)
   (effects (font (size 1.27 1.27)) (justify left bottom))
@@
   (effects (font (size 1.27 1.27)) (justify left bottom))
 )
-(label "MAKER_USB_DM"
+(label "MAKER_USB_DN"
   (at 359.41 247.65 0)
   (effects (font (size 1.27 1.27)) (justify left bottom))
 )
-(label "MAKER_USB_DM"
+(label "MAKER_USB_DN"
   (at 674.37 454.66 0)
   (effects (font (size 1.27 1.27)) (justify left bottom))
 )
-(label "EC_HOST_USB_DM"
+(label "EC_HOST_USB_DN"
   (at 359.41 252.73 0)
   (effects (font (size 1.27 1.27)) (justify left bottom))
 )
-(label "EC_HOST_USB_DM"
+(label "EC_HOST_USB_DN"
   (at 405.13 415.29 0)
   (effects (font (size 1.27 1.27)) (justify left bottom))
@@
   (effects (font (size 1.27 1.27)) (justify left bottom))
 )
-(label "TRACKPAD_USB_DM"
+(label "TRACKPAD_USB_DN"
   (at 359.41 267.97 0)
   (effects (font (size 1.27 1.27)) (justify left bottom))
 )
-(label "TRACKPAD_USB_DM"
+(label "TRACKPAD_USB_DN"
   (at 405.13 435.61 0)
   (effects (font (size 1.27 1.27)) (justify left bottom))
@@
   (effects (font (size 1.27 1.27)) (justify left bottom))
 )
-(label "HUB_DS4_DM"
+(label "HUB_DS4_DN"
   (at 480.06 125.73 0)
   (effects (font (size 1.27 1.27)) (justify left bottom))
 )
-(label "HUB_DS4_DM"
+(label "HUB_DS4_DN"
   (at 549.91 85.09 0)
   (effects (font (size 1.27 1.27)) (justify left bottom))
@@
   (effects (font (size 1.27 1.27)) (justify left bottom))
 )
-(label "HUB_DS1_DM"
+(label "HUB_DS1_DN"
   (at 480.06 161.29 0)
   (effects (font (size 1.27 1.27)) (justify left bottom))
 )
-(label "HUB_DS1_DM"
+(label "HUB_DS1_DN"
   (at 549.91 151.13 0)
   (effects (font (size 1.27 1.27)) (justify left bottom))
@@
   (effects (font (size 1.27 1.27)) (justify left bottom))
 )
-(label "RADIO_CODEC_USB_DP_HOST"
+(label "RADIO_CODEC_USB_HOST_DP"
   (at 535.94 255.27 0)
   (effects (font (size 1.27 1.27)) (justify left bottom))
 )
-(label "RADIO_CODEC_USB_DP_HOST"
+(label "RADIO_CODEC_USB_HOST_DP"
   (at 814.07 350.52 0)
   (effects (font (size 1.27 1.27)) (justify left bottom))
 )
-(label "RADIO_CODEC_USB_DM_HOST"
+(label "RADIO_CODEC_USB_HOST_DN"
   (at 535.94 260.35 0)
   (effects (font (size 1.27 1.27)) (justify left bottom))
 )
-(label "RADIO_CODEC_USB_DM_HOST"
+(label "RADIO_CODEC_USB_HOST_DN"
   (at 814.07 345.44 0)
   (effects (font (size 1.27 1.27)) (justify left bottom))
