File: ducktop2.kicad_sch (KiCad schematic)
At the start: 0 parts

Commit message: fix audit issues and move some connectors
Other:
- sheet FPC-3 (BMS) ports: added PACK_CHG_TEMP_OK; removed none
- sheet Power & Battery ports: added PACK_CHG_TEMP_OK; removed none
Changed lines of the file:
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@@
+    (effects (font (size 1.27 1.27)) (justify left))
+  )
+  (pin "PACK_CHG_TEMP_OK" bidirectional
+    (at 90.17 105.41 0)
+    (effects (font (size 1.27 1.27)) (justify left))
+  )
+  (pin "PACK_FAULT_N" bidirectional
+    (at 90.17 110.49 0)
     (effects (font (size 1.27 1.27)) (justify left))
   )
   (pin "AUX_DC_RAW" bidirectional
-    (at 90.17 105.41 0)
+    (at 90.17 115.57 0)
     (effects (font (size 1.27 1.27)) (justify left))
   )
   (pin "AUX_FAULT_N" bidirectional
-    (at 90.17 110.49 0)
+    (at 90.17 120.65 0)
     (effects (font (size 1.27 1.27)) (justify left))
   )
   (pin "AUX_PGOOD" bidirectional
-    (at 90.17 115.57 0)
+    (at 90.17 125.73 0)
     (effects (font (size 1.27 1.27)) (justify left))
   )
   (pin "AUX_DC_ADC" bidirectional
-    (at 90.17 120.65 0)
+    (at 90.17 130.81 0)
     (effects (font (size 1.27 1.27)) (justify left))
   )
   (pin "MAIN_USB_VALID_N" bidirectional
-    (at 90.17 125.73 0)
+    (at 90.17 135.89 0)
     (effects (font (size 1.27 1.27)) (justify left))
   )
   (pin "MAIN_AUX_VALID_N" bidirectional
-    (at 90.17 130.81 0)
+    (at 90.17 140.97 0)
     (effects (font (size 1.27 1.27)) (justify left))
   )
   (pin "USB_PD_SELECTED" bidirectional
-    (at 90.17 135.89 0)
+    (at 90.17 146.05 0)
     (effects (font (size 1.27 1.27)) (justify left))
   )
   (pin "PD2_VALID_N" bidirectional
-    (at 90.17 140.97 0)
+    (at 90.17 151.13 0)
     (effects (font (size 1.27 1.27)) (justify left))
   )
   (pin "PD2_VBUS_GATED" bidirectional
-    (at 90.17 146.05 0)
+    (at 90.17 156.21 0)
     (effects (font (size 1.27 1.27)) (justify left))
   )
   (pin "PD1_VBUS_RAW" bidirectional
-    (at 90.17 151.13 0)
+    (at 90.17 161.29 0)
     (effects (font (size 1.27 1.27)) (justify left))
   )
   (pin "PD2_VBUS_RAW" bidirectional
-    (at 90.17 156.21 0)
+    (at 90.17 166.37 0)
     (effects (font (size 1.27 1.27)) (justify left))
   )
   (pin "AON_FAULT_N" bidirectional
-    (at 90.17 161.29 0)
+    (at 90.17 171.45 0)
     (effects (font (size 1.27 1.27)) (justify left))
   )
   (pin "EC_AON_IN" bidirectional
-    (at 90.17 166.37 0)
-    (effects (font (size 1.27 1.27)) (justify left))
-  )
-  (pin "PACK_FAULT_N" bidirectional
-    (at 90.17 171.45 0)
+    (at 90.17 176.53 0)
     (effects (font (size 1.27 1.27)) (justify left))
   )
@@
     (effects (font (size 1.27 1.27)) (justify left top))
   )
-  (pin "FG_VSS" bidirectional
+  (pin "PACK_FAULT_N" bidirectional
     (at 619.76 44.45 0)
     (effects (font (size 1.27 1.27)) (justify left))
   )
+  (pin "PACK_RETRY_PULSE" bidirectional
+    (at 619.76 49.53 0)
+    (effects (font (size 1.27 1.27)) (justify left))
+  )
   (pin "MCU_3V3" bidirectional
-    (at 619.76 49.53 0)
-    (effects (font (size 1.27 1.27)) (justify left))
-  )
-  (pin "PACK_RETRY_PULSE" bidirectional
     (at 619.76 54.61 0)
     (effects (font (size 1.27 1.27)) (justify left))
   )
-  (pin "PACK_FAULT_N" bidirectional
+  (pin "PACK_CHG_TEMP_OK" bidirectional
     (at 619.76 59.69 0)
     (effects (font (size 1.27 1.27)) (justify left))
@@
     (effects (font (size 1.27 1.27)) (justify left))
   )
+  (pin "FG_VSS" bidirectional
+    (at 619.76 69.85 0)
+    (effects (font (size 1.27 1.27)) (justify left))
+  )
 )
 (label "BQ_ALERT"
@@
 )
 (label "MCU_3V3"
-  (at 619.76 49.53 0)
+  (at 619.76 54.61 0)
   (effects (font (size 1.27 1.27)) (justify left bottom))
 )
@@
 )
 (label "FG_VSS"
-  (at 619.76 44.45 0)
+  (at 619.76 69.85 0)
   (effects (font (size 1.27 1.27)) (justify left bottom))
 )
@@
   (effects (font (size 1.27 1.27)) (justify left bottom))
 )
+(label "PACK_CHG_TEMP_OK"
+  (at 90.17 105.41 0)
+  (effects (font (size 1.27 1.27)) (justify left bottom))
+)
+(label "PACK_CHG_TEMP_OK"
+  (at 619.76 59.69 0)
+  (effects (font (size 1.27 1.27)) (justify left bottom))
+)
+(label "PACK_FAULT_N"
+  (at 90.17 110.49 0)
+  (effects (font (size 1.27 1.27)) (justify left bottom))
+)
+(label "PACK_FAULT_N"
+  (at 219.71 471.17 0)
+  (effects (font (size 1.27 1.27)) (justify left bottom))
+)
+(label "PACK_FAULT_N"
+  (at 619.76 44.45 0)
+  (effects (font (size 1.27 1.27)) (justify left bottom))
+)
 (label "AUX_DC_RAW"
-  (at 90.17 105.41 0)
+  (at 90.17 115.57 0)
   (effects (font (size 1.27 1.27)) (justify left bottom))
 )
@@
 )
 (label "AUX_FAULT_N"
-  (at 90.17 110.49 0)
+  (at 90.17 120.65 0)
   (effects (font (size 1.27 1.27)) (justify left bottom))
 )
@@
 )
 (label "AUX_PGOOD"
-  (at 90.17 115.57 0)
+  (at 90.17 125.73 0)
   (effects (font (size 1.27 1.27)) (justify left bottom))
 )
@@
 )
 (label "AUX_DC_ADC"
-  (at 90.17 120.65 0)
+  (at 90.17 130.81 0)
   (effects (font (size 1.27 1.27)) (justify left bottom))
 )
@@
 )
 (label "MAIN_USB_VALID_N"
-  (at 90.17 125.73 0)
+  (at 90.17 135.89 0)
   (effects (font (size 1.27 1.27)) (justify left bottom))
 )
@@
 )
 (label "MAIN_AUX_VALID_N"
-  (at 90.17 130.81 0)
+  (at 90.17 140.97 0)
   (effects (font (size 1.27 1.27)) (justify left bottom))
 )
@@
 )
 (label "USB_PD_SELECTED"
-  (at 90.17 135.89 0)
+  (at 90.17 146.05 0)
   (effects (font (size 1.27 1.27)) (justify left bottom))
 )
@@
 )
 (label "PD2_VALID_N"
-  (at 90.17 140.97 0)
+  (at 90.17 151.13 0)
   (effects (font (size 1.27 1.27)) (justify left bottom))
 )
@@
 )
 (label "PD2_VBUS_GATED"
-  (at 90.17 146.05 0)
+  (at 90.17 156.21 0)
   (effects (font (size 1.27 1.27)) (justify left bottom))
 )
@@
 )
 (label "PD1_VBUS_RAW"
-  (at 90.17 151.13 0)
+  (at 90.17 161.29 0)
   (effects (font (size 1.27 1.27)) (justify left bottom))
 )
@@
 )
 (label "PD2_VBUS_RAW"
-  (at 90.17 156.21 0)
+  (at 90.17 166.37 0)
   (effects (font (size 1.27 1.27)) (justify left bottom))
 )
@@
 )
 (label "AON_FAULT_N"
-  (at 90.17 161.29 0)
+  (at 90.17 171.45 0)
   (effects (font (size 1.27 1.27)) (justify left bottom))
 )
@@
 )
 (label "EC_AON_IN"
-  (at 90.17 166.37 0)
+  (at 90.17 176.53 0)
   (effects (font (size 1.27 1.27)) (justify left bottom))
 )
@@
   (effects (font (size 1.27 1.27)) (justify left bottom))
 )
-(label "PACK_FAULT_N"
-  (at 90.17 171.45 0)
-  (effects (font (size 1.27 1.27)) (justify left bottom))
-)
-(label "PACK_FAULT_N"
-  (at 219.71 471.17 0)
-  (effects (font (size 1.27 1.27)) (justify left bottom))
-)
-(label "PACK_FAULT_N"
-  (at 619.76 59.69 0)
-  (effects (font (size 1.27 1.27)) (justify left bottom))
-)
 (label "KB_ROW2"
   (at 219.71 44.45 0)
@@
 )
 (label "PACK_RETRY_PULSE"
-  (at 619.76 54.61 0)
-  (effects (font (size 1.27 1.27)) (justify left bottom))
-)
+  (at 619.76 49.53 0)
+  (effects (font (size 1.27 1.27)) (justify left bottom))
+)

Commit message: fix the center layout and more board issues
Other:
- sheet FPC-1 (Left) ports: added PD2_SOURCE_PG, SERVICE_MUX_RESET_N, USB_J11_PERMIT, USB_J12_PERMIT; removed USB_PORT_5V
- sheet FPC-2 (Right) ports: added PD2_SOURCE_PG, USB_J11_PERMIT, USB_J12_PERMIT; removed USB_PORT_5V
