File: 09_radio_daughterboard_interface.kicad_sch (KiCad schematic)
At the start: 60 parts, among them J2300 FH12-30S 30-pin radio daughte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, Q2300 2N7002K radio-PG USB enable, U2300 TPS259470ARPW 2A reverse-bloc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, U2301 TLV803EA43 4.3V radio rail su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, U2302 SN74LVC1G17DBVR radio PG leve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, U2303 TS3USB30E default-disconnecte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, U2304 TPS2553D radio codec VBUS gat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, U2305 USBLC6-2P6 radio codec USB ESD

Commit message: get the main boards ready for routing
Connections:
- net RADIO_CODEC_USB_DM_DB renamed RADIO_CODEC_USB_DB_DN
- net RADIO_CODEC_USB_DM_HOST renamed RADIO_CODEC_USB_HOST_DN
- net RADIO_CODEC_USB_DP_DB renamed RADIO_CODEC_USB_DB_DP
- net RADIO_CODEC_USB_DP_HOST renamed RADIO_CODEC_USB_HOST_DP
Changed lines of the file:
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@@
   (effects (font (size 1.27 1.27)) (justify left bottom))
 )
-(hierarchical_label "RADIO_CODEC_USB_DP_HOST"
+(hierarchical_label "RADIO_CODEC_USB_HOST_DP"
   (shape bidirectional)
   (at 160.02 240.03 0)
@@
 )
 (no_connect (at 160.02 247.65))
-(label "RADIO_CODEC_USB_DP_DB"
+(label "RADIO_CODEC_USB_DB_DP"
   (at 139.7 240.03 0)
   (effects (font (size 1.27 1.27)) (justify left bottom))
@@
   (effects (font (size 1.27 1.27)) (justify left bottom))
 )
-(label "RADIO_CODEC_USB_DM_DB"
+(label "RADIO_CODEC_USB_DB_DN"
   (at 139.7 242.57 0)
   (effects (font (size 1.27 1.27)) (justify left bottom))
 )
 (no_connect (at 160.02 250.19))
-(hierarchical_label "RADIO_CODEC_USB_DM_HOST"
+(hierarchical_label "RADIO_CODEC_USB_HOST_DN"
   (shape bidirectional)
   (at 160.02 242.57 0)
@@
   )
 )
-(label "RADIO_CODEC_USB_DP_DB"
+(label "RADIO_CODEC_USB_DB_DP"
   (at 514.35 245.11 0)
   (effects (font (size 1.27 1.27)) (justify left bottom))
 )
-(label "RADIO_CODEC_USB_DP_DB"
+(label "RADIO_CODEC_USB_DB_DP"
   (at 524.51 245.11 0)
   (effects (font (size 1.27 1.27)) (justify left bottom))
 )
-(label "RADIO_CODEC_USB_DM_DB"
+(label "RADIO_CODEC_USB_DB_DN"
   (at 514.35 247.65 0)
   (effects (font (size 1.27 1.27)) (justify left bottom))
 )
-(label "RADIO_CODEC_USB_DM_DB"
+(label "RADIO_CODEC_USB_DB_DN"
   (at 524.51 247.65 0)
   (effects (font (size 1.27 1.27)) (justify left bottom))
@@
   (effects (font (size 1.27 1.27)) (justify left bottom))
 )
-(label "RADIO_CODEC_USB_DP_DB"
+(label "RADIO_CODEC_USB_DB_DP"
   (at 364.49 521.97 0)
   (effects (font (size 1.27 1.27)) (justify left bottom))
 )
-(label "RADIO_CODEC_USB_DM_DB"
+(label "RADIO_CODEC_USB_DB_DN"
   (at 364.49 524.51 0)
   (effects (font (size 1.27 1.27)) (justify left bottom))

Commit message: fix the center layout and more board issues
Parts:
- C2303: renamed from C2304; value 100n RADIO_DB_5V output HF -> 22u 25V RADIO_DB_5V bulk; TI characterized part; footprint Capacitor_SMD:C_0603_1608Metric -> Capacitor_SMD:C_1210_3225Metric; MPN GRM188R71H104KA93D -> GRM32ER71E226KE15L
- C2304: renamed from C2303; value 22u RADIO_DB_5V output bulk -> 100n RADIO_DB_5V output HF; footprint Capacitor_SMD:C_1206_3216Metric -> Capacitor_SMD:C_0603_1608Metric; MPN GRM31CZ71C226ME15L -> GRM188R71H104KA93D
Other:
- moved on the sheet: C2303, C2304
Changed lines of the file:
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@@
-(symbol
-  (lib_id "Device:C")
-  (at 20.32 139.7 0)
-  (unit 1)
-  (exclude_from_sim no)
-  (in_bom yes)
-  (on_board yes)
-  (dnp no)
-  (property "Reference" "C2303" (at 20.32 137.16 0) (effects (font (size 1.27 1.27))))
-  (property "Value" "22u RADIO_DB_5V output bulk" (at 20.32 142.24 0) (effects (font (size 1.27 1.27))))
-  (property "Footprint" "Capacitor_SMD:C_1206_3216Metric" (at 20.32 139.7 0) (effects (font (size 1.27 1.27)) (hide yes)))
-  (property "Datasheet" "" (at 20.32 139.7 0) (effects (font (size 1.27 1.27)) (hide yes)))
-  (property "Manufacturer" "Murata" (at 20.32 139.7 0) (effects (font (size 1.27 1.27)) (hide yes)))
-  (property "MPN" "GRM31CZ71C226ME15L" (at 20.32 139.7 0) (effects (font (size 1.27 1.27)) (hide yes)))
-  (pin "1")
-  (pin "2")
-  (instances
-    (project "ducktop2"
-      (path "/c1b99a0d-daca-57b5-85ae-3ffd9c9575e8"
-        (reference "C2303")
-        (unit 1)
-      )
-    )
-  )
-)
-(label "RADIO_DB_5V"
-  (at 20.32 135.89 0)
-  (effects (font (size 1.27 1.27)) (justify left bottom))
-)
-(label "GND"
-  (at 20.32 143.51 0)
-  (effects (font (size 1.27 1.27)) (justify left bottom))
-)
 (symbol
   (lib_id "Device:C")
@@
   (effects (font (size 1.27 1.27)) (justify left bottom))
 )
+(symbol
+  (lib_id "Device:C")
+  (at 20.32 139.7 0)
+  (unit 1)
+  (exclude_from_sim no)
+  (in_bom yes)
+  (on_board yes)
+  (dnp no)
+  (property "Reference" "C2303" (at 20.32 137.16 0) (effects (font (size 1.27 1.27))))
+  (property "Value" "22u 25V RADIO_DB_5V bulk; TI characterized part" (at 20.32 142.24 0) (effects (font (size 1.27 1.27))))
+  (property "Footprint" "Capacitor_SMD:C_1210_3225Metric" (at 20.32 139.7 0) (effects (font (size 1.27 1.27)) (hide yes)))
+  (property "Datasheet" "" (at 20.32 139.7 0) (effects (font (size 1.27 1.27)) (hide yes)))
+  (property "Manufacturer" "Murata" (at 20.32 139.7 0) (effects (font (size 1.27 1.27)) (hide yes)))
+  (property "MPN" "GRM32ER71E226KE15L" (at 20.32 139.7 0) (effects (font (size 1.27 1.27)) (hide yes)))
+  (pin "1")
+  (pin "2")
+  (instances
+    (project "ducktop2"
+      (path "/c1b99a0d-daca-57b5-85ae-3ffd9c9575e8"
+        (reference "C2303")
+        (unit 1)
+      )
+    )
+  )
+)
+(label "RADIO_DB_5V"
+  (at 20.32 135.89 0)
+  (effects (font (size 1.27 1.27)) (justify left bottom))
+)
+(label "GND"
+  (at 20.32 143.51 0)
+  (effects (font (size 1.27 1.27)) (justify left bottom))
+)
