File: 15_system_audio.kicad_sch (KiCad schematic)
At the start: 90 parts, among them J420 Left 8-ohm BTL speaker; pin 1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, J421 Right 8-ohm BTL speaker; pin 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, U400 USB2512B-AEZG-TR two-port HS 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, U401 TLV803EA29RDBZR 2.93V reset s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, U402 TPS2052BDR dual 500mA USB pow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, U410 PCM2900CDBR USB Audio Class s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, U420 TPA2012D2RTJR stereo BTL clas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, U421 SN74LVC1G08DBVR SSPND AND EC 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, U430 LP5907MFX-2.8/NOPB low-noise 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, U431 TLV9061IDBVR microphone pream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, Y400 ABM8-24.000MHZ-10-1-U-T 24MHz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, Y410 ABM8G-106-12.000MHZ-T 12MHz 1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

Commit message: Finish USB-C policy and split out radio board
Parts:
- C403: value 10u radio-codec VBUS -> 10u radio-codec host VBUS
- R402: value 10k NON_REM1 strap high -> 100k NON_REM1 strap low
- R403: value 100k NON_REM0 strap low -> 10k NON_REM0 strap high
- U400: Configuration CFG_SEL[1:0]=00 self-powered straps; NON_REM[1:0]=10 -> CFG_SEL[1:0]=00 self-powered; system-codec port 1 non-remov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
Connections:
- net RADIO_CODEC_USB_DM is gone; now on net SYSTEM_DAC_USB_DM: U400.1 (USBDM_DN1/PRT_DIS_M1)
- net RADIO_CODEC_USB_DP is gone; now on net SYSTEM_DAC_USB_DP: U400.2 (USBDP_DN1/PRT_DIS_P1)
- net GND: now also R402.2; no longer R403.2
- net SYSTEM_DAC_USB_DM: no longer U400.3 (USBDM_DN2/PRT_DIS_M2)
- net SYSTEM_DAC_USB_DP: no longer U400.4 (USBDP_DN2/PRT_DIS_P2)
- net SYSTEM_DAC_USB_VBUS: now also U402.7 (OUT1); no longer U402.6 (OUT2)
- net SYS_3V3: now also R403.2; no longer R402.2
- net RADIO_CODEC_USB_VBUS renamed RADIO_CODEC_USB_VBUS_HOST
- net RADIO_CODEC_USB_VBUS_HOST: now also U402.6 (OUT2); no longer U402.7 (OUT1)
- new net RADIO_CODEC_USB_DM_HOST: U400.3 (USBDM_DN2/PRT_DIS_M2)
- new net RADIO_CODEC_USB_DP_HOST: U400.4 (USBDP_DN2/PRT_DIS_P2)
Other:
- note added: "== U400 USB2512B-AEZG-TR: self-powered, port 1 non-removable, port 2 removable =="
- note added: "Mu USB2_P5 feeds a self-powered USB2512B multi-TT hub. Port 1 is the fixed PCM2900C system codec; port 2 is the optional radio daughterboard."
- note added: "Port 1 is non-removable. Port 2 is removable and may be empty; TPS2052B provides individual protected VBUS outputs."
- note removed: "== U400 USB2512B-AEZG-TR: self-powered, strap-configured, both ports non-removable =="
- note removed: "Both downstream devices are non-removable. TPS2052B implements host-controlled VBUS and individual overcurrent feedback."
- note removed: "Mu USB2_P5 feeds a self-powered USB2512B multi-TT hub. Port 1 is the existing radio codec; port 2 is the PCM2900C system codec."
Changed lines of the file:
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@@
   (paper "A2")
 (text "== System audio: embedded two-port USB hub, playback/record codec, microphone, and stereo BTL amplifier ==" (at 20.32 12.7 0) (effects (font (size 1.27 1.27))))
-(text "Mu USB2_P5 feeds a self-powered USB2512B multi-TT hub. Port 1 is the existing radio codec; port 2 is the PCM2900C system codec." (at 20.32 20.32 0) (effects (font (size 1.27 1.27))))
-(text "Both downstream devices are non-removable. TPS2052B implements host-controlled VBUS and individual overcurrent feedback." (at 20.32 27.94 0) (effects (font (size 1.27 1.27))))
+(text "Mu USB2_P5 feeds a self-powered USB2512B multi-TT hub. Port 1 is the fixed PCM2900C system codec; port 2 is the optional radio daughterboard." (at 20.32 20.32 0) (effects (font (size 1.27 1.27))))
+(text "Port 1 is non-removable. Port 2 is removable and may be empty; TPS2052B provides individual protected VBUS outputs." (at 20.32 27.94 0) (effects (font (size 1.27 1.27))))
 (text "== Protected 5V audio branch and downstream USB power ==" (at 20.32 45.72 0) (effects (font (size 1.27 1.27))))
 (symbol
@@
   (effects (font (size 1.27 1.27)) (justify left bottom))
 )
+(hierarchical_label "RADIO_CODEC_USB_VBUS_HOST"
+  (shape bidirectional)
+  (at 289.56 64.77 0)
+  (effects (font (size 1.27 1.27)) (justify left bottom))
+)
 (label "SYSTEM_DAC_USB_VBUS"
-  (at 289.56 64.77 0)
-  (effects (font (size 1.27 1.27)) (justify left bottom))
-)
-(hierarchical_label "RADIO_CODEC_USB_VBUS"
-  (shape bidirectional)
   (at 289.56 62.23 0)
   (effects (font (size 1.27 1.27)) (justify left bottom))
@@
   (dnp no)
   (property "Reference" "C403" (at 500.38 60.96 0) (effects (font (size 1.27 1.27))))
-  (property "Value" "10u radio-codec VBUS" (at 500.38 66.04 0) (effects (font (size 1.27 1.27))))
+  (property "Value" "10u radio-codec host VBUS" (at 500.38 66.04 0) (effects (font (size 1.27 1.27))))
   (property "Footprint" "Capacitor_SMD:C_1206_3216Metric" (at 500.38 63.5 0) (effects (font (size 1.27 1.27)) (hide yes)))
   (property "Datasheet" "" (at 500.38 63.5 0) (effects (font (size 1.27 1.27)) (hide yes)))
@@
   )
 )
-(hierarchical_label "RADIO_CODEC_USB_VBUS"
+(hierarchical_label "RADIO_CODEC_USB_VBUS_HOST"
   (shape bidirectional)
   (at 500.38 59.69 0)
@@
   )
 )
-(hierarchical_label "RADIO_CODEC_USB_VBUS"
+(hierarchical_label "RADIO_CODEC_USB_VBUS_HOST"
   (shape bidirectional)
   (at 500.38 72.39 0)
@@
   (effects (font (size 1.27 1.27)) (justify left bottom))
 )
-(text "== U400 USB2512B-AEZG-TR: self-powered, strap-configured, both ports non-removable ==" (at 20.32 93.98 0) (effects (font (size 1.27 1.27))))
+(text "== U400 USB2512B-AEZG-TR: self-powered, port 1 non-removable, port 2 removable ==" (at 20.32 93.98 0) (effects (font (size 1.27 1.27))))
 (symbol
   (lib_id "USB2512B:USB2512B")
@@
   (property "Manufacturer" "Microchip Technology" (at 299.72 160.02 0) (effects (font (size 1.27 1.27)) (hide yes)))
   (property "MPN" "USB2512B-AEZG-TR" (at 299.72 160.02 0) (effects (font (size 1.27 1.27)) (hide yes)))
-  (property "Configuration" "CFG_SEL[1:0]=00 self-powered straps; NON_REM[1:0]=10" (at 299.72 160.02 0) (effects (font (size 1.27 1.27)) (hide yes)))
+  (property "Configuration" "CFG_SEL[1:0]=00 self-powered; system-codec port 1 non-removable; radio port 2 removable" (at 299.72 160.02 0) (effects (font (size 1.27 1.27)) (hide yes)))
   (property "ReferenceCircuit" "Current DS00001692 plus DS00004539A hardware checklist" (at 299.72 160.02 0) (effects (font (size 1.27 1.27)) (hide yes)))
   (pin "1")
@@
   )
 )
-(hierarchical_label "RADIO_CODEC_USB_DM"
-  (shape bidirectional)
+(label "SYSTEM_DAC_USB_DM"
   (at 317.5 144.78 0)
   (effects (font (size 1.27 1.27)) (justify left bottom))
 )
-(hierarchical_label "RADIO_CODEC_USB_DP"
-  (shape bidirectional)
+(label "SYSTEM_DAC_USB_DP"
   (at 317.5 147.32 0)
   (effects (font (size 1.27 1.27)) (justify left bottom))
 )
-(label "SYSTEM_DAC_USB_DM"
+(hierarchical_label "RADIO_CODEC_USB_DM_HOST"
+  (shape bidirectional)
   (at 317.5 149.86 0)
   (effects (font (size 1.27 1.27)) (justify left bottom))
 )
-(label "SYSTEM_DAC_USB_DP"
+(hierarchical_label "RADIO_CODEC_USB_DP_HOST"
+  (shape bidirectional)
   (at 317.5 152.4 0)
   (effects (font (size 1.27 1.27)) (justify left bottom))
@@
   (dnp no)
   (property "Reference" "R402" (at 20.32 175.26 0) (effects (font (size 1.27 1.27))))
-  (property "Value" "10k NON_REM1 strap high" (at 20.32 180.34 0) (effects (font (size 1.27 1.27))))
+  (property "Value" "100k NON_REM1 strap low" (at 20.32 180.34 0) (effects (font (size 1.27 1.27))))
   (property "Footprint" "Resistor_SMD:R_0603_1608Metric" (at 20.32 177.8 0) (effects (font (size 1.27 1.27)) (hide yes)))
   (property "Datasheet" "" (at 20.32 177.8 0) (effects (font (size 1.27 1.27)) (hide yes)))
@@
   (effects (font (size 1.27 1.27)) (justify left bottom))
 )
-(hierarchical_label "SYS_3V3"
-  (shape bidirectional)
+(label "GND"
   (at 20.32 181.61 0)
   (effects (font (size 1.27 1.27)) (justify left bottom))
@@
   (dnp no)
   (property "Reference" "R403" (at 149.86 175.26 0) (effects (font (size 1.27 1.27))))
-  (property "Value" "100k NON_REM0 strap low" (at 149.86 180.34 0) (effects (font (size 1.27 1.27))))
+  (property "Value" "10k NON_REM0 strap high" (at 149.86 180.34 0) (effects (font (size 1.27 1.27))))
   (property "Footprint" "Resistor_SMD:R_0603_1608Metric" (at 149.86 177.8 0) (effects (font (size 1.27 1.27)) (hide yes)))
   (property "Datasheet" "" (at 149.86 177.8 0) (effects (font (size 1.27 1.27)) (hide yes)))
@@
   (effects (font (size 1.27 1.27)) (justify left bottom))
 )
-(label "GND"
+(hierarchical_label "SYS_3V3"
+  (shape bidirectional)
   (at 149.86 181.61 0)
   (effects (font (size 1.27 1.27)) (justify left bottom))

Commit message: Add rear 3.5mm headphone jack with plug-detect speaker mute (sheet 15)
Add the missing headphone output the user-verified behavior requires (row 11): rear CUI SJ1-3535NG stereo jack driven by a TPA6130A2RTJR DirectPath headphone amp, with automatic plug-detect speaker muting like a normal laptop.

- U425 TPA6130A2 (I2C @0x60, fixed): single-ended inputs from PCM2900C DAC_VOUT_L/R via 0.47u coupling (INM signal, INP AC-grounded per datasheet 9.2.2.1); capless ground-referenced HPLEFT/HPRIGHT outputs to jack T/R. Charge-pump flying + CPVSS + VDD bypass per 9.2.2.2/3.
- J422 SJ1-3535NG: RN ring normalling switch is plug detect (unplugged shorts RN to R = amp 0V -> low; plugged floats -> high).
- HP_DETECT is read by the EC on U44 (TCA9539 source manager) recovered spare input pin 6 (SOURCE_MGR_SPARE1 repurposed) with R782 100k pull-up to MCU_3V3. On plug-in the EC drives AUDIO_AMP_EC_EN low (U421 AND gate mutes the TPA2012D2 speaker amp) and I2C-unmutes U425.
- /SD tied to MU_HOST_ACTIVE so U425 is in hardware shutdown (0.4uA) outside S0; power-on default is muted with outputs disabled (fail-safe OFF until EC firmware enables over I2C).
- Datasheet-verified: TPA6130A2 is I2C-controlled (no G0/G1 hardware gain); reuses the TPA2012D2 WQFN-20-1EP 4x4mm EP2.7x2.7 footprint; AudioJack3_SwitchTR symbol matches the SJ1-3535NG 5-pad footprint (T/R/S/TN/RN).
- Contracts (verify_design_contracts, generate_pin_review_table x2, verify_schematic_closure) updated SPARE1->HP_DETECT. Added TPA6130A2 to sym-lib-table+LIBMAP.
- Enlarged System Audio root sheet block 60->85mm so all 14 hier pins fit; KiCad clamps sheet pins that overflow the block to the rectangle edge and merges them, which otherwise collapses I2C_SCL/HP_DETECT/AUDIO_MIC_EN into one net.
- ERC 0 errors/27 intentional warnings; schematic closure 1580/0; pin review 2603/2603.
Parts:
- added C452: 100n TLV9061 local bypass, Capacitor_SMD:C_0603_1608Metric, symbol Device:C
- added C453: 1.2n C0G feedback low-pass, Capacitor_SMD:C_0603_1608Metric, symbol Device:C
- added C454: 4.7u microphone gain-leg AC coupling, Capacitor_SMD:C_1206_3216Metric, symbol Device:C
- added C455: 4.7u microphone to PCM2900 VINL per TI analog fro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, Capacitor_SMD:C_1206_3216Metric, symbol Device:C
- added C456: 4.7u microphone to PCM2900 VINR per TI analog fro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, Capacitor_SMD:C_1206_3216Metric, symbol Device:C
- added C457: 0.47u L input coupling to LEFTINM, Capacitor_SMD:C_0805_2012Metric, symbol Device:C
- added C458: 0.47u L INP AC-ground reference, Capacitor_SMD:C_0805_2012Metric, symbol Device:C
- added C459: 0.47u R input coupling to RIGHTINM, Capacitor_SMD:C_0805_2012Metric, symbol Device:C
- added R432: 4.99k 1% microphone feedback, Resistor_SMD:R_0603_1608Metric, symbol Device:R
- added R433: 1.00k 1% microphone gain leg, Resistor_SMD:R_0603_1608Metric, symbol Device:R
- added U425: TPA6130A2RTJR DirectPath stereo headphone amp, Package_DFN_QFN:WQFN-20-1EP_4x4mm_P0.5mm_EP2.7x2.7mm_ThermalVias, symbol TPA6130A2:TPA6130A2
- C460: renamed from C452; value 100n TLV9061 local bypass -> 0.47u R INP AC-ground reference; footprint Capacitor_SMD:C_0603_1608Metric -> Capacitor_SMD:C_0805_2012Metric
- C461: renamed from R432; value 4.99k 1% microphone feedback -> 1u charge-pump flying CPP-CPN; footprint Resistor_SMD:R_0603_1608Metric -> Capacitor_SMD:C_0805_2012Metric; symbol Device:R -> Device:C
- C462: renamed from C453; value 1.2n C0G feedback low-pass -> 1u CPVSS negative-rail decoupling; footprint Capacitor_SMD:C_0603_1608Metric -> Capacitor_SMD:C_0805_2012Metric
- C463: renamed from R433; value 1.00k 1% microphone gain leg -> 1u VDD pin 12 analog bypass; footprint Resistor_SMD:R_0603_1608Metric -> Capacitor_SMD:C_0805_2012Metric; symbol Device:R -> Device:C
- C464: renamed from C454; value 4.7u microphone gain-leg AC coupling -> 1u VDD pin 20 charge-pump supply bypass; footprint Capacitor_SMD:C_1206_3216Metric -> Capacitor_SMD:C_0805_2012Metric
- C465: renamed from C455; value 4.7u microphone to PCM2900 VINL per TI analog front-end -> 100n VDD high-frequency bypass; footprint Capacitor_SMD:C_1206_3216Metric -> Capacitor_SMD:C_0603_1608Metric
- J422: renamed from C456; value 4.7u microphone to PCM2900 VINR per TI analog front-end -> CUI SJ1-3535NG rear 3.5mm stereo headphone jack; footprint Capacitor_SMD:C_1206_3216Metric -> Connector_Audio:Jack_3.5mm_CUI_SJ1-3535NG_Horizontal; symbol Device:C -> Connector_Audio:AudioJack3_SwitchTR; Detect (none) -> RN ring normalling switch: closed to R (amp 0V) when unplug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; MPN (none) -> SJ1-3535NG; Manufacturer (none) -> CUI Devices; SpeakerMute (none) -> EC reads HP_DETECT (U44 pin 6) and drives AUDIO_AMP_EC_EN l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
Connections:
- net AUDIO_5V: now also C463.1, C464.1, C465.1, U425.12 (VDD), U425.20 (VDD)
- net DAC_VOUT_L: now also C457.1
- net DAC_VOUT_R: now also C459.1
- net GND: now also C462.2, C463.2, C465.2, J422.S, C452.2, C454.2, C458.2, U425.10 (GND), U425.13 (GND), U425.19 (GND), U425.21 (PAD), U425.3 (GND), U425.9 (GND)
- net MIC_ADC_L: now also C455.2; no longer C465.2
- net MIC_ADC_R: now also C456.2; no longer J422.2
- net MIC_FB: now also C453.2, R432.2, R433.1; no longer C461.2, C462.2, C463.1
- net MIC_HP_NODE: now also C454.1, R433.2; no longer C463.2, C464.1
- net MIC_PREAMP: now also C453.1, C455.1, C456.1, R432.1; no longer C461.1, C462.1, C465.1, J422.1
- net SYS_3V3: now also C452.1; no longer C460.1
- new net CPN: C461.2, U425.17 (CPN)
- new net CPP: C461.1, U425.18 (CPP)
- new net CPVSS: C462.1, U425.15 (CPVSS), U425.16 (CPVSS)
- new net HP_DETECT: J422.RN
- new net HP_INM_L: C457.2, U425.1 (LEFTINM)
- new net HP_INM_R: C459.2, U425.5 (RIGHTINM)
- new net HP_INP_L: C458.1, U425.2 (LEFTINP)
- new net HP_INP_R: C460.1, U425.4 (RIGHTINP)
- new net HP_OUT_L: J422.T, U425.14 (HPLEFT)
- new net HP_OUT_R: J422.R, U425.11 (HPRIGHT)
- new net I2C_SCL: U425.8 (SCL)
- new net I2C_SDA: U425.7 (SDA)
- new net MU_HOST_ACTIVE: U425.6 (~{SD})
- no-connect marks 16 -> 17
Other:
- note added: "== Rear 3.5 mm headphone jack: TPA6130A2 DirectPath I2C headphone amp + plug-detect speaker mute =="
- note added: "DirectPath capless outputs HPLEFT/HPRIGHT drive jack J422 T/R. RN (ring normalling) = HP_DETECT: unplugged shorts RN to R (amp 0V) -> low; plugged floats -> R782 100k pull-up (sheet 02) -> high."
- note added: "EC reads HP_DETECT via U44 pin 6 over I2C; on plug-in it drives AUDIO_AMP_EC_EN low (U421 mutes speakers) and I2C-unmutes U425. /SD tied to MU_HOST_ACTIVE so U425 is in hardware shutdown (0.4uA) outside S0."
- note added: "HEADPHONE LAYOUT: keep the jack, VDD bypass, and charge-pump caps away from the mic preamp (MK430) and class-D speaker outputs."
- note added: "HEADPHONE STANDBY: /SD tied to MU_HOST_ACTIVE (S0-only) so U425 draws 0.4uA in S3; EC unmutes/enables over I2C only while host active."
- note added: "TPA6130A2 @0x60 (fixed). Power-on default = muted, outputs disabled (fail-safe OFF until EC firmware unmutes/enables over I2C). No G0/G1 hardware gain; 64-step I2C volume gives independent headphone level."
- note added: "U425 taps the PCM2900C DAC_VOUT_L/R line outputs single-ended (0.47u coupling into LEFTINM/RIGHTINM, INP AC-grounded)."
- moved on the sheet: C460, C462, C464, C465

Commit message: Stamp generation-time BOM catalog; close 378 procurement gaps
Parts:
- C400, C405, C406, C407, C408, C409, C410, C412, C413, C416, C428, C440, C450, C452, C465: MPN (none) -> GRM188R71H104KA93D; Manufacturer (none) -> Murata
- C401, C403, C404, C423, C429, C441: MPN (none) -> GRM31CR71E106KA12L; Manufacturer (none) -> Murata
- C402, C411, C422, C424, C425, C426, C427, C448, C449: MPN (none) -> GRM21BR71A105KA01L; Manufacturer (none) -> Murata
- C414, C415, C420, C421: MPN (none) -> GRM1885C1H180JA01; Manufacturer (none) -> Murata
- C430, C431: MPN (none) -> GRM188R71H473KA01; Manufacturer (none) -> Murata
- C432, C433, C434, C435, C461, C462, C463, C464: MPN (none) -> GRM21BR71H105KA01; Manufacturer (none) -> Murata
- C442, C443, C444, C445: MPN (none) -> GRM155R71H102KA01; Manufacturer (none) -> Murata
- C453: MPN (none) -> GRM1885C1H122JA01; Manufacturer (none) -> Murata
- C454, C455, C456: MPN (none) -> GRM31CR61C475KA01; Manufacturer (none) -> Murata
- C457, C458, C459, C460: MPN (none) -> GRM21BR71H474KA01; Manufacturer (none) -> Murata
- R400: MPN (none) -> RC0603FR-0712K0L; Manufacturer (none) -> Yageo
- R401, R403, R408, R409: MPN (none) -> RC0603FR-0710KL; Manufacturer (none) -> Yageo
- R402, R404, R405, R415, R416, R434: MPN (none) -> RC0603FR-07100KL; Manufacturer (none) -> Yageo
- R410, R411: MPN (none) -> RC0603FR-0722RL; Manufacturer (none) -> Yageo
- R412: MPN (none) -> RC0603FR-071K5L; Manufacturer (none) -> Yageo
- R413: MPN (none) -> RC0603FR-072R2L; Manufacturer (none) -> Yageo
- R414: MPN (none) -> RC0603FR-071ML; Manufacturer (none) -> Yageo
- R420, R421: MPN (none) -> RC0603FR-07100RL; Manufacturer (none) -> Yageo
- R432: MPN (none) -> RC0603FR-074K99L; Manufacturer (none) -> Yageo
- R433: MPN (none) -> RC0603FR-071KL; Manufacturer (none) -> Yageo
- R435: MPN (none) -> RC0603FR-072K2L; Manufacturer (none) -> Yageo

Commit message: get the main boards ready for routing
Parts:
- removed J421: Right 8-ohm BTL speaker; pin 1 +, pin 2 -, Connector_JST:JST_GH_SM02B-GHS-TB_1x02-1MP_P1.25mm_Horizontal, symbol Connector_Generic:Conn_01x02
- added J421: Right 8-ohm BTL speaker; pin 1 +, pin 2 -, Connector_JST:JST_GH_SM02B-GHS-TB_1x02-1MP_P1.25mm_Horizontal, symbol Conn_01x02_MP:Conn_01x02_MP
- J420: symbol Connector_Generic:Conn_01x02 -> Conn_01x02_MP:Conn_01x02_MP
Connections:
- net GND: now also J420.MP, J421.MP
- net SPK_R_N: now also J421.2 (Pin_2)
- net SPK_R_P: now also J421.1 (Pin_1)
- net AUDIO_USB_DM renamed AUDIO_USB_DN
- net CODEC_USB_DM renamed CODEC_USB_DN
- net RADIO_CODEC_USB_DM_HOST renamed RADIO_CODEC_USB_HOST_DN
- net RADIO_CODEC_USB_DP_HOST renamed RADIO_CODEC_USB_HOST_DP
- net SYSTEM_DAC_USB_DM renamed SYSTEM_DAC_USB_DN
Other:
- moved on the sheet: J420
Changed lines of the file:
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@@
   )
 )
-(label "SYSTEM_DAC_USB_DM"
+(label "SYSTEM_DAC_USB_DN"
   (at 317.5 144.78 0)
   (effects (font (size 1.27 1.27)) (justify left bottom))
@@
   (effects (font (size 1.27 1.27)) (justify left bottom))
 )
-(hierarchical_label "RADIO_CODEC_USB_DM_HOST"
+(hierarchical_label "RADIO_CODEC_USB_HOST_DN"
   (shape bidirectional)
   (at 317.5 149.86 0)
   (effects (font (size 1.27 1.27)) (justify left bottom))
 )
-(hierarchical_label "RADIO_CODEC_USB_DP_HOST"
+(hierarchical_label "RADIO_CODEC_USB_HOST_DP"
   (shape bidirectional)
   (at 317.5 152.4 0)
@@
   (effects (font (size 1.27 1.27)) (justify left bottom))
 )
-(hierarchical_label "AUDIO_USB_DM"
+(hierarchical_label "AUDIO_USB_DN"
   (shape bidirectional)
   (at 281.94 144.78 0)
@@
   (effects (font (size 1.27 1.27)) (justify left bottom))
 )
-(label "CODEC_USB_DM"
+(label "CODEC_USB_DN"
   (at 281.94 284.48 0)
   (effects (font (size 1.27 1.27)) (justify left bottom))
@@
   )
 )
-(label "SYSTEM_DAC_USB_DM"
+(label "SYSTEM_DAC_USB_DN"
   (at 20.32 229.87 0)
   (effects (font (size 1.27 1.27)) (justify left bottom))
 )
-(label "CODEC_USB_DM"
+(label "CODEC_USB_DN"
   (at 20.32 237.49 0)
   (effects (font (size 1.27 1.27)) (justify left bottom))
@@
 )
 (symbol
-  (lib_id "Connector_Generic:Conn_01x02")
+  (lib_id "Conn_01x02_MP:Conn_01x02_MP")
   (at 539.75 444.5 0)
   (unit 1)
@@
   (pin "1")
   (pin "2")
+  (pin "MP")
   (instances
     (project "ducktop2"
@@
   (effects (font (size 1.27 1.27)) (justify left bottom))
 )
-(symbol
-  (lib_id "Connector_Generic:Conn_01x02")
+(label "GND"
+  (at 544.83 445.77 0)
+  (effects (font (size 1.27 1.27)) (justify left bottom))
+)
+(symbol
+  (lib_id "Conn_01x02_MP:Conn_01x02_MP")
   (at 650.24 444.5 0)
   (unit 1)
@@
   (pin "1")
   (pin "2")
+  (pin "MP")
   (instances
     (project "ducktop2"
@@
   (effects (font (size 1.27 1.27)) (justify left bottom))
 )
+(label "GND"
+  (at 655.32 445.77 0)
+  (effects (font (size 1.27 1.27)) (justify left bottom))
+)
