File: radio_daughterboard/radio_daughterboard.kicad_pcb (KiCad board)
At the start: 4 copper layers, 120 x 40.5 mm, 126 parts, among them J1 DF40C 60-pin radio daughterbo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, J240 2m/VHF internal/PCB antenna f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, J241 2m/VHF rear external SMA/u.FL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, J250 70cm/UHF internal/PCB antenna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, J251 70cm/UHF rear external SMA/u.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, J42 GNSS passive antenna U.FL, J70 DRA818V 2m FM module, J71 DRA818U 70cm FM module, Q330 2N7002KT1G VHF PTT/suspend fa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, Q331 2N7002KT1G UHF PTT/suspend fa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, Q332 BSS84LT1G codec-loss force-mu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, U1 AP2112K-3.3 600mA daughterboa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, U240 PE42820B-X 2m/VHF 43dBm-CW RF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, U241 SN74LVC1G373DCKR VHF transmit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, U242 SN74LVC3G34DCUR VHF fail-safe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, U243 SN74LVC1T45 VHF TXD 4V-to-3V3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, U250 PE42820B-X 70cm/UHF 43dBm-CW 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, U251 SN74LVC1G373DCKR UHF transmit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, U252 SN74LVC3G34DCUR UHF fail-safe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, U253 SN74LVC1T45 UHF TXD 4V-to-3V3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, U260 SN74LVC2G04DCKR PTT request i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, U261 SN74LVC2G32DCUR dual-radio PT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, U330 PCM2902CDBR USB audio codec, U40 MAX-M10S GNSS, U41 SN74LVC3G34 GNSS input isolat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, U70 TPS54302 RADIO_DB_5V -> RADIO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, Y330 ABM8G-106-12.000MHZ-T 12MHz 1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

Commit message: Fix radio DB J1 layer (F.Cu->B.Cu) for mezzanine stack; add radio DB outline on mainboard Dwgs.User
Parts:
- J1: moved to B.Cu
