File: radio_daughterboard/radio_daughterboard.kicad_pcb (KiCad board)
At the start: 4 copper layers, 120 x 70 mm, 126 parts, among them J1 FH12-30S 30-pin radio daughte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, J240 2m/VHF internal/PCB antenna f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, J241 2m/VHF rear external SMA/u.FL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, J250 70cm/UHF internal/PCB antenna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, J251 70cm/UHF rear external SMA/u.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, J42 GNSS passive antenna U.FL, J70 DRA818V 2m FM module, J71 DRA818U 70cm FM module, Q330 2N7002KT1G VHF PTT/suspend fa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, Q331 2N7002KT1G UHF PTT/suspend fa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, Q332 BSS84LT1G codec-loss force-mu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, U1 AP2112K-3.3 600mA daughterboa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, U240 PE42820B-X 2m/VHF 43dBm-CW RF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, U241 SN74LVC1G373DCKR VHF transmit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, U242 SN74LVC3G34DCUR VHF fail-safe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, U243 SN74LVC1T45 VHF TXD 4V-to-3V3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, U250 PE42820B-X 70cm/UHF 43dBm-CW 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, U251 SN74LVC1G373DCKR UHF transmit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, U252 SN74LVC3G34DCUR UHF fail-safe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, U253 SN74LVC1T45 UHF TXD 4V-to-3V3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, U260 SN74LVC2G04DCKR PTT request i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, U261 SN74LVC2G32DCUR dual-radio PT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, U330 PCM2902CDBR USB audio codec, U40 MAX-M10S GNSS, U41 SN74LVC3G34 GNSS input isolat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, U70 TPS54302 RADIO_DB_5V -> RADIO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, Y330 ABM8G-106-12.000MHZ-T 12MHz 1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

Commit message: fix the center layout and more board issues
Parts:
- R221: value 100k 1% 4.0V FB hi -> 100k 0.02% 5ppm 4.0V FB hi
- R222: value 17.4k 1% 4.0V FB lo -> 17.4k 0.02% 5ppm 4.0V FB lo
- R227: value 47k 1% VHF antenna select default internal; PE42820 control divider low -> 47k 0.02% 5ppm VHF antenna select default internal; PE42820 control divider low
- R228: value 47k 1% UHF antenna select default internal; PE42820 control divider low -> 47k 0.02% 5ppm UHF antenna select default internal; PE42820 control divider low
- R242: value 10k 1% VHF PE42820 control divider top -> 10k 0.02% 5ppm VHF PE42820 control divider top
- R260: value 10k 1% UHF PE42820 control divider top -> 10k 0.02% 5ppm UHF PE42820 control divider top
Changed lines of the file:
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@@
 			(size 0.97 0.97)
 			(drill 0.46)
+			(property pad_prop_mechanical)
 			(layers "*.Cu")
 			(remove_unused_layers no)
@@
 			(size 0.97 0.97)
 			(drill 0.46)
+			(property pad_prop_mechanical)
 			(layers "*.Cu")
 			(remove_unused_layers no)
@@
 			(size 0.45 0.45)
 			(drill 0.2)
+			(property pad_prop_heatsink)
 			(layers "*.Cu")
 			(remove_unused_layers no)
@@
 			(size 0.45 0.45)
 			(drill 0.2)
+			(property pad_prop_heatsink)
 			(layers "*.Cu")
 			(remove_unused_layers no)
@@
 			(size 0.45 0.45)
 			(drill 0.2)
+			(property pad_prop_heatsink)
 			(layers "*.Cu")
 			(remove_unused_layers no)
@@
 			(size 0.45 0.45)
 			(drill 0.2)
+			(property pad_prop_heatsink)
 			(layers "*.Cu")
 			(remove_unused_layers no)
@@
 			(size 0.45 0.45)
 			(drill 0.2)
+			(property pad_prop_heatsink)
 			(layers "*.Cu")
 			(remove_unused_layers no)
@@
 			(at 0 0)
 			(size 2.8 2.8)
+			(property pad_prop_heatsink)
 			(layers "B.Cu")
 			(net "GND")
@@
 			(at 0 0)
 			(size 3.35 3.35)
+			(property pad_prop_heatsink)
 			(layers "F.Cu" "F.Mask")
 			(net "GND")
@@
 			(size 0.45 0.45)
 			(drill 0.2)
+			(property pad_prop_heatsink)
 			(layers "*.Cu")
 			(remove_unused_layers no)
@@
 			(size 0.45 0.45)
 			(drill 0.2)
+			(property pad_prop_heatsink)
 			(layers "*.Cu")
 			(remove_unused_layers no)
@@
 			(size 0.45 0.45)
 			(drill 0.2)
+			(property pad_prop_heatsink)
 			(layers "*.Cu")
 			(remove_unused_layers no)
@@
 			(size 0.45 0.45)
 			(drill 0.2)
+			(property pad_prop_heatsink)
 			(layers "*.Cu")
 			(remove_unused_layers no)
@@
 			(size 0.45 0.45)
 			(drill 0.2)
+			(property pad_prop_heatsink)
 			(layers "*.Cu")
 			(remove_unused_layers no)
@@
 			(size 0.45 0.45)
 			(drill 0.2)
+			(property pad_prop_heatsink)
 			(layers "*.Cu")
 			(remove_unused_layers no)
@@
 			(size 0.45 0.45)
 			(drill 0.2)
+			(property pad_prop_heatsink)
 			(layers "*.Cu")
 			(remove_unused_layers no)
@@
 			(size 0.45 0.45)
 			(drill 0.2)
+			(property pad_prop_heatsink)
 			(layers "*.Cu")
 			(remove_unused_layers no)
@@
 			(size 0.45 0.45)
 			(drill 0.2)
+			(property pad_prop_heatsink)
 			(layers "*.Cu")
 			(remove_unused_layers no)
@@
 			(at 0 0)
 			(size 2.8 2.8)
+			(property pad_prop_heatsink)
 			(layers "B.Cu")
 			(net "GND")
@@
 			(at 0 0)
 			(size 3.35 3.35)
+			(property pad_prop_heatsink)
 			(layers "F.Cu" "F.Mask")
 			(net "GND")
@@
 			(size 0.45 0.45)
 			(drill 0.2)
+			(property pad_prop_heatsink)
 			(layers "*.Cu")
 			(remove_unused_layers no)
@@
 			(size 0.45 0.45)
 			(drill 0.2)
+			(property pad_prop_heatsink)
 			(layers "*.Cu")
 			(remove_unused_layers no)
@@
 			(size 0.45 0.45)
 			(drill 0.2)
+			(property pad_prop_heatsink)
 			(layers "*.Cu")
 			(remove_unused_layers no)
@@
 			(size 0.45 0.45)
 			(drill 0.2)
+			(property pad_prop_heatsink)
 			(layers "*.Cu")
 			(remove_unused_layers no)
@@
 			)
 		)
-		(property "Value" "47k 1% VHF antenna select default internal; PE42820 control divider low"
+		(property "Value" "47k 0.02% 5ppm VHF antenna select default internal; PE42820 control divider low"
 			(at 0 1.43 0)
 			(layer "F.Fab")
@@
 			)
 		)
-		(property "Manufacturer" "Yageo"
+		(property "Manufacturer" "Vishay"
 			(at 0 0 0)
 			(unlocked yes)
@@
 			)
 		)
-		(property "MPN" "RC0603FR-0747KL"
+		(property "MPN" "TNPU060347K0HZEN00"
 			(at 0 0 0)
 			(unlocked yes)
@@
 			)
 		)
-		(property "Value" "10k 1% UHF PE42820 control divider top"
+		(property "Value" "10k 0.02% 5ppm UHF PE42820 control divider top"
 			(at 0 1.43 0)
 			(layer "F.Fab")
@@
 			)
 		)
-		(property "Manufacturer" "Yageo"
+		(property "Manufacturer" "Vishay"
 			(at 0 0 0)
 			(unlocked yes)
@@
 			)
 		)
-		(property "MPN" "RC0603FR-0710KL"
+		(property "MPN" "TNPU060310K0HZEN00"
 			(at 0 0 0)
 			(unlocked yes)
@@
 			(size 0.97 0.97)
 			(drill 0.46)
+			(property pad_prop_mechanical)
 			(layers "*.Cu")
 			(remove_unused_layers no)
@@
 			(size 0.97 0.97)
 			(drill 0.46)
+			(property pad_prop_mechanical)
 			(layers "*.Cu")
 			(remove_unused_layers no)
@@
 			)
 		)
-		(property "Value" "10k 1% VHF PE42820 control divider top"
+		(property "Value" "10k 0.02% 5ppm VHF PE42820 control divider top"
 			(at 0 1.43 0)
 			(layer "F.Fab")
@@
 			)
 		)
-		(property "Manufacturer" "Yageo"
+		(property "Manufacturer" "Vishay"
 			(at 0 0 0)
 			(unlocked yes)
@@
 			)
 		)
-		(property "MPN" "RC0603FR-0710KL"
+		(property "MPN" "TNPU060310K0HZEN00"
 			(at 0 0 0)
 			(unlocked yes)
@@
 			)
 		)
-		(property "Value" "17.4k 1% 4.0V FB lo"
+		(property "Value" "17.4k 0.02% 5ppm 4.0V FB lo"
 			(at 0 1.43 0)
 			(layer "F.Fab")
@@
 			)
 		)
-		(property "Manufacturer" "Yageo"
+		(property "Manufacturer" "Vishay"
 			(at 0 0 0)
 			(unlocked yes)
@@
 			)
 		)
-		(property "MPN" "RC0603FR-0717K4L"
+		(property "MPN" "TNPU060317K4HZEN00"
 			(at 0 0 0)
 			(unlocked yes)
@@
 			)
 		)
-		(property "Value" "100k 1% 4.0V FB hi"
+		(property "Value" "100k 0.02% 5ppm 4.0V FB hi"
 			(at 0 1.43 0)
 			(layer "F.Fab")
@@
 			)
 		)
-		(property "Manufacturer" "Yageo"
+		(property "Manufacturer" "Vishay"
 			(at 0 0 0)
 			(unlocked yes)
@@
 			)
 		)
-		(property "MPN" "RC0603FR-07100KL"
+		(property "MPN" "TNPU0603100KHZEN00"
 			(at 0 0 0)
 			(unlocked yes)
@@
 			)
 		)
-		(property "Value" "47k 1% UHF antenna select default internal; PE42820 control divider low"
+		(property "Value" "47k 0.02% 5ppm UHF antenna select default internal; PE42820 control divider low"
 			(at 0 1.43 0)
 			(layer "F.Fab")
@@
 			)
 		)
-		(property "Manufacturer" "Yageo"
+		(property "Manufacturer" "Vishay"
 			(at 0 0 0)
 			(unlocked yes)
@@
 			)
 		)
-		(property "MPN" "RC0603FR-0747KL"
+		(property "MPN" "TNPU060347K0HZEN00"
 			(at 0 0 0)
 			(unlocked yes)
