File: radio_daughterboard/02_radios.kicad_sch (KiCad schematic)
At the start: 72 parts, among them J240 2m/VHF internal/PCB antenna f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, J241 2m/VHF rear external SMA/u.FL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, J250 70cm/UHF internal/PCB antenna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, J251 70cm/UHF rear external SMA/u.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, J70 DRA818V 2m FM module, J71 DRA818U 70cm FM module, J72 DNP radio audio/codec harness, U240 PE42820B-X 2m/VHF 43dBm-CW RF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, U241 SN74LVC1G373DCKR VHF transmit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, U242 SN74LVC3G34DCUR VHF fail-safe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, U243 SN74LVC1T45 VHF TXD 4V-to-3V3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, U250 PE42820B-X 70cm/UHF 43dBm-CW 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, U251 SN74LVC1G373DCKR UHF transmit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, U252 SN74LVC3G34DCUR UHF fail-safe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, U253 SN74LVC1T45 UHF TXD 4V-to-3V3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, U260 SN74LVC2G04DCKR PTT request i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, U261 SN74LVC2G32DCUR dual-radio PT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, U70 TPS54302 RADIO_DB_5V -> RADIO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

Commit message: Apply BOM to radio + keyboard daughterboards, add Cherry MX switch 3D models
radio_daughterboard/:
- 74 MPNs assigned (33 resistors, 41 caps) across 4 schematic sheets
- 129 BOM gaps reduced to 7 (mounting holes H1-H4, DNP connectors J44/J72/J330)

12_keyboard_daughterboard/:
- 134 MPNs assigned: 65× 1N4148W-7-F diodes, 65× Cherry MX4A-L1NA switches,
  2× caps, 2× connectors
- BOM gaps eliminated: 134 → 0

3D models:
- Added Cherry_MX_ULP_SMD.step to ducktop2.3dshapes/ (65 Cherry MX switch
  footprints on keyboard daughterboard now have 3D models)
- Created gen/add_pcb_3d_models.py script for future 3D model assignments
- 57 footprints remain without models (MountingHole, TestPoint, Tag-Connect,
  and custom ducktop2 components — need manufacturer STEP files)

gen/:
- apply_bom_radio_daughterboard.py: radio daughterboard BOM catalog
- apply_bom_keyboard_daughterboard.py: keyboard daughterboard BOM catalog
- add_pcb_3d_models.py: automated 3D model path inserter
Parts:
- C221, C240, C246, C247, C248, C250, C256, C257, C258, C260, C261: MPN (none) -> GRM188R71H104KA93D; Manufacturer (none) -> Murata
- C224: MPN (none) -> GRM1885C1H560JA01D; Manufacturer (none) -> Murata
- C226, C227, C243, C253: MPN (none) -> GRM188R71H103KA01D; Manufacturer (none) -> Murata
- C244, C254: MPN (none) -> GRM1885C1H101JA01D; Manufacturer (none) -> Murata
- C245, C255: MPN (none) -> GRM1885C1H0R2CA01D; Manufacturer (none) -> Murata
- R220, R221, R225, R226, R230, R232: MPN (none) -> RC0603FR-07100KL; Manufacturer (none) -> Yageo
- R222: MPN (none) -> RC0603FR-0717K4L; Manufacturer (none) -> Yageo
- R227, R228: MPN (none) -> RC0603FR-0747KL; Manufacturer (none) -> Yageo
- R229, R231: MPN (none) -> RC0603FR-070RL; Manufacturer (none) -> Yageo
- R233, R234: MPN (none) -> RC0603FR-071KL; Manufacturer (none) -> Yageo
- R242, R260: MPN (none) -> RC0603FR-0710KL; Manufacturer (none) -> Yageo
- R243, R261: MPN (none) -> RC0603FR-07100RL; Manufacturer (none) -> Yageo

Commit message: Complete EC DFU port (J73) + DB power rework; verify schematic and board
- Add rear USB-C EC firmware programming port J73 (UFP/DFU) on Internal
  Services sheet: USBLC6-2P6 ESD (U63), 5.1k CC Rd resistors (R205/R211),
  22R series on D+/D- (R203/R204), mux-select hookup so BOOT0 high forces
  the USB mux to the DFU port
- Rename port ref J70->J73 after ham-radio collision; sync all net names
  (J73_CC1/J73_CC2)
- DB power rework: S5 gating + 3V3_STBY split, dual DCDC paths, GND
  returns on the standby rails; regenerate all sheets and re-verify
- sync_main_pcb_from_netlist: anchor placement for the 9 new footprints,
  scoped ECO support
- Board: rebuild main PCB with J73 footprint block (lib-sourced, net
  injection from netlist name attribute), sync pad nets for the 5 stale
  refs, remove duplicate R205/R211 copies
- Verified: check_schematic self-check OK (0 errors), radio DB contracts
  OK, ERC 0 errors, board DRC 0 electrical violations, board-vs-schematic
  net parity 0 conflicts, no duplicate refs
Parts:
- C221, C240, C246, C247, C248, C250, C256, C257, C258, C260, C261: MPN GRM188R71H104KA93D -> (none); Manufacturer Murata -> (none)
- C224: MPN GRM1885C1H560JA01D -> (none); Manufacturer Murata -> (none)
- C226, C227, C243, C253: MPN GRM188R71H103KA01D -> (none); Manufacturer Murata -> (none)
- C244, C254: MPN GRM1885C1H101JA01D -> (none); Manufacturer Murata -> (none)
- C245, C255: MPN GRM1885C1H0R2CA01D -> (none); Manufacturer Murata -> (none)
- R220, R221, R225, R226, R230, R232: MPN RC0603FR-07100KL -> (none); Manufacturer Yageo -> (none)
- R222: MPN RC0603FR-0717K4L -> (none); Manufacturer Yageo -> (none)
- R227, R228: MPN RC0603FR-0747KL -> (none); Manufacturer Yageo -> (none)
- R229, R231: MPN RC0603FR-070RL -> (none); Manufacturer Yageo -> (none)
- R233, R234: MPN RC0603FR-071KL -> (none); Manufacturer Yageo -> (none)
- R242, R260: MPN RC0603FR-0710KL -> (none); Manufacturer Yageo -> (none)
- R243, R261: MPN RC0603FR-07100RL -> (none); Manufacturer Yageo -> (none)
