File: radio_daughterboard/02_radios.kicad_sch (KiCad schematic)
At the start: 72 parts, among them J240 2m/VHF internal/PCB antenna f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, J241 2m/VHF rear external SMA/u.FL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, J250 70cm/UHF internal/PCB antenna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, J251 70cm/UHF rear external SMA/u.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, J70 DRA818V 2m FM module, J71 DRA818U 70cm FM module, J72 DNP radio audio/codec harness, U240 PE42820B-X 2m/VHF 43dBm-CW RF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, U241 SN74LVC1G373DCKR VHF transmit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, U242 SN74LVC3G34DCUR VHF fail-safe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, U243 SN74LVC1T45 VHF TXD 4V-to-3V3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, U250 PE42820B-X 70cm/UHF 43dBm-CW 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, U251 SN74LVC1G373DCKR UHF transmit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, U252 SN74LVC3G34DCUR UHF fail-safe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, U253 SN74LVC1T45 UHF TXD 4V-to-3V3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, U260 SN74LVC2G04DCKR PTT request i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, U261 SN74LVC2G32DCUR dual-radio PT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, U70 TPS54302 RADIO_DB_5V -> RADIO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

Commit message: fix the center layout and more board issues
Parts:
- R221: value 100k 1% 4.0V FB hi -> 100k 0.02% 5ppm 4.0V FB hi; MPN RC0603FR-07100KL -> TNPU0603100KHZEN00; Manufacturer Yageo -> Vishay
- R222: value 17.4k 1% 4.0V FB lo -> 17.4k 0.02% 5ppm 4.0V FB lo; MPN RC0603FR-0717K4L -> TNPU060317K4HZEN00; Manufacturer Yageo -> Vishay
- R227: value 47k 1% VHF antenna select default internal; PE42820 control divider low -> 47k 0.02% 5ppm VHF antenna select default internal; PE42820 control divider low; MPN RC0603FR-0747KL -> TNPU060347K0HZEN00; Manufacturer Yageo -> Vishay
- R228: value 47k 1% UHF antenna select default internal; PE42820 control divider low -> 47k 0.02% 5ppm UHF antenna select default internal; PE42820 control divider low; MPN RC0603FR-0747KL -> TNPU060347K0HZEN00; Manufacturer Yageo -> Vishay
- R242: value 10k 1% VHF PE42820 control divider top -> 10k 0.02% 5ppm VHF PE42820 control divider top; MPN RC0603FR-0710KL -> TNPU060310K0HZEN00; Manufacturer Yageo -> Vishay
- R260: value 10k 1% UHF PE42820 control divider top -> 10k 0.02% 5ppm UHF PE42820 control divider top; MPN RC0603FR-0710KL -> TNPU060310K0HZEN00; Manufacturer Yageo -> Vishay
Changed lines of the file:
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@@
   (dnp no)
   (property "Reference" "R221" (at 20.32 124.46 0) (effects (font (size 1.27 1.27))))
-  (property "Value" "100k 1% 4.0V FB hi" (at 20.32 129.54 0) (effects (font (size 1.27 1.27))))
+  (property "Value" "100k 0.02% 5ppm 4.0V FB hi" (at 20.32 129.54 0) (effects (font (size 1.27 1.27))))
   (property "Footprint" "Resistor_SMD:R_0603_1608Metric" (at 20.32 127 0) (effects (font (size 1.27 1.27)) (hide yes)))
   (property "Datasheet" "" (at 20.32 127 0) (effects (font (size 1.27 1.27)) (hide yes)))
-  (property "Manufacturer" "Yageo" (at 20.32 127 0) (effects (font (size 1.27 1.27)) (hide yes)))
-  (property "MPN" "RC0603FR-07100KL" (at 20.32 127 0) (effects (font (size 1.27 1.27)) (hide yes)))
+  (property "Manufacturer" "Vishay" (at 20.32 127 0) (effects (font (size 1.27 1.27)) (hide yes)))
+  (property "MPN" "TNPU0603100KHZEN00" (at 20.32 127 0) (effects (font (size 1.27 1.27)) (hide yes)))
   (pin "1")
   (pin "2")
@@
   (dnp no)
   (property "Reference" "R222" (at 20.32 137.16 0) (effects (font (size 1.27 1.27))))
-  (property "Value" "17.4k 1% 4.0V FB lo" (at 20.32 142.24 0) (effects (font (size 1.27 1.27))))
+  (property "Value" "17.4k 0.02% 5ppm 4.0V FB lo" (at 20.32 142.24 0) (effects (font (size 1.27 1.27))))
   (property "Footprint" "Resistor_SMD:R_0603_1608Metric" (at 20.32 139.7 0) (effects (font (size 1.27 1.27)) (hide yes)))
   (property "Datasheet" "" (at 20.32 139.7 0) (effects (font (size 1.27 1.27)) (hide yes)))
-  (property "Manufacturer" "Yageo" (at 20.32 139.7 0) (effects (font (size 1.27 1.27)) (hide yes)))
-  (property "MPN" "RC0603FR-0717K4L" (at 20.32 139.7 0) (effects (font (size 1.27 1.27)) (hide yes)))
+  (property "Manufacturer" "Vishay" (at 20.32 139.7 0) (effects (font (size 1.27 1.27)) (hide yes)))
+  (property "MPN" "TNPU060317K4HZEN00" (at 20.32 139.7 0) (effects (font (size 1.27 1.27)) (hide yes)))
   (pin "1")
   (pin "2")
@@
   (dnp no)
   (property "Reference" "R242" (at 549.91 193.04 0) (effects (font (size 1.27 1.27))))
-  (property "Value" "10k 1% VHF PE42820 control divider top" (at 549.91 198.12 0) (effects (font (size 1.27 1.27))))
+  (property "Value" "10k 0.02% 5ppm VHF PE42820 control divider top" (at 549.91 198.12 0) (effects (font (size 1.27 1.27))))
   (property "Footprint" "Resistor_SMD:R_0603_1608Metric" (at 549.91 195.58 0) (effects (font (size 1.27 1.27)) (hide yes)))
   (property "Datasheet" "" (at 549.91 195.58 0) (effects (font (size 1.27 1.27)) (hide yes)))
-  (property "Manufacturer" "Yageo" (at 549.91 195.58 0) (effects (font (size 1.27 1.27)) (hide yes)))
-  (property "MPN" "RC0603FR-0710KL" (at 549.91 195.58 0) (effects (font (size 1.27 1.27)) (hide yes)))
+  (property "Manufacturer" "Vishay" (at 549.91 195.58 0) (effects (font (size 1.27 1.27)) (hide yes)))
+  (property "MPN" "TNPU060310K0HZEN00" (at 549.91 195.58 0) (effects (font (size 1.27 1.27)) (hide yes)))
   (pin "1")
   (pin "2")
@@
   (dnp no)
   (property "Reference" "R260" (at 549.91 205.74 0) (effects (font (size 1.27 1.27))))
-  (property "Value" "10k 1% UHF PE42820 control divider top" (at 549.91 210.82 0) (effects (font (size 1.27 1.27))))
+  (property "Value" "10k 0.02% 5ppm UHF PE42820 control divider top" (at 549.91 210.82 0) (effects (font (size 1.27 1.27))))
   (property "Footprint" "Resistor_SMD:R_0603_1608Metric" (at 549.91 208.28 0) (effects (font (size 1.27 1.27)) (hide yes)))
   (property "Datasheet" "" (at 549.91 208.28 0) (effects (font (size 1.27 1.27)) (hide yes)))
-  (property "Manufacturer" "Yageo" (at 549.91 208.28 0) (effects (font (size 1.27 1.27)) (hide yes)))
-  (property "MPN" "RC0603FR-0710KL" (at 549.91 208.28 0) (effects (font (size 1.27 1.27)) (hide yes)))
+  (property "Manufacturer" "Vishay" (at 549.91 208.28 0) (effects (font (size 1.27 1.27)) (hide yes)))
+  (property "MPN" "TNPU060310K0HZEN00" (at 549.91 208.28 0) (effects (font (size 1.27 1.27)) (hide yes)))
   (pin "1")
   (pin "2")
@@
   (dnp no)
   (property "Reference" "R227" (at 250.19 269.24 0) (effects (font (size 1.27 1.27))))
-  (property "Value" "47k 1% VHF antenna select default internal; PE42820 control divider low" (at 250.19 274.32 0) (effects (font (size 1.27 1.27))))
+  (property "Value" "47k 0.02% 5ppm VHF antenna select default internal; PE42820 control divider low" (at 250.19 274.32 0) (effects (font (size 1.27 1.27))))
   (property "Footprint" "Resistor_SMD:R_0603_1608Metric" (at 250.19 271.78 0) (effects (font (size 1.27 1.27)) (hide yes)))
   (property "Datasheet" "" (at 250.19 271.78 0) (effects (font (size 1.27 1.27)) (hide yes)))
-  (property "Manufacturer" "Yageo" (at 250.19 271.78 0) (effects (font (size 1.27 1.27)) (hide yes)))
-  (property "MPN" "RC0603FR-0747KL" (at 250.19 271.78 0) (effects (font (size 1.27 1.27)) (hide yes)))
+  (property "Manufacturer" "Vishay" (at 250.19 271.78 0) (effects (font (size 1.27 1.27)) (hide yes)))
+  (property "MPN" "TNPU060347K0HZEN00" (at 250.19 271.78 0) (effects (font (size 1.27 1.27)) (hide yes)))
   (pin "1")
   (pin "2")
@@
   (dnp no)
   (property "Reference" "R228" (at 250.19 281.94 0) (effects (font (size 1.27 1.27))))
-  (property "Value" "47k 1% UHF antenna select default internal; PE42820 control divider low" (at 250.19 287.02 0) (effects (font (size 1.27 1.27))))
+  (property "Value" "47k 0.02% 5ppm UHF antenna select default internal; PE42820 control divider low" (at 250.19 287.02 0) (effects (font (size 1.27 1.27))))
   (property "Footprint" "Resistor_SMD:R_0603_1608Metric" (at 250.19 284.48 0) (effects (font (size 1.27 1.27)) (hide yes)))
   (property "Datasheet" "" (at 250.19 284.48 0) (effects (font (size 1.27 1.27)) (hide yes)))
-  (property "Manufacturer" "Yageo" (at 250.19 284.48 0) (effects (font (size 1.27 1.27)) (hide yes)))
-  (property "MPN" "RC0603FR-0747KL" (at 250.19 284.48 0) (effects (font (size 1.27 1.27)) (hide yes)))
-  (pin "1")
-  (pin "2")
+  (property "Manufacturer" "Vishay" (at 250.19 284.48 0) (effects (font (size 1.27 1.27)) (hide yes)))
+  (property "MPN" "TNPU060347K0HZEN00" (at 250.19 284.48 0) (effects (font (size 1.27 1.27)) (hide yes)))
+  (pin "1")
+  (pin "2")
