File: radio_daughterboard/radio_daughterboard.kicad_sch (KiCad schematic)
At the start: 0 parts

Commit message: get the main boards ready for routing
Other:
- sheet Core & Mainboard Connector ports: added RADIO_CODEC_USB_DN; removed RADIO_CODEC_USB_DM
- sheet USB Radio Audio ports: added RADIO_CODEC_USB_DN; removed RADIO_CODEC_USB_DM
Changed lines of the file:
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@@
     (effects (font (size 1.27 1.27)) (justify left))
   )
-  (pin "RADIO_CODEC_USB_DM" bidirectional
+  (pin "RADIO_CODEC_USB_DN" bidirectional
     (at 149.86 59.69 0)
     (effects (font (size 1.27 1.27)) (justify left))
@@
     (effects (font (size 1.27 1.27)) (justify left))
   )
-  (pin "RADIO_CODEC_USB_DM" bidirectional
+  (pin "RADIO_CODEC_USB_DN" bidirectional
     (at 599.44 49.53 0)
     (effects (font (size 1.27 1.27)) (justify left))
@@
   (effects (font (size 1.27 1.27)) (justify left bottom))
 )
-(label "RADIO_CODEC_USB_DM"
+(label "RADIO_CODEC_USB_DN"
   (at 149.86 59.69 0)
   (effects (font (size 1.27 1.27)) (justify left bottom))
 )
-(label "RADIO_CODEC_USB_DM"
+(label "RADIO_CODEC_USB_DN"
   (at 599.44 49.53 0)
   (effects (font (size 1.27 1.27)) (justify left bottom))
