File: radio_daughterboard/03_gnss.kicad_sch (KiCad schematic)
At the start: 10 parts, among them J42 GNSS passive antenna U.FL, J44 DNP MAX-M10S debug/program, U40 MAX-M10S GNSS, U41 SN74LVC3G34 GNSS input isolat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

Commit message: Complete EC DFU port (J73) + DB power rework; verify schematic and board
- Add rear USB-C EC firmware programming port J73 (UFP/DFU) on Internal
  Services sheet: USBLC6-2P6 ESD (U63), 5.1k CC Rd resistors (R205/R211),
  22R series on D+/D- (R203/R204), mux-select hookup so BOOT0 high forces
  the USB mux to the DFU port
- Rename port ref J70->J73 after ham-radio collision; sync all net names
  (J73_CC1/J73_CC2)
- DB power rework: S5 gating + 3V3_STBY split, dual DCDC paths, GND
  returns on the standby rails; regenerate all sheets and re-verify
- sync_main_pcb_from_netlist: anchor placement for the 9 new footprints,
  scoped ECO support
- Board: rebuild main PCB with J73 footprint block (lib-sourced, net
  injection from netlist name attribute), sync pad nets for the 5 stale
  refs, remove duplicate R205/R211 copies
- Verified: check_schematic self-check OK (0 errors), radio DB contracts
  OK, ERC 0 errors, board DRC 0 electrical violations, board-vs-schematic
  net parity 0 conflicts, no duplicate refs
Parts:
- C40, C42: MPN GRM188R71H104KA93D -> (none); Manufacturer Murata -> (none)
- C41: MPN GRM31CR71E106KA12L -> (none); Manufacturer Murata -> (none)
- R40: MPN RC0603FR-07100KL -> (none); Manufacturer Yageo -> (none)
- R41, R42: MPN RC0603FR-07100RL -> (none); Manufacturer Yageo -> (none)
Changed lines of the file:
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@@
   (property "Footprint" "Capacitor_SMD:C_0603_1608Metric" (at 199.39 106.68 0) (effects (font (size 1.27 1.27)) (hide yes)))
   (property "Datasheet" "" (at 199.39 106.68 0) (effects (font (size 1.27 1.27)) (hide yes)))
-  (property "Manufacturer" "Murata" (at 199.39 106.68 0) (effects (font (size 1.27 1.27)) (hide yes)))
-  (property "MPN" "GRM188R71H104KA93D" (at 199.39 106.68 0) (effects (font (size 1.27 1.27)) (hide yes)))
   (pin "1")
   (pin "2")
@@
   (property "Footprint" "Resistor_SMD:R_0603_1608Metric" (at 20.32 127 0) (effects (font (size 1.27 1.27)) (hide yes)))
   (property "Datasheet" "" (at 20.32 127 0) (effects (font (size 1.27 1.27)) (hide yes)))
-  (property "Manufacturer" "Yageo" (at 20.32 127 0) (effects (font (size 1.27 1.27)) (hide yes)))
-  (property "MPN" "RC0603FR-07100KL" (at 20.32 127 0) (effects (font (size 1.27 1.27)) (hide yes)))
   (pin "1")
   (pin "2")
@@
   (property "Footprint" "Resistor_SMD:R_0603_1608Metric" (at 20.32 152.4 0) (effects (font (size 1.27 1.27)) (hide yes)))
   (property "Datasheet" "" (at 20.32 152.4 0) (effects (font (size 1.27 1.27)) (hide yes)))
-  (property "Manufacturer" "Yageo" (at 20.32 152.4 0) (effects (font (size 1.27 1.27)) (hide yes)))
-  (property "MPN" "RC0603FR-07100RL" (at 20.32 152.4 0) (effects (font (size 1.27 1.27)) (hide yes)))
   (pin "1")
   (pin "2")
@@
   (property "Footprint" "Resistor_SMD:R_0603_1608Metric" (at 20.32 165.1 0) (effects (font (size 1.27 1.27)) (hide yes)))
   (property "Datasheet" "" (at 20.32 165.1 0) (effects (font (size 1.27 1.27)) (hide yes)))
-  (property "Manufacturer" "Yageo" (at 20.32 165.1 0) (effects (font (size 1.27 1.27)) (hide yes)))
-  (property "MPN" "RC0603FR-07100RL" (at 20.32 165.1 0) (effects (font (size 1.27 1.27)) (hide yes)))
   (pin "1")
   (pin "2")
@@
   (property "Footprint" "Capacitor_SMD:C_1206_3216Metric" (at 20.32 190.5 0) (effects (font (size 1.27 1.27)) (hide yes)))
   (property "Datasheet" "" (at 20.32 190.5 0) (effects (font (size 1.27 1.27)) (hide yes)))
-  (property "Manufacturer" "Murata" (at 20.32 190.5 0) (effects (font (size 1.27 1.27)) (hide yes)))
-  (property "MPN" "GRM31CR71E106KA12L" (at 20.32 190.5 0) (effects (font (size 1.27 1.27)) (hide yes)))
   (pin "1")
   (pin "2")
@@
   (property "Footprint" "Capacitor_SMD:C_0603_1608Metric" (at 20.32 203.2 0) (effects (font (size 1.27 1.27)) (hide yes)))
   (property "Datasheet" "" (at 20.32 203.2 0) (effects (font (size 1.27 1.27)) (hide yes)))
-  (property "Manufacturer" "Murata" (at 20.32 203.2 0) (effects (font (size 1.27 1.27)) (hide yes)))
-  (property "MPN" "GRM188R71H104KA93D" (at 20.32 203.2 0) (effects (font (size 1.27 1.27)) (hide yes)))
   (pin "1")
   (pin "2")

Commit message: fix audit issues and move some connectors
Parts:
- C40, C42: MPN (none) -> GRM188R71H104KA93D; Manufacturer (none) -> Murata
- C41: MPN (none) -> GRM31CR71E106KA12L; Manufacturer (none) -> Murata
- R40: MPN (none) -> RC0603FR-07100KL; Manufacturer (none) -> Yageo
- R41, R42: MPN (none) -> RC0603FR-07100RL; Manufacturer (none) -> Yageo
Changed lines of the file:
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@@
   (property "Footprint" "Capacitor_SMD:C_0603_1608Metric" (at 199.39 106.68 0) (effects (font (size 1.27 1.27)) (hide yes)))
   (property "Datasheet" "" (at 199.39 106.68 0) (effects (font (size 1.27 1.27)) (hide yes)))
+  (property "Manufacturer" "Murata" (at 199.39 106.68 0) (effects (font (size 1.27 1.27)) (hide yes)))
+  (property "MPN" "GRM188R71H104KA93D" (at 199.39 106.68 0) (effects (font (size 1.27 1.27)) (hide yes)))
   (pin "1")
   (pin "2")
@@
   (property "Footprint" "Resistor_SMD:R_0603_1608Metric" (at 20.32 127 0) (effects (font (size 1.27 1.27)) (hide yes)))
   (property "Datasheet" "" (at 20.32 127 0) (effects (font (size 1.27 1.27)) (hide yes)))
+  (property "Manufacturer" "Yageo" (at 20.32 127 0) (effects (font (size 1.27 1.27)) (hide yes)))
+  (property "MPN" "RC0603FR-07100KL" (at 20.32 127 0) (effects (font (size 1.27 1.27)) (hide yes)))
   (pin "1")
   (pin "2")
@@
   (property "Footprint" "Resistor_SMD:R_0603_1608Metric" (at 20.32 152.4 0) (effects (font (size 1.27 1.27)) (hide yes)))
   (property "Datasheet" "" (at 20.32 152.4 0) (effects (font (size 1.27 1.27)) (hide yes)))
+  (property "Manufacturer" "Yageo" (at 20.32 152.4 0) (effects (font (size 1.27 1.27)) (hide yes)))
+  (property "MPN" "RC0603FR-07100RL" (at 20.32 152.4 0) (effects (font (size 1.27 1.27)) (hide yes)))
   (pin "1")
   (pin "2")
@@
   (property "Footprint" "Resistor_SMD:R_0603_1608Metric" (at 20.32 165.1 0) (effects (font (size 1.27 1.27)) (hide yes)))
   (property "Datasheet" "" (at 20.32 165.1 0) (effects (font (size 1.27 1.27)) (hide yes)))
+  (property "Manufacturer" "Yageo" (at 20.32 165.1 0) (effects (font (size 1.27 1.27)) (hide yes)))
+  (property "MPN" "RC0603FR-07100RL" (at 20.32 165.1 0) (effects (font (size 1.27 1.27)) (hide yes)))
   (pin "1")
   (pin "2")
@@
   (property "Footprint" "Capacitor_SMD:C_1206_3216Metric" (at 20.32 190.5 0) (effects (font (size 1.27 1.27)) (hide yes)))
   (property "Datasheet" "" (at 20.32 190.5 0) (effects (font (size 1.27 1.27)) (hide yes)))
+  (property "Manufacturer" "Murata" (at 20.32 190.5 0) (effects (font (size 1.27 1.27)) (hide yes)))
+  (property "MPN" "GRM31CR71E106KA12L" (at 20.32 190.5 0) (effects (font (size 1.27 1.27)) (hide yes)))
   (pin "1")
   (pin "2")
@@
   (property "Footprint" "Capacitor_SMD:C_0603_1608Metric" (at 20.32 203.2 0) (effects (font (size 1.27 1.27)) (hide yes)))
   (property "Datasheet" "" (at 20.32 203.2 0) (effects (font (size 1.27 1.27)) (hide yes)))
+  (property "Manufacturer" "Murata" (at 20.32 203.2 0) (effects (font (size 1.27 1.27)) (hide yes)))
+  (property "MPN" "GRM188R71H104KA93D" (at 20.32 203.2 0) (effects (font (size 1.27 1.27)) (hide yes)))
   (pin "1")
   (pin "2")
