File: radio_daughterboard/04_codec.kicad_sch (KiCad schematic)
At the start: 36 parts, among them J330 DNP radio audio codec probe, Q330 2N7002KT1G VHF PTT/suspend fa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, Q331 2N7002KT1G UHF PTT/suspend fa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, Q332 BSS84LT1G codec-loss force-mu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, U330 PCM2902CDBR USB audio codec, Y330 ABM8G-106-12.000MHZ-T 12MHz 1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

Commit message: fix audit issues and move some connectors
Parts:
- C330, C332, C333, C334, C335, C340, C341, C342, C343: MPN (none) -> GRM21BR71A105KA01L; Manufacturer (none) -> Murata
- C331, C337: MPN (none) -> GRM31CR71E106KA12L; Manufacturer (none) -> Murata
- C338, C339: MPN (none) -> GRM1885C1H180JA01D; Manufacturer (none) -> Murata
- R330, R331: MPN (none) -> RC0603FR-0722RL; Manufacturer (none) -> Yageo
- R334, R335: MPN (none) -> RC0603FR-0782KL; Manufacturer (none) -> Yageo
- R336, R341: MPN (none) -> RC0603FR-071KL; Manufacturer (none) -> Yageo
- R337: MPN (none) -> RC0603FR-072R2L; Manufacturer (none) -> Yageo
- R338: MPN (none) -> RC0603FR-071K5L; Manufacturer (none) -> Yageo
- R340: MPN (none) -> RC0603FR-071ML; Manufacturer (none) -> Yageo
- R342, R343, R344, R345: MPN (none) -> RC0603FR-07100KL; Manufacturer (none) -> Yageo
