File: left_io/left_pd.kicad_sch (KiCad schematic)
At the start: 101 parts, among them J190 AUX/SOLAR protected screw ter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, J21 USB-C dual-role data/PD port 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, Q15 SiSS4409DN 40V reverse-blocki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, Q16 SiSS4409DN 40V reverse-blocki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, Q17 SiSS4409DN 40V reverse-blocki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, Q18 SiSS4409DN 40V reverse-blocki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, Q2001 2N7002K DFP USB2 enable inver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, U14 LTC4418IUF#PBF dual-input PD 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, U2000 TUSB1142 USB 3.2 Gen 2 orient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, U2001 TPD4S201 CC and USB2 short-to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, U2002 CAT24C256 32KB private TPS257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, U2003 TS3USB30E DFP-qualified USB2 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, U2004 SN74LVC2G07 partial-power-dow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, U2005 TVS2200 22V USB VBUS surge cl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, U2006 SN74LVC1G08 DFP and attached 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, U41 TPS25751AD USB-PD DRP control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, U720 TPS26630RGER PD1 default-off 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

Commit message: Phase 5: second-opinion audit remediation + rebuilt, verified board pipeline
Second-opinion AI audit found A-tier defects; remediation applied and the
board pipeline rebuilt on a known-good base with the fixes it needed:

- electrical: LTC4418IUF symbol pinout corrected (both selectors were
  dead as drawn); center charge cascade (U15 <- U15B, PD1 > PD2 > AUX);
  pack negative never crosses FPC-3, 15-pin FG_VSS return; power-budgeted
  FPC pin maps (0.4 A/pin derate); J12/DS4 completed; AUX source fuse
- FH41-68S footprint: 13 datasheet-correct SH pads + SH pin in symbol
- connector geometry settled against the Hirose FH12 2D drawing: FFC
  enters opposite the solder pins (mouth = local +Y); reversed side-B
  maps are correct for the 180-deg-mounted pairs; rotations set so mouths
  face across every seam
- pipeline (generate_split_boards.py): per-pin pad-net resync from the
  netlists (kills shadow nets for good), netlist-exact name
  normalization, netlist-only part injection (cascade, probe headers),
  zone refill after outline swap, read-before-write race fixed, orphan
  parts dropped loudly, non-zero exit on unresolved overlaps
- monolith board relocated to old/monolith_ducktop2.kicad_pcb (placement
  oracle for the center cut only)

verified end state: 4 boards 0 shorts / 0 clearance / 0 drill, 0 boundary
crossings, 6/6 connectors contract-exact with mouths facing, 0 shadow
nets, gates PASS x4, ERC 0 x4. routing next (499 nets/board).
Parts:
- removed C2144, C2145: 100n 50V selector local, Capacitor_SMD:C_0603_1608Metric, symbol Device:C
- removed Q18: SiSS4409DN 40V reverse-blocking PMOS, Package_SO:Vishay_PowerPAK_1212-8_Single, symbol Q_PMOS_1G_234S_5D:Q_PMOS_1G_234S_5D
- removed R2140, R2143: 1.00M 0.1% 15V UV top, Resistor_SMD:R_0603_1608Metric, symbol Device:R
- removed R2144: 19.6k 0.1% 15V window middle, Resistor_SMD:R_0603_1608Metric, symbol Device:R
- removed R2145: 63.4k 0.1% 15V OV bottom, Resistor_SMD:R_0603_1608Metric, symbol Device:R
- removed R2147: 10k PD2 VALID pull-up, Resistor_SMD:R_0603_1608Metric, symbol Device:R
- added C2140: 100n selector INTVCC, Capacitor_SMD:C_0603_1608Metric, symbol Device:C
- added F195: 3A MINI AUX source fuse: Littelfuse 0297003.WXNV, Fuse:Fuseholder_Blade_Mini_Keystone_3568, symbol Device:Fuse
- added H11, H12, H16: M2.5 isolated mainboard mounting hole, MountingHole:MountingHole_2.7mm_M2.5, symbol Mechanical:MountingHole
- H10: renamed from C2140; value 100n selector INTVCC -> M2.5 isolated mainboard mounting hole; footprint Capacitor_SMD:C_0603_1608Metric -> MountingHole:MountingHole_2.7mm_M2.5; symbol Device:C -> Mechanical:MountingHole; Hardware_Spec (none) -> 2.7mm isolated NPTH for M2.5 chassis screw; MPN GRM188R71H104KA93D -> (none); Manufacturer Murata -> (none); now left out of the parts list
- R2140: renamed from Q17; value SiSS4409DN 40V reverse-blocking PMOS -> 1.00M 0.1% 15V UV top; footprint Package_SO:Vishay_PowerPAK_1212-8_Single -> Resistor_SMD:R_0603_1608Metric; symbol Q_PMOS_1G_234S_5D:Q_PMOS_1G_234S_5D -> Device:R; MPN SiSS4409DN-T1-GE3 -> RT0603BRD071ML; Manufacturer Vishay -> Yageo
- U14: value LTC4418IUF#PBF dual-input PD selector -> LTC4418IUF#PBF dual-input PD selector (V1 = J21)
Connections:
- net PD2_SEL_OV is gone; now on net GND: U14.5 (OV2)
- net PD2_SEL_UV is gone; now on net GND: U14.4 (UV2)
- net PD2_VALID_N is gone; now on net PD_SEL_INTVCC: U14.10 (INTVCC)
- net AUX_DC_RAW: now also F195.2; no longer J190.1 (Pin_1)
- net GND: now also U14.12 (VS2), U14.16 (V2), U14.8 (GND), C2140.2; no longer H10.2, U14.7 (GND)
- net PD1_SEL_UV: now also R2140.2
- net PD1_VALID_N: now also U14.6 (~{VALID1}); no longer U14.9 (~{VALID1})
- net PD1_VBUS_GATED: now also R2140.1
- net PD_SEL_INTVCC: now also C2140.1; no longer H10.1, U14.8 (INTVCC)
- removed net PD2_SEL_FET_COMMON: R2140.2 (S), R2140.3 (S), R2140.4 (S), U14.12 (VS2)
- net PD2_SEL_GATE: no longer names the net of U14.11 (G2)
- net PD2_SEL_GATE: no longer R2140.1 (G)
- removed net PD2_VBUS_GATED: R2140.5 (D(5-8)), U14.16 (V2)
- new net AUX_DC_TERM: F195.1, J190.1 (Pin_1)
- no-connect marks 34 -> 36
Other:
- note added: "LTC4418 independently validates approximately 13.1V to 17.1V and prevents the attached adapter from backfeeding."
- note added: "Phase 5: J11 (PD2) charge power is selected on the CENTER board (U15B); this board exports its own gated VBUS only."
- note removed: "LTC4418 independently validates approximately 13.1V to 17.1V and prevents either attached adapter from backfeeding the other."

Commit message: get the main boards ready for routing
Parts:
- U2001: ChannelUse CC1_CC2_AND_USB2_DP_DM;DEAD_BATTERY_RD_ENABLED -> CC1_CC2_AND_USB2_DP_DN;DEAD_BATTERY_RD_ENABLED
Connections:
- net PD1_DM_CONN renamed PD1_CONN_DN
- net PD1_DM_HOST_SWITCHED renamed PD1_HOST_SWITCHED_DN
- net PD1_DP_CONN renamed PD1_CONN_DP
- net PD1_DP_HOST_SWITCHED renamed PD1_HOST_SWITCHED_DP
- net USBC1_DM renamed USBC1_DN
Changed lines of the file:
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@@
   (effects (font (size 1.27 1.27)) (justify left bottom))
 )
-(label "PD1_DP_CONN"
+(label "PD1_CONN_DP"
   (at 289.56 99.06 0)
   (effects (font (size 1.27 1.27)) (justify left bottom))
 )
-(label "PD1_DP_CONN"
+(label "PD1_CONN_DP"
   (at 289.56 101.6 0)
   (effects (font (size 1.27 1.27)) (justify left bottom))
 )
-(label "PD1_DM_CONN"
+(label "PD1_CONN_DN"
   (at 289.56 93.98 0)
   (effects (font (size 1.27 1.27)) (justify left bottom))
 )
-(label "PD1_DM_CONN"
+(label "PD1_CONN_DN"
   (at 289.56 96.52 0)
   (effects (font (size 1.27 1.27)) (justify left bottom))
@@
   (property "MPN" "TPD4S201RUKR" (at 226.06 106.68 0) (effects (font (size 1.27 1.27)) (hide yes)))
   (property "Datasheet" "https://www.ti.com/lit/ds/symlink/tpd4s201.pdf" (at 226.06 106.68 0) (effects (font (size 1.27 1.27)) (hide yes)))
-  (property "ChannelUse" "CC1_CC2_AND_USB2_DP_DM;DEAD_BATTERY_RD_ENABLED" (at 226.06 106.68 0) (effects (font (size 1.27 1.27)) (hide yes)))
+  (property "ChannelUse" "CC1_CC2_AND_USB2_DP_DN;DEAD_BATTERY_RD_ENABLED" (at 226.06 106.68 0) (effects (font (size 1.27 1.27)) (hide yes)))
   (pin "1")
   (pin "2")
@@
   )
 )
-(label "PD1_DP_CONN"
+(label "PD1_CONN_DP"
   (at 213.36 95.25 0)
   (effects (font (size 1.27 1.27)) (justify left bottom))
 )
-(label "PD1_DM_CONN"
+(label "PD1_CONN_DN"
   (at 213.36 97.79 0)
   (effects (font (size 1.27 1.27)) (justify left bottom))
@@
   (effects (font (size 1.27 1.27)) (justify left bottom))
 )
-(label "PD1_DM_HOST_SWITCHED"
+(label "PD1_HOST_SWITCHED_DN"
   (at 238.76 110.49 0)
   (effects (font (size 1.27 1.27)) (justify left bottom))
 )
-(label "PD1_DP_HOST_SWITCHED"
+(label "PD1_HOST_SWITCHED_DP"
   (at 238.76 107.95 0)
   (effects (font (size 1.27 1.27)) (justify left bottom))
@@
 )
 (no_connect (at 220.98 170.18))
-(label "PD1_DP_HOST_SWITCHED"
+(label "PD1_HOST_SWITCHED_DP"
   (at 200.66 162.56 0)
   (effects (font (size 1.27 1.27)) (justify left bottom))
@@
   (effects (font (size 1.27 1.27)) (justify left bottom))
 )
-(label "PD1_DM_HOST_SWITCHED"
+(label "PD1_HOST_SWITCHED_DN"
   (at 200.66 165.1 0)
   (effects (font (size 1.27 1.27)) (justify left bottom))
 )
 (no_connect (at 220.98 172.72))
-(hierarchical_label "USBC1_DM"
+(hierarchical_label "USBC1_DN"
   (shape bidirectional)
   (at 220.98 165.1 0)

Commit message: fix audit issues and move some connectors
Parts:
- C2146: footprint Capacitor_SMD:CP_Elec_6.3x5.8 -> Capacitor_SMD:CP_Elec_6.3x7.7
- R2080: value 887k 0.1% 15V eFuse UV/OV top -> 8.87k 0.1% 10ppm 15/20V eFuse UV/OV top; MPN RT0603BRD07887KL -> RT0603BRB078K87L
- R2081: value 27.4k 0.1% 15V eFuse UV/OV middle -> 562R 0.1% 10ppm 15/20V eFuse UV/OV middle; MPN RT0603BRD0727K4L -> RT0603BRB07562RL
- R2082: value 68.1k 0.1% 15V eFuse UV/OV bottom -> 511R 0.1% 10ppm 15/20V eFuse UV/OV bottom; MPN RT0603BRD0768K1L -> RT0603BRB07511RL
- R2140: value 1.00M 0.1% 15V UV top -> 1.00M 0.1% 25ppm 15/20V UV top
- R2141: value 19.6k 0.1% 15V window middle -> 35.7k 0.1% 25ppm 15/20V window middle; MPN RT0603BRD0719K6L -> RT0603BRD0735K7L
- R2142: value 63.4k 0.1% 15V OV bottom -> 47.5k 0.1% 25ppm 15/20V OV bottom; MPN RT0603BRD0763K4L -> RT0603BRD0747K5L
Other:
- note added: "J21: hardware accepts 15V/20V PD; use a verified 3A contract and 2.50A charger bootstrap limit. EEPROM/profile qualification remains required."
- note removed: "J21: EEPROM configures DRP prefer-sink, 15V/3A sink, 5V/0.9A source, default Rp, GPIO6 FLIP, GPIO4 DFP, and GPIO7 data-attached."

Commit message: fix more power stuff and update the left board
Parts:
- added C2403: 1u, Capacitor_SMD:C_0805_2012Metric, symbol Device:C
- added C2413: 4.7n C0G PP5V slew, Capacitor_SMD:C_0603_1608Metric, symbol Device:C
- added R2403: 100k, Resistor_SMD:R_0603_1608Metric, symbol Device:R
- added R2413: 10k, Resistor_SMD:R_0603_1608Metric, symbol Device:R
- added U2403: TPS22992SRXNR J21 PP5V gate, ducktop2:Texas_RXN0008A_WQFN-HR-8_1.25x1.25mm, symbol TPS22992S:TPS22992S
- R2080: value 8.87k 0.1% 10ppm 15/20V eFuse UV/OV top -> 8.87k 0.02% 5ppm 15/20V eFuse UV/OV top; MPN RT0603BRB078K87L -> TNPU06038K87HZEN00; Manufacturer Yageo -> Vishay
- R2081: value 562R 0.1% 10ppm 15/20V eFuse UV/OV middle -> 562R 0.02% 5ppm 15/20V eFuse UV/OV middle; MPN RT0603BRB07562RL -> TNPU0603562RHZEN00; Manufacturer Yageo -> Vishay
- R2082: value 511R 0.1% 10ppm 15/20V eFuse UV/OV bottom -> 511R 0.02% 5ppm 15/20V eFuse UV/OV bottom; MPN RT0603BRB07511RL -> TNPU0603511RHZEN00; Manufacturer Yageo -> Vishay
- R2141: value 35.7k 0.1% 25ppm 15/20V window middle -> 35.7k 0.02% 5ppm 15/20V window middle; MPN RT0603BRD0735K7L -> TNPU060335K7HZEN00; Manufacturer Yageo -> Vishay
- R2142: value 47.5k 0.1% 25ppm 15/20V OV bottom -> 47.5k 0.02% 5ppm 15/20V OV bottom; MPN RT0603BRD0747K5L -> TNPU060347K5HZEN00; Manufacturer Yageo -> Vishay
- U41: EEPROMSource firmware/tps25751a/ducktop2_dual_role_config.json -> firmware/tps25751a/ducktop2_pd1_config.json; PortPolicy DRP_PREFER_SINK;HOST_DATA_ONLY;15V_3A_SINK;5V_900MA_SOURCE;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 -> DRP;HOST_DATA_ONLY;5_9_15_20V_3A_SINK;5V_900MA_SOURCE;DEFAU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
Connections:
- net GND: now also C2403.2, C2413.2, R2403.2, U2403.4 (GND)
- net USB_PORT_5V: now also C2403.1, U2403.1 (VBIAS), U2403.2 (VIN); no longer C2025.1, C2026.1, C2027.1, U41.34 (PP5V_(34-35))
- new net J21_PP5V_CT: C2413.1, U2403.7 (CT)
- new net PD1_PP5V_GATED: C2025.1, C2026.1, C2027.1, R2413.1, U2403.5 (QOD), U2403.6 (VOUT), U41.34 (PP5V_(34-35))
- new net PD1_SOURCE_PG: R2413.2, U2403.3 (PG)
- new net USB_J21_PERMIT: R2403.1, U2403.8 (ON)
Other:
- note added: "J21: hardware accepts 15V/20V PD; use a verified 3A contract and 2.50A IINDPM bootstrap command. Actual current/headroom and EEPROM/profile qualification remain required."
- note added: "Phase 5: J11 (PD2) charge power is selected on the CENTER board (U16); this board exports its own gated VBUS only."
- note added: "Seven port permissions reserve VBUS, VCONN and branch losses before power is applied."
- note removed: "Five-port source budget: 5 x 0.9A maximum advertised load = 4.5A on the dedicated 6A USB_PORT_5V rail."
- note removed: "J21: hardware accepts 15V/20V PD; use a verified 3A contract and 2.50A charger bootstrap limit. EEPROM/profile qualification remains required."
- note removed: "Phase 5: J11 (PD2) charge power is selected on the CENTER board (U15B); this board exports its own gated VBUS only."
