File: left_io/left_usb.kicad_sch (KiCad schematic)
At the start: 161 parts, among them J22 USB-C source-only data port J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, J23 USB-C source-only data port J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, J24 USB 3.0 Type-A internal heade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, J25 USB 2.0 Type-A internal heade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, U1700 USB7206C-I/KDX six-port USB 3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, U1701 TPS62823DLC 3A USB7206C 1.146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, U1702 TLV803EA29 USB hub reset supe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, U1703 TPS56637RPAR VSYS to USB_PORT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, U1704 SN74LVC1G08 hub 3V3/core-PG r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, U1740 TPS2553DDBVR 1.3A USB branch, U1741 TPS25810RVCR Type-C DFP contr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, U1742 HD3SS6126RUAR USB3 orientatio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, U1743 TPD1S514-1YZR 5.9V VBUS OVP, U1745 TPD4E05U06 USB2/CC ESD, U1780 TPS2553DDBVR 1.3A USB branch, U1781 TPS25810RVCR Type-C DFP contr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, U1782 HD3SS6126RUAR USB3 orientatio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, U1783 TPD1S514-1YZR 5.9V VBUS OVP, U1785 TPD4E05U06 USB2/CC ESD, U1800 TPS2553DDBVR USB3-A VBUS bran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, U1801 USBLC6-2P6 USB3-A D+/D- ESD, U1802 TPD4E05U06 USB3-A SuperSpeed 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, U1803 TPS2553DDBVR USB2-A VBUS bran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, U1804 USBLC6-2P6 USB2-A D+/D- ESD, Y1700 25.000MHz 3.3V USB hub oscill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

Commit message: fix audit issues and move some connectors
Parts:
- removed C1786: 100n mux VDD, Capacitor_SMD:C_0603_1608Metric, symbol Device:C
- removed C1825: 100n USB7206C VCORE local, Capacitor_SMD:C_0603_1608Metric, symbol Device:C
- removed L1701: 3.3uH >=9A USB port buck, Inductor_SMD:L_Coilcraft_XAL7070-XXX, symbol Device:L
- removed R1700: 10k CFG_STRAP1, Resistor_SMD:R_0603_1608Metric, symbol Device:R
- removed R1710: 169k 1% USB5 EN top, Resistor_SMD:R_0603_1608Metric, symbol Device:R
- removed R1711: 36.1k 1% USB5 EN bottom, Resistor_SMD:R_0603_1608Metric, symbol Device:R
- removed R1712: 74.3k 0.1% USB5 FB top, Resistor_SMD:R_0603_1608Metric, symbol Device:R
- removed U1702: TLV803EA29 USB hub reset supervisor, Package_TO_SOT_SMD:SOT-23-3, symbol TLV803EA29RDBZR:TLV803EA29RDBZR
- added C1712: 10u 50V USB5 input, Capacitor_SMD:C_1206_3216Metric, symbol Device:C
- added C1713, C1867: 100n 50V USB5 input HF, Capacitor_SMD:C_0603_1608Metric, symbol Device:C
- added C1714, C1715: 22u 10V USB5 output, Capacitor_SMD:C_1210_3225Metric, symbol Device:C
- added C1833: 1n USB7206C VDD33 HF, Capacitor_SMD:C_0402_1005Metric, symbol Device:C
- added C1860: 22u 16V USB5 VCC; verify effective capacitance, Capacitor_SMD:C_1206_3216Metric, symbol Device:C
- added C1861: 100n 50V USB5 VDDA, Capacitor_SMD:C_0603_1608Metric, symbol Device:C
- added C1862: 220n 50V X7R USB5 COMP, Capacitor_SMD:C_0603_1608Metric, symbol Device:C
- added C1863: 2.2n 50V C0G USB5 COMP HF, Capacitor_SMD:C_0603_1608Metric, symbol Device:C
- added C1864, C1865: 330u 10V USB5 local reservoir; 4.3mm max height, Capacitor_Tantalum_SMD:CP_EIA-7343-43_Kemet-X, symbol Device:C_Polarized
- added C1866: DNP 68u 25V input damping option, Capacitor_Tantalum_SMD:CP_EIA-7343-20_Kemet-V, symbol Device:C_Polarized
- added R1860: 49.9k 0.1% 10ppm USB5 RT, Resistor_SMD:R_0603_1608Metric, symbol Device:R
- added R1861: 29.4k 1% standalone DRSS off, Resistor_SMD:R_0603_1608Metric, symbol Device:R
- added R1862: 6.8k 1% USB5 COMP, Resistor_SMD:R_0603_1608Metric, symbol Device:R
- added R1863: 1R USB5 bootstrap damping, Resistor_SMD:R_0603_1608Metric, symbol Device:R
- added U1701: TPS62823DLC 3A USB7206C 1.146V core buck, Package_SON:Texas_VSON-HR-8_1.5x2mm_P0.5mm, symbol Regulator_Switching:TPS62823DLC
- added U1740: TPS2553DDBVR 1.3A USB branch, Package_TO_SOT_SMD:SOT-23-6, symbol TPS2553D:TPS2553D
- added U1782: HD3SS6126RUAR USB3 orientation mux, Package_DFN_QFN:WQFN-42-1EP_3.5x9mm_P0.5mm_EP2.05x7.55mm_ThermalVias, symbol Interface_USB:HD3SS6126
- added U1802: TPD4E05U06 USB3-A SuperSpeed ESD, Package_SON:USON-10_2.5x1.0mm_P0.5mm, symbol Power_Protection:TPD4EUSB30
- C1710: value 100n USB5 bootstrap -> 47n 25V USB5 bootstrap; footprint Capacitor_SMD:C_0603_1608Metric -> Capacitor_SMD:C_0402_1005Metric; MPN GRM188R71H104KA93D -> GRM155R71E473KA88D
- C1711: Manufacturer Murata -> TDK
- C1786: renamed from U1740; value TPS2553DDBVR 1.3A USB branch -> 100n mux VDD; footprint Package_TO_SOT_SMD:SOT-23-6 -> Capacitor_SMD:C_0603_1608Metric; symbol TPS2553D:TPS2553D -> Device:C; MPN TPS2553DDBVR -> GRM188R71H104KA93D; Manufacturer Texas Instruments -> Murata
- C1825: renamed from U1782; value HD3SS6126RUAR USB3 orientation mux -> 100n USB7206C VCORE local; footprint Package_DFN_QFN:WQFN-42-1EP_3.5x9mm_P0.5mm_EP2.05x7.55mm_ThermalVias -> Capacitor_SMD:C_0603_1608Metric; symbol Interface_USB:HD3SS6126 -> Device:C; EnableState HS_OE_GND_NORMAL_OPERATION -> (none); MPN HD3SS6126RUAR -> GRM188R71H104KA93D; Manufacturer Texas Instruments -> Murata
- C1850, C1854: footprint Capacitor_SMD:C_1206_3216Metric -> Capacitor_SMD:C_0805_2012Metric
- L1701: renamed from C1712; value 10u 50V USB5 input -> 6.8uH 12.8A Isat30 / 6.8A Irms20; footprint Capacitor_SMD:C_1206_3216Metric -> Inductor_SMD:L_Coilcraft_XAL7070-XXX; symbol Device:C -> Device:L; MPN CGA5L1X7R1H106K160AC -> XAL7070-682MEC; Manufacturer Murata -> Coilcraft
- R1700: renamed from U1802; value TPD4E05U06 USB3-A SuperSpeed ESD -> 10k CFG_STRAP1; footprint Package_SON:USON-10_2.5x1.0mm_P0.5mm -> Resistor_SMD:R_0603_1608Metric; symbol Power_Protection:TPD4EUSB30 -> Device:R; MPN TPD4E05U06DQAR -> RC0603FR-0710KL; Manufacturer Texas Instruments -> Yageo
- R1710: renamed from C1714; value 22u 10V USB5 output -> 100k USB5 switched-3V3 EN top; footprint Capacitor_SMD:C_1210_3225Metric -> Resistor_SMD:R_0603_1608Metric; symbol Device:C -> Device:R; MPN GRM32ER71A226KE20L -> RC0603FR-07100KL; Manufacturer Murata -> Yageo
- R1711: renamed from C1715; value 22u 10V USB5 output -> 100k USB5 EN bottom; footprint Capacitor_SMD:C_1210_3225Metric -> Resistor_SMD:R_0603_1608Metric; symbol Device:C -> Device:R; MPN GRM32ER71A226KE20L -> RC0603FR-07100KL; Manufacturer Murata -> Yageo
- R1712: renamed from U1701; value TPS62823DLC 3A USB7206C 1.146V core buck -> 54.9k 0.1% 10ppm USB5 FB top; footprint Package_SON:Texas_VSON-HR-8_1.5x2mm_P0.5mm -> Resistor_SMD:R_0603_1608Metric; symbol Regulator_Switching:TPS62823DLC -> Device:R; MPN TPS62823DLC -> RT0603BRB0754K9L; Manufacturer Texas Instruments -> Yageo
- R1713: value 10.0k 0.1% USB5 FB bottom -> 10.2k 0.1% 10ppm USB5 FB bottom; MPN RT0603BRD0710KL -> RT0603BRB0710K2L
- RS1860: renamed from C1713; value 100n 50V USB5 input HF -> 5.6mOhm 1% 0.5W USB5 current sense; footprint Capacitor_SMD:C_0603_1608Metric -> ducktop2:Vishay_WSL2010_1to6m9; symbol Device:C -> Device:R; MPN GRM188R71H104KA93D -> WSL20105L600FEA; Manufacturer Murata -> Vishay Dale
- U1702: renamed from C1833; value 1n USB7206C VDD33 HF -> TLV803EA29 USB hub reset supervisor; footprint Capacitor_SMD:C_0402_1005Metric -> Package_TO_SOT_SMD:SOT-23-3; symbol Device:C -> TLV803EA29RDBZR:TLV803EA29RDBZR; MPN GRM155R71H102KA01D -> TLV803EA29RDBZR; Manufacturer Murata -> Texas Instruments
- U1703: value TPS56637RPAR VSYS to USB_PORT_5V 5.06V nominal -> LM706A0RRXR USB5 5.106V; 5.5A system limit; footprint ducktop2:Texas_RPA0010A_VQFN-HR-10_3x3mm -> ducktop2:Texas_RRX0029B_VQFN-29_6x6mm; symbol TPS56637:TPS56637 -> LM706A0:LM706A0; Compensation (none) -> external;6.8k+220n;2.2nHF;two330uF_local; Layout (none) -> separate_SW4_bootstrap_return;Kelvin_ISNS+_and_VOUT; MPN TPS56637RPAR -> LM706A0RRXR; Startup (none) -> ports_off_until_rails_settle
Connections:
- net GND: now also C1825.2, R1700.2, U1703.17 (AGND), U1703.23 (PGND1), U1703.24 (PGND2), U1703.25 (PGND3), U1703.26 (PGND4), U1703.30 (PGND), U1703.6 (BIAS), U1703.8 (PFM/SYNCIN), C1712.2, C1713.2, C1714.2, C1715.2, C1833.2, C1860.2, C1861.2, C1862.2, C1863.2, C1864.2, C1865.2, C1866.2, C1867.2, R1860.2, R1861.2, U1701.3 (AGND), U1701.5 (PGND), U1740.2 (GND), U1782.10 (GND), U1782.14 (GND), U1782.17 (GND), U1782.19 (GND), U1782.21 (GND), U1782.43 (EPAD), U1782.6 (HS_~{OE}), U1802.3 (GND), U1802.8 (GND); no longer C1825.10 (GND), C1825.14 (GND), C1825.17 (GND), C1825.19 (GND), C1825.21 (GND), C1825.43 (EPAD), C1825.6 (HS_~{OE}), L1701.2, R1700.3 (GND), R1700.8 (GND), R1710.2, R1712.3 (AGND), R1712.5 (PGND), RS1860.2, U1703.10 (MODE), U1703.3 (AGND), U1703.9 (PGND), U1801.5 (VBUS), U1804.5 (VBUS)
- net HUB_3V3_OK: now also U1702.1 (RESETz)
- net HUB_CFG1: now also R1700.1
- net HUB_CORE_FB: now also U1701.2 (FB); no longer R1712.2 (FB)
- net HUB_CORE_PG: now also U1701.8 (PG); no longer R1712.8 (PG)
- net HUB_CORE_SW: now also U1701.6 (SW); no longer R1712.6 (SW)
- net HUB_DIS5_RX_N: now also U1802.5 (D2-); no longer R1700.5 (D2-)
- net HUB_DIS5_RX_P: now also U1802.4 (D2+); no longer R1700.4 (D2+)
- net HUB_DIS5_TX_N: now also U1802.2 (D1-); no longer R1700.2 (D1-)
- net HUB_DIS5_TX_P: now also U1802.1 (D1+); no longer R1700.1 (D1+)
- net HUB_DS2_SSRX_N: now also U1782.16 (SSA1(n)); no longer C1825.16 (SSA1(n))
- net HUB_DS2_SSRX_P: now also U1782.15 (SSA1(p)); no longer C1825.15 (SSA1(p))
- net HUB_DS2_SSTX_N: now also U1782.12 (SSA0(n)); no longer C1825.12 (SSA0(n))
- net HUB_DS2_SSTX_P: now also U1782.11 (SSA0(p)); no longer C1825.11 (SSA0(p))
- net HUB_PRT_CTL3: now also U1740.3 (EN), U1740.4 (~{FAULT}); no longer C1786.3 (EN), C1786.4 (~{FAULT})
- net HUB_VCORE: now also C1825.1
- net J22_POL_N: now also U1782.9 (SEL); no longer C1825.9 (SEL)
- net J22_RX1_N: now also U1782.22 (SSC1(n)); no longer C1825.22 (SSC1(n))
- net J22_RX1_P: now also U1782.23 (SSC1(p)); no longer C1825.23 (SSC1(p))
- net J22_RX2_N: now also U1782.26 (SSB1(n)); no longer C1825.26 (SSB1(n))
- net J22_RX2_P: now also U1782.27 (SSB1(p)); no longer C1825.27 (SSB1(p))
- net J22_TX1_N: now also U1782.24 (SSC0(n)); no longer C1825.24 (SSC0(n))
- net J22_TX1_P: now also U1782.25 (SSC0(p)); no longer C1825.25 (SSC0(p))
- net J22_TX2_N: now also U1782.28 (SSB0(n)); no longer C1825.28 (SSB0(n))
- net J22_TX2_P: now also U1782.29 (SSB0(p)); no longer C1825.29 (SSB0(p))
- net J23_5V_PRE: now also U1740.6 (OUT); no longer C1786.6 (OUT)
- net J23_ILIM: now also U1740.5 (ILIM); no longer C1786.5 (ILIM)
- net J24_5V_PRE: now also U1801.5 (VBUS)
- net J25_5V_PRE: now also U1804.5 (VBUS)
- net SYS_3V3: now also C1786.1, R1710.1, U1702.3 (VDD), C1833.1, U1701.1 (EN), U1701.7 (VIN), U1782.13 (VDD), U1782.20 (VDD), U1782.30 (VDD); no longer C1825.13 (VDD), C1825.20 (VDD), C1825.30 (VDD), R1712.1 (EN), R1712.7 (VIN), U1702.1
- net USB5_BOOT: now also U1703.4 (CBOOT), R1863.1; no longer C1710.1, U1703.7 (BOOT)
- net USB5_EN: now also R1710.2, R1711.1, U1703.9 (EN/UVLO); no longer U1703.1 (EN)
- net USB5_FB: now also R1712.2, U1703.16 (FB); no longer U1703.2 (FB)
- net USB5_PG: now also U1703.7 (PG/SYNCOUT); no longer U1703.4 (PG)
- net USB5_SW: now also L1701.1, U1703.20 (SW1), U1703.21 (SW2), U1703.22 (SW3); no longer C1710.2, U1703.6 (SW)
- net USB_PORT_5V: now also R1712.1, RS1860.2, U1703.12 (VOUT), C1714.1, C1715.1, C1864.1, C1865.1, U1740.1 (IN); no longer C1786.1 (IN), R1710.1, R1711.1
- net VSYS: now also U1703.1 (VIN4), U1703.2 (VIN5), U1703.27 (VIN1), U1703.28 (VIN2), U1703.29 (VIN3), U1703.3 (VIN6), C1712.1, C1713.1, C1866.1, C1867.1; no longer L1701.1, RS1860.1, U1703.8 (VIN)
- net USB5_SW_BOOT: now reaches U1703.5 (SW4)
- net USB5_SW_BOOT: now also C1710.2
- new net USB5_BOOT_C: C1710.1, R1863.2
- new net USB5_COMP: C1863.1, R1862.1, U1703.15 (EXTCOMP)
- new net USB5_COMP_RC: C1862.1, R1862.2
- new net USB5_CONFIG: R1861.1, U1703.13 (CONFIG)
- new net USB5_PRE_SENSE: L1701.2, RS1860.1, U1703.11 (ISNS+)
- new net USB5_RT: R1860.1, U1703.14 (RT)
- new net USB5_VCC: C1860.1, U1703.19 (VCC)
- new net USB5_VDDA: C1861.1, U1703.18 (VDDA)
Other:
- note added: "5.5A is a system budget. Harness loss, capacitor corners, startup, load steps and thermal behavior still require qualification."
- note added: "== 5.5A system port budget and 1.15V hub-core rail =="
- note added: "USB5: external COMP 6.8k / 220n / 2.2n; include both local reservoirs and remote PP5V banks in the loop model."
- note removed: "== Dedicated 6A-class port rail and 1.15V hub-core rail =="

Commit message: fix more power stuff and update the left board
Parts:
- removed C1716: 100n oscillator bypass, Capacitor_SMD:C_0603_1608Metric, symbol Device:C
- removed C1722, C1723: 100n USB 3.2 TX AC coupling, Capacitor_SMD:C_0402_1005Metric, symbol Device:C
- removed C1740, C1780: 100n branch input, Capacitor_SMD:C_0603_1608Metric, symbol Device:C
- removed C1741, C1781: 100n TPS25810 IN HF, Capacitor_SMD:C_0603_1608Metric, symbol Device:C
- removed C1742, C1782: 150u 10V TPS25810 input reservoir, Capacitor_Tantalum_SMD:CP_EIA-7343-31_Kemet-D, symbol Device:C_Polarized
- removed L1700: 470nH >=3.9A USB hub core, ducktop2:TDK_TFM201610, symbol Device:L
- removed R1701: 200k CFG_STRAP2, Resistor_SMD:R_0603_1608Metric, symbol Device:R
- removed R1702: 200k CFG_STRAP3, Resistor_SMD:R_0603_1608Metric, symbol Device:R
- removed R1705: 91.0k 1% core FB top, Resistor_SMD:R_0603_1608Metric, symbol Device:R
- removed R1706: 100k 1% core FB bottom, Resistor_SMD:R_0603_1608Metric, symbol Device:R
- removed R1850, R1851: 20.0k 1% TPS2553 1.3A ILIM, Resistor_SMD:R_0603_1608Metric, symbol Device:R
- removed unit 5 of U1700
- added C1708, C1709: 10u core output, Capacitor_SMD:C_0805_2012Metric, symbol Device:C
- added C1828: 100n USB7206C VCORE local, Capacitor_SMD:C_0603_1608Metric, symbol Device:C
- added C1848: 1n USB7206C VCORE HF, Capacitor_SMD:C_0402_1005Metric, symbol Device:C
- added C1849: 10u USB7206C VDD33 bulk, Capacitor_SMD:C_0805_2012Metric, symbol Device:C
- added C1864, C1865: 330u 10V USB5 local reservoir; 4.3mm max height, Capacitor_Tantalum_SMD:CP_EIA-7343-43_Kemet-X, symbol Device:C_Polarized
- added C1866: DNP 68u 25V input damping option, Capacitor_Tantalum_SMD:CP_EIA-7343-20_Kemet-V, symbol Device:C_Polarized
- added C2400, C2401, C2402, C2405, C2406, C2407, C2408, C2410, C2411, C2415: 100n, Capacitor_SMD:C_0603_1608Metric, symbol Device:C
- added D1806, D1807, D1814, D1815: TPD1E0B04DPLR 0.13pF USB3 ESD, Diode_SMD:D_0201_0603Metric, symbol TPD1E0B04:TPD1E0B04
- added R1721, R1722, R1723: 100k unused SPI pull-down, Resistor_SMD:R_0603_1608Metric, symbol Device:R
- added R2400, R2401, R2402, R2412, R2429: 10k, Resistor_SMD:R_0603_1608Metric, symbol Device:R
- added R2405, R2406, R2407, R2408, R2410, R2420, R2421, R2422, R2423, R2426, R2427: 100k, Resistor_SMD:R_0603_1608Metric, symbol Device:R
- added R2424, R2425: 12.7k 1%, Resistor_SMD:R_0603_1608Metric, symbol Device:R
- added unit 1 of U1700
- added U1745, U1785: TPD4E05U06 USB2/CC ESD, Package_SON:USON-10_2.5x1.0mm_P0.5mm, symbol Power_Protection:TPD4E05U06DQA
- added U1801: USBLC6-2P6 USB3-A D+/D- ESD, Package_TO_SOT_SMD:SOT-666, symbol Power_Protection:USBLC6-2P6
- added U1804: USBLC6-2P6 USB2-A D+/D- ESD, Package_TO_SOT_SMD:SOT-666, symbol Power_Protection:USBLC6-2P6
- added U2400: TCA9539PWR USB permissions @0x76, Package_SO:TSSOP-24_4.4x7.8mm_P0.65mm, symbol Interface_Expansion:PCA9539xD
- added U2401: INA226AIDGSR USB5 monitor @0x40, Package_SO:TSSOP-10_3x3mm_P0.5mm, symbol Sensor_Energy:INA226
- added U2402: SN74LVC1G74DCUR USB fault latch, ducktop2:TI_DCU0008A_VSSOP8, symbol SN74LVC1G74DCU:SN74LVC1G74DCU
- added U2405: SN74LVC1G08DBVR J22 source permission, Package_TO_SOT_SMD:SOT-23-5, symbol 74xGxx:74LVC1G08
- added U2406: SN74LVC1G08DBVR J23 source permission, Package_TO_SOT_SMD:SOT-23-5, symbol 74xGxx:74LVC1G08
- added U2407: SN74LVC1G08DBVR J24 source permission, Package_TO_SOT_SMD:SOT-23-5, symbol 74xGxx:74LVC1G08
- added U2408: SN74LVC1G08DBVR J25 source permission, Package_TO_SOT_SMD:SOT-23-5, symbol 74xGxx:74LVC1G08
- added U2410: SN74LVC1G11DCKR USB5 permit AND, Package_TO_SOT_SMD:SOT-363_SC-70-6, symbol 74xGxx:74LVC1G11
- added U2411: SN74LVC1G08DBVR raw fault veto, Package_TO_SOT_SMD:SOT-23-5, symbol 74xGxx:74LVC1G08
- added U2413: SN74LVC1G08DBVR raw OC and SYS5 veto, Package_TO_SOT_SMD:SOT-23-5, symbol 74xGxx:74LVC1G08
- C1705: renamed from C1708; value 10u core output -> 120p core feed-forward; footprint Capacitor_SMD:C_0805_2012Metric -> Capacitor_SMD:C_0402_1005Metric; MPN GRM21BR71A106KE51L -> GRM1555C1H121JA01D
- C1706: renamed from C1709; value 10u core output -> 4.7u core input; MPN GRM21BR71A106KE51L -> GRM21BR71A475KA73L
- C1707: renamed from U1700; value USB7206C-I/KDX six-port USB 3.2 Gen 2 hub -> 100n core input HF; footprint Package_DFN_QFN:VQFN-100-1EP_12x12mm_P0.4mm_EP8x8mm_ThermalVias -> Capacitor_SMD:C_0603_1608Metric; symbol USB7206C:USB7206C -> Device:C; MPN USB7206C-I/KDX -> GRM188R71H104KA93D; Manufacturer Microchip -> Murata
- C1710: renamed from C1711; value 10u 50V USB5 input -> 47n 25V USB5 bootstrap; footprint Capacitor_SMD:C_1206_3216Metric -> Capacitor_SMD:C_0402_1005Metric; MPN CGA5L1X7R1H106K160AC -> GRM155R71E473KA88D; Manufacturer TDK -> Murata
- C1712: renamed from C1713; value 100n 50V USB5 input HF -> 10u 50V USB5 input; footprint Capacitor_SMD:C_0603_1608Metric -> Capacitor_SMD:C_1206_3216Metric; MPN GRM188R71H104KA93D -> CGA5L1X7R1H106K160AC; Manufacturer Murata -> TDK
- C1714: renamed from C1715; value 22u 10V USB5 output -> 22u 25V USB5 output; TI characterized part; MPN GRM32ER71A226KE20L -> GRM32ER71E226KE15L
- C1715: renamed from C1860; value 22u 16V USB5 VCC; verify effective capacitance -> 22u 25V USB5 output; TI characterized part; footprint Capacitor_SMD:C_1206_3216Metric -> Capacitor_SMD:C_1210_3225Metric; MPN GRM31CZ71C226ME15L -> GRM32ER71E226KE15L
- C1716: renamed from C1724; value 100n USB 3.2 TX AC coupling -> 100n oscillator bypass; footprint Capacitor_SMD:C_0402_1005Metric -> Capacitor_SMD:C_0603_1608Metric; MPN GRM155R71C104KA88D -> GRM188R71H104KA93D
- C1725: renamed from C1810; value 100n USB7206C VDD33 local -> 100n USB 3.2 TX AC coupling; footprint Capacitor_SMD:C_0603_1608Metric -> Capacitor_SMD:C_0402_1005Metric; MPN GRM188R71H104KA93D -> GRM155R71C104KA88D
- C1728: renamed from C1830; value 1n USB7206C VDD33 HF -> 100n USB 3.2 TX AC coupling; MPN GRM155R71H102KA01D -> GRM155R71C104KA88D
- C1729: renamed from C1811; value 100n USB7206C VDD33 local -> 100n USB 3.2 TX AC coupling; footprint Capacitor_SMD:C_0603_1608Metric -> Capacitor_SMD:C_0402_1005Metric; MPN GRM188R71H104KA93D -> GRM155R71C104KA88D
- C1740: renamed from C1743; value 10u protected VBUS_SYS -> 100n branch input; footprint Capacitor_SMD:C_1206_3216Metric -> Capacitor_SMD:C_0603_1608Metric; MPN GRM31CR71A106KA01L -> GRM188R71H104KA93D
- C1741: renamed from C1744; value 100n TPS25810 AUX -> 100n TPS25810 IN HF
- C1742: renamed from C1745; value 100n mux VDD -> 150u 10V TPS25810 input reservoir; footprint Capacitor_SMD:C_0603_1608Metric -> Capacitor_Tantalum_SMD:CP_EIA-7343-31_Kemet-D; symbol Device:C -> Device:C_Polarized; MPN GRM188R71H104KA93D -> T520D157M010ATE025; Manufacturer Murata -> KEMET
- C1743: renamed from C1746; value 100n mux VDD -> 10u protected VBUS_SYS; footprint Capacitor_SMD:C_0603_1608Metric -> Capacitor_SMD:C_1206_3216Metric; MPN GRM188R71H104KA93D -> GRM31CR71A106KA01L
- C1744: renamed from C1747; value 100n mux VDD -> 100n TPS25810 AUX
- C1745: renamed from C1748; value 1u mux local bulk -> 100n mux VDD; MPN GRM188R71A105KA61D -> GRM188R71H104KA93D
- C1746: renamed from C1749; value 10n mux HF -> 100n mux VDD; footprint Capacitor_SMD:C_0402_1005Metric -> Capacitor_SMD:C_0603_1608Metric; MPN GRM155R71H103KA88D -> GRM188R71H104KA93D
- C1747: renamed from R1741; value 4.99k POL pull-up -> 100n mux VDD; footprint Resistor_SMD:R_0603_1608Metric -> Capacitor_SMD:C_0603_1608Metric; symbol Device:R -> Device:C; MPN RC0603FR-074K99L -> GRM188R71H104KA93D; Manufacturer Yageo -> Murata
- C1748: renamed from R1742; value 100k 1% TPS25810 REF -> 1u mux local bulk; footprint Resistor_SMD:R_0603_1608Metric -> Capacitor_SMD:C_0603_1608Metric; symbol Device:R -> Device:C; MPN RC0603FR-07100KL -> GRM188R71A105KA61D; Manufacturer Yageo -> Murata
- C1749: renamed from R1750; value 249R 0.25W TPS25810 OUT discharge -> 10n mux HF; footprint Resistor_SMD:R_1206_3216Metric -> Capacitor_SMD:C_0402_1005Metric; symbol Device:R -> Device:C; MPN RC1206FR-07249RL -> GRM155R71H103KA88D; Manufacturer Yageo -> Murata
- C1750: renamed from D1809; value TPD1E0B04DPLR 0.13pF USB3 ESD -> 1u 50V connector-side VBUS; footprint Diode_SMD:D_0201_0603Metric -> Capacitor_SMD:C_0805_2012Metric; symbol TPD1E0B04:TPD1E0B04 -> Device:C; MPN TPD1E0B04DPLR -> GRM21BR71H105KA12L; Manufacturer Texas Instruments -> Murata
- C1751: renamed from D1810; value TPD1E0B04DPLR 0.13pF USB3 ESD -> 1u TPD1S514 VBUS_POWER stability; footprint Diode_SMD:D_0201_0603Metric -> Capacitor_SMD:C_0603_1608Metric; symbol TPD1E0B04:TPD1E0B04 -> Device:C; MPN TPD1E0B04DPLR -> GRM188R71A105KA61D; Manufacturer Texas Instruments -> Murata
- C1780: renamed from C1783; value 10u protected VBUS_SYS -> 100n branch input; footprint Capacitor_SMD:C_1206_3216Metric -> Capacitor_SMD:C_0603_1608Metric; MPN GRM31CR71A106KA01L -> GRM188R71H104KA93D
- C1781: renamed from C1784; value 100n TPS25810 AUX -> 100n TPS25810 IN HF
- C1782: renamed from C1785; value 100n mux VDD -> 150u 10V TPS25810 input reservoir; footprint Capacitor_SMD:C_0603_1608Metric -> Capacitor_Tantalum_SMD:CP_EIA-7343-31_Kemet-D; symbol Device:C -> Device:C_Polarized; MPN GRM188R71H104KA93D -> T520D157M010ATE025; Manufacturer Murata -> KEMET
- C1783: renamed from C1786; value 100n mux VDD -> 10u protected VBUS_SYS; footprint Capacitor_SMD:C_0603_1608Metric -> Capacitor_SMD:C_1206_3216Metric; MPN GRM188R71H104KA93D -> GRM31CR71A106KA01L
- C1784: renamed from C1787; value 100n mux VDD -> 100n TPS25810 AUX
- C1785: renamed from C1788; value 1u mux local bulk -> 100n mux VDD; MPN GRM188R71A105KA61D -> GRM188R71H104KA93D
- C1786: renamed from C1789; value 10n mux HF -> 100n mux VDD; footprint Capacitor_SMD:C_0402_1005Metric -> Capacitor_SMD:C_0603_1608Metric; MPN GRM155R71H103KA88D -> GRM188R71H104KA93D
- C1787: renamed from R1781; value 4.99k POL pull-up -> 100n mux VDD; footprint Resistor_SMD:R_0603_1608Metric -> Capacitor_SMD:C_0603_1608Metric; symbol Device:R -> Device:C; MPN RC0603FR-074K99L -> GRM188R71H104KA93D; Manufacturer Yageo -> Murata
- C1788: renamed from R1782; value 100k 1% TPS25810 REF -> 1u mux local bulk; footprint Resistor_SMD:R_0603_1608Metric -> Capacitor_SMD:C_0603_1608Metric; symbol Device:R -> Device:C; MPN RC0603FR-07100KL -> GRM188R71A105KA61D; Manufacturer Yageo -> Murata
- C1789: renamed from R1790; value 249R 0.25W TPS25810 OUT discharge -> 10n mux HF; footprint Resistor_SMD:R_1206_3216Metric -> Capacitor_SMD:C_0402_1005Metric; symbol Device:R -> Device:C; MPN RC1206FR-07249RL -> GRM155R71H103KA88D; Manufacturer Yageo -> Murata
- C1790: renamed from D1801; value TPD1E0B04DPLR 0.13pF USB3 ESD -> 1u 50V connector-side VBUS; footprint Diode_SMD:D_0201_0603Metric -> Capacitor_SMD:C_0805_2012Metric; symbol TPD1E0B04:TPD1E0B04 -> Device:C; MPN TPD1E0B04DPLR -> GRM21BR71H105KA12L; Manufacturer Texas Instruments -> Murata
- C1791: renamed from D1802; value TPD1E0B04DPLR 0.13pF USB3 ESD -> 1u TPD1S514 VBUS_POWER stability; footprint Diode_SMD:D_0201_0603Metric -> Capacitor_SMD:C_0603_1608Metric; symbol TPD1E0B04:TPD1E0B04 -> Device:C; MPN TPD1E0B04DPLR -> GRM188R71A105KA61D; Manufacturer Texas Instruments -> Murata
- C1810: renamed from C1831; value 1n USB7206C VDD33 HF -> 100n USB7206C VDD33 local; footprint Capacitor_SMD:C_0402_1005Metric -> Capacitor_SMD:C_0603_1608Metric; MPN GRM155R71H102KA01D -> GRM188R71H104KA93D
- C1811: renamed from C1832; value 1n USB7206C VDD33 HF -> 100n USB7206C VDD33 local; footprint Capacitor_SMD:C_0402_1005Metric -> Capacitor_SMD:C_0603_1608Metric; MPN GRM155R71H102KA01D -> GRM188R71H104KA93D
- C1812: renamed from C1833; value 1n USB7206C VDD33 HF -> 100n USB7206C VDD33 local; footprint Capacitor_SMD:C_0402_1005Metric -> Capacitor_SMD:C_0603_1608Metric; MPN GRM155R71H102KA01D -> GRM188R71H104KA93D
- C1813: renamed from C1834; value 1n USB7206C VDD33 HF -> 100n USB7206C VDD33 local; footprint Capacitor_SMD:C_0402_1005Metric -> Capacitor_SMD:C_0603_1608Metric; MPN GRM155R71H102KA01D -> GRM188R71H104KA93D
- C1814: renamed from C1835; value 1n USB7206C VDD33 HF -> 100n USB7206C VDD33 local; footprint Capacitor_SMD:C_0402_1005Metric -> Capacitor_SMD:C_0603_1608Metric; MPN GRM155R71H102KA01D -> GRM188R71H104KA93D
- C1815: renamed from C1836; value 1n USB7206C VDD33 HF -> 100n USB7206C VDD33 local; footprint Capacitor_SMD:C_0402_1005Metric -> Capacitor_SMD:C_0603_1608Metric; MPN GRM155R71H102KA01D -> GRM188R71H104KA93D
- C1816: renamed from C1837; value 1n USB7206C VDD33 HF -> 100n USB7206C VDD33 local; footprint Capacitor_SMD:C_0402_1005Metric -> Capacitor_SMD:C_0603_1608Metric; MPN GRM155R71H102KA01D -> GRM188R71H104KA93D
- C1817: renamed from C1840; value 1n USB7206C VCORE HF -> 100n USB7206C VDD33 local; footprint Capacitor_SMD:C_0402_1005Metric -> Capacitor_SMD:C_0603_1608Metric; MPN GRM155R71H102KA01D -> GRM188R71H104KA93D
- C1820: renamed from C1841; value 1n USB7206C VCORE HF -> 100n USB7206C VCORE local; footprint Capacitor_SMD:C_0402_1005Metric -> Capacitor_SMD:C_0603_1608Metric; MPN GRM155R71H102KA01D -> GRM188R71H104KA93D
- C1821: renamed from C1842; value 1n USB7206C VCORE HF -> 100n USB7206C VCORE local; footprint Capacitor_SMD:C_0402_1005Metric -> Capacitor_SMD:C_0603_1608Metric; MPN GRM155R71H102KA01D -> GRM188R71H104KA93D
- C1822: renamed from C1843; value 1n USB7206C VCORE HF -> 100n USB7206C VCORE local; footprint Capacitor_SMD:C_0402_1005Metric -> Capacitor_SMD:C_0603_1608Metric; MPN GRM155R71H102KA01D -> GRM188R71H104KA93D
- C1823: renamed from C1844; value 1n USB7206C VCORE HF -> 100n USB7206C VCORE local; footprint Capacitor_SMD:C_0402_1005Metric -> Capacitor_SMD:C_0603_1608Metric; MPN GRM155R71H102KA01D -> GRM188R71H104KA93D
- C1824: renamed from C1845; value 1n USB7206C VCORE HF -> 100n USB7206C VCORE local; footprint Capacitor_SMD:C_0402_1005Metric -> Capacitor_SMD:C_0603_1608Metric; MPN GRM155R71H102KA01D -> GRM188R71H104KA93D
- C1825: renamed from C1846; value 1n USB7206C VCORE HF -> 100n USB7206C VCORE local; footprint Capacitor_SMD:C_0402_1005Metric -> Capacitor_SMD:C_0603_1608Metric; MPN GRM155R71H102KA01D -> GRM188R71H104KA93D
- C1826: renamed from C1847; value 1n USB7206C VCORE HF -> 100n USB7206C VCORE local; footprint Capacitor_SMD:C_0402_1005Metric -> Capacitor_SMD:C_0603_1608Metric; MPN GRM155R71H102KA01D -> GRM188R71H104KA93D
- C1827: renamed from C1848; value 1n USB7206C VCORE HF -> 100n USB7206C VCORE local; footprint Capacitor_SMD:C_0402_1005Metric -> Capacitor_SMD:C_0603_1608Metric; MPN GRM155R71H102KA01D -> GRM188R71H104KA93D
- C1830: renamed from C1812; value 100n USB7206C VDD33 local -> 1n USB7206C VDD33 HF; footprint Capacitor_SMD:C_0603_1608Metric -> Capacitor_SMD:C_0402_1005Metric; MPN GRM188R71H104KA93D -> GRM155R71H102KA01D
- C1831: renamed from C1813; value 100n USB7206C VDD33 local -> 1n USB7206C VDD33 HF; footprint Capacitor_SMD:C_0603_1608Metric -> Capacitor_SMD:C_0402_1005Metric; MPN GRM188R71H104KA93D -> GRM155R71H102KA01D
- C1832: renamed from C1814; value 100n USB7206C VDD33 local -> 1n USB7206C VDD33 HF; footprint Capacitor_SMD:C_0603_1608Metric -> Capacitor_SMD:C_0402_1005Metric; MPN GRM188R71H104KA93D -> GRM155R71H102KA01D
- C1833: renamed from C1815; value 100n USB7206C VDD33 local -> 1n USB7206C VDD33 HF; footprint Capacitor_SMD:C_0603_1608Metric -> Capacitor_SMD:C_0402_1005Metric; MPN GRM188R71H104KA93D -> GRM155R71H102KA01D
- C1834: renamed from C1816; value 100n USB7206C VDD33 local -> 1n USB7206C VDD33 HF; footprint Capacitor_SMD:C_0603_1608Metric -> Capacitor_SMD:C_0402_1005Metric; MPN GRM188R71H104KA93D -> GRM155R71H102KA01D
- C1835: renamed from C1817; value 100n USB7206C VDD33 local -> 1n USB7206C VDD33 HF; footprint Capacitor_SMD:C_0603_1608Metric -> Capacitor_SMD:C_0402_1005Metric; MPN GRM188R71H104KA93D -> GRM155R71H102KA01D
- C1836: renamed from C1820; value 100n USB7206C VCORE local -> 1n USB7206C VDD33 HF; footprint Capacitor_SMD:C_0603_1608Metric -> Capacitor_SMD:C_0402_1005Metric; MPN GRM188R71H104KA93D -> GRM155R71H102KA01D
- C1837: renamed from C1821; value 100n USB7206C VCORE local -> 1n USB7206C VDD33 HF; footprint Capacitor_SMD:C_0603_1608Metric -> Capacitor_SMD:C_0402_1005Metric; MPN GRM188R71H104KA93D -> GRM155R71H102KA01D
- C1840: renamed from C1822; value 100n USB7206C VCORE local -> 1n USB7206C VCORE HF; footprint Capacitor_SMD:C_0603_1608Metric -> Capacitor_SMD:C_0402_1005Metric; MPN GRM188R71H104KA93D -> GRM155R71H102KA01D
- C1841: renamed from C1823; value 100n USB7206C VCORE local -> 1n USB7206C VCORE HF; footprint Capacitor_SMD:C_0603_1608Metric -> Capacitor_SMD:C_0402_1005Metric; MPN GRM188R71H104KA93D -> GRM155R71H102KA01D
- C1842: renamed from C1824; value 100n USB7206C VCORE local -> 1n USB7206C VCORE HF; footprint Capacitor_SMD:C_0603_1608Metric -> Capacitor_SMD:C_0402_1005Metric; MPN GRM188R71H104KA93D -> GRM155R71H102KA01D
- C1843: renamed from C1825; value 100n USB7206C VCORE local -> 1n USB7206C VCORE HF; footprint Capacitor_SMD:C_0603_1608Metric -> Capacitor_SMD:C_0402_1005Metric; MPN GRM188R71H104KA93D -> GRM155R71H102KA01D
- C1844: renamed from C1826; value 100n USB7206C VCORE local -> 1n USB7206C VCORE HF; footprint Capacitor_SMD:C_0603_1608Metric -> Capacitor_SMD:C_0402_1005Metric; MPN GRM188R71H104KA93D -> GRM155R71H102KA01D
- C1845: renamed from C1827; value 100n USB7206C VCORE local -> 1n USB7206C VCORE HF; footprint Capacitor_SMD:C_0603_1608Metric -> Capacitor_SMD:C_0402_1005Metric; MPN GRM188R71H104KA93D -> GRM155R71H102KA01D
- C1846: renamed from C1828; value 100n USB7206C VCORE local -> 1n USB7206C VCORE HF; footprint Capacitor_SMD:C_0603_1608Metric -> Capacitor_SMD:C_0402_1005Metric; MPN GRM188R71H104KA93D -> GRM155R71H102KA01D
- C1847: renamed from C1849; value 10u USB7206C VDD33 bulk -> 1n USB7206C VCORE HF; footprint Capacitor_SMD:C_0805_2012Metric -> Capacitor_SMD:C_0402_1005Metric; MPN GRM21BR71A106KE51L -> GRM155R71H102KA01D
- C1860: renamed from R1861; value 29.4k 1% standalone DRSS off -> 22u 25V USB5 VCC; effective minimum 4.7u; footprint Resistor_SMD:R_0603_1608Metric -> Capacitor_SMD:C_1210_3225Metric; symbol Device:R -> Device:C; MPN RC0603FR-0729K4L -> GRM32ER71E226KE15L; Manufacturer Yageo -> Murata
- C1861: renamed from R1862; value 6.8k 1% USB5 COMP -> 100n 50V USB5 VDDA; footprint Resistor_SMD:R_0603_1608Metric -> Capacitor_SMD:C_0603_1608Metric; symbol Device:R -> Device:C; MPN RC0603FR-076K8L -> GRM188R71H104KA93D; Manufacturer Yageo -> Murata
- C1862: renamed from C1865; value 330u 10V USB5 local reservoir; 4.3mm max height -> 220n 50V X7R USB5 COMP; footprint Capacitor_Tantalum_SMD:CP_EIA-7343-43_Kemet-X -> Capacitor_SMD:C_0603_1608Metric; symbol Device:C_Polarized -> Device:C; MPN T520X337M010ATE010 -> C0603C224K5RACTU
- C1863: renamed from C1866; value DNP 68u 25V input damping option -> 2.2n 50V C0G USB5 COMP HF; footprint Capacitor_Tantalum_SMD:CP_EIA-7343-20_Kemet-V -> Capacitor_SMD:C_0603_1608Metric; symbol Device:C_Polarized -> Device:C; MPN T521V686M025ATE050 -> C0603C222J5GACTU; now fitted; now in the parts list
- C1867: renamed from C1714; value 22u 10V USB5 output -> 100n 50V USB5 input HF; footprint Capacitor_SMD:C_1210_3225Metric -> Capacitor_SMD:C_0603_1608Metric; MPN GRM32ER71A226KE20L -> GRM188R71H104KA93D
- C1868: renamed from C1861; value 100n 50V USB5 VDDA -> 22u 25V USB5 output; TI characterized part; footprint Capacitor_SMD:C_0603_1608Metric -> Capacitor_SMD:C_1210_3225Metric; MPN GRM188R71H104KA93D -> GRM32ER71E226KE15L
- C1869: renamed from R1860; value 49.9k 0.1% 10ppm USB5 RT -> 22u 25V USB5 output; TI characterized part; footprint Resistor_SMD:R_0603_1608Metric -> Capacitor_SMD:C_1210_3225Metric; symbol Device:R -> Device:C; MPN RT0603BRB0749K9L -> GRM32ER71E226KE15L; Manufacturer Yageo -> Murata
- D1805: renamed from U1785; value TPD4E05U06 USB2/CC ESD -> TPD1E0B04DPLR 0.13pF USB3 ESD; footprint Package_SON:USON-10_2.5x1.0mm_P0.5mm -> Diode_SMD:D_0201_0603Metric; symbol Power_Protection:TPD4E05U06DQA -> TPD1E0B04:TPD1E0B04; MPN TPD4E05U06DQAR -> TPD1E0B04DPLR
- D1813: renamed from U1745; value TPD4E05U06 USB2/CC ESD -> TPD1E0B04DPLR 0.13pF USB3 ESD; footprint Package_SON:USON-10_2.5x1.0mm_P0.5mm -> Diode_SMD:D_0201_0603Metric; symbol Power_Protection:TPD4E05U06DQA -> TPD1E0B04:TPD1E0B04; MPN TPD4E05U06DQAR -> TPD1E0B04DPLR
- L1700: renamed from R1707; value 100k core PG pull-up -> 470nH >=3.9A USB hub core; footprint Resistor_SMD:R_0603_1608Metric -> ducktop2:TDK_TFM201610; symbol Device:R -> Device:L; MPN RC0603FR-07100KL -> TFM201610ALMA-R47MTAA; Manufacturer Yageo -> TDK
- L1701: value 6.8uH 12.8A Isat30 / 6.8A Irms20 -> 6.8uH 18.4A Isat30 / 10.9A Irms20; footprint Inductor_SMD:L_Coilcraft_XAL7070-XXX -> ducktop2:Coilcraft_XGL1060; Layout (none) -> pad1_is_marked_short_lead_to_SW;6mm_max_height; MPN XAL7070-682MEC -> XGL1060-682MEC
- R1700: renamed from R1703; value 200k all ports removable -> 10k CFG_STRAP1; MPN RC0603FR-07200KL -> RC0603FR-0710KL
- R1701: renamed from R1704; value 200k BC1.2 disabled -> 200k CFG_STRAP2
- R1702: renamed from R1708; value 12.0k 1% USB7206C RBIAS -> 200k CFG_STRAP3; MPN RC0603FR-0712KL -> RC0603FR-07200KL
- R1703: renamed from R1715; value 10k TEST pull-up -> 200k all ports removable; MPN RC0603FR-0710KL -> RC0603FR-07200KL
- R1704: renamed from R1716; value 10k TEST pull-up -> 200k BC1.2 disabled; MPN RC0603FR-0710KL -> RC0603FR-07200KL
- R1705: renamed from C1705; value 120p core feed-forward -> 91.0k 0.02% 5ppm core FB top; footprint Capacitor_SMD:C_0402_1005Metric -> Resistor_SMD:R_0603_1608Metric; symbol Device:C -> Device:R; MPN GRM1555C1H121JA01D -> TNPU060391K0HZEN00; Manufacturer Murata -> Vishay
- R1706: renamed from C1706; value 4.7u core input -> 100k 0.02% 5ppm core FB bottom; footprint Capacitor_SMD:C_0805_2012Metric -> Resistor_SMD:R_0603_1608Metric; symbol Device:C -> Device:R; MPN GRM21BR71A475KA73L -> TNPU0603100KHZEN00; Manufacturer Murata -> Vishay
- R1707: renamed from C1707; value 100n core input HF -> 100k core PG pull-up; footprint Capacitor_SMD:C_0603_1608Metric -> Resistor_SMD:R_0603_1608Metric; symbol Device:C -> Device:R; MPN GRM188R71H104KA93D -> RC0603FR-07100KL; Manufacturer Murata -> Yageo
- R1708: renamed from R1717; value 10k TEST pull-up -> 12.0k 1% USB7206C RBIAS; MPN RC0603FR-0710KL -> RC0603FR-0712KL
- R1710: renamed from R1711; value 100k USB5 EN bottom -> 100k USB5 hardware-qualified EN top
- R1711: renamed from R1712; value 54.9k 0.1% 10ppm USB5 FB top -> 100k USB5 EN bottom; MPN RT0603BRB0754K9L -> RC0603FR-07100KL
- R1712: renamed from R1713; value 10.2k 0.1% 10ppm USB5 FB bottom -> 55.6k 0.02% 5ppm USB5 FB top; MPN RT0603BRB0710K2L -> TNPU060355K6HZEN00; Manufacturer Yageo -> Vishay
- R1713: renamed from R1714; value 100k USB5 PG pull-up -> 10.2k 0.02% 5ppm USB5 FB bottom; MPN RC0603FR-07100KL -> TNPU060310K2HZEN00; Manufacturer Yageo -> Vishay
- R1714: renamed from R1863; value 1R USB5 bootstrap damping -> 100k USB5 PG pull-up; MPN RC0603FR-071RL -> RC0603FR-07100KL
- R1715: renamed from R1720; value 100k unused SPI pull-down -> 10k TEST pull-up; MPN RC0603FR-07100KL -> RC0603FR-0710KL
- R1716: renamed from R1721; value 100k unused SPI pull-down -> 10k TEST pull-up; MPN RC0603FR-07100KL -> RC0603FR-0710KL
- R1717: renamed from R1722; value 100k unused SPI pull-down -> 10k TEST pull-up; MPN RC0603FR-07100KL -> RC0603FR-0710KL
- R1740, R1780: value 20.0k 1% TPS2553 1.3A ILIM -> 19.1k 1% TPS2553 VBUS plus VCONN ILIM; MPN RC0603FR-0720KL -> RC0603FR-0719K1L
- R1741: renamed from C1750; value 1u 50V connector-side VBUS -> 4.99k POL pull-up; footprint Capacitor_SMD:C_0805_2012Metric -> Resistor_SMD:R_0603_1608Metric; symbol Device:C -> Device:R; MPN GRM21BR71H105KA12L -> RC0603FR-074K99L; Manufacturer Murata -> Yageo
- R1742: renamed from C1751; value 1u TPD1S514 VBUS_POWER stability -> 100k 1% TPS25810 REF; footprint Capacitor_SMD:C_0603_1608Metric -> Resistor_SMD:R_0603_1608Metric; symbol Device:C -> Device:R; MPN GRM188R71A105KA61D -> RC0603FR-07100KL; Manufacturer Murata -> Yageo
- R1750: renamed from D1808; value TPD1E0B04DPLR 0.13pF USB3 ESD -> 249R 0.25W TPS25810 OUT discharge; footprint Diode_SMD:D_0201_0603Metric -> Resistor_SMD:R_1206_3216Metric; symbol TPD1E0B04:TPD1E0B04 -> Device:R; MPN TPD1E0B04DPLR -> RC1206FR-07249RL; Manufacturer Texas Instruments -> Yageo
- R1781: renamed from C1790; value 1u 50V connector-side VBUS -> 4.99k POL pull-up; footprint Capacitor_SMD:C_0805_2012Metric -> Resistor_SMD:R_0603_1608Metric; symbol Device:C -> Device:R; MPN GRM21BR71H105KA12L -> RC0603FR-074K99L; Manufacturer Murata -> Yageo
- R1782: renamed from C1791; value 1u TPD1S514 VBUS_POWER stability -> 100k 1% TPS25810 REF; footprint Capacitor_SMD:C_0603_1608Metric -> Resistor_SMD:R_0603_1608Metric; symbol Device:C -> Device:R; MPN GRM188R71A105KA61D -> RC0603FR-07100KL; Manufacturer Murata -> Yageo
- R1790: renamed from D1800; value TPD1E0B04DPLR 0.13pF USB3 ESD -> 249R 0.25W TPS25810 OUT discharge; footprint Diode_SMD:D_0201_0603Metric -> Resistor_SMD:R_1206_3216Metric; symbol TPD1E0B04:TPD1E0B04 -> Device:R; MPN TPD1E0B04DPLR -> RC1206FR-07249RL; Manufacturer Texas Instruments -> Yageo
- R1850: renamed from U1801; value USBLC6-2P6 USB3-A D+/D- ESD -> 20.0k 1% TPS2553 1.3A ILIM; footprint Package_TO_SOT_SMD:SOT-666 -> Resistor_SMD:R_0603_1608Metric; symbol Power_Protection:USBLC6-2P6 -> Device:R; MPN USBLC6-2P6 -> RC0603FR-0720KL; Manufacturer STMicroelectronics -> Yageo
- R1851: renamed from U1804; value USBLC6-2P6 USB2-A D+/D- ESD -> 20.0k 1% TPS2553 1.3A ILIM; footprint Package_TO_SOT_SMD:SOT-666 -> Resistor_SMD:R_0603_1608Metric; symbol Power_Protection:USBLC6-2P6 -> Device:R; MPN USBLC6-2P6 -> RC0603FR-0720KL; Manufacturer STMicroelectronics -> Yageo
- renumbered C1712 to C1711, C1867 to C1713, C1725 to C1722, C1728 to C1723, C1729 to C1724, D1803 to D1800, D1804 to D1801, D1805 to D1802, D1806 to D1803, D1807 to D1804, D1811 to D1808, D1812 to D1809, D1813 to D1810, D1814 to D1811, D1815 to D1812, R1723 to R1720
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Connections:
- net GND: now also C1707.2, C1716.2, C1747.2, C1748.2, C1787.2, C1788.2, C1861.2, D1805.2 (IO), D1813.2 (IO), R1703.2, R1704.2, R1708.2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; no longer C1705.2, C1707.101 (GND), C1707.24 (TESTEN), C1710.2, C1725.2, C1728.2, C1729.2, D1805.3 (GND), D1805.8 (GND), D1813.3 (GND), D1813.8 (GND), R1707.2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
- net HUB_BC_EN: now also R1704.1, U1700.70 (SPI_D0/CFG_BC_EN/PF22); no longer C1707.70 (SPI_D0/CFG_BC_EN/PF22), R1701.1
- net HUB_CFG1: now also R1700.1, U1700.21 (CFG_STRAP1); no longer C1707.21 (CFG_STRAP1), U1700.1
- net HUB_CFG2: now also R1701.1, U1700.22 (CFG_STRAP2); no longer C1707.22 (CFG_STRAP2)
- net HUB_CFG3: now also R1702.1, U1700.23 (CFG_STRAP3); no longer C1707.23 (CFG_STRAP3)
- net HUB_CLK: now also U1700.98 (XTALI/CLK_IN); no longer C1707.98 (XTALI/CLK_IN)
- net HUB_CORE_FB: now also C1705.2, R1706.1
- net HUB_CORE_PG: now also R1707.2; no longer L1700.2
- net HUB_CORE_SW: now also L1700.1
- net HUB_DIS5_DN: now also U1801.3 (I/O2), U1801.4 (I/O2); no longer R1850.3 (I/O2), R1850.4 (I/O2)
- net HUB_DIS5_DP: now also U1801.1 (I/O1), U1801.6 (I/O1); no longer R1850.1 (I/O1), R1850.6 (I/O1)
- net HUB_DIS6_DN: now also U1804.3 (I/O2), U1804.4 (I/O2); no longer R1851.3 (I/O2), R1851.4 (I/O2)
- net HUB_DIS6_DP: now also U1804.1 (I/O1), U1804.6 (I/O1); no longer R1851.1 (I/O1), R1851.6 (I/O1)
- net HUB_DS1_PRT_CTL: now also U1700.60 (PF17); no longer C1707.60 (PF17)
- net HUB_DS2_DN: now also U1785.2 (D1-); no longer D1805.2 (D1-)
- net HUB_DS2_DP: now also U1785.1 (D1+); no longer D1805.1 (D1+)
- net HUB_DS2_SSTX_N: now also C1723.2
- net HUB_DS2_SSTX_P: now also C1722.2
- net HUB_DS2_TX_RAW_N: now also C1723.1
- net HUB_DS2_TX_RAW_P: now also C1722.1
- net HUB_DS3_DN: now also U1745.2 (D1-); no longer D1813.2 (D1-)
- net HUB_DS3_DP: now also U1745.1 (D1+); no longer D1813.1 (D1+)
- net HUB_DS3_SSTX_N: now also C1725.2; no longer C1722.2
- net HUB_DS3_SSTX_P: now also C1724.2; no longer C1716.2
- net HUB_DS3_TX_RAW_N: now also C1725.1; no longer C1722.1
- net HUB_DS3_TX_RAW_P: now also C1724.1; no longer C1716.1
- net HUB_NON_REM: now also R1703.1, U1700.69 (SPI_CE_N/CFG_NON_REM/PF20); no longer C1707.69 (SPI_CE_N/CFG_NON_REM/PF20), R1700.1
- net HUB_PRT_CTL2: now also U1700.59 (PF16), U2405.2; no longer C1707.59 (PF16), U1780.3 (EN), U1781.6 (EN)
- net HUB_PRT_CTL3: now also U1700.58 (PF15), U2406.2; no longer C1707.58 (PF15), U1740.3 (EN), U1741.6 (EN)
- net HUB_PRT_CTL4: now also U1700.57 (PF14); no longer C1707.57 (PF14)
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Other:
- note added: "6.5A includes VBUS and VCONN. Source admission, harness loss, capacitor corners, startup and thermal behavior require qualification."
- note added: "== 6.5A USB5 converter envelope and 1.15V hub-core rail =="
- note added: "Raw OC and SYS5 veto remain active during clear; any SYS5 loss latches USB off until explicit clear."
- note added: "USB permissions reset off; fault clear is active-low and defaults high."
- note added: "USB5: external COMP 2.49k / 220n / 2.2n; include each PP5V reservoir gate state and remote cable R/L in the loop model."
- note removed: "5.5A is a system budget. Harness loss, capacitor corners, startup, load steps and thermal behavior still require qualification."
- note removed: "== 5.5A system port budget and 1.15V hub-core rail =="
- note removed: "USB5: external COMP 6.8k / 220n / 2.2n; include both local reservoirs and remote PP5V banks in the loop model."
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