File: left_io/left_io.kicad_pcb (KiCad board)
At the start: 8 copper layers, 70 x 185 mm, 260 parts, among them J190 AUX/SOLAR protected screw ter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, J21 USB-C dual-role data/PD port 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, J22 USB-C source-only data port J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, J23 USB-C source-only data port J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, J24 USB 3.0 Type-A internal heade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, J25 USB 2.0 Type-A internal heade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, Q15 SiSS4409DN 40V reverse-blocki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, Q16 SiSS4409DN 40V reverse-blocki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, Q2001 2N7002K DFP USB2 enable inver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, U14 LTC4418IUF#PBF dual-input PD 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, U1700 USB7206C-I/KDX six-port USB 3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, U1701 TPS62823DLC 3A USB7206C 1.146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, U1702 TLV803EA29 USB hub reset supe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, U1703 TPS56637RPAR VSYS to USB_PORT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, U1704 SN74LVC1G08 hub 3V3/core-PG r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, U1740 TPS2553DDBVR 1.3A USB branch, U1741 TPS25810RVCR Type-C DFP contr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, U1742 HD3SS6126RUAR USB3 orientatio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, U1743 TPD1S514-1YZR 5.9V VBUS OVP, U1745 TPD4E05U06 USB2/CC ESD, U1780 TPS2553DDBVR 1.3A USB branch, U1781 TPS25810RVCR Type-C DFP contr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, U1782 HD3SS6126RUAR USB3 orientatio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, U1783 TPD1S514-1YZR 5.9V VBUS OVP, U1785 TPD4E05U06 USB2/CC ESD, U1800 TPS2553DDBVR USB3-A VBUS bran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, U1801 USBLC6-2P6 USB3-A D+/D- ESD, U1802 TPD4E05U06 USB3-A SuperSpeed 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, U1803 TPS2553DDBVR USB2-A VBUS bran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, U1804 USBLC6-2P6 USB2-A D+/D- ESD, U2000 TUSB1142 USB 3.2 Gen 2 orient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, U2001 TPD4S201 CC and USB2 short-to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, U2002 CAT24C256 32KB private TPS257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, U2003 TS3USB30E DFP-qualified USB2 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, U2004 SN74LVC2G07 partial-power-dow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, U2005 TVS2200 22V USB VBUS surge cl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, U2006 SN74LVC1G08 DFP and attached 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, U41 TPS25751AD USB-PD DRP control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, U720 TPS26630RGER PD1 default-off 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, Y1700 25.000MHz 3.3V USB hub oscill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

Commit message: fix audit issues and move some connectors
Parts:
- added C1860: 22u 16V USB5 VCC; verify effective capacitance, Capacitor_SMD:C_1206_3216Metric, F.Cu at (35.5, 83.2)
- added C1861: 100n 50V USB5 VDDA, Capacitor_SMD:C_0603_1608Metric, F.Cu at (33.5, 83.8)
- added C1862: 220n 50V X7R USB5 COMP, Capacitor_SMD:C_0603_1608Metric, F.Cu at (34.5, 91.0)
- added C1863: 2.2n 50V C0G USB5 COMP HF, Capacitor_SMD:C_0603_1608Metric, F.Cu at (34.5, 88.5)
- added C1864: 330u 10V USB5 local reservoir; 4.3mm max height, Capacitor_Tantalum_SMD:CP_EIA-7343-43_Kemet-X, F.Cu at (50.5, 71.5)
- added C1865: 330u 10V USB5 local reservoir; 4.3mm max height, Capacitor_Tantalum_SMD:CP_EIA-7343-43_Kemet-X, F.Cu at (50.5, 77.0)
- added C1866: DNP 68u 25V input damping option, Capacitor_Tantalum_SMD:CP_EIA-7343-20_Kemet-V, F.Cu at (29.5, 66.5)
- added C1867: 100n 50V USB5 input HF, Capacitor_SMD:C_0603_1608Metric, F.Cu at (24.4, 75.5)
- added R1860: 49.9k 0.1% 10ppm USB5 RT, Resistor_SMD:R_0603_1608Metric, F.Cu at (27.2, 87.0)
- added R1861: 29.4k 1% standalone DRSS off, Resistor_SMD:R_0603_1608Metric, F.Cu at (29.3, 87.0)
- added R1862: 6.8k 1% USB5 COMP, Resistor_SMD:R_0603_1608Metric, F.Cu at (31.3, 89.0)
- added R1863: 1R USB5 bootstrap damping, Resistor_SMD:R_0603_1608Metric, F.Cu at (23.8, 79.8)
- added RS1860: 5.6mOhm 1% 0.5W USB5 current sense, ducktop2:Vishay_WSL2010_1to6m9, F.Cu at (43.5, 76.5)
- C1710: value 100n USB5 bootstrap -> 47n 25V USB5 bootstrap; footprint Capacitor_SMD:C_0603_1608Metric -> Capacitor_SMD:C_0402_1005Metric
- C1850, C1854: footprint Capacitor_SMD:C_1206_3216Metric -> Capacitor_SMD:C_0805_2012Metric
- C2146: footprint Capacitor_SMD:CP_Elec_6.3x5.8 -> Capacitor_SMD:CP_Elec_6.3x7.7
- L1701: value 3.3uH >=9A USB port buck -> 6.8uH 12.8A Isat30 / 6.8A Irms20
- R1710: value 169k 1% USB5 EN top -> 100k USB5 switched-3V3 EN top
- R1711: value 36.1k 1% USB5 EN bottom -> 100k USB5 EN bottom
- R1712: value 74.3k 0.1% USB5 FB top -> 54.9k 0.1% 10ppm USB5 FB top
- R1713: value 10.0k 0.1% USB5 FB bottom -> 10.2k 0.1% 10ppm USB5 FB bottom
- R2080: value 887k 0.1% 15V eFuse UV/OV top -> 8.87k 0.1% 10ppm 15/20V eFuse UV/OV top
- R2081: value 27.4k 0.1% 15V eFuse UV/OV middle -> 562R 0.1% 10ppm 15/20V eFuse UV/OV middle
- R2082: value 68.1k 0.1% 15V eFuse UV/OV bottom -> 511R 0.1% 10ppm 15/20V eFuse UV/OV bottom
- R2140: value 1.00M 0.1% 15V UV top -> 1.00M 0.1% 25ppm 15/20V UV top
- R2141: value 19.6k 0.1% 15V window middle -> 35.7k 0.1% 25ppm 15/20V window middle
- R2142: value 63.4k 0.1% 15V OV bottom -> 47.5k 0.1% 25ppm 15/20V OV bottom
- U1703: value TPS56637RPAR VSYS to USB_PORT_5V 5.06V nominal -> LM706A0RRXR USB5 5.106V; 5.5A system limit; footprint ducktop2:Texas_RPA0010A_VQFN-HR-10_3x3mm -> ducktop2:Texas_RRX0029B_VQFN-29_6x6mm
- moved C1714 85.0 mm to (46.5, 83.0)
- moved R1712 66.6 mm to (38.5, 83.0), turned to 180 degrees
- moved R1713 59.9 mm to (37.0, 87.5)
- moved C1712 59.1 mm to (21.0, 78.5), turned to -90 degrees
- moved U1703 54.9 mm to (29.0, 80.0)
- moved C1710 52.7 mm to (23.0, 81.4), turned to -90 degrees
- moved C1713 50.4 mm to (28.7, 75.4), turned to 0 degrees
- moved L1701 49.5 mm to (37.0, 76.5)
- moved C1711 37.3 mm to (28.7, 72.9), turned to 0 degrees
- moved R1711 36.9 mm to (24.5, 89.3)
- moved C1715 26.8 mm to (51.5, 82.2), turned to 0 degrees
- moved C1751 14.4 mm to (21.2, 85.5)
- moved R1740 14.4 mm to (16.3, 80.7)
- moved U1740 14.4 mm to (16.3, 84.3)
- moved U1743 14.4 mm to (24.0, 85.5)
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Connections:
- C1710 pad 1: /USB Hub + Ports/USB5_BOOT -> /USB Hub + Ports/USB5_BOOT_C
- C1710 pad 2: /USB Hub + Ports/USB5_SW -> /USB Hub + Ports/USB5_SW_BOOT
- J21 pad A8: unconnected-(J21-SBU1-PadA8) -> (no net)
- J21 pad B8: unconnected-(J21-SBU2-PadB8) -> (no net)
- J22 pad A8: unconnected-(J22-SBU1-PadA8) -> (no net)
- J22 pad B8: unconnected-(J22-SBU2-PadB8) -> (no net)
- J23 pad A8: unconnected-(J23-SBU1-PadA8) -> (no net)
- J23 pad B8: unconnected-(J23-SBU2-PadB8) -> (no net)
- L1701 pad 2: /USB_PORT_5V -> /USB Hub + Ports/USB5_PRE_SENSE
- R1710 pad 1: /VSYS -> /SYS_3V3
- U14 pad 11: unconnected-(U14-G2-Pad11) -> (no net)
- U14 pad 7: unconnected-(U14-~{VALID2}-Pad7) -> (no net)
- U14 pad 9: unconnected-(U14-CAS-Pad9) -> (no net)
- U1700 pad 10: unconnected-(U1700B-RXDP1-Pad10) -> (no net)
- U1700 pad 11: unconnected-(U1700B-RXDM1-Pad11) -> (no net)
- U1700 pad 12: unconnected-(U1700B-NC-Pad12) -> (no net)
- U1700 pad 13: unconnected-(U1700B-NC-Pad13) -> (no net)
- U1700 pad 3: unconnected-(U1700A-PF31-Pad3) -> (no net)
- U1700 pad 36: unconnected-(U1700C-TXDP4-Pad36) -> (no net)
- U1700 pad 37: unconnected-(U1700C-TXDM4-Pad37) -> (no net)
- U1700 pad 39: unconnected-(U1700C-RXDP4-Pad39) -> (no net)
- U1700 pad 4: unconnected-(U1700A-NC-Pad4) -> (no net)
- U1700 pad 40: unconnected-(U1700C-RXDM4-Pad40) -> (no net)
- U1700 pad 44: unconnected-(U1700A-PF3-Pad44) -> (no net)
- U1700 pad 45: unconnected-(U1700A-PF4-Pad45) -> (no net)
- U1700 pad 46: unconnected-(U1700A-PF5-Pad46) -> (no net)
- U1700 pad 47: unconnected-(U1700A-PF6-Pad47) -> (no net)
- U1700 pad 48: unconnected-(U1700A-PF7-Pad48) -> (no net)
- U1700 pad 49: unconnected-(U1700A-PF8-Pad49) -> (no net)
- U1700 pad 50: unconnected-(U1700A-PF9-Pad50) -> (no net)
- U1700 pad 51: unconnected-(U1700A-PF10-Pad51) -> (no net)
- U1700 pad 52: unconnected-(U1700A-PF11-Pad52) -> (no net)
- U1700 pad 54: unconnected-(U1700A-PF12-Pad54) -> (no net)
- U1700 pad 56: unconnected-(U1700A-PF13-Pad56) -> (no net)
- U1700 pad 61: unconnected-(U1700A-PF18-Pad61) -> (no net)
- U1700 pad 66: unconnected-(U1700A-PF19-Pad66) -> (no net)
- U1700 pad 7: unconnected-(U1700B-TXDP1-Pad7) -> (no net)
- U1700 pad 74: unconnected-(U1700A-PF29-Pad74) -> (no net)
- U1700 pad 75: unconnected-(U1700A-PF26-Pad75) -> (no net)
- U1700 pad 76: unconnected-(U1700A-PF27-Pad76) -> (no net)
- U1700 pad 77: unconnected-(U1700A-PF28-Pad77) -> (no net)
- U1700 pad 8: unconnected-(U1700B-TXDM1-Pad8) -> (no net)
- U1700 pad 80: unconnected-(U1700A-NC-Pad80) -> (no net)
- U1700 pad 96: unconnected-(U1700A-ATEST-Pad96) -> (no net)
- U1700 pad 97: unconnected-(U1700A-XTALO-Pad97) -> (no net)
- U1701 pad 4: unconnected-(U1701-NC-Pad4) -> (no net)
- U1703 pad 1: /USB Hub + Ports/USB5_EN -> /VSYS
- U1703 pad 10: GND -> (no net)
- U1703 pad 2: /USB Hub + Ports/USB5_FB -> /VSYS
- U1703 pad 3: GND -> /VSYS
- U1703 pad 4: /USB Hub + Ports/USB5_PG -> /USB Hub + Ports/USB5_BOOT
- U1703 pad 5: unconnected-(U1703-NC-Pad5) -> /USB Hub + Ports/USB5_SW_BOOT
- U1703 pad 6: /USB Hub + Ports/USB5_SW -> GND
- U1703 pad 7: /USB Hub + Ports/USB5_BOOT -> /USB Hub + Ports/USB5_PG
- U1703 pad 8: /VSYS -> GND
- U1703 pad 9: GND -> /USB Hub + Ports/USB5_EN
- U1741 pad 16: unconnected-(U1741-~{DEBUG}-Pad16) -> (no net)
- U1741 pad 17: unconnected-(U1741-~{AUDIO}-Pad17) -> (no net)
- U1741 pad 19: unconnected-(U1741-~{UFP}-Pad19) -> (no net)
- U1741 pad 20: unconnected-(U1741-~{LD_DET}-Pad20) -> (no net)
- U1742 pad 1: unconnected-(U1742-NC-Pad1) -> (no net)
- U1742 pad 18: unconnected-(U1742-NC-Pad18) -> (no net)
- U1742 pad 2: unconnected-(U1742-NC-Pad2) -> (no net)
- U1742 pad 3: unconnected-(U1742-NC-Pad3) -> (no net)
- U1742 pad 31: unconnected-(U1742-HSB(p)-Pad31) -> (no net)
- U1742 pad 32: unconnected-(U1742-HSB(n)-Pad32) -> (no net)
- U1742 pad 33: unconnected-(U1742-HSC(p)-Pad33) -> (no net)
- U1742 pad 34: unconnected-(U1742-HSC(n)-Pad34) -> (no net)
- U1742 pad 35: unconnected-(U1742-NC-Pad35) -> (no net)
- U1742 pad 36: unconnected-(U1742-NC-Pad36) -> (no net)
- U1742 pad 37: unconnected-(U1742-NC-Pad37) -> (no net)
- U1742 pad 38: unconnected-(U1742-NC-Pad38) -> (no net)
- U1742 pad 39: unconnected-(U1742-NC-Pad39) -> (no net)
- U1742 pad 4: unconnected-(U1742-NC-Pad4) -> (no net)
- U1742 pad 40: unconnected-(U1742-NC-Pad40) -> (no net)
- U1742 pad 41: unconnected-(U1742-NC-Pad41) -> (no net)
- U1742 pad 42: unconnected-(U1742-NC-Pad42) -> (no net)
- U1742 pad 5: unconnected-(U1742-NC-Pad5) -> (no net)
- U1742 pad 7: unconnected-(U1742-HSA(n)-Pad7) -> (no net)
- U1742 pad 8: unconnected-(U1742-HSA(p)-Pad8) -> (no net)
- U1745 pad 10: unconnected-(U1745-NC-Pad10) -> (no net)
- U1745 pad 6: unconnected-(U1745-NC-Pad6) -> (no net)
- U1745 pad 7: unconnected-(U1745-NC-Pad7) -> (no net)
- U1745 pad 9: unconnected-(U1745-NC-Pad9) -> (no net)
- U1781 pad 16: unconnected-(U1781-~{DEBUG}-Pad16) -> (no net)
- U1781 pad 17: unconnected-(U1781-~{AUDIO}-Pad17) -> (no net)
- U1781 pad 19: unconnected-(U1781-~{UFP}-Pad19) -> (no net)
- U1781 pad 20: unconnected-(U1781-~{LD_DET}-Pad20) -> (no net)
- U1782 pad 1: unconnected-(U1782-NC-Pad1) -> (no net)
- U1782 pad 18: unconnected-(U1782-NC-Pad18) -> (no net)
- U1782 pad 2: unconnected-(U1782-NC-Pad2) -> (no net)
- U1782 pad 3: unconnected-(U1782-NC-Pad3) -> (no net)
- U1782 pad 31: unconnected-(U1782-HSB(p)-Pad31) -> (no net)
- U1782 pad 32: unconnected-(U1782-HSB(n)-Pad32) -> (no net)
- U1782 pad 33: unconnected-(U1782-HSC(p)-Pad33) -> (no net)
- U1782 pad 34: unconnected-(U1782-HSC(n)-Pad34) -> (no net)
- U1782 pad 35: unconnected-(U1782-NC-Pad35) -> (no net)
- U1782 pad 36: unconnected-(U1782-NC-Pad36) -> (no net)
- U1782 pad 37: unconnected-(U1782-NC-Pad37) -> (no net)
- U1782 pad 38: unconnected-(U1782-NC-Pad38) -> (no net)
- U1782 pad 39: unconnected-(U1782-NC-Pad39) -> (no net)
- U1782 pad 4: unconnected-(U1782-NC-Pad4) -> (no net)
- U1782 pad 40: unconnected-(U1782-NC-Pad40) -> (no net)
- U1782 pad 41: unconnected-(U1782-NC-Pad41) -> (no net)
- U1782 pad 42: unconnected-(U1782-NC-Pad42) -> (no net)
- U1782 pad 5: unconnected-(U1782-NC-Pad5) -> (no net)
- U1782 pad 7: unconnected-(U1782-HSA(n)-Pad7) -> (no net)
- U1782 pad 8: unconnected-(U1782-HSA(p)-Pad8) -> (no net)
- U1785 pad 10: unconnected-(U1785-NC-Pad10) -> (no net)
- U1785 pad 6: unconnected-(U1785-NC-Pad6) -> (no net)
- U1785 pad 7: unconnected-(U1785-NC-Pad7) -> (no net)
- U1785 pad 9: unconnected-(U1785-NC-Pad9) -> (no net)
- U1800 pad 4: unconnected-(U1800-~{FAULT}-Pad4) -> (no net)
- U1801 pad 5: GND -> /USB Hub + Ports/J24_5V_PRE
- U1802 pad 10: unconnected-(U1802-NC-Pad10) -> (no net)
- U1802 pad 6: unconnected-(U1802-NC-Pad6) -> (no net)
- U1802 pad 7: unconnected-(U1802-NC-Pad7) -> (no net)
- U1802 pad 9: unconnected-(U1802-NC-Pad9) -> (no net)
- U1803 pad 4: unconnected-(U1803-~{FAULT}-Pad4) -> (no net)
- U1804 pad 5: GND -> /USB Hub + Ports/J25_5V_PRE
- U2000 pad 10: unconnected-(U2000-RSVD2-Pad10) -> (no net)
- U2000 pad 11: unconnected-(U2000-NC-Pad11) -> (no net)
- U2000 pad 12: unconnected-(U2000-RSVD3-Pad12) -> (no net)
- U2000 pad 13: unconnected-(U2000-RSVD4-Pad13) -> (no net)
- U2000 pad 23: unconnected-(U2000-AEQCFG-Pad23) -> (no net)
- U2000 pad 24: unconnected-(U2000-NC-Pad24) -> (no net)
- U2000 pad 25: unconnected-(U2000-NC-Pad25) -> (no net)
- U2000 pad 29: unconnected-(U2000-CEQ1-Pad29) -> (no net)
- U2000 pad 32: unconnected-(U2000-NC-Pad32) -> (no net)
- U2000 pad 35: unconnected-(U2000-SSEQ0/A0-Pad35) -> (no net)
- U2000 pad 38: unconnected-(U2000-CEQ0-Pad38) -> (no net)
- U2000 pad 5: unconnected-(U2000-NC-Pad5) -> (no net)
- U2000 pad 7: unconnected-(U2000-TESTOUT1-Pad7) -> (no net)
- U2000 pad 8: unconnected-(U2000-TESTOUT2-Pad8) -> (no net)
- U2000 pad 9: unconnected-(U2000-RSVD1-Pad9) -> (no net)
- U2001 pad 16: unconnected-(U2001-NC-Pad16) -> (no net)
- U2001 pad 17: unconnected-(U2001-NC-Pad17) -> (no net)
- U2001 pad 19: unconnected-(U2001-NC-Pad19) -> (no net)
- U2001 pad 20: unconnected-(U2001-NC-Pad20) -> (no net)
- U2003 pad 3: unconnected-(U2003-D2+-Pad3) -> (no net)
- U2003 pad 7: unconnected-(U2003-D2--Pad7) -> (no net)
- U720 pad 13: unconnected-(U720-IMON-Pad13) -> (no net)
- U720 pad 16: unconnected-(U720-PGOOD-Pad16) -> (no net)
- U720 pad 19: unconnected-(U720-NC-Pad19) -> (no net)
- U720 pad 20: unconnected-(U720-NC-Pad20) -> (no net)
- U720 pad 21: unconnected-(U720-NC-Pad21) -> (no net)
- U720 pad 22: unconnected-(U720-NC-Pad22) -> (no net)
- U720 pad 23: unconnected-(U720-NC-Pad23) -> (no net)
- U720 pad 24: unconnected-(U720-NC-Pad24) -> (no net)
- U720 pad 3: unconnected-(U720-B_GATE-Pad3) -> (no net)
- U720 pad 4: unconnected-(U720-DRV-Pad4) -> (no net)
Routing:
- net /USB Hub + Ports/J23_TX2_N: track 11.4 -> 20.1 mm, vias 0 -> 2
- net /USB Hub + Ports/J23_RX1_P: track 12.2 -> 20.2 mm, vias 0 -> 2
- net /USB Hub + Ports/J23_RX1_N: track 13.4 -> 20.2 mm, vias 0 -> 2
- net /USB Hub + Ports/J23_TX2_P: track 14.1 -> 20.1 mm, vias 0 -> 2
- net /USB Hub + Ports/J23_TX1_P: track 6.09 -> 10.9 mm, vias 0 -> 2
- net GND: track 9.59 -> 6.35 mm, vias 0 -> 14
- net /USB Hub + Ports/J23_TX1_N: track 8.70 -> 10.9 mm, vias 0 -> 2
- net /USB Hub + Ports/HUB_DIS5_TX_N: track 1.35 -> 0.00 mm
- net /USB Hub + Ports/HUB_DIS5_DP: track 3.91 -> 4.53 mm, vias 0 -> 2
- net /USB Hub + Ports/HUB_DIS5_DN: track 3.87 -> 4.45 mm, vias 0 -> 2
- net /USB Hub + Ports/J23_RX2_P: track 9.02 -> 9.34 mm, vias 0 -> 2
- net /USB Hub + Ports/J23_RX2_N: track 9.58 -> 9.38 mm, vias 0 -> 2
- net /USB Hub + Ports/HUB_DIS6_DP: track 4.56 -> 4.61 mm, vias 0 -> 2
- net /USB Hub + Ports/HUB_DIS6_DN: track 4.52 -> 4.51 mm, vias 0 -> 2
- added copper zone on In1.Cu, net GND
- added copper zone on In3.Cu, net GND
- added copper zone on In6.Cu, net GND

Commit message: fix more power stuff and update the left board
Parts:
- added C1868: 22u 25V USB5 output; TI characterized part, Capacitor_SMD:C_1210_3225Metric, F.Cu at (43.0, 89.5)
- added C1869: 22u 25V USB5 output; TI characterized part, Capacitor_SMD:C_1210_3225Metric, F.Cu at (46.2, 90.8)
- added C2400: 100n, Capacitor_SMD:C_0603_1608Metric, F.Cu at (50.0, 135.0)
- added C2401: 100n, Capacitor_SMD:C_0603_1608Metric, F.Cu at (40.1, 94.0)
- added C2402: 100n, Capacitor_SMD:C_0603_1608Metric, F.Cu at (39.0, 98.2)
- added C2403: 1u, Capacitor_SMD:C_0805_2012Metric, F.Cu at (33.1, 35.5)
- added C2405: 100n, Capacitor_SMD:C_0603_1608Metric, F.Cu at (26.1, 36.3)
- added C2406: 100n, Capacitor_SMD:C_0603_1608Metric, F.Cu at (20.1, 89.8)
- added C2407: 100n, Capacitor_SMD:C_0603_1608Metric, F.Cu at (32.1, 125.8)
- added C2408: 100n, Capacitor_SMD:C_0603_1608Metric, F.Cu at (33.1, 137.8)
- added C2410: 100n, Capacitor_SMD:C_0603_1608Metric, F.Cu at (40.6, 107.0)
- added C2411: 100n, Capacitor_SMD:C_0603_1608Metric, F.Cu at (44.1, 100.8)
- added C2413: 4.7n C0G PP5V slew, Capacitor_SMD:C_0603_1608Metric, F.Cu at (33.6, 33.6)
- added C2415: 100n, Capacitor_SMD:C_0603_1608Metric, F.Cu at (47.6, 111.5)
- added J2431: left power loom, straight-numbered, Connector_Molex:Molex_Micro-Fit_3.0_43045-1212_2x06_P3.00mm_Vertical, F.Cu at (53.0, 59.5)
- added J2434: USB5 direct power loom, ducktop2:AMASS_XT30PW-F30_G_Y, F.Cu at (35.0, 150.0)
- added J2440: main ground strap, Connector_Wire:SolderWirePad_1x01_SMD_5x10mm, F.Cu at (62.5, 12.7)
- added J2442: main ground strap, Connector_Wire:SolderWirePad_1x01_SMD_5x10mm, F.Cu at (62.5, 70.0)
- added R2400: 10k, Resistor_SMD:R_0603_1608Metric, F.Cu at (44.9, 106.5)
- added R2401: 10k, Resistor_SMD:R_0603_1608Metric, F.Cu at (37.5, 93.5)
- added R2402: 10k, Resistor_SMD:R_0603_1608Metric, F.Cu at (40.5, 100.8)
- added R2403: 100k, Resistor_SMD:R_0603_1608Metric, F.Cu at (36.0, 32.9)
- added R2405: 100k, Resistor_SMD:R_0603_1608Metric, F.Cu at (23.9, 36.3)
- added R2406: 100k, Resistor_SMD:R_0603_1608Metric, F.Cu at (17.9, 89.8)
- added R2407: 100k, Resistor_SMD:R_0603_1608Metric, F.Cu at (42.6, 141.3)
- added R2408: 100k, Resistor_SMD:R_0603_1608Metric, F.Cu at (42.6, 142.9)
- added R2410: 100k, Resistor_SMD:R_0603_1608Metric, F.Cu at (42.6, 139.4)
- added R2412: 10k, Resistor_SMD:R_0603_1608Metric, F.Cu at (53.4, 141.6)
- added R2413: 10k, Resistor_SMD:R_0603_1608Metric, F.Cu at (35.7, 37.4)
- added R2420: 100k, Resistor_SMD:R_0603_1608Metric, F.Cu at (42.6, 137.7)
- added R2421: 100k, Resistor_SMD:R_0603_1608Metric, F.Cu at (33.7, 101.2)
- added R2422: 100k, Resistor_SMD:R_0603_1608Metric, F.Cu at (42.1, 109.3)
- added R2423: 100k, Resistor_SMD:R_0603_1608Metric, F.Cu at (53.4, 143.1)
- added R2424: 12.7k 1%, Resistor_SMD:R_0603_1608Metric, F.Cu at (52.6, 136.7)
- added R2425: 12.7k 1%, Resistor_SMD:R_0603_1608Metric, F.Cu at (54.9, 137.3)
- added R2426: 100k, Resistor_SMD:R_0603_1608Metric, F.Cu at (40.4, 112.5)
- added R2427: 100k, Resistor_SMD:R_0603_1608Metric, F.Cu at (53.4, 139.0)
- added R2429: 10k, Resistor_SMD:R_0603_1608Metric, F.Cu at (39.0, 103.8)
- added R2440: 0.33, Resistor_SMD:R_0603_1608Metric, F.Cu at (59.1, 26.5)
- added R2441: 0.33, Resistor_SMD:R_0603_1608Metric, F.Cu at (59.1, 42.5)
- added RS1861: 10mOhm 1% 1W USB5 sense; parallel pair gives 5mOhm, ducktop2:Panasonic_ERJ8CW_10to16m, F.Cu at (46.0, 84.5)
- added U2400: TCA9539PWR USB permissions @0x76, Package_SO:TSSOP-24_4.4x7.8mm_P0.65mm, F.Cu at (48.0, 140.0)
- added U2401: INA226AIDGSR USB5 monitor @0x40, Package_SO:TSSOP-10_3x3mm_P0.5mm, F.Cu at (37.5, 91.0)
- added U2402: SN74LVC1G74DCUR USB fault latch, ducktop2:TI_DCU0008A_VSSOP8, F.Cu at (37.5, 101.0)
- added U2403: TPS22992SRXNR J21 PP5V gate, ducktop2:Texas_RXN0008A_WQFN-HR-8_1.25x1.25mm, F.Cu at (36.0, 35.5)
- added U2405: SN74LVC1G08DBVR J22 source permission, Package_TO_SOT_SMD:SOT-23-5, F.Cu at (25.0, 39.5)
- added U2406: SN74LVC1G08DBVR J23 source permission, Package_TO_SOT_SMD:SOT-23-5, F.Cu at (19.0, 93.0)
- added U2407: SN74LVC1G08DBVR J24 source permission, Package_TO_SOT_SMD:SOT-23-5, F.Cu at (31.0, 129.0)
- added U2408: SN74LVC1G08DBVR J25 source permission, Package_TO_SOT_SMD:SOT-23-5, F.Cu at (32.0, 141.0)
- added U2410: SN74LVC1G11DCKR USB5 permit AND, Package_TO_SOT_SMD:SOT-363_SC-70-6, F.Cu at (37.5, 107.0)
- added U2411: SN74LVC1G08DBVR raw fault veto, Package_TO_SOT_SMD:SOT-23-5, F.Cu at (43.0, 104.0)
- added U2413: SN74LVC1G08DBVR raw OC and SYS5 veto, Package_TO_SOT_SMD:SOT-23-5, F.Cu at (44.0, 112.5)
- C1714, C1715: value 22u 10V USB5 output -> 22u 25V USB5 output; TI characterized part
- C1860: value 22u 16V USB5 VCC; verify effective capacitance -> 22u 25V USB5 VCC; effective minimum 4.7u; footprint Capacitor_SMD:C_1206_3216Metric -> Capacitor_SMD:C_1210_3225Metric
- FPC101: value FH41-68S-0.5SH (FPC-1) -> Molex5039084120 signal cable; footprint ducktop2:Hirose_FH41-68S-0.5SH_1x68_1MP_1SH_P0.5mm_Horizontal -> ducktop2:Molex_5039084120_1x41_P0.50mm_Horizontal
- L1701: value 6.8uH 12.8A Isat30 / 6.8A Irms20 -> 6.8uH 18.4A Isat30 / 10.9A Irms20; footprint Inductor_SMD:L_Coilcraft_XAL7070-XXX -> ducktop2:Coilcraft_XGL1060
- R1705: value 91.0k 1% core FB top -> 91.0k 0.02% 5ppm core FB top
- R1706: value 100k 1% core FB bottom -> 100k 0.02% 5ppm core FB bottom
- R1710: value 100k USB5 switched-3V3 EN top -> 100k USB5 hardware-qualified EN top
- R1712: value 54.9k 0.1% 10ppm USB5 FB top -> 55.6k 0.02% 5ppm USB5 FB top
- R1713: value 10.2k 0.1% 10ppm USB5 FB bottom -> 10.2k 0.02% 5ppm USB5 FB bottom
- R1740, R1780: value 20.0k 1% TPS2553 1.3A ILIM -> 19.1k 1% TPS2553 VBUS plus VCONN ILIM
- R1860: value 49.9k 0.1% 10ppm USB5 RT -> 22.1k 0.02% 5ppm USB5 RT
- R1862: value 6.8k 1% USB5 COMP -> 2.49k 0.02% 5ppm USB5 COMP
- R2080: value 8.87k 0.1% 10ppm 15/20V eFuse UV/OV top -> 8.87k 0.02% 5ppm 15/20V eFuse UV/OV top
- R2081: value 562R 0.1% 10ppm 15/20V eFuse UV/OV middle -> 562R 0.02% 5ppm 15/20V eFuse UV/OV middle
- R2082: value 511R 0.1% 10ppm 15/20V eFuse UV/OV bottom -> 511R 0.02% 5ppm 15/20V eFuse UV/OV bottom
- R2141: value 35.7k 0.1% 25ppm 15/20V window middle -> 35.7k 0.02% 5ppm 15/20V window middle
- R2142: value 47.5k 0.1% 25ppm 15/20V OV bottom -> 47.5k 0.02% 5ppm 15/20V OV bottom
- RS1860: value 5.6mOhm 1% 0.5W USB5 current sense -> 10mOhm 1% 1W USB5 sense; parallel pair gives 5mOhm; footprint ducktop2:Vishay_WSL2010_1to6m9 -> ducktop2:Panasonic_ERJ8CW_10to16m
- U1703: value LM706A0RRXR USB5 5.106V; 5.5A system limit -> LM706A0RRXR USB5 5.161V; 6.5A design envelope
- moved D2107 108.7 mm to (10.7, 50.5)
- moved D2103 105.6 mm to (5.17, 53.2), turned to 180 degrees
- moved D2105 105.4 mm to (9.41, 45.5), turned to 90 degrees
- moved R2085 103.6 mm to (50.4, 32.2), turned to 90 degrees
- moved C2019 102.7 mm to (56.4, 51.2), turned to 90 degrees
- moved D2102 99.1 mm to (9.41, 50.8), turned to -90 degrees
- moved R2014 98.7 mm to (29.8, 39.4), turned to -90 degrees
- moved FPC101 58.2 mm to (61.2, 34.5)
- moved R2005 57.3 mm to (26.6, 25.7)
- moved R1723 52.1 mm to (63.1, 90.5)
- moved R2009 52.1 mm to (18.0, 33.4), turned to 0 degrees
- moved R1721 45.5 mm to (66.1, 92.8)
- moved R1704 42.7 mm to (62.4, 97.7), turned to -90 degrees
- moved D1800 40.3 mm to (12.5, 45.2), turned to 180 degrees
- moved R1741 38.3 mm to (20.3, 70.6), turned to -90 degrees
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Connections:
- C2025 pad 1: /USB_PORT_5V -> /PD1 Dual-Role/PD1_PP5V_GATED
- C2026 pad 1: /USB_PORT_5V -> /PD1 Dual-Role/PD1_PP5V_GATED
- C2027 pad 1: /USB_PORT_5V -> /PD1 Dual-Role/PD1_PP5V_GATED
- FPC101 pad 1: /VSYS -> GND
- FPC101 pad 10: /USB_PORT_5V -> GND
- FPC101 pad 11: /USB_PORT_5V -> /USBC2_SSTX_P
- FPC101 pad 12: /USB_PORT_5V -> /USBC2_SSTX_N
- FPC101 pad 14: /SYS_3V3 -> /USBC1_DP
- FPC101 pad 15: /SYS_3V3 -> /USBC1_DN
- FPC101 pad 16: /MCU_3V3 -> GND
- FPC101 pad 17: /PD1_VBUS_RAW -> /USBC2_DP
- FPC101 pad 18: /PD1_VBUS_RAW -> /USBC2_DN
- FPC101 pad 19: /PD1_VBUS_RAW -> GND
- FPC101 pad 2: /VSYS -> /USBC1_SSRX_P
- FPC101 pad 20: /PD1_VBUS_RAW -> /HUB_DS1_DP
- FPC101 pad 21: /PD1_VBUS_RAW -> /HUB_DS1_DN
- FPC101 pad 22: /PD1_VBUS_RAW -> GND
- FPC101 pad 23: /USB_PD_SELECTED -> /HUB_DS4_DP
- FPC101 pad 24: /USB_PD_SELECTED -> /HUB_DS4_DN
- FPC101 pad 25: /USB_PD_SELECTED -> GND
- FPC101 pad 26: /USB_PD_SELECTED -> /PD1_I2C_SCL
- FPC101 pad 27: /USB_PD_SELECTED -> /PD1_I2C_SDA
- FPC101 pad 28: /USB_PD_SELECTED -> /PD1_TCPC_IRQ_N
- FPC101 pad 29: /AUX_DC_RAW -> GND
- FPC101 pad 3: /VSYS -> /USBC1_SSRX_N
- FPC101 pad 30: /AUX_DC_RAW -> /PD1_PATH_EN
- FPC101 pad 31: /AUX_DC_RAW -> /PD1_VALID_N
- FPC101 pad 32: /AUX_DC_RAW -> /PD1_EFUSE_FAULT_N
- FPC101 pad 33: /AUX_DC_RAW -> GND
- FPC101 pad 34: /AUX_DC_RAW -> /PD_PROTECT_FAULT_N
- FPC101 pad 35: GND -> /SERVICE_MUX_RESET_N
- FPC101 pad 36: GND -> /PD2_SOURCE_PG
- FPC101 pad 38: /INTERNAL_USB_VBUS_VALID -> /USB_J11_PERMIT
- FPC101 pad 39: /PD1_I2C_SCL -> /USB_J12_PERMIT
- FPC101 pad 4: /VSYS -> GND
- FPC101 pad 40: /PD1_I2C_SDA -> /HUB_PRT_CTL4
- FPC101 pad 41: /PD1_TCPC_IRQ_N -> /INTERNAL_USB_VBUS_VALID
- FPC101 pad 5: /VSYS -> /USBC1_SSTX_P
- FPC101 pad 6: /VSYS -> /USBC1_SSTX_N
- FPC101 pad 8: GND -> /USBC2_SSRX_P
- FPC101 pad 9: /USB_PORT_5V -> /USBC2_SSRX_N
- FPC101 pad SH: GND -> /FPC-1 (to Center)/FPC101_SHELL
- R1710 pad 1: /SYS_3V3 -> /USB Hub + Ports/USB5_HW_ENABLE
- U1740 pad 3: /USB Hub + Ports/HUB_PRT_CTL3 -> /USB Hub + Ports/USB_J23_SWITCH_EN
- U1741 pad 6: /USB Hub + Ports/HUB_PRT_CTL3 -> /USB Hub + Ports/USB_J23_SWITCH_EN
- U1780 pad 3: /USB Hub + Ports/HUB_PRT_CTL2 -> /USB Hub + Ports/USB_J22_SWITCH_EN
- U1781 pad 6: /USB Hub + Ports/HUB_PRT_CTL2 -> /USB Hub + Ports/USB_J22_SWITCH_EN
- U1800 pad 3: /INTERNAL_USB_VBUS_VALID -> /USB Hub + Ports/USB_J24_SWITCH_EN
- U1803 pad 3: /INTERNAL_USB_VBUS_VALID -> /USB Hub + Ports/USB_J25_SWITCH_EN
- U41 pad 34: /USB_PORT_5V -> /PD1 Dual-Role/PD1_PP5V_GATED

Commit message: work on the power redesign and case
Parts:
- added J2451: left power rails, ducktop2:WAGO_2060_453_SMD, F.Cu at (55.5, 129.2)
- added J2461: left power return, ducktop2:WAGO_2060_451_SMD, F.Cu at (62.5, 75.2)
- J2431: value left power loom, straight-numbered -> left power rails; footprint Connector_Molex:Molex_Micro-Fit_3.0_43045-1212_2x06_P3.00mm_Vertical -> ducktop2:WAGO_2060_453_SMD
- moved J2431 6.08 mm to (47.0, 60.8)
- moved C1715 6.01 mm to (51.8, 77.0)
- moved C2400 4.18 mm to (53.9, 136.5), turned to 0 degrees
- moved R1750 3.91 mm to (36.8, 62.3)
- moved R2424 3.78 mm to (56.4, 137.2)
- moved R2425 3.05 mm to (56.6, 139.8)
