File: left_io/left_fpc.kicad_sch (KiCad schematic)
At the start: 7 parts, among them J2431 left power loom, straight-num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, J2434 USB5 direct power loom, J2440 main ground strap, J2442 main ground strap

Commit message: work on the power redesign and case
Parts:
- added J2451: left power rails, ducktop2:WAGO_2060_453_SMD, symbol Connector_Generic:Conn_01x03
- added J2461: left power return, ducktop2:WAGO_2060_451_SMD, symbol Connector_Generic:Conn_01x01
- J2431: value left power loom, straight-numbered -> left power rails; footprint Connector_Molex:Molex_Micro-Fit_3.0_43045-1212_2x06_P3.00mm_Vertical -> ducktop2:WAGO_2060_453_SMD; symbol Connector_Generic:Conn_02x06_Odd_Even -> Connector_Generic:Conn_01x03; Assembly (none) -> strip 7..9 mm; hold the button to insert or remove stranded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; Contacts 43030-0038 tin 18 AWG -> (none); CurrentRatingBasis PS-43045 R; use 12-circuit 18 AWG 5.5 A reference screen; a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 -> 9 A IEC and UL; the 10 A ground-cut screen requires both se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; HarnessPinOrder pin n to pin n; continuity and isolation test every conduct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 -> match rail names in the harness drawing; each three-pole gr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; HarnessWireLength 90..100 mm between crimp barrels, including tolerance -> (none); MPN 43045-1212 -> 2060-453/998-404; Manufacturer Molex -> WAGO; MatedHeight 17.64 mm connector body; current 90..100 mm wire poses requ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 -> 4.5 mm terminal body; wire and release-tool envelopes are s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; MatingHousing 43025-1200 -> (none); ResistanceAcceptance termination <=45 mOhm hot/aged; wire <=30 mOhm/m hot; each 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 -> (none); ReturnAcceptance (none) -> remaining complete braid <=1 mOhm; each return wire >=0.12 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; Wire Alpha Wire 3253 UL1061 18 AWG tinned stranded -> Alpha 6715, 18 AWG 16/30 tinned copper; no ferrule
- J2434: CurrentRatingBasis AMASS 2025V0: 20 A at up to 85 K rise; project return design 8 A, qualification <=80 C -> AMASS 2025V0: 20 A at up to 85 K rise; project return design 10 A with 16 AWG wire, qualification <=80 C; MatedEnvelope 23.10 x 13.60 x 5.75 mm conservative; reserve sleeve and 18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 -> 23.10 x 13.60 x 5.75 mm conservative; reserve sleeve and 10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; Wire Alpha 5857 RD005/BK005; 18 AWG 19/30 silver-plated copper, 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 -> Alpha 6716 RD005/BK005; 16 AWG 26/30 tinned copper, mPPE
Connections:
- net AUX_DC_RAW: now also J2451.1 (Pin_1); no longer J2431.4 (Pin_4)
- net GND: now also J2461.1 (Pin_1); no longer J2431.10 (Pin_10), J2431.11 (Pin_11), J2431.12 (Pin_12), J2431.7 (Pin_7), J2431.8 (Pin_8), J2431.9 (Pin_9)
- net MCU_3V3: now also J2451.3 (Pin_3); no longer J2431.6 (Pin_6)
- net SYS_3V3: now also J2451.2 (Pin_2); no longer J2431.5 (Pin_5)

Commit message: rework the board placement and fix more power stuff
Connections:
- net PD1_EFUSE_FAULT_N renamed PD1_EFUSE_PG
Changed lines of the file:
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@@
   (effects (font (size 1.27 1.27)) (justify right bottom))
 )
-(hierarchical_label "PD1_EFUSE_FAULT_N"
+(hierarchical_label "PD1_EFUSE_PG"
   (shape bidirectional)
   (at 54.61 378.46 180)
