File: right_io/right_io.kicad_pcb (KiCad board)
At the start: 8 copper layers, 58 x 117 mm, 151 parts, among them J11 USB-C dual-role data/PD port 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, J12 USB-C source-only data port J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, J30 External HDMI-A from TCP0, J500 JXD1-1022NL recessed 1GbE RJ45, Q2002 2N7002K DFP USB2 enable inver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, Q50 BSS138 HDMI bias gate, U1760 TPS2553DDBVR 1.3A USB branch, U1761 TPS25810RVCR Type-C DFP contr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, U1763 TPD1S514-1YZR 5.9V VBUS OVP, U1765 TPD4E05U06 USB2/CC ESD, U2011 TPD4S201 CC and USB2 short-to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, U2012 CAT24C256 32KB private TPS257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, U2013 TS3USB30E DFP-qualified USB2 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, U2014 SN74LVC2G07 partial-power-dow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, U2015 TVS2200 22V USB VBUS surge cl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, U2016 SN74LVC1G08 DFP and attached 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, U42 TPS25751AD USB-PD DRP control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, U50 TPD4E05U06DQAR HDMI control a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, U500 RTL8111H-CG-RH PCIe Gigabit E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, U501 D3V3XA4B10LP-7 four-channel 0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, U502 D3V3XA4B10LP-7 four-channel 0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, U51 PCA9306DCTR HDMI DDC level tr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, U53 SN74LVC1G17DBVR HDMI HPD buff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, U54 TPS22948DCKR HDMI 5V current-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, U55 TPS22975NDSGR host-active SYS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, U721 TPS26630RGER PD2 default-off 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, Y500 ECS-250-8-33-AGN-TR 25MHz 8pF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

Commit message: fix the center layout and more board issues
Parts:
- added C2293: 22u 25V GbE input bulk; TI characterized part, Capacitor_SMD:C_1210_3225Metric, F.Cu at (321.4, 102.2)
- added C2404: 1u, Capacitor_SMD:C_0805_2012Metric, F.Cu at (323.4, 40.0)
- added C2409: 100n, Capacitor_SMD:C_0603_1608Metric, F.Cu at (314.5, 45.6)
- added C2414: 4.7n C0G PP5V slew, Capacitor_SMD:C_0603_1608Metric, F.Cu at (330.2, 37.0)
- added J2433: right power loom, straight-numbered, Connector_Molex:Molex_Micro-Fit_3.0_43045-1012_2x05_P3.00mm_Vertical, F.Cu at (313.5, 66.5)
- added J2435: USB5 direct power loom, ducktop2:AMASS_XT30PW-F30_G_Y, F.Cu at (328.0, 29.0)
- added J2445: main ground strap, Connector_Wire:SolderWirePad_1x01_SMD_5x10mm, F.Cu at (305.5, 42.5)
- added J2447: main ground strap, Connector_Wire:SolderWirePad_1x01_SMD_5x10mm, F.Cu at (305.5, 114.0)
- added R2404: 100k, Resistor_SMD:R_0603_1608Metric, F.Cu at (329.0, 39.6)
- added R2409: 100k, Resistor_SMD:R_0603_1608Metric, F.Cu at (307.0, 51.5)
- added R2414: 10k, Resistor_SMD:R_0603_1608Metric, F.Cu at (331.2, 40.8)
- added R2446: 0.33, Resistor_SMD:R_0603_1608Metric, F.Cu at (311.7, 72.3)
- added R2447: 0.33, Resistor_SMD:R_0603_1608Metric, F.Cu at (311.7, 109.6)
- added U2404: TPS22992SRXNR J11 PP5V gate, ducktop2:Texas_RXN0008A_WQFN-HR-8_1.25x1.25mm, F.Cu at (326.0, 40.0)
- added U2409: SN74LVC1G08DBVR J12 source permission, Package_TO_SOT_SMD:SOT-23-5, F.Cu at (311.0, 47.0)
- FPC104: value FH41-68S-0.5SH (FPC-2) -> Molex5039085120 signal cable; footprint ducktop2:Hirose_FH41-68S-0.5SH_1x68_1MP_1SH_P0.5mm_Horizontal -> ducktop2:Molex_5039085120_1x51_P0.50mm_Horizontal
- R1760: value 20.0k 1% TPS2553 1.3A ILIM -> 19.1k 1% TPS2553 VBUS plus VCONN ILIM
- R2090: value 8.87k 0.1% 10ppm 15/20V eFuse UV/OV top -> 8.87k 0.02% 5ppm 15/20V eFuse UV/OV top
- R2091: value 562R 0.1% 10ppm 15/20V eFuse UV/OV middle -> 562R 0.02% 5ppm 15/20V eFuse UV/OV middle
- R2092: value 511R 0.1% 10ppm 15/20V eFuse UV/OV bottom -> 511R 0.02% 5ppm 15/20V eFuse UV/OV bottom
- moved C2043 52.7 mm to (302.5, 11.7)
- moved C2062 48.5 mm to (322.1, 49.0), turned to 180 degrees
- moved C2070 45.1 mm to (308.7, 7.40), turned to 90 degrees
- moved C1771 44.4 mm to (346.0, 53.5)
- moved C2091 41.2 mm to (319.2, 78.8), turned to 90 degrees
- moved U1763 40.8 mm to (346.5, 51.3)
- moved C2059 36.2 mm to (347.0, 38.0), turned to 90 degrees
- moved C1762 35.2 mm to (327.0, 55.5), turned to 180 degrees
- moved C2041 34.4 mm to (340.5, 33.5)
- moved C2067 34.3 mm to (325.5, 37.0), turned to 180 degrees
- moved C2040 33.3 mm to (344.0, 34.5)
- moved C1763 29.8 mm to (342.8, 51.3), turned to 180 degrees
- moved C2064 29.7 mm to (331.2, 39.0), turned to 90 degrees
- moved C1761 27.7 mm to (331.8, 49.4), turned to 180 degrees
- moved C2042 26.2 mm to (333.5, 42.2), turned to 90 degrees
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Connections:
- C2065 pad 1: /USB_PORT_5V -> /PD2 Dual-Role/PD2_PP5V_GATED
- C2066 pad 1: /USB_PORT_5V -> /PD2 Dual-Role/PD2_PP5V_GATED
- C2067 pad 1: /USB_PORT_5V -> /PD2 Dual-Role/PD2_PP5V_GATED
- FPC104 pad 1: /SYS_5V -> GND
- FPC104 pad 10: /PD2_VBUS_GATED -> GND
- FPC104 pad 11: /PD2_VBUS_GATED -> /TCP0_TXRX1_P
- FPC104 pad 12: /PD2_VBUS_GATED -> /TCP0_TXRX1_N
- FPC104 pad 13: /PD2_VBUS_GATED -> GND
- FPC104 pad 14: /PD2_VBUS_RAW -> /GBE_HOST_RX_P
- FPC104 pad 15: /PD2_VBUS_RAW -> /GBE_HOST_RX_N
- FPC104 pad 16: /USB_PORT_5V -> GND
- FPC104 pad 17: /USB_PORT_5V -> /GBE_HOST_TX_P
- FPC104 pad 18: /USB_PORT_5V -> /GBE_HOST_TX_N
- FPC104 pad 19: /USB_PORT_5V -> GND
- FPC104 pad 2: /SYS_5V -> /TCP0_TX0_P
- FPC104 pad 20: GND -> /GBE_REFCLK_P
- FPC104 pad 21: GND -> /GBE_REFCLK_N
- FPC104 pad 22: /SYS_3V3 -> GND
- FPC104 pad 23: /SYS_3V3 -> /HUB_DS1_DP
- FPC104 pad 24: /PCIE_3V3 -> /HUB_DS1_DN
- FPC104 pad 25: /PCIE_3V3 -> GND
- FPC104 pad 26: /MCU_3V3 -> /HUB_DS4_DP
- FPC104 pad 27: /MCU_3V3 -> /HUB_DS4_DN
- FPC104 pad 29: /HUB_DS4_DP -> /TCP0_DDC_SCL
- FPC104 pad 3: /SYS_5V -> /TCP0_TX0_N
- FPC104 pad 30: /HUB_DS4_DN -> /TCP0_DDC_SDA
- FPC104 pad 31: /HUB_PRT_CTL4 -> /TCP0_HPD
- FPC104 pad 32: /MU_HOST_ACTIVE -> GND
- FPC104 pad 33: /PLTRST_SRC_N -> /PD2_I2C_SCL
- FPC104 pad 34: /PCIE_WAKE_N -> /PD2_I2C_SDA
- FPC104 pad 35: /GBE_CLKREQ_N -> /PD2_TCPC_IRQ_N
- FPC104 pad 36: /PD2_I2C_SCL -> GND
- FPC104 pad 37: /PD2_I2C_SDA -> /PD2_PATH_EN
- FPC104 pad 38: /PD2_TCPC_IRQ_N -> /PD2_EFUSE_FAULT_N
- FPC104 pad 39: /PD2_PATH_EN -> /PD_PROTECT_FAULT_N
- FPC104 pad 4: /SYS_5V -> GND
- FPC104 pad 40: /PD2_EFUSE_FAULT_N -> GND
- FPC104 pad 41: /PD_PROTECT_FAULT_N -> /PD2_SOURCE_PG
- FPC104 pad 42: GND -> /USB_J11_PERMIT
- FPC104 pad 43: /HUB_DS1_DP -> /USB_J12_PERMIT
- FPC104 pad 44: /HUB_DS1_DN -> GND
- FPC104 pad 45: GND -> /HUB_PRT_CTL4
- FPC104 pad 46: /TCP0_DDC_SCL -> /MU_HOST_ACTIVE
- FPC104 pad 47: /TCP0_DDC_SDA -> /PLTRST_SRC_N
- FPC104 pad 48: /TCP0_HPD -> GND
- FPC104 pad 49: GND -> /PCIE_WAKE_N
- FPC104 pad 5: GND -> /TCP0_TX1_P
- FPC104 pad 50: /GBE_REFCLK_P -> /GBE_CLKREQ_N
- FPC104 pad 51: /GBE_REFCLK_N -> GND
- FPC104 pad 6: GND -> /TCP0_TX1_N
- FPC104 pad 7: /PD2_VBUS_GATED -> GND
- FPC104 pad 8: /PD2_VBUS_GATED -> /TCP0_TXRX0_P
- FPC104 pad 9: /PD2_VBUS_GATED -> /TCP0_TXRX0_N
- FPC104 pad SH: GND -> /FPC-2 (to Center)/FPC104_SHELL
- U1760 pad 3: /HUB_PRT_CTL4 -> /PD2 Dual-Role/USB_J12_SWITCH_EN
- U1761 pad 6: /HUB_PRT_CTL4 -> /PD2 Dual-Role/USB_J12_SWITCH_EN
- U42 pad 34: /USB_PORT_5V -> /PD2 Dual-Role/PD2_PP5V_GATED
Routing:
- net /HDMI/EXT_HDMI_BIAS_RETURN: track 13.6 -> 65.1 mm, vias 5 -> 6
- net /PD2_VBUS_GATED: track 25.0 -> 0.00 mm
- net /PD2 Dual-Role/PD2_HOST_SWITCHED_DN: track 3.48 -> 9.87 mm
- net /HDMI/HDMI_DDC_REF5: track 8.68 -> 14.3 mm, vias 0 -> 3
- net /PD2 Dual-Role/PD2_CONN_DN: track 9.23 -> 14.3 mm
- net /HDMI/EXT_HDMI_CK_P: track 11.4 -> 8.39 mm, vias 2 -> 0
- net /HDMI/EXT_HDMI_D2_P: track 7.44 -> 9.30 mm
- net /HDMI/EXT_HDMI_D0_N: track 5.92 -> 7.78 mm, vias 2 -> 0
- net /PD2 Dual-Role/PD2_CONN_DP: track 13.7 -> 15.5 mm
- net /HDMI/EXT_HDMI_D1_P: track 6.58 -> 8.09 mm, vias 2 -> 0
- net GND: track 76.3 -> 74.9 mm, vias 36 -> 38
- net /TCP0_TXRX1_N: track 1.33 -> 0.00 mm, vias 1 -> 0
- net /HDMI/EXT_HDMI_D2_N: track 8.09 -> 9.30 mm, vias 1 -> 0
- net /MU_HOST_ACTIVE: track 2.80 -> 3.95 mm
- net /HDMI/EXT_HDMI_CK_N: track 9.54 -> 8.39 mm, vias 2 -> 0
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