File: right_io/right_hdmi.kicad_sch (KiCad schematic)
At the start: 50 parts, among them J30 External HDMI-A from TCP0, Q50 BSS138 HDMI bias gate, U50 TPD4E05U06DQAR HDMI control a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, U51 PCA9306DCTR HDMI DDC level tr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, U53 SN74LVC1G17DBVR HDMI HPD buff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, U54 TPS22948DCKR HDMI 5V current-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, U55 TPS22975NDSGR host-active SYS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

Commit message: start switching the carrier to mu ultra
Parts:
- J30: value External HDMI-A from TCP0 -> External HDMI-A from TCP2
Connections:
- net TCP0_DDC_SCL renamed TCP2_DDC_SCL
- net TCP0_DDC_SDA renamed TCP2_DDC_SDA
- net TCP0_HPD renamed TCP2_HPD
- net TCP0_TX0_N renamed TCP2_TX0_N
- net TCP0_TX0_P renamed TCP2_TX0_P
- net TCP0_TX1_N renamed TCP2_TX1_N
- net TCP0_TX1_P renamed TCP2_TX1_P
- net TCP0_TXRX0_N renamed TCP2_TXRX0_N
- net TCP0_TXRX0_P renamed TCP2_TXRX0_P
- net TCP0_TXRX1_N renamed TCP2_TXRX1_N
- net TCP0_TXRX1_P renamed TCP2_TXRX1_P
Other:
- note added: "== TCP2 external HDMI 2.0 output =="
- note added: "LattePanda Mu Ultra default BIOS maps TCP2 as HDMI 2.0; the internal panel uses the Mu module's onboard eDP connector."
- note removed: "== TCP0 external HDMI 2.0 output =="
- note removed: "LattePanda Mu default BIOS maps TCP0 as HDMI 2.0; the internal panel uses the Mu module's onboard eDP connector."
Changed lines of the file:
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@@
   (generator_version "10.0")
   (paper "A2")
-(text "== TCP0 external HDMI 2.0 output ==" (at 20.32 12.7 0) (effects (font (size 1.27 1.27))))
-(text "LattePanda Mu default BIOS maps TCP0 as HDMI 2.0; the internal panel uses the Mu module's onboard eDP connector." (at 20.32 20.32 0) (effects (font (size 1.27 1.27))))
+(text "== TCP2 external HDMI 2.0 output ==" (at 20.32 12.7 0) (effects (font (size 1.27 1.27))))
+(text "LattePanda Mu Ultra default BIOS maps TCP2 as HDMI 2.0; the internal panel uses the Mu module's onboard eDP connector." (at 20.32 20.32 0) (effects (font (size 1.27 1.27))))
 (text "Lane map, AC coupling, bias gating, DDC/HPD translation, and 5V isolation follow the Mu reference." (at 20.32 27.94 0) (effects (font (size 1.27 1.27))))
 (text "== J30 external HDMI-A connector ==" (at 20.32 50.8 0) (effects (font (size 1.27 1.27))))
@@
   (dnp no)
   (property "Reference" "J30" (at 115.57 90.17 0) (effects (font (size 1.27 1.27))))
-  (property "Value" "External HDMI-A from TCP0" (at 115.57 158.75 0) (effects (font (size 1.27 1.27))))
+  (property "Value" "External HDMI-A from TCP2" (at 115.57 158.75 0) (effects (font (size 1.27 1.27))))
   (property "Footprint" "Connector_Video:HDMI_A_Molex_208658-1001_Horizontal" (at 115.57 124.46 0) (effects (font (size 1.27 1.27)) (hide yes)))
   (property "Datasheet" "" (at 115.57 124.46 0) (effects (font (size 1.27 1.27)) (hide yes)))
@@
   )
 )
-(hierarchical_label "TCP0_TX0_P"
+(hierarchical_label "TCP2_TX0_P"
   (shape bidirectional)
   (at 250.19 78.74 0)
@@
   )
 )
-(hierarchical_label "TCP0_TX0_N"
+(hierarchical_label "TCP2_TX0_N"
   (shape bidirectional)
   (at 304.8 78.74 0)
@@
   )
 )
-(hierarchical_label "TCP0_TXRX0_P"
+(hierarchical_label "TCP2_TXRX0_P"
   (shape bidirectional)
   (at 359.41 78.74 0)
@@
   )
 )
-(hierarchical_label "TCP0_TXRX0_N"
+(hierarchical_label "TCP2_TXRX0_N"
   (shape bidirectional)
   (at 415.29 78.74 0)
@@
   )
 )
-(hierarchical_label "TCP0_TX1_P"
+(hierarchical_label "TCP2_TX1_P"
   (shape bidirectional)
   (at 250.19 104.14 0)
@@
   )
 )
-(hierarchical_label "TCP0_TX1_N"
+(hierarchical_label "TCP2_TX1_N"
   (shape bidirectional)
   (at 304.8 104.14 0)
@@
   )
 )
-(hierarchical_label "TCP0_TXRX1_P"
+(hierarchical_label "TCP2_TXRX1_P"
   (shape bidirectional)
   (at 359.41 104.14 0)
@@
   )
 )
-(hierarchical_label "TCP0_TXRX1_N"
+(hierarchical_label "TCP2_TXRX1_N"
   (shape bidirectional)
   (at 415.29 104.14 0)
@@
   (effects (font (size 1.27 1.27)) (justify right bottom))
 )
-(hierarchical_label "TCP0_DDC_SCL"
+(hierarchical_label "TCP2_DDC_SCL"
   (shape bidirectional)
   (at 492.76 118.11 180)
   (effects (font (size 1.27 1.27)) (justify right bottom))
 )
-(hierarchical_label "TCP0_DDC_SDA"
+(hierarchical_label "TCP2_DDC_SDA"
   (shape bidirectional)
   (at 492.76 120.65 180)
@@
   (effects (font (size 1.27 1.27)) (justify left bottom))
 )
-(hierarchical_label "TCP0_DDC_SCL"
+(hierarchical_label "TCP2_DDC_SCL"
   (shape bidirectional)
   (at 575.31 100.33 0)
@@
   (effects (font (size 1.27 1.27)) (justify left bottom))
 )
-(hierarchical_label "TCP0_DDC_SDA"
+(hierarchical_label "TCP2_DDC_SDA"
   (shape bidirectional)
   (at 575.31 113.03 0)
@@
   (effects (font (size 1.27 1.27)) (justify right bottom))
 )
-(hierarchical_label "TCP0_HPD"
+(hierarchical_label "TCP2_HPD"
   (shape bidirectional)
   (at 510.54 157.48 0)

Commit message: rework the board placement and fix more power stuff
Parts:
- added C2680: 1u 50V U55 input bypass, Capacitor_SMD:C_0603_1608Metric, symbol Device:C
Connections:
- net GND: now also C2680.2
- net SYS_3V3: now also C2680.1
Changed lines of the file:
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@@
 )
   (embedded_fonts no)
+(symbol
+  (lib_id "Device:C")
+  (at 405.13 142.24 0)
+  (unit 1)
+  (exclude_from_sim no)
+  (in_bom yes)
+  (on_board yes)
+  (dnp no)
+  (property "Reference" "C2680" (at 410.21 140.97 0) (effects (font (size 1.27 1.27)) (justify left)))
+  (property "Value" "1u 50V U55 input bypass" (at 410.21 143.51 0) (effects (font (size 1.27 1.27)) (justify left)))
+  (property "Footprint" "Capacitor_SMD:C_0603_1608Metric" (at 405.13 142.24 0) (effects (font (size 1.27 1.27)) (hide yes)))
+  (property "Datasheet" "" (at 405.13 142.24 0) (effects (font (size 1.27 1.27)) (hide yes)))
+  (property "Manufacturer" "Murata" (at 405.13 142.24 0) (effects (font (size 1.27 1.27)) (hide yes)))
+  (property "MPN" "GRT188R61H105ME13D" (at 405.13 142.24 0) (effects (font (size 1.27 1.27)) (hide yes)))
+  (property "DecouplingFor" "U55 VIN and VBIAS" (at 405.13 142.24 0) (effects (font (size 1.27 1.27)) (hide yes)))
+  (pin "1")
+  (pin "2")
+  (instances
+    (project "right_io"
+      (path "/49653426-5341-5295-bc21-ff9bd272935d"
+        (reference "C2680")
+        (unit 1)
+      )
+    )
+  )
 )
+(hierarchical_label "SYS_3V3"
+  (shape bidirectional)
+  (at 405.13 138.43 0)
+  (effects (font (size 1.27 1.27)) (justify left bottom))
+)
+(label "GND"
+  (at 405.13 146.05 0)
+  (effects (font (size 1.27 1.27)) (justify left bottom))
+)
+)
