File: keyboard/12_keyboard_daughterboard.kicad_pcb (KiCad board)
At the start: 2 copper layers, 273.5 x 80 mm, 131 parts, among them J320 Keyboard FFC: MX ULP 5x14 mat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, SW320 Esc 1u, SW321 1 1u, SW322 2 1u, SW323 3 1u, SW324 4 1u, SW325 5 1u, SW326 6 1u, SW327 7 1u, SW328 8 1u, SW329 9 1u, SW330 0 1u, SW331 Minus 1u, SW332 Equal 1u, SW333 Backspace 1.75u, SW334 Tab 1.25u, SW335 Q 1u, SW336 W 1u, SW337 E 1u, SW338 R 1u, SW339 T 1u, SW340 Y 1u, SW341 U 1u, SW342 I 1u, SW343 O 1u, SW344 P 1u, SW345 [ 1u, SW346 ] 1u, SW347 Backslash 1u, SW348 Caps 1.5u, SW349 A 1u, SW350 S 1u, SW351 D 1u, SW352 F 1u, SW353 G 1u, SW354 H 1u, SW355 J 1u, SW356 K 1u, SW357 L 1u, SW358 Semicolon 1u, SW359 Quote 1u, SW360 Enter 1.75u, SW361 Shift L 1.75u, SW362 Z 1u, SW363 X 1u, SW364 C 1u, SW365 V 1u, SW366 B 1u, SW367 N 1u, SW368 M 1u, SW369 Comma 1u, SW370 Period 1u, SW371 Slash 1u, SW372 Up 1u, SW373 Shift R 1.25u, SW374 Ctrl 1u, SW375 Fn 1u, SW376 Super 1u, SW377 Alt L 1u, SW378 Space L 2.25u, SW379 Space R 2.25u, SW380 Alt R 1u, SW381 Menu 1u, SW382 Left 1u, SW383 Down 1u, SW384 Right 1u

Commit message: add rgb to the keyboard and get it ready to route
Parts:
- added C320: 100n 50V buffer 3V3, Capacitor_SMD:C_0603_1608Metric, F.Cu at (289.2, 26.2)
- added C321: 10u 25V RGB input bulk, Capacitor_SMD:C_0805_2012Metric, F.Cu at (289.5, 8.00)
- added C322: 1u 25V RGB VCC, Capacitor_SMD:C_0603_1608Metric, F.Cu at (289.2, 23.2)
- added C323: 100n 50V RGB VCC, Capacitor_SMD:C_0603_1608Metric, F.Cu at (289.2, 21.4)
- added C324: 1u 25V RGB PVCC, Capacitor_SMD:C_0603_1608Metric, F.Cu at (280.4, 20.8)
- added C325: 100n 50V RGB PVCC / buffer A, Capacitor_SMD:C_0603_1608Metric, F.Cu at (280.4, 24.0)
- added C326: 100n 50V RGB startup delay, Capacitor_SMD:C_0603_1608Metric, F.Cu at (289.1, 13.5)
- added LED320: RGB ESC, ducktop2:LED_Everlight_19-337_1616, F.Cu at (26.2, 5.20)
- added LED321: RGB 1, ducktop2:LED_Everlight_19-337_1616, F.Cu at (44.2, 5.20)
- added LED322: RGB 2, ducktop2:LED_Everlight_19-337_1616, F.Cu at (62.2, 5.20)
- added LED323: RGB 3, ducktop2:LED_Everlight_19-337_1616, F.Cu at (80.2, 5.20)
- added LED324: RGB 4, ducktop2:LED_Everlight_19-337_1616, F.Cu at (98.2, 5.20)
- added LED325: RGB 5, ducktop2:LED_Everlight_19-337_1616, F.Cu at (116.2, 5.20)
- added LED326: RGB 6, ducktop2:LED_Everlight_19-337_1616, F.Cu at (134.2, 5.20)
- added LED327: RGB 7, ducktop2:LED_Everlight_19-337_1616, F.Cu at (152.2, 5.20)
- added LED328: RGB 8, ducktop2:LED_Everlight_19-337_1616, F.Cu at (170.2, 5.20)
- added LED329: RGB 9, ducktop2:LED_Everlight_19-337_1616, F.Cu at (188.2, 5.20)
- added LED330: RGB 0, ducktop2:LED_Everlight_19-337_1616, F.Cu at (206.2, 5.20)
- added LED331: RGB MINUS, ducktop2:LED_Everlight_19-337_1616, F.Cu at (224.2, 5.20)
- added LED332: RGB EQUAL, ducktop2:LED_Everlight_19-337_1616, F.Cu at (242.2, 5.20)
- added LED333: RGB BKSP, ducktop2:LED_Everlight_19-337_1616, F.Cu at (267.0, 5.20)
- added LED334: RGB TAB, ducktop2:LED_Everlight_19-337_1616, F.Cu at (33.0, 21.2)
- added LED335: RGB Q, ducktop2:LED_Everlight_19-337_1616, F.Cu at (53.2, 21.2)
- added LED336: RGB W, ducktop2:LED_Everlight_19-337_1616, F.Cu at (71.2, 21.2)
- added LED337: RGB E, ducktop2:LED_Everlight_19-337_1616, F.Cu at (89.2, 21.2)
- added LED338: RGB R, ducktop2:LED_Everlight_19-337_1616, F.Cu at (107.2, 21.2)
- added LED339: RGB T, ducktop2:LED_Everlight_19-337_1616, F.Cu at (125.2, 21.2)
- added LED340: RGB Y, ducktop2:LED_Everlight_19-337_1616, F.Cu at (143.2, 21.2)
- added LED341: RGB U, ducktop2:LED_Everlight_19-337_1616, F.Cu at (161.2, 21.2)
- added LED342: RGB I, ducktop2:LED_Everlight_19-337_1616, F.Cu at (179.2, 21.2)
- added LED343: RGB O, ducktop2:LED_Everlight_19-337_1616, F.Cu at (197.2, 21.2)
- added LED344: RGB P, ducktop2:LED_Everlight_19-337_1616, F.Cu at (215.2, 21.2)
- added LED345: RGB LBRACKET, ducktop2:LED_Everlight_19-337_1616, F.Cu at (233.2, 21.2)
- added LED346: RGB RBRACKET, ducktop2:LED_Everlight_19-337_1616, F.Cu at (251.2, 21.2)
- added LED347: RGB BSLASH, ducktop2:LED_Everlight_19-337_1616, F.Cu at (269.2, 21.2)
- added LED348: RGB CAPS, ducktop2:LED_Everlight_19-337_1616, F.Cu at (35.2, 37.2)
- added LED349: RGB A, ducktop2:LED_Everlight_19-337_1616, F.Cu at (57.8, 37.2)
- added LED350: RGB S, ducktop2:LED_Everlight_19-337_1616, F.Cu at (75.8, 37.2)
- added LED351: RGB D, ducktop2:LED_Everlight_19-337_1616, F.Cu at (93.8, 37.2)
- added LED352: RGB F, ducktop2:LED_Everlight_19-337_1616, F.Cu at (111.8, 37.2)
- added LED353: RGB G, ducktop2:LED_Everlight_19-337_1616, F.Cu at (129.8, 37.2)
- added LED354: RGB H, ducktop2:LED_Everlight_19-337_1616, F.Cu at (147.8, 37.2)
- added LED355: RGB J, ducktop2:LED_Everlight_19-337_1616, F.Cu at (165.8, 37.2)
- added LED356: RGB K, ducktop2:LED_Everlight_19-337_1616, F.Cu at (183.8, 37.2)
- added LED357: RGB L, ducktop2:LED_Everlight_19-337_1616, F.Cu at (201.8, 37.2)
- added LED358: RGB SEMICOLON, ducktop2:LED_Everlight_19-337_1616, F.Cu at (219.8, 37.2)
- added LED359: RGB QUOTE, ducktop2:LED_Everlight_19-337_1616, F.Cu at (237.8, 37.2)
- added LED360: RGB ENTER, ducktop2:LED_Everlight_19-337_1616, F.Cu at (262.5, 37.2)
- added LED361: RGB LSHIFT, ducktop2:LED_Everlight_19-337_1616, F.Cu at (39.8, 53.2)
- added LED362: RGB Z, ducktop2:LED_Everlight_19-337_1616, F.Cu at (64.5, 53.2)
- added LED363: RGB X, ducktop2:LED_Everlight_19-337_1616, F.Cu at (82.5, 53.2)
- added LED364: RGB C, ducktop2:LED_Everlight_19-337_1616, F.Cu at (100.5, 53.2)
- added LED365: RGB V, ducktop2:LED_Everlight_19-337_1616, F.Cu at (118.5, 53.2)
- added LED366: RGB B, ducktop2:LED_Everlight_19-337_1616, F.Cu at (136.5, 53.2)
- added LED367: RGB N, ducktop2:LED_Everlight_19-337_1616, F.Cu at (154.5, 53.2)
- added LED368: RGB M, ducktop2:LED_Everlight_19-337_1616, F.Cu at (172.5, 53.2)
- added LED369: RGB COMMA, ducktop2:LED_Everlight_19-337_1616, F.Cu at (190.5, 53.2)
- added LED370: RGB PERIOD, ducktop2:LED_Everlight_19-337_1616, F.Cu at (208.5, 53.2)
- added LED371: RGB SLASH, ducktop2:LED_Everlight_19-337_1616, F.Cu at (226.5, 53.2)
- added LED372: RGB UP, ducktop2:LED_Everlight_19-337_1616, F.Cu at (244.5, 53.2)
- added LED373: RGB RSHIFT, ducktop2:LED_Everlight_19-337_1616, F.Cu at (264.8, 53.2)
- added LED374: RGB CTRL, ducktop2:LED_Everlight_19-337_1616, F.Cu at (28.5, 69.2)
- added LED375: RGB FN, ducktop2:LED_Everlight_19-337_1616, F.Cu at (46.5, 69.2)
- added LED376: RGB SUPER, ducktop2:LED_Everlight_19-337_1616, F.Cu at (64.5, 69.2)
- added LED377: RGB LALT, ducktop2:LED_Everlight_19-337_1616, F.Cu at (82.5, 69.2)
- added LED378: RGB SPACE_L, ducktop2:LED_Everlight_19-337_1616, F.Cu at (111.8, 69.2)
- added LED379: RGB SPACE_R, ducktop2:LED_Everlight_19-337_1616, F.Cu at (152.2, 69.2)
- added LED380: RGB RALT, ducktop2:LED_Everlight_19-337_1616, F.Cu at (181.5, 69.2)
- added LED381: RGB MENU, ducktop2:LED_Everlight_19-337_1616, F.Cu at (199.5, 69.2)
- added LED382: RGB LEFT, ducktop2:LED_Everlight_19-337_1616, F.Cu at (235.5, 69.2)
- added LED383: RGB DOWN, ducktop2:LED_Everlight_19-337_1616, F.Cu at (253.5, 69.2)
- added LED384: RGB RIGHT, ducktop2:LED_Everlight_19-337_1616, F.Cu at (271.5, 69.2)
- added R320: 33.2k 1% RGB current limit, Resistor_SMD:R_0603_1608Metric, F.Cu at (289.2, 19.6)
- added R321: 2.2k RGB SCL pull-up, Resistor_SMD:R_0603_1608Metric, F.Cu at (279.8, 28.0)
- added R322: 2.2k RGB SDA pull-up, Resistor_SMD:R_0603_1608Metric, F.Cu at (289.2, 29.0)
- added R323: 100k RGB startup pull-up, Resistor_SMD:R_0603_1608Metric, F.Cu at (289.1, 16.7)
- added R330: 100R red-channel heat sharing, Resistor_SMD:R_0603_1608Metric, F.Cu at (283.4, 4.00)
- added R331: 100R red-channel heat sharing, Resistor_SMD:R_0603_1608Metric, F.Cu at (286.3, 4.00)
- added R332: 100R red-channel heat sharing, Resistor_SMD:R_0603_1608Metric, F.Cu at (286.3, 8.00)
- added R333: 100R red-channel heat sharing, Resistor_SMD:R_0603_1608Metric, F.Cu at (283.4, 8.00)
- added R334: 100R red-channel heat sharing, Resistor_SMD:R_0603_1608Metric, F.Cu at (283.4, 12.0)
- added R335: 100R red-channel heat sharing, Resistor_SMD:R_0603_1608Metric, F.Cu at (286.3, 12.0)
- added TPK1: KB_RGB_5V, TestPoint:TestPoint_Pad_D1.0mm, F.Cu at (284.5, 55.0)
- added TPK2: GND, TestPoint:TestPoint_Pad_D1.0mm, F.Cu at (288.0, 55.0)
- added TPK3: MCU_3V3, TestPoint:TestPoint_Pad_D1.0mm, F.Cu at (284.5, 60.0)
- added TPK4: RGB_SCL, TestPoint:TestPoint_Pad_D1.0mm, F.Cu at (288.0, 60.0)
- added TPK5: RGB_SDA, TestPoint:TestPoint_Pad_D1.0mm, F.Cu at (284.5, 65.0)
- added TPK6: RGB_SDB, TestPoint:TestPoint_Pad_D1.0mm, F.Cu at (288.0, 65.0)
- added U320: IS31FL3743A-QULS4-TR, ducktop2:IS31FL3743A_UQFN40, F.Cu at (284.5, 21.0)
- added U321: TCA9517ADGKR, Package_SO:VSSOP-8_3x3mm_P0.65mm, F.Cu at (284.5, 28.0)
Connections:
- J320 pad 10: KB_ROW5 -> (no net)
- J320 pad 11: KB_ROW6 -> (no net)
- J320 pad 12: KB_ROW7 -> (no net)
- J320 pad 27: KB_COL14 -> (no net)
- J320 pad 28: KB_COL15 -> (no net)
- J320 pad 29: SYS_5V -> KB_RGB_5V
Routing:
- net GND: track 413.5 -> 0.00 mm, vias 326 -> 0
- net KB_ROW4: track 363.9 -> 0.00 mm, vias 2 -> 0
- net KB_COL0: track 347.0 -> 0.00 mm, vias 4 -> 0
- net KB_COL1: track 319.8 -> 0.00 mm, vias 8 -> 0
- net KB_COL2: track 302.6 -> 0.00 mm, vias 6 -> 0
- net KB_ROW0: track 300.4 -> 0.00 mm
- net KB_ROW2: track 282.2 -> 0.00 mm, vias 24 -> 0
- net KB_ROW1: track 278.7 -> 0.00 mm, vias 14 -> 0
- net KB_COL3: track 278.6 -> 0.00 mm, vias 6 -> 0
- net KB_ROW3: track 266.0 -> 0.00 mm, vias 24 -> 0
- net KB_COL4: track 260.7 -> 0.00 mm, vias 4 -> 0
- net KB_COL5: track 240.8 -> 0.00 mm, vias 2 -> 0
- net KB_COL6: track 219.8 -> 0.00 mm, vias 2 -> 0
- net KB_COL7: track 199.9 -> 0.00 mm, vias 2 -> 0
- net KB_COL8: track 161.1 -> 0.00 mm, vias 2 -> 0
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- removed copper zone on B.Cu, net GND
- removed copper zone on F.Cu, net GND
Other:
- board text added: "Ducktop2 MX ULP keyboard daughterboard RGB: 273.5 x 80 mm Edge.Cuts"
- board text added: "J320 keeps the existing cable exit. Switches and LEDs are locked for routing."
- board text removed: "Ducktop2 MX ULP keyboard daughterboard rev A: 273.5 x 80 mm Edge.Cuts"
- board text removed: "J320 is parked in the right margin as a routing anchor; move only if the final flex exit requires it."

Commit message: keyboard stuff, lattepanda switching stuff
Parts:
- moved TPK1 22.6 mm to (281.8, 32.5)
- moved R334 14.0 mm to (289.2, 24.7), turned to 0 degrees
- moved C325 10.4 mm to (281.3, 34.4), turned to 180 degrees
- moved C321 8.07 mm to (289.0, 16.1), turned to 0 degrees
- moved C324 6.86 mm to (285.4, 25.5), turned to 0 degrees
- moved R321 1.46 mm to (280.6, 26.8), turned to -90 degrees
- moved R323 1.11 mm to (289.2, 17.8)
- moved R320 0.30 mm to (289.2, 19.3)
Routing:
- net KB_ROW4: track 0.00 -> 246.9 mm
- net KB_ROW0: track 0.00 -> 245.9 mm
- net KB_ROW1: track 0.00 -> 241.4 mm
- net KB_ROW2: track 0.00 -> 232.0 mm
- net KB_ROW3: track 0.00 -> 229.7 mm
- net RGB_SW10: track 0.00 -> 147.0 mm, vias 0 -> 1
- net RGB_SW09: track 0.00 -> 120.1 mm, vias 0 -> 1
- net RGB_SW01: track 0.00 -> 115.2 mm, vias 0 -> 1
- net RGB_SW02: track 0.00 -> 115.0 mm, vias 0 -> 1
- net RGB_SW04: track 0.00 -> 113.9 mm, vias 0 -> 1
- net RGB_SW06: track 0.00 -> 113.7 mm, vias 0 -> 1
- net RGB_SW08: track 0.00 -> 113.2 mm, vias 0 -> 1
- net RGB_SW11: track 0.00 -> 109.0 mm, vias 0 -> 1
- net RGB_SW03: track 0.00 -> 100.4 mm, vias 0 -> 1
- net RGB_SW05: track 0.00 -> 100.1 mm, vias 0 -> 1
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- added copper zone on B.Cu, net GND
- added copper zone on F.Cu, net GND
- added copper zone on In1.Cu, net GND
- added copper zone on In2.Cu, net GND
Other:
- copper layers 2 -> 4
- board text removed: "J320 keeps the existing cable exit. Switches and LEDs are locked for routing."

Commit message: sort out the keyboard leds and fix more bms routing
Connections:
- LED320 pad 1: RGB_SW01 -> RGB_SW11
- LED320 pad 3: RGB_SW01 -> RGB_SW11
- LED320 pad 5: RGB_SW01 -> RGB_SW11
- LED321 pad 2: RGB_CS06 -> RGB_CS18
- LED321 pad 4: RGB_RED04 -> RGB_RED16
- LED321 pad 6: RGB_CS05 -> RGB_CS17
- LED322 pad 2: RGB_CS09 -> RGB_CS03
- LED322 pad 4: RGB_RED07 -> RGB_RED01
- LED322 pad 6: RGB_CS08 -> RGB_CS02
- LED323 pad 1: RGB_SW01 -> RGB_SW02
- LED323 pad 2: RGB_CS12 -> RGB_CS03
- LED323 pad 3: RGB_SW01 -> RGB_SW02
- LED323 pad 4: RGB_RED10 -> RGB_RED01
- LED323 pad 5: RGB_SW01 -> RGB_SW02
- LED323 pad 6: RGB_CS11 -> RGB_CS02
- LED324 pad 1: RGB_SW01 -> RGB_SW03
- LED324 pad 2: RGB_CS15 -> RGB_CS03
- LED324 pad 3: RGB_SW01 -> RGB_SW03
- LED324 pad 4: RGB_RED13 -> RGB_RED01
- LED324 pad 5: RGB_SW01 -> RGB_SW03
- LED324 pad 6: RGB_CS14 -> RGB_CS02
- LED325 pad 1: RGB_SW01 -> RGB_SW04
- LED325 pad 2: RGB_CS18 -> RGB_CS03
- LED325 pad 3: RGB_SW01 -> RGB_SW04
- LED325 pad 4: RGB_RED16 -> RGB_RED01
- LED325 pad 5: RGB_SW01 -> RGB_SW04
- LED325 pad 6: RGB_CS17 -> RGB_CS02
- LED326 pad 1: RGB_SW02 -> RGB_SW04
- LED326 pad 2: RGB_CS03 -> RGB_CS18
- LED326 pad 3: RGB_SW02 -> RGB_SW04
- LED326 pad 4: RGB_RED01 -> RGB_RED16
- LED326 pad 5: RGB_SW02 -> RGB_SW04
- LED326 pad 6: RGB_CS02 -> RGB_CS17
- LED327 pad 1: RGB_SW02 -> RGB_SW05
- LED327 pad 2: RGB_CS06 -> RGB_CS03
- LED327 pad 3: RGB_SW02 -> RGB_SW05
- LED327 pad 4: RGB_RED04 -> RGB_RED01
- LED327 pad 5: RGB_SW02 -> RGB_SW05
- LED327 pad 6: RGB_CS05 -> RGB_CS02
- LED328 pad 1: RGB_SW02 -> RGB_SW06
- LED328 pad 2: RGB_CS09 -> RGB_CS03
- LED328 pad 3: RGB_SW02 -> RGB_SW06
- LED328 pad 4: RGB_RED07 -> RGB_RED01
- LED328 pad 5: RGB_SW02 -> RGB_SW06
- LED328 pad 6: RGB_CS08 -> RGB_CS02
- LED329 pad 1: RGB_SW02 -> RGB_SW07
- LED329 pad 2: RGB_CS12 -> RGB_CS03
- LED329 pad 3: RGB_SW02 -> RGB_SW07
- LED329 pad 4: RGB_RED10 -> RGB_RED01
- LED329 pad 5: RGB_SW02 -> RGB_SW07
- LED329 pad 6: RGB_CS11 -> RGB_CS02
- LED330 pad 1: RGB_SW02 -> RGB_SW08
- LED330 pad 2: RGB_CS15 -> RGB_CS18
- LED330 pad 3: RGB_SW02 -> RGB_SW08
- LED330 pad 4: RGB_RED13 -> RGB_RED16
- LED330 pad 5: RGB_SW02 -> RGB_SW08
- LED330 pad 6: RGB_CS14 -> RGB_CS17
- LED331 pad 1: RGB_SW02 -> RGB_SW08
- LED331 pad 2: RGB_CS18 -> RGB_CS03
- LED331 pad 3: RGB_SW02 -> RGB_SW08
- LED331 pad 4: RGB_RED16 -> RGB_RED01
- LED331 pad 5: RGB_SW02 -> RGB_SW08
- LED331 pad 6: RGB_CS17 -> RGB_CS02
- LED332 pad 1: RGB_SW03 -> RGB_SW09
- LED332 pad 3: RGB_SW03 -> RGB_SW09
- LED332 pad 5: RGB_SW03 -> RGB_SW09
- LED333 pad 1: RGB_SW03 -> RGB_SW10
- LED333 pad 2: RGB_CS06 -> RGB_CS03
- LED333 pad 3: RGB_SW03 -> RGB_SW10
- LED333 pad 4: RGB_RED04 -> RGB_RED01
- LED333 pad 5: RGB_SW03 -> RGB_SW10
- LED333 pad 6: RGB_CS05 -> RGB_CS02
- LED334 pad 1: RGB_SW05 -> RGB_SW11
- LED334 pad 2: RGB_CS12 -> RGB_CS06
- LED334 pad 3: RGB_SW05 -> RGB_SW11
- LED334 pad 4: RGB_RED10 -> RGB_RED04
- LED334 pad 5: RGB_SW05 -> RGB_SW11
- LED334 pad 6: RGB_CS11 -> RGB_CS05
- LED335 pad 1: RGB_SW05 -> RGB_SW01
- LED335 pad 2: RGB_CS09 -> RGB_CS06
- LED335 pad 3: RGB_SW05 -> RGB_SW01
- LED335 pad 4: RGB_RED07 -> RGB_RED04
- LED335 pad 5: RGB_SW05 -> RGB_SW01
- LED335 pad 6: RGB_CS08 -> RGB_CS05
- LED336 pad 1: RGB_SW05 -> RGB_SW02
- LED336 pad 3: RGB_SW05 -> RGB_SW02
- LED336 pad 5: RGB_SW05 -> RGB_SW02
- LED337 pad 1: RGB_SW05 -> RGB_SW02
- LED337 pad 2: RGB_CS03 -> RGB_CS18
- LED337 pad 3: RGB_SW05 -> RGB_SW02
- LED337 pad 4: RGB_RED01 -> RGB_RED16
- LED337 pad 5: RGB_SW05 -> RGB_SW02
- LED337 pad 6: RGB_CS02 -> RGB_CS17
- LED338 pad 1: RGB_SW04 -> RGB_SW03
- LED338 pad 2: RGB_CS18 -> RGB_CS06
- LED338 pad 3: RGB_SW04 -> RGB_SW03
- LED338 pad 4: RGB_RED16 -> RGB_RED04
- LED338 pad 5: RGB_SW04 -> RGB_SW03
- LED338 pad 6: RGB_CS17 -> RGB_CS05
- LED339 pad 2: RGB_CS15 -> RGB_CS06
- LED339 pad 4: RGB_RED13 -> RGB_RED04
- LED339 pad 6: RGB_CS14 -> RGB_CS05
- LED340 pad 1: RGB_SW04 -> RGB_SW05
- LED340 pad 2: RGB_CS12 -> RGB_CS06
- LED340 pad 3: RGB_SW04 -> RGB_SW05
- LED340 pad 4: RGB_RED10 -> RGB_RED04
- LED340 pad 5: RGB_SW04 -> RGB_SW05
- LED340 pad 6: RGB_CS11 -> RGB_CS05
- LED341 pad 1: RGB_SW04 -> RGB_SW06
- LED341 pad 2: RGB_CS09 -> RGB_CS18
- LED341 pad 3: RGB_SW04 -> RGB_SW06
- LED341 pad 4: RGB_RED07 -> RGB_RED16
- LED341 pad 5: RGB_SW04 -> RGB_SW06
- LED341 pad 6: RGB_CS08 -> RGB_CS17
- LED342 pad 1: RGB_SW04 -> RGB_SW06
- LED342 pad 3: RGB_SW04 -> RGB_SW06
- LED342 pad 5: RGB_SW04 -> RGB_SW06
- LED343 pad 1: RGB_SW04 -> RGB_SW07
- LED343 pad 2: RGB_CS03 -> RGB_CS06
- LED343 pad 3: RGB_SW04 -> RGB_SW07
- LED343 pad 4: RGB_RED01 -> RGB_RED04
- LED343 pad 5: RGB_SW04 -> RGB_SW07
- LED343 pad 6: RGB_CS02 -> RGB_CS05
- LED344 pad 1: RGB_SW03 -> RGB_SW08
- LED344 pad 2: RGB_CS18 -> RGB_CS06
- LED344 pad 3: RGB_SW03 -> RGB_SW08
- LED344 pad 4: RGB_RED16 -> RGB_RED04
- LED344 pad 5: RGB_SW03 -> RGB_SW08
- LED344 pad 6: RGB_CS17 -> RGB_CS05
- LED345 pad 1: RGB_SW03 -> RGB_SW09
- LED345 pad 2: RGB_CS15 -> RGB_CS06
- LED345 pad 3: RGB_SW03 -> RGB_SW09
- LED345 pad 4: RGB_RED13 -> RGB_RED04
- LED345 pad 5: RGB_SW03 -> RGB_SW09
- LED345 pad 6: RGB_CS14 -> RGB_CS05
- LED346 pad 1: RGB_SW03 -> RGB_SW10
- LED346 pad 2: RGB_CS12 -> RGB_CS18
- LED346 pad 3: RGB_SW03 -> RGB_SW10
- LED346 pad 4: RGB_RED10 -> RGB_RED16
- LED346 pad 5: RGB_SW03 -> RGB_SW10
- LED346 pad 6: RGB_CS11 -> RGB_CS17
- LED347 pad 1: RGB_SW03 -> RGB_SW10
- LED347 pad 2: RGB_CS09 -> RGB_CS06
- LED347 pad 3: RGB_SW03 -> RGB_SW10
- LED347 pad 4: RGB_RED07 -> RGB_RED04
- LED347 pad 5: RGB_SW03 -> RGB_SW10
- LED347 pad 6: RGB_CS08 -> RGB_CS05
- LED348 pad 1: RGB_SW05 -> RGB_SW11
- LED348 pad 2: RGB_CS15 -> RGB_CS09
- LED348 pad 3: RGB_SW05 -> RGB_SW11
- LED348 pad 4: RGB_RED13 -> RGB_RED07
- LED348 pad 5: RGB_SW05 -> RGB_SW11
- LED348 pad 6: RGB_CS14 -> RGB_CS08
- LED349 pad 1: RGB_SW05 -> RGB_SW01
- LED349 pad 2: RGB_CS18 -> RGB_CS09
- LED349 pad 3: RGB_SW05 -> RGB_SW01
- LED349 pad 4: RGB_RED16 -> RGB_RED07
- LED349 pad 5: RGB_SW05 -> RGB_SW01
- LED349 pad 6: RGB_CS17 -> RGB_CS08
- LED350 pad 1: RGB_SW06 -> RGB_SW02
- LED350 pad 2: RGB_CS03 -> RGB_CS09
- LED350 pad 3: RGB_SW06 -> RGB_SW02
- LED350 pad 4: RGB_RED01 -> RGB_RED07
- LED350 pad 5: RGB_SW06 -> RGB_SW02
- LED350 pad 6: RGB_CS02 -> RGB_CS08
- LED351 pad 1: RGB_SW06 -> RGB_SW03
- LED351 pad 2: RGB_CS06 -> RGB_CS09
- LED351 pad 3: RGB_SW06 -> RGB_SW03
- LED351 pad 4: RGB_RED04 -> RGB_RED07
- LED351 pad 5: RGB_SW06 -> RGB_SW03
- LED351 pad 6: RGB_CS05 -> RGB_CS08
- LED352 pad 1: RGB_SW06 -> RGB_SW03
- LED352 pad 2: RGB_CS09 -> RGB_CS18
- LED352 pad 3: RGB_SW06 -> RGB_SW03
- LED352 pad 4: RGB_RED07 -> RGB_RED16
- LED352 pad 5: RGB_SW06 -> RGB_SW03
- LED352 pad 6: RGB_CS08 -> RGB_CS17
- LED353 pad 1: RGB_SW06 -> RGB_SW04
- LED353 pad 2: RGB_CS12 -> RGB_CS09
- LED353 pad 3: RGB_SW06 -> RGB_SW04
- LED353 pad 4: RGB_RED10 -> RGB_RED07
- LED353 pad 5: RGB_SW06 -> RGB_SW04
- LED353 pad 6: RGB_CS11 -> RGB_CS08
- LED354 pad 1: RGB_SW06 -> RGB_SW05
- LED354 pad 2: RGB_CS15 -> RGB_CS09
- LED354 pad 3: RGB_SW06 -> RGB_SW05
- LED354 pad 4: RGB_RED13 -> RGB_RED07
- LED354 pad 5: RGB_SW06 -> RGB_SW05
- LED354 pad 6: RGB_CS14 -> RGB_CS08
- LED355 pad 2: RGB_CS18 -> RGB_CS09
- LED355 pad 4: RGB_RED16 -> RGB_RED07
- LED355 pad 6: RGB_CS17 -> RGB_CS08
- LED356 pad 2: RGB_CS03 -> RGB_CS18
- LED356 pad 4: RGB_RED01 -> RGB_RED16
- LED356 pad 6: RGB_CS02 -> RGB_CS17
- LED357 pad 2: RGB_CS06 -> RGB_CS09
- LED357 pad 4: RGB_RED04 -> RGB_RED07
- LED357 pad 6: RGB_CS05 -> RGB_CS08
- LED358 pad 1: RGB_SW07 -> RGB_SW08
- LED358 pad 3: RGB_SW07 -> RGB_SW08
- LED358 pad 5: RGB_SW07 -> RGB_SW08
- LED359 pad 1: RGB_SW07 -> RGB_SW09
- LED359 pad 2: RGB_CS12 -> RGB_CS09
- LED359 pad 3: RGB_SW07 -> RGB_SW09
- LED359 pad 4: RGB_RED10 -> RGB_RED07
- LED359 pad 5: RGB_SW07 -> RGB_SW09
- LED359 pad 6: RGB_CS11 -> RGB_CS08
- LED360 pad 1: RGB_SW07 -> RGB_SW10
- LED360 pad 2: RGB_CS15 -> RGB_CS09
- LED360 pad 3: RGB_SW07 -> RGB_SW10
- LED360 pad 4: RGB_RED13 -> RGB_RED07
- LED360 pad 5: RGB_SW07 -> RGB_SW10
- LED360 pad 6: RGB_CS14 -> RGB_CS08
- LED361 pad 1: RGB_SW09 -> RGB_SW11
- LED361 pad 2: RGB_CS18 -> RGB_CS12
- LED361 pad 3: RGB_SW09 -> RGB_SW11
- LED361 pad 4: RGB_RED16 -> RGB_RED10
- LED361 pad 5: RGB_SW09 -> RGB_SW11
- LED361 pad 6: RGB_CS17 -> RGB_CS11
- LED362 pad 1: RGB_SW09 -> RGB_SW01
- LED362 pad 2: RGB_CS15 -> RGB_CS12
- LED362 pad 3: RGB_SW09 -> RGB_SW01
- LED362 pad 4: RGB_RED13 -> RGB_RED10
- LED362 pad 5: RGB_SW09 -> RGB_SW01
- LED362 pad 6: RGB_CS14 -> RGB_CS11
- LED363 pad 1: RGB_SW09 -> RGB_SW02
- LED363 pad 3: RGB_SW09 -> RGB_SW02
- LED363 pad 5: RGB_SW09 -> RGB_SW02
- LED364 pad 1: RGB_SW09 -> RGB_SW03
- LED364 pad 2: RGB_CS09 -> RGB_CS12
- LED364 pad 3: RGB_SW09 -> RGB_SW03
- LED364 pad 4: RGB_RED07 -> RGB_RED10
- LED364 pad 5: RGB_SW09 -> RGB_SW03
- LED364 pad 6: RGB_CS08 -> RGB_CS11
- LED365 pad 1: RGB_SW09 -> RGB_SW04
- LED365 pad 2: RGB_CS06 -> RGB_CS12
- LED365 pad 3: RGB_SW09 -> RGB_SW04
- LED365 pad 4: RGB_RED04 -> RGB_RED10
- LED365 pad 5: RGB_SW09 -> RGB_SW04
- LED365 pad 6: RGB_CS05 -> RGB_CS11
- LED366 pad 1: RGB_SW09 -> RGB_SW05
- LED366 pad 2: RGB_CS03 -> RGB_CS18
- LED366 pad 3: RGB_SW09 -> RGB_SW05
- LED366 pad 4: RGB_RED01 -> RGB_RED16
- LED366 pad 5: RGB_SW09 -> RGB_SW05
- LED366 pad 6: RGB_CS02 -> RGB_CS17
- LED367 pad 1: RGB_SW08 -> RGB_SW05
- LED367 pad 2: RGB_CS18 -> RGB_CS12
- LED367 pad 3: RGB_SW08 -> RGB_SW05
- LED367 pad 4: RGB_RED16 -> RGB_RED10
- LED367 pad 5: RGB_SW08 -> RGB_SW05
- LED367 pad 6: RGB_CS17 -> RGB_CS11
- LED368 pad 1: RGB_SW08 -> RGB_SW06
- LED368 pad 2: RGB_CS15 -> RGB_CS12
- LED368 pad 3: RGB_SW08 -> RGB_SW06
- LED368 pad 4: RGB_RED13 -> RGB_RED10
- LED368 pad 5: RGB_SW08 -> RGB_SW06
- LED368 pad 6: RGB_CS14 -> RGB_CS11
- LED369 pad 1: RGB_SW08 -> RGB_SW07
- LED369 pad 3: RGB_SW08 -> RGB_SW07
- LED369 pad 5: RGB_SW08 -> RGB_SW07
- LED370 pad 2: RGB_CS09 -> RGB_CS12
- LED370 pad 4: RGB_RED07 -> RGB_RED10
- LED370 pad 6: RGB_CS08 -> RGB_CS11
- LED371 pad 1: RGB_SW08 -> RGB_SW09
- LED371 pad 2: RGB_CS06 -> RGB_CS18
- LED371 pad 3: RGB_SW08 -> RGB_SW09
- LED371 pad 4: RGB_RED04 -> RGB_RED16
- LED371 pad 5: RGB_SW08 -> RGB_SW09
- LED371 pad 6: RGB_CS05 -> RGB_CS17
- LED372 pad 1: RGB_SW08 -> RGB_SW09
- LED372 pad 2: RGB_CS03 -> RGB_CS12
- LED372 pad 3: RGB_SW08 -> RGB_SW09
- LED372 pad 4: RGB_RED01 -> RGB_RED10
- LED372 pad 5: RGB_SW08 -> RGB_SW09
- LED372 pad 6: RGB_CS02 -> RGB_CS11
- LED373 pad 1: RGB_SW07 -> RGB_SW10
- LED373 pad 2: RGB_CS18 -> RGB_CS12
- LED373 pad 3: RGB_SW07 -> RGB_SW10
- LED373 pad 4: RGB_RED16 -> RGB_RED10
- LED373 pad 5: RGB_SW07 -> RGB_SW10
- LED373 pad 6: RGB_CS17 -> RGB_CS11
- LED374 pad 1: RGB_SW10 -> RGB_SW11
- LED374 pad 2: RGB_CS03 -> RGB_CS15
- LED374 pad 3: RGB_SW10 -> RGB_SW11
- LED374 pad 4: RGB_RED01 -> RGB_RED13
- LED374 pad 5: RGB_SW10 -> RGB_SW11
- LED374 pad 6: RGB_CS02 -> RGB_CS14
- LED375 pad 1: RGB_SW10 -> RGB_SW01
- LED375 pad 2: RGB_CS06 -> RGB_CS15
- LED375 pad 3: RGB_SW10 -> RGB_SW01
- LED375 pad 4: RGB_RED04 -> RGB_RED13
- LED375 pad 5: RGB_SW10 -> RGB_SW01
- LED375 pad 6: RGB_CS05 -> RGB_CS14
- LED376 pad 1: RGB_SW10 -> RGB_SW02
- LED376 pad 2: RGB_CS09 -> RGB_CS15
- LED376 pad 3: RGB_SW10 -> RGB_SW02
- LED376 pad 4: RGB_RED07 -> RGB_RED13
- LED376 pad 5: RGB_SW10 -> RGB_SW02
- LED376 pad 6: RGB_CS08 -> RGB_CS14
- LED377 pad 1: RGB_SW10 -> RGB_SW03
- LED377 pad 2: RGB_CS12 -> RGB_CS15
- LED377 pad 3: RGB_SW10 -> RGB_SW03
- LED377 pad 4: RGB_RED10 -> RGB_RED13
- LED377 pad 5: RGB_SW10 -> RGB_SW03
- LED377 pad 6: RGB_CS11 -> RGB_CS14
- LED378 pad 1: RGB_SW10 -> RGB_SW04
- LED378 pad 3: RGB_SW10 -> RGB_SW04
- LED378 pad 5: RGB_SW10 -> RGB_SW04
- LED379 pad 1: RGB_SW10 -> RGB_SW05
- LED379 pad 2: RGB_CS18 -> RGB_CS15
- LED379 pad 3: RGB_SW10 -> RGB_SW05
- LED379 pad 4: RGB_RED16 -> RGB_RED13
- LED379 pad 5: RGB_SW10 -> RGB_SW05
- LED379 pad 6: RGB_CS17 -> RGB_CS14
- LED380 pad 1: RGB_SW11 -> RGB_SW06
- LED380 pad 2: RGB_CS03 -> RGB_CS15
- LED380 pad 3: RGB_SW11 -> RGB_SW06
- LED380 pad 4: RGB_RED01 -> RGB_RED13
- LED380 pad 5: RGB_SW11 -> RGB_SW06
- LED380 pad 6: RGB_CS02 -> RGB_CS14
- LED381 pad 1: RGB_SW11 -> RGB_SW07
- LED381 pad 2: RGB_CS06 -> RGB_CS15
- LED381 pad 3: RGB_SW11 -> RGB_SW07
- LED381 pad 4: RGB_RED04 -> RGB_RED13
- LED381 pad 5: RGB_SW11 -> RGB_SW07
- LED381 pad 6: RGB_CS05 -> RGB_CS14
- LED382 pad 1: RGB_SW11 -> RGB_SW08
- LED382 pad 2: RGB_CS09 -> RGB_CS15
- LED382 pad 3: RGB_SW11 -> RGB_SW08
- LED382 pad 4: RGB_RED07 -> RGB_RED13
- LED382 pad 5: RGB_SW11 -> RGB_SW08
- LED382 pad 6: RGB_CS08 -> RGB_CS14
- LED383 pad 1: RGB_SW11 -> RGB_SW09
- LED383 pad 2: RGB_CS12 -> RGB_CS15
- LED383 pad 3: RGB_SW11 -> RGB_SW09
- LED383 pad 4: RGB_RED10 -> RGB_RED13
- LED383 pad 5: RGB_SW11 -> RGB_SW09
- LED383 pad 6: RGB_CS11 -> RGB_CS14
- LED384 pad 1: RGB_SW11 -> RGB_SW10
- LED384 pad 3: RGB_SW11 -> RGB_SW10
- LED384 pad 5: RGB_SW11 -> RGB_SW10
Routing:
- net RGB_SW10: track 147.0 -> 44.0 mm
- net RGB_SW11: track 109.0 -> 28.0 mm
- net RGB_SW09: track 120.1 -> 60.1 mm
- net RGB_SW02: track 115.0 -> 61.8 mm
- net RGB_SW08: track 113.2 -> 60.1 mm
- net RGB_SW04: track 113.9 -> 61.2 mm
- net RGB_SW06: track 113.7 -> 61.7 mm
- net RGB_SW01: track 115.2 -> 68.1 mm
- net RGB_SW05: track 100.1 -> 56.8 mm
- net RGB_SW07: track 99.5 -> 60.4 mm
- net RGB_SW03: track 100.4 -> 65.3 mm

Commit message: keep routing
Parts:
- moved TPK6 49.1 mm to (285.8, 15.9)
- moved TPK5 35.3 mm to (278.4, 30.2)
- moved TPK4 31.7 mm to (280.2, 29.2)
- moved TPK3 28.8 mm to (280.0, 31.6)
- moved TPK2 25.2 mm to (281.8, 30.6)
- moved R330 7.22 mm to (289.2, 8.30), turned to 0 degrees
- moved R333 6.67 mm to (289.2, 11.3), turned to 0 degrees
- moved R331 6.48 mm to (289.2, 9.80), turned to 0 degrees
- moved R332 5.61 mm to (289.2, 12.8), turned to 180 degrees
- moved R335 1.68 mm to (286.9, 13.6)
- moved C326 0.81 mm to (289.2, 14.3), turned to 180 degrees
Routing:
- net RGB_RED01: track 0.00 -> 63.9 mm, vias 0 -> 1
- net RGB_CS02: track 1.53 -> 43.0 mm, vias 1 -> 2
- net RGB_CS03: track 2.10 -> 41.1 mm, vias 1 -> 2
- net RGB_SW06: track 61.7 -> 29.5 mm
- net RGB_SW02: track 61.8 -> 30.8 mm
- net RGB_CS06: track 1.70 -> 27.9 mm
- net RGB_SW03: track 65.3 -> 40.7 mm
- net RGB_RED04: track 0.00 -> 24.3 mm, vias 0 -> 1
- net RGB_SW10: track 44.0 -> 21.0 mm
- net RGB_CS05: track 1.84 -> 23.5 mm
- net RGB_SW08: track 60.1 -> 39.5 mm
- net RGB_SW05: track 56.8 -> 36.1 mm
- net RGB_SW04: track 61.2 -> 40.6 mm
- net RGB_SDB: track 0.73 -> 20.6 mm, vias 1 -> 3
- net RGB_SW01: track 68.1 -> 50.9 mm
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