File: keyboard/12_keyboard_daughterboard.kicad_sch (KiCad schematic)
At the start: 134 parts, among them J320 Keyboard FFC: MX ULP 5x14 mat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, J321 DNP keyboard bring-up/debug, SW320 Esc 1u, SW321 1 1u, SW322 2 1u, SW323 3 1u, SW324 4 1u, SW325 5 1u, SW326 6 1u, SW327 7 1u, SW328 8 1u, SW329 9 1u, SW330 0 1u, SW331 Minus 1u, SW332 Equal 1u, SW333 Backspace 1.75u, SW334 Tab 1.25u, SW335 Q 1u, SW336 W 1u, SW337 E 1u, SW338 R 1u, SW339 T 1u, SW340 Y 1u, SW341 U 1u, SW342 I 1u, SW343 O 1u, SW344 P 1u, SW345 [ 1u, SW346 ] 1u, SW347 Backslash 1u, SW348 Caps 1.5u, SW349 A 1u, SW350 S 1u, SW351 D 1u, SW352 F 1u, SW353 G 1u, SW354 H 1u, SW355 J 1u, SW356 K 1u, SW357 L 1u, SW358 Semicolon 1u, SW359 Quote 1u, SW360 Enter 1.75u, SW361 Shift L 1.75u, SW362 Z 1u, SW363 X 1u, SW364 C 1u, SW365 V 1u, SW366 B 1u, SW367 N 1u, SW368 M 1u, SW369 Comma 1u, SW370 Period 1u, SW371 Slash 1u, SW372 Up 1u, SW373 Shift R 1.25u, SW374 Ctrl 1u, SW375 Fn 1u, SW376 Super 1u, SW377 Alt L 1u, SW378 Space L 2.25u, SW379 Space R 2.25u, SW380 Alt R 1u, SW381 Menu 1u, SW382 Left 1u, SW383 Down 1u, SW384 Right 1u

Commit message: add rgb to the keyboard and get it ready to route
Parts:
- removed J321: DNP keyboard bring-up/debug, Connector_PinHeader_2.54mm:PinHeader_1x04_P2.54mm_Vertical, symbol Connector_Generic:Conn_01x04
- added C322: 1u 25V RGB VCC, Capacitor_SMD:C_0603_1608Metric, symbol Device:C
- added C323: 100n 50V RGB VCC, Capacitor_SMD:C_0603_1608Metric, symbol Device:C
- added C324: 1u 25V RGB PVCC, Capacitor_SMD:C_0603_1608Metric, symbol Device:C
- added C325: 100n 50V RGB PVCC / buffer A, Capacitor_SMD:C_0603_1608Metric, symbol Device:C
- added C326: 100n 50V RGB startup delay, Capacitor_SMD:C_0603_1608Metric, symbol Device:C
- added LED320: RGB ESC, ducktop2:LED_Everlight_19-337_1616, symbol Keyboard_RGB:LED_19_337_C02
- added LED321: RGB 1, ducktop2:LED_Everlight_19-337_1616, symbol Keyboard_RGB:LED_19_337_C02
- added LED322: RGB 2, ducktop2:LED_Everlight_19-337_1616, symbol Keyboard_RGB:LED_19_337_C02
- added LED323: RGB 3, ducktop2:LED_Everlight_19-337_1616, symbol Keyboard_RGB:LED_19_337_C02
- added LED324: RGB 4, ducktop2:LED_Everlight_19-337_1616, symbol Keyboard_RGB:LED_19_337_C02
- added LED325: RGB 5, ducktop2:LED_Everlight_19-337_1616, symbol Keyboard_RGB:LED_19_337_C02
- added LED326: RGB 6, ducktop2:LED_Everlight_19-337_1616, symbol Keyboard_RGB:LED_19_337_C02
- added LED327: RGB 7, ducktop2:LED_Everlight_19-337_1616, symbol Keyboard_RGB:LED_19_337_C02
- added LED328: RGB 8, ducktop2:LED_Everlight_19-337_1616, symbol Keyboard_RGB:LED_19_337_C02
- added LED329: RGB 9, ducktop2:LED_Everlight_19-337_1616, symbol Keyboard_RGB:LED_19_337_C02
- added LED330: RGB 0, ducktop2:LED_Everlight_19-337_1616, symbol Keyboard_RGB:LED_19_337_C02
- added LED331: RGB MINUS, ducktop2:LED_Everlight_19-337_1616, symbol Keyboard_RGB:LED_19_337_C02
- added LED332: RGB EQUAL, ducktop2:LED_Everlight_19-337_1616, symbol Keyboard_RGB:LED_19_337_C02
- added LED333: RGB BKSP, ducktop2:LED_Everlight_19-337_1616, symbol Keyboard_RGB:LED_19_337_C02
- added LED334: RGB TAB, ducktop2:LED_Everlight_19-337_1616, symbol Keyboard_RGB:LED_19_337_C02
- added LED335: RGB Q, ducktop2:LED_Everlight_19-337_1616, symbol Keyboard_RGB:LED_19_337_C02
- added LED336: RGB W, ducktop2:LED_Everlight_19-337_1616, symbol Keyboard_RGB:LED_19_337_C02
- added LED337: RGB E, ducktop2:LED_Everlight_19-337_1616, symbol Keyboard_RGB:LED_19_337_C02
- added LED338: RGB R, ducktop2:LED_Everlight_19-337_1616, symbol Keyboard_RGB:LED_19_337_C02
- added LED339: RGB T, ducktop2:LED_Everlight_19-337_1616, symbol Keyboard_RGB:LED_19_337_C02
- added LED340: RGB Y, ducktop2:LED_Everlight_19-337_1616, symbol Keyboard_RGB:LED_19_337_C02
- added LED341: RGB U, ducktop2:LED_Everlight_19-337_1616, symbol Keyboard_RGB:LED_19_337_C02
- added LED342: RGB I, ducktop2:LED_Everlight_19-337_1616, symbol Keyboard_RGB:LED_19_337_C02
- added LED343: RGB O, ducktop2:LED_Everlight_19-337_1616, symbol Keyboard_RGB:LED_19_337_C02
- added LED344: RGB P, ducktop2:LED_Everlight_19-337_1616, symbol Keyboard_RGB:LED_19_337_C02
- added LED345: RGB LBRACKET, ducktop2:LED_Everlight_19-337_1616, symbol Keyboard_RGB:LED_19_337_C02
- added LED346: RGB RBRACKET, ducktop2:LED_Everlight_19-337_1616, symbol Keyboard_RGB:LED_19_337_C02
- added LED347: RGB BSLASH, ducktop2:LED_Everlight_19-337_1616, symbol Keyboard_RGB:LED_19_337_C02
- added LED348: RGB CAPS, ducktop2:LED_Everlight_19-337_1616, symbol Keyboard_RGB:LED_19_337_C02
- added LED349: RGB A, ducktop2:LED_Everlight_19-337_1616, symbol Keyboard_RGB:LED_19_337_C02
- added LED350: RGB S, ducktop2:LED_Everlight_19-337_1616, symbol Keyboard_RGB:LED_19_337_C02
- added LED351: RGB D, ducktop2:LED_Everlight_19-337_1616, symbol Keyboard_RGB:LED_19_337_C02
- added LED352: RGB F, ducktop2:LED_Everlight_19-337_1616, symbol Keyboard_RGB:LED_19_337_C02
- added LED353: RGB G, ducktop2:LED_Everlight_19-337_1616, symbol Keyboard_RGB:LED_19_337_C02
- added LED354: RGB H, ducktop2:LED_Everlight_19-337_1616, symbol Keyboard_RGB:LED_19_337_C02
- added LED355: RGB J, ducktop2:LED_Everlight_19-337_1616, symbol Keyboard_RGB:LED_19_337_C02
- added LED356: RGB K, ducktop2:LED_Everlight_19-337_1616, symbol Keyboard_RGB:LED_19_337_C02
- added LED357: RGB L, ducktop2:LED_Everlight_19-337_1616, symbol Keyboard_RGB:LED_19_337_C02
- added LED358: RGB SEMICOLON, ducktop2:LED_Everlight_19-337_1616, symbol Keyboard_RGB:LED_19_337_C02
- added LED359: RGB QUOTE, ducktop2:LED_Everlight_19-337_1616, symbol Keyboard_RGB:LED_19_337_C02
- added LED360: RGB ENTER, ducktop2:LED_Everlight_19-337_1616, symbol Keyboard_RGB:LED_19_337_C02
- added LED361: RGB LSHIFT, ducktop2:LED_Everlight_19-337_1616, symbol Keyboard_RGB:LED_19_337_C02
- added LED362: RGB Z, ducktop2:LED_Everlight_19-337_1616, symbol Keyboard_RGB:LED_19_337_C02
- added LED363: RGB X, ducktop2:LED_Everlight_19-337_1616, symbol Keyboard_RGB:LED_19_337_C02
- added LED364: RGB C, ducktop2:LED_Everlight_19-337_1616, symbol Keyboard_RGB:LED_19_337_C02
- added LED365: RGB V, ducktop2:LED_Everlight_19-337_1616, symbol Keyboard_RGB:LED_19_337_C02
- added LED366: RGB B, ducktop2:LED_Everlight_19-337_1616, symbol Keyboard_RGB:LED_19_337_C02
- added LED367: RGB N, ducktop2:LED_Everlight_19-337_1616, symbol Keyboard_RGB:LED_19_337_C02
- added LED368: RGB M, ducktop2:LED_Everlight_19-337_1616, symbol Keyboard_RGB:LED_19_337_C02
- added LED369: RGB COMMA, ducktop2:LED_Everlight_19-337_1616, symbol Keyboard_RGB:LED_19_337_C02
- added LED370: RGB PERIOD, ducktop2:LED_Everlight_19-337_1616, symbol Keyboard_RGB:LED_19_337_C02
- added LED371: RGB SLASH, ducktop2:LED_Everlight_19-337_1616, symbol Keyboard_RGB:LED_19_337_C02
- added LED372: RGB UP, ducktop2:LED_Everlight_19-337_1616, symbol Keyboard_RGB:LED_19_337_C02
- added LED373: RGB RSHIFT, ducktop2:LED_Everlight_19-337_1616, symbol Keyboard_RGB:LED_19_337_C02
- added LED374: RGB CTRL, ducktop2:LED_Everlight_19-337_1616, symbol Keyboard_RGB:LED_19_337_C02
- added LED375: RGB FN, ducktop2:LED_Everlight_19-337_1616, symbol Keyboard_RGB:LED_19_337_C02
- added LED376: RGB SUPER, ducktop2:LED_Everlight_19-337_1616, symbol Keyboard_RGB:LED_19_337_C02
- added LED377: RGB LALT, ducktop2:LED_Everlight_19-337_1616, symbol Keyboard_RGB:LED_19_337_C02
- added LED378: RGB SPACE_L, ducktop2:LED_Everlight_19-337_1616, symbol Keyboard_RGB:LED_19_337_C02
- added LED379: RGB SPACE_R, ducktop2:LED_Everlight_19-337_1616, symbol Keyboard_RGB:LED_19_337_C02
- added LED380: RGB RALT, ducktop2:LED_Everlight_19-337_1616, symbol Keyboard_RGB:LED_19_337_C02
- added LED381: RGB MENU, ducktop2:LED_Everlight_19-337_1616, symbol Keyboard_RGB:LED_19_337_C02
- added LED382: RGB LEFT, ducktop2:LED_Everlight_19-337_1616, symbol Keyboard_RGB:LED_19_337_C02
- added LED383: RGB DOWN, ducktop2:LED_Everlight_19-337_1616, symbol Keyboard_RGB:LED_19_337_C02
- added LED384: RGB RIGHT, ducktop2:LED_Everlight_19-337_1616, symbol Keyboard_RGB:LED_19_337_C02
- added R320: 33.2k 1% RGB current limit, Resistor_SMD:R_0603_1608Metric, symbol Device:R
- added R321: 2.2k RGB SCL pull-up, Resistor_SMD:R_0603_1608Metric, symbol Device:R
- added R322: 2.2k RGB SDA pull-up, Resistor_SMD:R_0603_1608Metric, symbol Device:R
- added R323: 100k RGB startup pull-up, Resistor_SMD:R_0603_1608Metric, symbol Device:R
- added R330, R331, R332, R333, R334, R335: 100R red-channel heat sharing, Resistor_SMD:R_0603_1608Metric, symbol Device:R
- added TPK1: KB_RGB_5V, TestPoint:TestPoint_Pad_D1.0mm, symbol Connector:TestPoint
- added TPK2: GND, TestPoint:TestPoint_Pad_D1.0mm, symbol Connector:TestPoint
- added TPK3: MCU_3V3, TestPoint:TestPoint_Pad_D1.0mm, symbol Connector:TestPoint
- added TPK4: RGB_SCL, TestPoint:TestPoint_Pad_D1.0mm, symbol Connector:TestPoint
- added TPK5: RGB_SDA, TestPoint:TestPoint_Pad_D1.0mm, symbol Connector:TestPoint
- added TPK6: RGB_SDB, TestPoint:TestPoint_Pad_D1.0mm, symbol Connector:TestPoint
- added U320: IS31FL3743A-QULS4-TR, ducktop2:IS31FL3743A_UQFN40, symbol Keyboard_RGB:IS31FL3743A
- added U321: TCA9517ADGKR, Package_SO:VSSOP-8_3x3mm_P0.65mm, symbol Keyboard_RGB:TCA9517A
- C320: value DNP 100n keyboard 3V3 reserve -> 100n 50V buffer 3V3; MPN (none) -> CL10B104KB8NNNC; Manufacturer (none) -> Samsung Electro-Mechanics; ReleasedRevA Not fitted; footprint omitted from manufactured PCB -> (none); now fitted; now in the parts list
- C321: value DNP 10u optional 5V/backlight -> 10u 25V RGB input bulk; footprint Capacitor_SMD:C_1206_3216Metric -> Capacitor_SMD:C_0805_2012Metric; MPN (none) -> CL21A106KAYNNNE; Manufacturer (none) -> Samsung Electro-Mechanics; ReleasedRevA Not fitted; footprint omitted from manufactured PCB -> (none); now fitted; now in the parts list
- J320: Assembly (none) -> connector MP hold-downs are mechanical and netless; ReleasedRevA Populated; connector MP hold-down pads are mechanical and n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 -> (none)
- SW320, SW321, SW322, SW323, SW324, SW325, SW326, SW327, SW328, SW329, SW330, SW331, SW332, SW333, SW334, SW335, SW336, SW337, SW338, SW339, SW340, SW341, SW342, SW343, SW344, SW345, SW346, SW347, SW348, SW349, SW350, SW351, SW352, SW353, SW354, SW355, SW356, SW357, SW358, SW359, SW360, SW361, SW362, SW363, SW364, SW365, SW366, SW367, SW368, SW369, SW370, SW371, SW372, SW373, SW374, SW375, SW376, SW377, SW378, SW379, SW380, SW381, SW382, SW383, SW384: Assembly customer assembly after diode and FFC assembly -> fit after LEDs, diodes, connector and support parts
Connections:
- net GND: now also C322.2, C323.2, C324.2, C325.2, C326.2, R320.2, TPK2.1, U320.16 (PGND), U320.23 (GND), U320.41 (EP), U321.4 (GND)
- net I2C_SCL: now also U321.7 (SCLB)
- net I2C_SDA: now also U321.6 (SDAB)
- net MCU_3V3: now also TPK3.1, U321.8 (VCCB)
- net KB_COL14: no longer names the net of J320.27 (Pin_27)
- net KB_COL15: no longer names the net of J320.28 (Pin_28)
- net KB_ROW5: no longer names the net of J320.10 (Pin_10)
- net KB_ROW6: no longer names the net of J320.11 (Pin_11)
- net KB_ROW7: no longer names the net of J320.12 (Pin_12)
- net SYS_5V renamed KB_RGB_5V
- net KB_RGB_5V: now also C322.1, C323.1, C324.1, C325.1, R321.1, R322.1, R323.1, TPK1.1, U320.22 (VCC), U320.24 (ADDR2), U320.25 (ADDR1), U320.5 (PVCC), U321.1 (VCCA), U321.5 (EN)
- new net RGB_CS01: R330.1, U320.39 (CS01)
- new net RGB_CS02: LED320.6 (G_K), LED326.6 (G_K), LED332.6 (G_K), LED337.6 (G_K), LED343.6 (G_K), LED350.6 (G_K), LED356.6 (G_K), LED366.6 (G_K), LED372.6 (G_K), LED374.6 (G_K), LED380.6 (G_K), U320.38 (CS02)
- new net RGB_CS03: LED320.2 (B_K), LED326.2 (B_K), LED332.2 (B_K), LED337.2 (B_K), LED343.2 (B_K), LED350.2 (B_K), LED356.2 (B_K), LED366.2 (B_K), LED372.2 (B_K), LED374.2 (B_K), LED380.2 (B_K), U320.37 (CS03)
- new net RGB_CS04: R331.1, U320.36 (CS04)
- new net RGB_CS05: LED321.6 (G_K), LED327.6 (G_K), LED333.6 (G_K), LED336.6 (G_K), LED342.6 (G_K), LED351.6 (G_K), LED357.6 (G_K), LED365.6 (G_K), LED371.6 (G_K), LED375.6 (G_K), LED381.6 (G_K), U320.35 (CS05)
- new net RGB_CS06: LED321.2 (B_K), LED327.2 (B_K), LED333.2 (B_K), LED336.2 (B_K), LED342.2 (B_K), LED351.2 (B_K), LED357.2 (B_K), LED365.2 (B_K), LED371.2 (B_K), LED375.2 (B_K), LED381.2 (B_K), U320.34 (CS06)
- new net RGB_CS07: R332.1, U320.33 (CS07)
- new net RGB_CS08: LED322.6 (G_K), LED328.6 (G_K), LED335.6 (G_K), LED341.6 (G_K), LED347.6 (G_K), LED352.6 (G_K), LED358.6 (G_K), LED364.6 (G_K), LED370.6 (G_K), LED376.6 (G_K), LED382.6 (G_K), U320.32 (CS08)
- new net RGB_CS09: LED322.2 (B_K), LED328.2 (B_K), LED335.2 (B_K), LED341.2 (B_K), LED347.2 (B_K), LED352.2 (B_K), LED358.2 (B_K), LED364.2 (B_K), LED370.2 (B_K), LED376.2 (B_K), LED382.2 (B_K), U320.31 (CS09)
- new net RGB_CS10: R333.1, U320.21 (CS10)
- new net RGB_CS11: LED323.6 (G_K), LED329.6 (G_K), LED334.6 (G_K), LED340.6 (G_K), LED346.6 (G_K), LED353.6 (G_K), LED359.6 (G_K), LED363.6 (G_K), LED369.6 (G_K), LED377.6 (G_K), LED383.6 (G_K), U320.20 (CS11)
- new net RGB_CS12: LED323.2 (B_K), LED329.2 (B_K), LED334.2 (B_K), LED340.2 (B_K), LED346.2 (B_K), LED353.2 (B_K), LED359.2 (B_K), LED363.2 (B_K), LED369.2 (B_K), LED377.2 (B_K), LED383.2 (B_K), U320.19 (CS12)
- new net RGB_CS13: R334.1, U320.18 (CS13)
- new net RGB_CS14: LED324.6 (G_K), LED330.6 (G_K), LED339.6 (G_K), LED345.6 (G_K), LED348.6 (G_K), LED354.6 (G_K), LED360.6 (G_K), LED362.6 (G_K), LED368.6 (G_K), LED378.6 (G_K), LED384.6 (G_K), U320.17 (CS14)
- new net RGB_CS15: LED324.2 (B_K), LED330.2 (B_K), LED339.2 (B_K), LED345.2 (B_K), LED348.2 (B_K), LED354.2 (B_K), LED360.2 (B_K), LED362.2 (B_K), LED368.2 (B_K), LED378.2 (B_K), LED384.2 (B_K), U320.15 (CS15)
- new net RGB_CS16: R335.1, U320.14 (CS16)
- new net RGB_CS17: LED325.6 (G_K), LED331.6 (G_K), LED338.6 (G_K), LED344.6 (G_K), LED349.6 (G_K), LED355.6 (G_K), LED361.6 (G_K), LED367.6 (G_K), LED373.6 (G_K), LED379.6 (G_K), U320.13 (CS17)
- new net RGB_CS18: LED325.2 (B_K), LED331.2 (B_K), LED338.2 (B_K), LED344.2 (B_K), LED349.2 (B_K), LED355.2 (B_K), LED361.2 (B_K), LED367.2 (B_K), LED373.2 (B_K), LED379.2 (B_K), U320.12 (CS18)
- new net RGB_ISET: R320.1, U320.29 (ISET)
- new net RGB_RED01: LED320.4 (R_K), LED326.4 (R_K), LED332.4 (R_K), LED337.4 (R_K), LED343.4 (R_K), LED350.4 (R_K), LED356.4 (R_K), LED366.4 (R_K), LED372.4 (R_K), LED374.4 (R_K), LED380.4 (R_K), R330.2
- new net RGB_RED04: LED321.4 (R_K), LED327.4 (R_K), LED333.4 (R_K), LED336.4 (R_K), LED342.4 (R_K), LED351.4 (R_K), LED357.4 (R_K), LED365.4 (R_K), LED371.4 (R_K), LED375.4 (R_K), LED381.4 (R_K), R331.2
- new net RGB_RED07: LED322.4 (R_K), LED328.4 (R_K), LED335.4 (R_K), LED341.4 (R_K), LED347.4 (R_K), LED352.4 (R_K), LED358.4 (R_K), LED364.4 (R_K), LED370.4 (R_K), LED376.4 (R_K), LED382.4 (R_K), R332.2
- new net RGB_RED10: LED323.4 (R_K), LED329.4 (R_K), LED334.4 (R_K), LED340.4 (R_K), LED346.4 (R_K), LED353.4 (R_K), LED359.4 (R_K), LED363.4 (R_K), LED369.4 (R_K), LED377.4 (R_K), LED383.4 (R_K), R333.2
- new net RGB_RED13: LED324.4 (R_K), LED330.4 (R_K), LED339.4 (R_K), LED345.4 (R_K), LED348.4 (R_K), LED354.4 (R_K), LED360.4 (R_K), LED362.4 (R_K), LED368.4 (R_K), LED378.4 (R_K), LED384.4 (R_K), R334.2
- new net RGB_RED16: LED325.4 (R_K), LED331.4 (R_K), LED338.4 (R_K), LED344.4 (R_K), LED349.4 (R_K), LED355.4 (R_K), LED361.4 (R_K), LED367.4 (R_K), LED373.4 (R_K), LED379.4 (R_K), R335.2
- new net RGB_SCL: R321.2, TPK4.1, U320.27 (SCL), U321.2 (SCLA)
- new net RGB_SDA: R322.2, TPK5.1, U320.28 (SDA), U321.3 (SDAA)
- new net RGB_SDB: C326.1, R323.2, TPK6.1, U320.26 (SDB)
- new net RGB_SW01: LED320.1 (B_A), LED320.3 (R_A), LED320.5 (G_A), LED321.1 (B_A), LED321.3 (R_A), LED321.5 (G_A), LED322.1 (B_A), LED322.3 (R_A), LED322.5 (G_A), LED323.1 (B_A), LED323.3 (R_A), LED323.5 (G_A), LED324.1 (B_A), LED324.3 (R_A), LED324.5 (G_A), LED325.1 (B_A), LED325.3 (R_A), LED325.5 (G_A), U320.6 (SW01)
- new net RGB_SW02: LED326.1 (B_A), LED326.3 (R_A), LED326.5 (G_A), LED327.1 (B_A), LED327.3 (R_A), LED327.5 (G_A), LED328.1 (B_A), LED328.3 (R_A), LED328.5 (G_A), LED329.1 (B_A), LED329.3 (R_A), LED329.5 (G_A), LED330.1 (B_A), LED330.3 (R_A), LED330.5 (G_A), LED331.1 (B_A), LED331.3 (R_A), LED331.5 (G_A), U320.4 (SW02)
- new net RGB_SW03: LED332.1 (B_A), LED332.3 (R_A), LED332.5 (G_A), LED333.1 (B_A), LED333.3 (R_A), LED333.5 (G_A), LED344.1 (B_A), LED344.3 (R_A), LED344.5 (G_A), LED345.1 (B_A), LED345.3 (R_A), LED345.5 (G_A), LED346.1 (B_A), LED346.3 (R_A), LED346.5 (G_A), LED347.1 (B_A), LED347.3 (R_A), LED347.5 (G_A), U320.7 (SW03)
- new net RGB_SW04: LED338.1 (B_A), LED338.3 (R_A), LED338.5 (G_A), LED339.1 (B_A), LED339.3 (R_A), LED339.5 (G_A), LED340.1 (B_A), LED340.3 (R_A), LED340.5 (G_A), LED341.1 (B_A), LED341.3 (R_A), LED341.5 (G_A), LED342.1 (B_A), LED342.3 (R_A), LED342.5 (G_A), LED343.1 (B_A), LED343.3 (R_A), LED343.5 (G_A), U320.3 (SW04)
- new net RGB_SW05: LED334.1 (B_A), LED334.3 (R_A), LED334.5 (G_A), LED335.1 (B_A), LED335.3 (R_A), LED335.5 (G_A), LED336.1 (B_A), LED336.3 (R_A), LED336.5 (G_A), LED337.1 (B_A), LED337.3 (R_A), LED337.5 (G_A), LED348.1 (B_A), LED348.3 (R_A), LED348.5 (G_A), LED349.1 (B_A), LED349.3 (R_A), LED349.5 (G_A), U320.8 (SW05)
- new net RGB_SW06: LED350.1 (B_A), LED350.3 (R_A), LED350.5 (G_A), LED351.1 (B_A), LED351.3 (R_A), LED351.5 (G_A), LED352.1 (B_A), LED352.3 (R_A), LED352.5 (G_A), LED353.1 (B_A), LED353.3 (R_A), LED353.5 (G_A), LED354.1 (B_A), LED354.3 (R_A), LED354.5 (G_A), LED355.1 (B_A), LED355.3 (R_A), LED355.5 (G_A), U320.2 (SW06)
- new net RGB_SW07: LED356.1 (B_A), LED356.3 (R_A), LED356.5 (G_A), LED357.1 (B_A), LED357.3 (R_A), LED357.5 (G_A), LED358.1 (B_A), LED358.3 (R_A), LED358.5 (G_A), LED359.1 (B_A), LED359.3 (R_A), LED359.5 (G_A), LED360.1 (B_A), LED360.3 (R_A), LED360.5 (G_A), LED373.1 (B_A), LED373.3 (R_A), LED373.5 (G_A), U320.9 (SW07)
- new net RGB_SW08: LED367.1 (B_A), LED367.3 (R_A), LED367.5 (G_A), LED368.1 (B_A), LED368.3 (R_A), LED368.5 (G_A), LED369.1 (B_A), LED369.3 (R_A), LED369.5 (G_A), LED370.1 (B_A), LED370.3 (R_A), LED370.5 (G_A), LED371.1 (B_A), LED371.3 (R_A), LED371.5 (G_A), LED372.1 (B_A), LED372.3 (R_A), LED372.5 (G_A), U320.1 (SW08)
- new net RGB_SW09: LED361.1 (B_A), LED361.3 (R_A), LED361.5 (G_A), LED362.1 (B_A), LED362.3 (R_A), LED362.5 (G_A), LED363.1 (B_A), LED363.3 (R_A), LED363.5 (G_A), LED364.1 (B_A), LED364.3 (R_A), LED364.5 (G_A), LED365.1 (B_A), LED365.3 (R_A), LED365.5 (G_A), LED366.1 (B_A), LED366.3 (R_A), LED366.5 (G_A), U320.10 (SW09)
- new net RGB_SW10: LED374.1 (B_A), LED374.3 (R_A), LED374.5 (G_A), LED375.1 (B_A), LED375.3 (R_A), LED375.5 (G_A), LED376.1 (B_A), LED376.3 (R_A), LED376.5 (G_A), LED377.1 (B_A), LED377.3 (R_A), LED377.5 (G_A), LED378.1 (B_A), LED378.3 (R_A), LED378.5 (G_A), LED379.1 (B_A), LED379.3 (R_A), LED379.5 (G_A), U320.40 (SW10)
- new net RGB_SW11: LED380.1 (B_A), LED380.3 (R_A), LED380.5 (G_A), LED381.1 (B_A), LED381.3 (R_A), LED381.5 (G_A), LED382.1 (B_A), LED382.3 (R_A), LED382.5 (G_A), LED383.1 (B_A), LED383.3 (R_A), LED383.5 (G_A), LED384.1 (B_A), LED384.3 (R_A), LED384.5 (G_A), U320.11 (SW11)
- no-connect marks 1 -> 7
Other:
- note added: "ADDR1/ADDR2 at VCC select 7-bit address 0x2F. SDB rises through R323/C326; wait 20 ms before setup."
- note added: "Each group has up to six nearby keys. Follow the RGB_SW and RGB_CS labels when routing."
- note added: "Everlight 19-337/R6GHBHC-C02/2T, 1.6 x 1.6 x 0.35 mm; LEDs are fitted before the switches."
- note added: "Fit LEDs and support parts before the MX ULP switches. Follow CHERRY's assembly process and check a first article."
- note added: "J320 mirrors mainboard J310. Fit mainboard R387 for the RGB I2C buffer; keep R386 absent so the 5 V current limit cannot be bypassed."
- note added: "J320 pin 29 is the switched 5 V rail. Pin 2 needs mainboard R387 fitted for the I2C buffer."
- note added: "Keep C322/C323 close to VCC, C324/C325 close to PVCC, and R320 close to ISET. Connect the exposed pad to ground."
- note added: "R320 limits peak sink current to about 11.3 mA at the datasheet corner: 18 active sinks stay below the cable budget."
- note added: "RGB revision: same 273.5 x 80.0 mm outline, key positions and active matrix contacts."
- note added: "The split space layout is unchanged. Check the large keycaps and stabilizers with the actual switch/plate stack."
- note added: "U321 A side is switched 5 V; B side is 3.3 V. Its power-off isolation keeps the unpowered LED driver off the EC bus."
- note added: "keyboard rgb: 65 separate colours, hardware-limited current"
- note removed: "J320 mirrors mainboard J310. Its MP hold-down pads are intentionally netless on manufactured Rev A; C320/C321/J321 are DNP and excluded from that PCB."
- note removed: "Keyboard envelope is 273.5 x 80.0 mm; corrected candidate retains the rev A population and connector contract."
- note removed: "MX ULP hotswap is not planned: use stencil + reflow/hot plate for production and validate rework on a small coupon first."
- note removed: "Use split space in rev A. Treat Backspace, Enter, left Shift, and both Space keys as mechanical stabilizer/keycap-risk items before full board release."
- moved on the sheet: D320, D321, D322, D323, D324, D325, D326, D327, D328, D329, D330, D331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

Commit message: sort out the keyboard leds and fix more bms routing
Parts:
- LED320: RGB_bank 1 -> 11
- LED323: RGB_bank 1 -> 2
- LED324: RGB_bank 1 -> 3
- LED325: RGB_bank 1 -> 4
- LED326: RGB_bank 2 -> 4
- LED327: RGB_bank 2 -> 5
- LED328: RGB_bank 2 -> 6
- LED329: RGB_bank 2 -> 7
- LED330, LED331: RGB_bank 2 -> 8
- LED332, LED345: RGB_bank 3 -> 9
- LED333, LED346, LED347: RGB_bank 3 -> 10
- LED334, LED348: RGB_bank 5 -> 11
- LED335, LED349: RGB_bank 5 -> 1
- LED336, LED337: RGB_bank 5 -> 2
- LED338: RGB_bank 4 -> 3
- LED340: RGB_bank 4 -> 5
- LED341, LED342: RGB_bank 4 -> 6
- LED343: RGB_bank 4 -> 7
- LED344: RGB_bank 3 -> 8
- LED350: RGB_bank 6 -> 2
- LED351, LED352: RGB_bank 6 -> 3
- LED353: RGB_bank 6 -> 4
- LED354: RGB_bank 6 -> 5
- LED358: RGB_bank 7 -> 8
- LED359: RGB_bank 7 -> 9
- LED360, LED373: RGB_bank 7 -> 10
- LED361: RGB_bank 9 -> 11
- LED362: RGB_bank 9 -> 1
- LED363: RGB_bank 9 -> 2
- LED364: RGB_bank 9 -> 3
- LED365: RGB_bank 9 -> 4
- LED366: RGB_bank 9 -> 5
- LED367: RGB_bank 8 -> 5
- LED368: RGB_bank 8 -> 6
- LED369: RGB_bank 8 -> 7
- LED371, LED372: RGB_bank 8 -> 9
- LED374: RGB_bank 10 -> 11
- LED375: RGB_bank 10 -> 1
- LED376: RGB_bank 10 -> 2
- LED377: RGB_bank 10 -> 3
- LED378: RGB_bank 10 -> 4
- LED379: RGB_bank 10 -> 5
- LED380: RGB_bank 11 -> 6
- LED381: RGB_bank 11 -> 7
- LED382: RGB_bank 11 -> 8
- LED383: RGB_bank 11 -> 9
- LED384: RGB_bank 11 -> 10
Connections:
- net RGB_CS02: now also LED322.6 (G_K), LED323.6 (G_K), LED324.6 (G_K), LED325.6 (G_K), LED327.6 (G_K), LED328.6 (G_K), LED329.6 (G_K), LED331.6 (G_K), LED333.6 (G_K); no longer LED326.6 (G_K), LED337.6 (G_K), LED343.6 (G_K), LED350.6 (G_K), LED356.6 (G_K), LED366.6 (G_K), LED372.6 (G_K), LED374.6 (G_K), LED380.6 (G_K)
- net RGB_CS03: now also LED322.2 (B_K), LED323.2 (B_K), LED324.2 (B_K), LED325.2 (B_K), LED327.2 (B_K), LED328.2 (B_K), LED329.2 (B_K), LED331.2 (B_K), LED333.2 (B_K); no longer LED326.2 (B_K), LED337.2 (B_K), LED343.2 (B_K), LED350.2 (B_K), LED356.2 (B_K), LED366.2 (B_K), LED372.2 (B_K), LED374.2 (B_K), LED380.2 (B_K)
- net RGB_CS05: now also LED334.6 (G_K), LED335.6 (G_K), LED338.6 (G_K), LED339.6 (G_K), LED340.6 (G_K), LED343.6 (G_K), LED344.6 (G_K), LED345.6 (G_K), LED347.6 (G_K); no longer LED321.6 (G_K), LED327.6 (G_K), LED333.6 (G_K), LED351.6 (G_K), LED357.6 (G_K), LED365.6 (G_K), LED371.6 (G_K), LED375.6 (G_K), LED381.6 (G_K)
- net RGB_CS06: now also LED334.2 (B_K), LED335.2 (B_K), LED338.2 (B_K), LED339.2 (B_K), LED340.2 (B_K), LED343.2 (B_K), LED344.2 (B_K), LED345.2 (B_K), LED347.2 (B_K); no longer LED321.2 (B_K), LED327.2 (B_K), LED333.2 (B_K), LED351.2 (B_K), LED357.2 (B_K), LED365.2 (B_K), LED371.2 (B_K), LED375.2 (B_K), LED381.2 (B_K)
- net RGB_CS08: now also LED348.6 (G_K), LED349.6 (G_K), LED350.6 (G_K), LED351.6 (G_K), LED353.6 (G_K), LED354.6 (G_K), LED355.6 (G_K), LED357.6 (G_K), LED359.6 (G_K), LED360.6 (G_K); no longer LED322.6 (G_K), LED328.6 (G_K), LED335.6 (G_K), LED341.6 (G_K), LED347.6 (G_K), LED352.6 (G_K), LED364.6 (G_K), LED370.6 (G_K), LED376.6 (G_K), LED382.6 (G_K)
- net RGB_CS09: now also LED348.2 (B_K), LED349.2 (B_K), LED350.2 (B_K), LED351.2 (B_K), LED353.2 (B_K), LED354.2 (B_K), LED355.2 (B_K), LED357.2 (B_K), LED359.2 (B_K), LED360.2 (B_K); no longer LED322.2 (B_K), LED328.2 (B_K), LED335.2 (B_K), LED341.2 (B_K), LED347.2 (B_K), LED352.2 (B_K), LED364.2 (B_K), LED370.2 (B_K), LED376.2 (B_K), LED382.2 (B_K)
- net RGB_CS11: now also LED361.6 (G_K), LED362.6 (G_K), LED364.6 (G_K), LED365.6 (G_K), LED367.6 (G_K), LED368.6 (G_K), LED370.6 (G_K), LED372.6 (G_K), LED373.6 (G_K); no longer LED323.6 (G_K), LED329.6 (G_K), LED334.6 (G_K), LED340.6 (G_K), LED346.6 (G_K), LED353.6 (G_K), LED359.6 (G_K), LED377.6 (G_K), LED383.6 (G_K)
- net RGB_CS12: now also LED361.2 (B_K), LED362.2 (B_K), LED364.2 (B_K), LED365.2 (B_K), LED367.2 (B_K), LED368.2 (B_K), LED370.2 (B_K), LED372.2 (B_K), LED373.2 (B_K); no longer LED323.2 (B_K), LED329.2 (B_K), LED334.2 (B_K), LED340.2 (B_K), LED346.2 (B_K), LED353.2 (B_K), LED359.2 (B_K), LED377.2 (B_K), LED383.2 (B_K)
- net RGB_CS14: now also LED374.6 (G_K), LED375.6 (G_K), LED376.6 (G_K), LED377.6 (G_K), LED379.6 (G_K), LED380.6 (G_K), LED381.6 (G_K), LED382.6 (G_K), LED383.6 (G_K); no longer LED324.6 (G_K), LED330.6 (G_K), LED339.6 (G_K), LED345.6 (G_K), LED348.6 (G_K), LED354.6 (G_K), LED360.6 (G_K), LED362.6 (G_K), LED368.6 (G_K)
- net RGB_CS15: now also LED374.2 (B_K), LED375.2 (B_K), LED376.2 (B_K), LED377.2 (B_K), LED379.2 (B_K), LED380.2 (B_K), LED381.2 (B_K), LED382.2 (B_K), LED383.2 (B_K); no longer LED324.2 (B_K), LED330.2 (B_K), LED339.2 (B_K), LED345.2 (B_K), LED348.2 (B_K), LED354.2 (B_K), LED360.2 (B_K), LED362.2 (B_K), LED368.2 (B_K)
- net RGB_CS17: now also LED321.6 (G_K), LED326.6 (G_K), LED330.6 (G_K), LED337.6 (G_K), LED341.6 (G_K), LED346.6 (G_K), LED352.6 (G_K), LED356.6 (G_K), LED366.6 (G_K), LED371.6 (G_K); no longer LED325.6 (G_K), LED331.6 (G_K), LED338.6 (G_K), LED344.6 (G_K), LED349.6 (G_K), LED355.6 (G_K), LED361.6 (G_K), LED367.6 (G_K), LED373.6 (G_K), LED379.6 (G_K)
- net RGB_CS18: now also LED321.2 (B_K), LED326.2 (B_K), LED330.2 (B_K), LED337.2 (B_K), LED341.2 (B_K), LED346.2 (B_K), LED352.2 (B_K), LED356.2 (B_K), LED366.2 (B_K), LED371.2 (B_K); no longer LED325.2 (B_K), LED331.2 (B_K), LED338.2 (B_K), LED344.2 (B_K), LED349.2 (B_K), LED355.2 (B_K), LED361.2 (B_K), LED367.2 (B_K), LED373.2 (B_K), LED379.2 (B_K)
- net RGB_RED01: now also LED322.4 (R_K), LED323.4 (R_K), LED324.4 (R_K), LED325.4 (R_K), LED327.4 (R_K), LED328.4 (R_K), LED329.4 (R_K), LED331.4 (R_K), LED333.4 (R_K); no longer LED326.4 (R_K), LED337.4 (R_K), LED343.4 (R_K), LED350.4 (R_K), LED356.4 (R_K), LED366.4 (R_K), LED372.4 (R_K), LED374.4 (R_K), LED380.4 (R_K)
- net RGB_RED04: now also LED334.4 (R_K), LED335.4 (R_K), LED338.4 (R_K), LED339.4 (R_K), LED340.4 (R_K), LED343.4 (R_K), LED344.4 (R_K), LED345.4 (R_K), LED347.4 (R_K); no longer LED321.4 (R_K), LED327.4 (R_K), LED333.4 (R_K), LED351.4 (R_K), LED357.4 (R_K), LED365.4 (R_K), LED371.4 (R_K), LED375.4 (R_K), LED381.4 (R_K)
- net RGB_RED07: now also LED348.4 (R_K), LED349.4 (R_K), LED350.4 (R_K), LED351.4 (R_K), LED353.4 (R_K), LED354.4 (R_K), LED355.4 (R_K), LED357.4 (R_K), LED359.4 (R_K), LED360.4 (R_K); no longer LED322.4 (R_K), LED328.4 (R_K), LED335.4 (R_K), LED341.4 (R_K), LED347.4 (R_K), LED352.4 (R_K), LED364.4 (R_K), LED370.4 (R_K), LED376.4 (R_K), LED382.4 (R_K)
- net RGB_RED10: now also LED361.4 (R_K), LED362.4 (R_K), LED364.4 (R_K), LED365.4 (R_K), LED367.4 (R_K), LED368.4 (R_K), LED370.4 (R_K), LED372.4 (R_K), LED373.4 (R_K); no longer LED323.4 (R_K), LED329.4 (R_K), LED334.4 (R_K), LED340.4 (R_K), LED346.4 (R_K), LED353.4 (R_K), LED359.4 (R_K), LED377.4 (R_K), LED383.4 (R_K)
- net RGB_RED13: now also LED374.4 (R_K), LED375.4 (R_K), LED376.4 (R_K), LED377.4 (R_K), LED379.4 (R_K), LED380.4 (R_K), LED381.4 (R_K), LED382.4 (R_K), LED383.4 (R_K); no longer LED324.4 (R_K), LED330.4 (R_K), LED339.4 (R_K), LED345.4 (R_K), LED348.4 (R_K), LED354.4 (R_K), LED360.4 (R_K), LED362.4 (R_K), LED368.4 (R_K)
- net RGB_RED16: now also LED321.4 (R_K), LED326.4 (R_K), LED330.4 (R_K), LED337.4 (R_K), LED341.4 (R_K), LED346.4 (R_K), LED352.4 (R_K), LED356.4 (R_K), LED366.4 (R_K), LED371.4 (R_K); no longer LED325.4 (R_K), LED331.4 (R_K), LED338.4 (R_K), LED344.4 (R_K), LED349.4 (R_K), LED355.4 (R_K), LED361.4 (R_K), LED367.4 (R_K), LED373.4 (R_K), LED379.4 (R_K)
- net RGB_SW01: now also LED335.1 (B_A), LED335.3 (R_A), LED335.5 (G_A), LED349.1 (B_A), LED349.3 (R_A), LED349.5 (G_A), LED362.1 (B_A), LED362.3 (R_A), LED362.5 (G_A), LED375.1 (B_A), LED375.3 (R_A), LED375.5 (G_A); no longer LED320.1 (B_A), LED320.3 (R_A), LED320.5 (G_A), LED323.1 (B_A), LED323.3 (R_A), LED323.5 (G_A), LED324.1 (B_A), LED324.3 (R_A), LED324.5 (G_A), LED325.1 (B_A), LED325.3 (R_A), LED325.5 (G_A)
- net RGB_SW02: now also LED323.1 (B_A), LED323.3 (R_A), LED323.5 (G_A), LED336.1 (B_A), LED336.3 (R_A), LED336.5 (G_A), LED337.1 (B_A), LED337.3 (R_A), LED337.5 (G_A), LED350.1 (B_A), LED350.3 (R_A), LED350.5 (G_A), LED363.1 (B_A), LED363.3 (R_A), LED363.5 (G_A), LED376.1 (B_A), LED376.3 (R_A), LED376.5 (G_A); no longer LED326.1 (B_A), LED326.3 (R_A), LED326.5 (G_A), LED327.1 (B_A), LED327.3 (R_A), LED327.5 (G_A), LED328.1 (B_A), LED328.3 (R_A), LED328.5 (G_A), LED329.1 (B_A), LED329.3 (R_A), LED329.5 (G_A), LED330.1 (B_A), LED330.3 (R_A), LED330.5 (G_A), LED331.1 (B_A), LED331.3 (R_A), LED331.5 (G_A)
- net RGB_SW03: now also LED324.1 (B_A), LED324.3 (R_A), LED324.5 (G_A), LED338.1 (B_A), LED338.3 (R_A), LED338.5 (G_A), LED351.1 (B_A), LED351.3 (R_A), LED351.5 (G_A), LED352.1 (B_A), LED352.3 (R_A), LED352.5 (G_A), LED364.1 (B_A), LED364.3 (R_A), LED364.5 (G_A), LED377.1 (B_A), LED377.3 (R_A), LED377.5 (G_A); no longer LED332.1 (B_A), LED332.3 (R_A), LED332.5 (G_A), LED333.1 (B_A), LED333.3 (R_A), LED333.5 (G_A), LED344.1 (B_A), LED344.3 (R_A), LED344.5 (G_A), LED345.1 (B_A), LED345.3 (R_A), LED345.5 (G_A), LED346.1 (B_A), LED346.3 (R_A), LED346.5 (G_A), LED347.1 (B_A), LED347.3 (R_A), LED347.5 (G_A)
- net RGB_SW04: now also LED325.1 (B_A), LED325.3 (R_A), LED325.5 (G_A), LED326.1 (B_A), LED326.3 (R_A), LED326.5 (G_A), LED353.1 (B_A), LED353.3 (R_A), LED353.5 (G_A), LED365.1 (B_A), LED365.3 (R_A), LED365.5 (G_A), LED378.1 (B_A), LED378.3 (R_A), LED378.5 (G_A); no longer LED338.1 (B_A), LED338.3 (R_A), LED338.5 (G_A), LED340.1 (B_A), LED340.3 (R_A), LED340.5 (G_A), LED341.1 (B_A), LED341.3 (R_A), LED341.5 (G_A), LED342.1 (B_A), LED342.3 (R_A), LED342.5 (G_A), LED343.1 (B_A), LED343.3 (R_A), LED343.5 (G_A)
- net RGB_SW05: now also LED327.1 (B_A), LED327.3 (R_A), LED327.5 (G_A), LED340.1 (B_A), LED340.3 (R_A), LED340.5 (G_A), LED354.1 (B_A), LED354.3 (R_A), LED354.5 (G_A), LED366.1 (B_A), LED366.3 (R_A), LED366.5 (G_A), LED367.1 (B_A), LED367.3 (R_A), LED367.5 (G_A), LED379.1 (B_A), LED379.3 (R_A), LED379.5 (G_A); no longer LED334.1 (B_A), LED334.3 (R_A), LED334.5 (G_A), LED335.1 (B_A), LED335.3 (R_A), LED335.5 (G_A), LED336.1 (B_A), LED336.3 (R_A), LED336.5 (G_A), LED337.1 (B_A), LED337.3 (R_A), LED337.5 (G_A), LED348.1 (B_A), LED348.3 (R_A), LED348.5 (G_A), LED349.1 (B_A), LED349.3 (R_A), LED349.5 (G_A)
- net RGB_SW06: now also LED328.1 (B_A), LED328.3 (R_A), LED328.5 (G_A), LED341.1 (B_A), LED341.3 (R_A), LED341.5 (G_A), LED342.1 (B_A), LED342.3 (R_A), LED342.5 (G_A), LED368.1 (B_A), LED368.3 (R_A), LED368.5 (G_A), LED380.1 (B_A), LED380.3 (R_A), LED380.5 (G_A); no longer LED350.1 (B_A), LED350.3 (R_A), LED350.5 (G_A), LED351.1 (B_A), LED351.3 (R_A), LED351.5 (G_A), LED352.1 (B_A), LED352.3 (R_A), LED352.5 (G_A), LED353.1 (B_A), LED353.3 (R_A), LED353.5 (G_A), LED354.1 (B_A), LED354.3 (R_A), LED354.5 (G_A)
- net RGB_SW07: now also LED329.1 (B_A), LED329.3 (R_A), LED329.5 (G_A), LED343.1 (B_A), LED343.3 (R_A), LED343.5 (G_A), LED369.1 (B_A), LED369.3 (R_A), LED369.5 (G_A), LED381.1 (B_A), LED381.3 (R_A), LED381.5 (G_A); no longer LED358.1 (B_A), LED358.3 (R_A), LED358.5 (G_A), LED359.1 (B_A), LED359.3 (R_A), LED359.5 (G_A), LED360.1 (B_A), LED360.3 (R_A), LED360.5 (G_A), LED373.1 (B_A), LED373.3 (R_A), LED373.5 (G_A)
- net RGB_SW08: now also LED330.1 (B_A), LED330.3 (R_A), LED330.5 (G_A), LED331.1 (B_A), LED331.3 (R_A), LED331.5 (G_A), LED344.1 (B_A), LED344.3 (R_A), LED344.5 (G_A), LED358.1 (B_A), LED358.3 (R_A), LED358.5 (G_A), LED382.1 (B_A), LED382.3 (R_A), LED382.5 (G_A); no longer LED367.1 (B_A), LED367.3 (R_A), LED367.5 (G_A), LED368.1 (B_A), LED368.3 (R_A), LED368.5 (G_A), LED369.1 (B_A), LED369.3 (R_A), LED369.5 (G_A), LED371.1 (B_A), LED371.3 (R_A), LED371.5 (G_A), LED372.1 (B_A), LED372.3 (R_A), LED372.5 (G_A)
- net RGB_SW09: now also LED332.1 (B_A), LED332.3 (R_A), LED332.5 (G_A), LED345.1 (B_A), LED345.3 (R_A), LED345.5 (G_A), LED359.1 (B_A), LED359.3 (R_A), LED359.5 (G_A), LED371.1 (B_A), LED371.3 (R_A), LED371.5 (G_A), LED372.1 (B_A), LED372.3 (R_A), LED372.5 (G_A), LED383.1 (B_A), LED383.3 (R_A), LED383.5 (G_A); no longer LED361.1 (B_A), LED361.3 (R_A), LED361.5 (G_A), LED362.1 (B_A), LED362.3 (R_A), LED362.5 (G_A), LED363.1 (B_A), LED363.3 (R_A), LED363.5 (G_A), LED364.1 (B_A), LED364.3 (R_A), LED364.5 (G_A), LED365.1 (B_A), LED365.3 (R_A), LED365.5 (G_A), LED366.1 (B_A), LED366.3 (R_A), LED366.5 (G_A)
- net RGB_SW10: now also LED333.1 (B_A), LED333.3 (R_A), LED333.5 (G_A), LED346.1 (B_A), LED346.3 (R_A), LED346.5 (G_A), LED347.1 (B_A), LED347.3 (R_A), LED347.5 (G_A), LED360.1 (B_A), LED360.3 (R_A), LED360.5 (G_A), LED373.1 (B_A), LED373.3 (R_A), LED373.5 (G_A), LED384.1 (B_A), LED384.3 (R_A), LED384.5 (G_A); no longer LED374.1 (B_A), LED374.3 (R_A), LED374.5 (G_A), LED375.1 (B_A), LED375.3 (R_A), LED375.5 (G_A), LED376.1 (B_A), LED376.3 (R_A), LED376.5 (G_A), LED377.1 (B_A), LED377.3 (R_A), LED377.5 (G_A), LED378.1 (B_A), LED378.3 (R_A), LED378.5 (G_A), LED379.1 (B_A), LED379.3 (R_A), LED379.5 (G_A)
- net RGB_SW11: now also LED320.1 (B_A), LED320.3 (R_A), LED320.5 (G_A), LED334.1 (B_A), LED334.3 (R_A), LED334.5 (G_A), LED348.1 (B_A), LED348.3 (R_A), LED348.5 (G_A), LED361.1 (B_A), LED361.3 (R_A), LED361.5 (G_A), LED374.1 (B_A), LED374.3 (R_A), LED374.5 (G_A); no longer LED380.1 (B_A), LED380.3 (R_A), LED380.5 (G_A), LED381.1 (B_A), LED381.3 (R_A), LED381.5 (G_A), LED382.1 (B_A), LED382.3 (R_A), LED382.5 (G_A), LED383.1 (B_A), LED383.3 (R_A), LED383.5 (G_A), LED384.1 (B_A), LED384.3 (R_A), LED384.5 (G_A)
Other:
- note added: "Physical rows use sink groups 1..5; the ten extra keys use group 6. Scan banks follow nearby columns."
- note removed: "Each group has up to six nearby keys. Follow the RGB_SW and RGB_CS labels when routing."
- moved on the sheet: LED320, LED321, LED322, LED323, LED324, LED325, LED326, LED327, LED328, LED329, LED330, LED331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

Commit message: finish the new bms and move the connectors up top
Parts:
- C325: value 100n 50V RGB PVCC / buffer A -> 100n 50V RGB PVCC / buffer B
Connections:
- net I2C_SCL: now also U321.2 (SCLA); no longer U321.7 (SCLB)
- net I2C_SDA: now also U321.3 (SDAA); no longer U321.6 (SDAB)
- net KB_RGB_5V: now also U321.8 (VCCB); no longer U321.1 (VCCA), U321.5 (EN)
- net MCU_3V3: now also U321.1 (VCCA), U321.5 (EN); no longer U321.8 (VCCB)
- net RGB_SCL: now also U321.7 (SCLB); no longer U321.2 (SCLA)
- net RGB_SDA: now also U321.6 (SDAB); no longer U321.3 (SDAA)
Other:
- note added: "U321 A side is the main 3.3 V bus; B side is the switched 5 V RGB bus. Its power-off isolation keeps the unpowered LED driver off the EC bus."
- note removed: "U321 A side is switched 5 V; B side is 3.3 V. Its power-off isolation keeps the unpowered LED driver off the EC bus."

Commit message: finish the keyboard and update the case and power
Parts:
- J320: footprint Connector_FFC-FPC:Hirose_FH12-30S-0.5SH_1x30-1MP_P0.50mm_Horizontal -> Keyboard_Connector:Hirose_FH12_30_Separate_Mounts; symbol Conn_01x30_FFC_MP:Conn_01x30_FFC_MP -> Keyboard_Connector:FFC_30_Separate_Mounts; Assembly connector MP hold-downs are mechanical and netless -> MP1 and MP2 are separate unused mechanical hold-downs
Connections:
- no-connect marks 7 -> 8
Changed lines of the file:
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@@
 (text "== J320 keyboard FFC / board-to-board connector ==" (at 20.32 335.28 0) (effects (font (size 1.27 1.27)) (justify left)))
 (symbol
-  (lib_id "Conn_01x30_FFC_MP:Conn_01x30_FFC_MP")
+  (lib_id "Keyboard_Connector:FFC_30_Separate_Mounts")
   (at 165.1 400.05 0)
   (unit 1)
@@
   (property "Reference" "J320" (at 165.1 353.06 0) (effects (font (size 1.27 1.27))))
   (property "Value" "Keyboard FFC: MX ULP 5x14 matrix on 30-pin EC contract" (at 165.1 447.04 0) (effects (font (size 1.27 1.27))))
-  (property "Footprint" "Connector_FFC-FPC:Hirose_FH12-30S-0.5SH_1x30-1MP_P0.50mm_Horizontal" (at 165.1 400.05 0) (effects (font (size 1.27 1.27)) (hide yes)))
+  (property "Footprint" "Keyboard_Connector:Hirose_FH12_30_Separate_Mounts" (at 165.1 400.05 0) (effects (font (size 1.27 1.27)) (hide yes)))
   (property "Datasheet" "" (at 165.1 400.05 0) (effects (font (size 1.27 1.27)) (hide yes)))
   (property "Manufacturer" "Hirose" (at 165.1 400.05 0) (effects (font (size 1.27 1.27)) (hide yes)))
@@
   (property "LCSC" "C506793" (at 165.1 400.05 0) (effects (font (size 1.27 1.27)) (hide yes)))
   (property "JLCPCB Part #" "C506793" (at 165.1 400.05 0) (effects (font (size 1.27 1.27)) (hide yes)))
-  (property "Assembly" "connector MP hold-downs are mechanical and netless" (at 165.1 400.05 0) (effects (font (size 1.27 1.27)) (hide yes)))
+  (property "Assembly" "MP1 and MP2 are separate unused mechanical hold-downs" (at 165.1 400.05 0) (effects (font (size 1.27 1.27)) (hide yes)))
   (pin "1")
   (pin "2")
@@
   (pin "29")
   (pin "30")
-  (pin "MP")
+  (pin "MP1")
+  (pin "MP2")
   (instances
     (project "ducktop2"
@@
 )
   (embedded_fonts no)
+(no_connect (at 170.18 443.23))
 )
