File: bms/bms.kicad_sch (KiCad schematic)
At the start: 62 parts, among them J2 3S pack power + cell-tap harn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, Q11 CSD18540Q5B reverse-pack FET A, Q12 CSD18540Q5B reverse-pack FET B, Q701 BSS138 pack protector latch r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, Q703 CSD18540Q5B BQ77915 discharge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, Q704 CSD18540Q5B BQ77915 charge FET, U11 LTC4368IMS-1 bidirectional pa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, U719 BQ7791500PWR autonomous 3S pr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

Commit message: route more of the bms
Parts:
- removed FPC106: FH12-30S-0.5SH (FPC-3), Connector_FFC-FPC:Hirose_FH12-30S-0.5SH_1x30-1MP_P0.50mm_Horizontal, symbol Conn_01x30_FFC_MP:Conn_01x30_FFC_MP
- added C2200: 100n 50V thermal regulator input, Capacitor_SMD:C_0603_1608Metric, symbol Device:C
- added C2201: 10u 50V thermal bias; require Ceff >=2u, Capacitor_SMD:C_1206_3216Metric, symbol Device:C
- added C2211, C2212, C2213: 10n 50V NTC sense filter, Capacitor_SMD:C_0603_1608Metric, symbol Device:C
- added C2221, C2222, C2223: 100n 50V comparator supply, Capacitor_SMD:C_0603_1608Metric, symbol Device:C
- added C2230: 100n 50V thermal supervisor supply, Capacitor_SMD:C_0603_1608Metric, symbol Device:C
- added C2231: 100n 50V thermal buffer supply, Capacitor_SMD:C_0603_1608Metric, symbol Device:C
- added C2240, C2241, C2242: 10n 50V thermal reference filter, Capacitor_SMD:C_0603_1608Metric, symbol Device:C
- added C2243: 10n 50V thermal reference filter, Capacitor_SMD:C_0402_1005Metric, symbol Device:C
- added C2250: 100n 50V raw isolator supply, Capacitor_SMD:C_0603_1608Metric, symbol Device:C
- added C2251: 100n 50V control-island isolator supply, Capacitor_SMD:C_0603_1608Metric, symbol Device:C
- added C2252: 100n 50V control fault-buffer supply, Capacitor_SMD:C_0603_1608Metric, symbol Device:C
- added C2253: 100n 50V protected control regulator input, Capacitor_SMD:C_0603_1608Metric, symbol Device:C
- added C2254: 10u 50V protected local bias; Ceff >=2u, Capacitor_SMD:C_1206_3216Metric, symbol Device:C
- added C2255: 100n 50V protected transceiver supply, Capacitor_SMD:C_0603_1608Metric, symbol Device:C
- added C2256: 100n 50V control transceiver supply, Capacitor_SMD:C_0603_1608Metric, symbol Device:C
- added D2200: BAT54WS protected control reverse-input block, Diode_SMD:D_SOD-323, symbol Device:D_Schottky
- added D2201, D2202: BAT54S control-island pin clamps, Package_TO_SOT_SMD:SOT-23, symbol BMS_Thermal:BAT54S_AKC
- added J2072: protected pack power, Connector_Molex:Molex_Micro-Fit_3.0_43650-0224_1x02-1MP_P3.00mm_Vertical, symbol Conn_01x02_MP:Conn_01x02_MP
- added J2074: isolated bms control, Connector_JST:JST_SH_SM05B-SRSS-TB_1x05-1MP_P1.00mm_Horizontal, symbol Connector_Generic_MountingPin:Conn_01x05_MountingPin
- added J2200: three cell probes: paired 1/2, 3/4, 5/6, Connector_JST:JST_SH_SM06B-SRSS-TB_1x06-1MP_P1.00mm_Horizontal, symbol BMS_Thermal:Conn_01x06_Thermal_MP
- added Q2200: BSS138 CHG thermal CTR pull-down, Package_TO_SOT_SMD:SOT-23, symbol Q_NMOS_SOT23_GSD:Q_NMOS_SOT23_GSD
- added Q2201: BSS138 DSG thermal CTR pull-down, Package_TO_SOT_SMD:SOT-23, symbol Q_NMOS_SOT23_GSD:Q_NMOS_SOT23_GSD
- added R2200: 1k 1% 0.75W raw thermal supply limiter, Resistor_SMD:R_2010_5025Metric, symbol Device:R
- added R2201: 9.53k 0.1% 25ppm thermal bias fault bleed, Resistor_SMD:R_0603_1608Metric, symbol Device:R
- added R2210, R2213, R2216: 100k 0.1% 25ppm cell NTC pull-up, Resistor_SMD:R_0603_1608Metric, symbol Device:R
- added R2211, R2214: 10k 0.1% 25ppm NTC sense-lead limit, Resistor_SMD:R_0603_1608Metric, symbol Device:R
- added R2212, R2215, R2218: 10k 0.1% 25ppm NTC return-lead limit, Resistor_SMD:R_0603_1608Metric, symbol Device:R
- added R2217: 10k 0.1% 25ppm NTC sense-lead limit, Resistor_SMD:R_0402_1005Metric, symbol Device:R
- added R2230: 100k thermal charge-health pull-up, Resistor_SMD:R_0603_1608Metric, symbol Device:R
- added R2231: 100k thermal discharge-health pull-up, Resistor_SMD:R_0603_1608Metric, symbol Device:R
- added R2232: 100k thermal-ready pull-up, Resistor_SMD:R_0603_1608Metric, symbol Device:R
- added R2233: 1M thermal-ready default-low, Resistor_SMD:R_0603_1608Metric, symbol Device:R
- added R2234, R2237: 1k thermal CTR gate series, Resistor_SMD:R_0603_1608Metric, symbol Device:R
- added R2235, R2238: 100k thermal CTR gate default-off, Resistor_SMD:R_0603_1608Metric, symbol Device:R
- added R2236, R2239: 470k 0.1% 25ppm CTR fault pull-up, Resistor_SMD:R_0603_1608Metric, symbol Device:R
- added R2240: 243k 0.1% 25ppm CHG_COLD top, Resistor_SMD:R_0603_1608Metric, symbol Device:R
- added R2242: 634k 0.1% 25ppm CHG_HOT top, Resistor_SMD:R_0603_1608Metric, symbol Device:R
- added R2244: 147k 0.1% 25ppm DSG_COLD top, Resistor_SMD:R_0603_1608Metric, symbol Device:R
- added R2246: 845k 0.1% 25ppm DSG_HOT top, Resistor_SMD:R_0603_1608Metric, symbol Device:R
- added R2247: 499k 0.1% 25ppm thermal reference bottom, Resistor_SMD:R_0603_1608Metric, symbol Device:R
- added R2250: 100k isolated discharge-health default-low, Resistor_SMD:R_0603_1608Metric, symbol Device:R
- added R2251: 100k isolated charge-permit default-low, Resistor_SMD:R_0603_1608Metric, symbol Device:R
- added R2252: 2.49k 1% 0.25W protected control supply limiter, Resistor_SMD:R_1206_3216Metric, symbol Device:R
- added R2253: 30.1k 0.1% protected bias minimum load, Resistor_SMD:R_0603_1608Metric, symbol Device:R
- added R2254: 1k local retry gate series, Resistor_SMD:R_0402_1005Metric, symbol Device:R
- added R2255: 100k isolated LTC-health default-low, Resistor_SMD:R_0603_1608Metric, symbol Device:R
- added R2256: 3.3k control fault pull-up, Resistor_SMD:R_0603_1608Metric, symbol Device:R
- added R2257: 100R 1% 0.25W control-island current limiter, Resistor_SMD:R_1206_3216Metric, symbol Device:R
- added R2258: 4.7k fault interface current limit, Resistor_SMD:R_0603_1608Metric, symbol Device:R
- added R2259: 4.7k retry interface current limit, Resistor_SMD:R_0603_1608Metric, symbol Device:R
- added R2264: 100k retry input default-low, Resistor_SMD:R_0603_1608Metric, symbol Device:R
- added R2265: 4.7k charge-permit interface current limit, Resistor_SMD:R_0603_1608Metric, symbol Device:R
- added TH2201: 104JT-025 cell 1 insulated probe, symbol Device:Thermistor_NTC
- added TH2202: 104JT-025 cell 2 insulated probe, symbol Device:Thermistor_NTC
- added TH2203: 104JT-025 cell 3 insulated probe, symbol Device:Thermistor_NTC
- added TPB12: BMS_SRP, TestPoint:TestPoint_Pad_1.5x1.5mm, symbol Connector:TestPoint
- added TPB2: BAT_PROT_VIN, TestPoint:TestPoint_Pad_1.5x1.5mm, symbol Connector:TestPoint
- added TPB20: THERM_3V3, TestPoint:TestPoint_Pad_1.5x1.5mm, symbol Connector:TestPoint
- added TPB21: THERM_READY, TestPoint:TestPoint_Pad_1.5x1.5mm, symbol Connector:TestPoint
- added TPB22: THERM_SENSE_1, TestPoint:TestPoint_Pad_1.5x1.5mm, symbol Connector:TestPoint
- added TPB23: THERM_SENSE_2, TestPoint:TestPoint_Pad_1.5x1.5mm, symbol Connector:TestPoint
- added TPB24: THERM_SENSE_3, TestPoint:TestPoint_Pad_1.5x1.5mm, symbol Connector:TestPoint
- added TPB25: BMS_CTRC, TestPoint:TestPoint_Pad_1.5x1.5mm, symbol Connector:TestPoint
- added TPB26: BMS_CTRD, TestPoint:TestPoint_Pad_1.5x1.5mm, symbol Connector:TestPoint
- added TPB27: PACK_CHG_TEMP_OK, TestPoint:TestPoint_Pad_1.5x1.5mm, symbol Connector:TestPoint
- added TPB7: PACK_FAULT_N, TestPoint:TestPoint_Pad_1.5x1.5mm, symbol Connector:TestPoint
- added U2200: TPS70933DBVR raw-pack thermal bias, Package_TO_SOT_SMD:SOT-23-5, symbol BMS_Thermal:TPS70933DBV
- added U2201: TLV1864PWR cell 1 thermal windows, Package_SO:TSSOP-14_4.4x5mm_P0.65mm, symbol BMS_Thermal:TLV1864PW
- added U2202: TLV1864PWR cell 2 thermal windows, Package_SO:TSSOP-14_4.4x5mm_P0.65mm, symbol BMS_Thermal:TLV1864PW
- added U2203: TLV1864PWR cell 3 thermal windows, Package_SO:TSSOP-14_4.4x5mm_P0.65mm, symbol BMS_Thermal:TLV1864PW
- added U2204: TLV803EA29RDBZR thermal startup hold, Package_TO_SOT_SMD:SOT-23, symbol TLV803EA29RDBZR:TLV803EA29RDBZR
- added U2205: SN74AUP2G126DCUR thermal startup gate, ducktop2:TI_DCU0008A_VSSOP8, symbol BMS_Thermal:SN74AUP2G126DCU
- added U2206: ISO7041FDBQR separate charge/discharge permits; d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, Package_SO:QSOP-16_3.9x4.9mm_P0.635mm, symbol BMS_Thermal:ISO7041FDBQ
- added U2207: SN74AUP2G07DCKR thermal and LTC fault wired-OR, Package_TO_SOT_SMD:SOT-363_SC-70-6, symbol BMS_Thermal:SN74AUP2G07DCK
- added U2208: TPS70933DBVR protected-side local bias, Package_TO_SOT_SMD:SOT-23-5, symbol BMS_Thermal:TPS70933DBV
- added U2209: ISO7021FDR LTC fault and retry isolation, Package_SO:SOIC-8_3.9x4.9mm_P1.27mm, symbol BMS_Thermal:ISO7021FD
- R2241: renamed from TPB2; value BAT_PROT_VIN -> 499k 0.1% 25ppm thermal reference bottom; footprint TestPoint:TestPoint_Pad_1.5x1.5mm -> Resistor_SMD:R_0603_1608Metric; symbol Connector:TestPoint -> Device:R; MPN (none) -> RT0603BRD07499KL; Manufacturer - -> Yageo; Note test point, no MPN -> (none); now in the parts list
- R2243: renamed from TPB7; value PACK_FAULT_N -> 499k 0.1% 25ppm thermal reference bottom; footprint TestPoint:TestPoint_Pad_1.5x1.5mm -> Resistor_SMD:R_0603_1608Metric; symbol Connector:TestPoint -> Device:R; MPN (none) -> RT0603BRD07499KL; Manufacturer - -> Yageo; Note test point, no MPN -> (none); now in the parts list
- R2245: renamed from TPB12; value BMS_SRP -> 499k 0.1% 25ppm thermal reference bottom; footprint TestPoint:TestPoint_Pad_1.5x1.5mm -> Resistor_SMD:R_0603_1608Metric; symbol Connector:TestPoint -> Device:R; MPN (none) -> RT0603BRD07499KL; Manufacturer - -> Yageo; Note test point, no MPN -> (none); now in the parts list
- R708: value 10k pack FAULT pull-up -> 100k protected-side LTC fault pull-up; MPN RC0603FR-0710KL -> RC0603FR-07100KL
- TPB5: footprint TestPoint:TestPoint_Pad_1.5x1.5mm -> TestPoint:TestPoint_Pad_1.0x1.0mm
Connections:
- net BAT_PROT_VIN: now also R2252.1, TPB2.1; no longer R2241.1
- net BMS_SRP: now also TPB12.1; no longer R2245.1
- net BMS_VDD: now also R2236.1, R2239.1
- net FG_VSS: now also C2253.2, C2254.2, C2255.2, J2072.2 (Pin_2), R2253.2, U2208.2 (GND), U2209.4 (GND1)
- net MCU_3V3: now also J2074.3 (Pin_3), R2257.1; no longer R708.1
- net PACK_FAULT_N: now also J2074.1 (Pin_1), R2258.2, TPB7.1; no longer R2243.1, R708.2, U11.7 (FAULT)
- net PACK_NEG_RAW: now also R2241.2, R2243.2, R2245.2, C2200.2, C2201.2, C2211.2, C2212.2, C2213.2, C2221.2, C2222.2, C2223.2, C2230.2, C2231.2, C2240.2, C2241.2, C2242.2, C2243.2, C2250.2, J2200.MP, Q2200.2 (S), Q2201.2 (S), R2201.2, R2212.2, R2215.2, R2218.2, R2233.2, R2235.2, R2238.2, R2247.2, U2200.2 (GND), U2201.11 (V-), U2202.11 (V-), U2203.11 (V-), U2204.2 (GND), U2205.4 (GND), U2206.2 (GND1), U2206.5 (INC), U2206.7 (EN1), U2206.8 (GND1); no longer U719.23 (CTRC), U719.24 (CTRD)
- net PACK_POS_FUSED: now also J2072.1 (Pin_1)
- net PACK_POS_RAW: now also R2200.1
- net PACK_RETRY_PULSE: now also J2074.2 (Pin_2), R2259.1; no longer Q701.1 (G), R709.1
- new net BMS_CTRC: Q2200.3 (D), R2236.2, TPB25.1, U719.23 (CTRC)
- new net BMS_CTRD: Q2201.3 (D), R2239.2, TPB26.1, U719.24 (CTRD)
- new net BMS_PROTECT_FAULT_N: R708.2, U11.7 (FAULT), U2209.3 (INB)
- new net CTRL_3V3: C2251.1, C2252.1, C2256.1, D2201.2 (K2), D2202.2 (K2), R2256.1, R2257.2, U2206.16 (VCC2), U2207.5 (VCC), U2209.8 (VCC2)
- new net CTRL_FAULT_LOCAL_N: R2256.2, R2258.1, U2207.4 (2Y), U2207.6 (1Y)
- new net CTRL_GND: C2251.2, C2252.2, C2256.2, D2201.1 (A1), D2202.1 (A1), J2074.5 (Pin_5), J2074.MP (MountPin), R2250.2, R2251.2, R2255.2, R2264.2, U2206.10 (EN2), U2206.11 (IND), U2206.15 (GND2), U2206.9 (GND2), U2207.2 (GND), U2209.5 (GND2)
- new net CTRL_RETRY_IN: D2201.3 (K1_A2), R2259.2, R2264.1, U2209.7 (INA)
- new net PACK_CHG_TEMP_OK: J2074.4 (Pin_4), R2265.2, TPB27.1
- new net PACK_PROTECT_OK: R2255.1, U2207.3 (2A), U2209.6 (OUTB)
- new net PACK_RETRY_LOCAL: R2254.1, U2209.2 (OUTA)
- new net PACK_RETRY_LOCAL_GATE: Q701.1 (G), R2254.2, R709.1
- new net PROT_CTRL_3V3: C2254.1, C2255.1, R2253.1, R708.1, U2208.5 (OUT), U2209.1 (VCC1)
- new net PROT_CTRL_FEED: D2200.2 (A), R2252.2
- new net PROT_CTRL_IN: C2253.1, D2200.1 (K), U2208.1 (IN)
- new net THERM_3V3: C2201.1, C2221.1, C2222.1, C2223.1, C2230.1, C2231.1, C2250.1, R2201.1, R2210.1, R2213.1, R2216.1, R2230.1, R2231.1, R2232.1, R2240.1, R2242.1, R2244.1, R2246.1, TPB20.1, U2200.5 (OUT), U2201.4 (V+), U2202.4 (V+), U2203.4 (V+), U2204.3 (VDD), U2205.8 (VCC), U2206.1 (VCC1)
- new net THERM_CHG_COLD_REF: C2240.1, R2240.2, R2241.1, U2201.3 (IN1+), U2202.3 (IN1+), U2203.3 (IN1+)
- new net THERM_CHG_GATE: Q2200.1 (G), R2234.2, R2235.1, U2206.3 (INA)
- new net THERM_CHG_HEALTH: R2230.2, U2201.1 (OUT1), U2201.7 (OUT2), U2202.1 (OUT1), U2202.7 (OUT2), U2203.1 (OUT1), U2203.7 (OUT2), U2205.2 (1A)
- new net THERM_CHG_HEALTH_ISO: D2202.3 (K1_A2), R2251.1, R2265.1, U2206.14 (OUTA)
- new net THERM_CHG_HOT_REF: C2241.1, R2242.2, R2243.1, U2201.6 (IN2-), U2202.6 (IN2-), U2203.6 (IN2-)
- new net THERM_CHG_PERMIT: R2234.1, U2205.6 (1Y)
- new net THERM_DSG_COLD_REF: C2242.1, R2244.2, R2245.1, U2201.12 (IN4+), U2202.12 (IN4+), U2203.12 (IN4+)
- new net THERM_DSG_GATE: Q2201.1 (G), R2237.2, R2238.1, U2206.4 (INB)
- new net THERM_DSG_HEALTH: R2231.2, U2201.14 (OUT4), U2201.8 (OUT3), U2202.14 (OUT4), U2202.8 (OUT3), U2203.14 (OUT4), U2203.8 (OUT3), U2205.5 (2A)
- new net THERM_DSG_HEALTH_ISO: R2250.1, U2206.13 (OUTB), U2207.1 (1A)
- new net THERM_DSG_HOT_REF: C2243.1, R2246.2, R2247.1, U2201.9 (IN3-), U2202.9 (IN3-), U2203.9 (IN3-)
- new net THERM_DSG_PERMIT: R2237.1, U2205.3 (2Y)
- new net THERM_PROBE_1_A: J2200.1 (Pin_1), R2211.2, TH2201.1
- new net THERM_PROBE_1_B: J2200.2 (Pin_2), R2212.1, TH2201.2
- new net THERM_PROBE_2_A: J2200.3 (Pin_3), R2214.2, TH2202.1
- new net THERM_PROBE_2_B: J2200.4 (Pin_4), R2215.1, TH2202.2
- new net THERM_PROBE_3_A: J2200.5 (Pin_5), R2217.2, TH2203.1
- new net THERM_PROBE_3_B: J2200.6 (Pin_6), R2218.1, TH2203.2
- new net THERM_RAW_IN: C2200.1, R2200.2, U2200.1 (IN)
- new net THERM_READY: R2232.2, R2233.1, TPB21.1, U2204.1 (RESETz), U2205.1 (1OE), U2205.7 (2OE)
- new net THERM_SENSE_1: C2211.1, R2210.2, R2211.1, TPB22.1, U2201.10 (IN3+), U2201.13 (IN4-), U2201.2 (IN1-), U2201.5 (IN2+)
- new net THERM_SENSE_2: C2212.1, R2213.2, R2214.1, TPB23.1, U2202.10 (IN3+), U2202.13 (IN4-), U2202.2 (IN1-), U2202.5 (IN2+)
- new net THERM_SENSE_3: C2213.1, R2216.2, R2217.1, TPB24.1, U2203.10 (IN3+), U2203.13 (IN4-), U2203.2 (IN1-), U2203.5 (IN2+)
- no-connect marks 3 -> 10
Other:
- note added: "== three-cell temperature inhibit: raw reference, independent of firmware =="
- note added: "CTRL_GND belongs only to the isolated control island. Power-return disconnect cannot reach the center through fault/retry pins."
- note added: "J2200 and its hold-downs are raw-pack referenced; no system-ground wire."
- note added: "discharge faults assert PACK_FAULT_N; charge-only faults lower PACK_CHG_TEMP_OK. no raw-ground bypass."
- note added: "j2072 carries protected pack power and return. j2074 pin 5 and its mounting tabs serve only the isolated ctrl_gnd island."
- note added: "never join ctrl_gnd to fg_vss or pack_neg_raw. raw pack negative remains inside the bms and pack harness."
- note added: "provisional charge 10..40C / discharge 0..50C screen; actual cell profile and installed probe response remain unqualified."

Commit message: work on the power redesign and case
Parts:
- F1: value 10A MINI pack fuse: Littelfuse 0297010.WXNV -> 5A fast pack fuse: Schurter HCF, 1kA at 125VDC; footprint Fuse:Fuseholder_Blade_Mini_Keystone_3568 -> ducktop2:Schurter_HCF_8.05x5mm; Height (none) -> 5 mm; InterruptRating (none) -> 1000 A at 125 VDC, L/R <1 ms; MPN 0297010.WXNV + 3568 -> 3-101-056; Manufacturer Littelfuse / Keystone -> SCHURTER
- J2: footprint Connector_Molex:Molex_Mega-Fit_76829-0006_2x03_P5.70mm_Vertical -> Connector_Molex:Molex_Micro-Fit_3.0_43045-0400_2x02_P3.00mm_Horizontal; symbol Connector_Generic:Conn_02x03_Odd_Even -> Connector_Generic:Conn_02x02_Odd_Even; Contacts (none) -> 43030-0038 tin 18 AWG; CurrentRatingBasis (none) -> PS-43045: use conservative six-circuit 18 AWG 6.5 A screen;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; HarnessPinOrder (none) -> 1 raw negative, 2 cell 2 tap, 3 raw positive, 4 cell 1 tap;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; MPN 76829-0006 -> 43045-0400; MatedHeight (none) -> 10.29 mm nominal; horizontal exit; independent harness clamp; MatingHousing (none) -> 43025-0400; Wire (none) -> Alpha 6715, 18 AWG, minimum bend radius 8.763 mm
- J2072: footprint Connector_Molex:Molex_Micro-Fit_3.0_43650-0224_1x02-1MP_P3.00mm_Vertical -> ducktop2:WAGO_2060_452_SMD; symbol Conn_01x02_MP:Conn_01x02_MP -> Connector_Generic:Conn_01x02; Contacts 43030-0038 tin, 18 awg; insulation diameter <=1.85 mm -> spring contact; CurrentRatingBasis PS-43650-001 N4: 2 circuits, 18 awg, 8.5 A at 30 C rise; va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 -> WAGO 2060, 9 A IEC/UL rating with 18 AWG; assembled tempera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; Harness 18 awg; pin 1 red; pin 2 black; straight-numbered; 75 mm le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 -> center: 1 FG_VSS, 2 PACK_POS_FUSED; BMS: 1 PACK_POS_FUSED, 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; MPN 43650-0224 -> 2060-452/998-404; Manufacturer Molex -> WAGO; MatedHeight reserve 17.56 mm per drawing, plus wire exit and bend -> 4.5 mm terminal body; reserve release-tool access; MatingHousing 43645-0200 -> bare wire; Wire (none) -> Alpha 6715 RD005/BK005, 18 AWG; minimum bend radius 8.763 mm
Connections:
- net CELL1_TAP: now also J2.4 (Pin_4); no longer J2.5 (Pin_5)
- net CELL2_TAP: now also J2.2 (Pin_2); no longer J2.6 (Pin_6)
- net PACK_NEG_RAW: now also J2.1 (Pin_1); no longer J2.3 (Pin_3), J2.4 (Pin_4)
- net PACK_POS_RAW: now also J2.3 (Pin_3); no longer J2.1 (Pin_1), J2.2 (Pin_2)
- no-connect marks 10 -> 9
Other:
- moved on the sheet: J2072

Commit message: sort out the keyboard leds and fix more bms routing
Parts:
- TPB13: footprint TestPoint:TestPoint_Pad_1.5x1.5mm -> TestPoint:TestPoint_Pad_D1.0mm
Changed lines of the file:
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@@
   (property "Reference" "TPB13" (at 599.44 162.56 0) (effects (font (size 1.27 1.27))))
   (property "Value" "BMS_SRN" (at 599.44 167.64 0) (effects (font (size 1.27 1.27))))
-  (property "Footprint" "TestPoint:TestPoint_Pad_1.5x1.5mm" (at 599.44 165.1 0) (effects (font (size 1.27 1.27)) (hide yes)))
+  (property "Footprint" "TestPoint:TestPoint_Pad_D1.0mm" (at 599.44 165.1 0) (effects (font (size 1.27 1.27)) (hide yes)))
   (property "Datasheet" "" (at 599.44 165.1 0) (effects (font (size 1.27 1.27)) (hide yes)))
   (property "Manufacturer" "-" (at 599.44 165.1 0) (effects (font (size 1.27 1.27)) (hide yes)))

Commit message: work on standby power and update the pd configs
Parts:
- RS10: MPN WSLP2512R0110FEA -> WSL2512R0110FEA18
Changed lines of the file:
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@@
   (property "Datasheet" "" (at 335.28 59.69 0) (effects (font (size 1.27 1.27)) (hide yes)))
   (property "Manufacturer" "Vishay Dale" (at 335.28 59.69 0) (effects (font (size 1.27 1.27)) (hide yes)))
-  (property "MPN" "WSLP2512R0110FEA" (at 335.28 59.69 0) (effects (font (size 1.27 1.27)) (hide yes)))
+  (property "MPN" "WSL2512R0110FEA18" (at 335.28 59.69 0) (effects (font (size 1.27 1.27)) (hide yes)))
   (pin "1")
   (pin "2")

Commit message: finish the new bms and move the connectors up top
Parts:
- removed C2254: 10u 50V protected local bias; Ceff >=2u, Capacitor_SMD:C_1206_3216Metric, symbol Device:C
- removed C725: 10u 25V X7R LTC4368 VOUT, Capacitor_SMD:C_0805_2012Metric, symbol Device:C
- removed C842, C843, C844, C848: 1u 10V X7R BQ77915 internal-balance filter, Capacitor_SMD:C_0805_2012Metric, symbol Device:C
- removed C847: 100n BQ77915 SRN-VSS filter, Capacitor_SMD:C_0603_1608Metric, symbol Device:C
- removed D2200: BAT54WS protected control reverse-input block, Diode_SMD:D_SOD-323, symbol Device:D_Schottky
- removed D2201, D2202: BAT54S control-island pin clamps, Package_TO_SOT_SMD:SOT-23, symbol BMS_Thermal:BAT54S_AKC
- removed J2074: isolated bms control, Connector_JST:JST_SH_SM05B-SRSS-TB_1x05-1MP_P1.00mm_Horizontal, symbol Connector_Generic_MountingPin:Conn_01x05_MountingPin
- removed Q2200: BSS138 CHG thermal CTR pull-down, Package_TO_SOT_SMD:SOT-23, symbol Q_NMOS_SOT23_GSD:Q_NMOS_SOT23_GSD
- removed Q701: BSS138 pack protector latch reset, Package_TO_SOT_SMD:SOT-23, symbol Q_NMOS_SOT23_GSD:Q_NMOS_SOT23_GSD
- removed Q703: CSD18540Q5B BQ77915 discharge FET, ducktop2:CSD18540Q5B_DNK, symbol Q_NMOS_123S_4G_5678D:Q_NMOS_123S_4G_5678D
- removed R2200: 1k 1% 0.75W raw thermal supply limiter, Resistor_SMD:R_2010_5025Metric, symbol Device:R
- removed R2201: 9.53k 0.1% 25ppm thermal bias fault bleed, Resistor_SMD:R_0603_1608Metric, symbol Device:R
- removed R2210, R2213: 100k 0.1% 25ppm cell NTC pull-up, Resistor_SMD:R_0603_1608Metric, symbol Device:R
- removed R2211, R2214: 10k 0.1% 25ppm NTC sense-lead limit, Resistor_SMD:R_0603_1608Metric, symbol Device:R
- removed R2212, R2215, R2218: 10k 0.1% 25ppm NTC return-lead limit, Resistor_SMD:R_0603_1608Metric, symbol Device:R
- removed R2217: 10k 0.1% 25ppm NTC sense-lead limit, Resistor_SMD:R_0402_1005Metric, symbol Device:R
- removed R2230: 100k thermal charge-health pull-up, Resistor_SMD:R_0603_1608Metric, symbol Device:R
- removed R2231: 100k thermal discharge-health pull-up, Resistor_SMD:R_0603_1608Metric, symbol Device:R
- removed R2232: 100k thermal-ready pull-up, Resistor_SMD:R_0603_1608Metric, symbol Device:R
- removed R2233: 1M thermal-ready default-low, Resistor_SMD:R_0603_1608Metric, symbol Device:R
- removed R2234: 1k thermal CTR gate series, Resistor_SMD:R_0603_1608Metric, symbol Device:R
- removed R2235: 100k thermal CTR gate default-off, Resistor_SMD:R_0603_1608Metric, symbol Device:R
- removed R2236: 470k 0.1% 25ppm CTR fault pull-up, Resistor_SMD:R_0603_1608Metric, symbol Device:R
- removed R2240: 243k 0.1% 25ppm CHG_COLD top, Resistor_SMD:R_0603_1608Metric, symbol Device:R
- removed R2241, R2243, R2245, R2247: 499k 0.1% 25ppm thermal reference bottom, Resistor_SMD:R_0603_1608Metric, symbol Device:R
- removed R2242: 634k 0.1% 25ppm CHG_HOT top, Resistor_SMD:R_0603_1608Metric, symbol Device:R
- removed R2244: 147k 0.1% 25ppm DSG_COLD top, Resistor_SMD:R_0603_1608Metric, symbol Device:R
- removed R2246: 845k 0.1% 25ppm DSG_HOT top, Resistor_SMD:R_0603_1608Metric, symbol Device:R
- removed R2250: 100k isolated discharge-health default-low, Resistor_SMD:R_0603_1608Metric, symbol Device:R
- removed R2251: 100k isolated charge-permit default-low, Resistor_SMD:R_0603_1608Metric, symbol Device:R
- removed R2252: 2.49k 1% 0.25W protected control supply limiter, Resistor_SMD:R_1206_3216Metric, symbol Device:R
- removed R2253: 30.1k 0.1% protected bias minimum load, Resistor_SMD:R_0603_1608Metric, symbol Device:R
- removed R2254: 1k local retry gate series, Resistor_SMD:R_0402_1005Metric, symbol Device:R
- removed R2255: 100k isolated LTC-health default-low, Resistor_SMD:R_0603_1608Metric, symbol Device:R
- removed R2256: 3.3k control fault pull-up, Resistor_SMD:R_0603_1608Metric, symbol Device:R
- removed R2257: 100R 1% 0.25W control-island current limiter, Resistor_SMD:R_1206_3216Metric, symbol Device:R
- removed R2258: 4.7k fault interface current limit, Resistor_SMD:R_0603_1608Metric, symbol Device:R
- removed R2264: 100k retry input default-low, Resistor_SMD:R_0603_1608Metric, symbol Device:R
- removed R2265: 4.7k charge-permit interface current limit, Resistor_SMD:R_0603_1608Metric, symbol Device:R
- removed R700: 3.09M 1% BAT UV/OV top, Resistor_SMD:R_0603_1608Metric, symbol Device:R
- removed R702: 121k 1% BAT UV/OV bottom, Resistor_SMD:R_0603_1608Metric, symbol Device:R
- removed R703: 22k LTC4368 CGATE series, Resistor_SMD:R_0603_1608Metric, symbol Device:R
- removed R707: 100k pack protector SHDN pull-up, Resistor_SMD:R_0603_1608Metric, symbol Device:R
- removed R708: 100k protected-side LTC fault pull-up, Resistor_SMD:R_0603_1608Metric, symbol Device:R
- removed R709: 100k pack retry gate pulldown, Resistor_SMD:R_0603_1608Metric, symbol Device:R
- removed R840: 1k 1% BQ77915 VDD filter, Resistor_SMD:R_0603_1608Metric, symbol Device:R
- removed R841, R842, R843, R844: 75R 1% BQ77915 cell/balance filter, Resistor_SMD:R_0603_1608Metric, symbol Device:R
- removed R845: 100R BQ77915 SRP filter, Resistor_SMD:R_0603_1608Metric, symbol Device:R
- removed R846: 100R BQ77915 SRN filter, Resistor_SMD:R_0603_1608Metric, symbol Device:R
- removed R847: 4.53k 1% DSG gate resistor, Resistor_SMD:R_0603_1608Metric, symbol Device:R
- removed R848: 1k 1% CHG gate resistor, Resistor_SMD:R_0603_1608Metric, symbol Device:R
- removed R849: 1M 5% DSG gate-source, Resistor_SMD:R_0603_1608Metric, symbol Device:R
- removed R850: 3.3M 5% CHG gate-source, Resistor_SMD:R_0603_1608Metric, symbol Device:R
- removed RS11: 8mOhm 1% 2W BQ77915 current shunt, Resistor_SMD:R_2512_6332Metric, symbol Device:R
- removed TPB1: PACK_POS_RAW, TestPoint:TestPoint_Pad_1.5x1.5mm, symbol Connector:TestPoint
- removed TPB10: BMS_AVDD, TestPoint:TestPoint_Pad_1.5x1.5mm, symbol Connector:TestPoint
- removed TPB11: BMS_VDD, TestPoint:TestPoint_Pad_1.5x1.5mm, symbol Connector:TestPoint
- removed TPB13: BMS_SRN, TestPoint:TestPoint_Pad_D1.0mm, symbol Connector:TestPoint
- removed TPB14: BMS_PRES, TestPoint:TestPoint_Pad_1.5x1.5mm, symbol Connector:TestPoint
- removed TPB15: BMS_LD, TestPoint:TestPoint_Pad_1.5x1.5mm, symbol Connector:TestPoint
- removed TPB16: FG_VSS, TestPoint:TestPoint_Pad_1.5x1.5mm, symbol Connector:TestPoint
- removed TPB20: THERM_3V3, TestPoint:TestPoint_Pad_1.5x1.5mm, symbol Connector:TestPoint
- removed TPB21: THERM_READY, TestPoint:TestPoint_Pad_1.5x1.5mm, symbol Connector:TestPoint
- removed TPB22: THERM_SENSE_1, TestPoint:TestPoint_Pad_1.5x1.5mm, symbol Connector:TestPoint
- removed TPB23: THERM_SENSE_2, TestPoint:TestPoint_Pad_1.5x1.5mm, symbol Connector:TestPoint
- removed TPB24: THERM_SENSE_3, TestPoint:TestPoint_Pad_1.5x1.5mm, symbol Connector:TestPoint
- removed TPB26: BMS_CTRD, TestPoint:TestPoint_Pad_1.5x1.5mm, symbol Connector:TestPoint
- removed TPB27: PACK_CHG_TEMP_OK, TestPoint:TestPoint_Pad_1.5x1.5mm, symbol Connector:TestPoint
- removed TPB3: PACK_POS_FUSED, TestPoint:TestPoint_Pad_1.5x1.5mm, symbol Connector:TestPoint
- removed TPB4: BAT_PROT_FET_COMMON, TestPoint:TestPoint_Pad_1.5x1.5mm, symbol Connector:TestPoint
- removed TPB5: BAT_PROT_GATE, TestPoint:TestPoint_Pad_1.0x1.0mm, symbol Connector:TestPoint
- removed TPB6: BAT_PROT_CGATE, TestPoint:TestPoint_Pad_1.5x1.5mm, symbol Connector:TestPoint
- removed TPB8: PACK_RETRY_PULSE, TestPoint:TestPoint_Pad_1.5x1.5mm, symbol Connector:TestPoint
- removed TPB9: MCU_3V3, TestPoint:TestPoint_Pad_1.5x1.5mm, symbol Connector:TestPoint
- removed U2204: TLV803EA29RDBZR thermal startup hold, Package_TO_SOT_SMD:SOT-23, symbol TLV803EA29RDBZR:TLV803EA29RDBZR
- removed U2206: ISO7041FDBQR separate charge/discharge permits; d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, Package_SO:QSOP-16_3.9x4.9mm_P0.635mm, symbol BMS_Thermal:ISO7041FDBQ
- removed U2207: SN74AUP2G07DCKR thermal and LTC fault wired-OR, Package_TO_SOT_SMD:SOT-363_SC-70-6, symbol BMS_Thermal:SN74AUP2G07DCK
- removed U2208: TPS70933DBVR protected-side local bias, Package_TO_SOT_SMD:SOT-23-5, symbol BMS_Thermal:TPS70933DBV
- removed U719: BQ7791500PWR autonomous 3S primary protector, Package_SO:TSSOP-24_4.4x7.8mm_P0.65mm, symbol BQ77915:BQ77915
- added C2222, C2223: 100n 50V comparator supply, Capacitor_SMD:C_0603_1608Metric, symbol Device:C
- added C2231: 100n 50V thermal buffer supply, Capacitor_SMD:C_0603_1608Metric, symbol Device:C
- added C2232: 100n 50V OFF-bias bypass, Capacitor_SMD:C_0603_1608Metric, symbol Device:C
- added C2257: 1u 10V control input, Capacitor_SMD:C_0603_1608Metric, symbol Device:C
- added C2258: 1u 10V control output, Capacitor_SMD:C_0603_1608Metric, symbol Device:C
- added C2270, C2271: 10n 50V C0G differential filter, Capacitor_SMD:C_0603_1608Metric, symbol Device:C
- added C2272: 1u 10V reference input, Capacitor_SMD:C_0603_1608Metric, symbol Device:C
- added C2274, C2275: 100n 50V current guard supply, Capacitor_SMD:C_0603_1608Metric, symbol Device:C
- added C2276, C2277: 10n 50V current reference filter, Capacitor_SMD:C_0603_1608Metric, symbol Device:C
- added C2278: 100n 50V current supervisor supply, Capacitor_SMD:C_0603_1608Metric, symbol Device:C
- added C2279: 100n 50V readiness logic supply, Capacitor_SMD:C_0603_1608Metric, symbol Device:C
- added C2281: 1u 50V thermal switch input, Capacitor_SMD:C_0805_2012Metric, symbol Device:C
- added C852, C853, C854, C855: 220n 50V cell filter, Capacitor_SMD:C_0603_1608Metric, symbol Device:C
- added C882: 100n 25V C0G startup ramp, Capacitor_SMD:C_1206_3216Metric, symbol Device:C
- added C883: 1u 50V startup input, Capacitor_SMD:C_0805_2012Metric, symbol Device:C
- added C884: 220n 50V startup output; effective >=100n, Capacitor_SMD:C_0603_1608Metric, symbol Device:C
- added D2220, D2221: BAT54WS OFF-bias supply OR, Diode_SMD:D_SOD-323, symbol Device:D_Schottky
- added D840: BAT54WS BAT supply reverse block, Diode_SMD:D_SOD-323, symbol Device:D_Schottky
- added D847, D848: BZT52C15 gate-source clamp, Diode_SMD:D_SOD-123, symbol Device:D_Zener
- added D849: BZT52C5V1 startup permit VGS clamp, Diode_SMD:D_SOD-123, symbol Device:D_Zener
- added J2072: protected pack power, ducktop2:WAGO_2060_452_SMD, symbol Connector_Generic:Conn_01x02
- added J2200: three cell probes: paired 1/2, 3/4, 5/6, Connector_JST:JST_SH_SM06B-SRSS-TB_1x06-1MP_P1.00mm_Horizontal, symbol BMS_Thermal:Conn_01x06_Thermal_MP
- added J2201: cell taps: 1 cell 1, 2 cell 2, Connector_JST:JST_GH_SM02B-GHS-TB_1x02-1MP_P1.25mm_Horizontal, symbol Conn_01x02_MP:Conn_01x02_MP
- added Q2211: ZXMP6A13FTA PDSG signal translator, Package_TO_SOT_SMD:SOT-23, symbol Transistor_FET:Q_PMOS_GSD
- added Q2212: BSS138 independent discharge inhibit, Package_TO_SOT_SMD:SOT-23, symbol Q_NMOS_SOT23_GSD:Q_NMOS_SOT23_GSD
- added R2200: 1k 1% 0.75W raw thermal supply limiter, Resistor_SMD:R_2010_5025Metric, symbol BMS_Passives:R
- added R2210, R2213, R2216: 100k 0.1% 25ppm cell NTC pull-up, Resistor_SMD:R_0603_1608Metric, symbol BMS_Passives:R
- added R2211, R2214: 10k 0.1% 25ppm NTC sense-lead limit, Resistor_SMD:R_0603_1608Metric, symbol BMS_Passives:R
- added R2212, R2215, R2218: 10k 0.1% 25ppm NTC return-lead limit, Resistor_SMD:R_0603_1608Metric, symbol BMS_Passives:R
- added R2217: 10k 0.1% 25ppm NTC sense-lead limit, Resistor_SMD:R_0402_1005Metric, symbol BMS_Passives:R
- added R2232: 47k thermal-ready pull-up, Resistor_SMD:R_0603_1608Metric, symbol BMS_Passives:R
- added R2233: 1M thermal-ready default-low, Resistor_SMD:R_0603_1608Metric, symbol BMS_Passives:R
- added R2234, R2237: 1k thermal CTR gate series, Resistor_SMD:R_0603_1608Metric, symbol BMS_Passives:R
- added R2238: 100k thermal CTR gate default-off, Resistor_SMD:R_0603_1608Metric, symbol BMS_Passives:R
- added R2239: 10k hardware OFF default-high, Resistor_SMD:R_0603_1608Metric, symbol BMS_Passives:R
- added R2240: 243k 0.1% 25ppm CHG_COLD top, Resistor_SMD:R_0603_1608Metric, symbol BMS_Passives:R
- added R2242: 634k 0.1% 25ppm CHG_HOT top, Resistor_SMD:R_0603_1608Metric, symbol BMS_Passives:R
- added R2244: 147k 0.1% 25ppm DSG_COLD top, Resistor_SMD:R_0603_1608Metric, symbol BMS_Passives:R
- added R2246: 845k 0.1% 25ppm DSG_HOT top, Resistor_SMD:R_0603_1608Metric, symbol BMS_Passives:R
- added R2247: 499k 0.1% 25ppm thermal reference bottom, Resistor_SMD:R_0603_1608Metric, symbol BMS_Passives:R
- added R2251: 100k raw health default-low, Resistor_SMD:R_0603_1608Metric, symbol BMS_Passives:R
- added R2255: 100k control health default-low, Resistor_SMD:R_0603_1608Metric, symbol BMS_Passives:R
- added R2258: 4.7k readiness output current limit, Resistor_SMD:R_0603_1608Metric, symbol BMS_Passives:R
- added R2260, R2261: 4.7k 1% I2C pull-up, Resistor_SMD:R_0603_1608Metric, symbol BMS_Passives:R
- added R2262, R2263, R2266, R2267: 2.2k 1% I2C pull-up, Resistor_SMD:R_0603_1608Metric, symbol BMS_Passives:R
- added R2270: 10.2k 0.1% 25ppm current limit, Resistor_SMD:R_0603_1608Metric, symbol BMS_Passives:R
- added R2271: 26.7k 0.1% 25ppm current limit, Resistor_SMD:R_0603_1608Metric, symbol BMS_Passives:R
- added R2272: 16.9k 0.1% 25ppm current limit, Resistor_SMD:R_0603_1608Metric, symbol BMS_Passives:R
- added R2273: 31.6k 0.1% 25ppm current limit, Resistor_SMD:R_0603_1608Metric, symbol BMS_Passives:R
- added R2274: 10k current-ready pull-up, Resistor_SMD:R_0603_1608Metric, symbol BMS_Passives:R
- added R2275: 100k current-ready default-low, Resistor_SMD:R_0603_1608Metric, symbol BMS_Passives:R
- added R2276: 100k current reset pull-up, Resistor_SMD:R_0603_1608Metric, symbol BMS_Passives:R
- added R2277: 100k 180..420ms current hold, Resistor_SMD:R_0603_1608Metric, symbol BMS_Passives:R
- added R2278: 100k permission default-low, Resistor_SMD:R_0603_1608Metric, symbol BMS_Passives:R
- added R2280, R2281, R2282, R2283: 4.99R 0.1% 25ppm sense filter, Resistor_SMD:R_0603_1608Metric, symbol BMS_Passives:R
- added R2290: 390k thermal switch default-off, Resistor_SMD:R_0603_1608Metric, symbol BMS_Passives:R
- added R840: 100R BAT input filter, Resistor_SMD:R_0603_1608Metric, symbol BMS_Passives:R
- added R841, R842, R843, R844: 75R 1% cell input/balance filter, Resistor_SMD:R_0603_1608Metric, symbol BMS_Passives:R
- added R845: 100R SRP filter, Resistor_SMD:R_0603_1608Metric, symbol BMS_Passives:R
- added R847, R848: 100R gate series, Resistor_SMD:R_0603_1608Metric, symbol BMS_Passives:R
- added R849, R850: 1M gate-source, Resistor_SMD:R_0603_1608Metric, symbol BMS_Passives:R
- added R851: 10k PACK sense, Resistor_SMD:R_0603_1608Metric, symbol BMS_Passives:R
- added R852: 10k LD sense, Resistor_SMD:R_0603_1608Metric, symbol BMS_Passives:R
- added R870: DNP 0R drive release, Resistor_SMD:R_0603_1608Metric, symbol BMS_Passives:R
- added R872: DNP 0R startup drive release, Resistor_SMD:R_0603_1608Metric, symbol BMS_Passives:R
- added R880, R881: 430R 1% 1.5W REGIN supply limiter, Resistor_SMD:R_2512_6332Metric, symbol BMS_Passives:R
- added R884: 100k UVLO top, Resistor_SMD:R_0603_1608Metric, symbol BMS_Passives:R
- added R885: 24.9k UVLO bottom, Resistor_SMD:R_0603_1608Metric, symbol BMS_Passives:R
- added R886: 402k latched current-limit mode, Resistor_SMD:R_0603_1608Metric, symbol BMS_Passives:R
- added R887: 12k 0.1% 25ppm ILIM, Resistor_SMD:R_0603_1608Metric, symbol BMS_Passives:R
- added R888: 24k 0.1% 25ppm ILIM, Resistor_SMD:R_0603_1608Metric, symbol BMS_Passives:R
- added R889: 100k startup fault pull-up, Resistor_SMD:R_0603_1608Metric, symbol BMS_Passives:R
- added R890: 1k PDSG translator gate, Resistor_SMD:R_0603_1608Metric, symbol BMS_Passives:R
- added R891: 1M translator gate-source, Resistor_SMD:R_0603_1608Metric, symbol BMS_Passives:R
- added R892: 100k startup shutdown top, Resistor_SMD:R_0603_1608Metric, symbol BMS_Passives:R
- added R893: 33.2k startup shutdown default-low, Resistor_SMD:R_0603_1608Metric, symbol BMS_Passives:R
- added R894: 100k startup permit gate series, Resistor_SMD:R_0603_1608Metric, symbol BMS_Passives:R
- added RS11: 2mOhm 1% 6W four-terminal pack shunt, ducktop2:Bourns_CSS4J_4026_Kelvin, symbol BMS_Current:BMS_Shunt4
- added TH2202: 104JT-025 cell 2 insulated probe, symbol Device:Thermistor_NTC
- added TH2203: 104JT-025 cell 3 insulated probe, symbol Device:Thermistor_NTC
- added TPB1: PACK_POS_RAW, TestPoint:TestPoint_Pad_D1.0mm, symbol BMS_Passives:TestPoint
- added TPB10: BQ_REG1, TestPoint:TestPoint_Pad_D1.0mm, symbol BMS_Passives:TestPoint
- added TPB11: BMS_SRP, TestPoint:TestPoint_Pad_D1.0mm, symbol BMS_Passives:TestPoint
- added TPB13: BMS_RAW_SCL, TestPoint:TestPoint_Pad_D1.0mm, symbol BMS_Passives:TestPoint
- added TPB14: BMS_RAW_SDA, TestPoint:TestPoint_Pad_D1.0mm, symbol BMS_Passives:TestPoint
- added TPB15: BQ_ALERT_AWAKE, TestPoint:TestPoint_Pad_D1.0mm, symbol BMS_Passives:TestPoint
- added TPB16: BQ_REGIN, TestPoint:TestPoint_Pad_D1.0mm, symbol BMS_Passives:TestPoint
- added TPB20: THERM_3V3, TestPoint:TestPoint_Pad_D1.0mm, symbol BMS_Passives:TestPoint
- added TPB21: THERM_READY, TestPoint:TestPoint_Pad_D1.0mm, symbol BMS_Passives:TestPoint
- added TPB22: THERM_SENSE_1, TestPoint:TestPoint_Pad_D1.0mm, symbol BMS_Passives:TestPoint
- added TPB23: THERM_SENSE_2, TestPoint:TestPoint_Pad_D1.0mm, symbol BMS_Passives:TestPoint
- added TPB24: THERM_SENSE_3, TestPoint:TestPoint_Pad_D1.0mm, symbol BMS_Passives:TestPoint
- added TPB25: BMS_CFETOFF, TestPoint:TestPoint_Pad_D1.0mm, symbol BMS_Passives:TestPoint
- added TPB27: BMS_PERMIT_READY, TestPoint:TestPoint_Pad_D1.0mm, symbol BMS_Passives:TestPoint
- added TPB3: PACK_POS_FUSED, TestPoint:TestPoint_Pad_D1.0mm, symbol BMS_Passives:TestPoint
- added TPB30: PDSG_FLT_N, TestPoint:TestPoint_Pad_D1.0mm, symbol BMS_Passives:TestPoint
- added TPB31: PDSG_SHDN, TestPoint:TestPoint_Pad_D1.0mm, symbol BMS_Passives:TestPoint
- added TPB32: PDSG_RTN, TestPoint:TestPoint_Pad_D1.0mm, symbol BMS_Passives:TestPoint
- added TPB33: CURRENT_READY, TestPoint:TestPoint_Pad_D1.0mm, symbol BMS_Passives:TestPoint
- added TPB35: BMS_CURRENT_REF, TestPoint:TestPoint_Pad_D1.0mm, symbol BMS_Passives:TestPoint
- added TPB4: BAT_PROT_FET_COMMON, TestPoint:TestPoint_Pad_D1.0mm, symbol BMS_Passives:TestPoint
- added TPB5: PACK_NEG_RAW, TestPoint:TestPoint_Pad_D1.0mm, symbol BMS_Passives:TestPoint
- added TPB6: FG_VSS, TestPoint:TestPoint_Pad_D1.0mm, symbol BMS_Passives:TestPoint
- added TPB8: BQ_WAKE, TestPoint:TestPoint_Pad_D1.0mm, symbol BMS_Passives:TestPoint
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Connections:
- net BAT_PROT_CGATE is gone; now on net BMS_SRN: TPB12.1
- net BMS_PRES is gone; now on net PACK_NEG_RAW: C881.2
- net PACK_FAULT_N is gone; now on net THERM_CHG_HOT_REF: R2243.1
- net PROT_CTRL_IN is gone; now on net BQ_REG1: C2253.1
- net BAT_PROT_FET_COMMON: now also Q11.5 (D(5-8)), Q12.5 (D(5-8)), TPB4.1; no longer C724.2, Q11.1 (S), Q11.2 (S), Q11.3 (S), Q12.1 (S), Q12.2 (S), Q12.3 (S)
- net BAT_PROT_VIN: now also Q11.1 (S), Q11.2 (S), Q11.3 (S), TPB2.1, C883.1, D847.2 (A), R849.2, R884.1, U2218.1 (IN), U2218.2 (IN); no longer J2074.1 (VIN), Q11.5 (D(5-8)), R2241.1
- net BMS_SRN: now also R846.2, U719.12 (SRN)
- net BMS_SRP: now also R845.2, TPB11.1, U719.11 (SRP); no longer C845.1, R2245.1
- net CELL1_TAP: now also J2201.1 (Pin_1), R842.1; no longer J2.4 (Pin_4)
- net CELL2_TAP: now also J2201.2 (Pin_2), R843.1; no longer J2.2 (Pin_2)
- net CTRL_3V3: now also C2258.1, R2262.1, R2263.1, R2266.1, R2267.1, U2206.1 (VCC1), U2207.1 (VCCA), U2207.5 (EN), U2207.8 (VCCB), U2216.1 (VOUT)
- net CTRL_GND: now also J2074.5 (Pin_5), J2074.MP (MountPin), U2209.7 (INA), C2257.2, C2258.2, R2255.2, U2206.4 (GND1), U2207.4 (GND), U2216.2 (GND), U2216.4 (ON_N)
- net FG_VSS: now also C884.2, J2072.2 (Pin_2), RS11.2 (FORCE_FET), TPB6.1; no longer C2253.2, C2255.2, C880.2, J2074.4 (RETRY), J2074.5 (GND), R2201.2 (Pin_2), R846.1 (S), R846.2 (S), R846.3 (S), TPB12.2, U2209.4 (GND1)
- net MCU_3V3: now also J2074.3 (Pin_3), C2257.1, U2216.5 (VIN)
- net PACK_NEG_RAW: now also C2253.2, C2255.2, C2273.2, C880.2, Q2200.2 (S), R2201.2, R2241.2, R2243.2, R2245.2, U2204.2 (GND), U2209.4 (GND1), U2210.5 (GND)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; no longer Q2200.MP, R2230.2, TPB26.2
- net PACK_POS_FUSED: now also Q12.1 (S), Q12.2 (S), Q12.3 (S), C884.1, D848.2 (A), J2072.1 (Pin_1), R850.2, R851.1, R852.1, TPB3.1, U2218.15 (OUT), U2218.16 (OUT); no longer J2074.8 (VOUT), R2201.1 (Pin_1), TPB2.2
- net PACK_POS_RAW: now also J2.2 (Pin_2), D840.2 (A), R2200.1, R844.1, R880.1, R881.1, TPB1.1; no longer C881.1, J2.3 (Pin_3)
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Other:
- note added: "8 A discharge / 3 A charge design targets; installed current, startup and temperature limits need bench verification."
- note added: "== current guards: signed low-side sense, hardware latches =="
- note added: "== isolated control interface: I2C and monitor readiness =="
- note added: "== startup branch: active current limit, thermal latch-off =="
- note added: "== three-cell BMS: high-side protection, cell monitoring and independent inhibits =="
- note added: "BQ uses isolator side2. Side1 is a short local bus; the buffer carries the longer harness load."
- note added: "CLR is a raw-side service input. The five-wire control harness does not reset these latches."
- note added: "CTRL_GND stays isolated from RAW and FG. All external pack current crosses RS11 and the center gauge shunt."
- note added: "Charge10..40C / discharge0..50C design windows. Cell limits and installed probe response need tests."
- note added: "High readiness means REG1 and the thermal supervisor are powered. Faults and freshness come from verified I2C samples."
- note added: "Leave the three drive-release links open until configuration and fault tests pass."
- note added: "Loss of either READY signal removes permission. The hardware inhibit covers main FETs and the startup branch."
- note added: "Nominal trips: about9.1A discharge and4.1A charge. These are fault trips, not operating ratings."
- note added: "PDSG timeout stays0; only voltage completion may enable the main DSG path."
- note added: "PDSG_RTN is the local eFuse reference. Do not bond it to RAW, FG, CTRL or a mounting hole."
- note added: "Raw service pads: use an isolated programmer. Do not attach system-ground equipment across either shunt."
- note added: "The control connector supplies only CTRL_GND. Programming and current-clear pads belong to RAW."
- note added: "The independent discharge permit also covers PDSG; a disabled main FET cannot leave an unchecked bypass."
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